File: audio.sch (KiCad schematic (older format))
At the start: 7 parts, among them U12 PCM5100

Commit message: Small fixes
Parts:
- added C? (x2): 1u, Capacitor_SMD:C_0402_1005Metric, symbol Device:C
Connections:
- net AUDIO_L: now also C?.1; no longer U12.6 (OUTL)
- net AUDIO_R: now also C?.1; no longer U12.7 (OUTR)
- new net: C?.2, U12.6 (OUTL)
- new net: C?.2, U12.7 (OUTR)
Changed lines of the file:
@@
 $Descr A4 11693 8268
 encoding utf-8
-Sheet 9 10
+Sheet 7 10
 Title ""
 Date ""
@@
 Text Notes 550  650  0    79   ~ 0
 I2S Audio DAC
-Text HLabel 6150 3350 2    39   Output ~ 0
+Text HLabel 6550 3250 2    39   Output ~ 0
 AUDIO_L
-Text HLabel 6150 3450 2    39   Output ~ 0
+Text HLabel 6550 3550 2    39   Output ~ 0
 AUDIO_R
 Wire Wire Line
@@
 Wire Wire Line
 	4800 3550 5150 3550
+$Comp
+L Device:C C?
+U 1 1 5F37D2B1
+P 6400 3250
+F 0 "C?" V 6250 3200 50  0000 L CNN
+F 1 "1u" V 6350 3100 50  0000 L CNN
+F 2 "Capacitor_SMD:C_0402_1005Metric" H 6438 3100 50  0001 C CNN
+F 3 "~" H 6400 3250 50  0001 C CNN
+	1    6400 3250
+	0    1    1    0
+$EndComp
+$Comp
+L Device:C C?
+U 1 1 5F37F925
+P 6400 3550
+F 0 "C?" V 6250 3500 50  0000 L CNN
+F 1 "1u" V 6350 3400 50  0000 L CNN
+F 2 "Capacitor_SMD:C_0402_1005Metric" H 6438 3400 50  0001 C CNN
+F 3 "~" H 6400 3550 50  0001 C CNN
+	1    6400 3550
+	0    1    1    0
+$EndComp
+Wire Wire Line
+	6150 3350 6200 3350
+Wire Wire Line
+	6200 3350 6200 3250
+Wire Wire Line
+	6200 3250 6250 3250
+Wire Wire Line
+	6150 3450 6200 3450
+Wire Wire Line
+	6200 3450 6200 3550
+Wire Wire Line
+	6200 3550 6250 3550
 $EndSCHEMATC
