File: touch.sch (KiCad schematic (older format))
At the start: 3 parts, among them U8 MPR121Q

Commit message: Small fixes
Parts:
- added C42: 100n, Capacitor_SMD:C_0603_1608Metric, symbol Device:C_Small
- added C43: 10u, Capacitor_SMD:C_0603_1608Metric, symbol Device:C_Small
Connections:
- net +3V3: now also C42.1, C43.1
- net GND: now also C42.2, C43.2
Changed lines of the file:
@@
 $Descr A4 11693 8268
 encoding utf-8
-Sheet 6 10
+Sheet 4 10
 Title ""
 Date ""
@@
 Text HLabel 5350 3400 0    39   Output ~ 0
 IRQ
+$Comp
+L Device:C_Small C43
+U 1 1 5F339FD0
+P 10950 6200
+F 0 "C43" H 11042 6246 50  0000 L CNN
+F 1 "10u" H 11042 6155 50  0000 L CNN
+F 2 "Capacitor_SMD:C_0603_1608Metric" H 10950 6200 50  0001 C CNN
+F 3 "~" H 10950 6200 50  0001 C CNN
+	1    10950 6200
+	1    0    0    -1
+$EndComp
+$Comp
+L power:GND #PWR0164
+U 1 1 5F33A63D
+P 10950 6300
+F 0 "#PWR0164" H 10950 6050 50  0001 C CNN
+F 1 "GND" H 10955 6127 50  0000 C CNN
+F 2 "" H 10950 6300 50  0001 C CNN
+F 3 "" H 10950 6300 50  0001 C CNN
+	1    10950 6300
+	1    0    0    -1
+$EndComp
+$Comp
+L power:+3.3V #PWR0165
+U 1 1 5F33AC79
+P 10950 6100
+F 0 "#PWR0165" H 10950 5950 50  0001 C CNN
+F 1 "+3.3V" H 10950 6250 50  0000 C CNN
+F 2 "" H 10950 6100 50  0001 C CNN
+F 3 "" H 10950 6100 50  0001 C CNN
+	1    10950 6100
+	1    0    0    -1
+$EndComp
+$Comp
+L Device:C_Small C42
+U 1 1 5F33C3B2
+P 10550 6200
+F 0 "C42" H 10642 6246 50  0000 L CNN
+F 1 "100n" H 10642 6155 50  0000 L CNN
+F 2 "Capacitor_SMD:C_0603_1608Metric" H 10550 6200 50  0001 C CNN
+F 3 "~" H 10550 6200 50  0001 C CNN
+	1    10550 6200
+	1    0    0    -1
+$EndComp
+$Comp
+L power:GND #PWR0166
+U 1 1 5F33C3B8
+P 10550 6300
+F 0 "#PWR0166" H 10550 6050 50  0001 C CNN
+F 1 "GND" H 10555 6127 50  0000 C CNN
+F 2 "" H 10550 6300 50  0001 C CNN
+F 3 "" H 10550 6300 50  0001 C CNN
+	1    10550 6300
+	1    0    0    -1
+$EndComp
+$Comp
+L power:+3.3V #PWR0167
+U 1 1 5F33C3BE
+P 10550 6100
+F 0 "#PWR0167" H 10550 5950 50  0001 C CNN
+F 1 "+3.3V" H 10550 6250 50  0000 C CNN
+F 2 "" H 10550 6100 50  0001 C CNN
+F 3 "" H 10550 6100 50  0001 C CNN
+	1    10550 6100
+	1    0    0    -1
+$EndComp
 $EndSCHEMATC

Commit message: Fixes, removed I2S DAC
Connections:
- net FPGA_CDONE renamed TOUCH_START
- net FPGA_RESET renamed TOUCH_SELECT
Other:
- note removed: "Output type:\nopen drain"
Changed lines of the file:
@@
 $Descr A4 11693 8268
 encoding utf-8
-Sheet 4 10
+Sheet 4 9
 Title ""
 Date ""
@@
 Wire Wire Line
 	4800 3850 5350 3850
-Text HLabel 6150 4300 2    39   Output ~ 0
-FPGA_RESET
-Text HLabel 6150 4200 2    39   Input ~ 0
-FPGA_CDONE
-Text Notes 6600 4350 0    35   ~ 0
-Output type:\nopen drain
 Text HLabel 5350 3500 0    39   Input ~ 0
 I2C_SCL
@@
 	1    0    0    -1
 $EndComp
+Text GLabel 6150 4200 2    35   Input ~ 0
+TOUCH_START
+Text GLabel 6150 4300 2    35   Input ~ 0
+TOUCH_SELECT
 $EndSCHEMATC

Commit message: Dump.
Parts:
- added U?: PCA9555PW, Package_SO:TSSOP-24_4.4x7.8mm_P0.65mm, symbol Interface_Expansion:PCA9555PW
- C22: renamed from C20; footprint Capacitor_SMD:C_0402_1005Metric -> Capacitor_SMD:C_0603_1608Metric; LCSC (none) -> C14663; Mouser (none) -> -; Price (none) -> 0.0020; Sponsored (none) -> N
- C23: renamed from C42; LCSC (none) -> C14663; Mouser (none) -> -; Price (none) -> 0.0020; Sponsored (none) -> N
- C24: renamed from C43; Price (none) -> 0.0020; Sponsored (none) -> N
- R17: renamed from R19; LCSC (none) -> C325654; Mouser (none) -> -; Price (none) -> 0.0016; Sponsored (none) -> N
- U8: LCSC (none) -> C91322; Mouser (none) -> -; Price (none) -> 0.77; Sponsored (none) -> N
Changed lines of the file:
@@
 F 2 "Package_DFN_QFN:QFN-20-1EP_3x3mm_P0.4mm_EP1.65x1.65mm" H 5800 3700 50  0001 C CNN
 F 3 "" H 5800 3700 50  0001 C CNN
+F 4 "C91322" H 5800 3700 50  0001 C CNN "LCSC"
+F 5 "-" H 5800 3700 50  0001 C CNN "Mouser"
+F 6 "0.77" H 5800 3700 50  0001 C CNN "Price"
+F 7 "N" H 5800 3700 50  0001 C CNN "Sponsored"
 	1    5800 3700
 	1    0    0    -1
 $EndComp
 $Comp
-L Device:R R19
+L Device:R R17
 U 1 1 605342FC
 P 5100 4700
-F 0 "R19" V 4893 4700 50  0000 C CNN
+F 0 "R17" V 4893 4700 50  0000 C CNN
 F 1 "75k" V 4984 4700 50  0000 C CNN
 F 2 "Resistor_SMD:R_0603_1608Metric" V 5030 4700 50  0001 C CNN
 F 3 "~" H 5100 4700 50  0001 C CNN
+F 4 "0.0016" H 5100 4700 50  0001 C CNN "Price"
+F 5 "C325654" H 5100 4700 50  0001 C CNN "LCSC"
+F 6 "-" H 5100 4700 50  0001 C CNN "Mouser"
+F 7 "N" H 5100 4700 50  0001 C CNN "Sponsored"
 	1    5100 4700
 	1    0    0    -1
 $EndComp
 $Comp
-L Device:C C20
+L Device:C C22
 U 1 1 6053432A
 P 5300 4700
-F 0 "C20" V 5048 4700 50  0000 C CNN
+F 0 "C22" V 5048 4700 50  0000 C CNN
 F 1 "100n" V 5139 4700 50  0000 C CNN
-F 2 "Capacitor_SMD:C_0402_1005Metric" H 5338 4550 50  0001 C CNN
+F 2 "Capacitor_SMD:C_0603_1608Metric" H 5338 4550 50  0001 C CNN
 F 3 "~" H 5300 4700 50  0001 C CNN
+F 4 "C14663" H 5300 4700 50  0001 C CNN "LCSC"
+F 5 "0.0020" H 5300 4700 50  0001 C CNN "Price"
+F 6 "-" H 5300 4700 50  0001 C CNN "Mouser"
+F 7 "N" H 5300 4700 50  0001 C CNN "Sponsored"
 	1    5300 4700
 	-1   0    0    1
 $EndComp
 $Comp
-L power:GND #PWR084
+L power:GND #PWR089
 U 1 1 6053432B
 P 5100 4850
-F 0 "#PWR084" H 5100 4600 50  0001 C CNN
+F 0 "#PWR089" H 5100 4600 50  0001 C CNN
 F 1 "GND" H 5105 4677 50  0000 C CNN
 F 2 "" H 5100 4850 50  0001 C CNN
@@
 $EndComp
 $Comp
-L power:+3.3V #PWR086
+L power:+3.3V #PWR091
 U 1 1 5F90D187
 P 5750 3200
-F 0 "#PWR086" H 5750 3050 50  0001 C CNN
+F 0 "#PWR091" H 5750 3050 50  0001 C CNN
 F 1 "+3.3V" H 5750 3350 50  0000 C CNN
 F 2 "" H 5750 3200 50  0001 C CNN
@@
 $EndComp
 $Comp
-L power:GND #PWR083
+L power:GND #PWR088
 U 1 1 6053432E
 P 4800 4850
-F 0 "#PWR083" H 4800 4600 50  0001 C CNN
+F 0 "#PWR088" H 4800 4600 50  0001 C CNN
 F 1 "GND" H 4805 4677 50  0000 C CNN
 F 2 "" H 4800 4850 50  0001 C CNN
@@
 $EndComp
 $Comp
-L power:GND #PWR085
+L power:GND #PWR090
 U 1 1 6053432F
 P 5300 4850
-F 0 "#PWR085" H 5300 4600 50  0001 C CNN
+F 0 "#PWR090" H 5300 4600 50  0001 C CNN
 F 1 "GND" H 5305 4677 50  0000 C CNN
 F 2 "" H 5300 4850 50  0001 C CNN
@@
 $EndComp
 $Comp
-L power:GND #PWR087
+L power:GND #PWR092
 U 1 1 60534330
 P 5750 4850
-F 0 "#PWR087" H 5750 4600 50  0001 C CNN
+F 0 "#PWR092" H 5750 4600 50  0001 C CNN
 F 1 "GND" H 5755 4677 50  0000 C CNN
 F 2 "" H 5750 4850 50  0001 C CNN
@@
 IRQ
 $Comp
-L Device:C_Small C43
+L Device:C_Small C24
 U 1 1 5F339FD0
 P 10950 6200
-F 0 "C43" H 11042 6246 50  0000 L CNN
+F 0 "C24" H 11042 6246 50  0000 L CNN
 F 1 "10u" H 11042 6155 50  0000 L CNN
 F 2 "Capacitor_SMD:C_0603_1608Metric" H 10950 6200 50  0001 C CNN
 F 3 "~" H 10950 6200 50  0001 C CNN
+F 4 "0.0020" H 10950 6200 50  0001 C CNN "Price"
+F 5 "N" H 10950 6200 50  0001 C CNN "Sponsored"
 	1    10950 6200
 	1    0    0    -1
 $EndComp
 $Comp
-L power:GND #PWR0164
+L power:GND #PWR096
 U 1 1 5F33A63D
 P 10950 6300
-F 0 "#PWR0164" H 10950 6050 50  0001 C CNN
+F 0 "#PWR096" H 10950 6050 50  0001 C CNN
 F 1 "GND" H 10955 6127 50  0000 C CNN
 F 2 "" H 10950 6300 50  0001 C CNN
@@
 $EndComp
 $Comp
-L power:+3.3V #PWR0165
+L power:+3.3V #PWR095
 U 1 1 5F33AC79
 P 10950 6100
-F 0 "#PWR0165" H 10950 5950 50  0001 C CNN
+F 0 "#PWR095" H 10950 5950 50  0001 C CNN
 F 1 "+3.3V" H 10950 6250 50  0000 C CNN
 F 2 "" H 10950 6100 50  0001 C CNN
@@
 $EndComp
 $Comp
-L Device:C_Small C42
+L Device:C_Small C23
 U 1 1 5F33C3B2
 P 10550 6200
-F 0 "C42" H 10642 6246 50  0000 L CNN
+F 0 "C23" H 10642 6246 50  0000 L CNN
 F 1 "100n" H 10642 6155 50  0000 L CNN
 F 2 "Capacitor_SMD:C_0603_1608Metric" H 10550 6200 50  0001 C CNN
 F 3 "~" H 10550 6200 50  0001 C CNN
+F 4 "C14663" H 10550 6200 50  0001 C CNN "LCSC"
+F 5 "0.0020" H 10550 6200 50  0001 C CNN "Price"
+F 6 "-" H 10550 6200 50  0001 C CNN "Mouser"
+F 7 "N" H 10550 6200 50  0001 C CNN "Sponsored"
 	1    10550 6200
 	1    0    0    -1
 $EndComp
 $Comp
-L power:GND #PWR0166
+L power:GND #PWR094
 U 1 1 5F33C3B8
 P 10550 6300
-F 0 "#PWR0166" H 10550 6050 50  0001 C CNN
+F 0 "#PWR094" H 10550 6050 50  0001 C CNN
 F 1 "GND" H 10555 6127 50  0000 C CNN
 F 2 "" H 10550 6300 50  0001 C CNN
@@
 $EndComp
 $Comp
-L power:+3.3V #PWR0167
+L power:+3.3V #PWR093
 U 1 1 5F33C3BE
 P 10550 6100
-F 0 "#PWR0167" H 10550 5950 50  0001 C CNN
+F 0 "#PWR093" H 10550 5950 50  0001 C CNN
 F 1 "+3.3V" H 10550 6250 50  0000 C CNN
 F 2 "" H 10550 6100 50  0001 C CNN
@@
 Text GLabel 6150 4300 2    35   Input ~ 0
 TOUCH_SELECT
+$Comp
+L Interface_Expansion:PCA9555PW U?
+U 1 1 5F5BEEA4
+P 7400 3650
+F 0 "U?" H 7400 4831 50  0000 C CNN
+F 1 "PCA9555PW" H 7400 4740 50  0000 C CNN
+F 2 "Package_SO:TSSOP-24_4.4x7.8mm_P0.65mm" H 7400 3650 50  0001 C CNN
+F 3 "https://www.nxp.com/docs/en/data-sheet/PCA9555.pdf" H 7400 3650 50  0001 C CNN
+	1    7400 3650
+	1    0    0    -1
+$EndComp
 $EndSCHEMATC
