File: fpga.sch (KiCad schematic (older format))
At the start: 22 parts, among them U8 ICE40UP5K-SG48ITR, U9 LY68L6400

Commit message: Dump.
Parts:
- renumbered R21 to R33, R22 to R34, R23 to R35, R24 to R36, R25 to R37, R26 to R38, R27 to R39, R28 to R40, RN9 to RN5, RN10 to RN6
Changed lines of the file:
@@
 $EndComp
 $Comp
-L Device:R_Small R22
+L Device:R_Small R34
 U 1 1 5F537E5C
 P 1050 1500
-F 0 "R22" V 1246 1500 50  0000 C CNN
+F 0 "R34" V 1246 1500 50  0000 C CNN
 F 1 "100" V 1155 1500 50  0000 C CNN
 F 2 "Resistor_SMD:R_0603_1608Metric" H 1050 1500 50  0001 C CNN
@@
 $EndComp
 $Comp
-L power:GND #PWR0114
+L power:GND #PWR0113
 U 1 1 5F553535
 P 1650 1800
-F 0 "#PWR0114" H 1650 1550 50  0001 C CNN
+F 0 "#PWR0113" H 1650 1550 50  0001 C CNN
 F 1 "GND" H 1655 1627 50  0000 C CNN
 F 2 "" H 1650 1800 50  0001 C CNN
@@
 $EndComp
 $Comp
-L power:GND #PWR0112
+L power:GND #PWR0111
 U 1 1 5F553952
 P 1250 1800
-F 0 "#PWR0112" H 1250 1550 50  0001 C CNN
+F 0 "#PWR0111" H 1250 1550 50  0001 C CNN
 F 1 "GND" H 1255 1627 50  0000 C CNN
 F 2 "" H 1250 1800 50  0001 C CNN
@@
 $EndComp
 $Comp
-L power:GND #PWR0110
+L power:GND #PWR0109
 U 1 1 5F553E39
 P 850 1800
-F 0 "#PWR0110" H 850 1550 50  0001 C CNN
+F 0 "#PWR0109" H 850 1550 50  0001 C CNN
 F 1 "GND" H 855 1627 50  0000 C CNN
 F 2 "" H 850 1800 50  0001 C CNN
@@
 	850  1500 850  1600
 $Comp
-L power:+2V5 #PWR0116
+L power:+2V5 #PWR0115
 U 1 1 5F561535
 P 1800 1100
-F 0 "#PWR0116" H 1800 950 50  0001 C CNN
+F 0 "#PWR0115" H 1800 950 50  0001 C CNN
 F 1 "+2V5" V 1815 1228 50  0000 L CNN
 F 2 "" H 1800 1100 50  0001 C CNN
@@
 Connection ~ 850  1200
 $Comp
-L power:+1V2 #PWR0109
+L power:+1V2 #PWR0108
 U 1 1 5F564804
 P 850 1000
-F 0 "#PWR0109" H 850 850 50  0001 C CNN
+F 0 "#PWR0108" H 850 850 50  0001 C CNN
 F 1 "+1V2" H 865 1173 50  0000 C CNN
 F 2 "" H 850 1000 50  0001 C CNN
@@
 $EndComp
 $Comp
-L power:GND #PWR0117
+L power:GND #PWR0116
 U 1 1 5F565850
 P 2700 1800
-F 0 "#PWR0117" H 2700 1550 50  0001 C CNN
+F 0 "#PWR0116" H 2700 1550 50  0001 C CNN
 F 1 "GND" H 2705 1627 50  0000 C CNN
 F 2 "" H 2700 1800 50  0001 C CNN
@@
 	2700 1200 2600 1200
 $Comp
-L power:+3.3V #PWR0122
+L power:+3.3V #PWR0121
 U 1 1 5F57B8C0
 P 6100 2150
-F 0 "#PWR0122" H 6100 2000 50  0001 C CNN
+F 0 "#PWR0121" H 6100 2000 50  0001 C CNN
 F 1 "+3.3V" H 6115 2323 50  0000 C CNN
 F 2 "" H 6100 2150 50  0001 C CNN
@@
 FPGA_CDONE
 $Comp
-L power:GND #PWR0111
+L power:GND #PWR0110
 U 1 1 5F58383F
 P 1100 3150
-F 0 "#PWR0111" H 1100 2900 50  0001 C CNN
+F 0 "#PWR0110" H 1100 2900 50  0001 C CNN
 F 1 "GND" H 1105 2977 50  0000 C CNN
 F 2 "" H 1100 3150 50  0001 C CNN
@@
 $EndComp
 $Comp
-L Device:R_Small R23
+L Device:R_Small R35
 U 1 1 5F59314F
 P 1100 3050
-F 0 "R23" H 1159 3096 50  0000 L CNN
+F 0 "R35" H 1159 3096 50  0000 L CNN
 F 1 "100k" H 1159 3005 50  0000 L CNN
 F 2 "Resistor_SMD:R_0603_1608Metric" H 1100 3050 50  0001 C CNN
@@
 FPGA_RESET
 $Comp
-L Device:R_Small R24
+L Device:R_Small R36
 U 1 1 5F5BBEB5
 P 1400 2700
-F 0 "R24" H 1459 2746 50  0000 L CNN
+F 0 "R36" H 1459 2746 50  0000 L CNN
 F 1 "100k" H 1459 2655 50  0000 L CNN
 F 2 "Resistor_SMD:R_0603_1608Metric" H 1400 2700 50  0001 C CNN
@@
 FPGA_CDONE
 $Comp
-L power:+3.3V #PWR0113
+L power:+3.3V #PWR0112
 U 1 1 5F5BD259
 P 1400 2600
-F 0 "#PWR0113" H 1400 2450 50  0001 C CNN
+F 0 "#PWR0112" H 1400 2450 50  0001 C CNN
 F 1 "+3.3V" H 1415 2773 50  0000 C CNN
 F 2 "" H 1400 2600 50  0001 C CNN
@@
 LCD_FMARK
 $Comp
-L power:+3.3V #PWR0118
+L power:+3.3V #PWR0117
 U 1 1 60CF7467
 P 3300 5150
-F 0 "#PWR0118" H 3300 5000 50  0001 C CNN
+F 0 "#PWR0117" H 3300 5000 50  0001 C CNN
 F 1 "+3.3V" H 3315 5323 50  0000 C CNN
 F 2 "" H 3300 5150 50  0001 C CNN
@@
 RGB2
 $Comp
-L power:+3.3V #PWR0121
+L power:+3.3V #PWR0120
 U 1 1 5F32B7AB
 P 4950 5950
-F 0 "#PWR0121" H 4950 5800 50  0001 C CNN
+F 0 "#PWR0120" H 4950 5800 50  0001 C CNN
 F 1 "+3.3V" H 4965 6123 50  0000 C CNN
 F 2 "" H 4950 5950 50  0001 C CNN
@@
 	10500 1750 10500 1800
 $Comp
-L power:GND #PWR0131
+L power:GND #PWR0130
 U 1 1 5F3AAB21
 P 10500 1800
-F 0 "#PWR0131" H 10500 1550 50  0001 C CNN
+F 0 "#PWR0130" H 10500 1550 50  0001 C CNN
 F 1 "GND" H 10505 1627 50  0000 C CNN
 F 2 "" H 10500 1800 50  0001 C CNN
@@
 $EndComp
 $Comp
-L Device:R_Small R28
+L Device:R_Small R40
 U 1 1 5F436AA9
 P 9450 1050
-F 0 "R28" H 9509 1096 50  0000 L CNN
+F 0 "R40" H 9509 1096 50  0000 L CNN
 F 1 "10k" H 9509 1005 50  0000 L CNN
 F 2 "Resistor_SMD:R_0603_1608Metric" H 9450 1050 50  0001 C CNN
@@
 	9450 1250 9450 1150
 $Comp
-L power:+3.3V #PWR0125
+L power:+3.3V #PWR0124
 U 1 1 5F439DDC
 P 9450 950
-F 0 "#PWR0125" H 9450 800 50  0001 C CNN
+F 0 "#PWR0124" H 9450 800 50  0001 C CNN
 F 1 "+3.3V" H 9465 1123 50  0000 C CNN
 F 2 "" H 9450 950 50  0001 C CNN
@@
 $EndComp
 $Comp
-L power:+3.3V #PWR0130
+L power:+3.3V #PWR0129
 U 1 1 5F43A076
 P 10500 950
-F 0 "#PWR0130" H 10500 800 50  0001 C CNN
+F 0 "#PWR0129" H 10500 800 50  0001 C CNN
 F 1 "+3.3V" H 10515 1123 50  0000 C CNN
 F 2 "" H 10500 950 50  0001 C CNN
@@
 $EndComp
 $Comp
-L power:GND #PWR0129
+L power:GND #PWR0128
 U 1 1 5F473D9D
 P 10100 6250
-F 0 "#PWR0129" H 10100 6000 50  0001 C CNN
+F 0 "#PWR0128" H 10100 6000 50  0001 C CNN
 F 1 "GND" H 10105 6077 50  0000 C CNN
 F 2 "" H 10100 6250 50  0001 C CNN
@@
 $EndComp
 $Comp
-L power:+3.3V #PWR0128
+L power:+3.3V #PWR0127
 U 1 1 5F473F7E
 P 10100 6050
-F 0 "#PWR0128" H 10100 5900 50  0001 C CNN
+F 0 "#PWR0127" H 10100 5900 50  0001 C CNN
 F 1 "+3.3V" H 10115 6223 50  0000 C CNN
 F 2 "" H 10100 6050 50  0001 C CNN
@@
 $EndComp
 $Comp
-L power:GND #PWR0135
+L power:GND #PWR0134
 U 1 1 5F47D06A
 P 10900 6250
-F 0 "#PWR0135" H 10900 6000 50  0001 C CNN
+F 0 "#PWR0134" H 10900 6000 50  0001 C CNN
 F 1 "GND" H 10905 6077 50  0000 C CNN
 F 2 "" H 10900 6250 50  0001 C CNN
@@
 $EndComp
 $Comp
-L power:+3.3V #PWR0134
+L power:+3.3V #PWR0133
 U 1 1 5F47D070
 P 10900 6050
-F 0 "#PWR0134" H 10900 5900 50  0001 C CNN
+F 0 "#PWR0133" H 10900 5900 50  0001 C CNN
 F 1 "+3.3V" H 10915 6223 50  0000 C CNN
 F 2 "" H 10900 6050 50  0001 C CNN
@@
 $EndComp
 $Comp
-L power:GND #PWR0133
+L power:GND #PWR0132
 U 1 1 5F47E270
 P 10500 6250
-F 0 "#PWR0133" H 10500 6000 50  0001 C CNN
+F 0 "#PWR0132" H 10500 6000 50  0001 C CNN
 F 1 "GND" H 10505 6077 50  0000 C CNN
 F 2 "" H 10500 6250 50  0001 C CNN
@@
 $EndComp
 $Comp
-L power:+3.3V #PWR0132
+L power:+3.3V #PWR0131
 U 1 1 5F47E276
 P 10500 6050
-F 0 "#PWR0132" H 10500 5900 50  0001 C CNN
+F 0 "#PWR0131" H 10500 5900 50  0001 C CNN
 F 1 "+3.3V" H 10515 6223 50  0000 C CNN
 F 2 "" H 10500 6050 50  0001 C CNN
@@
 $EndComp
 $Comp
-L power:GND #PWR0127
+L power:GND #PWR0126
 U 1 1 5F489EEC
 P 9700 6250
-F 0 "#PWR0127" H 9700 6000 50  0001 C CNN
+F 0 "#PWR0126" H 9700 6000 50  0001 C CNN
 F 1 "GND" H 9705 6077 50  0000 C CNN
 F 2 "" H 9700 6250 50  0001 C CNN
@@
 $EndComp
 $Comp
-L power:+3.3V #PWR0126
+L power:+3.3V #PWR0125
 U 1 1 5F489EF2
 P 9700 6050
-F 0 "#PWR0126" H 9700 5900 50  0001 C CNN
+F 0 "#PWR0125" H 9700 5900 50  0001 C CNN
 F 1 "+3.3V" H 9715 6223 50  0000 C CNN
 F 2 "" H 9700 6050 50  0001 C CNN
@@
 $EndComp
 $Comp
-L power:GND #PWR0124
+L power:GND #PWR0123
 U 1 1 5F48A8FA
 P 9300 6250
-F 0 "#PWR0124" H 9300 6000 50  0001 C CNN
+F 0 "#PWR0123" H 9300 6000 50  0001 C CNN
 F 1 "GND" H 9305 6077 50  0000 C CNN
 F 2 "" H 9300 6250 50  0001 C CNN
@@
 $EndComp
 $Comp
-L power:+3.3V #PWR0123
+L power:+3.3V #PWR0122
 U 1 1 5F48A900
 P 9300 6050
-F 0 "#PWR0123" H 9300 5900 50  0001 C CNN
+F 0 "#PWR0122" H 9300 5900 50  0001 C CNN
 F 1 "+3.3V" H 9315 6223 50  0000 C CNN
 F 2 "" H 9300 6050 50  0001 C CNN
@@
 $EndComp
 $Comp
-L power:GND #PWR0108
+L power:GND #PWR0107
 U 1 1 5F503F48
 P 800 3150
-F 0 "#PWR0108" H 800 2900 50  0001 C CNN
+F 0 "#PWR0107" H 800 2900 50  0001 C CNN
 F 1 "GND" H 805 2977 50  0000 C CNN
 F 2 "" H 800 3150 50  0001 C CNN
@@
 $EndComp
 $Comp
-L Device:R_Small R21
+L Device:R_Small R33
 U 1 1 5F503F4E
 P 800 3050
-F 0 "R21" H 859 3096 50  0000 L CNN
+F 0 "R33" H 859 3096 50  0000 L CNN
 F 1 "100k" H 859 3005 50  0000 L CNN
 F 2 "Resistor_SMD:R_0603_1608Metric" H 800 3050 50  0001 C CNN
@@
 	5600 3150 4850 3150
 $Comp
-L Device:R_Small R26
+L Device:R_Small R38
 U 1 1 5F67E775
 P 4750 3050
-F 0 "R26" V 4850 3050 50  0000 C CNN
+F 0 "R38" V 4850 3050 50  0000 C CNN
 F 1 "TBD" V 4750 3050 50  0000 C CNN
 F 2 "Resistor_SMD:R_0603_1608Metric" H 4750 3050 50  0001 C CNN
@@
 $EndComp
 $Comp
-L Device:R_Small R27
+L Device:R_Small R39
 U 1 1 5F684417
 P 4750 3150
-F 0 "R27" V 4650 3150 50  0000 C CNN
+F 0 "R39" V 4650 3150 50  0000 C CNN
 F 1 "TBD" V 4750 3150 50  0000 C CNN
 F 2 "Resistor_SMD:R_0603_1608Metric" H 4750 3150 50  0001 C CNN
@@
 	4050 3050 4050 3300
 $Comp
-L power:GND #PWR0120
+L power:GND #PWR0119
 U 1 1 5F68C71B
 P 4550 3500
-F 0 "#PWR0120" H 4550 3250 50  0001 C CNN
+F 0 "#PWR0119" H 4550 3250 50  0001 C CNN
 F 1 "GND" H 4555 3327 50  0000 C CNN
 F 2 "" H 4550 3500 50  0001 C CNN
@@
 $EndComp
 $Comp
-L power:GND #PWR0119
+L power:GND #PWR0118
 U 1 1 5F68DF1A
 P 4050 3500
-F 0 "#PWR0119" H 4050 3250 50  0001 C CNN
+F 0 "#PWR0118" H 4050 3250 50  0001 C CNN
 F 1 "GND" H 4055 3327 50  0000 C CNN
 F 2 "" H 4050 3500 50  0001 C CNN
@@
 PMOD_7
 $Comp
-L Device:R_Pack04 RN10
+L Device:R_Pack04 RN6
 U 1 1 5FD85945
 P 4350 6950
-F 0 "RN10" V 4050 6950 50  0000 C CNN
+F 0 "RN6" V 4050 6950 50  0000 C CNN
 F 1 "47" V 3950 6950 50  0000 C CNN
 F 2 "Resistor_SMD:R_Array_Convex_4x0603" V 4625 6950 50  0001 C CNN
@@
 $EndComp
 $Comp
-L Device:R_Pack04 RN9
+L Device:R_Pack04 RN5
 U 1 1 5FD84D43
 P 4350 6650
-F 0 "RN9" V 3933 6650 50  0000 C CNN
+F 0 "RN5" V 3933 6650 50  0000 C CNN
 F 1 "47" V 4024 6650 50  0000 C CNN
 F 2 "Resistor_SMD:R_Array_Convex_4x0603" V 4625 6650 50  0001 C CNN
@@
 IRQ
 $Comp
-L Device:R_Small R25
+L Device:R_Small R37
 U 1 1 5F54C08B
 P 1750 2700
-F 0 "R25" H 1809 2746 50  0000 L CNN
+F 0 "R37" H 1809 2746 50  0000 L CNN
 F 1 "4k7" H 1809 2655 50  0000 L CNN
 F 2 "Resistor_SMD:R_0603_1608Metric" H 1750 2700 50  0001 C CNN
@@
 $EndComp
 $Comp
-L power:+3.3V #PWR0115
+L power:+3.3V #PWR0114
 U 1 1 5F54C091
 P 1750 2600
-F 0 "#PWR0115" H 1750 2450 50  0001 C CNN
+F 0 "#PWR0114" H 1750 2450 50  0001 C CNN
 F 1 "+3.3V" H 1765 2773 50  0000 C CNN
 F 2 "" H 1750 2600 50  0001 C CNN

Commit message: Dump.
Connections:
- net SPIRAM_CS: now also U8.13 (IOB_24a); no longer U8.12 (IOB_22b)
- net SPIRAM_D0: now also U8.19 (IOB_29b); no longer U8.18 (IOB_31b)
- net SPIRAM_D1: now also U8.12 (IOB_22b); no longer U8.19 (IOB_29b)
- net SPIRAM_D2: now also U8.18 (IOB_31b); no longer U8.20 (IOB_25b_G3)
- net SPIRAM_SCK: now also U8.20 (IOB_25b_G3); no longer U8.13 (IOB_24a)
Changed lines of the file:
@@
 $Descr A4 11693 8268
 encoding utf-8
-Sheet 6 9
+Sheet 5 9
 Title ""
 Date ""
@@
 Text GLabel 9350 1750 0    39   3State ~ 0
 SPIRAM_D3
-Text GLabel 5600 3450 0    39   Output ~ 0
+Text GLabel 5600 3550 0    39   Output ~ 0
 SPIRAM_SCK
+Text GLabel 5600 3650 0    39   3State ~ 0
+SPIRAM_D0
+Text GLabel 5600 3250 0    39   3State ~ 0
+SPIRAM_D1
 Text GLabel 5600 3750 0    39   3State ~ 0
-SPIRAM_D0
-Text GLabel 5600 3650 0    39   3State ~ 0
-SPIRAM_D1
-Text GLabel 5600 3550 0    39   3State ~ 0
 SPIRAM_D2
 Text GLabel 5600 3350 0    39   3State ~ 0
@@
 	9450 1250 9350 1250
 Connection ~ 9450 1250
-Text GLabel 5600 3250 0    39   Output ~ 0
+Text GLabel 5600 3450 0    39   Output ~ 0
 SPIRAM_CS
 Wire Wire Line
