File: fpga.sch (KiCad schematic (older format))
At the start: 22 parts, among them U8 ICE40UP5K-SG48ITR, U9 LY68L6400

Commit message: Dump!
Connections:
- wire segments 33 -> 56
Other:
- moved on the sheet: C30, C31, R38, R39, U8C
Changed lines of the file:
@@
 L FPGA_Lattice:ICE40UP5K-SG48ITR U8
 U 3 1 5F52F020
-P 4950 6650
-F 0 "U8" H 4850 5950 50  0000 L CNN
-F 1 "ICE40UP5K-SG48ITR" H 4550 5850 50  0000 L CNN
-F 2 "Package_DFN_QFN:QFN-48-1EP_7x7mm_P0.5mm_EP5.6x5.6mm" H 4950 5300 50  0001 C CNN
-F 3 "http://www.latticesemi.com/Products/FPGAandCPLD/iCE40Ultra" H 4550 7650 50  0001 C CNN
-F 4 "-" H 4950 6650 50  0001 C CNN "LCSC"
-F 5 "842-40UP5KSG48ITR" H 4950 6650 50  0001 C CNN "Mouser"
-F 6 "5.29" H 4950 6650 50  0001 C CNN "Price"
-F 7 "N" H 4950 6650 50  0001 C CNN "Sponsored"
-	3    4950 6650
+P 5550 6650
+F 0 "U8" H 5450 5950 50  0000 L CNN
+F 1 "ICE40UP5K-SG48ITR" H 5150 5850 50  0000 L CNN
+F 2 "Package_DFN_QFN:QFN-48-1EP_7x7mm_P0.5mm_EP5.6x5.6mm" H 5550 5300 50  0001 C CNN
+F 3 "http://www.latticesemi.com/Products/FPGAandCPLD/iCE40Ultra" H 5150 7650 50  0001 C CNN
+F 4 "-" H 5550 6650 50  0001 C CNN "LCSC"
+F 5 "842-40UP5KSG48ITR" H 5550 6650 50  0001 C CNN "Mouser"
+F 6 "5.29" H 5550 6650 50  0001 C CNN "Price"
+F 7 "N" H 5550 6650 50  0001 C CNN "Sponsored"
+	3    5550 6650
 	1    0    0    -1
 $EndComp
@@
 	1    0    0    -1
 $EndComp
-Text HLabel 2900 6850 0    39   Output ~ 0
+Text HLabel 5600 3150 0    39   Output ~ 0
 LCD_RS
-Text HLabel 2900 6950 0    39   Output ~ 0
+Text HLabel 2900 5750 0    39   Output ~ 0
 LCD_WR
 Text HLabel 2900 5650 0    39   Input ~ 0
@@
 L power:+3.3V #PWR0120
 U 1 1 5F32B7AB
-P 4950 5950
-F 0 "#PWR0120" H 4950 5800 50  0001 C CNN
-F 1 "+3.3V" H 4965 6123 50  0000 C CNN
-F 2 "" H 4950 5950 50  0001 C CNN
-F 3 "" H 4950 5950 50  0001 C CNN
-	1    4950 5950
+P 5300 5950
+F 0 "#PWR0120" H 5300 5800 50  0001 C CNN
+F 1 "+3.3V" H 5315 6123 50  0000 C CNN
+F 2 "" H 5300 5950 50  0001 C CNN
+F 3 "" H 5300 5950 50  0001 C CNN
+	1    5300 5950
 	1    0    0    -1
 $EndComp
@@
 $EndComp
 $Comp
-L power:+3.3V #PWR0122
-U 1 1 5F48A900
-P 9300 6050
-F 0 "#PWR0122" H 9300 5900 50  0001 C CNN
-F 1 "+3.3V" H 9315 6223 50  0000 C CNN
-F 2 "" H 9300 6050 50  0001 C CNN
-F 3 "" H 9300 6050 50  0001 C CNN
-	1    9300 6050
-	1    0    0    -1
-$EndComp
-$Comp
 L power:GND #PWR0107
 U 1 1 5F503F48
@@
 Text HLabel 800  2950 1    39   UnSpc ~ 0
 SPI_CS
-Text HLabel 2900 6750 0    39   Output ~ 0
+Text HLabel 5600 3050 0    39   Output ~ 0
 IRQ
 $Comp
 L Device:C_Small C30
 U 1 1 5F618B63
-P 4050 3400
-F 0 "C30" H 3958 3354 50  0000 R CNN
-F 1 "C_Small" H 3958 3445 50  0000 R CNN
-F 2 "Capacitor_SMD:C_0603_1608Metric" H 4050 3400 50  0001 C CNN
-F 3 "~" H 4050 3400 50  0001 C CNN
-F 4 "0.0020" H 4050 3400 50  0001 C CNN "Price"
-F 5 "N" H 4050 3400 50  0001 C CNN "Sponsored"
-	1    4050 3400
+P 1350 7200
+F 0 "C30" H 1258 7154 50  0000 R CNN
+F 1 "C_Small" H 1258 7245 50  0000 R CNN
+F 2 "Capacitor_SMD:C_0603_1608Metric" H 1350 7200 50  0001 C CNN
+F 3 "~" H 1350 7200 50  0001 C CNN
+F 4 "0.0020" H 1350 7200 50  0001 C CNN "Price"
+F 5 "N" H 1350 7200 50  0001 C CNN "Sponsored"
+	1    1350 7200
 	-1   0    0    1
 $EndComp
 Wire Wire Line
-	5600 3050 4850 3050
-Wire Wire Line
-	5600 3150 4850 3150
+	2900 6750 2150 6750
+Wire Wire Line
+	2900 6950 2150 6950
 $Comp
 L Device:R_Small R38
 U 1 1 5F67E775
-P 4750 3050
-F 0 "R38" V 4850 3050 50  0000 C CNN
-F 1 "TBD" V 4750 3050 50  0000 C CNN
-F 2 "Resistor_SMD:R_0603_1608Metric" H 4750 3050 50  0001 C CNN
-F 3 "~" H 4750 3050 50  0001 C CNN
-F 4 "0.0005" H 4750 3050 50  0001 C CNN "Price"
-F 5 "-" H 4750 3050 50  0001 C CNN "LCSC"
-F 6 "-" H 4750 3050 50  0001 C CNN "Mouser"
-F 7 "N" H 4750 3050 50  0001 C CNN "Sponsored"
-	1    4750 3050
+P 2050 6750
+F 0 "R38" V 2150 6750 50  0000 C CNN
+F 1 "TBD" V 2050 6750 50  0000 C CNN
+F 2 "Resistor_SMD:R_0603_1608Metric" H 2050 6750 50  0001 C CNN
+F 3 "~" H 2050 6750 50  0001 C CNN
+F 4 "0.0005" H 2050 6750 50  0001 C CNN "Price"
+F 5 "-" H 2050 6750 50  0001 C CNN "LCSC"
+F 6 "-" H 2050 6750 50  0001 C CNN "Mouser"
+F 7 "N" H 2050 6750 50  0001 C CNN "Sponsored"
+	1    2050 6750
 	0    -1   -1   0
 $EndComp
@@
 L Device:R_Small R39
 U 1 1 5F684417
-P 4750 3150
-F 0 "R39" V 4650 3150 50  0000 C CNN
-F 1 "TBD" V 4750 3150 50  0000 C CNN
-F 2 "Resistor_SMD:R_0603_1608Metric" H 4750 3150 50  0001 C CNN
-F 3 "~" H 4750 3150 50  0001 C CNN
-F 4 "0.0005" H 4750 3150 50  0001 C CNN "Price"
-F 5 "-" H 4750 3150 50  0001 C CNN "LCSC"
-F 6 "-" H 4750 3150 50  0001 C CNN "Mouser"
-F 7 "N" H 4750 3150 50  0001 C CNN "Sponsored"
-	1    4750 3150
+P 2050 6950
+F 0 "R39" V 1950 6950 50  0000 C CNN
+F 1 "TBD" V 2050 6950 50  0000 C CNN
+F 2 "Resistor_SMD:R_0603_1608Metric" H 2050 6950 50  0001 C CNN
+F 3 "~" H 2050 6950 50  0001 C CNN
+F 4 "0.0005" H 2050 6950 50  0001 C CNN "Price"
+F 5 "-" H 2050 6950 50  0001 C CNN "LCSC"
+F 6 "-" H 2050 6950 50  0001 C CNN "Mouser"
+F 7 "N" H 2050 6950 50  0001 C CNN "Sponsored"
+	1    2050 6950
 	0    -1   -1   0
 $EndComp
@@
 L Device:C_Small C31
 U 1 1 5F688EB1
-P 4550 3400
-F 0 "C31" H 4458 3354 50  0000 R CNN
-F 1 "C_Small" H 4458 3445 50  0000 R CNN
-F 2 "Capacitor_SMD:C_0603_1608Metric" H 4550 3400 50  0001 C CNN
-F 3 "~" H 4550 3400 50  0001 C CNN
-F 4 "0.0020" H 4550 3400 50  0001 C CNN "Price"
-F 5 "N" H 4550 3400 50  0001 C CNN "Sponsored"
-	1    4550 3400
+P 1850 7200
+F 0 "C31" H 1758 7154 50  0000 R CNN
+F 1 "C_Small" H 1758 7245 50  0000 R CNN
+F 2 "Capacitor_SMD:C_0603_1608Metric" H 1850 7200 50  0001 C CNN
+F 3 "~" H 1850 7200 50  0001 C CNN
+F 4 "0.0020" H 1850 7200 50  0001 C CNN "Price"
+F 5 "N" H 1850 7200 50  0001 C CNN "Sponsored"
+	1    1850 7200
 	-1   0    0    1
 $EndComp
 Wire Wire Line
-	4650 3150 4550 3150
-Wire Wire Line
-	4550 3150 4550 3300
-Wire Wire Line
-	4650 3050 4050 3050
-Wire Wire Line
-	4050 3050 4050 3300
+	1950 6950 1850 6950
+Wire Wire Line
+	1850 6950 1850 7100
+Wire Wire Line
+	1950 6750 1350 6750
 $Comp
 L power:GND #PWR0119
 U 1 1 5F68C71B
-P 4550 3500
-F 0 "#PWR0119" H 4550 3250 50  0001 C CNN
-F 1 "GND" H 4555 3327 50  0000 C CNN
-F 2 "" H 4550 3500 50  0001 C CNN
-F 3 "" H 4550 3500 50  0001 C CNN
-	1    4550 3500
+P 1850 7300
+F 0 "#PWR0119" H 1850 7050 50  0001 C CNN
+F 1 "GND" H 1855 7127 50  0000 C CNN
+F 2 "" H 1850 7300 50  0001 C CNN
+F 3 "" H 1850 7300 50  0001 C CNN
+	1    1850 7300
 	1    0    0    -1
 $EndComp
@@
 L power:GND #PWR0118
 U 1 1 5F68DF1A
-P 4050 3500
-F 0 "#PWR0118" H 4050 3250 50  0001 C CNN
-F 1 "GND" H 4055 3327 50  0000 C CNN
-F 2 "" H 4050 3500 50  0001 C CNN
-F 3 "" H 4050 3500 50  0001 C CNN
-	1    4050 3500
-	1    0    0    -1
-$EndComp
-Wire Wire Line
-	4550 3150 3950 3150
-Connection ~ 4550 3150
-Wire Wire Line
-	4050 3050 3950 3050
-Connection ~ 4050 3050
-Text HLabel 3950 3050 0    39   Output ~ 0
+P 1350 7300
+F 0 "#PWR0118" H 1350 7050 50  0001 C CNN
+F 1 "GND" H 1355 7127 50  0000 C CNN
+F 2 "" H 1350 7300 50  0001 C CNN
+F 3 "" H 1350 7300 50  0001 C CNN
+	1    1350 7300
+	1    0    0    -1
+$EndComp
+Wire Wire Line
+	1850 6950 1250 6950
+Connection ~ 1850 6950
+Wire Wire Line
+	1350 6750 1250 6750
+Connection ~ 1350 6750
+Text HLabel 1250 6750 0    39   Output ~ 0
 AUDO_L
-Text HLabel 3950 3150 0    39   Output ~ 0
+Text HLabel 1250 6950 0    39   Output ~ 0
 AUDO_R
 Text HLabel 4150 6650 0    50   BiDi ~ 0
@@
 Text HLabel 4150 6850 0    50   BiDi ~ 0
 PMOD_4
-Text HLabel 4150 6750 0    50   BiDi ~ 0
-PMOD_5
 Text HLabel 4150 6550 0    50   BiDi ~ 0
 PMOD_6
@@
 Text HLabel 4150 6950 0    50   BiDi ~ 0
 PMOD_8
-Text HLabel 4150 7050 0    50   BiDi ~ 0
-PMOD_3
 Text HLabel 2900 6150 0    39   Output ~ 0
 LCD_D3
@@
 Text HLabel 2900 6650 0    39   Output ~ 0
 LCD_D7
-Text HLabel 2900 5750 0    39   Output ~ 0
+Text HLabel 2900 6850 0    39   Output ~ 0
 LCD_ENABLE
 Text HLabel 2900 6450 0    39   Input ~ 0
@@
 	1    0    0    -1
 $EndComp
+$Comp
+L power:+1V2 #PWR0122
+U 1 1 5FB6D63F
+P 9300 6050
+F 0 "#PWR0122" H 9300 5900 50  0001 C CNN
+F 1 "+1V2" H 9315 6223 50  0000 C CNN
+F 2 "" H 9300 6050 50  0001 C CNN
+F 3 "" H 9300 6050 50  0001 C CNN
+	1    9300 6050
+	1    0    0    -1
+$EndComp
+Wire Wire Line
+	1350 6750 1350 7100
+Text HLabel 4150 6750 0    50   BiDi ~ 0
+PMOD_5
+Text HLabel 4150 7050 0    50   BiDi ~ 0
+PMOD_3
+Wire Wire Line
+	4550 6750 4700 6750
+Wire Wire Line
+	4700 6750 4900 7050
+Wire Wire Line
+	4900 7050 5150 7050
+Wire Wire Line
+	5150 7150 5050 7150
+Wire Wire Line
+	4700 6650 4550 6650
+Wire Wire Line
+	4700 6650 5050 7150
+Wire Wire Line
+	5150 6950 5000 6950
+Wire Wire Line
+	5000 6950 4750 6550
+Wire Wire Line
+	4750 6550 4550 6550
+Wire Wire Line
+	5150 6750 5000 6750
+Wire Wire Line
+	5000 6750 4800 6450
+Wire Wire Line
+	4800 6450 4550 6450
+Wire Wire Line
+	5150 6550 5050 6550
+Wire Wire Line
+	5050 6550 4700 7150
+Wire Wire Line
+	4700 7150 4550 7150
+Wire Wire Line
+	5000 6450 4650 7050
+Wire Wire Line
+	4650 7050 4550 7050
+Wire Wire Line
+	5000 6450 5150 6450
+Wire Wire Line
+	5150 6850 4700 6850
+Wire Wire Line
+	4700 6850 4600 6950
+Wire Wire Line
+	4600 6950 4550 6950
+Wire Wire Line
+	4750 6650 5150 6650
+Wire Wire Line
+	4550 6850 4750 6650
 $EndSCHEMATC

Commit message: Routed and 0 DRC errors
Changed lines of the file:
@@
 L power:+3.3V #PWR0120
 U 1 1 5F32B7AB
-P 5300 5950
-F 0 "#PWR0120" H 5300 5800 50  0001 C CNN
-F 1 "+3.3V" H 5315 6123 50  0000 C CNN
-F 2 "" H 5300 5950 50  0001 C CNN
-F 3 "" H 5300 5950 50  0001 C CNN
-	1    5300 5950
+P 5550 5950
+F 0 "#PWR0120" H 5550 5800 50  0001 C CNN
+F 1 "+3.3V" H 5565 6123 50  0000 C CNN
+F 2 "" H 5550 5950 50  0001 C CNN
+F 3 "" H 5550 5950 50  0001 C CNN
+	1    5550 5950
 	1    0    0    -1
 $EndComp

Commit message: Dump.
Parts:
- C27, C29, C32, C33, C34, C35, C36: Price 0.0020 -> (none)
- C28: LCSC (none) -> C307461; Price 0.0020 -> (none)
- C30, C31: value C_Small -> TBD; LCSC (none) -> -; Price 0.0020 -> (none)
- R33, R35, R36: LCSC - -> C15458; Price 0.0005 -> (none)
- R34, R38, R39: Price 0.0005 -> (none)
- R37: LCSC - -> C269694; Price 0.0005 -> (none)
- R40: LCSC - -> C115324; Price 0.0005 -> (none)
- RN5, RN6: LCSC - -> C327045; Price 0.0042 -> (none)
- U8: Price 5.29 -> (none)
- U9: Price 0.64 -> (none)
Connections:
- net labels added: AUDIO_L, AUDIO_R
- net labels removed: AUDO_L, AUDO_R
Changed lines of the file:
@@
 F 4 "-" H 3300 6250 50  0001 C CNN "LCSC"
 F 5 "842-40UP5KSG48ITR" H 3300 6250 50  0001 C CNN "Mouser"
-F 6 "5.29" H 3300 6250 50  0001 C CNN "Price"
+F 6 "" H 3300 6250 50  0001 C CNN "Price"
 F 7 "N" H 3300 6250 50  0001 C CNN "Sponsored"
 	1    3300 6250
@@
 F 4 "-" H 6100 3250 50  0001 C CNN "LCSC"
 F 5 "842-40UP5KSG48ITR" H 6100 3250 50  0001 C CNN "Mouser"
-F 6 "5.29" H 6100 3250 50  0001 C CNN "Price"
+F 6 "" H 6100 3250 50  0001 C CNN "Price"
 F 7 "N" H 6100 3250 50  0001 C CNN "Sponsored"
 	2    6100 3250
@@
 F 4 "-" H 5550 6650 50  0001 C CNN "LCSC"
 F 5 "842-40UP5KSG48ITR" H 5550 6650 50  0001 C CNN "Mouser"
-F 6 "5.29" H 5550 6650 50  0001 C CNN "Price"
+F 6 "" H 5550 6650 50  0001 C CNN "Price"
 F 7 "N" H 5550 6650 50  0001 C CNN "Sponsored"
 	3    5550 6650
@@
 F 4 "-" H 2200 1200 50  0001 C CNN "LCSC"
 F 5 "842-40UP5KSG48ITR" H 2200 1200 50  0001 C CNN "Mouser"
-F 6 "5.29" H 2200 1200 50  0001 C CNN "Price"
+F 6 "" H 2200 1200 50  0001 C CNN "Price"
 F 7 "N" H 2200 1200 50  0001 C CNN "Sponsored"
 	4    2200 1200
@@
 F 2 "Resistor_SMD:R_0603_1608Metric" H 1050 1500 50  0001 C CNN
 F 3 "~" H 1050 1500 50  0001 C CNN
-F 4 "0.0005" H 1050 1500 50  0001 C CNN "Price"
+F 4 "" H 1050 1500 50  0001 C CNN "Price"
 F 5 "C25201" H 1050 1500 50  0001 C CNN "LCSC"
 F 6 "-" H 1050 1500 50  0001 C CNN "Mouser"
@@
 F 3 "~" H 850 1700 50  0001 C CNN
 F 4 "C14663" H 850 1700 50  0001 C CNN "LCSC"
-F 5 "0.0020" H 850 1700 50  0001 C CNN "Price"
+F 5 "" H 850 1700 50  0001 C CNN "Price"
 F 6 "-" H 850 1700 50  0001 C CNN "Mouser"
 F 7 "N" H 850 1700 50  0001 C CNN "Sponsored"
@@
 F 2 "Capacitor_SMD:C_0603_1608Metric" H 1250 1700 50  0001 C CNN
 F 3 "~" H 1250 1700 50  0001 C CNN
-F 4 "0.0020" H 1250 1700 50  0001 C CNN "Price"
+F 4 "" H 1250 1700 50  0001 C CNN "Price"
 F 5 "N" H 1250 1700 50  0001 C CNN "Sponsored"
+F 6 "C307461" H 1250 1700 50  0001 C CNN "LCSC"
 	1    1250 1700
 	1    0    0    -1
@@
 F 3 "~" H 1650 1700 50  0001 C CNN
 F 4 "C14663" H 1650 1700 50  0001 C CNN "LCSC"
-F 5 "0.0020" H 1650 1700 50  0001 C CNN "Price"
+F 5 "" H 1650 1700 50  0001 C CNN "Price"
 F 6 "-" H 1650 1700 50  0001 C CNN "Mouser"
 F 7 "N" H 1650 1700 50  0001 C CNN "Sponsored"
@@
 F 2 "Resistor_SMD:R_0603_1608Metric" H 1100 3050 50  0001 C CNN
 F 3 "~" H 1100 3050 50  0001 C CNN
-F 4 "0.0005" H 1100 3050 50  0001 C CNN "Price"
-F 5 "-" H 1100 3050 50  0001 C CNN "LCSC"
+F 4 "" H 1100 3050 50  0001 C CNN "Price"
+F 5 "C15458" H 1100 3050 50  0001 C CNN "LCSC"
 F 6 "-" H 1100 3050 50  0001 C CNN "Mouser"
 F 7 "N" H 1100 3050 50  0001 C CNN "Sponsored"
@@
 F 2 "Resistor_SMD:R_0603_1608Metric" H 1400 2700 50  0001 C CNN
 F 3 "~" H 1400 2700 50  0001 C CNN
-F 4 "0.0005" H 1400 2700 50  0001 C CNN "Price"
-F 5 "-" H 1400 2700 50  0001 C CNN "LCSC"
+F 4 "" H 1400 2700 50  0001 C CNN "Price"
+F 5 "C15458" H 1400 2700 50  0001 C CNN "LCSC"
 F 6 "-" H 1400 2700 50  0001 C CNN "Mouser"
 F 7 "N" H 1400 2700 50  0001 C CNN "Sponsored"
@@
 F 4 "C261881" H 10000 1500 50  0001 C CNN "LCSC"
 F 5 "-" H 10000 1500 50  0001 C CNN "Mouser"
-F 6 "0.64" H 10000 1500 50  0001 C CNN "Price"
+F 6 "" H 10000 1500 50  0001 C CNN "Price"
 F 7 "Y" H 10000 1500 50  0001 C CNN "Sponsored"
 	1    10000 1500
@@
 F 2 "Resistor_SMD:R_0603_1608Metric" H 9450 1050 50  0001 C CNN
 F 3 "~" H 9450 1050 50  0001 C CNN
-F 4 "0.0005" H 9450 1050 50  0001 C CNN "Price"
-F 5 "-" H 9450 1050 50  0001 C CNN "LCSC"
+F 4 "" H 9450 1050 50  0001 C CNN "Price"
+F 5 "C115324" H 9450 1050 50  0001 C CNN "LCSC"
 F 6 "-" H 9450 1050 50  0001 C CNN "Mouser"
 F 7 "N" H 9450 1050 50  0001 C CNN "Sponsored"
@@
 F 3 "~" H 10100 6150 50  0001 C CNN
 F 4 "C14663" H 10100 6150 50  0001 C CNN "LCSC"
-F 5 "0.0020" H 10100 6150 50  0001 C CNN "Price"
+F 5 "" H 10100 6150 50  0001 C CNN "Price"
 F 6 "-" H 10100 6150 50  0001 C CNN "Mouser"
 F 7 "N" H 10100 6150 50  0001 C CNN "Sponsored"
@@
 F 3 "~" H 10900 6150 50  0001 C CNN
 F 4 "C14663" H 10900 6150 50  0001 C CNN "LCSC"
-F 5 "0.0020" H 10900 6150 50  0001 C CNN "Price"
+F 5 "" H 10900 6150 50  0001 C CNN "Price"
 F 6 "-" H 10900 6150 50  0001 C CNN "Mouser"
 F 7 "N" H 10900 6150 50  0001 C CNN "Sponsored"
@@
 F 3 "~" H 10500 6150 50  0001 C CNN
 F 4 "C14663" H 10500 6150 50  0001 C CNN "LCSC"
-F 5 "0.0020" H 10500 6150 50  0001 C CNN "Price"
+F 5 "" H 10500 6150 50  0001 C CNN "Price"
 F 6 "-" H 10500 6150 50  0001 C CNN "Mouser"
 F 7 "N" H 10500 6150 50  0001 C CNN "Sponsored"
@@
 F 3 "~" H 9700 6150 50  0001 C CNN
 F 4 "C14663" H 9700 6150 50  0001 C CNN "LCSC"
-F 5 "0.0020" H 9700 6150 50  0001 C CNN "Price"
+F 5 "" H 9700 6150 50  0001 C CNN "Price"
 F 6 "-" H 9700 6150 50  0001 C CNN "Mouser"
 F 7 "N" H 9700 6150 50  0001 C CNN "Sponsored"
@@
 F 3 "~" H 9300 6150 50  0001 C CNN
 F 4 "C14663" H 9300 6150 50  0001 C CNN "LCSC"
-F 5 "0.0020" H 9300 6150 50  0001 C CNN "Price"
+F 5 "" H 9300 6150 50  0001 C CNN "Price"
 F 6 "-" H 9300 6150 50  0001 C CNN "Mouser"
 F 7 "N" H 9300 6150 50  0001 C CNN "Sponsored"
@@
 F 2 "Resistor_SMD:R_0603_1608Metric" H 800 3050 50  0001 C CNN
 F 3 "~" H 800 3050 50  0001 C CNN
-F 4 "0.0005" H 800 3050 50  0001 C CNN "Price"
-F 5 "-" H 800 3050 50  0001 C CNN "LCSC"
+F 4 "" H 800 3050 50  0001 C CNN "Price"
+F 5 "C15458" H 800 3050 50  0001 C CNN "LCSC"
 F 6 "-" H 800 3050 50  0001 C CNN "Mouser"
 F 7 "N" H 800 3050 50  0001 C CNN "Sponsored"
@@
 P 1350 7200
 F 0 "C30" H 1258 7154 50  0000 R CNN
-F 1 "C_Small" H 1258 7245 50  0000 R CNN
+F 1 "TBD" H 1258 7245 50  0000 R CNN
 F 2 "Capacitor_SMD:C_0603_1608Metric" H 1350 7200 50  0001 C CNN
 F 3 "~" H 1350 7200 50  0001 C CNN
-F 4 "0.0020" H 1350 7200 50  0001 C CNN "Price"
+F 4 "" H 1350 7200 50  0001 C CNN "Price"
 F 5 "N" H 1350 7200 50  0001 C CNN "Sponsored"
+F 6 "-" H 1350 7200 50  0001 C CNN "LCSC"
 	1    1350 7200
 	-1   0    0    1
@@
 F 2 "Resistor_SMD:R_0603_1608Metric" H 2050 6750 50  0001 C CNN
 F 3 "~" H 2050 6750 50  0001 C CNN
-F 4 "0.0005" H 2050 6750 50  0001 C CNN "Price"
+F 4 "" H 2050 6750 50  0001 C CNN "Price"
 F 5 "-" H 2050 6750 50  0001 C CNN "LCSC"
 F 6 "-" H 2050 6750 50  0001 C CNN "Mouser"
@@
 F 2 "Resistor_SMD:R_0603_1608Metric" H 2050 6950 50  0001 C CNN
 F 3 "~" H 2050 6950 50  0001 C CNN
-F 4 "0.0005" H 2050 6950 50  0001 C CNN "Price"
+F 4 "" H 2050 6950 50  0001 C CNN "Price"
 F 5 "-" H 2050 6950 50  0001 C CNN "LCSC"
 F 6 "-" H 2050 6950 50  0001 C CNN "Mouser"
@@
 P 1850 7200
 F 0 "C31" H 1758 7154 50  0000 R CNN
-F 1 "C_Small" H 1758 7245 50  0000 R CNN
+F 1 "TBD" H 1758 7245 50  0000 R CNN
 F 2 "Capacitor_SMD:C_0603_1608Metric" H 1850 7200 50  0001 C CNN
 F 3 "~" H 1850 7200 50  0001 C CNN
-F 4 "0.0020" H 1850 7200 50  0001 C CNN "Price"
+F 4 "" H 1850 7200 50  0001 C CNN "Price"
 F 5 "N" H 1850 7200 50  0001 C CNN "Sponsored"
+F 6 "-" H 1850 7200 50  0001 C CNN "LCSC"
 	1    1850 7200
 	-1   0    0    1
@@
 Connection ~ 1350 6750
 Text HLabel 1250 6750 0    39   Output ~ 0
-AUDO_L
+AUDIO_L
 Text HLabel 1250 6950 0    39   Output ~ 0
-AUDO_R
-Text HLabel 4150 6650 0    50   BiDi ~ 0
+AUDIO_R
+Text HLabel 4150 6750 0    50   BiDi ~ 0
 PMOD_1
+Text HLabel 4150 6550 0    50   BiDi ~ 0
+PMOD_2
+Text HLabel 4150 6950 0    50   BiDi ~ 0
+PMOD_4
 Text HLabel 4150 6450 0    50   BiDi ~ 0
-PMOD_2
-Text HLabel 4150 6850 0    50   BiDi ~ 0
-PMOD_4
-Text HLabel 4150 6550 0    50   BiDi ~ 0
 PMOD_6
-Text HLabel 4150 7150 0    50   BiDi ~ 0
+Text HLabel 4150 7050 0    50   BiDi ~ 0
 PMOD_7
 $Comp
@@
 F 2 "Resistor_SMD:R_Array_Convex_4x0603" V 4625 6950 50  0001 C CNN
 F 3 "~" H 4350 6950 50  0001 C CNN
-F 4 "-" H 4350 6950 50  0001 C CNN "LCSC"
+F 4 "C327045" H 4350 6950 50  0001 C CNN "LCSC"
 F 5 "-" H 4350 6950 50  0001 C CNN "Mouser"
-F 6 "0.0042" H 4350 6950 50  0001 C CNN "Price"
+F 6 "" H 4350 6950 50  0001 C CNN "Price"
 F 7 "N" H 4350 6950 50  0001 C CNN "Sponsored"
 	1    4350 6950
@@
 F 2 "Resistor_SMD:R_Array_Convex_4x0603" V 4625 6650 50  0001 C CNN
 F 3 "~" H 4350 6650 50  0001 C CNN
-F 4 "-" H 4350 6650 50  0001 C CNN "LCSC"
+F 4 "C327045" H 4350 6650 50  0001 C CNN "LCSC"
 F 5 "-" H 4350 6650 50  0001 C CNN "Mouser"
-F 6 "0.0042" H 4350 6650 50  0001 C CNN "Price"
+F 6 "" H 4350 6650 50  0001 C CNN "Price"
 F 7 "N" H 4350 6650 50  0001 C CNN "Sponsored"
 	1    4350 6650
 	0    1    1    0
 $EndComp
-Text HLabel 4150 6950 0    50   BiDi ~ 0
+Text HLabel 4150 6850 0    50   BiDi ~ 0
 PMOD_8
 Text HLabel 2900 6150 0    39   Output ~ 0
@@
 F 2 "Resistor_SMD:R_0603_1608Metric" H 1750 2700 50  0001 C CNN
 F 3 "~" H 1750 2700 50  0001 C CNN
-F 4 "0.0005" H 1750 2700 50  0001 C CNN "Price"
-F 5 "-" H 1750 2700 50  0001 C CNN "LCSC"
+F 4 "" H 1750 2700 50  0001 C CNN "Price"
+F 5 "C269694" H 1750 2700 50  0001 C CNN "LCSC"
 F 6 "-" H 1750 2700 50  0001 C CNN "Mouser"
 F 7 "N" H 1750 2700 50  0001 C CNN "Sponsored"
@@
 Wire Wire Line
 	1350 6750 1350 7100
-Text HLabel 4150 6750 0    50   BiDi ~ 0
+Text HLabel 4150 6650 0    50   BiDi ~ 0
 PMOD_5
-Text HLabel 4150 7050 0    50   BiDi ~ 0
+Text HLabel 4150 7150 0    50   BiDi ~ 0
 PMOD_3
 Wire Wire Line

Commit message: Work in progress: prototype 2
Parts:
- removed C30, C31: TBD, Capacitor_SMD:C_0603_1608Metric, symbol Device:C_Small
- removed R38, R39: TBD, Resistor_SMD:R_0603_1608Metric, symbol Device:R_Small
- R33, R35: value 100k -> 10k
- R36: value 100k -> DNP
Connections:
- net labels removed: +2V5, AUDIO_L, AUDIO_R, LCD_ENABLE
- wire segments 56 -> 48
Other:
- moved on the sheet: R33, RN5, RN6, U8A, U8B, U8C

Commit message: More work on prototype 2
Other:
- note added: "Sorry, will clean this up later :-)"
Changed lines of the file:
@@
 $Descr A4 11693 8268
 encoding utf-8
-Sheet 8 9
+Sheet 7 9
 Title ""
-Date ""
-Rev ""
-Comp ""
+Date "2020-11-22"
+Rev "2"
+Comp "BADGE.TEAM"
 Comment1 ""
 Comment2 ""
@@
 $EndComp
 $Comp
-L power:+3.3V #PWR?
+L power:+3.3V #PWR0195
 U 1 1 5F8E28AC
 P 1800 1100
-F 0 "#PWR?" H 1800 950 50  0001 C CNN
+F 0 "#PWR0195" H 1800 950 50  0001 C CNN
 F 1 "+3.3V" H 1815 1273 50  0000 C CNN
 F 2 "" H 1800 1100 50  0001 C CNN
@@
 	0    -1   -1   0
 $EndComp
+Text Notes 7500 4150 3    50   ~ 0
+Sorry, will clean this up later :-)
 $EndSCHEMATC

Commit message: Schematic for prototype 2 is now complete, time for review! :D
Connections:
- net I2S_CLK: now reaches U8.38 (IOT_50b)
- net I2S_LR: now reaches U8.42 (IOT_51a)
- net I2S_DATA: now reaches U8.43 (IOT_49a)
Changed lines of the file:
@@
 Text Notes 7500 4150 3    50   ~ 0
 Sorry, will clean this up later :-)
+Text HLabel 3250 4650 0    39   Output ~ 0
+I2S_DATA
+Text HLabel 3250 4750 0    39   Output ~ 0
+I2S_CLK
+Text HLabel 3250 4850 0    39   Output ~ 0
+I2S_LR
 $EndSCHEMATC
