File: mch2021.sch (KiCad schematic (older format))
At the start: 55 parts, among them J2 USB_C_Receptacle_USB2.0, J3 QG-2864KLBEG01, SW4 SW_SPDT, U11 SY6280AAC, U3 SY6280AAC, U8 IR1261

Commit message: Finished work on initial schematic
Parts:
- removed C1, C12, C18, C19, C23, C28, C29, C30, C31, C33, C34, C35, C36, C37, C38, C39, C4, C7: 1u, Capacitor_SMD:C_0402_1005Metric, symbol Device:C
- removed C26: 4.7u, Capacitor_SMD:C_0603_1608Metric, symbol Device:C
- removed C27: 2.2u, Capacitor_SMD:C_0603_1608Metric, symbol Device:C
- removed D1, D10, D11, D12, D13, D14, D15, D2, D3, D4, D5, D6: WS2812B, corelib:SK6212SIDE, symbol LED:WS2812B
- removed D7: LED, LED_SMD:LED_0805_2012Metric_Castellated, symbol Device:LED
- removed J3: QG-2864KLBEG01, corelib:hotbar_30x0.7, symbol mch2021-rescue:QG-2864KLBEG01-corelib
- removed LS1: Speaker_Crystal, Buzzer_Beeper:Buzzer_Murata_PKMCS0909E4000-R1, symbol Device:Speaker_Crystal
- removed MK1: SPH0641LM4H-1, corelib:Knowles-SPH0641LM4H-1, symbol mch2021-rescue:SPH0641LM4H-1-corelib
- removed R10: 910k, Resistor_SMD:R_0603_1608Metric, symbol Device:R
- removed R11: 3.4k, Resistor_SMD:R_0603_1608Metric, symbol Device:R
- removed R12, R18, R19, R25, R26: 10k, Resistor_SMD:R_0603_1608Metric, symbol Device:R
- removed R9: 100R, Resistor_SMD:R_0603_1608Metric, symbol Device:R
- removed RN1: 100k, Resistor_SMD:R_Array_Convex_4x0603, symbol Device:R_Pack04
- removed SW4: SW_SPDT, Button_Switch_SMD:SW_SPDT_PCM12, symbol Switch:SW_SPDT
- removed TP10, TP11, TP9: TestPoint, TestPoint:TestPoint_Pad_D2.0mm, symbol Connector:TestPoint
- removed U11, U3: SY6280AAC, Package_TO_SOT_SMD:SOT-23-5, symbol Power_Management:AAT4610BIGV-1-T1
- removed U8: IR1261, OptoDevice:Vishay_MINICAST-3Pin, symbol Interface_Optical:TSMP58000
- added D1: RGB-5050, symbol led:RGB-5050
- added J2, J4: SAO, Connector_PinSocket_2.54mm:PinSocket_2x03_P2.54mm_Vertical, symbol Connector_Generic:Conn_02x03_Odd_Even
- added J3: AudioJack3, corelib:Boom-audiojack-PJ-320B, symbol Connector:AudioJack3
- added J5: Micro_SD_Card, corelib:MicroSD-SOFNG-TF-002-H18, symbol Connector:Micro_SD_Card
- added R3: 47, Resistor_SMD:R_0603_1608Metric, symbol Device:R_Small
- renumbered J2 to J1, R9 to R1, R10 to R2
Connections:
- net labels added: PWR_SDCARD
- net labels removed: 3V3, BUZZER, GATEDPOWER, GATEDPOWER_ENABLE, I2C_SCL, I2C_SDA, IR_RECV, IR_SEND, LEDPWR, LED_DIN_GATED, MIC, MICCLK, PWR_LED_ENABLE, SENSE_VBAT, SENSE_VUSB, VBAT
- wire segments 246 -> 235
- no-connect marks 1 -> 0
Other:
- moved on the sheet: J1, R1, R2

Commit message: Small fixes
Connections:
- net GND: now also J1.A1 (GND), J1.A12 (GND), J1.B1 (GND), J1.B12 (GND), J1.S1 (SHIELD)

Commit message: SPI RAM for the FPGA
Parts:
- added RN?: R_Pack04, symbol Device:R_Pack04
Connections:
- net AUDIO/I2S_BCLK: now also RN?.7 (R2.2)
- net AUDIO/I2S_DATA: now also RN?.5 (R4.2)
- net AUDIO/I2S_LRCK: now also RN?.6 (R3.2)
- net ESP32/I2S_BCLK: now also RN?.2 (R2.1)
- net ESP32/I2S_DATA: now also RN?.4 (R4.1)
- net ESP32/I2S_LRCK: now also RN?.3 (R3.1)
Other:
- moved on the sheet: D1
Changed lines of the file:
@@
 	6800 2600 6800 3300
 Wire Wire Line
-	6600 6100 6600 7300
-Wire Wire Line
 	6600 7300 6500 7300
 Wire Wire Line
-	6700 7400 6700 6200
-Wire Wire Line
 	6500 7400 6700 7400
 Wire Wire Line
-	6800 6300 6800 7500
-Wire Wire Line
 	6800 7500 6500 7500
 Wire Wire Line
@@
 	8600 2500 10000 2500
 Wire Wire Line
-	10000 2500 10000 5850
+	10000 2500 10000 5750
 Wire Wire Line
 	10100 2600 8600 2600
@@
 	9400 3700 9400 5200
 Wire Wire Line
-	8600 3000 8700 3000
-Wire Wire Line
-	8700 3000 8700 4500
-Wire Wire Line
 	8600 3100 8800 3100
 Wire Wire Line
@@
 Wire Wire Line
 	9300 3600 9300 5100
-Wire Wire Line
-	5750 3650 5750 5150
-Wire Wire Line
-	5850 3750 5850 5250
 Wire Wire Line
 	6900 4550 6500 4550
@@
 	3150 5350 6900 5350
 Wire Wire Line
-	6900 5150 5750 5150
-Connection ~ 5750 5150
-Wire Wire Line
-	5750 5150 5750 6350
-Wire Wire Line
-	5850 5250 6900 5250
-Connection ~ 5850 5250
-Wire Wire Line
-	5850 5250 5850 6350
-Wire Wire Line
-	6900 6100 6600 6100
-Wire Wire Line
-	6900 6200 6700 6200
-Wire Wire Line
-	6900 6300 6800 6300
-Wire Wire Line
-	8600 5750 9900 5750
-Wire Wire Line
 	9900 5750 9900 2400
 Wire Wire Line
-	8600 5850 10000 5850
-Wire Wire Line
-	8600 5950 10100 5950
-Wire Wire Line
-	10100 5950 10100 2600
-Wire Wire Line
 	9500 3800 9500 5300
 Wire Wire Line
@@
 Wire Wire Line
 	8800 4600 8600 4600
-Wire Wire Line
-	8700 4500 8600 4500
 Wire Wire Line
 	8600 4800 9000 4800
@@
 L led:RGB-5050 D1
 U 1 1 611CFAC6
-P 9000 6200
-F 0 "D1" V 9307 6075 50  0000 C CNN
-F 1 "RGB-5050" V 9216 6075 50  0000 C CNN
-F 2 "" H 9000 6050 60  0001 C CNN
-F 3 "" H 9000 6050 60  0001 C CNN
-	1    9000 6200
+P 9000 5900
+F 0 "D1" V 9307 5775 50  0000 C CNN
+F 1 "RGB-5050" V 9216 5775 50  0000 C CNN
+F 2 "" H 9000 5750 60  0001 C CNN
+F 3 "" H 9000 5750 60  0001 C CNN
+	1    9000 5900
 	0    1    1    0
 $EndComp
 Wire Wire Line
-	9000 6100 9100 6100
-Wire Wire Line
-	9100 6100 9100 6200
-Wire Wire Line
-	9100 6200 9000 6200
-Wire Wire Line
-	9000 6300 9100 6300
-Wire Wire Line
-	9100 6300 9100 6200
-Connection ~ 9100 6200
+	9000 5800 9100 5800
+Wire Wire Line
+	9100 5800 9100 5900
+Wire Wire Line
+	9100 5900 9000 5900
+Wire Wire Line
+	9000 6000 9100 6000
+Wire Wire Line
+	9100 6000 9100 5900
+Connection ~ 9100 5900
 $Comp
 L power:+3.3V #PWR09
 U 1 1 611F8813
-P 9100 6200
-F 0 "#PWR09" H 9100 6050 50  0001 C CNN
-F 1 "+3.3V" H 9000 6350 50  0000 L CNN
-F 2 "" H 9100 6200 50  0001 C CNN
-F 3 "" H 9100 6200 50  0001 C CNN
-	1    9100 6200
+P 9100 5900
+F 0 "#PWR09" H 9100 5750 50  0001 C CNN
+F 1 "+3.3V" H 9000 6050 50  0000 L CNN
+F 2 "" H 9100 5900 50  0001 C CNN
+F 3 "" H 9100 5900 50  0001 C CNN
+	1    9100 5900
 	0    1    1    0
 $EndComp
 Wire Wire Line
-	8600 6100 8750 6100
-Wire Wire Line
-	8750 6200 8600 6200
-Wire Wire Line
-	8600 6300 8750 6300
+	8600 5800 8750 5800
+Wire Wire Line
+	8750 5900 8600 5900
+Wire Wire Line
+	8600 6000 8750 6000
 $Sheet
 S 1000 3550 900  200
@@
 	1    0    0    -1
 $EndComp
+Wire Wire Line
+	6900 4950 3250 4950
+Wire Wire Line
+	5850 3750 5850 6350
+Wire Wire Line
+	5750 3650 5750 6350
 $Sheet
-S 6900 4450 1700 1950
+S 6900 4450 1700 1650
 U 5F526357
 F0 "FPGA" 50
@@
 F15 "LCD_RS" O R 8600 4600 50
 F16 "LCD_WR" O R 8600 4700 50
-F17 "LCD_CS" O R 8600 4500 50
-F18 "LCD_FMARK" I R 8600 5600 50
-F19 "LCD_ENABLE" O L 6900 5350 50
-F20 "I2C_SDA" T L 6900 5150 50
-F21 "I2C_SCL" I L 6900 5250 50
-F22 "I2S_IN_DATA" I R 8600 5750 50
-F23 "I2S_IN_LRCK" I R 8600 5850 50
-F24 "I2S_IN_BCLK" I R 8600 5950 50
-F25 "I2S_OUT_DATA" I L 6900 6100 50
-F26 "I2S_OUT_LRCK" I L 6900 6200 50
-F27 "I2S_OUT_BCLK" I L 6900 6300 50
-F28 "SPI_CS" I L 6900 4850 50
-F29 "UART_RX" I L 6900 5450 50
-F30 "UART_TX" O L 6900 5550 50
-F31 "CLK" I L 6900 5650 50
-F32 "RGB0" O R 8600 6100 50
-F33 "RGB1" O R 8600 6200 50
-F34 "RGB2" O R 8600 6300 50
+F17 "LCD_FMARK" I R 8600 5600 50
+F18 "LCD_ENABLE" O L 6900 5350 50
+F19 "I2S_OUT_DATA" I L 6900 5800 50
+F20 "I2S_OUT_LRCK" I L 6900 5900 50
+F21 "I2S_OUT_BCLK" I L 6900 6000 50
+F22 "SPI_CS" I L 6900 4850 50
+F23 "UART_RX" I L 6900 5450 50
+F24 "UART_TX" O L 6900 5550 50
+F25 "CLK" I L 6900 5650 50
+F26 "RGB0" O R 8600 5800 50
+F27 "RGB1" O R 8600 5900 50
+F28 "RGB2" O R 8600 6000 50
 $EndSheet
 Wire Wire Line
-	6900 4950 3250 4950
+	6600 5800 6900 5800
+Wire Wire Line
+	6700 5900 6900 5900
+Wire Wire Line
+	6900 6000 6800 6000
+Wire Wire Line
+	6800 6000 6800 6450
+Wire Wire Line
+	6700 5900 6700 6350
+Wire Wire Line
+	6600 5800 6600 6250
+$Comp
+L Device:R_Pack04 RN?
+U 1 1 5F3FEAC4
+P 10000 5950
+F 0 "RN?" H 9720 5904 50  0000 R CNN
+F 1 "R_Pack04" H 9720 5995 50  0000 R CNN
+F 2 "" V 10275 5950 50  0001 C CNN
+F 3 "~" H 10000 5950 50  0001 C CNN
+	1    10000 5950
+	-1   0    0    1
+$EndComp
+Wire Wire Line
+	10100 5750 10100 2600
+Wire Wire Line
+	9900 6150 9900 6250
+Wire Wire Line
+	9900 6250 6600 6250
+Connection ~ 6600 6250
+Wire Wire Line
+	6600 6250 6600 7300
+Wire Wire Line
+	10000 6150 10000 6350
+Wire Wire Line
+	10000 6350 6700 6350
+Connection ~ 6700 6350
+Wire Wire Line
+	6700 6350 6700 7400
+Wire Wire Line
+	10100 6450 6800 6450
+Wire Wire Line
+	10100 6150 10100 6450
+Connection ~ 6800 6450
+Wire Wire Line
+	6800 6450 6800 7500
 $EndSCHEMATC

Commit message: Fixes, removed I2S DAC
Parts:
- added C? (x2): C_Small, symbol Device:C_Small
- added J?: PMOD, symbol Connector_Generic:Conn_02x06_Counter_Clockwise
- RN?: value R_Pack04 -> TBD
Connections:
- net AUDIO/I2S_BCLK is gone; now on an unnamed net: RN?.7 (R2.2)
- net AUDIO/I2S_LRCK is gone; now on an unnamed net: RN?.6 (R3.2)
- net +3V3: now also J?.6 (Pin_6), J?.7 (Pin_7)
- net GND: now also J?.5 (Pin_5), J?.8 (Pin_8)
- net FPGA/AUDO_L: now reaches RN?.1 (R1.1)
- net at RN?.8 (R1.2): now also C?.1
- net AUDIO/AUDIO_L: no longer names the net of J3.T
- net AUDIO/AUDIO_L: now also C?.2
- net AUDIO/AUDIO_R: no longer names the net of J3.R
- net AUDIO/AUDIO_R: now also C?.1
- net AUDIO/I2S_DATA: no longer names the net of RN?.5 (R4.2)
- net AUDIO/I2S_DATA: now also C?.2
- net ESP32/I2S_BCLK renamed ESP32_AUDIO_L
- net ESP32/I2S_DATA renamed ESP32_AUDIO_R
- net ESP32/I2S_LRCK renamed FPGA/AUDO_R
- new net FPGA/PMOD_1: J?.1 (Pin_1)
- new net FPGA/PMOD_2: J?.2 (Pin_2)
- new net FPGA/PMOD_3: J?.3 (Pin_3)
- new net FPGA/PMOD_4: J?.4 (Pin_4)
- new net FPGA/PMOD_5: J?.12 (Pin_12)
- new net FPGA/PMOD_6: J?.11 (Pin_11)
- new net FPGA/PMOD_7: J?.10 (Pin_10)
- new net FPGA/PMOD_8: J?.9 (Pin_9)
- no-connect marks 0 -> 1
Other:
- moved on the sheet: D1, J2, J4, RN?

Commit message: Dump.
Parts:
- added D2: LED, LED_SMD:LED_0805_2012Metric_Castellated, symbol Device:LED
- added H1, H2, H3, H4: MountingHole_Pad, corecode:HOLE-M3-COND, symbol Mechanical:MountingHole_Pad
- added LS1: Speaker_Crystal, Buzzer_Beeper:Buzzer_Murata_PKMCS0909E4000-R1, symbol Device:Speaker_Crystal
- added R4: 100, Resistor_SMD:R_0603_1608Metric, symbol Device:R
- C1, C2: renamed from C?; footprint (none) -> Capacitor_SMD:C_0603_1608Metric; Price (none) -> 0.0020; Sponsored (none) -> N
- D1: footprint (none) -> LED_SMD:LED_RGB_5050-6; LCSC (none) -> C219409; Mouser (none) -> -; Price (none) -> 0.024; Sponsored (none) -> N
- J1: LCSC (none) -> C165948; Mouser (none) -> -; Price (none) -> 0.19; Sponsored (none) -> N
- J2, J4: LCSC (none) -> -; Mouser (none) -> -; Price (none) -> 0.03; Sponsored (none) -> N
- J3: footprint corelib:Boom-audiojack-PJ-320B -> custom:Boom-audiojack-PJ-320B; LCSC (none) -> C431535; Mouser (none) -> -; Price (none) -> 0.018; Sponsored (none) -> N
- J5: value Micro_SD_Card -> Micro SD card; footprint corelib:MicroSD-SOFNG-TF-002-H18 -> custom:MicroSD-SOFNG-TF-002-H18; LCSC (none) -> C125814; Mouser (none) -> -; Price (none) -> 0.044; Sponsored (none) -> N
- J6: renamed from J?; footprint (none) -> Connector_PinSocket_2.54mm:PinSocket_2x06_P2.54mm_Horizontal; symbol Connector_Generic:Conn_02x06_Counter_Clockwise -> Connector_Generic:Conn_02x06_Odd_Even; LCSC (none) -> C239357; Mouser (none) -> -; Price (none) -> 0.13; Sponsored (none) -> N
- R1, R2, R3: LCSC (none) -> -; Mouser (none) -> -; Price (none) -> 0.0005; Sponsored (none) -> N
- RN1: renamed from RN?; footprint (none) -> Resistor_SMD:R_Array_Convex_4x0603; LCSC (none) -> -; Mouser (none) -> -; Price (none) -> 0.0042; Sponsored (none) -> N
Connections:
- net +3V3: now also J6.1 (Pin_1), J6.2 (Pin_2); no longer J6.6 (Pin_6), J6.7 (Pin_7)
- net ESP32_AUDIO_L: now also RN1.7 (R2.2); no longer RN1.2 (R2.1)
- net ESP32_AUDIO_R: now also RN1.5 (R4.2); no longer RN1.4 (R4.1)
- net FPGA/AUDO_L: now also RN1.8 (R1.2); no longer RN1.1 (R1.1)
- net FPGA/AUDO_R: now also RN1.6 (R3.2); no longer RN1.3 (R3.1)
- net FPGA/PMOD_1: now also J6.12 (Pin_12); no longer J6.1 (Pin_1)
- net FPGA/PMOD_2: now also J6.10 (Pin_10); no longer J6.2 (Pin_2)
- net FPGA/PMOD_3: now also J6.8 (Pin_8); no longer J6.3 (Pin_3)
- net FPGA/PMOD_4: now also J6.6 (Pin_6); no longer J6.4 (Pin_4)
- net FPGA/PMOD_5: now also J6.11 (Pin_11); no longer J6.12 (Pin_12)
- net FPGA/PMOD_6: now also J6.9 (Pin_9); no longer J6.11 (Pin_11)
- net FPGA/PMOD_7: now also J6.7 (Pin_7); no longer J6.10 (Pin_10)
- net FPGA/PMOD_8: now also J6.5 (Pin_5); no longer J6.9 (Pin_9)
- net GND: now also J6.3 (Pin_3), J6.4 (Pin_4), D2.1 (K), H1.1, H2.1, H3.1, H4.1, LS1.1; no longer J6.5 (Pin_5), J6.8 (Pin_8)
- new net: C1.1, RN1.1 (R1.1), RN1.2 (R2.1)
- new net: C2.2, RN1.3 (R3.1), RN1.4 (R4.1)
- new net: D2.2 (A), R4.1
- new net ESP32/IR_TX: R4.2
- new net SPK: LS1.2
- no-connect marks 1 -> 0
Other:
- moved on the sheet: J5

Commit message: Dump.
Changed lines of the file:
@@
 	8700 750  8700 550
-Wire Wire Line
-	3450 750  3650 750
 Wire Wire Line
 	3650 850  3450 850
@@
 	8600 2400 9900 2400
 $Comp
-L power:GND #PWR026
+L power:GND #PWR022
 U 1 1 60AAA727
 P 10950 1800
-F 0 "#PWR026" H 10950 1550 50  0001 C CNN
+F 0 "#PWR022" H 10950 1550 50  0001 C CNN
 F 1 "GND" H 10955 1627 50  0000 C CNN
 F 2 "" H 10950 1800 50  0001 C CNN
@@
 $EndComp
 $Comp
-L power:GND #PWR021
+L power:GND #PWR019
 U 1 1 5FC38556
 P 10350 6050
-F 0 "#PWR021" H 10350 5800 50  0001 C CNN
+F 0 "#PWR019" H 10350 5800 50  0001 C CNN
 F 1 "GND" V 10355 5922 50  0000 R CNN
 F 2 "" H 10350 6050 50  0001 C CNN
@@
 $EndComp
 $Comp
-L power:+3.3V #PWR022
+L power:+3.3V #PWR020
 U 1 1 5FC4AEFB
 P 10350 6150
-F 0 "#PWR022" H 10350 6000 50  0001 C CNN
+F 0 "#PWR020" H 10350 6000 50  0001 C CNN
 F 1 "+3.3V" V 10365 6278 50  0000 L CNN
 F 2 "" H 10350 6150 50  0001 C CNN
@@
 F21 "SAO_IO0" B R 5400 2750 50
 F22 "SAO_IO1" B R 5400 2850 50
-F23 "CHARGING" I L 3650 750 50
-F24 "LCD_ENABLE_PAR" I L 3650 1950 50
-F25 "LCD_RESET" O L 3650 2150 50
-F26 "LCD_MODE" O L 3650 2250 50
-F27 "LCD_BACKLIGHT" O L 3650 2050 50
-F28 "MCO" O L 3650 1550 50
-F29 "SPI_CS_A" I R 5400 1850 50
-F30 "LCD_CS" O L 3650 2350 50
-F31 "FPGA_CS" O R 5400 2550 50
-F32 "SPI_CS_B" I R 5400 1950 50
-F33 "SPK" O R 5400 2200 50
+F23 "LCD_ENABLE_PAR" I L 3650 1950 50
+F24 "LCD_RESET" O L 3650 2150 50
+F25 "LCD_MODE" O L 3650 2250 50
+F26 "LCD_BACKLIGHT" O L 3650 2050 50
+F27 "MCO" O L 3650 1550 50
+F28 "SPI_CS_A" I R 5400 1850 50
+F29 "LCD_CS" O L 3650 2350 50
+F30 "FPGA_CS" O R 5400 2550 50
+F31 "SPI_CS_B" I R 5400 1950 50
+F32 "SPK" O R 5400 2200 50
 $EndSheet
 Wire Wire Line
@@
 F7 "FPGA_RESET" O L 3650 4000 50
 F8 "FPGA_CDONE" O L 3650 4100 50
+F9 "CHARGING" I R 5400 4100 50
 $EndSheet
 Wire Wire Line
@@
 $EndComp
 $Comp
-L power:GND #PWR023
+L power:GND #PWR021
 U 1 1 60CE727A
 P 10450 2100
-F 0 "#PWR023" H 10450 1850 50  0001 C CNN
+F 0 "#PWR021" H 10450 1850 50  0001 C CNN
 F 1 "GND" H 10455 1927 50  0000 C CNN
 F 2 "" H 10450 2100 50  0001 C CNN
@@
 	1    0    0    -1
 $EndComp
+Wire Wire Line
+	5400 4100 5450 4100
+Wire Wire Line
+	5450 4100 5450 4450
+Wire Wire Line
+	5450 4450 3400 4450
+Wire Wire Line
+	3400 4450 3400 1100
+Wire Wire Line
+	3400 1100 3550 1100
+Wire Wire Line
+	3550 1100 3550 750
+Wire Wire Line
+	3550 750  3450 750
 $EndSCHEMATC

Commit message: Dump.
Parts:
- removed D2: LED, LED_SMD:LED_0805_2012Metric_Castellated, symbol Device:LED
- removed R4: 100, Resistor_SMD:R_0603_1608Metric, symbol Device:R
Connections:
- net at J2.6 (Pin_6): no longer R3.1
Changed lines of the file:
@@
 $EndComp
-Wire Wire Line
-	6050 2100 6900 2100
-Wire Wire Line
-	6900 2200 5950 2200
 Wire Wire Line
 	6800 2600 6900 2600
@@
 	8600 2400 9900 2400
 $Comp
-L power:GND #PWR022
+L power:GND #PWR021
 U 1 1 60AAA727
 P 10950 1800
-F 0 "#PWR022" H 10950 1550 50  0001 C CNN
+F 0 "#PWR021" H 10950 1550 50  0001 C CNN
 F 1 "GND" H 10955 1627 50  0000 C CNN
 F 2 "" H 10950 1800 50  0001 C CNN
@@
 Wire Wire Line
 	2250 3650 2350 3650
-Wire Wire Line
-	2350 3300 2250 3300
 $Comp
 L power:GND #PWR02
@@
 	5400 4000 6050 4000
 Wire Wire Line
-	6050 2100 6050 4000
-Wire Wire Line
 	5400 3800 5750 3800
 Wire Wire Line
@@
 Wire Wire Line
 	5400 3400 5950 3400
-Wire Wire Line
-	5950 2200 5950 3400
 Wire Wire Line
 	5400 3300 5850 3300
@@
 Wire Wire Line
 	5750 1250 5750 3200
-Wire Wire Line
-	2350 3650 2350 3300
 Wire Wire Line
 	5300 7300 5750 7300
@@
 Wire Wire Line
 	2950 2050 3650 2050
-Wire Wire Line
-	6900 3800 6650 3800
-Wire Wire Line
-	6650 3800 6650 4250
-Wire Wire Line
-	6650 4250 3000 4250
-Wire Wire Line
-	3000 4250 3000 2350
 $Sheet
 S 3650 650  1750 2250
@@
 F26 "LCD_BACKLIGHT" O L 3650 2050 50
 F27 "MCO" O L 3650 1550 50
-F28 "SPI_CS_A" I R 5400 1850 50
-F29 "LCD_CS" O L 3650 2350 50
-F30 "FPGA_CS" O R 5400 2550 50
-F31 "SPI_CS_B" I R 5400 1950 50
-F32 "SPK" O R 5400 2200 50
+F28 "SPK" O R 5400 2200 50
+F29 "SPI_CS" I R 5400 1850 50
 $EndSheet
 Wire Wire Line
-	6900 1850 5400 1850
-Wire Wire Line
-	5400 1950 6900 1950
-Wire Wire Line
 	3650 2450 1500 2450
 Wire Wire Line
 	1500 2450 1500 3400
 Wire Wire Line
-	3650 2350 3000 2350
-Wire Wire Line
 	6950 4750 6200 4750
-Wire Wire Line
-	6200 4750 6200 2550
-Wire Wire Line
-	6200 2550 5400 2550
 Wire Wire Line
 	8600 850  9200 850
@@
 F11 "SPI_MOSI" O L 6900 1550 50
 F12 "SPI_MISO" I L 6900 1650 50
-F13 "IRQ_TOUCH" I L 6900 2100 50
-F14 "IRQ_ACCEL" I L 6900 2200 50
+F13 "IRQ_TOUCH" I L 6900 2250 50
+F14 "IRQ_ACCEL" I L 6900 2350 50
 F15 "SD_D0" B R 8600 1450 50
 F16 "SD_D1" B R 8600 1550 50
@@
 F22 "AUDIO_L" O R 8600 2500 50
 F23 "AUDIO_R" O R 8600 2600 50
-F24 "SPI_CS_A" O L 6900 1850 50
-F25 "SPI_CS_B" O L 6900 1950 50
-F26 "IR_TX" O R 8600 2100 50
+F24 "SPI_CS_LCD" O L 6900 2050 50
+F25 "SPI_CS_FPGA" O L 6900 1950 50
+F26 "SPI_CS_STM32" O L 6900 1850 50
 $EndSheet
 Wire Wire Line
-	9850 2100 8600 2100
-$Comp
-L Device:R R4
-U 1 1 60C79CD0
-P 10000 2100
-F 0 "R4" V 9793 2100 50  0000 C CNN
-F 1 "100" V 9884 2100 50  0000 C CNN
-F 2 "Resistor_SMD:R_0603_1608Metric" V 9930 2100 50  0001 C CNN
-F 3 "~" H 10000 2100 50  0001 C CNN
-F 4 "0.0005" H 10000 2100 50  0001 C CNN "Price"
-F 5 "C25201" H 10000 2100 50  0001 C CNN "LCSC"
-F 6 "-" H 10000 2100 50  0001 C CNN "Mouser"
-F 7 "N" H 10000 2100 50  0001 C CNN "Sponsored"
-	1    10000 2100
-	0    1    1    0
-$EndComp
-$Comp
-L Device:LED D2
-U 1 1 60C79CD1
-P 10300 2100
-F 0 "D2" H 10293 1845 50  0000 C CNN
-F 1 "LED" H 10293 1936 50  0000 C CNN
-F 2 "LED_SMD:LED_0805_2012Metric_Castellated" H 10300 2100 50  0001 C CNN
-F 3 "~" H 10300 2100 50  0001 C CNN
-F 4 "N" H 10300 2100 50  0001 C CNN "Sponsored"
-F 5 "C396645" H 10300 2100 50  0001 C CNN "LCSC"
-F 6 "-" H 10300 2100 50  0001 C CNN "Mouser"
-F 7 "0.022" H 10300 2100 50  0001 C CNN "Price"
-	1    10300 2100
-	-1   0    0    1
-$EndComp
-$Comp
-L power:GND #PWR021
-U 1 1 60CE727A
-P 10450 2100
-F 0 "#PWR021" H 10450 1850 50  0001 C CNN
-F 1 "GND" H 10455 1927 50  0000 C CNN
-F 2 "" H 10450 2100 50  0001 C CNN
-F 3 "" H 10450 2100 50  0001 C CNN
-	1    10450 2100
-	1    0    0    -1
-$EndComp
-Wire Wire Line
 	5400 4100 5450 4100
 Wire Wire Line
@@
 Wire Wire Line
 	3550 750  3450 750
+Wire Wire Line
+	6900 2350 5950 2350
+Wire Wire Line
+	5950 2350 5950 3400
+Wire Wire Line
+	6900 2250 6050 2250
+Wire Wire Line
+	6050 2250 6050 4000
+Wire Wire Line
+	6900 1950 6200 1950
+Wire Wire Line
+	6200 1950 6200 4750
+Wire Wire Line
+	6900 2050 6600 2050
+Wire Wire Line
+	6600 2050 6600 3800
+Wire Wire Line
+	6600 3800 6900 3800
+Wire Wire Line
+	6900 1850 5400 1850
 $EndSCHEMATC

Commit message: Dump.
Connections:
- net STM32/SAO_IO2: now reaches J2.5 (Pin_5)
- net STM32/SAO_IO3: now reaches J2.6 (Pin_6)
Changed lines of the file:
@@
 Connection ~ 6500 1550
 Connection ~ 6300 1750
-$Sheet
-S 3650 3100 1750 400
-U 6057522A
-F0 "ACCELEROMETER" 50
-F1 "accelerometer.sch" 50
-F2 "I2C_SDA" B R 5400 3200 50
-F3 "I2C_SCL" I R 5400 3300 50
-F4 "IRQ" O R 5400 3400 50
-F5 "AUX_SDA" T L 3650 3200 50
-F6 "AUX_SCL" O L 3650 3300 50
-$EndSheet
 Wire Wire Line
 	6500 1550 6900 1550
@@
 Wire Wire Line
 	9000 3300 9000 4650
-Wire Wire Line
-	1600 3200 1600 2800
-Wire Wire Line
-	1600 3200 1750 3200
-Wire Wire Line
-	1600 2800 2450 2800
 Connection ~ 1600 1700
 Connection ~ 1600 1800
@@
 	1    0    0    -1
 $EndComp
-Wire Wire Line
-	2450 2800 2450 3300
 Wire Wire Line
 	2850 4400 2850 2250
@@
 F15 "SPI_MISO" O R 5400 1650 50
 F16 "SPI_MOSI" I R 5400 1550 50
-F17 "LED_DATA" O L 3650 2450 50
+F17 "LED_DATA" O L 3650 2350 50
 F18 "PWR_LED_ENABLE" O L 3650 1150 50
 F19 "SENSE_VBAT" O L 3650 850 50
@@
 F28 "SPK" O R 5400 2200 50
 F29 "SPI_CS" I R 5400 1850 50
+F30 "SAO_IO2" B L 3650 2450 50
+F31 "SAO_IO3" B L 3650 2550 50
 $EndSheet
-Wire Wire Line
-	3650 2450 1500 2450
-Wire Wire Line
-	1500 2450 1500 3400
 Wire Wire Line
 	6950 4750 6200 4750
@@
 Wire Wire Line
 	6900 1850 5400 1850
+Wire Wire Line
+	3650 2350 1500 2350
+Wire Wire Line
+	1500 2350 1500 3400
+Wire Wire Line
+	3650 2450 1550 2450
+Wire Wire Line
+	1550 2450 1550 3300
+Wire Wire Line
+	1550 3300 1750 3300
+Wire Wire Line
+	2250 3300 2400 3300
+Wire Wire Line
+	2400 3300 2400 2550
+Wire Wire Line
+	2400 2550 3650 2550
+Wire Wire Line
+	2450 3300 2450 3400
+Wire Wire Line
+	2450 3400 1700 3400
+Wire Wire Line
+	1700 3400 1700 3200
+Wire Wire Line
+	1700 3200 1750 3200
+$Sheet
+S 3650 3100 1750 400
+U 6057522A
+F0 "ACCELEROMETER" 50
+F1 "accelerometer.sch" 50
+F2 "I2C_SDA" B R 5400 3200 50
+F3 "I2C_SCL" I R 5400 3300 50
+F4 "IRQ" O R 5400 3400 50
+F5 "AUX_SDA" T L 3650 3200 50
+F6 "AUX_SCL" O L 3650 3300 50
+$EndSheet
 $EndSCHEMATC
