File: mch2021.sch (KiCad schematic (older format))
At the start: 41 parts, among them J1 USB_C_Receptacle_USB2.0, J2 QWIIC_CONNECTORJS-1MM, J3 AudioJack3, J4 QWIIC_CONNECTORJS-1MM, J5 Micro SD card, J6 PMOD, U6 PCM5100, X1 Simple_Addon_v2

Commit message: Add chokes to usb lines
Parts:
- added L?: L_Core_Ferrite_Coupled_Small_GND, custom:MCE1012E900FBP, symbol L_Core_Ferrite_Coupled_Small_GND:L_Core_Ferrite_Coupled_Small_GND
- added L?: L_Core_Ferrite_Coupled_Small_1243, symbol Device:L_Core_Ferrite_Coupled_Small_1243
Connections:
- net labels added: VUSB_EXT
- wire segments 300 -> 309

Commit message: Add jumpers
Parts:
- added JP? (x4): Jumper_NO_Small, symbol Device:Jumper_NO_Small
Connections:
- wire segments 309 -> 331
Changed lines of the file:
@@
 F27 "SENSE_VUSB" I L 3650 950 50
 F28 "PWR_SDCARD_ENABLE" O L 3650 1150 50
-F29 "USB_DET" I L 3650 1600 50
+F29 "USB_DET" I L 3650 1550 50
 F30 "ESP32_WK" O R 5400 2250 50
 F31 "LED_DATA" O L 3650 1400 50
@@
 $EndComp
 Wire Wire Line
-	2200 3100 2500 3100
+	2200 3100 2450 3100
 Wire Wire Line
 	2200 3000 2200 3100
@@
 Wire Wire Line
 	1700 1150 1700 1300
-Wire Wire Line
-	2150 1150 1700 1150
-Wire Wire Line
-	2150 1600 2150 1150
 Wire Wire Line
 	2550 1400 3650 1400
@@
 P 2000 2500
 F 0 "D10" H 1750 2900 60  0000 R CNN
-F 1 "USBLC6-4SC6" H 2250 2050 60  0000 R CNN
+F 1 "USBLC6-4SC6" H 2300 1950 60  0000 R CNN
 F 2 "digikey-footprints:SOT23-6L" H 2200 2700 60  0001 L CNN
 F 3 "http://www.st.com/content/ccc/resource/technical/document/datasheet/9a/e6/1c/4f/b6/9a/44/e6/CD00047494.pdf/files/CD00047494.pdf/jcr:content/translations/en.CD00047494.pdf" H 2200 2800 60  0001 L CNN
@@
 $EndSheet
 Wire Wire Line
-	3650 1800 2750 1800
-Wire Wire Line
-	1800 1700 2550 1700
+	3650 1800 2800 1800
 $Comp
 L L_Core_Ferrite_Coupled_Small_GND:L_Core_Ferrite_Coupled_Small_GND L?
@@
 	1    0    0    -1
 $EndComp
-Wire Wire Line
-	2500 1600 2500 3100
-Connection ~ 2500 1600
-Wire Wire Line
-	2500 1600 2150 1600
-Wire Wire Line
-	2500 1600 3650 1600
 $Comp
 L power:GND #PWR?
@@
 $EndComp
 Wire Wire Line
-	2750 1700 3650 1700
-Wire Wire Line
-	2550 1800 2200 1800
+	2750 1700 2800 1700
+Wire Wire Line
+	2550 1800 2500 1800
 Wire Wire Line
 	2650 3000 2650 1950
@@
 U 1 1 5FE90F71
 P 1050 2850
-F 0 "L?" V 1050 2944 50  0000 L CNN
+F 0 "L?" V 1250 2600 50  0000 L CNN
 F 1 "L_Core_Ferrite_Coupled_Small_1243" V 1095 2944 50  0001 L CNN
 F 2 "" H 1050 2850 50  0001 C CNN
@@
 	1200 2550 1100 2550
 Wire Wire Line
-	1100 2550 1100 2750
-Wire Wire Line
-	1000 2600 1000 2750
-Wire Wire Line
-	1000 2950 1000 3050
+	1100 2550 1100 2700
+Wire Wire Line
+	1000 2600 1000 2700
+Wire Wire Line
+	1000 2950 1000 3000
+$Comp
+L Device:Jumper_NO_Small JP?
+U 1 1 5FF4CB69
+P 2650 1600
+F 0 "JP?" H 2400 1650 50  0000 C CNN
+F 1 "Jumper_NO_Small" H 2650 1506 50  0001 C CNN
+F 2 "" H 2650 1600 50  0001 C CNN
+F 3 "~" H 2650 1600 50  0001 C CNN
+	1    2650 1600
+	-1   0    0    1
+$EndComp
+Wire Wire Line
+	1700 1150 2450 1150
+$Comp
+L Device:Jumper_NO_Small JP?
+U 1 1 5FFB3A8B
+P 2650 1950
+F 0 "JP?" H 2400 1850 50  0000 C CNN
+F 1 "Jumper_NO_Small" H 2650 1856 50  0001 C CNN
+F 2 "" H 2650 1950 50  0001 C CNN
+F 3 "~" H 2650 1950 50  0001 C CNN
+	1    2650 1950
+	-1   0    0    1
+$EndComp
+Wire Wire Line
+	1800 1700 2500 1700
+Wire Wire Line
+	2450 3100 2450 1550
+Wire Wire Line
+	2500 1700 2500 1600
+Wire Wire Line
+	2500 1600 2550 1600
+Connection ~ 2500 1700
+Wire Wire Line
+	2500 1700 2550 1700
+Wire Wire Line
+	2500 1800 2500 1950
+Wire Wire Line
+	2500 1950 2550 1950
+Connection ~ 2500 1800
+Wire Wire Line
+	2500 1800 2200 1800
+Wire Wire Line
+	2750 1950 2800 1950
+Wire Wire Line
+	2800 1950 2800 1800
+Connection ~ 2800 1800
+Wire Wire Line
+	2800 1800 2750 1800
+Wire Wire Line
+	2800 1700 2800 1600
+Wire Wire Line
+	2800 1600 2750 1600
+Connection ~ 2800 1700
+Wire Wire Line
+	2800 1700 3650 1700
+Wire Wire Line
+	3650 1550 2450 1550
+Connection ~ 2450 1550
+Wire Wire Line
+	2450 1150 2450 1550
+$Comp
+L Device:Jumper_NO_Small JP?
+U 1 1 600F350C
+P 900 2850
+F 0 "JP?" H 900 2950 50  0000 C CNN
+F 1 "Jumper_NO_Small" H 900 2756 50  0001 C CNN
+F 2 "" H 900 2850 50  0001 C CNN
+F 3 "~" H 900 2850 50  0001 C CNN
+	1    900  2850
+	0    -1   -1   0
+$EndComp
+Wire Wire Line
+	900  2750 900  2700
+Wire Wire Line
+	900  2700 1000 2700
+Connection ~ 1000 2700
+Wire Wire Line
+	1000 2700 1000 2750
+Wire Wire Line
+	900  2950 900  3000
+Wire Wire Line
+	900  3000 1000 3000
+Connection ~ 1000 3000
+Wire Wire Line
+	1000 3000 1000 3050
+$Comp
+L Device:Jumper_NO_Small JP?
+U 1 1 60139684
+P 1150 2850
+F 0 "JP?" H 1150 2950 50  0000 C CNN
+F 1 "Jumper_NO_Small" H 1150 2756 50  0001 C CNN
+F 2 "" H 1150 2850 50  0001 C CNN
+F 3 "~" H 1150 2850 50  0001 C CNN
+	1    1150 2850
+	0    1    1    0
+$EndComp
+Wire Wire Line
+	1150 2750 1150 2700
+Wire Wire Line
+	1150 2700 1100 2700
+Connection ~ 1100 2700
+Wire Wire Line
+	1100 2700 1100 2750
 Wire Wire Line
 	1350 2750 1350 3000
 Wire Wire Line
-	1350 3000 1100 3000
-Wire Wire Line
-	1100 3000 1100 2950
+	1150 2950 1150 3000
+Wire Wire Line
+	1100 2950 1100 3000
+Wire Wire Line
+	1150 3000 1100 3000
+Wire Wire Line
+	1150 3000 1350 3000
+Connection ~ 1150 3000
 $EndSCHEMATC

Commit message: Updated schematic, add design file
Parts:
- removed JP? (x2): Jumper_NO_Small, symbol Device:Jumper_NO_Small
- removed L?: L_Core_Ferrite_Coupled_Small_1243, symbol Device:L_Core_Ferrite_Coupled_Small_1243
- removed R15, R17, R65: 220, Resistor_SMD:R_0603_1608Metric, symbol Device:R
- added F1: 1A, Fuse:Fuse_0805_2012Metric, symbol Device:Polyfuse_Small
- added L3: 22 Ohm, Resistor_SMD:R_0805_2012Metric, symbol Device:L_Core_Ferrite_Small
- added N1: Artwork, custom:draft2, symbol Mechanical:Housing
- added N2: Badge.team, custom:badgeteam, symbol Mechanical:Housing
- JP3, JP4: renamed from JP?; footprint (none) -> Jumpers:SMT-JUMPER_2_NO_NO-SILK_ROUND
- R16, R50, R66: value 220 -> 470
- X1: footprint (none) -> Simple_Addon_v2:Simple_Addon_v2-BADGE-2x3
- gave numbers to parts that had none: 1
Connections:
- net labels removed: VUSB_EXT
- wire segments 331 -> 316

Commit message: Update artwork
Parts:
- N1: footprint custom:draft2 -> custom:draft2_renze
Changed lines of the file:
@@
 F 0 "N1" H 6603 7584 50  0000 L CNN
 F 1 "Artwork" H 6603 7493 50  0000 L CNN
-F 2 "custom:draft2" H 6500 7600 50  0001 C CNN
+F 2 "custom:draft2_renze" H 6500 7600 50  0001 C CNN
 F 3 "~" H 6500 7600 50  0001 C CNN
 	1    6450 7550
@@
 	1    0    0    -1
 $EndComp
+$Comp
+L power:GND #PWR0242
+U 1 1 5FEF0000
+P 4100 7500
+F 0 "#PWR0242" H 4100 7250 50  0001 C CNN
+F 1 "GND" H 4105 7327 50  0000 C CNN
+F 2 "" H 4100 7500 50  0001 C CNN
+F 3 "" H 4100 7500 50  0001 C CNN
+	1    4100 7500
+	-1   0    0    -1
+$EndComp
+Text GLabel 4100 7500 1    50   Input ~ 0
+GND
 $EndSCHEMATC

Commit message: First steps of routing prototype 2, switch to 0402 for most passives
Parts:
- C16, C18, C19, C20: LCSC (none) -> C107372
- C17, C30: LCSC (none) -> C83056
- N1: footprint custom:draft2_renze -> custom:vector4
- R1, R2: footprint Resistor_SMD:R_0603_1608Metric -> Resistor_SMD:R_0402_1005Metric; LCSC C269696 -> C103086
- R16, R3, R30, R38, R39, R50, R53, R66, R7: footprint Resistor_SMD:R_0603_1608Metric -> Resistor_SMD:R_0402_1005Metric; LCSC C115324 -> (none)
Changed lines of the file:
@@
 F 0 "R53" V 9250 900 50  0000 C CNN
 F 1 "10k" V 9200 1050 50  0000 C CNN
-F 2 "Resistor_SMD:R_0603_1608Metric" V 9130 1050 50  0001 C CNN
+F 2 "Resistor_SMD:R_0402_1005Metric" V 9130 1050 50  0001 C CNN
 F 3 "~" H 9200 1050 50  0001 C CNN
 F 4 "" H 9200 1050 50  0001 C CNN "Price"
-F 5 "C115324" H 9200 1050 50  0001 C CNN "LCSC"
+F 5 "" H 9200 1050 50  0001 C CNN "LCSC"
 F 6 "-" H 9200 1050 50  0001 C CNN "Mouser"
 F 7 "N" H 9200 1050 50  0001 C CNN "Sponsored"
@@
 F 0 "R39" V 9150 900 50  0000 C CNN
 F 1 "10k" V 9100 1050 50  0000 C CNN
-F 2 "Resistor_SMD:R_0603_1608Metric" V 9030 1050 50  0001 C CNN
+F 2 "Resistor_SMD:R_0402_1005Metric" V 9030 1050 50  0001 C CNN
 F 3 "~" H 9100 1050 50  0001 C CNN
 F 4 "" H 9100 1050 50  0001 C CNN "Price"
-F 5 "C115324" H 9100 1050 50  0001 C CNN "LCSC"
+F 5 "" H 9100 1050 50  0001 C CNN "LCSC"
 F 6 "-" H 9100 1050 50  0001 C CNN "Mouser"
 F 7 "N" H 9100 1050 50  0001 C CNN "Sponsored"
@@
 F 0 "R38" V 9050 900 50  0000 C CNN
 F 1 "10k" V 9000 1050 50  0000 C CNN
-F 2 "Resistor_SMD:R_0603_1608Metric" V 8930 1050 50  0001 C CNN
+F 2 "Resistor_SMD:R_0402_1005Metric" V 8930 1050 50  0001 C CNN
 F 3 "~" H 9000 1050 50  0001 C CNN
 F 4 "" H 9000 1050 50  0001 C CNN "Price"
-F 5 "C115324" H 9000 1050 50  0001 C CNN "LCSC"
+F 5 "" H 9000 1050 50  0001 C CNN "LCSC"
 F 6 "-" H 9000 1050 50  0001 C CNN "Mouser"
 F 7 "N" H 9000 1050 50  0001 C CNN "Sponsored"
@@
 F 0 "R7" V 8850 900 50  0000 C CNN
 F 1 "10k" V 8800 1050 50  0000 C CNN
-F 2 "Resistor_SMD:R_0603_1608Metric" V 8730 1050 50  0001 C CNN
+F 2 "Resistor_SMD:R_0402_1005Metric" V 8730 1050 50  0001 C CNN
 F 3 "~" H 8800 1050 50  0001 C CNN
 F 4 "" H 8800 1050 50  0001 C CNN "Price"
-F 5 "C115324" H 8800 1050 50  0001 C CNN "LCSC"
+F 5 "" H 8800 1050 50  0001 C CNN "LCSC"
 F 6 "-" H 8800 1050 50  0001 C CNN "Mouser"
 F 7 "N" H 8800 1050 50  0001 C CNN "Sponsored"
@@
 F 0 "R30" V 8950 900 50  0000 C CNN
 F 1 "10k" V 8900 1050 50  0000 C CNN
-F 2 "Resistor_SMD:R_0603_1608Metric" V 8830 1050 50  0001 C CNN
+F 2 "Resistor_SMD:R_0402_1005Metric" V 8830 1050 50  0001 C CNN
 F 3 "~" H 8900 1050 50  0001 C CNN
 F 4 "" H 8900 1050 50  0001 C CNN "Price"
-F 5 "C115324" H 8900 1050 50  0001 C CNN "LCSC"
+F 5 "" H 8900 1050 50  0001 C CNN "LCSC"
 F 6 "-" H 8900 1050 50  0001 C CNN "Mouser"
 F 7 "N" H 8900 1050 50  0001 C CNN "Sponsored"
@@
 F 0 "R3" V 8750 900 50  0000 C CNN
 F 1 "10k" V 8700 1050 50  0000 C CNN
-F 2 "Resistor_SMD:R_0603_1608Metric" V 8630 1050 50  0001 C CNN
+F 2 "Resistor_SMD:R_0402_1005Metric" V 8630 1050 50  0001 C CNN
 F 3 "~" H 8700 1050 50  0001 C CNN
 F 4 "" H 8700 1050 50  0001 C CNN "Price"
-F 5 "C115324" H 8700 1050 50  0001 C CNN "LCSC"
+F 5 "" H 8700 1050 50  0001 C CNN "LCSC"
 F 6 "-" H 8700 1050 50  0001 C CNN "Mouser"
 F 7 "N" H 8700 1050 50  0001 C CNN "Sponsored"
@@
 F 1 "1u" H 1765 6705 50  0000 L CNN
 F 2 "Capacitor_SMD:C_0402_1005Metric" H 1688 6600 50  0001 C CNN
-F 3 "~" H 1650 6750 50  0001 C CNN
+F 3 "" H 1650 6750 50  0001 C CNN
+F 4 "C107372" H 1650 6750 50  0001 C CNN "LCSC"
 	1    1650 6750
 	-1   0    0    -1
@@
 F 1 "1u" H 1765 7305 50  0000 L CNN
 F 2 "Capacitor_SMD:C_0402_1005Metric" H 1688 7200 50  0001 C CNN
-F 3 "~" H 1650 7350 50  0001 C CNN
+F 3 "" H 1650 7350 50  0001 C CNN
+F 4 "C107372" H 1650 7350 50  0001 C CNN "LCSC"
 	1    1650 7350
 	-1   0    0    -1
@@
 F 1 "100n" H 1415 7305 50  0000 L CNN
 F 2 "Capacitor_SMD:C_0402_1005Metric" H 1338 7200 50  0001 C CNN
-F 3 "~" H 1300 7350 50  0001 C CNN
+F 3 "" H 1300 7350 50  0001 C CNN
+F 4 "C83056 " H 1300 7350 50  0001 C CNN "LCSC"
 	1    1300 7350
 	-1   0    0    -1
@@
 F 1 "1u" H 1015 7305 50  0000 L CNN
 F 2 "Capacitor_SMD:C_0402_1005Metric" H 938 7200 50  0001 C CNN
-F 3 "~" H 900 7350 50  0001 C CNN
+F 3 "" H 900 7350 50  0001 C CNN
+F 4 "C107372" H 900 7350 50  0001 C CNN "LCSC"
 	1    900  7350
 	-1   0    0    -1
@@
 F 1 "1u" H 3165 7305 50  0000 L CNN
 F 2 "Capacitor_SMD:C_0402_1005Metric" H 3088 7200 50  0001 C CNN
-F 3 "~" H 3050 7350 50  0001 C CNN
+F 3 "" H 3050 7350 50  0001 C CNN
+F 4 "C107372" H 3050 7350 50  0001 C CNN "LCSC"
 	1    3050 7350
 	-1   0    0    -1
@@
 F 1 "100n" H 3615 7305 50  0000 L CNN
 F 2 "Capacitor_SMD:C_0402_1005Metric" H 3538 7200 50  0001 C CNN
-F 3 "~" H 3500 7350 50  0001 C CNN
+F 3 "" H 3500 7350 50  0001 C CNN
+F 4 "C83056 " H 3500 7350 50  0001 C CNN "LCSC"
 	1    3500 7350
 	-1   0    0    -1
@@
 F 0 "R16" V 3200 6050 50  0000 C CNN
 F 1 "470" V 3150 6200 50  0000 C CNN
-F 2 "Resistor_SMD:R_0603_1608Metric" V 3080 6200 50  0001 C CNN
+F 2 "Resistor_SMD:R_0402_1005Metric" V 3080 6200 50  0001 C CNN
 F 3 "~" H 3150 6200 50  0001 C CNN
 F 4 "" H 3150 6200 50  0001 C CNN "Price"
-F 5 "C115324" H 3150 6200 50  0001 C CNN "LCSC"
+F 5 "" H 3150 6200 50  0001 C CNN "LCSC"
 F 6 "-" H 3150 6200 50  0001 C CNN "Mouser"
 F 7 "N" H 3150 6200 50  0001 C CNN "Sponsored"
@@
 F 0 "R50" V 3200 6250 50  0000 C CNN
 F 1 "470" V 3150 6400 50  0000 C CNN
-F 2 "Resistor_SMD:R_0603_1608Metric" V 3080 6400 50  0001 C CNN
+F 2 "Resistor_SMD:R_0402_1005Metric" V 3080 6400 50  0001 C CNN
 F 3 "~" H 3150 6400 50  0001 C CNN
 F 4 "" H 3150 6400 50  0001 C CNN "Price"
-F 5 "C115324" H 3150 6400 50  0001 C CNN "LCSC"
+F 5 "" H 3150 6400 50  0001 C CNN "LCSC"
 F 6 "-" H 3150 6400 50  0001 C CNN "Mouser"
 F 7 "N" H 3150 6400 50  0001 C CNN "Sponsored"
@@
 F 0 "R66" V 3200 6450 50  0000 C CNN
 F 1 "470" V 3150 6600 50  0000 C CNN
-F 2 "Resistor_SMD:R_0603_1608Metric" V 3080 6600 50  0001 C CNN
+F 2 "Resistor_SMD:R_0402_1005Metric" V 3080 6600 50  0001 C CNN
 F 3 "~" H 3150 6600 50  0001 C CNN
 F 4 "" H 3150 6600 50  0001 C CNN "Price"
-F 5 "C115324" H 3150 6600 50  0001 C CNN "LCSC"
+F 5 "" H 3150 6600 50  0001 C CNN "LCSC"
 F 6 "-" H 3150 6600 50  0001 C CNN "Mouser"
 F 7 "N" H 3150 6600 50  0001 C CNN "Sponsored"
@@
 F 0 "R2" V 1750 1550 50  0000 C CNN
 F 1 "5k1" V 1800 1400 50  0000 C CNN
-F 2 "Resistor_SMD:R_0603_1608Metric" H 1800 1400 50  0001 C CNN
+F 2 "Resistor_SMD:R_0402_1005Metric" H 1800 1400 50  0001 C CNN
 F 3 "~" H 1800 1400 50  0001 C CNN
 F 4 "" H 1800 1400 50  0001 C CNN "Price"
-F 5 "C269696" H 1800 1400 50  0001 C CNN "LCSC"
+F 5 "C103086" H 1800 1400 50  0001 C CNN "LCSC"
 F 6 "-" H 1800 1400 50  0001 C CNN "Mouser"
 F 7 "N" H 1800 1400 50  0001 C CNN "Sponsored"
@@
 F 0 "R1" V 1750 1450 50  0000 C CNN
 F 1 "5k1" V 1800 1300 50  0000 C CNN
-F 2 "Resistor_SMD:R_0603_1608Metric" H 1800 1300 50  0001 C CNN
+F 2 "Resistor_SMD:R_0402_1005Metric" H 1800 1300 50  0001 C CNN
 F 3 "~" H 1800 1300 50  0001 C CNN
 F 4 "" H 1800 1300 50  0001 C CNN "Price"
-F 5 "C269696" H 1800 1300 50  0001 C CNN "LCSC"
+F 5 "C103086" H 1800 1300 50  0001 C CNN "LCSC"
 F 6 "-" H 1800 1300 50  0001 C CNN "Mouser"
 F 7 "N" H 1800 1300 50  0001 C CNN "Sponsored"
@@
 F 0 "N1" H 6603 7584 50  0000 L CNN
 F 1 "Artwork" H 6603 7493 50  0000 L CNN
-F 2 "custom:draft2_renze" H 6500 7600 50  0001 C CNN
+F 2 "custom:vector4" H 6500 7600 50  0001 C CNN
 F 3 "~" H 6500 7600 50  0001 C CNN
 	1    6450 7550

Commit message: Some more work
Parts:
- removed JP3, JP4: Jumper_NO_Small, Jumpers:SMT-JUMPER_2_NO_NO-SILK_ROUND, symbol Device:Jumper_NO_Small
- removed N1: Artwork, custom:vector4, symbol Mechanical:Housing
- added C51, C52: 2.2n, Capacitor_SMD:C_0402_1005Metric, symbol Device:C
- added C53: 1u, Capacitor_SMD:C_0402_1005Metric, symbol Device:C
- added C54: 100n, Capacitor_SMD:C_0402_1005Metric, symbol Device:C
- added N2: Artwork, custom:vector4, symbol Mechanical:Housing
- added R69, R70: DNP, Resistor_SMD:R_0402_1005Metric, symbol Device:R
- added R71, R72: 0, Resistor_SMD:R_0402_1005Metric, symbol Device:R
- added R73, R74: 470, Resistor_SMD:R_0402_1005Metric, symbol Device:R
- C3: renamed from C18; value 1u -> 2.2u; LCSC C107372 -> (none)
- C4: renamed from C19; value 1u -> 2.2u; LCSC C107372 -> (none)
- X1: footprint Simple_Addon_v2:Simple_Addon_v2-BADGE-2x3 -> Simple_Addon_v2:Simple_Addon_v2-BADGE-2x3-nosilk
- renumbered C16 to C1, C17 to C2, C20 to C5, C30 to C6, D10 to D1, D1 to D2, J3 to J1, J1 to J2, J2 to J3, J6 to J4, J4 to J6, L3 to L1, L4 to L2, N2 to N1, R39 to R10, R53 to R11, R16 to R3, R50 to R4, R66 to R5, R3 to R6, R30 to R8, R38 to R9, U6 to U1
Connections:
- net +3V3: now also C53.1, C54.1
- net 6: now also C51.2, C52.2, C53.2, C54.2, R69.1, R70.1
- net USB_VBUS: now reaches J2.A4 (VBUS), J2.A9 (VBUS), J2.B4 (VBUS), J2.B9 (VBUS), L1.2
- net USB_D+: now reaches J2.A6 (D+), J2.B6 (D+), L2.3
- net USB_D+: now also D1.6; no longer D1.4
- net USB_D-: now reaches J2.A7 (D-), J2.B7 (D-), L2.1
- net USB_D-: now also D1.4; no longer D1.6
- net PCM5100_LDOO: now reaches C1.1, C2.1, U1.18 (LDOO)
- net PCM5100_CAPP: now reaches C3.1, U1.2 (CAPP)
- net PCM5100_CAPN: now reaches C3.2, U1.4 (CAPM)
- net PCM5100_VNEG: now reaches C4.1, U1.5 (VNEG)
- net at J1.T: now also R69.2, R71.2; no longer U1.6 (OUTL)
- net at J1.R: now also R70.2, R72.2; no longer U1.7 (OUTR)
- new net: C52.1, R71.1, R73.2
- new net: C51.1, R72.1, R74.2
- new net PCM5100_OUTL: R73.1, U1.6 (OUTL)
- new net PCM5100_OUTR: R74.1, U1.7 (OUTR)
Other:
- moved on the sheet: C1, C2, C3, C4, C5, C6, J1, N1, R3, R4, R5, U1

Commit message: Layout+initial full routing
Parts:
- D2: symbol led:RGB-5050 -> mch2021-rescue:RGB-5050-led
- J2: symbol Connector:USB_C_Receptacle_USB2.0 -> mch2021-rescue:USB_C_Receptacle_USB2.0-Connector
- J3, J6: symbol SparkFun-Connectors:QWIIC_CONNECTORJS-1MM -> mch2021-rescue:QWIIC_CONNECTORJS-1MM-SparkFun-Connectors
- N2: footprint custom:vector4 -> custom:vector5
Connections:
- net USB_VBUS: now also D1.5
- net VUSB: no longer D1.5
Changed lines of the file:
@@
 	2850 4400 6800 4400
 $Comp
-L led:RGB-5050 D2
+L mch2021-rescue:RGB-5050-led D2
 U 1 1 611CFAC6
 P 6500 5250
@@
 	5550 6150 5550 6250
 $Comp
-L SparkFun-Connectors:QWIIC_CONNECTORJS-1MM J3
+L mch2021-rescue:QWIIC_CONNECTORJS-1MM-SparkFun-Connectors J3
 U 1 1 5FC35963
 P 5550 6350
@@
 	10350 2550 10450 2550
 $Comp
-L SparkFun-Connectors:QWIIC_CONNECTORJS-1MM J6
+L mch2021-rescue:QWIIC_CONNECTORJS-1MM-SparkFun-Connectors J6
 U 1 1 604137E0
 P 10550 2550
@@
 F 3 "" H 2000 3000 50  0001 C CNN
 	1    2000 3000
-	1    0    0    -1
-$EndComp
-$Comp
-L vusb:VUSB #PWR08
-U 1 1 5F50A06B
-P 2000 2000
-F 0 "#PWR08" H 2010 2000 20  0001 C CNN
-F 1 "VUSB" H 2000 2096 40  0000 C CNN
-F 2 "" H 2000 2000 60  0001 C CNN
-F 3 "" H 2000 2000 60  0001 C CNN
-	1    2000 2000
 	1    0    0    -1
 $EndComp
@@
 	1600 1800 1600 1900
 $Comp
-L vusb:VUSB #PWR012
+L mch2021-rescue:VUSB-vusb #PWR012
 U 1 1 5FCD69E4
 P 2350 1050
@@
 Connection ~ 1600 1800
 $Comp
-L Connector:USB_C_Receptacle_USB2.0 J2
+L mch2021-rescue:USB_C_Receptacle_USB2.0-Connector J2
 U 1 1 5E94CF38
 P 1000 1700
@@
 F 0 "N2" H 6403 7584 50  0000 L CNN
 F 1 "Artwork" H 6403 7493 50  0000 L CNN
-F 2 "custom:vector4" H 6300 7600 50  0001 C CNN
+F 2 "custom:vector5" H 6300 7600 50  0001 C CNN
 F 3 "~" H 6300 7600 50  0001 C CNN
 	1    6250 7550
 	1    0    0    -1
 $EndComp
+Text Label 1750 1050 2    50   ~ 0
+USB_VBUS
+Wire Wire Line
+	1750 1050 1750 1100
+Connection ~ 1750 1100
+Text Label 2000 1900 0    50   ~ 0
+USB_VBUS
+Wire Wire Line
+	2000 1900 2000 2000
 $EndSCHEMATC

Commit message: Moar fixes
Parts:
- added TP12, TP13: LED OUT, TestPoint:TestPoint_Pad_1.0x1.0mm, symbol Connector:TestPoint_Small
- N2: footprint custom:vector5 -> custom:vector6
Connections:
- net 6: now also TP12.1
- new net PWR_LED: TP13.1
Changed lines of the file:
@@
 F 0 "N2" H 6403 7584 50  0000 L CNN
 F 1 "Artwork" H 6403 7493 50  0000 L CNN
-F 2 "custom:vector5" H 6300 7600 50  0001 C CNN
+F 2 "custom:vector6" H 6300 7600 50  0001 C CNN
 F 3 "~" H 6300 7600 50  0001 C CNN
 	1    6250 7550
@@
 Wire Wire Line
 	2000 1900 2000 2000
+$Comp
+L Connector:TestPoint_Small TP12
+U 1 1 600A5D31
+P 750 600
+F 0 "TP12" H 550 600 50  0000 L CNN
+F 1 "LED OUT" H 798 555 50  0001 L CNN
+F 2 "TestPoint:TestPoint_Pad_1.0x1.0mm" H 950 600 50  0001 C CNN
+F 3 "~" H 950 600 50  0001 C CNN
+	1    750  600
+	1    0    0    -1
+$EndComp
+$Comp
+L Connector:TestPoint_Small TP13
+U 1 1 600A6E9D
+P 1050 600
+F 0 "TP13" H 850 600 50  0000 L CNN
+F 1 "LED OUT" H 1098 555 50  0001 L CNN
+F 2 "TestPoint:TestPoint_Pad_1.0x1.0mm" H 1250 600 50  0001 C CNN
+F 3 "~" H 1250 600 50  0001 C CNN
+	1    1050 600
+	1    0    0    -1
+$EndComp
+Text GLabel 1100 550  2    31   Input ~ 0
+PWR_LED
+Wire Wire Line
+	1100 550  1050 550
+Wire Wire Line
+	1050 550  1050 600
+Wire Wire Line
+	750  600  750  650
+$Comp
+L power:GND #PWR0220
+U 1 1 600F1D69
+P 750 650
+F 0 "#PWR0220" H 750 400 50  0001 C CNN
+F 1 "GND" H 755 477 50  0000 C CNN
+F 2 "" H 750 650 50  0001 C CNN
+F 3 "" H 750 650 50  0001 C CNN
+	1    750  650
+	1    0    0    -1
+$EndComp
 $EndSCHEMATC
