File: mch2021.sch (KiCad schematic (older format))
At the start: 62 parts, among them J1 AudioJack3, J10 CONN-3, J11 CONN-7, J2 USB_C_Receptacle_USB2.0, J3 QWIIC_CONNECTORJS-1MM, J4 PMOD, J5 Micro SD card, J6 QWIIC_CONNECTORJS-1MM, J9 CONN-7, U1 PCM5100, X1 Simple_Addon_v2

Commit message: Small tweaks
Parts:
- N3: value Prototyping area 1 -> May Contain Hardware
- N4: value Prototyping area 2 -> More Cool Hardware
Changed lines of the file:
@@
 P 3200 5500
 F 0 "N3" H 3353 5534 50  0000 L CNN
-F 1 "Prototyping area 1" H 3353 5443 50  0000 L CNN
+F 1 "May Contain Hardware" H 3353 5443 50  0000 L CNN
 F 2 "custom:protoboard-squares" H 3250 5550 50  0001 C CNN
 F 3 "~" H 3250 5550 50  0001 C CNN
@@
 P 4400 5500
 F 0 "N4" H 4553 5534 50  0000 L CNN
-F 1 "Prototyping area 2" H 4553 5443 50  0000 L CNN
+F 1 "More Cool Hardware" H 4553 5443 50  0000 L CNN
 F 2 "custom:protoboard-squares-big" H 4450 5550 50  0001 C CNN
 F 3 "~" H 4450 5550 50  0001 C CNN

Commit message: Small last minute fixes
Parts:
- added N?: Logo, custom:badgeteam, symbol Mechanical:Housing
- C3, C4: LCSC (none) -> C12530
- C51, C52: LCSC (none) -> C915853
- J3, J6: footprint Connectors:1X04_1MM_RA -> custom:1X04_1MM_RA_GND; symbol mch2021-rescue:QWIIC_CONNECTORJS-1MM-SparkFun-Connectors -> mch2021-rescue:QWIIC_MCH
Changed lines of the file:
@@
 Sheet 1 9
 Title "MCH2021 badge - Overview"
-Date "2020-12-22"
+Date "2021-01-14"
 Rev "2"
 Comp "BADGE.TEAM"
@@
 	5550 6150 5550 6250
 $Comp
-L mch2021-rescue:QWIIC_CONNECTORJS-1MM-SparkFun-Connectors J3
+L mch2021-rescue:QWIIC_MCH J3
 U 1 1 5FC35963
 P 5550 6350
 F 0 "J3" H 5400 6750 45  0000 C CNN
 F 1 "QWIIC_CONNECTORJS-1MM" V 5150 6500 45  0000 C CNN
-F 2 "Connectors:1X04_1MM_RA" H 5550 6850 20  0001 C CNN
+F 2 "custom:1X04_1MM_RA_GND" H 5550 6850 20  0001 C CNN
 F 3 "" H 5550 6350 50  0001 C CNN
 F 4 "CONN-13694" V 5250 6500 60  0000 C CNN "Field4"
@@
 F 2 "Capacitor_SMD:C_0402_1005Metric" H 3138 6600 50  0001 C CNN
 F 3 "" H 3100 6750 50  0001 C CNN
-F 4 "" H 3100 6750 50  0001 C CNN "LCSC"
+F 4 "C12530" H 3100 6750 50  0001 C CNN "LCSC"
 	1    3100 6750
 	-1   0    0    -1
@@
 F 2 "Capacitor_SMD:C_0402_1005Metric" H 3138 7200 50  0001 C CNN
 F 3 "" H 3100 7350 50  0001 C CNN
-F 4 "" H 3100 7350 50  0001 C CNN "LCSC"
+F 4 "C12530" H 3100 7350 50  0001 C CNN "LCSC"
 	1    3100 7350
 	-1   0    0    -1
@@
 	10350 2550 10450 2550
 $Comp
-L mch2021-rescue:QWIIC_CONNECTORJS-1MM-SparkFun-Connectors J6
+L mch2021-rescue:QWIIC_MCH J6
 U 1 1 604137E0
 P 10550 2550
 F 0 "J6" H 10400 2950 45  0000 C CNN
 F 1 "QWIIC_CONNECTORJS-1MM" V 10150 2700 45  0000 C CNN
-F 2 "Connectors:1X04_1MM_RA" H 10550 3050 20  0001 C CNN
+F 2 "custom:1X04_1MM_RA_GND" H 10550 3050 20  0001 C CNN
 F 3 "" H 10550 2550 50  0001 C CNN
 F 4 "CONN-13694" V 10250 2700 60  0000 C CNN "Field4"
@@
 F 2 "Capacitor_SMD:C_0402_1005Metric" H 2238 7200 50  0001 C CNN
 F 3 "" H 2200 7350 50  0001 C CNN
-F 4 "" H 2200 7350 50  0001 C CNN "LCSC"
+F 4 "C915853" H 2200 7350 50  0001 C CNN "LCSC"
 	1    2200 7350
 	-1   0    0    -1
@@
 F 2 "Capacitor_SMD:C_0402_1005Metric" H 1938 7200 50  0001 C CNN
 F 3 "" H 1900 7350 50  0001 C CNN
-F 4 "" H 1900 7350 50  0001 C CNN "LCSC"
+F 4 "C915853" H 1900 7350 50  0001 C CNN "LCSC"
 	1    1900 7350
 	-1   0    0    -1
@@
 Wire Wire Line
 	1600 4500 5750 4500
+$Comp
+L Mechanical:Housing N?
+U 1 1 600E8BB4
+P 2200 5900
+F 0 "N?" H 2353 5934 50  0000 L CNN
+F 1 "Logo" H 2353 5843 50  0000 L CNN
+F 2 "custom:badgeteam" H 2250 5950 50  0001 C CNN
+F 3 "~" H 2250 5950 50  0001 C CNN
+	1    2200 5900
+	1    0    0    -1
+$EndComp
 $EndSCHEMATC

Commit message: Update LCSC code for the 32kHz crystals
Parts:
- gave numbers to parts that had none: 1
Changed lines of the file:
@@
 	1600 4500 5750 4500
 $Comp
-L Mechanical:Housing N?
+L Mechanical:Housing N5
 U 1 1 600E8BB4
 P 2200 5900
-F 0 "N?" H 2353 5934 50  0000 L CNN
+F 0 "N5" H 2353 5934 50  0000 L CNN
 F 1 "Logo" H 2353 5843 50  0000 L CNN
 F 2 "custom:badgeteam" H 2250 5950 50  0001 C CNN

Commit message: Fix most of the bugs found on prototype 2 board
Parts:
- removed J5: Micro SD card, custom:MicroSD-SOFNG-TF-002-H18, symbol Connector:Micro_SD_Card
- removed L1: 22 Ohm, Resistor_SMD:R_0805_2012Metric, symbol Device:L_Core_Ferrite_Small
- removed L2: L_Core_Ferrite_Coupled_Small_GND, custom:MCE1012E900FBP, symbol L_Core_Ferrite_Coupled_Small_GND:L_Core_Ferrite_Coupled_Small_GND
- removed R10, R11, R6, R7, R8, R9: 10k, Resistor_SMD:R_0402_1005Metric, symbol Device:R
- removed TP2, TP3: LED IN, TestPoint:TestPoint_Pad_1.0x1.0mm, symbol Connector:TestPoint_Small
Connections:
- net labels removed: PWR_SDCARD
- wire segments 376 -> 337

Commit message: Change pinout of expansion header close to board edge to be fully ground instead of gnd + 3.3v (& update component references)
Parts:
- C1, C2, C3, C4, C5, C51, C52, C53, C54, C57, C6: symbol Device:C -> mch2021-rescue:C-Device
- D1: symbol dk_TVS-Diodes:USBLC6-4SC6 -> mch2021-rescue:USBLC6-4SC6-dk_TVS-Diodes
- F1: symbol Device:Polyfuse_Small -> mch2021-rescue:Polyfuse_Small-Device
- J1: symbol Connector:AudioJack3 -> mch2021-rescue:AudioJack3-Connector
- J10: symbol conn-3:CONN-3 -> mch2021-rescue:CONN-3-conn-3
- J11, J9: symbol conn-7:CONN-7 -> mch2021-rescue:CONN-7-conn-7
- J4: symbol Connector_Generic:Conn_02x06_Odd_Even -> mch2021-rescue:Conn_02x06_Odd_Even-Connector_Generic
- N1, N2, N3, N4, N5: symbol Mechanical:Housing -> mch2021-rescue:Housing-Mechanical
- R1, R2: symbol Device:R_Small -> mch2021-rescue:R_Small-Device
- R3, R4, R5, R69, R70, R71, R72, R73, R74, R75: symbol Device:R -> mch2021-rescue:R-Device
- TP1, TP10, TP11, TP12, TP13, TP4, TP5, TP6, TP7, TP8, TP9: symbol Connector:TestPoint_Small -> mch2021-rescue:TestPoint_Small-Connector
- U1: symbol Audio:PCM5100 -> mch2021-rescue:PCM5100-Audio

Commit message: Fix symbol of 5050 led and rotate footprint to match actual LED pinout
Parts:
- D2: symbol mch2021-rescue:RGB-5050-led -> custom:RGB-5050-MCH
Connections:
- net +3V3: now also D2.1 (G), D2.2 (R), D2.3 (B); no longer D2.4 (G), D2.5 (R), D2.6 (B)
- net FPGA/RGB0: now also D2.4; no longer D2.1
- net FPGA/RGB1: now also D2.5; no longer D2.3
- net FPGA/RGB2: now also D2.6; no longer D2.2
Changed lines of the file:
@@
 Sheet 1 9
 Title "MCH2021 badge - Overview"
-Date "2021-10-09"
+Date "2021-11-13"
 Rev "3"
 Comp "BADGE.TEAM"
@@
 	2850 4400 6800 4400
 $Comp
-L mch2021-rescue:RGB-5050-led D2
+L custom:RGB-5050-MCH D2
 U 1 1 611CFAC6
 P 6500 5250

Commit message: Add hooks
Parts:
- added J12: Hook 1, TestPoint:TestPoint_Keystone_5019_Minature, symbol Connector_Generic:Conn_01x01
- added J13: Hook 2, TestPoint:TestPoint_Keystone_5019_Minature, symbol Connector_Generic:Conn_01x01
Connections:
- net GND: now also J12.1 (Pin_1), J13.1 (Pin_1)
Changed lines of the file:
@@
 Sheet 1 9
 Title "MCH2021 badge - Overview"
-Date "2021-11-13"
+Date "2021-11-14"
 Rev "3"
 Comp "BADGE.TEAM"
@@
 Wire Wire Line
 	2550 5100 2550 5200
+$Comp
+L Connector_Generic:Conn_01x01 J13
+U 1 1 61937729
+P 2750 4850
+F 0 "J13" H 2830 4892 50  0000 L CNN
+F 1 "Hook 2" H 2830 4801 50  0000 L CNN
+F 2 "TestPoint:TestPoint_Keystone_5019_Minature" H 2750 4850 50  0001 C CNN
+F 3 "~" H 2750 4850 50  0001 C CNN
+	1    2750 4850
+	1    0    0    -1
+$EndComp
+$Comp
+L Connector_Generic:Conn_01x01 J12
+U 1 1 61937DD9
+P 2750 4650
+F 0 "J12" H 2830 4692 50  0000 L CNN
+F 1 "Hook 1" H 2830 4601 50  0000 L CNN
+F 2 "TestPoint:TestPoint_Keystone_5019_Minature" H 2750 4650 50  0001 C CNN
+F 3 "~" H 2750 4650 50  0001 C CNN
+	1    2750 4650
+	1    0    0    -1
+$EndComp
+Wire Wire Line
+	2550 4850 2550 5000
+Connection ~ 2550 5000
+Wire Wire Line
+	2550 4650 2550 4850
+Connection ~ 2550 4850
 $EndSCHEMATC
