File: mch2021.kicad_pcb (KiCad board)
At the start: 4 copper layers, 100 x 100 mm, 160 parts, among them J1 USB_C_Receptacle_USB2.0, J2 SAO, J3 AudioJack3, J4 SAO, J5 Micro SD card, J6 PMOD, J7 LCD, J8 GPIO, Q1 Q_PMOS_GSD, Q2 Q_NMOS_GSD, Q3 Q_NMOS_GSD, SW1 Power switch, SW2 Start, SW3 Select, SW4 Menu, SW5 Home, SW6 Back, SW7 Accept, U1 SY8079AAC, U10 SN74LVC1G125DCKR, U11 STM32F103C8Tx, U12 PCA9555PW, U13 ESP32-WROVER, U2 SY8079AAC, U3 XT4054K421MR-G, U4 SY6280AAC, U5 SY6280AAC, U6 MPU-6050, U7 74LVC1G125, U8 ICE40UP5K-SG48ITR, U9 LY68L6400, Y1 16MHz

Commit message: 33 DRC errors to go...
Parts:
- R27, R28, R32, R45: moved to B.Cu
- moved R32 35.4 mm to (47.4, 35.2), turned to 90 degrees
- moved R28 34.0 mm to (48.4, 31.2)
- moved R27 21.5 mm to (69.9, 23.3), turned to 0 degrees
- moved R29 21.1 mm to (27.9, 13.9), turned to 0 degrees
- moved R11 15.4 mm to (20.6, 66.2), turned to 0 degrees
- moved C28 13.6 mm to (94.3, 37.5)
- moved R25 12.9 mm to (70.7, 21.7)
- moved R34 12.1 mm to (92.7, 36.0), turned to 0 degrees
- moved R45 10.9 mm to (41.9, 62.4), turned to 90 degrees
- moved RN2 8.33 mm to (85.2, 97.6), turned to 90 degrees
- moved R24 5.29 mm to (76.9, 21.6), turned to 0 degrees
- moved C27 5.28 mm to (88.2, 35.6), turned to 180 degrees
- moved C35 4.36 mm to (86.7, 34.0)
- moved R33 4.35 mm to (81.1, 53.6), turned to 270 degrees
- moved C29 4.35 mm to (86.7, 32.6)
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Connections:
- D1 pad 2: /FPGA/RGB0 -> /FPGA/RGB1
- D1 pad 3: /FPGA/RGB1 -> /FPGA/RGB0
- S1 pad SH1: Net-(S1-PadSH1) -> GND
- S1 pad SH2: Net-(S1-PadSH1) -> GND
Routing:
- net /STM32/FPGA_RX: track 19.2 -> 107.4 mm, vias 2 -> 5
- net /STM32/FPGA_TX: track 15.5 -> 100.5 mm, vias 2 -> 5
- net /FPGA/CLK: track 13.6 -> 89.9 mm, vias 2 -> 5
- net /FPGA/LCD_ENABLE: track 7.21 -> 80.2 mm
- net /LCD/BACKLIGHT: track 8.18 -> 59.3 mm
- net /STM32/LCD_MODE: track 6.81 -> 53.8 mm, vias 0 -> 2
- net Net-(C28-Pad1): track 10.3 -> 30.1 mm
- net /LCD/LCD_IM0: track 0.00 -> 15.1 mm
- net /FPGA/RGB1: track 34.1 -> 48.2 mm, vias 0 -> 1
- net /POWER/SENSE_VBAT: track 132.2 -> 144.3 mm
- net /FPGA/RGB2: track 39.1 -> 51.1 mm, vias 0 -> 1
- net /LCD/LCD_RS_SCK_SWITCH: track 26.2 -> 37.4 mm
- net /STM32/LCD_RESET: track 72.0 -> 83.1 mm
- net +3V3: track 124.9 -> 135.0 mm, vias 27 -> 30
- net /POWER/SENSE_VUSB: track 134.2 -> 143.7 mm
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- added copper zone on F.Cu, net GND
