File: mch2021.kicad_pcb (KiCad board)
At the start: 4 copper layers, 100 x 100 mm, 160 parts, among them J1 USB_C_Receptacle_USB2.0, J2 SAO, J3 AudioJack3, J4 SAO, J5 Micro SD card, J6 PMOD, J7 LCD, J8 GPIO, Q1 Q_PMOS_GSD, Q2 Q_NMOS_GSD, Q3 Q_NMOS_GSD, SW1 Power switch, SW2 Start, SW3 Select, SW4 Menu, SW5 Home, SW6 Back, SW7 Accept, U1 SY8079AAC, U10 SN74LVC1G125DCKR, U11 STM32F103C8Tx, U12 PCA9555PW, U13 ESP32-WROVER, U2 SY8079AAC, U3 XT4054K421MR-G, U4 SY6280AAC, U5 SY6280AAC, U6 MPU-6050, U7 74LVC1G125, U8 ICE40UP5K-SG48ITR, U9 LY68L6400, Y1 16MHz

Commit message: Routed and 0 DRC errors
Parts:
- moved RN5 7.28 mm to (92.1, 18.2)
- moved RN6 7.16 mm to (86.9, 18.2)
- moved C29 6.23 mm to (92.7, 34.1), turned to 180 degrees
- moved R31 3.15 mm to (76.1, 24.2), turned to 90 degrees
- moved C16 2.17 mm to (91.8, 32.9), turned to 0 degrees
- moved C33 1.01 mm to (76.3, 14.4)
- moved C40 0.85 mm to (12.0, 25.9)
- moved R25 0.75 mm to (70.0, 21.7)
- moved Q3 0.67 mm to (73.4, 24.4), turned to 180 degrees
- moved R17 0.60 mm to (13.1, 73.2)
- moved R16 0.42 mm to (7.61, 70.9)
- moved C18 0.40 mm to (18.1, 72.7)
- moved U7 0.40 mm to (76.6, 46.4)
- moved C37 0.40 mm to (13.8, 27.2)
- moved R27 0.07 mm to (70.0, 23.3)
Connections:
- RN5 pad 1: /FPGA/PMOD_2 -> /FPGA/PMOD_6
- RN5 pad 2: /FPGA/PMOD_6 -> /FPGA/PMOD_2
- RN5 pad 3: /FPGA/PMOD_1 -> /FPGA/PMOD_5
- RN5 pad 4: /FPGA/PMOD_5 -> /FPGA/PMOD_1
- RN6 pad 5: /FPGA/PMOD_4 -> /FPGA/PMOD_8
- RN6 pad 6: /FPGA/PMOD_8 -> /FPGA/PMOD_4
- RN6 pad 7: /FPGA/PMOD_3 -> /FPGA/PMOD_7
- RN6 pad 8: /FPGA/PMOD_7 -> /FPGA/PMOD_3
- U13 pad 39: (no net) -> GND
- U8 pad 1: (no net) -> +3V3
Routing:
- net Net-(RN5-Pad8): track 19.5 -> 31.2 mm
- net Net-(RN5-Pad6): track 35.6 -> 24.6 mm
- net Net-(RN5-Pad7): track 35.3 -> 24.6 mm
- net /FPGA/PMOD_6: track 2.71 -> 13.4 mm
- net /FPGA/PMOD_8: track 2.74 -> 13.4 mm
- net /FPGA/PMOD_7: track 2.91 -> 13.4 mm
- net /FPGA/PMOD_5: track 2.94 -> 13.4 mm
- net Net-(RN5-Pad5): track 36.0 -> 26.2 mm
- net /FPGA/PMOD_4: track 5.90 -> 13.6 mm
- net /FPGA/PMOD_3: track 5.79 -> 13.4 mm
- net /FPGA/PMOD_1: track 5.81 -> 13.4 mm
- net /FPGA/PMOD_2: track 5.87 -> 13.4 mm
- net GND: track 256.6 -> 262.0 mm, vias 72 -> 81
- net /LCD/LCD_RS_SCK_SWITCH: track 37.4 -> 33.9 mm
- net Net-(RN6-Pad1): track 21.0 -> 24.6 mm
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
Commit message: Small tweaks
Parts:
- moved R33 34.9 mm to (48.9, 40.0), turned to 180 degrees
Routing:
- net /ESP32/SPI_MOSI: track 162.1 -> 246.3 mm
- net /FPGA/SPI_CS: track 99.4 -> 137.6 mm
- net /LCD/LCD_WR_RS: track 108.2 -> 132.0 mm
- net /ACCELEROMETER/I2C_SCL: track 126.4 -> 139.9 mm
- net /ESP32/SPI_CLK: track 158.2 -> 155.9 mm
- net /ESP32/SPI_MISO: track 129.9 -> 128.1 mm
- net GND: track 262.0 -> 263.2 mm
- net /FPGA/LCD_RS: track 22.9 -> 24.0 mm

Commit message: Final touches
Parts:
- added G***: LOGO, custom:badgeteam, B.Cu at (-12.0, 43.3)
- added Ref**: Val**, custom:artwork, F.Cu at (50.0, 50.0)

Commit message: Moved SAO2/3, I2C_SDA/SCL away from antenna, and LCD/CS away from hole in PCB.
Routing:
- net /FPGA/RGB0: track 45.6 -> 43.8 mm
- net /LCD/CS: track 95.0 -> 96.0 mm
- net /FPGA/RGB1: track 48.0 -> 47.1 mm
- net /STM32/SAO_IO2: track 61.9 -> 62.6 mm
- net /ACCELEROMETER/I2C_SDA: track 130.3 -> 129.7 mm
- net /STM32/SAO_IO3: track 65.5 -> 66.1 mm

Commit message: Dump.
Parts:
- removed G***: LOGO, custom:badgeteam
- added C45: 100n, Capacitor_SMD:C_0603_1608Metric, B.Cu at (74.2, 62.4)
- added C46: 100n, Capacitor_SMD:C_0603_1608Metric, B.Cu at (77.1, 62.4)
- added D10: USBLC6-4SC6, digikey-footprints:SOT23-6L, B.Cu at (23.1, 5.50)
- added R61: DNP, Resistor_SMD:R_0603_1608Metric, B.Cu at (8.31, 11.0)
- added R62: DNP, Resistor_SMD:R_0603_1608Metric, B.Cu at (8.42, 7.78)
- C10, C11, C12, C15, C4, C5, C9: footprint Capacitor_SMD:C_0603_1608Metric -> Capacitor_SMD:C_0805_2012Metric
- moved RN4 20.8 mm to (62.6, 34.0), turned to 0 degrees
- moved RN3 17.1 mm to (62.6, 38.0), turned to 0 degrees
- moved R1 14.4 mm to (9.90, 11.0), turned to 270 degrees
- moved R2 5.16 mm to (20.4, 10.3)
- moved R12 1.31 mm to (11.2, 12.8)
- moved C11 0.75 mm to (94.2, 76.7)
- moved C12 0.71 mm to (94.2, 66.1)
- moved C10 0.37 mm to (92.1, 66.2)
- moved C9 0.20 mm to (92.0, 76.7)
Connections:
- net /FPGA/AUDO_L renamed /FPGA/AUDIO_L
- net /FPGA/AUDO_R renamed /FPGA/AUDIO_R
- J1 pad A8: (no net) -> SBU1
- J1 pad B8: (no net) -> SBU2
Routing:
- net /FPGA/LCD_D7: track 36.3 -> 19.3 mm
- net /FPGA/LCD_D6: track 35.6 -> 19.2 mm
- net /FPGA/LCD_D5: track 34.6 -> 19.0 mm
- net /FPGA/LCD_D4: track 33.9 -> 19.0 mm
- net /FPGA/LCD_D3: track 32.7 -> 18.9 mm
- net SBU1: track 0.00 -> 13.2 mm, vias 0 -> 2
- net /FPGA/LCD_D2: track 32.4 -> 19.6 mm
- net Net-(C1-Pad2): track 9.73 -> 21.5 mm
- net /FPGA/LCD_D1: track 31.4 -> 20.1 mm
- net /FPGA/LCD_D0: track 31.0 -> 19.8 mm
- net SBU2: track 0.00 -> 9.47 mm
- net /ACCELEROMETER/I2C_SDA: track 129.7 -> 138.6 mm
- net /STM32/USB_D+: track 10.6 -> 18.2 mm
- net /STM32/USB_D-: track 10.6 -> 18.0 mm
- net /ACCELEROMETER/I2C_SCL: track 139.5 -> 146.8 mm
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Other:
- board text added: "JLCJLCJLCJLC"
