File: mch2021.kicad_pcb (KiCad board)
At the start: 4 copper layers, 100 x 100 mm, 166 parts, among them J1 USB_C_Receptacle_USB2.0, J2 SAO, J3 AudioJack3, J4 SAO, J5 Micro SD card, J6 PMOD, J7 LCD, J8 GPIO, Q1 Q_PMOS_GSD, Q2 Q_NMOS_GSD, Q3 Q_NMOS_GSD, SW1 Power switch, SW2 Start, SW3 Select, SW4 Menu, SW5 Home, SW6 Back, SW7 Accept, U1 SY8079AAC, U10 SN74LVC1G125DCKR, U11 STM32F103C8Tx, U12 PCA9555PW, U13 ESP32-WROVER, U2 SY8079AAC, U3 XT4054K421MR-G, U4 SY6280AAC, U5 SY6280AAC, U6 MPU-6050, U7 74LVC1G125, U8 ICE40UP5K-SG48ITR, U9 LY68L6400, Y1 16MHz

Commit message: Work in progress: prototype 2
Parts:
- removed C14: 100n, Capacitor_SMD:C_0603_1608Metric
- removed D3: CDBU0130R, Diode_SMD:D_0603_1608Metric
- removed R3: 47, Resistor_SMD:R_0603_1608Metric
- removed Ref**: Val**, custom:artwork
- C1, C2, C30, C31: value C_Small -> TBD
- C37, C38: value 20p -> 22p
- R33, R35: value 100k -> 10k
- R36: value 100k -> DNP
- U10: value SN74LVC1G125DCKR -> 74LVC1G125; footprint digikey-footprints:SOT-353 -> Package_TO_SOT_SMD:SOT-353_SC-70-5
- moved U10 0.06 mm to (25.8, 9.18), turned to 0 degrees
- turned R33 to 0 degrees
- turned S1 to 45 degrees
Connections:
- BT1 pad 1: VBAT -> (no net)
- BT1 pad 3: (no net) -> VBAT
- D10 pad 1: Net-(C2-Pad1) -> (no net)
- D10 pad 3: Net-(C1-Pad2) -> (no net)
- D9 pad 2: /LED/DATA_OUT -> (no net)
- J7 pad 39: /LCD/LCD_RS_SCK_SWITCH -> Net-(J7-Pad39)
- J7 pad 40: /LCD/LCD_RS_SCK_SWITCH -> Net-(J7-Pad39)
- Q3 pad 3: /LCD/LCD_RS_SCK_SWITCH -> Net-(J7-Pad39)
- R27 pad 2: /LCD/LCD_RS_SCK_SWITCH -> Net-(J7-Pad39)
- R33 pad 1: /FPGA/SPI_CS -> +3V3
- R33 pad 2: GND -> /FPGA/SPI_CS
- U10 pad 1: /POWER/PWR_LED_ENABLE -> GND
- U7 pad 1: /LCD/LCD_RS_SCK_SWITCH -> /STM32/LCD_MODE
- U8 pad 24: +2V5 -> +3V3
Routing:
- net /STM32/LCD_MODE: track 53.0 -> 87.9 mm, vias 2 -> 4
- net /LCD/LCD_RS_SCK_SWITCH: track 33.9 -> 0.00 mm, vias 2 -> 0
- net Net-(C1-Pad2): track 21.5 -> 9.73 mm
- net Net-(J7-Pad39): track 0.00 -> 11.7 mm
- net /POWER/PWR_LED_ENABLE: track 30.4 -> 19.4 mm
- net +3V3: track 138.8 -> 146.4 mm, vias 30 -> 31
- net GND: track 269.8 -> 276.6 mm
- net +2V5: track 4.32 -> 0.00 mm
- net Net-(C2-Pad1): track 18.7 -> 14.6 mm
- net VBAT: track 17.1 -> 20.6 mm
- net /LED/DATA_OUT: track 3.18 -> 0.00 mm
- net (no net): track 0.00 -> 3.18 mm
- net JOY_D: track 30.7 -> 32.1 mm
- net JOY_A: track 37.4 -> 38.5 mm
- net /STM32/LCD_RESET: track 83.1 -> 84.2 mm
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
Commit message: More work on prototype 2
Parts:
- added C1: 100n, Capacitor_SMD:C_0603_1608Metric, F.Cu at (137.3, 11.2)
- added C14: 22p, Capacitor_SMD:C_0603_1608Metric, F.Cu at (159.1, 17.1)
- added C2: 22p, Capacitor_SMD:C_0603_1608Metric, F.Cu at (150.7, 19.1)
- added D2: NSVR0320MW2T1G, Diode_SMD:D_SOD-323, F.Cu at (125.1, 10.5)
- added J2: QWIIC_CONNECTORJS-1MM, Connectors:1X04_1MM_RA, F.Cu at (154.2, 38.6)
- added Q1: Q_NMOS_GSD, Package_TO_SOT_SMD:SOT-23, F.Cu at (135.1, 7.70)
- added Q4: Q_NMOS_GSD, Package_TO_SOT_SMD:SOT-23, F.Cu at (150.9, 15.6)
- added R3: 10k, Resistor_SMD:R_0603_1608Metric, F.Cu at (158.4, 2.03)
- added R30: 10k, Resistor_SMD:R_0603_1608Metric, F.Cu at (158.4, 4.54)
- added R38: 10k, Resistor_SMD:R_0603_1608Metric, F.Cu at (162.5, 2.03)
- added R39: 10k, Resistor_SMD:R_0603_1608Metric, F.Cu at (158.7, 7.05)
- added R53: 10k, Resistor_SMD:R_0603_1608Metric, F.Cu at (150.7, 8.43)
- added R54: 10k, Resistor_SMD:R_0603_1608Metric, F.Cu at (139.7, 2.03)
- added R55: 10k, Resistor_SMD:R_0603_1608Metric, F.Cu at (129.3, 10.3)
- added R56: 10k, Resistor_SMD:R_0603_1608Metric, F.Cu at (133.3, 11.2)
- added R57: 100k, Resistor_SMD:R_0603_1608Metric, F.Cu at (139.7, 4.54)
- added R58: 10k, Resistor_SMD:R_0603_1608Metric, F.Cu at (139.3, 7.05)
- added R61: 47, Resistor_SMD:R_0603_1608Metric, F.Cu at (154.7, 19.6)
- added R62: 47, Resistor_SMD:R_0603_1608Metric, F.Cu at (159.1, 14.6)
- added R63: 10k, Resistor_SMD:R_0603_1608Metric, F.Cu at (155.1, 17.1)
- added R64: 10k, Resistor_SMD:R_0603_1608Metric, F.Cu at (155.1, 14.6)
- added R7: 10k, Resistor_SMD:R_0603_1608Metric, F.Cu at (154.7, 8.43)
- added U14: SY6280AAC, Package_TO_SOT_SMD:SOT-23-5, F.Cu at (135.3, 3.10)
- added U15: AMS1117-3.3, Package_TO_SOT_SMD:SOT-223-3_TabPin2, F.Cu at (127.9, 4.90)
- R43: value 10k -> DNP
Connections:
- C1 pad 2: Net-(C1-Pad2) -> (no net)
- D10 pad 3: (no net) -> /CC1
- J1 pad A8: SBU1 -> (no net)
- J1 pad B8: SBU2 -> (no net)
- J2 pad 5: /STM32/SAO_IO2 -> (no net)
- J2 pad 6: /STM32/SAO_IO3 -> (no net)
- J3 pad R: Net-(C2-Pad1) -> (no net)
- J3 pad T: Net-(C1-Pad2) -> (no net)
- J5 pad 1: SD_D2 -> Net-(J5-Pad1)
- J5 pad 2: /ESP32/SD_D3 -> Net-(J5-Pad2)
- J5 pad 3: SD_CMD -> /ESP32/SD_CMD
- J5 pad 7: SD_D0 -> /ESP32/SD_D0
- J5 pad 8: /ESP32/SD_D1 -> Net-(J5-Pad8)
- J8 pad 2: Net-(J8-Pad2) -> (no net)
- J8 pad 3: Net-(J8-Pad3) -> (no net)
- LS1 pad 2: SPK -> (no net)
- R10 pad 1: /BUTTONS/CHARGING -> /POWER/CHARGING
- R11 pad 2: /ESP32/PWR_SDCARD_ENABLE -> /POWER/PWR_SDCARD_ENABLE
- R38 pad 2: Net-(R38-Pad2) -> (no net)
- R39 pad 2: Net-(R39-Pad2) -> (no net)
- R46 pad 1: SD_D0 -> /ESP32/SD_D0
- R49 pad 2: SD_D2 -> Net-(R49-Pad2)
- R50 pad 1: SD_D2 -> Net-(R49-Pad2)
- R54 pad 2: SD_CMD -> (no net)
- R55 pad 2: SD_D0 -> (no net)
- R56 pad 2: /ESP32/SD_D1 -> (no net)
- R57 pad 2: SD_D2 -> (no net)
- R58 pad 2: /ESP32/SD_D3 -> (no net)
- R59 pad 2: SD_CMD -> /ESP32/SD_CMD
- R60 pad 1: SD_CMD -> /ESP32/SD_CMD
- R61 pad 1: SBU1 -> (no net)
- R62 pad 2: SBU2 -> (no net)
- RN1 pad 5: ESP32_AUDIO_R -> (no net)
- RN1 pad 7: ESP32_AUDIO_L -> (no net)
- SW1 pad 1: Net-(D2-Pad1) -> Net-(R55-Pad1)
- SW1 pad 2: VIN -> VBAT
- SW1 pad 3: VUSB -> (no net)
- U11 pad 1: +3V3 -> BAT_3.3
- U11 pad 12: /ESP32/ESP32_RX -> /STM32/FPGA_RX
- U11 pad 13: /ESP32/ESP32_TX -> /STM32/FPGA_TX
- U11 pad 18: /STM32/SAO_IO3 -> /ESP32/ESP32_EN
- U11 pad 19: /STM32/SAO_IO2 -> Net-(R62-Pad2)
- U11 pad 2: /ESP32/ESP32_EN -> Net-(Q4-Pad3)
- U11 pad 20: /STM32/SAO_IO1 -> /POWER/CHARGING
- U11 pad 21: /STM32/SAO_IO0 -> /ACCELEROMETER/I2C_SCL
- U11 pad 22: Net-(U10-Pad2) -> /ACCELEROMETER/I2C_SDA
- U11 pad 25: Net-(J8-Pad3) -> /STM32/SAO_IO0
- U11 pad 26: Net-(J8-Pad2) -> /STM32/SAO_IO1
- U11 pad 28: Net-(U10-Pad2) -> /POWER/PWR_SDCARD_ENABLE
- U11 pad 3: /ESP32/ESP32_BL -> Net-(C14-Pad1)
- U11 pad 30: /STM32/FPGA_RX -> /ESP32/ESP32_RX
- U11 pad 31: /STM32/FPGA_TX -> /ESP32/ESP32_TX
- U11 pad 38: SPK -> Net-(R64-Pad2)
- U11 pad 4: (no net) -> Net-(C2-Pad1)
- U11 pad 42: /ACCELEROMETER/I2C_SCL -> Net-(U10-Pad2)
- U11 pad 43: /ACCELEROMETER/I2C_SDA -> (no net)
- U11 pad 45: /FPGA/LCD_ENABLE -> (no net)
- U12 pad 8: /BUTTONS/CHARGING -> (no net)
- U13 pad 10: ESP32_AUDIO_L -> (no net)
- U13 pad 11: ESP32_AUDIO_R -> (no net)
- U13 pad 14: SD_D2 -> Net-(R49-Pad2)
- U13 pad 16: /ESP32/SD_D3 -> (no net)
- U13 pad 23: SD_CMD -> /ESP32/SD_CMD
- U13 pad 24: SD_D0 -> /ESP32/SD_D0
- U13 pad 26: /ESP32/SD_D1 -> (no net)
- U13 pad 29: /ESP32/PWR_SDCARD_ENABLE -> (no net)
- U3 pad 1: /BUTTONS/CHARGING -> /POWER/CHARGING
- U4 pad 4: /ESP32/PWR_SDCARD_ENABLE -> /POWER/PWR_SDCARD_ENABLE
- U7 pad 1: /STM32/LCD_MODE -> /LCD/LCD_IM0
- U8 pad 38: /FPGA/LCD_ENABLE -> (no net)
- U8 pad 42: Net-(R39-Pad2) -> (no net)
- U8 pad 43: Net-(R38-Pad2) -> (no net)
Routing:
- net (no net): track 3.18 -> 376.4 mm, vias 0 -> 10
- net /FPGA/LCD_ENABLE: track 80.2 -> 0.00 mm
- net ESP32_AUDIO_L: track 68.2 -> 0.00 mm, vias 2 -> 0
- net ESP32_AUDIO_R: track 65.4 -> 0.00 mm, vias 2 -> 0
- net Net-(R39-Pad2): track 65.4 -> 0.00 mm, vias 2 -> 0
- net Net-(R38-Pad2): track 61.6 -> 0.00 mm, vias 2 -> 0
- net SBU1: track 13.2 -> 0.00 mm, vias 2 -> 0
- net Net-(C1-Pad2): track 9.73 -> 0.00 mm
- net SBU2: track 9.47 -> 0.00 mm

Commit message: Schematic for prototype 2 is now complete, time for review! :D
Parts:
- removed the C1 at (137.3, 11.2)
- removed the C1 at (40.7, 4.06)
- removed the C2 at (150.7, 19.1)
- removed the C2 at (40.7, 2.29)
- removed the D2 at (125.1, 10.5)
- removed the D2 at (89.9, 94.4)
- removed the J2 at (154.2, 38.6)
- removed the J2 at (4.93, 68.0)
- removed LS1: Speaker_Crystal, Buzzer_Beeper:Buzzer_Murata_PKMCS0909E4000-R1
- removed the Q1 at (135.1, 7.70)
- removed the Q1 at (89.8, 97.5)
- removed the R30 at (158.4, 4.54)
- removed the R30 at (26.2, 19.2)
- removed the R38 at (162.5, 2.03)
- removed the R38 at (48.0, 4.83)
- removed the R39 at (158.7, 7.05)
- removed the R39 at (48.0, 3.30)
- removed the R53 at (150.7, 8.43)
- removed the R53 at (22.7, 38.6)
- removed the R54 at (139.7, 2.03)
- removed the R54 at (27.6, 63.6)
- removed the R55 at (129.3, 10.3)
- removed the R55 at (24.5, 60.6)
- removed the R56 at (133.3, 11.2)
- removed the R56 at (24.5, 63.6)
- removed the R57 at (139.7, 4.54)
- removed the R57 at (25.1, 36.3)
- removed the R58 at (139.3, 7.05)
- removed the R58 at (28.1, 39.3)
- removed the R61 at (154.7, 19.6)
- removed the R61 at (8.31, 11.0)
- removed the R62 at (159.1, 14.6)
- removed the R62 at (8.42, 7.78)
- removed the R7 at (154.7, 8.43)
- removed the R7 at (12.3, 11.3)
- removed RN1: TBD, Resistor_SMD:R_Array_Convex_4x0603
- added C1: 100n, Capacitor_SMD:C_0603_1608Metric, F.Cu at (140.5, 58.5)
- added C2: 22p, Capacitor_SMD:C_0603_1608Metric, F.Cu at (177.1, 47.3)
- added C47: 100n, Capacitor_SMD:C_0603_1608Metric, F.Cu at (166.0, 53.4)
- added C48: 22p, Capacitor_SMD:C_0603_1608Metric, F.Cu at (159.4, 59.1)
- added C49: 22p, Capacitor_SMD:C_0603_1608Metric, F.Cu at (163.4, 55.9)
- added C50: 100n, Capacitor_SMD:C_0603_1608Metric, F.Cu at (170.0, 50.9)
- added D2: NSVR0320MW2T1G, Diode_SMD:D_SOD-323, F.Cu at (136.6, 55.8)
- added J2: QWIIC_CONNECTORJS-1MM, Connectors:1X04_1MM_RA, F.Cu at (140.2, 34.5)
- added Q1: Q_NMOS_GSD, Package_TO_SOT_SMD:SOT-23, F.Cu at (132.3, 56.6)
- added R30: 10k, Resistor_SMD:R_0603_1608Metric, F.Cu at (154.8, 26.5)
- added R38: 10k, Resistor_SMD:R_0603_1608Metric, F.Cu at (130.2, 41.7)
- added R39: 10k, Resistor_SMD:R_0603_1608Metric, F.Cu at (126.2, 44.2)
- added R53: 10k, Resistor_SMD:R_0603_1608Metric, F.Cu at (122.2, 44.2)
- added R54: 10k, Resistor_SMD:R_0603_1608Metric, F.Cu at (136.1, 61.0)
- added R55: 10k, Resistor_SMD:R_0603_1608Metric, F.Cu at (145.8, 50.9)
- added R56: 10k, Resistor_SMD:R_0603_1608Metric, F.Cu at (140.7, 55.5)
- added R57: 100k, Resistor_SMD:R_0603_1608Metric, F.Cu at (132.0, 62.6)
- added R58: 10k, Resistor_SMD:R_0603_1608Metric, F.Cu at (136.1, 63.5)
- added R61: 47, Resistor_SMD:R_0603_1608Metric, F.Cu at (181.1, 47.8)
- added R62: 47, Resistor_SMD:R_0603_1608Metric, F.Cu at (185.5, 42.8)
- added R65: 47, Resistor_SMD:R_0603_1608Metric, F.Cu at (138.3, 40.9)
- added R66: 47, Resistor_SMD:R_0603_1608Metric, F.Cu at (122.2, 41.7)
- added R67: 47, Resistor_SMD:R_0603_1608Metric, F.Cu at (194.1, 29.0)
- added R68: 47, Resistor_SMD:R_0603_1608Metric, F.Cu at (194.1, 26.5)
- added R69: 4.7k, Resistor_SMD:R_0603_1608Metric, F.Cu at (163.2, 26.5)
- added R7: 10k, Resistor_SMD:R_0603_1608Metric, F.Cu at (138.2, 43.5)
- added R70: 4k7, Resistor_SMD:R_0603_1608Metric, F.Cu at (162.0, 50.9)
- added R71: 4k7, Resistor_SMD:R_0603_1608Metric, F.Cu at (162.0, 53.4)
- added R72: 4k7, Resistor_SMD:R_0603_1608Metric, F.Cu at (159.4, 56.6)
- added TP1: LED OUT, TestPoint:TestPoint_Pad_1.0x1.0mm, F.Cu at (152.7, 36.2)
- added TP10: STM32 RESET, TestPoint:TestPoint_Pad_1.0x1.0mm, F.Cu at (149.6, 33.2)
- added TP11: STM32 BOOT0, TestPoint:TestPoint_Pad_1.0x1.0mm, F.Cu at (149.6, 36.2)
- added TP12: ESP EN, TestPoint:TestPoint_Pad_1.0x1.0mm, F.Cu at (166.8, 26.8)
- added TP13: IRQ SENSOR, TestPoint:TestPoint_Pad_1.0x1.0mm, F.Cu at (162.7, 32.3)
- added TP14: IRQ FPGA, TestPoint:TestPoint_Pad_1.0x1.0mm, F.Cu at (165.8, 29.8)
- added TP15: ESP32 BL, TestPoint:TestPoint_Pad_1.0x1.0mm, F.Cu at (169.8, 26.8)
- added TP16: ESP32 TX, TestPoint:TestPoint_Pad_1.0x1.0mm, F.Cu at (162.7, 35.4)
- added TP17: ESP32 RX, TestPoint:TestPoint_Pad_1.0x1.0mm, F.Cu at (174.9, 29.8)
- added TP18: ESP32 TDI, TestPoint:TestPoint_Pad_1.0x1.0mm, F.Cu at (165.8, 32.9)
- added TP19: ESP32 TDI, TestPoint:TestPoint_Pad_1.0x1.0mm, F.Cu at (168.8, 29.8)
- added TP2: LED IN, TestPoint:TestPoint_Pad_1.0x1.0mm, F.Cu at (144.9, 43.4)
- added TP20: ESP32 TDI, TestPoint:TestPoint_Pad_1.0x1.0mm, F.Cu at (172.9, 26.8)
- added TP21: ESP32 TCK, TestPoint:TestPoint_Pad_1.0x1.0mm, F.Cu at (165.8, 35.9)
- added TP22: ESP32 TMS, TestPoint:TestPoint_Pad_1.0x1.0mm, F.Cu at (168.8, 32.9)
- added TP23: ESP32 TDO, TestPoint:TestPoint_Pad_1.0x1.0mm, F.Cu at (162.7, 29.3)
- added TP24: SPI CLK, TestPoint:TestPoint_Pad_1.0x1.0mm, F.Cu at (175.9, 26.8)
- added TP25: SPI CS STM32, TestPoint:TestPoint_Pad_1.0x1.0mm, F.Cu at (171.9, 29.8)
- added TP26: SPI MOSI, TestPoint:TestPoint_Pad_1.0x1.0mm, F.Cu at (174.9, 35.9)
- added TP27: SPI MOSI, TestPoint:TestPoint_Pad_1.0x1.0mm, F.Cu at (182.0, 26.8)
- added TP28: SPI MOSI, TestPoint:TestPoint_Pad_1.0x1.0mm, F.Cu at (178.0, 29.8)
- added TP29: SPI CS FPGA, TestPoint:TestPoint_Pad_1.0x1.0mm, F.Cu at (174.9, 32.9)
- added TP3: LED IN, TestPoint:TestPoint_Pad_1.0x1.0mm, F.Cu at (148.7, 39.3)
- added TP30: SPI CS LCD, TestPoint:TestPoint_Pad_1.0x1.0mm, F.Cu at (171.9, 35.9)
- added TP31: LCD DC, TestPoint:TestPoint_Pad_1.0x1.0mm, F.Cu at (179.0, 26.8)
- added TP32: IRQ BTN, TestPoint:TestPoint_Pad_1.0x1.0mm, F.Cu at (171.9, 32.9)
- added TP33: SPI MISO, TestPoint:TestPoint_Pad_1.0x1.0mm, F.Cu at (168.8, 35.9)
- added TP4: LCD MODE, TestPoint:TestPoint_Pad_1.0x1.0mm, F.Cu at (145.6, 40.4)
- added TP5: LCD RESET, TestPoint:TestPoint_Pad_1.0x1.0mm, F.Cu at (145.6, 37.3)
- added TP6: LCD BACKLIGHT, TestPoint:TestPoint_Pad_1.0x1.0mm, F.Cu at (141.8, 41.2)
- added TP7: FPGA RX, TestPoint:TestPoint_Pad_1.0x1.0mm, F.Cu at (154.4, 29.3)
- added TP8: FPGA TX, TestPoint:TestPoint_Pad_1.0x1.0mm, F.Cu at (141.8, 44.3)
- added TP9: MCO, TestPoint:TestPoint_Pad_1.0x1.0mm, F.Cu at (152.7, 33.2)
- added U16: BNO055, digikey-footprints:LGA-28_5.2x3.8mm_BNO0055, F.Cu at (156.3, 52.5)
- added U17: BME680, Package_LGA:Bosch_LGA-8_3x3mm_P0.8mm_ClockwisePinNumbering, F.Cu at (155.1, 57.7)
- C16: value 100n -> 1u; footprint Capacitor_SMD:C_0603_1608Metric -> Capacitor_SMD:C_0402_1005Metric; moved to F.Cu
- C17: footprint Capacitor_SMD:C_0603_1608Metric -> Capacitor_SMD:C_0402_1005Metric
- C18: value 2.2n -> 1u; footprint Capacitor_SMD:C_0603_1608Metric -> Capacitor_SMD:C_0402_1005Metric
- C19: value 100n -> 1u; footprint Capacitor_SMD:C_0603_1608Metric -> Capacitor_SMD:C_0402_1005Metric
- C20: value 10u -> 1u; footprint Capacitor_SMD:C_0603_1608Metric -> Capacitor_SMD:C_0402_1005Metric
- C30: value TBD -> 100n; footprint Capacitor_SMD:C_0603_1608Metric -> Capacitor_SMD:C_0402_1005Metric; moved to F.Cu
- C31: value TBD -> 100n; moved to F.Cu
- C6, L1, R11, R5, U1: moved to F.Cu
- J4: value SAO -> QWIIC_CONNECTORJS-1MM; footprint Connector_PinSocket_2.54mm:PinSocket_2x03_P2.54mm_Vertical -> Connectors:1X04_1MM_RA
- R15, R16, R17: value 4k7 -> 47
- R49: value 45.3k -> 4.7k
- R50: value DNP -> 47; moved to F.Cu
- U6: value MPU-6050 -> PCM5100; footprint Sensor_Motion:InvenSense_QFN-24_4x4mm_P0.5mm -> Package_SO:TSSOP-20_4.4x6.5mm_P0.65mm
- moved U10 165.2 mm to (190.0, 27.2)
- moved C19 145.4 mm to (155.6, 33.8)
- moved J4 144.8 mm to (148.9, 26.4)
- moved C20 141.9 mm to (148.6, 41.8), turned to 0 degrees
- moved C17 138.5 mm to (147.9, 43.8), turned to 0 degrees
- moved C18 137.8 mm to (151.6, 38.7), turned to 0 degrees
- moved U6 131.2 mm to (140.7, 29.3), turned to 0 degrees
- moved R12 129.7 mm to (132.0, 60.1)
- moved C31 127.8 mm to (166.0, 50.9), turned to 0 degrees
- moved R16 125.5 mm to (130.2, 44.2), turned to 0 degrees
- moved R11 124.8 mm to (144.8, 53.4)
- moved R15 121.7 mm to (134.2, 44.2), turned to 0 degrees
- moved R50 121.1 mm to (146.1, 34.5)
- moved R17 117.4 mm to (126.2, 41.7), turned to 0 degrees
- moved C30 110.6 mm to (155.6, 31.8), turned to 0 degrees
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Connections:
- net /BUTTONS/STM32_BOOT0 renamed /BOSCH/BOOT
- net /LED/DATA_IN renamed Net-(D4-Pad4)
- C16 pad 1: +3V3 -> Net-(C16-Pad1)
- C17 pad 1: GND -> Net-(C16-Pad1)
- C17 pad 2: Net-(C17-Pad2) -> GND
- C18 pad 1: GND -> Net-(C18-Pad1)
- C19 pad 1: +3V3 -> Net-(C19-Pad1)
- C30 pad 1: GND -> +3V3
- C30 pad 2: /FPGA/AUDIO_L -> GND
- C31 pad 1: GND -> +3V3
- C31 pad 2: /FPGA/AUDIO_R -> GND
- D9 pad 2: (no net) -> /LED/DATA_OUT
- J3 pad R: (no net) -> Net-(J3-PadR)
- J3 pad T: (no net) -> Net-(J3-PadT)
- J4 pad 3: /ACCELEROMETER/I2C_SCL -> /ESP32/EXT_I2C_SDA
- J4 pad 4: /ACCELEROMETER/I2C_SDA -> /ESP32/EXT_I2C_SCL
- J8 pad 2: (no net) -> Net-(J8-Pad2)
- J8 pad 3: (no net) -> Net-(J8-Pad3)
- R15 pad 1: +3V3 -> ESP_I2S_LR
- R15 pad 2: /ACCELEROMETER/AUX_SDA -> Net-(R15-Pad2)
- R16 pad 1: +3V3 -> FPGA_I2S_LR
- R16 pad 2: /ACCELEROMETER/AUX_SCL -> Net-(R15-Pad2)
- R17 pad 1: +3V3 -> ESP_I2S_DATA
- R17 pad 2: /ACCELEROMETER/IRQ -> Net-(R17-Pad2)
- R45 pad 2: /BUTTONS/IRQ -> /STM32/ESP32_WK
- R49 pad 2: Net-(R49-Pad2) -> /ESP32/EXT_I2C_SDA
- R50 pad 1: Net-(R49-Pad2) -> FPGA_I2S_DATA
- R50 pad 2: GND -> Net-(R17-Pad2)
- R51 pad 2: /ACCELEROMETER/I2C_SCL -> /BUTTONS/I2C_SCL
- R52 pad 2: /ACCELEROMETER/I2C_SDA -> /BUTTONS/I2C_SDA
- U10 pad 2: Net-(U10-Pad2) -> Net-(R67-Pad1)
- U11 pad 21: /ACCELEROMETER/I2C_SCL -> /BUTTONS/I2C_SCL
- U11 pad 22: /ACCELEROMETER/I2C_SDA -> /BUTTONS/I2C_SDA
- U11 pad 25: /STM32/SAO_IO0 -> (no net)
- U11 pad 26: /STM32/SAO_IO1 -> (no net)
- U11 pad 39: (no net) -> /STM32/ESP32_WK
- U11 pad 42: Net-(U10-Pad2) -> /LED/DATA_IN2
- U11 pad 43: (no net) -> Net-(J8-Pad2)
- U11 pad 45: (no net) -> Net-(J8-Pad3)
- U12 pad 1: /BUTTONS/IRQ -> /STM32/ESP32_WK
- U12 pad 22: /ACCELEROMETER/I2C_SCL -> /BUTTONS/I2C_SCL
- U12 pad 23: /ACCELEROMETER/I2C_SDA -> /BUTTONS/I2C_SDA
- U12 pad 8: (no net) -> /BUTTONS/BNO055_RESET
- U13 pad 10: (no net) -> ESP_I2S_CLK
- U13 pad 11: (no net) -> ESP_I2S_DATA
- U13 pad 14: Net-(R49-Pad2) -> /ESP32/EXT_I2C_SDA
- U13 pad 16: (no net) -> /ESP32/EXT_I2C_SCL
- U13 pad 26: (no net) -> ESP_I2S_LR
- U13 pad 29: (no net) -> /LED/DATA_IN1
- U13 pad 33: /ACCELEROMETER/I2C_SCL -> /BUTTONS/I2C_SCL
- U13 pad 36: /ACCELEROMETER/I2C_SDA -> /BUTTONS/I2C_SDA
- U13 pad 4: /ACCELEROMETER/IRQ -> /BOSCH/INT
- U13 pad 6: /BUTTONS/IRQ -> /STM32/ESP32_WK
- U6 pad 1: GND -> +3V3
- U6 pad 10: Net-(C17-Pad2) -> GND
- U6 pad 12: /ACCELEROMETER/IRQ -> GND
- U6 pad 13: +3V3 -> Net-(R65-Pad2)
- U6 pad 14: (no net) -> Net-(R17-Pad2)
- U6 pad 15: (no net) -> Net-(R15-Pad2)
- U6 pad 16: (no net) -> GND
- U6 pad 17: (no net) -> +3V3
- U6 pad 18: GND -> Net-(C16-Pad1)
- U6 pad 19: (no net) -> GND
- U6 pad 2: (no net) -> Net-(C18-Pad1)
- U6 pad 20: Net-(C18-Pad2) -> +3V3
- U6 pad 3: (no net) -> GND
- U6 pad 4: (no net) -> Net-(C18-Pad2)
- U6 pad 5: (no net) -> Net-(C19-Pad1)
- U6 pad 6: /ACCELEROMETER/AUX_SDA -> Net-(J3-PadT)
- U6 pad 7: /ACCELEROMETER/AUX_SCL -> Net-(J3-PadR)
- U8 pad 38: (no net) -> FPGA_I2S_CLK
- U8 pad 42: (no net) -> FPGA_I2S_LR
- U8 pad 43: (no net) -> FPGA_I2S_DATA
Routing:
- net (no net): track 376.4 -> 80.2 mm, vias 10 -> 0
- net /ACCELEROMETER/I2C_SCL: track 146.8 -> 0.00 mm, vias 4 -> 0
- net /ACCELEROMETER/I2C_SDA: track 138.6 -> 0.00 mm, vias 4 -> 0
- net /STM32/SAO_IO3: track 66.1 -> 0.00 mm, vias 1 -> 0
- net ESP_I2S_CLK: track 0.00 -> 64.7 mm, vias 0 -> 2
- net ESP_I2S_DATA: track 0.00 -> 64.2 mm, vias 0 -> 2
- net /STM32/SAO_IO2: track 62.6 -> 0.00 mm, vias 1 -> 0
- net /STM32/ESP32_WK: track 0.00 -> 60.7 mm, vias 0 -> 2
- net /BUTTONS/IRQ: track 60.7 -> 0.00 mm, vias 2 -> 0
- net FPGA_I2S_LR: track 0.00 -> 59.2 mm, vias 0 -> 2
- net /BUTTONS/I2C_SDA: track 0.00 -> 57.3 mm, vias 0 -> 1
- net FPGA_I2S_DATA: track 0.00 -> 55.9 mm, vias 0 -> 2
- net /BUTTONS/I2C_SCL: track 0.00 -> 54.5 mm, vias 0 -> 1
- net SPK: track 52.0 -> 0.00 mm
- net Net-(R64-Pad2): track 0.00 -> 52.0 mm
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
Commit message: Updated schematic, add design file
Parts:
- removed H1, H2, H3, H4: MountingHole_Pad, corecode:HOLE-M3-COND
- removed R65, R68: 47, Resistor_SMD:R_0603_1608Metric
- removed TP27, TP28: SPI MOSI, TestPoint:TestPoint_Pad_1.0x1.0mm
- removed U15: AMS1117-3.3, Package_TO_SOT_SMD:SOT-223-3_TabPin2
- added D11: 3V3, Diode_SMD:D_SOD-323, F.Cu at (237.5, -265.5)
- added D3: 1N4148W, Diode_SMD:D_SOD-123, F.Cu at (-25.1, -85.2)
- added F1: 1A, Fuse:Fuse_0805_2012Metric, F.Cu at (213.1, -257.0)
- added JP3: Jumper_NO_Small, Jumpers:SMT-JUMPER_2_NO_NO-SILK_ROUND, F.Cu at (227.0, -261.9)
- added JP4: Jumper_NO_Small, Jumpers:SMT-JUMPER_2_NO_NO-SILK_ROUND, F.Cu at (227.0, -257.9)
- added L3: 22 Ohm, Resistor_SMD:R_0805_2012Metric, F.Cu at (227.2, -265.5)
- added L4: L_Core_Ferrite_Coupled_Small_GND, custom:MCE1012E900FBP, F.Cu at (-26.3, -78.7)
- added N1: Artwork, custom:draft2, F.Cu at (0.00, 0.00)
- added N2: Badge.team, custom:badgeteam, F.Cu at (-99.1, -15.6)
- added R73: 4.7k, Resistor_SMD:R_0603_1608Metric, F.Cu at (-33.7, -85.7)
- added R74: 100k, Resistor_SMD:R_0603_1608Metric, F.Cu at (245.4, -263.2)
- added X1: Simple_Addon_v2, Simple_Addon_v2:Simple_Addon_v2-BADGE-2x3, F.Cu at (217.9, -262.2)
- added Y2: 32kHz, Crystal:Crystal_SMD_3215-2Pin_3.2x1.5mm, F.Cu at (213.4, -250.1)
- added Y3: 32kHz, Crystal:Crystal_SMD_3215-2Pin_3.2x1.5mm, F.Cu at (237.9, -255.1)
- C24: value 1u -> 100n
- C25, C26: value 1u -> DNP
- D4, D5, D6, D7, D8, D9: value WS2812B -> WS2812B-2020; footprint LED_SMD:LED_WS2812B_PLCC4_5.0x5.0mm_P3.2mm -> custom:ws2812-2020
- R15, R17: value 47 -> 0
- R16, R50, R66, R67: value 47 -> 470
- R51, R52: value 10k -> 4.7k
- moved BT1 340.8 mm to (320.9, -153.2)
- moved C10 340.8 mm to (330.7, -177.2)
- moved C3 340.8 mm to (328.8, -157.8)
- moved C4 340.8 mm to (330.3, -162.5)
- moved C46 340.8 mm to (315.6, -180.9)
- moved C5 340.8 mm to (330.3, -172.8)
- moved R10 340.8 mm to (332.3, -153.7)
- moved R35 340.8 mm to (298.7, -180.8)
- moved R36 340.8 mm to (298.7, -182.2)
- moved R4 340.8 mm to (331.4, -156.6)
- moved RN2 340.8 mm to (323.8, -145.7)
- moved C11 340.8 mm to (332.8, -166.7)
- moved C12 340.8 mm to (332.7, -177.2)
- moved C13 340.8 mm to (328.2, -151.9)
- moved C45 340.8 mm to (312.8, -180.9)
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Connections:
- BT1 pad 2: GND -> 6
- C1 pad 2: GND -> 6
- C10 pad 2: GND -> 6
- C11 pad 2: GND -> 6
- C12 pad 2: GND -> 6
- C13 pad 2: GND -> 6
- C14 pad 2: GND -> 6
- C15 pad 2: GND -> 6
- C16 pad 2: GND -> 6
- C17 pad 2: GND -> 6
- C19 pad 2: GND -> 6
- C2 pad 2: GND -> 6
- C20 pad 2: GND -> 6
- C21 pad 2: GND -> 6
- C22 pad 2: GND -> 6
- C23 pad 2: GND -> 6
- C24 pad 1: PWR_LED -> /ESP32/ESP32_EN
- C24 pad 2: GND -> 6
- C25 pad 1: PWR_LED -> Net-(C25-Pad1)
- C25 pad 2: GND -> 6
- C26 pad 1: PWR_LED -> Net-(C26-Pad1)
- C26 pad 2: GND -> 6
- C27 pad 2: GND -> 6
- C28 pad 2: GND -> 6
- C29 pad 2: GND -> 6
- C3 pad 1: GND -> 6
- C30 pad 2: GND -> 6
- C31 pad 2: GND -> 6
- C32 pad 2: GND -> 6
- C33 pad 2: GND -> 6
- C34 pad 2: GND -> 6
- C35 pad 2: GND -> 6
- C36 pad 2: GND -> 6
- C37 pad 2: GND -> 6
- C38 pad 2: GND -> 6
- C39 pad 2: GND -> 6
- C4 pad 1: VIN -> Net-(C25-Pad1)
- C4 pad 2: GND -> 6
- C40 pad 2: GND -> 6
- C41 pad 2: GND -> 6
- C42 pad 2: GND -> 6
- C43 pad 2: GND -> 6
- C44 pad 2: GND -> 6
- C45 pad 2: GND -> 6
- C46 pad 2: GND -> 6
- C47 pad 2: GND -> 6
- C48 pad 2: GND -> 6
- C49 pad 2: GND -> 6
- C5 pad 1: VIN -> Net-(C26-Pad1)
- C5 pad 2: GND -> 6
- C50 pad 2: GND -> 6
- C6 pad 1: GND -> 6
- C9 pad 2: GND -> 6
- D1 pad 1: /FPGA/RGB2 -> /FPGA/RGB0
- D1 pad 2: /FPGA/RGB1 -> /FPGA/RGB2
- D1 pad 3: /FPGA/RGB0 -> /FPGA/RGB1
- D10 pad 2: GND -> 6
- D10 pad 4: /STM32/USB_D+ -> Net-(D10-Pad4)
- D10 pad 6: /STM32/USB_D- -> Net-(D10-Pad6)
- D4 pad 3: GND -> 6
- D5 pad 3: GND -> 6
- D6 pad 3: GND -> 6
- D7 pad 3: GND -> 6
- D8 pad 3: GND -> 6
- D9 pad 3: GND -> 6
- J1 pad A1: GND -> 6
- J1 pad A12: GND -> 6
- J1 pad A4: VUSB -> Net-(J1-PadA4)
- J1 pad A6: /STM32/USB_D+ -> Net-(D10-Pad4)
- J1 pad A7: /STM32/USB_D- -> Net-(D10-Pad6)
- J1 pad A9: VUSB -> Net-(J1-PadA4)
- J1 pad B1: GND -> 6
- J1 pad B12: GND -> 6
- J1 pad B4: VUSB -> Net-(J1-PadA4)
- J1 pad B6: /STM32/USB_D+ -> Net-(D10-Pad4)
- J1 pad B7: /STM32/USB_D- -> Net-(D10-Pad6)
- J1 pad B9: VUSB -> Net-(J1-PadA4)
- J1 pad S1: GND -> 6
- J2 pad 1: GND -> 6
- J3 pad S: GND -> 6
- J4 pad 1: GND -> 6
- J5 pad 6: GND -> 6
- J5 pad 9: GND -> 6
- J6 pad 11: /FPGA/PMOD_5 -> /FPGA/PMOD_7
- J6 pad 3: GND -> 6
- J6 pad 4: GND -> 6
- J6 pad 5: /FPGA/PMOD_8 -> /FPGA/PMOD_10
- J6 pad 7: /FPGA/PMOD_7 -> /FPGA/PMOD_9
- J6 pad 9: /FPGA/PMOD_6 -> /FPGA/PMOD_8
- J7 pad 16: GND -> 6
- J7 pad 17: GND -> 6
- J7 pad 18: GND -> 6
- J7 pad 19: GND -> 6
- J7 pad 20: GND -> 6
- J7 pad 21: GND -> 6
- J7 pad 22: GND -> 6
- J7 pad 23: GND -> 6
- J7 pad 24: GND -> 6
- J7 pad 37: GND -> 6
- J7 pad 5: GND -> 6
- J8 pad 6: GND -> 6
- Q1 pad 2: GND -> 6
- Q2 pad 2: GND -> 6
- Q3 pad 2: GND -> 6
- Q4 pad 2: GND -> 6
- R1 pad 1: GND -> 6
- R11 pad 1: GND -> 6
- R12 pad 1: GND -> 6
- R13 pad 1: GND -> 6
- R14 pad 2: GND -> 6
- R15 pad 1: ESP_I2S_LR -> Net-(C25-Pad1)
- R15 pad 2: Net-(R15-Pad2) -> VIN
- R16 pad 2: Net-(R15-Pad2) -> ESP_I2S_LR
- R17 pad 1: ESP_I2S_DATA -> Net-(C26-Pad1)
- R17 pad 2: Net-(R17-Pad2) -> VIN
- R2 pad 1: GND -> 6
- R31 pad 1: GND -> 6
- R32 pad 1: GND -> 6
- R35 pad 2: GND -> 6
- R4 pad 2: GND -> 6
- R41 pad 1: GND -> 6
- R46 pad 2: GND -> 6
- R49 pad 1: +3V3 -> ESP_I2S_CLK
- R49 pad 2: /ESP32/EXT_I2C_SDA -> 6
- R5 pad 2: GND -> 6
- R50 pad 2: Net-(R17-Pad2) -> ESP_I2S_DATA
- R54 pad 2: GND -> 6
- R57 pad 1: GND -> 6
- R58 pad 1: GND -> 6
- R6 pad 2: GND -> 6
- R60 pad 2: GND -> 6
- R66 pad 2: Net-(R65-Pad2) -> ESP_I2S_CLK
- R67 pad 1: Net-(R67-Pad1) -> /LED/DATA_IN2
- RN2 pad 2: GND -> 6
- RN2 pad 4: GND -> 6
- RN3 pad 1: GND -> 6
- RN3 pad 2: GND -> 6
- RN3 pad 3: GND -> 6
- RN3 pad 4: GND -> 6
- RN4 pad 1: GND -> 6
- RN4 pad 2: GND -> 6
- RN4 pad 3: GND -> 6
- RN4 pad 4: GND -> 6
- RN5 pad 1: /FPGA/PMOD_6 -> /FPGA/PMOD_7
- RN5 pad 2: /FPGA/PMOD_2 -> /FPGA/PMOD_1
- RN5 pad 3: /FPGA/PMOD_5 -> /FPGA/PMOD_2
- RN5 pad 4: /FPGA/PMOD_1 -> /FPGA/PMOD_8
- RN5 pad 5: Net-(RN5-Pad5) -> /FPGA/PMOD_8i
- RN5 pad 6: Net-(RN5-Pad6) -> /FPGA/PMOD_2i
- RN5 pad 7: Net-(RN5-Pad7) -> /FPGA/PMOD_1i
- RN5 pad 8: Net-(RN5-Pad8) -> /FPGA/PMOD_7i
- RN6 pad 1: Net-(RN6-Pad1) -> /FPGA/PMOD_9
- RN6 pad 2: Net-(RN6-Pad2) -> /FPGA/PMOD_3
- RN6 pad 3: Net-(RN6-Pad3) -> /FPGA/PMOD_10
- RN6 pad 4: Net-(RN6-Pad4) -> /FPGA/PMOD_4
- RN6 pad 5: /FPGA/PMOD_8 -> /FPGA/PMOD_4i
- RN6 pad 6: /FPGA/PMOD_4 -> /FPGA/PMOD_10i
- RN6 pad 7: /FPGA/PMOD_7 -> /FPGA/PMOD_3i
- RN6 pad 8: /FPGA/PMOD_3 -> /FPGA/PMOD_9i
- S1 pad 5: GND -> 6
- S1 pad SH1: GND -> 6
- S1 pad SH2: GND -> 6
- SW2 pad 2: GND -> 6
- SW3 pad 2: GND -> 6
- SW4 pad 2: GND -> 6
- SW5 pad 2: GND -> 6
- SW6 pad 2: GND -> 6
- SW7 pad 2: GND -> 6
- TP20 pad 1: /ESP32/EXT_I2C_SDA -> ESP_I2S_CLK
- TP21 pad 1: /ESP32/EXT_I2C_SCL -> ESP_I2S_DATA
- U1 pad 1: VIN -> Net-(C25-Pad1)
- U1 pad 2: GND -> 6
- U1 pad 4: VIN -> Net-(C25-Pad1)
- U10 pad 1: GND -> 6
- U10 pad 2: Net-(R67-Pad1) -> /LED/DATA_IN2
- U10 pad 3: GND -> 6
- U10 pad 5: VIN -> PWR_LED
- U11 pad 23: GND -> 6
- U11 pad 25: (no net) -> SAO0
- U11 pad 26: (no net) -> SAO1
- U11 pad 35: GND -> 6
- U11 pad 47: GND -> 6
- U11 pad 8: GND -> 6
- U12 pad 12: GND -> 6
- U12 pad 21: GND -> 6
- U13 pad 1: GND -> 6
- U13 pad 10: ESP_I2S_CLK -> /ESP32/EXT_I2C_SCL
- U13 pad 11: ESP_I2S_DATA -> /ESP32/EXT_I2C_SDA
- U13 pad 14: /ESP32/EXT_I2C_SDA -> ESP_I2S_CLK
- U13 pad 15: GND -> 6
- U13 pad 16: /ESP32/EXT_I2C_SCL -> ESP_I2S_DATA
- U13 pad 38: GND -> 6
- U13 pad 39: GND -> 6
- U14 pad 2: GND -> 6
- U16 pad 10: GND -> 6
- U16 pad 15: GND -> 6
- U16 pad 16: GND -> 6
- U16 pad 17: GND -> 6
- U16 pad 18: GND -> 6
- U16 pad 2: GND -> 6
- U16 pad 25: GND -> 6
- U16 pad 5: GND -> 6
- U16 pad 6: GND -> 6
- U17 pad 1: GND -> 6
- U17 pad 7: GND -> 6
- U2 pad 1: VIN -> Net-(C26-Pad1)
- U2 pad 2: GND -> 6
- U2 pad 4: VIN -> Net-(C26-Pad1)
- U3 pad 2: GND -> 6
- U4 pad 2: GND -> 6
- U5 pad 2: GND -> 6
- U6 pad 10: GND -> 6
- U6 pad 11: GND -> 6
- U6 pad 12: GND -> 6
- U6 pad 13: Net-(R65-Pad2) -> ESP_I2S_CLK
- U6 pad 14: Net-(R17-Pad2) -> ESP_I2S_DATA
- U6 pad 15: Net-(R15-Pad2) -> ESP_I2S_LR
- U6 pad 16: GND -> 6
- U6 pad 19: GND -> 6
- U6 pad 3: GND -> 6
- U6 pad 9: GND -> 6
- U7 pad 3: GND -> 6
- U8 pad 12: SPIRAM_D1 -> SPIRAM_D2
- U8 pad 13: SPIRAM_CS -> SPIRAM_D1
- U8 pad 18: SPIRAM_D2 -> SPIRAM_CS
- U8 pad 19: SPIRAM_D0 -> SPIRAM_SCK
- U8 pad 2: Net-(RN5-Pad7) -> /FPGA/PMOD_4i
- U8 pad 20: SPIRAM_SCK -> SPIRAM_D3
- U8 pad 21: SPIRAM_D3 -> SPIRAM_D0
- U8 pad 28: /FPGA/LCD_D2 -> FPGA_I2S_CLK
- U8 pad 3: Net-(RN5-Pad6) -> /FPGA/PMOD_9i
- U8 pad 31: /FPGA/LCD_D3 -> /FPGA/LCD_D2
- U8 pad 32: /FPGA/LCD_D4 -> /FPGA/LCD_D3
- U8 pad 34: /FPGA/LCD_D5 -> /FPGA/LCD_D4
- U8 pad 35: /FPGA/LCD_D6 -> /FPGA/CLK
- U8 pad 36: /FPGA/LCD_D7 -> FPGA_I2S_DATA
- U8 pad 37: /FPGA/CLK -> /FPGA/LCD_D5
- U8 pad 38: FPGA_I2S_CLK -> /FPGA/LCD_D6
- U8 pad 4: Net-(RN5-Pad5) -> /FPGA/PMOD_3i
- U8 pad 42: FPGA_I2S_LR -> /FPGA/LCD_D7
- U8 pad 43: FPGA_I2S_DATA -> FPGA_I2S_LR
- U8 pad 44: Net-(RN6-Pad4) -> /FPGA/PMOD_7i
- U8 pad 45: Net-(RN6-Pad3) -> /FPGA/PMOD_8i
- U8 pad 46: Net-(RN6-Pad2) -> /FPGA/PMOD_10i
- U8 pad 47: Net-(RN6-Pad1) -> /FPGA/PMOD_1i
- U8 pad 48: Net-(RN5-Pad8) -> /FPGA/PMOD_2i
- U8 pad 49: GND -> 6
- U9 pad 4: GND -> 6
- Y1 pad 2: GND -> 6
- Y1 pad 4: GND -> 6
Routing:
- net GND: track 265.0 -> 11.0 mm, vias 102 -> 27
- net 6: track 0.00 -> 231.2 mm, vias 0 -> 59
- net /ESP32/SPI_MOSI: track 246.3 -> 31.3 mm, vias 8 -> 3
- net VIN: track 209.5 -> 39.1 mm, vias 6 -> 5
- net VUSB: track 220.6 -> 61.9 mm, vias 6 -> 5
- net /ESP32/SPI_CLK: track 155.9 -> 31.1 mm, vias 6 -> 2
- net /FPGA/SPI_CS: track 137.6 -> 13.0 mm, vias 4 -> 2
- net /LCD/LCD_WR_RS: track 132.0 -> 17.5 mm
- net /FPGA/IRQ: track 108.1 -> 2.19 mm, vias 2 -> 0
- net /ESP32/SPI_MISO: track 128.1 -> 25.0 mm, vias 4 -> 2
- net /STM32/FPGA_RX: track 107.4 -> 5.04 mm, vias 5 -> 0
- net /STM32/FPGA_TX: track 100.5 -> 2.13 mm, vias 5 -> 0
- net /LCD/CS: track 98.2 -> 1.73 mm, vias 2 -> 0
- net /POWER/SENSE_VBAT: track 148.1 -> 59.7 mm, vias 4 -> 2
- net /FPGA/CLK: track 89.9 -> 2.63 mm, vias 5 -> 0
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- added copper zone on B.Cu, net 6
- added copper zone on In1.Cu, net 6
- removed copper zone on F.Cu, net GND
- removed copper zone on In1.Cu, net GND
Other:
- board size 100 x 100 mm -> 253.2 x 64.2 mm
