File: mch2021.kicad_pcb (KiCad board)
At the start: 4 copper layers, 253.2 x 64.2 mm, 219 parts, among them J1 USB_C_Receptacle_USB2.0, J2 QWIIC_CONNECTORJS-1MM, J3 AudioJack3, J4 QWIIC_CONNECTORJS-1MM, J5 Micro SD card, J6 PMOD, J7 LCD, J8 GPIO, Q1 Q_NMOS_GSD, Q2 Q_NMOS_GSD, Q3 Q_NMOS_GSD, Q4 Q_NMOS_GSD, SW1 Power switch, SW2 Start, SW3 Select, SW4 Menu, SW5 Home, SW6 Back, SW7 Accept, U1 SY8079AAC, U10 74LVC1G125, U11 STM32F103C8Tx, U12 PCA9555PW, U13 ESP32-WROVER, U14 SY6280AAC, U16 BNO055, U17 BME680, U2 SY8079AAC, U3 XT4054K421MR-G, U4 SY6280AAC, U5 SY6280AAC, U6 PCM5100, U7 74LVC1G125, U8 ICE40UP5K-SG48ITR, U9 LY68L6400, X1 Simple_Addon_v2, Y1 16MHz, Y2 32kHz, Y3 32kHz

Commit message: Update artwork
Parts:
- C23: moved to B.Cu
- D4, D5, D6, D7, D8, D9: value WS2812B-2020 -> SK6812-EC15; footprint custom:ws2812-2020 -> LED_SMD:LED_SK6812_EC15_1.5x1.5mm
- N1: footprint custom:draft2 -> custom:draft2_renze
- moved C33 410.3 mm to (-216.4, 8.73)
- moved Y3 377.8 mm to (-102.1, -90.4), turned to 180 degrees
- moved J6 287.1 mm to (-59.8, 20.7), turned to 0 degrees
- moved D7 229.8 mm to (-49.7, -39.5)
- moved D8 223.7 mm to (-33.4, -41.4)
- moved D5 217.3 mm to (-40.4, -25.6)
- moved D6 216.4 mm to (-37.1, -33.6)
- moved C23 183.1 mm to (-8.50, -83.5), turned to 180 degrees
- moved D9 176.4 mm to (3.15, -85.3)
- moved X1 148.2 mm to (80.0, -208.1)
- moved C49 70.5 mm to (-105.8, -91.2), turned to 90 degrees
- moved U16 60.4 mm to (-103.0, -97.1), turned to 180 degrees
- moved C48 58.5 mm to (-98.1, -91.4), turned to 90 degrees
- moved N2 46.1 mm to (-142.3, -31.9)
- moved D4 40.3 mm to (-17.1, -25.6), turned to 0 degrees
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Connections:
- BT1 pad 2: 6 -> GND
- C1 pad 2: 6 -> GND
- C10 pad 2: 6 -> GND
- C11 pad 2: 6 -> GND
- C12 pad 2: 6 -> GND
- C13 pad 2: 6 -> GND
- C14 pad 2: 6 -> GND
- C15 pad 2: 6 -> GND
- C16 pad 2: 6 -> GND
- C17 pad 2: 6 -> GND
- C19 pad 2: 6 -> GND
- C2 pad 2: 6 -> GND
- C20 pad 2: 6 -> GND
- C21 pad 2: 6 -> GND
- C22 pad 2: 6 -> GND
- C23 pad 2: 6 -> GND
- C24 pad 2: 6 -> GND
- C25 pad 2: 6 -> GND
- C26 pad 2: 6 -> GND
- C27 pad 2: 6 -> GND
- C28 pad 2: 6 -> GND
- C29 pad 2: 6 -> GND
- C3 pad 1: 6 -> GND
- C30 pad 2: 6 -> GND
- C31 pad 2: 6 -> GND
- C32 pad 2: 6 -> GND
- C33 pad 2: 6 -> GND
- C34 pad 2: 6 -> GND
- C35 pad 2: 6 -> GND
- C36 pad 2: 6 -> GND
- C37 pad 2: 6 -> GND
- C38 pad 2: 6 -> GND
- C39 pad 2: 6 -> GND
- C4 pad 2: 6 -> GND
- C40 pad 2: 6 -> GND
- C41 pad 2: 6 -> GND
- C42 pad 2: 6 -> GND
- C43 pad 2: 6 -> GND
- C44 pad 2: 6 -> GND
- C45 pad 2: 6 -> GND
- C46 pad 2: 6 -> GND
- C47 pad 2: 6 -> GND
- C48 pad 2: 6 -> GND
- C49 pad 2: 6 -> GND
- C5 pad 2: 6 -> GND
- C50 pad 2: 6 -> GND
- C6 pad 1: 6 -> GND
- C9 pad 2: 6 -> GND
- D10 pad 2: 6 -> GND
- D11 pad 2: 6 -> GND
- D4 pad 3: 6 -> GND
- D5 pad 3: 6 -> GND
- D6 pad 3: 6 -> GND
- D7 pad 3: 6 -> GND
- D8 pad 3: 6 -> GND
- D9 pad 3: 6 -> GND
- J1 pad A1: 6 -> GND
- J1 pad A12: 6 -> GND
- J1 pad B1: 6 -> GND
- J1 pad B12: 6 -> GND
- J1 pad S1: 6 -> GND
- J2 pad 1: 6 -> GND
- J3 pad S: 6 -> GND
- J4 pad 1: 6 -> GND
- J5 pad 6: 6 -> GND
- J5 pad 9: 6 -> GND
- J6 pad 3: 6 -> GND
- J6 pad 4: 6 -> GND
- J7 pad 16: 6 -> GND
- J7 pad 17: 6 -> GND
- J7 pad 18: 6 -> GND
- J7 pad 19: 6 -> GND
- J7 pad 20: 6 -> GND
- J7 pad 21: 6 -> GND
- J7 pad 22: 6 -> GND
- J7 pad 23: 6 -> GND
- J7 pad 24: 6 -> GND
- J7 pad 37: 6 -> GND
- J7 pad 5: 6 -> GND
- J8 pad 6: 6 -> GND
- L4 pad 5: 6 -> GND
- L4 pad 6: 6 -> GND
- Q1 pad 2: 6 -> GND
- Q2 pad 2: 6 -> GND
- Q3 pad 2: 6 -> GND
- Q4 pad 2: 6 -> GND
- R1 pad 1: 6 -> GND
- R11 pad 1: 6 -> GND
- R12 pad 1: 6 -> GND
- R13 pad 1: 6 -> GND
- R14 pad 2: 6 -> GND
- R2 pad 1: 6 -> GND
- R31 pad 1: 6 -> GND
- R32 pad 1: 6 -> GND
- R35 pad 2: 6 -> GND
- R4 pad 2: 6 -> GND
- R41 pad 1: 6 -> GND
- R46 pad 2: 6 -> GND
- R49 pad 2: 6 -> GND
- R5 pad 2: 6 -> GND
- R54 pad 2: 6 -> GND
- R57 pad 1: 6 -> GND
- R58 pad 1: 6 -> GND
- R6 pad 2: 6 -> GND
- R60 pad 2: 6 -> GND
- RN2 pad 2: 6 -> GND
- RN2 pad 4: 6 -> GND
- RN3 pad 1: 6 -> GND
- RN3 pad 2: 6 -> GND
- RN3 pad 3: 6 -> GND
- RN3 pad 4: 6 -> GND
- RN4 pad 1: 6 -> GND
- RN4 pad 2: 6 -> GND
- RN4 pad 3: 6 -> GND
- RN4 pad 4: 6 -> GND
- S1 pad 5: 6 -> GND
- S1 pad SH1: 6 -> GND
- S1 pad SH2: 6 -> GND
- SW2 pad 2: 6 -> GND
- SW3 pad 2: 6 -> GND
- SW4 pad 2: 6 -> GND
- SW5 pad 2: 6 -> GND
- SW6 pad 2: 6 -> GND
- SW7 pad 2: 6 -> GND
- U1 pad 2: 6 -> GND
- U10 pad 1: 6 -> GND
- U10 pad 3: 6 -> GND
- U11 pad 23: 6 -> GND
- U11 pad 35: 6 -> GND
- U11 pad 47: 6 -> GND
- U11 pad 8: 6 -> GND
- U12 pad 12: 6 -> GND
- U12 pad 21: 6 -> GND
- U13 pad 1: 6 -> GND
- U13 pad 15: 6 -> GND
- U13 pad 38: 6 -> GND
- U13 pad 39: 6 -> GND
- U14 pad 2: 6 -> GND
- U16 pad 10: 6 -> GND
- U16 pad 15: 6 -> GND
- U16 pad 16: 6 -> GND
- U16 pad 17: 6 -> GND
- U16 pad 18: 6 -> GND
- U16 pad 2: 6 -> GND
- U16 pad 25: 6 -> GND
- U16 pad 5: 6 -> GND
- U16 pad 6: 6 -> GND
- U17 pad 1: 6 -> GND
- U17 pad 7: 6 -> GND
- U2 pad 2: 6 -> GND
- U3 pad 2: 6 -> GND
- U4 pad 2: 6 -> GND
- U5 pad 2: 6 -> GND
- U6 pad 10: 6 -> GND
- U6 pad 11: 6 -> GND
- U6 pad 12: 6 -> GND
- U6 pad 16: 6 -> GND
- U6 pad 19: 6 -> GND
- U6 pad 3: 6 -> GND
- U6 pad 9: 6 -> GND
- U7 pad 3: 6 -> GND
- U8 pad 49: 6 -> GND
- U9 pad 4: 6 -> GND
- X1 pad 2: 6 -> GND
- Y1 pad 2: 6 -> GND
- Y1 pad 4: 6 -> GND
Routing:
- net 6: track 231.2 -> 11.1 mm, vias 59 -> 1
- net GND: track 11.0 -> 210.1 mm, vias 27 -> 76
- net PWR_LED: track 57.8 -> 2.80 mm, vias 3 -> 0
- net Net-(D8-Pad2): track 17.4 -> 0.00 mm
- net Net-(D6-Pad2): track 10.9 -> 0.00 mm, vias 2 -> 0
- net FPGA_I2S_LR: track 5.73 -> 0.00 mm, vias 1 -> 0
- net /LED/DATA_OUT: track 3.18 -> 0.00 mm
- net VIN: track 39.1 -> 37.3 mm
- added copper zone on B.Cu, net GND
- added copper zone on In1.Cu, net GND
- removed copper zone on B.Cu, net 6
- removed copper zone on In1.Cu, net 6

Commit message: First steps of routing prototype 2, switch to 0402 for most passives
Parts:
- removed N1: Artwork, custom:draft2_renze
- removed R21, R22, R23, R24: 47, Resistor_SMD:R_0603_1608Metric
- added RN1: 47, Resistor_SMD:R_Array_Convex_4x0603, B.Cu at (28.8, -9.17)
- C1, C13, C14, C2, C21, C22, C23, C24, C25, C26, C3, C31, C32, C33, C34, C36, C37, C38, C39, C40, C41, C43, C44, C45, C46, C47, C50, C6, C7, C8: footprint Capacitor_SMD:C_0603_1608Metric -> Capacitor_SMD:C_0402_1005Metric
- C27, C28, C29, C35, C42, C48, C49: footprint Capacitor_SMD:C_0603_1608Metric -> Capacitor_SMD:C_0402_1005Metric; moved to B.Cu
- N2, U12, U16, U17, U6, Y3: moved to B.Cu
- R1, R10, R11, R12, R13, R14, R15, R17, R18, R19, R2, R20, R25, R26, R27, R28, R29, R3, R30, R31, R32, R33, R35, R36, R37, R38, R39, R4, R40, R41, R42, R43, R44, R46, R47, R48, R49, R5, R50, R51, R52, R53, R55, R56, R57, R58, R59, R6, R60, R61, R62, R63, R64, R66, R67, R69, R7, R70, R71, R72, R73, R74, R8, R9: footprint Resistor_SMD:R_0603_1608Metric -> Resistor_SMD:R_0402_1005Metric
- R16: footprint Resistor_SMD:R_0603_1608Metric -> Resistor_SMD:R_0402_1005Metric; moved to B.Cu
- R34: value 100 -> 47; footprint Resistor_SMD:R_0603_1608Metric -> Resistor_SMD:R_0402_1005Metric; moved to B.Cu
- R45: footprint Resistor_SMD:R_0603_1608Metric -> Resistor_SMD:R_0402_1005Metric; moved to F.Cu
- R54: value 10k -> 100k; footprint Resistor_SMD:R_0603_1608Metric -> Resistor_SMD:R_0402_1005Metric
- moved SW1 411.2 mm to (-19.7, 44.0), turned to 180 degrees
- moved R10 408.7 mm to (-27.6, 39.9), turned to 270 degrees
- moved R4 406.3 mm to (-24.7, 39.0), turned to 0 degrees
- moved C11 404.4 mm to (-14.7, 40.4), turned to 180 degrees
- moved C13 403.8 mm to (-29.4, 35.8), turned to 270 degrees
- moved U3 403.6 mm to (-26.5, 36.5), turned to 0 degrees
- moved C4 402.6 mm to (-18.8, 38.0), turned to 0 degrees
- moved C3 402.3 mm to (-23.5, 36.5), turned to 90 degrees
- moved C9 401.3 mm to (-14.7, 38.1), turned to 180 degrees
- moved RN2 400.7 mm to (-35.6, 31.4), turned to 0 degrees
- moved C7 398.0 mm to (-20.7, 34.0), turned to 0 degrees
- moved R8 395.5 mm to (-20.7, 32.2), turned to 0 degrees
- moved BT1 393.5 mm to (-28.1, 28.5), turned to 0 degrees
- moved C12 336.8 mm to (78.7, 44.0), turned to 180 degrees
- moved C5 333.9 mm to (74.3, 41.5), turned to 0 degrees
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Connections:
- net Net-(C28-Pad1) renamed /FPGA/VCCPLL
Routing:
- net /POWER/SENSE_VUSB: track 62.3 -> 2.60 mm, vias 2 -> 1
- net /POWER/SENSE_VBAT: track 59.7 -> 0.80 mm, vias 2 -> 0
- net GND: track 210.1 -> 173.4 mm, vias 76 -> 51
- net /STM32/LCD_MODE: track 34.9 -> 0.00 mm, vias 2 -> 0
- net /ESP32/SPI_MOSI: track 31.3 -> 0.00 mm, vias 3 -> 0
- net /ESP32/SPI_CLK: track 31.1 -> 0.00 mm, vias 2 -> 0
- net /FPGA/LCD_D6: track 51.7 -> 22.0 mm
- net +3V3: track 107.5 -> 78.8 mm, vias 22 -> 17
- net /FPGA/VCCPLL: track 30.0 -> 2.00 mm, vias 1 -> 0
- net /ESP32/EXT_I2C_SCL: track 27.6 -> 0.00 mm
- net /ESP32/SD_CLK: track 26.8 -> 0.00 mm
- net /ESP32/EXT_I2C_SDA: track 26.8 -> 0.00 mm
- net ESP_I2S_LR: track 26.7 -> 0.00 mm
- net /ESP32/SD_D0: track 30.5 -> 3.72 mm
- net /ESP32/SD_CMD: track 31.9 -> 5.14 mm
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Other:
- board size 253.2 x 64.2 mm -> 5 x 28.7 mm
- rule via_min_drill: 0.3 -> 0.2
- rule via_min_size: 0.4 -> 0.45

Commit message: More routing...
Parts:
- added N1: Artwork, custom:vector4, F.Cu at (0.00, 0.00)
- C21, C26, C31, C47, L1, R14, R17, R70, R71, R72, U1, U10, U5: moved to B.Cu
- moved R17 324.0 mm to (157.0, 46.0), turned to 180 degrees
- moved C26 322.4 mm to (159.0, 46.0)
- moved U1 284.0 mm to (176.0, 40.3), turned to 180 degrees
- moved L1 268.4 mm to (179.4, 41.2), turned to 180 degrees
- moved R53 247.4 mm to (12.3, -28.5)
- moved R66 247.4 mm to (12.3, -31.0)
- moved R33 242.2 mm to (9.18, -14.8)
- moved C11 193.0 mm to (178.3, 45.6)
- moved C4 193.0 mm to (174.1, 43.2)
- moved C9 193.0 mm to (178.2, 43.3)
- moved C7 193.0 mm to (172.2, 39.3)
- moved R8 193.0 mm to (172.2, 37.4)
- moved C31 123.5 mm to (-4.17, 12.4), turned to 270 degrees
- moved R70 121.9 mm to (-0.50, 8.50)
- moved R71 120.8 mm to (-5.39, 11.3), turned to 90 degrees
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Connections:
- net Net-(C26-Pad1) renamed /POWER/1V2REG_VIN
- net Net-(C47-Pad1) renamed /BOSCH/BNO055_CAP
- net Net-(C48-Pad1) renamed /BOSCH/BNO055_XIN32
- net Net-(C49-Pad1) renamed /BOSCH/BNO055_XOUT32
Routing:
- net VUSB: track 61.9 -> 0.00 mm, vias 5 -> 0
- net GND: track 173.4 -> 139.8 mm, vias 51 -> 42
- net SPIRAM_D2: track 0.00 -> 21.5 mm
- net Net-(R55-Pad1): track 21.2 -> 0.00 mm, vias 2 -> 0
- net VBAT: track 20.6 -> 0.00 mm
- net SPIRAM_D1: track 0.00 -> 19.7 mm
- net /POWER/PWR_LED_ENABLE: track 19.4 -> 0.00 mm, vias 1 -> 0
- net Net-(U10-Pad2): track 18.2 -> 0.00 mm, vias 2 -> 0
- net /STM32/USB_D+: track 18.2 -> 0.00 mm
- net /STM32/USB_D-: track 18.0 -> 0.00 mm
- net VIN: track 19.4 -> 1.65 mm, vias 2 -> 1
- net SPIRAM_CS: track 0.00 -> 16.0 mm
- net /BUTTONS/STM32_RESET: track 11.9 -> 0.00 mm, vias 2 -> 0
- net SPIRAM_SCK: track 0.00 -> 11.6 mm
- net +3V3: track 78.8 -> 67.3 mm, vias 17 -> 13
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Other:
- board size 5 x 28.7 mm -> 144.8 x 94.3 mm
