File: stm32.sch (KiCad schematic (older format))
At the start: 16 parts

Commit message: Finished work on initial schematic
Parts:
- added R27: 10k, Resistor_SMD:R_0603_1608Metric, symbol Device:R
- gave numbers to parts that had none: 7
- renumbered C18 to C23, C1 to C24, C19 to C25, C20 to C26, C21 to C27, R27 to R29, R25 to R30
Connections:
- net FPGA_CTS is gone; now on net SENSE_VBAT: U11.10 (PA0)
- net +3V3: now also R27.2
- net IRQ: now also U11.18 (PB0), R27.1; no longer R26.2, U11.29 (PA8)
- net SENSE_VBAT: no longer U11.18 (PB0)
- net SENSE_VUSB: now also U11.11 (PA1); no longer U11.19 (PB1)
- net at U11.22 (PB11): now also U10.2, U11.28 (PB15)
- net LCD_MODE: now reaches U11.41 (PB5)
- net STM32_JNTRST renamed LCD_RESET
- net STM32_JTCK: no longer names the net of J7.2 (Pin_2), U11.37 (PA14)
- net STM32_JTDI: no longer names the net of U11.38 (PA15)
- net STM32_JTDO renamed LCD_ENABLE_PAR
- net STM32_JTMS: no longer names the net of J7.1 (Pin_1), U11.34 (PA13)
- new net LCD_BACKLIGHT: U11.19 (PB1)
- new net MCO: U11.29 (PA8)
Other:
- moved on the sheet: J7, R26

Commit message: Small fixes
Parts:
- removed R26: 10k, Resistor_SMD:R_0603_1608Metric, symbol Device:R
Other:
- note added: "if using hardware time and the aproach of DMA > TIMer Output\ncompare register you will need bridge pb15 and pb11 so we can\nselect or spi or tim"
Changed lines of the file:
@@
 $Descr A4 11693 8268
 encoding utf-8
-Sheet 7 10
+Sheet 6 10
 Title "MCH2021 badge - STM32 microcontroller"
 Date "2020-08-08"
@@
 Text HLabel 2700 3500 0    50   Output ~ 0
 IRQ
-$Comp
-L Device:R R?
-U 1 1 5FB3552C
-P 1400 2100
-AR Path="/5DC753C3/5FB3552C" Ref="R?"  Part="1"
-AR Path="/5FB3552C" Ref="R?"  Part="1"
-AR Path="/5E3BA64A/5FB3552C" Ref="R?"  Part="1"
-AR Path="/5F51E414/5FB3552C" Ref="R26"  Part="1"
-F 0 "R26" V 1300 2100 50  0000 C CNN
-F 1 "10k" V 1400 2100 50  0000 C CNN
-F 2 "Resistor_SMD:R_0603_1608Metric" V 1330 2100 50  0001 C CNN
-F 3 "~" H 1400 2100 50  0001 C CNN
-F 4 "C25804" H 1400 2100 50  0001 C CNN "LCSC"
-	1    1400 2100
-	1    0    0    -1
-$EndComp
-$Comp
-L power:+3.3V #PWR0101
-U 1 1 5FB36090
-P 1400 1950
-F 0 "#PWR0101" H 1400 1800 50  0001 C CNN
-F 1 "+3.3V" H 1415 2123 50  0000 C CNN
-F 2 "" H 1400 1950 50  0001 C CNN
-F 3 "" H 1400 1950 50  0001 C CNN
-	1    1400 1950
-	1    0    0    -1
-$EndComp
 Text HLabel 8050 3500 2    50   Input ~ 0
 SENSE_VBAT
@@
 Text HLabel 8050 4300 2    50   Output ~ 0
 MCO
+Text Notes 700  7650 0    79   ~ 0
+if using hardware time and the aproach of DMA > TIMer Output\ncompare register you will need bridge pb15 and pb11 so we can\nselect or spi or tim
 $EndSCHEMATC

Commit message: Fixes, removed I2S DAC
Parts:
- removed R27: 10k, Resistor_SMD:R_0603_1608Metric, symbol Device:R
Connections:
- net FPGA_RESET: now reaches U11.21 (PB10)
- net FPGA_CDONE: now reaches U11.25 (PB12)
- net IRQ: no longer names the net of U11.18 (PB0)
Other:
- note added: "The ESP32 BL pin also serves as IRQ"
Changed lines of the file:
@@
 $Descr A4 11693 8268
 encoding utf-8
-Sheet 6 10
+Sheet 6 9
 Title "MCH2021 badge - STM32 microcontroller"
 Date "2020-08-08"
@@
 Wire Wire Line
 	6650 4800 8050 4800
-Text HLabel 2700 3500 0    50   Output ~ 0
-IRQ
 Text HLabel 8050 3500 2    50   Input ~ 0
 SENSE_VBAT
@@
 Wire Wire Line
 	6650 4300 8050 4300
-$Comp
-L Device:R R?
-U 1 1 60D92E94
-P 3450 2200
-AR Path="/5DC753C3/60D92E94" Ref="R?"  Part="1"
-AR Path="/60D92E94" Ref="R?"  Part="1"
-AR Path="/5E3BA64A/60D92E94" Ref="R?"  Part="1"
-AR Path="/5F51E414/60D92E94" Ref="R27"  Part="1"
-F 0 "R27" V 3550 2200 50  0000 C CNN
-F 1 "10k" V 3450 2200 50  0000 C CNN
-F 2 "Resistor_SMD:R_0603_1608Metric" V 3380 2200 50  0001 C CNN
-F 3 "~" H 3450 2200 50  0001 C CNN
-F 4 "C25804" H 3450 2200 50  0001 C CNN "LCSC"
-	1    3450 2200
-	-1   0    0    1
-$EndComp
-$Comp
-L power:+3.3V #PWR0104
-U 1 1 60D92E9A
-P 3450 2050
-F 0 "#PWR0104" H 3450 1900 50  0001 C CNN
-F 1 "+3.3V" H 3465 2223 50  0000 C CNN
-F 2 "" H 3450 2050 50  0001 C CNN
-F 3 "" H 3450 2050 50  0001 C CNN
-	1    3450 2050
-	1    0    0    -1
-$EndComp
-Wire Wire Line
-	2700 3500 3450 3500
-Wire Wire Line
-	3450 2350 3450 3500
-Connection ~ 3450 3500
-Wire Wire Line
-	3450 3500 5350 3500
 Text HLabel 8050 4300 2    50   Output ~ 0
 MCO
 Text Notes 700  7650 0    79   ~ 0
 if using hardware time and the aproach of DMA > TIMer Output\ncompare register you will need bridge pb15 and pb11 so we can\nselect or spi or tim
+Text HLabel 2700 4500 0    50   Output ~ 0
+FPGA_RESET
+Text HLabel 2700 4600 0    50   Input ~ 0
+FPGA_CDONE
+Wire Wire Line
+	2700 4500 5350 4500
+Wire Wire Line
+	5350 4700 5200 4700
+Wire Wire Line
+	5200 4700 5200 4600
+Wire Wire Line
+	5200 4600 2700 4600
+Text Notes 750  3200 0    50   ~ 0
+The ESP32 BL pin also serves as IRQ
 $EndSCHEMATC

Commit message: Dump.
Parts:
- removed R29, R30: 10k, Resistor_SMD:R_0603_1608Metric, symbol Device:R
- added J9: GPIO, Connector_PinHeader_2.54mm:PinHeader_1x04_P2.54mm_Vertical, symbol Connector:Conn_01x04_Male
- added R34: 10k, Resistor_SMD:R_0603_1608Metric, symbol Device:R
- C43: renamed from C23; value 20pF -> 20p; LCSC C1648 -> (none); Price (none) -> 0.0020; Sponsored (none) -> N
- C44: renamed from C24; value 20pF -> 20p; LCSC C1648 -> (none); Price (none) -> 0.0020; Sponsored (none) -> N
- C45: renamed from C25; value 100nF -> 100n; Mouser (none) -> -; Price (none) -> 0.0020; Sponsored (none) -> N
- C46: renamed from C26; value 100nF -> 100n; Mouser (none) -> -; Price (none) -> 0.0020; Sponsored (none) -> N
- C47: renamed from C27; value 100nF -> 100n; Mouser (none) -> -; Price (none) -> 0.0020; Sponsored (none) -> N
- J8: renamed from J7; LCSC (none) -> -; Mouser (none) -> -; Price (none) -> 0; Sponsored (none) -> -
- R32: renamed from R28; LCSC C25804 -> -; Mouser (none) -> -; Price (none) -> 0.0005; Sponsored (none) -> N
- R33: LCSC C25804 -> -; Mouser (none) -> -; Price (none) -> 0.0005; Sponsored (none) -> N
- R35: renamed from R31; LCSC C25804 -> -; Mouser (none) -> -; Price (none) -> 0.0005; Sponsored (none) -> N
- R36: renamed from R32; LCSC C25804 -> -; Mouser (none) -> -; Price (none) -> 0.0005; Sponsored (none) -> N
- U13: renamed from U10; footprint (none) -> Package_TO_SOT_SMD:SOT-353_SC-70-5; LCSC (none) -> C703585; Mouser (none) -> -; Price (none) -> 0.020; Sponsored (none) -> N
- U14: renamed from U11; Mouser (none) -> -; Price (none) -> 0.97; Sponsored (none) -> N
- Y1: Mouser (none) -> -; Price (none) -> 0.045; Sponsored (none) -> N
Connections:
- net labels added: FPGA_CS, LCD_CS, SPI_CS_A, SPI_CS_B, SPK
- net labels removed: FPGA_CDONE, FPGA_RESET, SPI_CS_STM32
- wire segments 88 -> 95
- no-connect marks 1 -> 0
Other:
- note added: "SPI DEVICE SELECTION\n\nP: LCD_ENABLE_PAR input from the FPGA\nA: input from the ESP32 (1)\nB: input from the ESP32 (2)\nL: LCD CS output\nF: FPGA CS output\n\nPAB LF Description\n----\n000 11 None\n001 11 STM32 selected\n010 01 LCD selected\n011 10 FPGA selected\n100 01 None\n101 01 STM32 selected\n110 01 None\n111 00 FPGA selected\n\nNote:\nWhen LCD is in parallel mode the LCD\nchip-select pin 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"

Commit message: Dump.
Parts:
- removed J8: PROG, Connector:Tag-Connect_TC2030-IDC-NL_2x03_P1.27mm_Vertical, symbol Connector_Generic:Conn_01x06
- removed U13: 74LVC1G125, Package_TO_SOT_SMD:SOT-353_SC-70-5, symbol 74xGxx:74LVC1G125
- added U10: SN74LVC1G125DCKR, digikey-footprints:SOT-353, symbol dk_Logic-Buffers-Drivers-Receivers-Transceivers:SN74LVC1G125DCKR
- J8: renamed from J9; footprint Connector_PinHeader_2.54mm:PinHeader_1x04_P2.54mm_Vertical -> Connector_PinHeader_2.54mm:PinHeader_1x06_P2.54mm_Vertical; symbol Connector:Conn_01x04_Male -> Connector_Generic:Conn_01x06
- renumbered C43 to C37, C44 to C38, C45 to C39, C46 to C40, C47 to C41, R32 to R29, R33 to R30, R34 to R31, R35 to R32, R36 to R33, U14 to U11
Connections:
- net labels added: VIN
- net labels removed: CHARGING, VBAT
- wire segments 95 -> 106

Commit message: Dump.
Parts:
- removed R30, R31: 10k, Resistor_SMD:R_0603_1608Metric, symbol Device:R
- added R44: 100k, Resistor_SMD:R_0603_1608Metric, symbol Device:R
- renumbered R29 to R41, R32 to R42, R33 to R43
Connections:
- net SPI_CS_A is gone; now on net SAO_IO1: U11.20 (PB2)
- net +3V3: now also R44.1
- net ESP32_RX: now also U11.12 (PA2); no longer U11.30 (PA9)
- net ESP32_TX: now also U11.13 (PA3); no longer U11.31 (PA10)
- net FPGA_RX: now also U11.30 (PA9); no longer U11.12 (PA2)
- net FPGA_TX: now also U11.31 (PA10); no longer U11.13 (PA3)
- net LCD_ENABLE_PAR: now also U11.45 (PB8); no longer U11.26 (PB13)
- net SAO_IO0: now also U11.21 (PB10); no longer U11.45 (PB8)
- net SAO_IO1: no longer U11.46 (PB9)
- net at J8.2 (Pin_2): now also U11.26 (PB13); no longer U11.21 (PB10)
- net FPGA_CS renamed SPI_CS
- net SPI_CS: now also R44.2
- net LCD_CS: no longer names the net of U11.4 (PC15)
- net SPI_CS_B: no longer names the net of U11.39 (PB3)
Other:
- note removed: "SPI DEVICE SELECTION\n\nP: LCD_ENABLE_PAR input from the FPGA\nA: input from the ESP32 (1)\nB: input from the ESP32 (2)\nL: LCD CS output\nF: FPGA CS output\n\nPAB LF Description\n----\n000 11 None\n001 11 STM32 selected\n010 01 LCD selected\n011 10 FPGA selected\n100 01 None\n101 01 STM32 selected\n110 01 None\n111 00 FPGA selected\n\nNote:\nWhen LCD is in parallel mode the LCD\nchip-select pin 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"

Commit message: Dump.
Connections:
- net LCD_BACKLIGHT: now also U11.46 (PB9); no longer U11.19 (PB1)
- net SENSE_VBAT: now also U11.11 (PA1); no longer U11.10 (PA0)
- net SENSE_VUSB: now also U11.10 (PA0); no longer U11.11 (PA1)
- net SAO_IO3: now reaches U11.18 (PB0)
- new net SAO_IO2: U11.19 (PB1)
Changed lines of the file:
@@
 $Descr A4 11693 8268
 encoding utf-8
-Sheet 7 9
+Sheet 6 9
 Title "MCH2021 badge - STM32 microcontroller"
 Date "2020-08-08"
@@
 Wire Wire Line
 	6650 4800 7100 4800
+Text HLabel 8050 3600 2    50   Input ~ 0
+SENSE_VBAT
 Text HLabel 8050 3500 2    50   Input ~ 0
-SENSE_VBAT
-Text HLabel 8050 3600 2    50   Input ~ 0
 SENSE_VUSB
 Wire Wire Line
@@
 	5350 4000 2700 4000
 Wire Wire Line
-	2700 3600 5350 3600
-Wire Wire Line
 	6650 4300 8050 4300
 Text HLabel 8050 4300 2    50   Output ~ 0
@@
 Wire Wire Line
 	5100 4800 5350 4800
-Text HLabel 2700 3600 0    50   Output ~ 0
+Text HLabel 2700 4400 0    50   Output ~ 0
 LCD_BACKLIGHT
 Wire Wire Line
@@
 	2750 3850 2750 3900
 Wire Notes Line
-	2700 3600 2750 3550
-Wire Notes Line
-	2750 3550 2750 3600
+	2700 4400 2750 4350
+Wire Notes Line
+	2750 4350 2750 4400
 Wire Notes Line
 	2700 3200 2750 3150
@@
 Wire Wire Line
 	7000 2350 7000 3900
+Wire Wire Line
+	5350 4400 2700 4400
+Wire Wire Line
+	5350 3500 2700 3500
+Wire Wire Line
+	5350 3600 2700 3600
+Text HLabel 2700 3600 0    50   BiDi ~ 0
+SAO_IO2
+Text HLabel 2700 3500 0    50   BiDi ~ 0
+SAO_IO3
 $EndSCHEMATC

Commit message: Dump.
Parts:
- C37, C38: value 20p -> 22p; LCSC (none) -> C388041; Price 0.0020 -> (none)
- C39, C40, C41: Price 0.0020 -> (none)
- J8: LCSC (none) -> -; Sponsored (none) -> N
- R41, R42, R43: LCSC - -> C115324; Price 0.0005 -> (none)
- R44: LCSC - -> C15458; Price 0.0005 -> (none)
- U10: LCSC (none) -> C7833; Sponsored (none) -> N
- U11: Price 0.97 -> (none)
- Y1: Price 0.045 -> (none)
Changed lines of the file:
@@
 F 3 "~" H 9600 5950 50  0001 C CNN
 F 4 "C14663" H 9600 5950 50  0001 C CNN "LCSC"
-F 5 "0.0020" H 9600 5950 50  0001 C CNN "Price"
+F 5 "" H 9600 5950 50  0001 C CNN "Price"
 F 6 "-" H 9600 5950 50  0001 C CNN "Mouser"
 F 7 "N" H 9600 5950 50  0001 C CNN "Sponsored"
@@
 F 3 "~" H 10100 5950 50  0001 C CNN
 F 4 "C14663" H 10100 5950 50  0001 C CNN "LCSC"
-F 5 "0.0020" H 10100 5950 50  0001 C CNN "Price"
+F 5 "" H 10100 5950 50  0001 C CNN "Price"
 F 6 "-" H 10100 5950 50  0001 C CNN "Mouser"
 F 7 "N" H 10100 5950 50  0001 C CNN "Sponsored"
@@
 F 3 "~" H 10600 5950 50  0001 C CNN
 F 4 "C14663" H 10600 5950 50  0001 C CNN "LCSC"
-F 5 "0.0020" H 10600 5950 50  0001 C CNN "Price"
+F 5 "" H 10600 5950 50  0001 C CNN "Price"
 F 6 "-" H 10600 5950 50  0001 C CNN "Mouser"
 F 7 "N" H 10600 5950 50  0001 C CNN "Sponsored"
@@
 AR Path="/5F51E414/5E3EFF6B" Ref="C38"  Part="1"
 F 0 "C38" H 4900 5300 50  0000 L CNN
-F 1 "20p" H 4900 5100 50  0000 L CNN
+F 1 "22p" H 4900 5100 50  0000 L CNN
 F 2 "Capacitor_SMD:C_0603_1608Metric" H 4938 5050 50  0001 C CNN
 F 3 "~" H 4900 5200 50  0001 C CNN
-F 4 "" H 4900 5200 50  0001 C CNN "LCSC"
-F 5 "0.0020" H 4900 5200 50  0001 C CNN "Price"
+F 4 "C388041" H 4900 5200 50  0001 C CNN "LCSC"
+F 5 "" H 4900 5200 50  0001 C CNN "Price"
 F 6 "N" H 4900 5200 50  0001 C CNN "Sponsored"
 	1    4900 5200
@@
 AR Path="/5F51E414/5E3F1F93" Ref="C37"  Part="1"
 F 0 "C37" H 4500 5300 50  0000 L CNN
-F 1 "20p" H 4450 5100 50  0000 L CNN
+F 1 "22p" H 4450 5100 50  0000 L CNN
 F 2 "Capacitor_SMD:C_0603_1608Metric" H 4688 5050 50  0001 C CNN
 F 3 "~" H 4650 5200 50  0001 C CNN
-F 4 "" H 4650 5200 50  0001 C CNN "LCSC"
-F 5 "0.0020" H 4650 5200 50  0001 C CNN "Price"
+F 4 "C388041" H 4650 5200 50  0001 C CNN "LCSC"
+F 5 "" H 4650 5200 50  0001 C CNN "Price"
 F 6 "N" H 4650 5200 50  0001 C CNN "Sponsored"
 	1    4650 5200
@@
 F 3 "~" H 4050 2850 50  0001 C CNN
 F 4 "C13738" H 4050 2850 50  0001 C CNN "LCSC"
-F 5 "0.045" H 4050 2850 50  0001 C CNN "Price"
+F 5 "" H 4050 2850 50  0001 C CNN "Price"
 F 6 "-" H 4050 2850 50  0001 C CNN "Mouser"
 F 7 "N" H 4050 2850 50  0001 C CNN "Sponsored"
@@
 F 2 "Resistor_SMD:R_0603_1608Metric" V 3580 5200 50  0001 C CNN
 F 3 "~" H 3650 5200 50  0001 C CNN
-F 4 "-" H 3650 5200 50  0001 C CNN "LCSC"
-F 5 "0.0005" H 3650 5200 50  0001 C CNN "Price"
+F 4 "C115324" H 3650 5200 50  0001 C CNN "LCSC"
+F 5 "" H 3650 5200 50  0001 C CNN "Price"
 F 6 "-" H 3650 5200 50  0001 C CNN "Mouser"
 F 7 "N" H 3650 5200 50  0001 C CNN "Sponsored"
@@
 F 2 "Resistor_SMD:R_0603_1608Metric" V 5230 2200 50  0001 C CNN
 F 3 "~" H 5300 2200 50  0001 C CNN
-F 4 "-" H 5300 2200 50  0001 C CNN "LCSC"
-F 5 "0.0005" H 5300 2200 50  0001 C CNN "Price"
+F 4 "C115324" H 5300 2200 50  0001 C CNN "LCSC"
+F 5 "" H 5300 2200 50  0001 C CNN "Price"
 F 6 "-" H 5300 2200 50  0001 C CNN "Mouser"
 F 7 "N" H 5300 2200 50  0001 C CNN "Sponsored"
@@
 F 2 "Connector_PinHeader_2.54mm:PinHeader_1x06_P2.54mm_Vertical" H 950 4600 50  0001 C CNN
 F 3 "~" H 950 4600 50  0001 C CNN
+F 4 "N" H 950 4600 50  0001 C CNN "Sponsored"
+F 5 "-" H 950 4600 50  0001 C CNN "LCSC"
 	1    950  4600
 	-1   0    0    -1
@@
 F 11 "Texas Instruments" H 3200 6300 60  0001 L CNN "Manufacturer"
 F 12 "Active" H 3200 6400 60  0001 L CNN "Status"
+F 13 "N" H 3000 5200 50  0001 C CNN "Sponsored"
+F 14 "C7833" H 3000 5200 50  0001 C CNN "LCSC"
+F 15 "" H 3000 5200 50  0001 C CNN "Price"
 	1    3000 5200
 	-1   0    0    -1
@@
 F 2 "Resistor_SMD:R_0603_1608Metric" V 6630 2200 50  0001 C CNN
 F 3 "~" H 6700 2200 50  0001 C CNN
-F 4 "-" H 6700 2200 50  0001 C CNN "LCSC"
-F 5 "0.0005" H 6700 2200 50  0001 C CNN "Price"
+F 4 "C115324" H 6700 2200 50  0001 C CNN "LCSC"
+F 5 "" H 6700 2200 50  0001 C CNN "Price"
 F 6 "-" H 6700 2200 50  0001 C CNN "Mouser"
 F 7 "N" H 6700 2200 50  0001 C CNN "Sponsored"
@@
 F 3 "http://www.st.com/st-web-ui/static/active/en/resource/technical/document/datasheet/CD00161566.pdf" H 6050 3700 50  0001 C CNN
 F 4 "C8734" H 6050 3700 50  0001 C CNN "LCSC"
-F 5 "0.97" H 6050 3700 50  0001 C CNN "Price"
+F 5 "" H 6050 3700 50  0001 C CNN "Price"
 F 6 "-" H 6050 3700 50  0001 C CNN "Mouser"
 F 7 "N" H 6050 3700 50  0001 C CNN "Sponsored"
@@
 F 2 "Resistor_SMD:R_0603_1608Metric" V 6930 2200 50  0001 C CNN
 F 3 "~" H 7000 2200 50  0001 C CNN
-F 4 "-" H 7000 2200 50  0001 C CNN "LCSC"
-F 5 "0.0005" H 7000 2200 50  0001 C CNN "Price"
+F 4 "C15458" H 7000 2200 50  0001 C CNN "LCSC"
+F 5 "" H 7000 2200 50  0001 C CNN "Price"
 F 6 "-" H 7000 2200 50  0001 C CNN "Mouser"
 F 7 "N" H 7000 2200 50  0001 C CNN "Sponsored"
