File: stm32.sch (KiCad schematic (older format))
At the start: 13 parts, among them J8 GPIO, U10 SN74LVC1G125DCKR, U11 STM32F103C8Tx, Y1 16MHz

Commit message: Work in progress: prototype 2
Parts:
- added C? (x2): 22p, Capacitor_SMD:C_0603_1608Metric, symbol Device:C
- added R?: 47, Resistor_SMD:R_0603_1608Metric, symbol Device:R
- added Y?: 32kHz, symbol Device:Crystal_Small
- U10: value SN74LVC1G125DCKR -> 74LVC1G125; footprint digikey-footprints:SOT-353 -> Package_TO_SOT_SMD:SOT-353_SC-70-5
Connections:
- net SAO_IO3 is gone; now on net ESP32_EN: U11.18 (PB0)
- net +3V3: no longer U11.1 (VBAT)
- net ESP32_BL: now also R?.1; no longer U11.3 (PC14)
- net ESP32_EN: no longer U11.2 (PC13)
- net GND: now also U10.1 (~OE), C?.2, C?.2
- net I2C_SCL: now also U11.21 (PB10); no longer U11.42 (PB6)
- net I2C_SDA: now also U11.22 (PB11); no longer U11.43 (PB7)
- net PWR_LED_ENABLE: no longer U10.1 (~OE)
- net SAO_IO0: now also U11.25 (PB12); no longer U11.21 (PB10)
- net SAO_IO1: now also U11.26 (PB13); no longer U11.20 (PB2)
- net at J8.3 (Pin_3): no longer U11.25 (PB12)
- net at J8.2 (Pin_2): no longer U11.26 (PB13)
- net at U11.4 (PC15): now also C?.1, Y?.2
- net LCD_ENABLE_PAR: no longer names the net of U11.45 (PB8)
- net SAO_IO2: no longer names the net of U11.19 (PB1)
- net SAO_IO2: now also R?.2
- net SPK: no longer names the net of U11.38 (PA15)
- new net: C?.1, U11.3 (PC14), Y?.1
- new net: U10.2 (A), U11.42 (PB6)
- new net BAT_3.3: U11.1 (VBAT)
- new net CHARGING: U11.20 (PB2)
- new net PWR_SDCARD_ENABLE: U11.28 (PB15)
Other:
- note added: "Sink only"
- note added: "if using hardware time and the aproach of DMA > Timer Output\ncompare register you will need bridge pb15 and pb11 so we can\nselect or spi or tim"
- note removed: "if using hardware time and the aproach of DMA > TIMer Output\ncompare register you will need bridge pb15 and pb11 so we can\nselect or spi or tim"
- moved on the sheet: C37, C38, J8, U10, Y1

Commit message: More work on prototype 2
Parts:
- added Q4: Q_NMOS_GSD, Package_TO_SOT_SMD:SOT-23, symbol Device:Q_NMOS_GSD
- added R61: 47, Resistor_SMD:R_0603_1608Metric, symbol Device:R
- added R63, R64: 10k, Resistor_SMD:R_0603_1608Metric, symbol Device:R
- R43: value 10k -> DNP
- gave numbers to parts that had none: 4
Connections:
- net +3V3: now also R63.2
- net ESP32_RX: now also U11.30 (PA9); no longer U11.12 (PA2)
- net ESP32_TX: now also U11.31 (PA10); no longer U11.13 (PA3)
- net FPGA_RX: now also U11.12 (PA2); no longer U11.30 (PA9)
- net FPGA_TX: now also U11.13 (PA3); no longer U11.31 (PA10)
- net GND: now also Q4.2 (S)
- net USB_D+: now also R64.1
- net at U11.2 (PC13): now also Q4.3 (D), R63.1
- net at U11.38 (PA15): now also R64.2
- new net: Q4.1 (G), R61.1
- new net USB_DET: R61.2
Other:
- note added: "Bootloader UART"
Changed lines of the file:
@@
 Sheet 5 9
 Title "MCH2021 badge - STM32 microcontroller"
-Date "2020-08-08"
-Rev "1"
+Date "2020-11-22"
+Rev "2"
 Comp "BADGE.TEAM"
 Comment1 ""
@@
 Text HLabel 2700 4500 0    50   Input ~ 0
 I2C_SCL
-Text HLabel 8050 4400 2    50   Output ~ 0
-FPGA_RX
-Text HLabel 8050 4500 2    50   Input ~ 0
-FPGA_TX
-Text HLabel 8050 3700 2    50   Output ~ 0
-ESP32_RX
-Text HLabel 8050 3800 2    50   Input ~ 0
-ESP32_TX
 $Comp
 L Device:Crystal_GND24_Small Y1
@@
 Connection ~ 6700 4700
 Wire Wire Line
-	6700 4700 8050 4700
+	6700 4700 7550 4700
 Text Notes 550  650  0    79   ~ 0
 STM32 microcontroller
@@
 AR Path="/5F51E414/5E4109CF" Ref="R43"  Part="1"
 F 0 "R43" V 6600 2200 50  0000 C CNN
-F 1 "10k" V 6700 2200 50  0000 C CNN
+F 1 "DNP" V 6700 2200 50  0000 C CNN
 F 2 "Resistor_SMD:R_0603_1608Metric" V 6630 2200 50  0001 C CNN
 F 3 "~" H 6700 2200 50  0001 C CNN
@@
 AR Path="/6015B06D" Ref="R?"  Part="1"
 AR Path="/5E3BA64A/6015B06D" Ref="R?"  Part="1"
-AR Path="/5F51E414/6015B06D" Ref="R?"  Part="1"
-F 0 "R?" V 3300 3750 50  0000 C CNN
+AR Path="/5F51E414/6015B06D" Ref="R62"  Part="1"
+F 0 "R62" V 3300 3750 50  0000 C CNN
 F 1 "47" V 3250 3600 50  0000 C CNN
 F 2 "Resistor_SMD:R_0603_1608Metric" V 3180 3600 50  0001 C CNN
@@
 $EndComp
 $Comp
-L Device:Crystal_Small Y?
+L Device:Crystal_Small Y2
 U 1 1 5FC777BF
 P 4350 3250
-F 0 "Y?" V 4304 3338 50  0000 L CNN
+F 0 "Y2" V 4304 3338 50  0000 L CNN
 F 1 "32kHz" V 4395 3338 50  0000 L CNN
 F 2 "" H 4350 3250 50  0001 C CNN
@@
 AR Path="/5FCCE7C7" Ref="C?"  Part="1"
 AR Path="/5E3BA64A/5FCCE7C7" Ref="C?"  Part="1"
-AR Path="/5F51E414/5FCCE7C7" Ref="C?"  Part="1"
-F 0 "C?" H 4650 5300 50  0000 L CNN
+AR Path="/5F51E414/5FCCE7C7" Ref="C14"  Part="1"
+F 0 "C14" H 4650 5300 50  0000 L CNN
 F 1 "22p" H 4650 5100 50  0000 L CNN
 F 2 "Capacitor_SMD:C_0603_1608Metric" H 4688 5050 50  0001 C CNN
@@
 AR Path="/5FCCE7D0" Ref="C?"  Part="1"
 AR Path="/5E3BA64A/5FCCE7D0" Ref="C?"  Part="1"
-AR Path="/5F51E414/5FCCE7D0" Ref="C?"  Part="1"
-F 0 "C?" H 4300 5300 50  0000 L CNN
+AR Path="/5F51E414/5FCCE7D0" Ref="C2"  Part="1"
+F 0 "C2" H 4300 5300 50  0000 L CNN
 F 1 "22p" H 4250 5100 50  0000 L CNN
 F 2 "Capacitor_SMD:C_0603_1608Metric" H 4488 5050 50  0001 C CNN
@@
 $EndComp
 $Comp
-L power:GND #PWR?
+L power:GND #PWR0191
 U 1 1 5FCCE7D6
 P 4650 5350
-F 0 "#PWR?" H 4650 5100 50  0001 C CNN
+F 0 "#PWR0191" H 4650 5100 50  0001 C CNN
 F 1 "GND" H 4655 5177 50  0000 C CNN
 F 2 "" H 4650 5350 50  0001 C CNN
@@
 $EndComp
 $Comp
-L power:GND #PWR?
+L power:GND #PWR0192
 U 1 1 5FCCE7DC
 P 4450 5350
-F 0 "#PWR?" H 4450 5100 50  0001 C CNN
+F 0 "#PWR0192" H 4450 5100 50  0001 C CNN
 F 1 "GND" H 4455 5177 50  0000 C CNN
 F 2 "" H 4450 5350 50  0001 C CNN
@@
 Text GLabel 5850 2200 1    50   Input ~ 0
 BAT_3.3
+$Comp
+L Device:R R?
+U 1 1 5FB263DC
+P 7550 4850
+AR Path="/5DC753C3/5FB263DC" Ref="R?"  Part="1"
+AR Path="/5FB263DC" Ref="R?"  Part="1"
+AR Path="/5E3BA64A/5FB263DC" Ref="R?"  Part="1"
+AR Path="/5F51E414/5FB263DC" Ref="R64"  Part="1"
+F 0 "R64" V 7450 4850 50  0000 C CNN
+F 1 "10k" V 7550 4850 50  0000 C CNN
+F 2 "Resistor_SMD:R_0603_1608Metric" V 7480 4850 50  0001 C CNN
+F 3 "~" H 7550 4850 50  0001 C CNN
+F 4 "C115324" H 7550 4850 50  0001 C CNN "LCSC"
+F 5 "" H 7550 4850 50  0001 C CNN "Price"
+F 6 "-" H 7550 4850 50  0001 C CNN "Mouser"
+F 7 "N" H 7550 4850 50  0001 C CNN "Sponsored"
+	1    7550 4850
+	1    0    0    -1
+$EndComp
+Connection ~ 7550 4700
+Wire Wire Line
+	7550 4700 8050 4700
+Wire Wire Line
+	7550 5000 6650 5000
+Text HLabel 8050 4400 2    50   Output ~ 0
+ESP32_RX
+Text HLabel 8050 4500 2    50   Input ~ 0
+ESP32_TX
+Text HLabel 8050 3700 2    50   Output ~ 0
+FPGA_RX
+Text HLabel 8050 3800 2    50   Input ~ 0
+FPGA_TX
+Wire Notes Line
+	8500 4350 8500 4550
+Text Notes 8550 4450 0    50   ~ 0
+Bootloader UART
+Wire Wire Line
+	5350 3100 3500 3100
+$Comp
+L Device:R R?
+U 1 1 5FB5E63D
+P 3050 6250
+AR Path="/5DC753C3/5FB5E63D" Ref="R?"  Part="1"
+AR Path="/5FB5E63D" Ref="R?"  Part="1"
+AR Path="/5E3BA64A/5FB5E63D" Ref="R?"  Part="1"
+AR Path="/5F51E414/5FB5E63D" Ref="R61"  Part="1"
+AR Path="/5FDC6C76/5FB5E63D" Ref="R?"  Part="1"
+F 0 "R61" V 2950 6250 50  0000 C CNN
+F 1 "47" V 3050 6250 50  0000 C CNN
+F 2 "Resistor_SMD:R_0603_1608Metric" V 2980 6250 50  0001 C CNN
+F 3 "~" H 3050 6250 50  0001 C CNN
+F 4 "C1211" H 3050 6250 50  0001 C CNN "LCSC"
+F 5 "" H 3050 6250 50  0001 C CNN "Price"
+F 6 "-" H 3050 6250 50  0001 C CNN "Mouser"
+F 7 "N" H 3050 6250 50  0001 C CNN "Sponsored"
+	1    3050 6250
+	0    1    1    0
+$EndComp
+$Comp
+L Device:Q_NMOS_GSD Q?
+U 1 1 5FB5E630
+P 3400 6250
+AR Path="/5FDC6C76/5FB5E630" Ref="Q?"  Part="1"
+AR Path="/5F51E414/5FB5E630" Ref="Q4"  Part="1"
+F 0 "Q4" H 3350 6050 50  0000 C CNN
+F 1 "Q_NMOS_GSD" H 3150 6150 50  0000 C CNN
+F 2 "Package_TO_SOT_SMD:SOT-23" H 3600 6350 50  0001 C CNN
+F 3 "~" H 3400 6250 50  0001 C CNN
+F 4 "C406812" H 3400 6250 50  0001 C CNN "LCSC"
+F 5 "-" H 3400 6250 50  0001 C CNN "Mouser"
+F 6 "" H 3400 6250 50  0001 C CNN "Price"
+F 7 "N" H 3400 6250 50  0001 C CNN "Sponsored"
+	1    3400 6250
+	1    0    0    -1
+$EndComp
+$Comp
+L Device:R R?
+U 1 1 5FB7AAB6
+P 3500 2200
+AR Path="/5DC753C3/5FB7AAB6" Ref="R?"  Part="1"
+AR Path="/5FB7AAB6" Ref="R?"  Part="1"
+AR Path="/5E3BA64A/5FB7AAB6" Ref="R?"  Part="1"
+AR Path="/5F51E414/5FB7AAB6" Ref="R63"  Part="1"
+F 0 "R63" V 3600 2200 50  0000 C CNN
+F 1 "10k" V 3500 2200 50  0000 C CNN
+F 2 "Resistor_SMD:R_0603_1608Metric" V 3430 2200 50  0001 C CNN
+F 3 "~" H 3500 2200 50  0001 C CNN
+F 4 "C115324" H 3500 2200 50  0001 C CNN "LCSC"
+F 5 "" H 3500 2200 50  0001 C CNN "Price"
+F 6 "-" H 3500 2200 50  0001 C CNN "Mouser"
+F 7 "N" H 3500 2200 50  0001 C CNN "Sponsored"
+	1    3500 2200
+	-1   0    0    1
+$EndComp
+$Comp
+L power:+3.3V #PWR0193
+U 1 1 5FB7E8B5
+P 3500 2050
+F 0 "#PWR0193" H 3500 1900 50  0001 C CNN
+F 1 "+3.3V" H 3515 2223 50  0000 C CNN
+F 2 "" H 3500 2050 50  0001 C CNN
+F 3 "" H 3500 2050 50  0001 C CNN
+	1    3500 2050
+	1    0    0    -1
+$EndComp
+Wire Wire Line
+	3500 2350 3500 3100
+Wire Wire Line
+	3500 3100 3500 6050
+Connection ~ 3500 3100
+$Comp
+L power:GND #PWR0194
+U 1 1 5FB9040E
+P 3500 6450
+F 0 "#PWR0194" H 3500 6200 50  0001 C CNN
+F 1 "GND" H 3505 6277 50  0000 C CNN
+F 2 "" H 3500 6450 50  0001 C CNN
+F 3 "" H 3500 6450 50  0001 C CNN
+	1    3500 6450
+	1    0    0    -1
+$EndComp
+Wire Wire Line
+	2700 6250 2900 6250
+Text HLabel 2700 6250 0    50   Input ~ 0
+USB_DET
 $EndSCHEMATC

Commit message: Add testpoints, add way for STM32 to wake-up ESP32 from deep sleep
Connections:
- net ESP32_WK: now reaches U11.39 (PB3)
- net at U11.43 (PB7): now also J8.2 (Pin_2)
- net at U11.45 (PB8): now also J8.3 (Pin_3)
Changed lines of the file:
@@
 Sheet 5 9
 Title "MCH2021 badge - STM32 microcontroller"
-Date "2020-11-22"
+Date "2020-11-29"
 Rev "2"
 Comp "BADGE.TEAM"
@@
 Text HLabel 2700 6250 0    50   Input ~ 0
 USB_DET
+Wire Wire Line
+	5350 3800 2700 3800
+Text HLabel 2700 3800 0    50   Output ~ 0
+ESP32_WK
+Wire Wire Line
+	5350 4300 3300 4300
+Wire Wire Line
+	3300 4300 3300 5600
+Wire Wire Line
+	3300 5600 1150 5600
+Wire Wire Line
+	1150 5500 3200 5500
+Wire Wire Line
+	3200 5500 3200 4200
+Wire Wire Line
+	3200 4200 5350 4200
 $EndSCHEMATC

Commit message: Schematic for prototype 2 is now complete, time for review! :D
Parts:
- removed U10: 74LVC1G125, Package_TO_SOT_SMD:SOT-353_SC-70-5, symbol dk_Logic-Buffers-Drivers-Receivers-Transceivers:SN74LVC1G125DCKR
Connections:
- net LED_DATA: now also U11.42 (PB6)
Changed lines of the file:
@@
 Text HLabel 8050 4200 2    50   Input ~ 0
 SPI_MOSI
-Text HLabel 1050 4100 0    50   Output ~ 0
-LED_DATA
 Text HLabel 2700 4900 0    50   Output ~ 0
 PWR_LED_ENABLE
@@
 	1    0    0    -1
 $EndComp
-$Comp
-L power:GND #PWR0138
-U 1 1 5F9F3DCC
-P 1350 4300
-F 0 "#PWR0138" H 1350 4050 50  0001 C CNN
-F 1 "GND" H 1355 4127 50  0000 C CNN
-F 2 "" H 1350 4300 50  0001 C CNN
-F 3 "" H 1350 4300 50  0001 C CNN
-	1    1350 4300
-	1    0    0    -1
-$EndComp
 Wire Notes Line
 	2750 3850 2750 3900
@@
 Wire Notes Line
 	2800 4050 2750 4000
-$Comp
-L Connector_Generic:Conn_01x06 J8
-U 1 1 5F5C2047
-P 950 5600
-F 0 "J8" H 1058 5881 50  0000 C CNN
-F 1 "GPIO" H 1058 5790 50  0000 C CNN
-F 2 "Connector_PinHeader_2.54mm:PinHeader_1x06_P2.54mm_Vertical" H 950 5600 50  0001 C CNN
-F 3 "~" H 950 5600 50  0001 C CNN
-F 4 "N" H 950 5600 50  0001 C CNN "Sponsored"
-F 5 "-" H 950 5600 50  0001 C CNN "LCSC"
-	1    950  5600
-	-1   0    0    -1
-$EndComp
 $Comp
 L power:GND #PWR0136
@@
 	1    0    0    -1
 $EndComp
-$Comp
-L power:+3.3V #PWR0135
-U 1 1 5F5CC1A1
-P 1250 5300
-F 0 "#PWR0135" H 1250 5150 50  0001 C CNN
-F 1 "+3.3V" H 1265 5473 50  0000 C CNN
-F 2 "" H 1250 5300 50  0001 C CNN
-F 3 "" H 1250 5300 50  0001 C CNN
-	1    1250 5300
-	1    0    0    -1
-$EndComp
-Wire Wire Line
-	1250 5400 1250 5300
-Wire Wire Line
-	1250 5400 1150 5400
 Wire Wire Line
 	1150 5900 1250 5900
@@
 Wire Wire Line
 	7150 5800 7150 4900
-$Comp
-L vin:VIN #PWR0137
-U 1 1 5F61F3B1
-P 1350 3700
-F 0 "#PWR0137" H 1360 3700 20  0001 C CNN
-F 1 "VIN" H 1350 3796 40  0000 C CNN
-F 2 "" H 1350 3700 60  0001 C CNN
-F 3 "" H 1350 3700 60  0001 C CNN
-	1    1350 3700
-	1    0    0    -1
-$EndComp
-$Comp
-L dk_Logic-Buffers-Drivers-Receivers-Transceivers:SN74LVC1G125DCKR U10
-U 1 1 5F6503C3
-P 1350 4000
-F 0 "U10" H 1600 4200 60  0000 C CNN
-F 1 "74LVC1G125" H 1800 4100 60  0000 C CNN
-F 2 "Package_TO_SOT_SMD:SOT-353_SC-70-5" H 1550 4200 60  0001 L CNN
-F 3 "http://www.ti.com/general/docs/suppproductinfo.tsp?distId=10&gotoUrl=http%3A%2F%2Fwww.ti.com%2Flit%2Fgpn%2Fsn74lvc1g125" H 1550 4300 60  0001 L CNN
-F 4 "296-11604-1-ND" H 1550 4400 60  0001 L CNN "Digi-Key_PN"
-F 5 "SN74LVC1G125DCKR" H 1550 4500 60  0001 L CNN "MPN"
-F 6 "Integrated Circuits (ICs)" H 1550 4600 60  0001 L CNN "Category"
-F 7 "Logic - Buffers, Drivers, Receivers, Transceivers" H 1550 4700 60  0001 L CNN "Family"
-F 8 "http://www.ti.com/general/docs/suppproductinfo.tsp?distId=10&gotoUrl=http%3A%2F%2Fwww.ti.com%2Flit%2Fgpn%2Fsn74lvc1g125" H 1550 4800 60  0001 L CNN "DK_Datasheet_Link"
-F 9 "/product-detail/en/texas-instruments/SN74LVC1G125DCKR/296-11604-1-ND/385743" H 1550 4900 60  0001 L CNN "DK_Detail_Page"
-F 10 "IC BUF NON-INVERT 5.5V SC70-5" H 1550 5000 60  0001 L CNN "Description"
-F 11 "Texas Instruments" H 1550 5100 60  0001 L CNN "Manufacturer"
-F 12 "Active" H 1550 5200 60  0001 L CNN "Status"
-F 13 "N" H 1350 4000 50  0001 C CNN "Sponsored"
-F 14 "C7833" H 1350 4000 50  0001 C CNN "LCSC"
-F 15 "" H 1350 4000 50  0001 C CNN "Price"
-	1    1350 4000
-	-1   0    0    -1
-$EndComp
-Wire Wire Line
-	1150 4100 1050 4100
-Wire Wire Line
-	1650 3900 1700 3900
 Wire Wire Line
 	2700 4500 5350 4500
@@
 Wire Wire Line
 	5350 4400 2700 4400
-$Comp
-L power:GND #PWR0182
-U 1 1 5F8A4D62
-P 1700 4300
-F 0 "#PWR0182" H 1700 4050 50  0001 C CNN
-F 1 "GND" H 1705 4127 50  0000 C CNN
-F 2 "" H 1700 4300 50  0001 C CNN
-F 3 "" H 1700 4300 50  0001 C CNN
-	1    1700 4300
-	1    0    0    -1
-$EndComp
-Wire Wire Line
-	1700 3900 1700 4300
 Text HLabel 2700 3700 0    50   Input ~ 0
 CHARGING
@@
 Wire Wire Line
 	1150 5700 7100 5700
-Wire Wire Line
-	1650 4100 5350 4100
 Wire Notes Line
 	5450 3000 5700 3000
@@
 ESP32_WK
 Wire Wire Line
+	5350 4100 2700 4100
+Text HLabel 2700 4100 0    50   Output ~ 0
+LED_DATA
+Wire Wire Line
 	5350 4300 3300 4300
 Wire Wire Line
+	3200 4200 5350 4200
+Wire Wire Line
+	3200 5500 3200 4200
+Wire Wire Line
 	3300 4300 3300 5600
+$Comp
+L power:+3.3V #PWR0135
+U 1 1 5F5CC1A1
+P 1250 5300
+F 0 "#PWR0135" H 1250 5150 50  0001 C CNN
+F 1 "+3.3V" H 1265 5473 50  0000 C CNN
+F 2 "" H 1250 5300 50  0001 C CNN
+F 3 "" H 1250 5300 50  0001 C CNN
+	1    1250 5300
+	1    0    0    -1
+$EndComp
+Wire Wire Line
+	1250 5400 1250 5300
+Wire Wire Line
+	1250 5400 1150 5400
+$Comp
+L Connector_Generic:Conn_01x06 J8
+U 1 1 5F5C2047
+P 950 5600
+F 0 "J8" H 1058 5881 50  0000 C CNN
+F 1 "GPIO" H 1058 5790 50  0000 C CNN
+F 2 "Connector_PinHeader_2.54mm:PinHeader_1x06_P2.54mm_Vertical" H 950 5600 50  0001 C CNN
+F 3 "~" H 950 5600 50  0001 C CNN
+F 4 "N" H 950 5600 50  0001 C CNN "Sponsored"
+F 5 "-" H 950 5600 50  0001 C CNN "LCSC"
+	1    950  5600
+	-1   0    0    -1
+$EndComp
 Wire Wire Line
 	3300 5600 1150 5600
 Wire Wire Line
 	1150 5500 3200 5500
-Wire Wire Line
-	3200 5500 3200 4200
-Wire Wire Line
-	3200 4200 5350 4200
 $EndSCHEMATC
