File: stm32.sch (KiCad schematic (older format))
At the start: 20 parts, among them J8 GPIO, Q4 Q_NMOS_GSD, U11 STM32F103C8Tx, Y1 16MHz, Y2 32kHz

Commit message: Updated schematic, add design file
Parts:
- Y2: footprint (none) -> Crystal:Crystal_SMD_3215-2Pin_3.2x1.5mm
Changed lines of the file:
@@
 F 0 "Y2" V 4304 3338 50  0000 L CNN
 F 1 "32kHz" V 4395 3338 50  0000 L CNN
-F 2 "" H 4350 3250 50  0001 C CNN
+F 2 "Crystal:Crystal_SMD_3215-2Pin_3.2x1.5mm" H 4350 3250 50  0001 C CNN
 F 3 "~" H 4350 3250 50  0001 C CNN
 	1    4350 3250

Commit message: First steps of routing prototype 2, switch to 0402 for most passives
Parts:
- C14, C2, C37, C38: footprint Capacitor_SMD:C_0603_1608Metric -> Capacitor_SMD:C_0402_1005Metric; LCSC C388041 -> C696906
- C39, C40, C41: footprint Capacitor_SMD:C_0603_1608Metric -> Capacitor_SMD:C_0402_1005Metric; LCSC C14663 -> C83056
- R41, R42, R43, R62, R63, R64: footprint Resistor_SMD:R_0603_1608Metric -> Resistor_SMD:R_0402_1005Metric; LCSC C115324 -> (none)
- R44: footprint Resistor_SMD:R_0603_1608Metric -> Resistor_SMD:R_0402_1005Metric; LCSC C15458 -> (none)
- R61: footprint Resistor_SMD:R_0603_1608Metric -> Resistor_SMD:R_0402_1005Metric; LCSC C1211 -> (none)
Changed lines of the file:
@@
 F 0 "C39" H 9715 5996 50  0000 L CNN
 F 1 "100n" H 9715 5905 50  0000 L CNN
-F 2 "Capacitor_SMD:C_0603_1608Metric" H 9638 5800 50  0001 C CNN
-F 3 "~" H 9600 5950 50  0001 C CNN
-F 4 "C14663" H 9600 5950 50  0001 C CNN "LCSC"
+F 2 "Capacitor_SMD:C_0402_1005Metric" H 9638 5800 50  0001 C CNN
+F 3 "" H 9600 5950 50  0001 C CNN
+F 4 "C83056 " H 9600 5950 50  0001 C CNN "LCSC"
 F 5 "" H 9600 5950 50  0001 C CNN "Price"
 F 6 "-" H 9600 5950 50  0001 C CNN "Mouser"
@@
 F 0 "C40" H 10215 5996 50  0000 L CNN
 F 1 "100n" H 10215 5905 50  0000 L CNN
-F 2 "Capacitor_SMD:C_0603_1608Metric" H 10138 5800 50  0001 C CNN
-F 3 "~" H 10100 5950 50  0001 C CNN
-F 4 "C14663" H 10100 5950 50  0001 C CNN "LCSC"
+F 2 "Capacitor_SMD:C_0402_1005Metric" H 10138 5800 50  0001 C CNN
+F 3 "" H 10100 5950 50  0001 C CNN
+F 4 "C83056 " H 10100 5950 50  0001 C CNN "LCSC"
 F 5 "" H 10100 5950 50  0001 C CNN "Price"
 F 6 "-" H 10100 5950 50  0001 C CNN "Mouser"
@@
 F 0 "C41" H 10715 5996 50  0000 L CNN
 F 1 "100n" H 10715 5905 50  0000 L CNN
-F 2 "Capacitor_SMD:C_0603_1608Metric" H 10638 5800 50  0001 C CNN
-F 3 "~" H 10600 5950 50  0001 C CNN
-F 4 "C14663" H 10600 5950 50  0001 C CNN "LCSC"
+F 2 "Capacitor_SMD:C_0402_1005Metric" H 10638 5800 50  0001 C CNN
+F 3 "" H 10600 5950 50  0001 C CNN
+F 4 "C83056 " H 10600 5950 50  0001 C CNN "LCSC"
 F 5 "" H 10600 5950 50  0001 C CNN "Price"
 F 6 "-" H 10600 5950 50  0001 C CNN "Mouser"
@@
 F 0 "C38" H 5250 5300 50  0000 L CNN
 F 1 "22p" H 5250 5100 50  0000 L CNN
-F 2 "Capacitor_SMD:C_0603_1608Metric" H 5288 5050 50  0001 C CNN
-F 3 "~" H 5250 5200 50  0001 C CNN
-F 4 "C388041" H 5250 5200 50  0001 C CNN "LCSC"
+F 2 "Capacitor_SMD:C_0402_1005Metric" H 5288 5050 50  0001 C CNN
+F 3 "" H 5250 5200 50  0001 C CNN
+F 4 "C696906" H 5250 5200 50  0001 C CNN "LCSC"
 F 5 "" H 5250 5200 50  0001 C CNN "Price"
 F 6 "N" H 5250 5200 50  0001 C CNN "Sponsored"
@@
 F 0 "C37" H 4900 5300 50  0000 L CNN
 F 1 "22p" H 4850 5100 50  0000 L CNN
-F 2 "Capacitor_SMD:C_0603_1608Metric" H 5088 5050 50  0001 C CNN
-F 3 "~" H 5050 5200 50  0001 C CNN
-F 4 "C388041" H 5050 5200 50  0001 C CNN "LCSC"
+F 2 "Capacitor_SMD:C_0402_1005Metric" H 5088 5050 50  0001 C CNN
+F 3 "" H 5050 5200 50  0001 C CNN
+F 4 "C696906" H 5050 5200 50  0001 C CNN "LCSC"
 F 5 "" H 5050 5200 50  0001 C CNN "Price"
 F 6 "N" H 5050 5200 50  0001 C CNN "Sponsored"
@@
 F 0 "R41" V 3750 5200 50  0000 C CNN
 F 1 "10k" V 3650 5200 50  0000 C CNN
-F 2 "Resistor_SMD:R_0603_1608Metric" V 3580 5200 50  0001 C CNN
+F 2 "Resistor_SMD:R_0402_1005Metric" V 3580 5200 50  0001 C CNN
 F 3 "~" H 3650 5200 50  0001 C CNN
-F 4 "C115324" H 3650 5200 50  0001 C CNN "LCSC"
+F 4 "" H 3650 5200 50  0001 C CNN "LCSC"
 F 5 "" H 3650 5200 50  0001 C CNN "Price"
 F 6 "-" H 3650 5200 50  0001 C CNN "Mouser"
@@
 F 0 "R42" V 5200 2200 50  0000 C CNN
 F 1 "10k" V 5300 2200 50  0000 C CNN
-F 2 "Resistor_SMD:R_0603_1608Metric" V 5230 2200 50  0001 C CNN
+F 2 "Resistor_SMD:R_0402_1005Metric" V 5230 2200 50  0001 C CNN
 F 3 "~" H 5300 2200 50  0001 C CNN
-F 4 "C115324" H 5300 2200 50  0001 C CNN "LCSC"
+F 4 "" H 5300 2200 50  0001 C CNN "LCSC"
 F 5 "" H 5300 2200 50  0001 C CNN "Price"
 F 6 "-" H 5300 2200 50  0001 C CNN "Mouser"
@@
 F 0 "R43" V 6600 2200 50  0000 C CNN
 F 1 "DNP" V 6700 2200 50  0000 C CNN
-F 2 "Resistor_SMD:R_0603_1608Metric" V 6630 2200 50  0001 C CNN
+F 2 "Resistor_SMD:R_0402_1005Metric" V 6630 2200 50  0001 C CNN
 F 3 "~" H 6700 2200 50  0001 C CNN
-F 4 "C115324" H 6700 2200 50  0001 C CNN "LCSC"
+F 4 "" H 6700 2200 50  0001 C CNN "LCSC"
 F 5 "" H 6700 2200 50  0001 C CNN "Price"
 F 6 "-" H 6700 2200 50  0001 C CNN "Mouser"
@@
 F 0 "R44" V 6900 2200 50  0000 C CNN
 F 1 "100k" V 7000 2200 50  0000 C CNN
-F 2 "Resistor_SMD:R_0603_1608Metric" V 6930 2200 50  0001 C CNN
+F 2 "Resistor_SMD:R_0402_1005Metric" V 6930 2200 50  0001 C CNN
 F 3 "~" H 7000 2200 50  0001 C CNN
-F 4 "C15458" H 7000 2200 50  0001 C CNN "LCSC"
+F 4 "" H 7000 2200 50  0001 C CNN "LCSC"
 F 5 "" H 7000 2200 50  0001 C CNN "Price"
 F 6 "-" H 7000 2200 50  0001 C CNN "Mouser"
@@
 F 0 "R62" V 3300 3750 50  0000 C CNN
 F 1 "47" V 3250 3600 50  0000 C CNN
-F 2 "Resistor_SMD:R_0603_1608Metric" V 3180 3600 50  0001 C CNN
+F 2 "Resistor_SMD:R_0402_1005Metric" V 3180 3600 50  0001 C CNN
 F 3 "~" H 3250 3600 50  0001 C CNN
-F 4 "C115324" H 3250 3600 50  0001 C CNN "LCSC"
+F 4 "" H 3250 3600 50  0001 C CNN "LCSC"
 F 5 "" H 3250 3600 50  0001 C CNN "Price"
 F 6 "-" H 3250 3600 50  0001 C CNN "Mouser"
@@
 F 0 "C14" H 4650 5300 50  0000 L CNN
 F 1 "22p" H 4650 5100 50  0000 L CNN
-F 2 "Capacitor_SMD:C_0603_1608Metric" H 4688 5050 50  0001 C CNN
-F 3 "~" H 4650 5200 50  0001 C CNN
-F 4 "C388041" H 4650 5200 50  0001 C CNN "LCSC"
+F 2 "Capacitor_SMD:C_0402_1005Metric" H 4688 5050 50  0001 C CNN
+F 3 "" H 4650 5200 50  0001 C CNN
+F 4 "C696906" H 4650 5200 50  0001 C CNN "LCSC"
 F 5 "" H 4650 5200 50  0001 C CNN "Price"
 F 6 "N" H 4650 5200 50  0001 C CNN "Sponsored"
@@
 F 0 "C2" H 4300 5300 50  0000 L CNN
 F 1 "22p" H 4250 5100 50  0000 L CNN
-F 2 "Capacitor_SMD:C_0603_1608Metric" H 4488 5050 50  0001 C CNN
-F 3 "~" H 4450 5200 50  0001 C CNN
-F 4 "C388041" H 4450 5200 50  0001 C CNN "LCSC"
+F 2 "Capacitor_SMD:C_0402_1005Metric" H 4488 5050 50  0001 C CNN
+F 3 "" H 4450 5200 50  0001 C CNN
+F 4 "C696906" H 4450 5200 50  0001 C CNN "LCSC"
 F 5 "" H 4450 5200 50  0001 C CNN "Price"
 F 6 "N" H 4450 5200 50  0001 C CNN "Sponsored"
@@
 F 0 "R64" V 7450 4850 50  0000 C CNN
 F 1 "10k" V 7550 4850 50  0000 C CNN
-F 2 "Resistor_SMD:R_0603_1608Metric" V 7480 4850 50  0001 C CNN
+F 2 "Resistor_SMD:R_0402_1005Metric" V 7480 4850 50  0001 C CNN
 F 3 "~" H 7550 4850 50  0001 C CNN
-F 4 "C115324" H 7550 4850 50  0001 C CNN "LCSC"
+F 4 "" H 7550 4850 50  0001 C CNN "LCSC"
 F 5 "" H 7550 4850 50  0001 C CNN "Price"
 F 6 "-" H 7550 4850 50  0001 C CNN "Mouser"
@@
 F 0 "R61" V 2950 6250 50  0000 C CNN
 F 1 "47" V 3050 6250 50  0000 C CNN
-F 2 "Resistor_SMD:R_0603_1608Metric" V 2980 6250 50  0001 C CNN
+F 2 "Resistor_SMD:R_0402_1005Metric" V 2980 6250 50  0001 C CNN
 F 3 "~" H 3050 6250 50  0001 C CNN
-F 4 "C1211" H 3050 6250 50  0001 C CNN "LCSC"
+F 4 "" H 3050 6250 50  0001 C CNN "LCSC"
 F 5 "" H 3050 6250 50  0001 C CNN "Price"
 F 6 "-" H 3050 6250 50  0001 C CNN "Mouser"
@@
 F 0 "R63" V 3600 2200 50  0000 C CNN
 F 1 "10k" V 3500 2200 50  0000 C CNN
-F 2 "Resistor_SMD:R_0603_1608Metric" V 3430 2200 50  0001 C CNN
+F 2 "Resistor_SMD:R_0402_1005Metric" V 3430 2200 50  0001 C CNN
 F 3 "~" H 3500 2200 50  0001 C CNN
-F 4 "C115324" H 3500 2200 50  0001 C CNN "LCSC"
+F 4 "" H 3500 2200 50  0001 C CNN "LCSC"
 F 5 "" H 3500 2200 50  0001 C CNN "Price"
 F 6 "-" H 3500 2200 50  0001 C CNN "Mouser"

Commit message: Some more work
Parts:
- removed J8: GPIO, Connector_PinHeader_2.54mm:PinHeader_1x06_P2.54mm_Vertical, symbol Connector_Generic:Conn_01x06
- added J8: JTAG, Connector:Tag-Connect_TC2030-IDC-FP_2x03_P1.27mm_Vertical, symbol Connector_Generic:Conn_02x03_Odd_Even
- renumbered C38 to C10, C39 to C11, C40 to C12, C41 to C13, C2 to C7, C14 to C8, C37 to C9, Q4 to Q3, R61 to R22, R62 to R23, R63 to R24, R41 to R25, R42 to R26, R43 to R27, R44 to R28, R64 to R29, U11 to U3, Y2 to Y1, Y1 to Y2
Connections:
- net labels added: STM32_SWCLK, STM32_SWDIO
- wire segments 102 -> 96
- no-connect marks 0 -> 1

Commit message: Add extra IO header, add battery NTC connection
Connections:
- net SAO_IO0: now also U3.26 (PB13); no longer U3.25 (PB12)
- net SAO_IO1: now also U3.25 (PB12); no longer U3.26 (PB13)
- net at R23.2: now also U3.45 (PB8); no longer U3.19 (PB1)
- net SAO_IO2: now reaches U3.43 (PB7)
- new net BATT_TEMP: U3.19 (PB1)
Other:
- moved on the sheet: R23
Changed lines of the file:
@@
 Text HLabel 2700 3500 0    50   Output ~ 0
 ESP32_EN
-Text HLabel 2700 3600 0    50   Output ~ 0
+Text HLabel 2700 4300 0    50   Output ~ 0
 ESP32_BL
 Wire Wire Line
@@
 Text HLabel 8050 3500 2    50   Input ~ 0
 SENSE_VUSB
+Text HLabel 2700 4800 0    50   BiDi ~ 0
+SAO_IO0
 Text HLabel 2700 4700 0    50   BiDi ~ 0
-SAO_IO0
-Text HLabel 2700 4800 0    50   BiDi ~ 0
 SAO_IO1
 Wire Wire Line
@@
 Text HLabel 2700 4400 0    50   Output ~ 0
 LCD_BACKLIGHT
-Wire Wire Line
-	2700 3600 3100 3600
 Wire Wire Line
 	2700 2400 2800 2400
@@
 L Device:R R?
 U 1 1 6015B06D
-P 3250 3600
+P 3250 4300
 AR Path="/5DC753C3/6015B06D" Ref="R?"  Part="1"
 AR Path="/6015B06D" Ref="R?"  Part="1"
 AR Path="/5E3BA64A/6015B06D" Ref="R?"  Part="1"
 AR Path="/5F51E414/6015B06D" Ref="R23"  Part="1"
-F 0 "R23" V 3300 3750 50  0000 C CNN
-F 1 "47" V 3250 3600 50  0000 C CNN
-F 2 "Resistor_SMD:R_0402_1005Metric" V 3180 3600 50  0001 C CNN
-F 3 "~" H 3250 3600 50  0001 C CNN
-F 4 "" H 3250 3600 50  0001 C CNN "LCSC"
-F 5 "" H 3250 3600 50  0001 C CNN "Price"
-F 6 "-" H 3250 3600 50  0001 C CNN "Mouser"
-F 7 "N" H 3250 3600 50  0001 C CNN "Sponsored"
-	1    3250 3600
+F 0 "R23" V 3300 4450 50  0000 C CNN
+F 1 "47" V 3250 4300 50  0000 C CNN
+F 2 "Resistor_SMD:R_0402_1005Metric" V 3180 4300 50  0001 C CNN
+F 3 "~" H 3250 4300 50  0001 C CNN
+F 4 "" H 3250 4300 50  0001 C CNN "LCSC"
+F 5 "" H 3250 4300 50  0001 C CNN "Price"
+F 6 "-" H 3250 4300 50  0001 C CNN "Mouser"
+F 7 "N" H 3250 4300 50  0001 C CNN "Sponsored"
+	1    3250 4300
 	0    -1   -1   0
 $EndComp
@@
 Wire Wire Line
 	2700 3700 5350 3700
-Wire Wire Line
-	5350 3600 3400 3600
 Text GLabel 5850 2000 1    31   Input ~ 0
 BAT_3.3
@@
 	5350 4400 2700 4400
 Wire Wire Line
-	2700 4300 5350 4300
-Wire Wire Line
-	2700 4200 5350 4200
+	2700 4300 3100 4300
 Text GLabel 6650 4800 2    31   Input ~ 0
 STM32_SWDIO
@@
 Wire Wire Line
 	5850 2200 5850 2000
+Wire Wire Line
+	2700 3600 5350 3600
+Wire Wire Line
+	3400 4300 5350 4300
+Text HLabel 2700 3600 0    50   Input ~ 0
+BATT_TEMP
+Wire Wire Line
+	2700 4200 5350 4200
+Text GLabel 2700 4200 0    50   BiDi ~ 0
+SAO_IO2
 $EndSCHEMATC

Commit message: Update LCSC code for the 32kHz crystals
Parts:
- Y1: LCSC (none) -> C271654
Changed lines of the file:
@@
 F 2 "Crystal:Crystal_SMD_3215-2Pin_3.2x1.5mm" H 4350 3250 50  0001 C CNN
 F 3 "~" H 4350 3250 50  0001 C CNN
+F 4 "C271654" H 4350 3250 50  0001 C CNN "LCSC"
 	1    4350 3250
 	0    1    1    0

Commit message: Fix most of the bugs found on prototype 2 board
Parts:
- removed R27: DNP, Resistor_SMD:R_0402_1005Metric, symbol Device:R
- added R6, R7: 22, Resistor_SMD:R_0402_1005Metric, symbol Device:R_Small
- added TP14: UNUSED PIN, TestPoint:TestPoint_Pad_1.0x1.0mm, symbol Connector:TestPoint
Connections:
- net USB_D+: now also R7.2; no longer U3.33 (PA12)
- net USB_D-: now also R6.1; no longer U3.32 (PA11)
- net PWR_SDCARD_ENABLE: no longer names the net of U3.28 (PB15)
- net PWR_SDCARD_ENABLE: now also TP14.1
- new net: R6.2, U3.32 (PA11)
- new net: R7.1, U3.33 (PA12)
Other:
- moved on the sheet: R29
Changed lines of the file:
@@
 Sheet 3 9
 Title "MCH2021 badge - STM32 microcontroller"
-Date "2021-01-14"
-Rev "2"
+Date "2021-10-09"
+Rev "3"
 Comp "BADGE.TEAM"
 Comment1 ""
@@
 Text HLabel 8050 4600 2    50   BiDi ~ 0
 USB_D-
-Wire Wire Line
-	6650 4700 6700 4700
 Text HLabel 2700 4500 0    50   Input ~ 0
 I2C_SCL
@@
 	6650 3800 8050 3800
 Wire Wire Line
-	6650 4600 8050 4600
+	6650 4600 7700 4600
 Wire Wire Line
 	6650 4500 8050 4500
 Wire Wire Line
 	6650 4400 8050 4400
-Wire Wire Line
-	6700 4700 6700 2350
-Connection ~ 6700 4700
-Wire Wire Line
-	6700 4700 7550 4700
 Text Notes 550  650  0    79   ~ 0
 STM32 microcontroller
@@
 SPI_CS
 $Comp
-L power:+3.3V #PWR057
-U 1 1 5F85DFEF
-P 6700 2050
-F 0 "#PWR057" H 6700 1900 50  0001 C CNN
-F 1 "+3.3V" H 6715 2223 50  0000 C CNN
-F 2 "" H 6700 2050 50  0001 C CNN
-F 3 "" H 6700 2050 50  0001 C CNN
-	1    6700 2050
-	1    0    0    -1
-$EndComp
-$Comp
-L Device:R R?
-U 1 1 5E4109CF
-P 6700 2200
-AR Path="/5DC753C3/5E4109CF" Ref="R?"  Part="1"
-AR Path="/5E4109CF" Ref="R?"  Part="1"
-AR Path="/5E3BA64A/5E4109CF" Ref="R?"  Part="1"
-AR Path="/5F51E414/5E4109CF" Ref="R27"  Part="1"
-F 0 "R27" V 6600 2200 50  0000 C CNN
-F 1 "DNP" V 6700 2200 50  0000 C CNN
-F 2 "Resistor_SMD:R_0402_1005Metric" V 6630 2200 50  0001 C CNN
-F 3 "~" H 6700 2200 50  0001 C CNN
-F 4 "" H 6700 2200 50  0001 C CNN "LCSC"
-F 5 "" H 6700 2200 50  0001 C CNN "Price"
-F 6 "-" H 6700 2200 50  0001 C CNN "Mouser"
-F 7 "N" H 6700 2200 50  0001 C CNN "Sponsored"
-	1    6700 2200
-	1    0    0    -1
-$EndComp
-$Comp
 L MCU_ST_STM32F1:STM32F103C8Tx U3
 U 1 1 5E3BAF1D
@@
 Text Notes 5800 3350 1    39   ~ 0
 Sink only
-Text HLabel 2700 5000 0    50   Output ~ 0
-PWR_SDCARD_ENABLE
 Wire Wire Line
 	5350 5000 2700 5000
@@
 L Device:R R?
 U 1 1 5FB263DC
-P 7550 4850
+P 7950 4850
 AR Path="/5DC753C3/5FB263DC" Ref="R?"  Part="1"
 AR Path="/5FB263DC" Ref="R?"  Part="1"
 AR Path="/5E3BA64A/5FB263DC" Ref="R?"  Part="1"
 AR Path="/5F51E414/5FB263DC" Ref="R29"  Part="1"
-F 0 "R29" V 7450 4850 50  0000 C CNN
-F 1 "10k" V 7550 4850 50  0000 C CNN
-F 2 "Resistor_SMD:R_0402_1005Metric" V 7480 4850 50  0001 C CNN
-F 3 "~" H 7550 4850 50  0001 C CNN
-F 4 "" H 7550 4850 50  0001 C CNN "LCSC"
-F 5 "" H 7550 4850 50  0001 C CNN "Price"
-F 6 "-" H 7550 4850 50  0001 C CNN "Mouser"
-F 7 "N" H 7550 4850 50  0001 C CNN "Sponsored"
-	1    7550 4850
-	1    0    0    -1
-$EndComp
-Connection ~ 7550 4700
-Wire Wire Line
-	7550 4700 8050 4700
-Wire Wire Line
-	7550 5000 6650 5000
+F 0 "R29" V 7850 4850 50  0000 C CNN
+F 1 "10k" V 7950 4850 50  0000 C CNN
+F 2 "Resistor_SMD:R_0402_1005Metric" V 7880 4850 50  0001 C CNN
+F 3 "~" H 7950 4850 50  0001 C CNN
+F 4 "" H 7950 4850 50  0001 C CNN "LCSC"
+F 5 "" H 7950 4850 50  0001 C CNN "Price"
+F 6 "-" H 7950 4850 50  0001 C CNN "Mouser"
+F 7 "N" H 7950 4850 50  0001 C CNN "Sponsored"
+	1    7950 4850
+	1    0    0    -1
+$EndComp
 Text HLabel 8050 4400 2    50   Output ~ 0
 ESP32_RX
@@
 Text GLabel 2700 4200 0    50   BiDi ~ 0
 SAO_IO2
+$Comp
+L Connector:TestPoint TP14
+U 1 1 6173E651
+P 2700 5000
+F 0 "TP14" H 2642 5026 50  0000 R CNN
+F 1 "UNUSED PIN" H 2642 5117 50  0000 R CNN
+F 2 "TestPoint:TestPoint_Pad_1.0x1.0mm" H 2900 5000 50  0001 C CNN
+F 3 "~" H 2900 5000 50  0001 C CNN
+	1    2700 5000
+	-1   0    0    1
+$EndComp
+$Comp
+L Device:R_Small R?
+U 1 1 61BC9ED7
+P 7800 4600
+AR Path="/61BC9ED7" Ref="R?"  Part="1"
+AR Path="/5F51E414/61BC9ED7" Ref="R6"  Part="1"
+F 0 "R6" V 7750 4450 50  0000 C CNN
+F 1 "22" V 7800 4600 35  0000 C CNN
+F 2 "Resistor_SMD:R_0402_1005Metric" H 7800 4600 50  0001 C CNN
+F 3 "~" H 7800 4600 50  0001 C CNN
+F 4 "" H 7800 4600 50  0001 C CNN "Price"
+F 5 "C103086" H 7800 4600 50  0001 C CNN "LCSC"
+F 6 "-" H 7800 4600 50  0001 C CNN "Mouser"
+F 7 "N" H 7800 4600 50  0001 C CNN "Sponsored"
+	1    7800 4600
+	0    1    1    0
+$EndComp
+$Comp
+L Device:R_Small R?
+U 1 1 61BC9EE1
+P 7800 4700
+AR Path="/61BC9EE1" Ref="R?"  Part="1"
+AR Path="/5F51E414/61BC9EE1" Ref="R7"  Part="1"
+F 0 "R7" V 7850 4850 50  0000 C CNN
+F 1 "22" V 7800 4700 35  0000 C CNN
+F 2 "Resistor_SMD:R_0402_1005Metric" H 7800 4700 50  0001 C CNN
+F 3 "~" H 7800 4700 50  0001 C CNN
+F 4 "" H 7800 4700 50  0001 C CNN "Price"
+F 5 "C103086" H 7800 4700 50  0001 C CNN "LCSC"
+F 6 "-" H 7800 4700 50  0001 C CNN "Mouser"
+F 7 "N" H 7800 4700 50  0001 C CNN "Sponsored"
+	1    7800 4700
+	0    -1   -1   0
+$EndComp
+Wire Wire Line
+	7900 4600 8050 4600
+Wire Wire Line
+	7900 4700 7950 4700
+Connection ~ 7950 4700
+Wire Wire Line
+	7950 4700 8050 4700
+Wire Wire Line
+	6650 5000 7950 5000
+Wire Wire Line
+	6650 4700 7700 4700
 $EndSCHEMATC
