File: accelerometer.sch (KiCad schematic (older format))
At the start: 6 parts, among them U7 MPU-6050

Commit message: Small fixes
Parts:
- added C40: 100n, Capacitor_SMD:C_0603_1608Metric, symbol Device:C_Small
- added C41: 10u, Capacitor_SMD:C_0603_1608Metric, symbol Device:C_Small
Connections:
- net +3V3: now also C40.1, C41.1
- net GND: now also C40.2, C41.2
Changed lines of the file:
@@
 $Descr A4 11693 8268
 encoding utf-8
-Sheet 5 10
+Sheet 3 10
 Title ""
 Date ""
@@
 Wire Wire Line
 	6850 4000 7000 4000
+$Comp
+L Device:C_Small C41
+U 1 1 5F345F18
+P 10900 6200
+F 0 "C41" H 10992 6246 50  0000 L CNN
+F 1 "10u" H 10992 6155 50  0000 L CNN
+F 2 "Capacitor_SMD:C_0603_1608Metric" H 10900 6200 50  0001 C CNN
+F 3 "~" H 10900 6200 50  0001 C CNN
+	1    10900 6200
+	1    0    0    -1
+$EndComp
+$Comp
+L Device:C_Small C40
+U 1 1 5F34624F
+P 10550 6200
+F 0 "C40" H 10642 6246 50  0000 L CNN
+F 1 "100n" H 10642 6155 50  0000 L CNN
+F 2 "Capacitor_SMD:C_0603_1608Metric" H 10550 6200 50  0001 C CNN
+F 3 "~" H 10550 6200 50  0001 C CNN
+	1    10550 6200
+	1    0    0    -1
+$EndComp
+$Comp
+L power:GND #PWR0160
+U 1 1 5F347135
+P 10900 6300
+F 0 "#PWR0160" H 10900 6050 50  0001 C CNN
+F 1 "GND" H 10905 6127 50  0000 C CNN
+F 2 "" H 10900 6300 50  0001 C CNN
+F 3 "" H 10900 6300 50  0001 C CNN
+	1    10900 6300
+	1    0    0    -1
+$EndComp
+$Comp
+L power:GND #PWR0161
+U 1 1 5F34742D
+P 10550 6300
+F 0 "#PWR0161" H 10550 6050 50  0001 C CNN
+F 1 "GND" H 10555 6127 50  0000 C CNN
+F 2 "" H 10550 6300 50  0001 C CNN
+F 3 "" H 10550 6300 50  0001 C CNN
+	1    10550 6300
+	1    0    0    -1
+$EndComp
+$Comp
+L power:+3.3V #PWR0162
+U 1 1 5F349445
+P 10900 6100
+F 0 "#PWR0162" H 10900 5950 50  0001 C CNN
+F 1 "+3.3V" V 10915 6228 50  0000 L CNN
+F 2 "" H 10900 6100 50  0001 C CNN
+F 3 "" H 10900 6100 50  0001 C CNN
+	1    10900 6100
+	1    0    0    -1
+$EndComp
+$Comp
+L power:+3.3V #PWR0163
+U 1 1 5F349A13
+P 10550 6100
+F 0 "#PWR0163" H 10550 5950 50  0001 C CNN
+F 1 "+3.3V" V 10565 6228 50  0000 L CNN
+F 2 "" H 10550 6100 50  0001 C CNN
+F 3 "" H 10550 6100 50  0001 C CNN
+	1    10550 6100
+	1    0    0    -1
+$EndComp
 $EndSCHEMATC

Commit message: Dump.
Parts:
- added R17: 4k7, Resistor_SMD:R_0603_1608Metric, symbol Device:R_Small
- C17, C18: LCSC (none) -> C14663; Mouser (none) -> -; Price (none) -> 0.0020; Sponsored (none) -> N
- C19: Price (none) -> 0.0020; Sponsored (none) -> N
- C20: renamed from C40; LCSC (none) -> C14663; Mouser (none) -> -; Price (none) -> 0.0020; Sponsored (none) -> N
- C21: renamed from C41; Price (none) -> 0.0020; Sponsored (none) -> N
- R15: renamed from R17; footprint (none) -> Resistor_SMD:R_0603_1608Metric; LCSC (none) -> -; Mouser (none) -> -; Price (none) -> 0.0005; Sponsored (none) -> N
- R16: renamed from R18; footprint (none) -> Resistor_SMD:R_0603_1608Metric; LCSC (none) -> -; Mouser (none) -> -; Price (none) -> 0.0005; Sponsored (none) -> N
- U7: LCSC (none) -> C24112; Mouser (none) -> -; Price (none) -> 1.27; Sponsored (none) -> N
Connections:
- net +3V3: now also R17.1
- net IRQ: now also R17.2
Changed lines of the file:
@@
 $EndDescr
 $Comp
-L power:+3.3V #PWR078
+L power:+3.3V #PWR079
 U 1 1 5FC7218B
 P 5850 3300
-F 0 "#PWR078" H 5850 3150 50  0001 C CNN
+F 0 "#PWR079" H 5850 3150 50  0001 C CNN
 F 1 "+3.3V" V 5865 3428 50  0000 L CNN
 F 2 "" H 5850 3300 50  0001 C CNN
@@
 F 2 "Capacitor_SMD:C_0603_1608Metric" H 6600 4550 50  0001 C CNN
 F 3 "~" H 6600 4550 50  0001 C CNN
+F 4 "0.0020" H 6600 4550 50  0001 C CNN "Price"
+F 5 "N" H 6600 4550 50  0001 C CNN "Sponsored"
 	1    6600 4550
 	1    0    0    1
@@
 F 2 "Capacitor_SMD:C_0603_1608Metric" H 6450 4550 50  0001 C CNN
 F 3 "~" H 6450 4550 50  0001 C CNN
+F 4 "C14663" H 6450 4550 50  0001 C CNN "LCSC"
+F 5 "0.0020" H 6450 4550 50  0001 C CNN "Price"
+F 6 "-" H 6450 4550 50  0001 C CNN "Mouser"
+F 7 "N" H 6450 4550 50  0001 C CNN "Sponsored"
 	1    6450 4550
 	-1   0    0    1
@@
 	6600 4200 6600 4450
 $Comp
-L power:GND #PWR081
+L power:GND #PWR082
 U 1 1 605756E7
 P 6600 4700
-F 0 "#PWR081" H 6600 4450 50  0001 C CNN
+F 0 "#PWR082" H 6600 4450 50  0001 C CNN
 F 1 "GND" H 6605 4527 50  0000 C CNN
 F 2 "" H 6600 4700 50  0001 C CNN
@@
 $EndComp
 $Comp
-L power:GND #PWR079
+L power:GND #PWR080
 U 1 1 605756E8
 P 6450 4700
-F 0 "#PWR079" H 6450 4450 50  0001 C CNN
+F 0 "#PWR080" H 6450 4450 50  0001 C CNN
 F 1 "GND" H 6455 4527 50  0000 C CNN
 F 2 "" H 6450 4700 50  0001 C CNN
@@
 $EndComp
 $Comp
-L power:GND #PWR077
+L power:GND #PWR078
 U 1 1 60534309
 P 5750 4700
-F 0 "#PWR077" H 5750 4450 50  0001 C CNN
+F 0 "#PWR078" H 5750 4450 50  0001 C CNN
 F 1 "GND" H 5755 4527 50  0000 C CNN
 F 2 "" H 5750 4700 50  0001 C CNN
@@
 	6450 4700 6450 4650
 $Comp
-L power:GND #PWR075
+L power:GND #PWR076
 U 1 1 6053430A
 P 5050 4700
-F 0 "#PWR075" H 5050 4450 50  0001 C CNN
+F 0 "#PWR076" H 5050 4450 50  0001 C CNN
 F 1 "GND" H 5055 4527 50  0000 C CNN
 F 2 "" H 5050 4700 50  0001 C CNN
@@
 $EndComp
 $Comp
-L power:+3.3V #PWR076
+L power:+3.3V #PWR077
 U 1 1 605756D6
 P 5650 3300
-F 0 "#PWR076" H 5650 3150 50  0001 C CNN
+F 0 "#PWR077" H 5650 3150 50  0001 C CNN
 F 1 "+3.3V" V 5665 3428 50  0000 L CNN
 F 2 "" H 5650 3300 50  0001 C CNN
@@
 F 2 "Capacitor_SMD:C_0603_1608Metric" H 4700 4550 50  0001 C CNN
 F 3 "~" H 4700 4550 50  0001 C CNN
+F 4 "C14663" H 4700 4550 50  0001 C CNN "LCSC"
+F 5 "0.0020" H 4700 4550 50  0001 C CNN "Price"
+F 6 "-" H 4700 4550 50  0001 C CNN "Mouser"
+F 7 "N" H 4700 4550 50  0001 C CNN "Sponsored"
 	1    4700 4550
 	1    0    0    -1
 $EndComp
 $Comp
-L power:GND #PWR074
+L power:GND #PWR075
 U 1 1 605756D7
 P 4700 4700
-F 0 "#PWR074" H 4700 4450 50  0001 C CNN
+F 0 "#PWR075" H 4700 4450 50  0001 C CNN
 F 1 "GND" H 4705 4527 50  0000 C CNN
 F 2 "" H 4700 4700 50  0001 C CNN
@@
 	4700 4700 4700 4650
 $Comp
-L power:+3.3V #PWR073
+L power:+3.3V #PWR074
 U 1 1 605756D8
 P 4700 3300
-F 0 "#PWR073" H 4700 3150 50  0001 C CNN
+F 0 "#PWR074" H 4700 3150 50  0001 C CNN
 F 1 "+3.3V" V 4715 3428 50  0000 L CNN
 F 2 "" H 4700 3300 50  0001 C CNN
@@
 F 2 "Sensor_Motion:InvenSense_QFN-24_4x4mm_P0.5mm" H 5750 3200 50  0001 C CNN
 F 3 "https://store.invensense.com/datasheets/invensense/MPU-6050_DataSheet_V3%204.pdf" H 5750 3850 50  0001 C CNN
+F 4 "C24112" H 5750 4000 50  0001 C CNN "LCSC"
+F 5 "-" H 5750 4000 50  0001 C CNN "Mouser"
+F 6 "1.27" H 5750 4000 50  0001 C CNN "Price"
+F 7 "N" H 5750 4000 50  0001 C CNN "Sponsored"
 	1    5750 4000
 	1    0    0    -1
@@
 Wire Wire Line
 	4700 3300 4700 4450
-Text HLabel 7000 3700 2    39   Output ~ 0
+Text HLabel 7250 3700 2    39   Output ~ 0
 IRQ
-Text HLabel 7000 3900 2    39   3State ~ 0
+Text HLabel 7250 3900 2    39   3State ~ 0
 AUX_SDA
-Text HLabel 7000 4000 2    39   Output ~ 0
+Text HLabel 7250 4000 2    39   Output ~ 0
 AUX_SCL
 $Comp
-L Device:R_Small R17
+L Device:R_Small R15
 U 1 1 605967DC
 P 6550 3400
-F 0 "R17" H 6609 3446 50  0000 L CNN
+F 0 "R15" H 6609 3446 50  0000 L CNN
 F 1 "4k7" H 6609 3355 50  0000 L CNN
-F 2 "" H 6550 3400 50  0001 C CNN
+F 2 "Resistor_SMD:R_0603_1608Metric" H 6550 3400 50  0001 C CNN
 F 3 "~" H 6550 3400 50  0001 C CNN
+F 4 "0.0005" H 6550 3400 50  0001 C CNN "Price"
+F 5 "-" H 6550 3400 50  0001 C CNN "LCSC"
+F 6 "-" H 6550 3400 50  0001 C CNN "Mouser"
+F 7 "N" H 6550 3400 50  0001 C CNN "Sponsored"
 	1    6550 3400
 	1    0    0    -1
 $EndComp
 $Comp
-L power:+3.3V #PWR080
+L power:+3.3V #PWR081
 U 1 1 6059915F
 P 6550 3300
-F 0 "#PWR080" H 6550 3150 50  0001 C CNN
+F 0 "#PWR081" H 6550 3150 50  0001 C CNN
 F 1 "+3.3V" V 6565 3428 50  0000 L CNN
 F 2 "" H 6550 3300 50  0001 C CNN
@@
 $EndComp
 $Comp
-L Device:R_Small R18
+L Device:R_Small R16
 U 1 1 6059D815
 P 6850 3400
-F 0 "R18" H 6909 3446 50  0000 L CNN
+F 0 "R16" H 6909 3446 50  0000 L CNN
 F 1 "4k7" H 6909 3355 50  0000 L CNN
-F 2 "" H 6850 3400 50  0001 C CNN
+F 2 "Resistor_SMD:R_0603_1608Metric" H 6850 3400 50  0001 C CNN
 F 3 "~" H 6850 3400 50  0001 C CNN
+F 4 "0.0005" H 6850 3400 50  0001 C CNN "Price"
+F 5 "-" H 6850 3400 50  0001 C CNN "LCSC"
+F 6 "-" H 6850 3400 50  0001 C CNN "Mouser"
+F 7 "N" H 6850 3400 50  0001 C CNN "Sponsored"
 	1    6850 3400
 	1    0    0    -1
 $EndComp
 $Comp
-L power:+3.3V #PWR082
+L power:+3.3V #PWR083
 U 1 1 6059D81B
 P 6850 3300
-F 0 "#PWR082" H 6850 3150 50  0001 C CNN
+F 0 "#PWR083" H 6850 3150 50  0001 C CNN
 F 1 "+3.3V" V 6865 3428 50  0000 L CNN
 F 2 "" H 6850 3300 50  0001 C CNN
@@
 $EndComp
 Wire Wire Line
-	7000 3700 6450 3700
-Wire Wire Line
 	6450 3900 6550 3900
 Wire Wire Line
@@
 Connection ~ 6550 3900
 Wire Wire Line
-	6550 3900 7000 3900
-Wire Wire Line
 	6850 3500 6850 4000
 Connection ~ 6850 4000
-Wire Wire Line
-	6850 4000 7000 4000
-$Comp
-L Device:C_Small C41
+$Comp
+L Device:C_Small C21
 U 1 1 5F345F18
 P 10900 6200
-F 0 "C41" H 10992 6246 50  0000 L CNN
+F 0 "C21" H 10992 6246 50  0000 L CNN
 F 1 "10u" H 10992 6155 50  0000 L CNN
 F 2 "Capacitor_SMD:C_0603_1608Metric" H 10900 6200 50  0001 C CNN
 F 3 "~" H 10900 6200 50  0001 C CNN
+F 4 "0.0020" H 10900 6200 50  0001 C CNN "Price"
+F 5 "N" H 10900 6200 50  0001 C CNN "Sponsored"
 	1    10900 6200
 	1    0    0    -1
 $EndComp
 $Comp
-L Device:C_Small C40
+L Device:C_Small C20
 U 1 1 5F34624F
 P 10550 6200
-F 0 "C40" H 10642 6246 50  0000 L CNN
+F 0 "C20" H 10642 6246 50  0000 L CNN
 F 1 "100n" H 10642 6155 50  0000 L CNN
 F 2 "Capacitor_SMD:C_0603_1608Metric" H 10550 6200 50  0001 C CNN
 F 3 "~" H 10550 6200 50  0001 C CNN
+F 4 "C14663" H 10550 6200 50  0001 C CNN "LCSC"
+F 5 "0.0020" H 10550 6200 50  0001 C CNN "Price"
+F 6 "-" H 10550 6200 50  0001 C CNN "Mouser"
+F 7 "N" H 10550 6200 50  0001 C CNN "Sponsored"
 	1    10550 6200
 	1    0    0    -1
 $EndComp
 $Comp
-L power:GND #PWR0160
+L power:GND #PWR087
 U 1 1 5F347135
 P 10900 6300
-F 0 "#PWR0160" H 10900 6050 50  0001 C CNN
+F 0 "#PWR087" H 10900 6050 50  0001 C CNN
 F 1 "GND" H 10905 6127 50  0000 C CNN
 F 2 "" H 10900 6300 50  0001 C CNN
@@
 $EndComp
 $Comp
-L power:GND #PWR0161
+L power:GND #PWR085
 U 1 1 5F34742D
 P 10550 6300
-F 0 "#PWR0161" H 10550 6050 50  0001 C CNN
+F 0 "#PWR085" H 10550 6050 50  0001 C CNN
 F 1 "GND" H 10555 6127 50  0000 C CNN
 F 2 "" H 10550 6300 50  0001 C CNN
@@
 $EndComp
 $Comp
-L power:+3.3V #PWR0162
+L power:+3.3V #PWR086
 U 1 1 5F349445
 P 10900 6100
-F 0 "#PWR0162" H 10900 5950 50  0001 C CNN
+F 0 "#PWR086" H 10900 5950 50  0001 C CNN
 F 1 "+3.3V" V 10915 6228 50  0000 L CNN
 F 2 "" H 10900 6100 50  0001 C CNN
@@
 $EndComp
 $Comp
-L power:+3.3V #PWR0163
+L power:+3.3V #PWR084
 U 1 1 5F349A13
 P 10550 6100
-F 0 "#PWR0163" H 10550 5950 50  0001 C CNN
+F 0 "#PWR084" H 10550 5950 50  0001 C CNN
 F 1 "+3.3V" V 10565 6228 50  0000 L CNN
 F 2 "" H 10550 6100 50  0001 C CNN
@@
 	1    0    0    -1
 $EndComp
+$Comp
+L Device:R_Small R17
+U 1 1 5F484279
+P 7150 3400
+F 0 "R17" H 7209 3446 50  0000 L CNN
+F 1 "4k7" H 7209 3355 50  0000 L CNN
+F 2 "Resistor_SMD:R_0603_1608Metric" H 7150 3400 50  0001 C CNN
+F 3 "~" H 7150 3400 50  0001 C CNN
+F 4 "0.0005" H 7150 3400 50  0001 C CNN "Price"
+F 5 "-" H 7150 3400 50  0001 C CNN "LCSC"
+F 6 "-" H 7150 3400 50  0001 C CNN "Mouser"
+F 7 "N" H 7150 3400 50  0001 C CNN "Sponsored"
+	1    7150 3400
+	1    0    0    -1
+$EndComp
+Wire Wire Line
+	6450 3700 7150 3700
+Wire Wire Line
+	7150 3500 7150 3700
+Connection ~ 7150 3700
+Wire Wire Line
+	7150 3700 7250 3700
+$Comp
+L power:+3.3V #PWR0103
+U 1 1 5F4853B8
+P 7150 3300
+F 0 "#PWR0103" H 7150 3150 50  0001 C CNN
+F 1 "+3.3V" V 7165 3428 50  0000 L CNN
+F 2 "" H 7150 3300 50  0001 C CNN
+F 3 "" H 7150 3300 50  0001 C CNN
+	1    7150 3300
+	1    0    0    -1
+$EndComp
+Wire Wire Line
+	6550 3900 7250 3900
+Wire Wire Line
+	6850 4000 7250 4000
 $EndSCHEMATC

Commit message: Dump.
Parts:
- renumbered C17 to C16, C18 to C17, C19 to C18, C20 to C19, C21 to C20, R15 to R16, R16 to R17, R17 to R18, U7 to U6
Changed lines of the file:
@@
 $EndDescr
 $Comp
-L power:+3.3V #PWR079
+L power:+3.3V #PWR076
 U 1 1 5FC7218B
 P 5850 3300
-F 0 "#PWR079" H 5850 3150 50  0001 C CNN
+F 0 "#PWR076" H 5850 3150 50  0001 C CNN
 F 1 "+3.3V" V 5865 3428 50  0000 L CNN
 F 2 "" H 5850 3300 50  0001 C CNN
@@
 $EndComp
 $Comp
-L Device:C_Small C19
+L Device:C_Small C18
 U 1 1 5FC7218C
 P 6600 4550
-F 0 "C19" H 6600 4450 50  0000 L CNN
+F 0 "C18" H 6600 4450 50  0000 L CNN
 F 1 "2.2n" H 6600 4650 50  0000 L CNN
 F 2 "Capacitor_SMD:C_0603_1608Metric" H 6600 4550 50  0001 C CNN
@@
 $EndComp
 $Comp
-L Device:C_Small C18
+L Device:C_Small C17
 U 1 1 605756F6
 P 6450 4550
-F 0 "C18" H 6450 4450 50  0000 L CNN
+F 0 "C17" H 6450 4450 50  0000 L CNN
 F 1 "100n" H 6450 4650 50  0000 L CNN
 F 2 "Capacitor_SMD:C_0603_1608Metric" H 6450 4550 50  0001 C CNN
@@
 	6600 4200 6600 4450
 $Comp
-L power:GND #PWR082
+L power:GND #PWR079
 U 1 1 605756E7
 P 6600 4700
-F 0 "#PWR082" H 6600 4450 50  0001 C CNN
+F 0 "#PWR079" H 6600 4450 50  0001 C CNN
 F 1 "GND" H 6605 4527 50  0000 C CNN
 F 2 "" H 6600 4700 50  0001 C CNN
@@
 $EndComp
 $Comp
-L power:GND #PWR080
+L power:GND #PWR077
 U 1 1 605756E8
 P 6450 4700
-F 0 "#PWR080" H 6450 4450 50  0001 C CNN
+F 0 "#PWR077" H 6450 4450 50  0001 C CNN
 F 1 "GND" H 6455 4527 50  0000 C CNN
 F 2 "" H 6450 4700 50  0001 C CNN
@@
 $EndComp
 $Comp
-L power:GND #PWR078
+L power:GND #PWR075
 U 1 1 60534309
 P 5750 4700
-F 0 "#PWR078" H 5750 4450 50  0001 C CNN
+F 0 "#PWR075" H 5750 4450 50  0001 C CNN
 F 1 "GND" H 5755 4527 50  0000 C CNN
 F 2 "" H 5750 4700 50  0001 C CNN
@@
 	6450 4700 6450 4650
 $Comp
-L power:GND #PWR076
+L power:GND #PWR073
 U 1 1 6053430A
 P 5050 4700
-F 0 "#PWR076" H 5050 4450 50  0001 C CNN
+F 0 "#PWR073" H 5050 4450 50  0001 C CNN
 F 1 "GND" H 5055 4527 50  0000 C CNN
 F 2 "" H 5050 4700 50  0001 C CNN
@@
 $EndComp
 $Comp
-L power:+3.3V #PWR077
+L power:+3.3V #PWR074
 U 1 1 605756D6
 P 5650 3300
-F 0 "#PWR077" H 5650 3150 50  0001 C CNN
+F 0 "#PWR074" H 5650 3150 50  0001 C CNN
 F 1 "+3.3V" V 5665 3428 50  0000 L CNN
 F 2 "" H 5650 3300 50  0001 C CNN
@@
 $EndComp
 $Comp
-L Device:C_Small C17
+L Device:C_Small C16
 U 1 1 5FC72193
 P 4700 4550
-F 0 "C17" H 4792 4596 50  0000 L CNN
+F 0 "C16" H 4792 4596 50  0000 L CNN
 F 1 "100n" H 4792 4505 50  0000 L CNN
 F 2 "Capacitor_SMD:C_0603_1608Metric" H 4700 4550 50  0001 C CNN
@@
 $EndComp
 $Comp
-L power:GND #PWR075
+L power:GND #PWR072
 U 1 1 605756D7
 P 4700 4700
-F 0 "#PWR075" H 4700 4450 50  0001 C CNN
+F 0 "#PWR072" H 4700 4450 50  0001 C CNN
 F 1 "GND" H 4705 4527 50  0000 C CNN
 F 2 "" H 4700 4700 50  0001 C CNN
@@
 	4700 4700 4700 4650
 $Comp
-L power:+3.3V #PWR074
+L power:+3.3V #PWR071
 U 1 1 605756D8
 P 4700 3300
-F 0 "#PWR074" H 4700 3150 50  0001 C CNN
+F 0 "#PWR071" H 4700 3150 50  0001 C CNN
 F 1 "+3.3V" V 4715 3428 50  0000 L CNN
 F 2 "" H 4700 3300 50  0001 C CNN
@@
 Connection ~ 5050 4300
 $Comp
-L Sensor_Motion:MPU-6050 U7
+L Sensor_Motion:MPU-6050 U6
 U 1 1 605756E6
 P 5750 4000
-F 0 "U7" H 5300 4550 50  0000 C CNN
+F 0 "U6" H 5300 4550 50  0000 C CNN
 F 1 "MPU-6050" H 5650 4000 50  0000 C CNN
 F 2 "Sensor_Motion:InvenSense_QFN-24_4x4mm_P0.5mm" H 5750 3200 50  0001 C CNN
@@
 AUX_SCL
 $Comp
-L Device:R_Small R15
+L Device:R_Small R16
 U 1 1 605967DC
 P 6550 3400
-F 0 "R15" H 6609 3446 50  0000 L CNN
+F 0 "R16" H 6609 3446 50  0000 L CNN
 F 1 "4k7" H 6609 3355 50  0000 L CNN
 F 2 "Resistor_SMD:R_0603_1608Metric" H 6550 3400 50  0001 C CNN
@@
 $EndComp
 $Comp
-L power:+3.3V #PWR081
+L power:+3.3V #PWR078
 U 1 1 6059915F
 P 6550 3300
-F 0 "#PWR081" H 6550 3150 50  0001 C CNN
+F 0 "#PWR078" H 6550 3150 50  0001 C CNN
 F 1 "+3.3V" V 6565 3428 50  0000 L CNN
 F 2 "" H 6550 3300 50  0001 C CNN
@@
 $EndComp
 $Comp
-L Device:R_Small R16
+L Device:R_Small R17
 U 1 1 6059D815
 P 6850 3400
-F 0 "R16" H 6909 3446 50  0000 L CNN
+F 0 "R17" H 6909 3446 50  0000 L CNN
 F 1 "4k7" H 6909 3355 50  0000 L CNN
 F 2 "Resistor_SMD:R_0603_1608Metric" H 6850 3400 50  0001 C CNN
@@
 $EndComp
 $Comp
-L power:+3.3V #PWR083
+L power:+3.3V #PWR080
 U 1 1 6059D81B
 P 6850 3300
-F 0 "#PWR083" H 6850 3150 50  0001 C CNN
+F 0 "#PWR080" H 6850 3150 50  0001 C CNN
 F 1 "+3.3V" V 6865 3428 50  0000 L CNN
 F 2 "" H 6850 3300 50  0001 C CNN
@@
 Connection ~ 6850 4000
 $Comp
-L Device:C_Small C21
+L Device:C_Small C20
 U 1 1 5F345F18
 P 10900 6200
-F 0 "C21" H 10992 6246 50  0000 L CNN
+F 0 "C20" H 10992 6246 50  0000 L CNN
 F 1 "10u" H 10992 6155 50  0000 L CNN
 F 2 "Capacitor_SMD:C_0603_1608Metric" H 10900 6200 50  0001 C CNN
@@
 $EndComp
 $Comp
-L Device:C_Small C20
+L Device:C_Small C19
 U 1 1 5F34624F
 P 10550 6200
-F 0 "C20" H 10642 6246 50  0000 L CNN
+F 0 "C19" H 10642 6246 50  0000 L CNN
 F 1 "100n" H 10642 6155 50  0000 L CNN
 F 2 "Capacitor_SMD:C_0603_1608Metric" H 10550 6200 50  0001 C CNN
@@
 $EndComp
 $Comp
-L power:GND #PWR087
+L power:GND #PWR085
 U 1 1 5F347135
 P 10900 6300
-F 0 "#PWR087" H 10900 6050 50  0001 C CNN
+F 0 "#PWR085" H 10900 6050 50  0001 C CNN
 F 1 "GND" H 10905 6127 50  0000 C CNN
 F 2 "" H 10900 6300 50  0001 C CNN
@@
 $EndComp
 $Comp
-L power:GND #PWR085
+L power:GND #PWR083
 U 1 1 5F34742D
 P 10550 6300
-F 0 "#PWR085" H 10550 6050 50  0001 C CNN
+F 0 "#PWR083" H 10550 6050 50  0001 C CNN
 F 1 "GND" H 10555 6127 50  0000 C CNN
 F 2 "" H 10550 6300 50  0001 C CNN
@@
 $EndComp
 $Comp
-L power:+3.3V #PWR086
+L power:+3.3V #PWR084
 U 1 1 5F349445
 P 10900 6100
-F 0 "#PWR086" H 10900 5950 50  0001 C CNN
+F 0 "#PWR084" H 10900 5950 50  0001 C CNN
 F 1 "+3.3V" V 10915 6228 50  0000 L CNN
 F 2 "" H 10900 6100 50  0001 C CNN
@@
 $EndComp
 $Comp
-L power:+3.3V #PWR084
+L power:+3.3V #PWR082
 U 1 1 5F349A13
 P 10550 6100
-F 0 "#PWR084" H 10550 5950 50  0001 C CNN
+F 0 "#PWR082" H 10550 5950 50  0001 C CNN
 F 1 "+3.3V" V 10565 6228 50  0000 L CNN
 F 2 "" H 10550 6100 50  0001 C CNN
@@
 $EndComp
 $Comp
-L Device:R_Small R17
+L Device:R_Small R18
 U 1 1 5F484279
 P 7150 3400
-F 0 "R17" H 7209 3446 50  0000 L CNN
+F 0 "R18" H 7209 3446 50  0000 L CNN
 F 1 "4k7" H 7209 3355 50  0000 L CNN
 F 2 "Resistor_SMD:R_0603_1608Metric" H 7150 3400 50  0001 C CNN
@@
 	7150 3700 7250 3700
 $Comp
-L power:+3.3V #PWR0103
+L power:+3.3V #PWR081
 U 1 1 5F4853B8
 P 7150 3300
-F 0 "#PWR0103" H 7150 3150 50  0001 C CNN
+F 0 "#PWR081" H 7150 3150 50  0001 C CNN
 F 1 "+3.3V" V 7165 3428 50  0000 L CNN
 F 2 "" H 7150 3300 50  0001 C CNN

Commit message: Dump.
Parts:
- renumbered R16 to R15, R17 to R16, R18 to R17
Changed lines of the file:
@@
 $EndDescr
 $Comp
-L power:+3.3V #PWR076
+L power:+3.3V #PWR075
 U 1 1 5FC7218B
 P 5850 3300
-F 0 "#PWR076" H 5850 3150 50  0001 C CNN
+F 0 "#PWR075" H 5850 3150 50  0001 C CNN
 F 1 "+3.3V" V 5865 3428 50  0000 L CNN
 F 2 "" H 5850 3300 50  0001 C CNN
@@
 	6600 4200 6600 4450
 $Comp
-L power:GND #PWR079
+L power:GND #PWR078
 U 1 1 605756E7
 P 6600 4700
-F 0 "#PWR079" H 6600 4450 50  0001 C CNN
+F 0 "#PWR078" H 6600 4450 50  0001 C CNN
 F 1 "GND" H 6605 4527 50  0000 C CNN
 F 2 "" H 6600 4700 50  0001 C CNN
@@
 $EndComp
 $Comp
-L power:GND #PWR077
+L power:GND #PWR076
 U 1 1 605756E8
 P 6450 4700
-F 0 "#PWR077" H 6450 4450 50  0001 C CNN
+F 0 "#PWR076" H 6450 4450 50  0001 C CNN
 F 1 "GND" H 6455 4527 50  0000 C CNN
 F 2 "" H 6450 4700 50  0001 C CNN
@@
 $EndComp
 $Comp
-L power:GND #PWR075
+L power:GND #PWR074
 U 1 1 60534309
 P 5750 4700
-F 0 "#PWR075" H 5750 4450 50  0001 C CNN
+F 0 "#PWR074" H 5750 4450 50  0001 C CNN
 F 1 "GND" H 5755 4527 50  0000 C CNN
 F 2 "" H 5750 4700 50  0001 C CNN
@@
 	6450 4700 6450 4650
 $Comp
-L power:GND #PWR073
+L power:GND #PWR072
 U 1 1 6053430A
 P 5050 4700
-F 0 "#PWR073" H 5050 4450 50  0001 C CNN
+F 0 "#PWR072" H 5050 4450 50  0001 C CNN
 F 1 "GND" H 5055 4527 50  0000 C CNN
 F 2 "" H 5050 4700 50  0001 C CNN
@@
 $EndComp
 $Comp
-L power:+3.3V #PWR074
+L power:+3.3V #PWR073
 U 1 1 605756D6
 P 5650 3300
-F 0 "#PWR074" H 5650 3150 50  0001 C CNN
+F 0 "#PWR073" H 5650 3150 50  0001 C CNN
 F 1 "+3.3V" V 5665 3428 50  0000 L CNN
 F 2 "" H 5650 3300 50  0001 C CNN
@@
 $EndComp
 $Comp
-L power:GND #PWR072
+L power:GND #PWR071
 U 1 1 605756D7
 P 4700 4700
-F 0 "#PWR072" H 4700 4450 50  0001 C CNN
+F 0 "#PWR071" H 4700 4450 50  0001 C CNN
 F 1 "GND" H 4705 4527 50  0000 C CNN
 F 2 "" H 4700 4700 50  0001 C CNN
@@
 	4700 4700 4700 4650
 $Comp
-L power:+3.3V #PWR071
+L power:+3.3V #PWR070
 U 1 1 605756D8
 P 4700 3300
-F 0 "#PWR071" H 4700 3150 50  0001 C CNN
+F 0 "#PWR070" H 4700 3150 50  0001 C CNN
 F 1 "+3.3V" V 4715 3428 50  0000 L CNN
 F 2 "" H 4700 3300 50  0001 C CNN
@@
 AUX_SCL
 $Comp
-L Device:R_Small R16
+L Device:R_Small R15
 U 1 1 605967DC
 P 6550 3400
-F 0 "R16" H 6609 3446 50  0000 L CNN
+F 0 "R15" H 6609 3446 50  0000 L CNN
 F 1 "4k7" H 6609 3355 50  0000 L CNN
 F 2 "Resistor_SMD:R_0603_1608Metric" H 6550 3400 50  0001 C CNN
@@
 $EndComp
 $Comp
-L power:+3.3V #PWR078
+L power:+3.3V #PWR077
 U 1 1 6059915F
 P 6550 3300
-F 0 "#PWR078" H 6550 3150 50  0001 C CNN
+F 0 "#PWR077" H 6550 3150 50  0001 C CNN
 F 1 "+3.3V" V 6565 3428 50  0000 L CNN
 F 2 "" H 6550 3300 50  0001 C CNN
@@
 $EndComp
 $Comp
-L Device:R_Small R17
+L Device:R_Small R16
 U 1 1 6059D815
 P 6850 3400
-F 0 "R17" H 6909 3446 50  0000 L CNN
+F 0 "R16" H 6909 3446 50  0000 L CNN
 F 1 "4k7" H 6909 3355 50  0000 L CNN
 F 2 "Resistor_SMD:R_0603_1608Metric" H 6850 3400 50  0001 C CNN
@@
 $EndComp
 $Comp
-L power:+3.3V #PWR080
+L power:+3.3V #PWR079
 U 1 1 6059D81B
 P 6850 3300
-F 0 "#PWR080" H 6850 3150 50  0001 C CNN
+F 0 "#PWR079" H 6850 3150 50  0001 C CNN
 F 1 "+3.3V" V 6865 3428 50  0000 L CNN
 F 2 "" H 6850 3300 50  0001 C CNN
@@
 $EndComp
 $Comp
-L power:GND #PWR085
+L power:GND #PWR084
 U 1 1 5F347135
 P 10900 6300
-F 0 "#PWR085" H 10900 6050 50  0001 C CNN
+F 0 "#PWR084" H 10900 6050 50  0001 C CNN
 F 1 "GND" H 10905 6127 50  0000 C CNN
 F 2 "" H 10900 6300 50  0001 C CNN
@@
 $EndComp
 $Comp
-L power:GND #PWR083
+L power:GND #PWR082
 U 1 1 5F34742D
 P 10550 6300
-F 0 "#PWR083" H 10550 6050 50  0001 C CNN
+F 0 "#PWR082" H 10550 6050 50  0001 C CNN
 F 1 "GND" H 10555 6127 50  0000 C CNN
 F 2 "" H 10550 6300 50  0001 C CNN
@@
 $EndComp
 $Comp
-L power:+3.3V #PWR084
+L power:+3.3V #PWR083
 U 1 1 5F349445
 P 10900 6100
-F 0 "#PWR084" H 10900 5950 50  0001 C CNN
+F 0 "#PWR083" H 10900 5950 50  0001 C CNN
 F 1 "+3.3V" V 10915 6228 50  0000 L CNN
 F 2 "" H 10900 6100 50  0001 C CNN
@@
 $EndComp
 $Comp
-L power:+3.3V #PWR082
+L power:+3.3V #PWR081
 U 1 1 5F349A13
 P 10550 6100
-F 0 "#PWR082" H 10550 5950 50  0001 C CNN
+F 0 "#PWR081" H 10550 5950 50  0001 C CNN
 F 1 "+3.3V" V 10565 6228 50  0000 L CNN
 F 2 "" H 10550 6100 50  0001 C CNN
@@
 $EndComp
 $Comp
-L Device:R_Small R18
+L Device:R_Small R17
 U 1 1 5F484279
 P 7150 3400
-F 0 "R18" H 7209 3446 50  0000 L CNN
+F 0 "R17" H 7209 3446 50  0000 L CNN
 F 1 "4k7" H 7209 3355 50  0000 L CNN
 F 2 "Resistor_SMD:R_0603_1608Metric" H 7150 3400 50  0001 C CNN
@@
 	7150 3700 7250 3700
 $Comp
-L power:+3.3V #PWR081
+L power:+3.3V #PWR080
 U 1 1 5F4853B8
 P 7150 3300
-F 0 "#PWR081" H 7150 3150 50  0001 C CNN
+F 0 "#PWR080" H 7150 3150 50  0001 C CNN
 F 1 "+3.3V" V 7165 3428 50  0000 L CNN
 F 2 "" H 7150 3300 50  0001 C CNN
