File: accelerometer.sch (KiCad schematic (older format))
At the start: 9 parts, among them U6 MPU-6050

Commit message: Dump.
Parts:
- C16, C17, C19: Price 0.0020 -> (none)
- C18: LCSC (none) -> C466783; Price 0.0020 -> (none)
- C20: LCSC (none) -> C307461; Price 0.0020 -> (none)
- R15, R16, R17: LCSC - -> C269694; Price 0.0005 -> (none)
- U6: Price 1.27 -> (none)
Changed lines of the file:
@@
 F 2 "Capacitor_SMD:C_0603_1608Metric" H 6600 4550 50  0001 C CNN
 F 3 "~" H 6600 4550 50  0001 C CNN
-F 4 "0.0020" H 6600 4550 50  0001 C CNN "Price"
+F 4 "" H 6600 4550 50  0001 C CNN "Price"
 F 5 "N" H 6600 4550 50  0001 C CNN "Sponsored"
+F 6 "C466783" H 6600 4550 50  0001 C CNN "LCSC"
 	1    6600 4550
 	1    0    0    1
@@
 F 3 "~" H 6450 4550 50  0001 C CNN
 F 4 "C14663" H 6450 4550 50  0001 C CNN "LCSC"
-F 5 "0.0020" H 6450 4550 50  0001 C CNN "Price"
+F 5 "" H 6450 4550 50  0001 C CNN "Price"
 F 6 "-" H 6450 4550 50  0001 C CNN "Mouser"
 F 7 "N" H 6450 4550 50  0001 C CNN "Sponsored"
@@
 F 3 "~" H 4700 4550 50  0001 C CNN
 F 4 "C14663" H 4700 4550 50  0001 C CNN "LCSC"
-F 5 "0.0020" H 4700 4550 50  0001 C CNN "Price"
+F 5 "" H 4700 4550 50  0001 C CNN "Price"
 F 6 "-" H 4700 4550 50  0001 C CNN "Mouser"
 F 7 "N" H 4700 4550 50  0001 C CNN "Sponsored"
@@
 F 4 "C24112" H 5750 4000 50  0001 C CNN "LCSC"
 F 5 "-" H 5750 4000 50  0001 C CNN "Mouser"
-F 6 "1.27" H 5750 4000 50  0001 C CNN "Price"
+F 6 "" H 5750 4000 50  0001 C CNN "Price"
 F 7 "N" H 5750 4000 50  0001 C CNN "Sponsored"
 	1    5750 4000
@@
 F 2 "Resistor_SMD:R_0603_1608Metric" H 6550 3400 50  0001 C CNN
 F 3 "~" H 6550 3400 50  0001 C CNN
-F 4 "0.0005" H 6550 3400 50  0001 C CNN "Price"
-F 5 "-" H 6550 3400 50  0001 C CNN "LCSC"
+F 4 "" H 6550 3400 50  0001 C CNN "Price"
+F 5 "C269694" H 6550 3400 50  0001 C CNN "LCSC"
 F 6 "-" H 6550 3400 50  0001 C CNN "Mouser"
 F 7 "N" H 6550 3400 50  0001 C CNN "Sponsored"
@@
 F 2 "Resistor_SMD:R_0603_1608Metric" H 6850 3400 50  0001 C CNN
 F 3 "~" H 6850 3400 50  0001 C CNN
-F 4 "0.0005" H 6850 3400 50  0001 C CNN "Price"
-F 5 "-" H 6850 3400 50  0001 C CNN "LCSC"
+F 4 "" H 6850 3400 50  0001 C CNN "Price"
+F 5 "C269694" H 6850 3400 50  0001 C CNN "LCSC"
 F 6 "-" H 6850 3400 50  0001 C CNN "Mouser"
 F 7 "N" H 6850 3400 50  0001 C CNN "Sponsored"
@@
 F 2 "Capacitor_SMD:C_0603_1608Metric" H 10900 6200 50  0001 C CNN
 F 3 "~" H 10900 6200 50  0001 C CNN
-F 4 "0.0020" H 10900 6200 50  0001 C CNN "Price"
+F 4 "" H 10900 6200 50  0001 C CNN "Price"
 F 5 "N" H 10900 6200 50  0001 C CNN "Sponsored"
+F 6 "C307461" H 10900 6200 50  0001 C CNN "LCSC"
 	1    10900 6200
 	1    0    0    -1
@@
 F 3 "~" H 10550 6200 50  0001 C CNN
 F 4 "C14663" H 10550 6200 50  0001 C CNN "LCSC"
-F 5 "0.0020" H 10550 6200 50  0001 C CNN "Price"
+F 5 "" H 10550 6200 50  0001 C CNN "Price"
 F 6 "-" H 10550 6200 50  0001 C CNN "Mouser"
 F 7 "N" H 10550 6200 50  0001 C CNN "Sponsored"
@@
 F 2 "Resistor_SMD:R_0603_1608Metric" H 7150 3400 50  0001 C CNN
 F 3 "~" H 7150 3400 50  0001 C CNN
-F 4 "0.0005" H 7150 3400 50  0001 C CNN "Price"
-F 5 "-" H 7150 3400 50  0001 C CNN "LCSC"
+F 4 "" H 7150 3400 50  0001 C CNN "Price"
+F 5 "C269694" H 7150 3400 50  0001 C CNN "LCSC"
 F 6 "-" H 7150 3400 50  0001 C CNN "Mouser"
 F 7 "N" H 7150 3400 50  0001 C CNN "Sponsored"
