File: esp32.sch (KiCad schematic (older format))
At the start: 18 parts, among them U13 ESP32-WROVER

Commit message: Dump.
Parts:
- renumbered R35 to R46, R36 to R47, R37 to R48, R38 to R49, R39 to R50, R40 to R51, R41 to R52, R42 to R53, R43 to R54, R44 to R55, R45 to R56, R46 to R57, R47 to R58, R48 to R59, R49 to R60
Connections:
- net IRQ_ACCEL: now also U13.4 (SENSOR_VP); no longer U13.6 (IO34)
- net IRQ_TOUCH: now also U13.6 (IO34); no longer U13.4 (SENSOR_VP)
- net LCD_DC: now also U13.9 (IO33); no longer U13.29 (IO5)
- net PWR_SDCARD_ENABLE: now also U13.29 (IO5); no longer U13.9 (IO33)
- net IR_TX renamed SPI_CS_STM32
- net SPI_CS_A renamed SPI_CS_FPGA
- net SPI_CS_B renamed SPI_CS_LCD
Changed lines of the file:
@@
 $EndDescr
 $Comp
-L power:+3.3V #PWR0165
+L power:+3.3V #PWR0163
 U 1 1 605756DE
 P 3650 2800
-F 0 "#PWR0165" H 3650 2650 50  0001 C CNN
+F 0 "#PWR0163" H 3650 2650 50  0001 C CNN
 F 1 "+3.3V" H 3650 2950 50  0000 C CNN
 F 2 "" H 3650 2800 50  0001 C CNN
@@
 NoConn ~ 3050 4200
 $Comp
-L power:GND #PWR0166
+L power:GND #PWR0164
 U 1 1 60721513
 P 3650 5600
-F 0 "#PWR0166" H 3650 5350 50  0001 C CNN
+F 0 "#PWR0164" H 3650 5350 50  0001 C CNN
 F 1 "GND" H 3655 5427 50  0000 C CNN
 F 2 "" H 3650 5600 50  0001 C CNN
@@
 $EndComp
 $Comp
-L power:+3.3V #PWR0169
+L power:+3.3V #PWR0167
 U 1 1 60AFAF9F
 P 6600 7150
-F 0 "#PWR0169" H 6600 7000 50  0001 C CNN
+F 0 "#PWR0167" H 6600 7000 50  0001 C CNN
 F 1 "+3.3V" H 6600 7300 50  0000 C CNN
 F 2 "" H 6600 7150 50  0001 C CNN
@@
 $EndComp
 $Comp
-L power:+3.3V #PWR0167
+L power:+3.3V #PWR0165
 U 1 1 60575709
 P 6150 7150
-F 0 "#PWR0167" H 6150 7000 50  0001 C CNN
+F 0 "#PWR0165" H 6150 7000 50  0001 C CNN
 F 1 "+3.3V" H 6150 7300 50  0000 C CNN
 F 2 "" H 6150 7150 50  0001 C CNN
@@
 	9150 4500 9050 4500
 $Comp
-L power:GND #PWR0170
+L power:GND #PWR0168
 U 1 1 605756D0
 P 6600 7450
-F 0 "#PWR0170" H 6600 7200 50  0001 C CNN
+F 0 "#PWR0168" H 6600 7200 50  0001 C CNN
 F 1 "GND" H 6605 7277 50  0000 C CNN
 F 2 "" H 6600 7450 50  0001 C CNN
@@
 $EndComp
 $Comp
-L power:GND #PWR0168
+L power:GND #PWR0166
 U 1 1 5F61964A
 P 6150 7450
-F 0 "#PWR0168" H 6150 7200 50  0001 C CNN
+F 0 "#PWR0166" H 6150 7200 50  0001 C CNN
 F 1 "GND" H 6155 7277 50  0000 C CNN
 F 2 "" H 6150 7450 50  0001 C CNN
@@
 $EndComp
 $Comp
-L power:GND #PWR0176
+L power:GND #PWR0174
 U 1 1 605756F0
 P 9800 2400
-F 0 "#PWR0176" H 9800 2150 50  0001 C CNN
+F 0 "#PWR0174" H 9800 2150 50  0001 C CNN
 F 1 "GND" H 9805 2227 50  0000 C CNN
 F 2 "" H 9800 2400 50  0001 C CNN
@@
 $EndComp
 $Comp
-L Device:R R49
+L Device:R R60
 U 1 1 605756E5
 P 9800 2250
-F 0 "R49" V 9700 2250 50  0000 C CNN
+F 0 "R60" V 9700 2250 50  0000 C CNN
 F 1 "45.3k" V 9900 2250 50  0000 C CNN
 F 2 "Resistor_SMD:R_0603_1608Metric" V 9730 2250 50  0001 C CNN
@@
 SD_D0
 $Comp
-L Device:R R35
+L Device:R R46
 U 1 1 6072151D
 P 8250 2250
-F 0 "R35" V 8150 2250 50  0000 C CNN
+F 0 "R46" V 8150 2250 50  0000 C CNN
 F 1 "45.3k" V 8350 2250 50  0000 C CNN
 F 2 "Resistor_SMD:R_0603_1608Metric" V 8180 2250 50  0001 C CNN
@@
 $EndComp
 $Comp
-L power:GND #PWR0171
+L power:GND #PWR0169
 U 1 1 6072151E
 P 8250 2400
-F 0 "#PWR0171" H 8250 2150 50  0001 C CNN
+F 0 "#PWR0169" H 8250 2150 50  0001 C CNN
 F 1 "GND" H 8255 2227 50  0000 C CNN
 F 2 "" H 8250 2400 50  0001 C CNN
@@
 	9800 2050 9750 2050
 $Comp
-L Device:R R48
+L Device:R R59
 U 1 1 60534310
 P 9800 1850
-F 0 "R48" V 9700 1850 50  0000 C CNN
+F 0 "R59" V 9700 1850 50  0000 C CNN
 F 1 "DNP" V 9900 1850 50  0000 C CNN
 F 2 "Resistor_SMD:R_0603_1608Metric" V 9730 1850 50  0001 C CNN
@@
 $EndComp
 $Comp
-L power:+3.3V #PWR0175
+L power:+3.3V #PWR0173
 U 1 1 605756EE
 P 9800 1700
-F 0 "#PWR0175" H 9800 1550 50  0001 C CNN
+F 0 "#PWR0173" H 9800 1550 50  0001 C CNN
 F 1 "+3.3V" H 9800 1850 50  0000 C CNN
 F 2 "" H 9800 1700 50  0001 C CNN
@@
 Connection ~ 9800 2050
 $Comp
-L power:GND #PWR0173
+L power:GND #PWR0171
 U 1 1 60721519
 P 9000 2400
-F 0 "#PWR0173" H 9000 2150 50  0001 C CNN
+F 0 "#PWR0171" H 9000 2150 50  0001 C CNN
 F 1 "GND" H 9005 2227 50  0000 C CNN
 F 2 "" H 9000 2400 50  0001 C CNN
@@
 	9000 2050 8950 2050
 $Comp
-L Device:R R39
+L Device:R R50
 U 1 1 605756DA
 P 9000 2250
-F 0 "R39" V 8900 2250 50  0000 C CNN
+F 0 "R50" V 8900 2250 50  0000 C CNN
 F 1 "DNP" V 9100 2250 50  0000 C CNN
 F 2 "Resistor_SMD:R_0603_1608Metric" V 8930 2250 50  0001 C CNN
@@
 $EndComp
 $Comp
-L power:+3.3V #PWR0172
+L power:+3.3V #PWR0170
 U 1 1 60721533
 P 9000 1700
-F 0 "#PWR0172" H 9000 1550 50  0001 C CNN
+F 0 "#PWR0170" H 9000 1550 50  0001 C CNN
 F 1 "+3.3V" H 9000 1850 50  0000 C CNN
 F 2 "" H 9000 1700 50  0001 C CNN
@@
 Connection ~ 9000 2050
 $Comp
-L Device:R R38
+L Device:R R49
 U 1 1 60721539
 P 9000 1850
-F 0 "R38" V 8900 1850 50  0000 C CNN
+F 0 "R49" V 8900 1850 50  0000 C CNN
 F 1 "45.3k" V 9100 1850 50  0000 C CNN
 F 2 "Resistor_SMD:R_0603_1608Metric" V 8930 1850 50  0001 C CNN
@@
 Unknown\nLow = UART DL\nHigh = ???
 $Comp
-L power:+3.3V #PWR0174
+L power:+3.3V #PWR0172
 U 1 1 605756F5
 P 9000 4450
-F 0 "#PWR0174" H 9000 4300 50  0001 C CNN
+F 0 "#PWR0172" H 9000 4300 50  0001 C CNN
 F 1 "+3.3V" H 9000 4600 50  0000 C CNN
 F 2 "" H 9000 4450 50  0001 C CNN
@@
 	1    0    0    -1
 $EndComp
-Text HLabel 4250 5100 2    39   Output ~ 0
+Text HLabel 4250 3500 2    39   Output ~ 0
 PWR_SDCARD_ENABLE
 Text HLabel 2800 3000 0    39   Input ~ 0
@@
 Text HLabel 4250 4200 2    39   Output ~ 0
 SPI_CLK
-Text HLabel 4250 3500 2    39   Output ~ 0
+Text HLabel 4250 5100 2    39   Output ~ 0
 LCD_DC
 Text HLabel 4250 4400 2    39   Output ~ 0
@@
 Text HLabel 4250 3000 2    39   Input ~ 0
 ESP32_BL
+Text HLabel 4250 5200 2    39   Input ~ 0
+IRQ_TOUCH
 Text HLabel 2800 3200 0    39   Input ~ 0
-IRQ_TOUCH
-Text HLabel 4250 5200 2    39   Input ~ 0
 IRQ_ACCEL
 Wire Notes Line
@@
 	2800 3200 3050 3200
 $Comp
-L Device:R R47
+L Device:R R58
 U 1 1 5F4625FA
 P 9750 4750
-F 0 "R47" V 9800 4600 50  0000 C CNN
+F 0 "R58" V 9800 4600 50  0000 C CNN
 F 1 "10k" V 9750 4750 50  0000 C CNN
 F 2 "Resistor_SMD:R_0603_1608Metric" V 9680 4750 50  0001 C CNN
@@
 $EndComp
 $Comp
-L Device:R R46
+L Device:R R57
 U 1 1 5F462EA1
 P 9650 4750
-F 0 "R46" V 9700 4600 50  0000 C CNN
+F 0 "R57" V 9700 4600 50  0000 C CNN
 F 1 "10k" V 9650 4750 50  0000 C CNN
 F 2 "Resistor_SMD:R_0603_1608Metric" V 9580 4750 50  0001 C CNN
@@
 $EndComp
 $Comp
-L Device:R R45
+L Device:R R56
 U 1 1 5F463A31
 P 9550 4750
-F 0 "R45" V 9600 4600 50  0000 C CNN
+F 0 "R56" V 9600 4600 50  0000 C CNN
 F 1 "10k" V 9550 4750 50  0000 C CNN
 F 2 "Resistor_SMD:R_0603_1608Metric" V 9480 4750 50  0001 C CNN
@@
 $EndComp
 $Comp
-L Device:R R44
+L Device:R R55
 U 1 1 5F464767
 P 9450 4750
-F 0 "R44" V 9500 4600 50  0000 C CNN
+F 0 "R55" V 9500 4600 50  0000 C CNN
 F 1 "10k" V 9450 4750 50  0000 C CNN
 F 2 "Resistor_SMD:R_0603_1608Metric" V 9380 4750 50  0001 C CNN
@@
 $EndComp
 $Comp
-L Device:R R43
+L Device:R R54
 U 1 1 5F4653F4
 P 9350 4750
-F 0 "R43" V 9400 4600 50  0000 C CNN
+F 0 "R54" V 9400 4600 50  0000 C CNN
 F 1 "10k" V 9350 4750 50  0000 C CNN
 F 2 "Resistor_SMD:R_0603_1608Metric" V 9280 4750 50  0001 C CNN
@@
 $EndComp
 $Comp
-L Device:R R42
+L Device:R R53
 U 1 1 5F465E5B
 P 9250 4750
-F 0 "R42" V 9300 4600 50  0000 C CNN
+F 0 "R53" V 9300 4600 50  0000 C CNN
 F 1 "10k" V 9250 4750 50  0000 C CNN
 F 2 "Resistor_SMD:R_0603_1608Metric" V 9180 4750 50  0001 C CNN
@@
 	9250 4900 9250 4950
 $Comp
-L Device:R R41
+L Device:R R52
 U 1 1 5F472114
 P 9150 4750
-F 0 "R41" V 9200 4600 50  0000 C CNN
+F 0 "R52" V 9200 4600 50  0000 C CNN
 F 1 "10k" V 9150 4750 50  0000 C CNN
 F 2 "Resistor_SMD:R_0603_1608Metric" V 9080 4750 50  0001 C CNN
@@
 $EndComp
 $Comp
-L Device:R R40
+L Device:R R51
 U 1 1 5F47253D
 P 9050 4750
-F 0 "R40" V 9100 4600 50  0000 C CNN
+F 0 "R51" V 9100 4600 50  0000 C CNN
 F 1 "10k" V 9050 4750 50  0000 C CNN
 F 2 "Resistor_SMD:R_0603_1608Metric" V 8980 4750 50  0001 C CNN
@@
 $EndComp
 $Comp
-L Device:R R37
+L Device:R R48
 U 1 1 5F472778
 P 8950 4750
-F 0 "R37" V 9000 4600 50  0000 C CNN
+F 0 "R48" V 9000 4600 50  0000 C CNN
 F 1 "10k" V 8950 4750 50  0000 C CNN
 F 2 "Resistor_SMD:R_0603_1608Metric" V 8880 4750 50  0001 C CNN
@@
 $EndComp
 $Comp
-L Device:R R36
+L Device:R R47
 U 1 1 5F47298B
 P 8850 4750
-F 0 "R36" V 8900 4600 50  0000 C CNN
+F 0 "R47" V 8900 4600 50  0000 C CNN
 F 1 "10k" V 8850 4750 50  0000 C CNN
 F 2 "Resistor_SMD:R_0603_1608Metric" V 8780 4750 50  0001 C CNN
@@
 	8850 4500 8850 4600
 Text HLabel 4250 5000 2    39   Output ~ 0
-SPI_CS_B
+SPI_CS_LCD
 Text HLabel 4250 4900 2    39   Output ~ 0
-SPI_CS_A
+SPI_CS_FPGA
 Text Notes 7000 3450 0    79   ~ 0
 Pull-up resistors for\n - I2C bus\n - Download mode (IO0)\n - SDIO bus
 Text HLabel 4250 4300 2    39   Output ~ 0
-IR_TX
+SPI_CS_STM32
 $EndSCHEMATC

Commit message: Dump.
Parts:
- C43: Price 0.0020 -> (none)
- C44: LCSC (none) -> C307461; Price 0.0020 -> (none)
- R46, R49, R60: LCSC - -> C23058; Price 0.0005 -> (none)
- R47, R48, R51, R52, R53, R54, R55, R56, R57, R58: LCSC - -> C115324; Price 0.0005 -> (none)
- R50, R59: Price 0.0005 -> (none)
- U13: Price 0 -> (none)
Connections:
- net GND: now also U13.39 (GND)
Changed lines of the file:
@@
 F 3 "~" H 6150 7300 50  0001 C CNN
 F 4 "C14663" H 6150 7300 50  0001 C CNN "LCSC"
-F 5 "0.0020" H 6150 7300 50  0001 C CNN "Price"
+F 5 "" H 6150 7300 50  0001 C CNN "Price"
 F 6 "-" H 6150 7300 50  0001 C CNN "Mouser"
 F 7 "N" H 6150 7300 50  0001 C CNN "Sponsored"
@@
 F 2 "Capacitor_SMD:C_0603_1608Metric" H 6638 7150 50  0001 C CNN
 F 3 "~" H 6600 7300 50  0001 C CNN
-F 4 "0.0020" H 6600 7300 50  0001 C CNN "Price"
+F 4 "" H 6600 7300 50  0001 C CNN "Price"
 F 5 "N" H 6600 7300 50  0001 C CNN "Sponsored"
+F 6 "C307461" H 6600 7300 50  0001 C CNN "LCSC"
 	1    6600 7300
 	1    0    0    -1
@@
 F 2 "Resistor_SMD:R_0603_1608Metric" V 9730 2250 50  0001 C CNN
 F 3 "~" H 9800 2250 50  0001 C CNN
-F 4 "0.0005" H 9800 2250 50  0001 C CNN "Price"
-F 5 "-" H 9800 2250 50  0001 C CNN "LCSC"
+F 4 "" H 9800 2250 50  0001 C CNN "Price"
+F 5 "C23058" H 9800 2250 50  0001 C CNN "LCSC"
 F 6 "-" H 9800 2250 50  0001 C CNN "Mouser"
 F 7 "N" H 9800 2250 50  0001 C CNN "Sponsored"
@@
 F 2 "Resistor_SMD:R_0603_1608Metric" V 8180 2250 50  0001 C CNN
 F 3 "~" H 8250 2250 50  0001 C CNN
-F 4 "0.0005" H 8250 2250 50  0001 C CNN "Price"
-F 5 "-" H 8250 2250 50  0001 C CNN "LCSC"
+F 4 "" H 8250 2250 50  0001 C CNN "Price"
+F 5 "C23058" H 8250 2250 50  0001 C CNN "LCSC"
 F 6 "-" H 8250 2250 50  0001 C CNN "Mouser"
 F 7 "N" H 8250 2250 50  0001 C CNN "Sponsored"
@@
 F 2 "Resistor_SMD:R_0603_1608Metric" V 9730 1850 50  0001 C CNN
 F 3 "~" H 9800 1850 50  0001 C CNN
-F 4 "0.0005" H 9800 1850 50  0001 C CNN "Price"
+F 4 "" H 9800 1850 50  0001 C CNN "Price"
 F 5 "-" H 9800 1850 50  0001 C CNN "LCSC"
 F 6 "-" H 9800 1850 50  0001 C CNN "Mouser"
@@
 F 2 "Resistor_SMD:R_0603_1608Metric" V 8930 2250 50  0001 C CNN
 F 3 "~" H 9000 2250 50  0001 C CNN
-F 4 "0.0005" H 9000 2250 50  0001 C CNN "Price"
+F 4 "" H 9000 2250 50  0001 C CNN "Price"
 F 5 "-" H 9000 2250 50  0001 C CNN "LCSC"
 F 6 "-" H 9000 2250 50  0001 C CNN "Mouser"
@@
 F 2 "Resistor_SMD:R_0603_1608Metric" V 8930 1850 50  0001 C CNN
 F 3 "~" H 9000 1850 50  0001 C CNN
-F 4 "0.0005" H 9000 1850 50  0001 C CNN "Price"
-F 5 "-" H 9000 1850 50  0001 C CNN "LCSC"
+F 4 "" H 9000 1850 50  0001 C CNN "Price"
+F 5 "C23058" H 9000 1850 50  0001 C CNN "LCSC"
 F 6 "-" H 9000 1850 50  0001 C CNN "Mouser"
 F 7 "N" H 9000 1850 50  0001 C CNN "Sponsored"
@@
 F 2 "custom:ESP32-WROVER" H 3650 2700 50  0001 C CNN
 F 3 "https://www.espressif.com/sites/default/files/documentation/esp32-wroom-32_datasheet_en.pdf" H 3350 4250 50  0001 C CNN
-F 4 "0" H 3650 4200 50  0001 C CNN "Price"
+F 4 "" H 3650 4200 50  0001 C CNN "Price"
 F 5 "-" H 3650 4200 50  0001 C CNN "LCSC"
 F 6 "-" H 3650 4200 50  0001 C CNN "Mouser"
@@
 F 2 "Resistor_SMD:R_0603_1608Metric" V 9680 4750 50  0001 C CNN
 F 3 "~" H 9750 4750 50  0001 C CNN
-F 4 "0.0005" H 9750 4750 50  0001 C CNN "Price"
-F 5 "-" H 9750 4750 50  0001 C CNN "LCSC"
+F 4 "" H 9750 4750 50  0001 C CNN "Price"
+F 5 "C115324" H 9750 4750 50  0001 C CNN "LCSC"
 F 6 "-" H 9750 4750 50  0001 C CNN "Mouser"
 F 7 "N" H 9750 4750 50  0001 C CNN "Sponsored"
@@
 F 2 "Resistor_SMD:R_0603_1608Metric" V 9580 4750 50  0001 C CNN
 F 3 "~" H 9650 4750 50  0001 C CNN
-F 4 "0.0005" H 9650 4750 50  0001 C CNN "Price"
-F 5 "-" H 9650 4750 50  0001 C CNN "LCSC"
+F 4 "" H 9650 4750 50  0001 C CNN "Price"
+F 5 "C115324" H 9650 4750 50  0001 C CNN "LCSC"
 F 6 "-" H 9650 4750 50  0001 C CNN "Mouser"
 F 7 "N" H 9650 4750 50  0001 C CNN "Sponsored"
@@
 F 2 "Resistor_SMD:R_0603_1608Metric" V 9480 4750 50  0001 C CNN
 F 3 "~" H 9550 4750 50  0001 C CNN
-F 4 "0.0005" H 9550 4750 50  0001 C CNN "Price"
-F 5 "-" H 9550 4750 50  0001 C CNN "LCSC"
+F 4 "" H 9550 4750 50  0001 C CNN "Price"
+F 5 "C115324" H 9550 4750 50  0001 C CNN "LCSC"
 F 6 "-" H 9550 4750 50  0001 C CNN "Mouser"
 F 7 "N" H 9550 4750 50  0001 C CNN "Sponsored"
@@
 F 2 "Resistor_SMD:R_0603_1608Metric" V 9380 4750 50  0001 C CNN
 F 3 "~" H 9450 4750 50  0001 C CNN
-F 4 "0.0005" H 9450 4750 50  0001 C CNN "Price"
-F 5 "-" H 9450 4750 50  0001 C CNN "LCSC"
+F 4 "" H 9450 4750 50  0001 C CNN "Price"
+F 5 "C115324" H 9450 4750 50  0001 C CNN "LCSC"
 F 6 "-" H 9450 4750 50  0001 C CNN "Mouser"
 F 7 "N" H 9450 4750 50  0001 C CNN "Sponsored"
@@
 F 2 "Resistor_SMD:R_0603_1608Metric" V 9280 4750 50  0001 C CNN
 F 3 "~" H 9350 4750 50  0001 C CNN
-F 4 "0.0005" H 9350 4750 50  0001 C CNN "Price"
-F 5 "-" H 9350 4750 50  0001 C CNN "LCSC"
+F 4 "" H 9350 4750 50  0001 C CNN "Price"
+F 5 "C115324" H 9350 4750 50  0001 C CNN "LCSC"
 F 6 "-" H 9350 4750 50  0001 C CNN "Mouser"
 F 7 "N" H 9350 4750 50  0001 C CNN "Sponsored"
@@
 F 2 "Resistor_SMD:R_0603_1608Metric" V 9180 4750 50  0001 C CNN
 F 3 "~" H 9250 4750 50  0001 C CNN
-F 4 "0.0005" H 9250 4750 50  0001 C CNN "Price"
-F 5 "-" H 9250 4750 50  0001 C CNN "LCSC"
+F 4 "" H 9250 4750 50  0001 C CNN "Price"
+F 5 "C115324" H 9250 4750 50  0001 C CNN "LCSC"
 F 6 "-" H 9250 4750 50  0001 C CNN "Mouser"
 F 7 "N" H 9250 4750 50  0001 C CNN "Sponsored"
@@
 F 2 "Resistor_SMD:R_0603_1608Metric" V 9080 4750 50  0001 C CNN
 F 3 "~" H 9150 4750 50  0001 C CNN
-F 4 "0.0005" H 9150 4750 50  0001 C CNN "Price"
-F 5 "-" H 9150 4750 50  0001 C CNN "LCSC"
+F 4 "" H 9150 4750 50  0001 C CNN "Price"
+F 5 "C115324" H 9150 4750 50  0001 C CNN "LCSC"
 F 6 "-" H 9150 4750 50  0001 C CNN "Mouser"
 F 7 "N" H 9150 4750 50  0001 C CNN "Sponsored"
@@
 F 2 "Resistor_SMD:R_0603_1608Metric" V 8980 4750 50  0001 C CNN
 F 3 "~" H 9050 4750 50  0001 C CNN
-F 4 "0.0005" H 9050 4750 50  0001 C CNN "Price"
-F 5 "-" H 9050 4750 50  0001 C CNN "LCSC"
+F 4 "" H 9050 4750 50  0001 C CNN "Price"
+F 5 "C115324" H 9050 4750 50  0001 C CNN "LCSC"
 F 6 "-" H 9050 4750 50  0001 C CNN "Mouser"
 F 7 "N" H 9050 4750 50  0001 C CNN "Sponsored"
@@
 F 2 "Resistor_SMD:R_0603_1608Metric" V 8880 4750 50  0001 C CNN
 F 3 "~" H 8950 4750 50  0001 C CNN
-F 4 "0.0005" H 8950 4750 50  0001 C CNN "Price"
-F 5 "-" H 8950 4750 50  0001 C CNN "LCSC"
+F 4 "" H 8950 4750 50  0001 C CNN "Price"
+F 5 "C115324" H 8950 4750 50  0001 C CNN "LCSC"
 F 6 "-" H 8950 4750 50  0001 C CNN "Mouser"
 F 7 "N" H 8950 4750 50  0001 C CNN "Sponsored"
@@
 F 2 "Resistor_SMD:R_0603_1608Metric" V 8780 4750 50  0001 C CNN
 F 3 "~" H 8850 4750 50  0001 C CNN
-F 4 "0.0005" H 8850 4750 50  0001 C CNN "Price"
-F 5 "-" H 8850 4750 50  0001 C CNN "LCSC"
+F 4 "" H 8850 4750 50  0001 C CNN "Price"
+F 5 "C115324" H 8850 4750 50  0001 C CNN "LCSC"
 F 6 "-" H 8850 4750 50  0001 C CNN "Mouser"
 F 7 "N" H 8850 4750 50  0001 C CNN "Sponsored"
@@
 Text HLabel 4250 4300 2    39   Output ~ 0
 SPI_CS_STM32
+Wire Wire Line
+	3050 5100 2950 5100
+$Comp
+L power:GND #PWR0181
+U 1 1 5F69C61B
+P 2950 5600
+F 0 "#PWR0181" H 2950 5350 50  0001 C CNN
+F 1 "GND" H 2955 5427 50  0000 C CNN
+F 2 "" H 2950 5600 50  0001 C CNN
+F 3 "" H 2950 5600 50  0001 C CNN
+	1    2950 5600
+	1    0    0    -1
+$EndComp
+Wire Wire Line
+	2950 5100 2950 5600
 $EndSCHEMATC

Commit message: Work in progress: prototype 2
Parts:
- removed R53, R54, R55, R56, R57, R58: 10k, Resistor_SMD:R_0603_1608Metric, symbol Device:R
Connections:
- net labels removed: AUDIO_L, AUDIO_R, PWR_SDCARD, PWR_SDCARD_ENABLE, SD_D1, SD_D2, SD_D3
Other:
- note added: "*"
- note added: "* Bootstrapping pins\nIO 0:Low for UART DL mode, pull high for normal boot\nIO 2: Pull down to select UART DL mode when GPIO 0 is LOW\nIO 12: Selects internal flash/ram voltage. Pull-up for 3.3v, pull-down for 1.8v\nIO 15: Pull down for silent bootloader"
- note added: "JTAG TCK"
- note added: "JTAG TDI"
- note added: "JTAG TDO"
- note added: "JTAG TMS"
- note removed: "Also used as STM32 IRQ"
- note removed: "Bootloader\nLow = silent\nHigh = debug"
- note removed: "ESP32 bootstapping pins"
- note removed: "Flash/RAM voltage\nLow = 1.8v\nHigh = 3.3v"
- note removed: "IO 0:Low for uart dl, high for normal boot\nIO 2: Always pull-down during boot\nIO 12: Selects internal flash/ram voltage. Pull-up for 3.3v, pull-down for 1.8v\nIO 15: Pull down for silent bootloader"
- note removed: "IO 12"
- note removed: "IO 15"
- note removed: "IO 2"
- note removed: "Pull-up resistors for\n - I2C bus\n - Download mode (IO0)\n - SDIO bus"
- note removed: "Unknown\nLow = UART DL\nHigh = ???"
- moved on the sheet: R46, R47, R48, R49, R50, R51, R52, R59, R60
