File: esp32.sch (KiCad schematic (older format))
At the start: 34 parts, among them U13 ESP32-WROVER

Commit message: Updated schematic, add design file
Parts:
- gave numbers to parts that had none: 2
Changed lines of the file:
@@
 EXT_I2C_SCL
 $Comp
-L power:GND #PWR?
+L power:GND #PWR0105
 U 1 1 5FDD9C6F
 P 4650 5700
-F 0 "#PWR?" H 4650 5450 50  0001 C CNN
+F 0 "#PWR0105" H 4650 5450 50  0001 C CNN
 F 1 "GND" H 4655 5527 50  0000 C CNN
 F 2 "" H 4650 5700 50  0001 C CNN
@@
 Connection ~ 5850 4700
 $Comp
-L Device:R R?
+L Device:R R73
 U 1 1 5FDFAB98
 P 6150 2700
-F 0 "R?" V 6050 2700 50  0000 C CNN
+F 0 "R73" V 6050 2700 50  0000 C CNN
 F 1 "4.7k" V 6250 2700 50  0000 C CNN
 F 2 "Resistor_SMD:R_0603_1608Metric" V 6080 2700 50  0001 C CNN
@@
 $EndComp
 $Comp
-L power:+3.3V #PWR?
+L power:+3.3V #PWR0106
 U 1 1 5FDFB48F
 P 6150 2550
-F 0 "#PWR?" H 6150 2400 50  0001 C CNN
+F 0 "#PWR0106" H 6150 2400 50  0001 C CNN
 F 1 "+3.3V" H 6150 2700 50  0000 C CNN
 F 2 "" H 6150 2550 50  0001 C CNN
@@
 	5850 4700 6700 4700
 $Comp
-L Device:C C?
+L Device:C C24
 U 1 1 5FE0AEBE
 P 2550 3750
-F 0 "C?" H 2665 3796 50  0000 L CNN
+F 0 "C24" H 2665 3796 50  0000 L CNN
 F 1 "100n" H 2665 3705 50  0000 L CNN
 F 2 "Capacitor_SMD:C_0603_1608Metric" H 2588 3600 50  0001 C CNN
@@
 	2550 3000 2950 3000
 $Comp
-L power:GND #PWR?
+L power:GND #PWR0170
 U 1 1 5FE22DD7
 P 2550 5700
-F 0 "#PWR?" H 2550 5450 50  0001 C CNN
+F 0 "#PWR0170" H 2550 5450 50  0001 C CNN
 F 1 "GND" H 2555 5527 50  0000 C CNN
 F 2 "" H 2550 5700 50  0001 C CNN

Commit message: First steps of routing prototype 2, switch to 0402 for most passives
Parts:
- C24, C43: footprint Capacitor_SMD:C_0603_1608Metric -> Capacitor_SMD:C_0402_1005Metric; LCSC C14663 -> C83056
- C44: footprint Capacitor_SMD:C_0603_1608Metric -> Capacitor_SMD:C_0402_1005Metric; LCSC C307461 -> C15525
- R46, R49, R60, R69, R73: footprint Resistor_SMD:R_0603_1608Metric -> Resistor_SMD:R_0402_1005Metric; LCSC C23058 -> (none)
- R47, R48, R51, R52: footprint Resistor_SMD:R_0603_1608Metric -> Resistor_SMD:R_0402_1005Metric; LCSC C115324 -> (none)
- R59: footprint Resistor_SMD:R_0603_1608Metric -> Resistor_SMD:R_0402_1005Metric; LCSC - -> (none)
Changed lines of the file:
@@
 F 0 "C43" H 6265 7346 50  0000 L CNN
 F 1 "100n" H 6265 7255 50  0000 L CNN
-F 2 "Capacitor_SMD:C_0603_1608Metric" H 6188 7150 50  0001 C CNN
-F 3 "~" H 6150 7300 50  0001 C CNN
-F 4 "C14663" H 6150 7300 50  0001 C CNN "LCSC"
+F 2 "Capacitor_SMD:C_0402_1005Metric" H 6188 7150 50  0001 C CNN
+F 3 "" H 6150 7300 50  0001 C CNN
+F 4 "C83056 " H 6150 7300 50  0001 C CNN "LCSC"
 F 5 "" H 6150 7300 50  0001 C CNN "Price"
 F 6 "-" H 6150 7300 50  0001 C CNN "Mouser"
@@
 F 0 "C44" H 6715 7346 50  0000 L CNN
 F 1 "10u" H 6715 7255 50  0000 L CNN
-F 2 "Capacitor_SMD:C_0603_1608Metric" H 6638 7150 50  0001 C CNN
-F 3 "~" H 6600 7300 50  0001 C CNN
+F 2 "Capacitor_SMD:C_0402_1005Metric" H 6638 7150 50  0001 C CNN
+F 3 "" H 6600 7300 50  0001 C CNN
 F 4 "" H 6600 7300 50  0001 C CNN "Price"
 F 5 "N" H 6600 7300 50  0001 C CNN "Sponsored"
-F 6 "C307461" H 6600 7300 50  0001 C CNN "LCSC"
+F 6 "C15525" H 6600 7300 50  0001 C CNN "LCSC"
 	1    6600 7300
 	1    0    0    -1
@@
 F 0 "R60" V 4850 5550 50  0000 C CNN
 F 1 "45.3k" V 5050 5550 50  0000 C CNN
-F 2 "Resistor_SMD:R_0603_1608Metric" V 4880 5550 50  0001 C CNN
+F 2 "Resistor_SMD:R_0402_1005Metric" V 4880 5550 50  0001 C CNN
 F 3 "~" H 4950 5550 50  0001 C CNN
 F 4 "" H 4950 5550 50  0001 C CNN "Price"
-F 5 "C23058" H 4950 5550 50  0001 C CNN "LCSC"
+F 5 "" H 4950 5550 50  0001 C CNN "LCSC"
 F 6 "-" H 4950 5550 50  0001 C CNN "Mouser"
 F 7 "N" H 4950 5550 50  0001 C CNN "Sponsored"
@@
 F 0 "R46" V 4250 5550 50  0000 C CNN
 F 1 "45.3k" V 4450 5550 50  0000 C CNN
-F 2 "Resistor_SMD:R_0603_1608Metric" V 4280 5550 50  0001 C CNN
+F 2 "Resistor_SMD:R_0402_1005Metric" V 4280 5550 50  0001 C CNN
 F 3 "~" H 4350 5550 50  0001 C CNN
 F 4 "" H 4350 5550 50  0001 C CNN "Price"
-F 5 "C23058" H 4350 5550 50  0001 C CNN "LCSC"
+F 5 "" H 4350 5550 50  0001 C CNN "LCSC"
 F 6 "-" H 4350 5550 50  0001 C CNN "Mouser"
 F 7 "N" H 4350 5550 50  0001 C CNN "Sponsored"
@@
 F 0 "R49" V 4550 5550 50  0000 C CNN
 F 1 "4.7k" V 4750 5550 50  0000 C CNN
-F 2 "Resistor_SMD:R_0603_1608Metric" V 4580 5550 50  0001 C CNN
+F 2 "Resistor_SMD:R_0402_1005Metric" V 4580 5550 50  0001 C CNN
 F 3 "~" H 4650 5550 50  0001 C CNN
 F 4 "" H 4650 5550 50  0001 C CNN "Price"
-F 5 "C23058" H 4650 5550 50  0001 C CNN "LCSC"
+F 5 "" H 4650 5550 50  0001 C CNN "LCSC"
 F 6 "-" H 4650 5550 50  0001 C CNN "Mouser"
 F 7 "N" H 4650 5550 50  0001 C CNN "Sponsored"
@@
 F 0 "R52" V 5450 2700 50  0000 C CNN
 F 1 "4.7k" V 5650 2700 50  0000 C CNN
-F 2 "Resistor_SMD:R_0603_1608Metric" V 5480 2700 50  0001 C CNN
+F 2 "Resistor_SMD:R_0402_1005Metric" V 5480 2700 50  0001 C CNN
 F 3 "~" H 5550 2700 50  0001 C CNN
 F 4 "" H 5550 2700 50  0001 C CNN "Price"
-F 5 "C115324" H 5550 2700 50  0001 C CNN "LCSC"
+F 5 "" H 5550 2700 50  0001 C CNN "LCSC"
 F 6 "-" H 5550 2700 50  0001 C CNN "Mouser"
 F 7 "N" H 5550 2700 50  0001 C CNN "Sponsored"
@@
 F 0 "R51" V 5150 2700 50  0000 C CNN
 F 1 "4.7k" V 5350 2700 50  0000 C CNN
-F 2 "Resistor_SMD:R_0603_1608Metric" V 5180 2700 50  0001 C CNN
+F 2 "Resistor_SMD:R_0402_1005Metric" V 5180 2700 50  0001 C CNN
 F 3 "~" H 5250 2700 50  0001 C CNN
 F 4 "" H 5250 2700 50  0001 C CNN "Price"
-F 5 "C115324" H 5250 2700 50  0001 C CNN "LCSC"
+F 5 "" H 5250 2700 50  0001 C CNN "LCSC"
 F 6 "-" H 5250 2700 50  0001 C CNN "Mouser"
 F 7 "N" H 5250 2700 50  0001 C CNN "Sponsored"
@@
 F 0 "R48" V 4250 2700 50  0000 C CNN
 F 1 "10k" V 4450 2700 50  0000 C CNN
-F 2 "Resistor_SMD:R_0603_1608Metric" V 4280 2700 50  0001 C CNN
+F 2 "Resistor_SMD:R_0402_1005Metric" V 4280 2700 50  0001 C CNN
 F 3 "~" H 4350 2700 50  0001 C CNN
 F 4 "" H 4350 2700 50  0001 C CNN "Price"
-F 5 "C115324" H 4350 2700 50  0001 C CNN "LCSC"
+F 5 "" H 4350 2700 50  0001 C CNN "LCSC"
 F 6 "-" H 4350 2700 50  0001 C CNN "Mouser"
 F 7 "N" H 4350 2700 50  0001 C CNN "Sponsored"
@@
 F 0 "R47" V 2850 2650 50  0000 C CNN
 F 1 "10k" V 3050 2650 50  0000 C CNN
-F 2 "Resistor_SMD:R_0603_1608Metric" V 2880 2650 50  0001 C CNN
+F 2 "Resistor_SMD:R_0402_1005Metric" V 2880 2650 50  0001 C CNN
 F 3 "~" H 2950 2650 50  0001 C CNN
 F 4 "" H 2950 2650 50  0001 C CNN "Price"
-F 5 "C115324" H 2950 2650 50  0001 C CNN "LCSC"
+F 5 "" H 2950 2650 50  0001 C CNN "LCSC"
 F 6 "-" H 2950 2650 50  0001 C CNN "Mouser"
 F 7 "N" H 2950 2650 50  0001 C CNN "Sponsored"
@@
 F 0 "R59" V 4850 2700 50  0000 C CNN
 F 1 "DNP" V 5050 2700 50  0000 C CNN
-F 2 "Resistor_SMD:R_0603_1608Metric" V 4880 2700 50  0001 C CNN
+F 2 "Resistor_SMD:R_0402_1005Metric" V 4880 2700 50  0001 C CNN
 F 3 "~" H 4950 2700 50  0001 C CNN
 F 4 "" H 4950 2700 50  0001 C CNN "Price"
-F 5 "-" H 4950 2700 50  0001 C CNN "LCSC"
+F 5 "" H 4950 2700 50  0001 C CNN "LCSC"
 F 6 "-" H 4950 2700 50  0001 C CNN "Mouser"
 F 7 "N" H 4950 2700 50  0001 C CNN "Sponsored"
@@
 F 0 "R69" V 5750 2700 50  0000 C CNN
 F 1 "4.7k" V 5950 2700 50  0000 C CNN
-F 2 "Resistor_SMD:R_0603_1608Metric" V 5780 2700 50  0001 C CNN
+F 2 "Resistor_SMD:R_0402_1005Metric" V 5780 2700 50  0001 C CNN
 F 3 "~" H 5850 2700 50  0001 C CNN
 F 4 "" H 5850 2700 50  0001 C CNN "Price"
-F 5 "C23058" H 5850 2700 50  0001 C CNN "LCSC"
+F 5 "" H 5850 2700 50  0001 C CNN "LCSC"
 F 6 "-" H 5850 2700 50  0001 C CNN "Mouser"
 F 7 "N" H 5850 2700 50  0001 C CNN "Sponsored"
@@
 F 0 "R73" V 6050 2700 50  0000 C CNN
 F 1 "4.7k" V 6250 2700 50  0000 C CNN
-F 2 "Resistor_SMD:R_0603_1608Metric" V 6080 2700 50  0001 C CNN
+F 2 "Resistor_SMD:R_0402_1005Metric" V 6080 2700 50  0001 C CNN
 F 3 "~" H 6150 2700 50  0001 C CNN
 F 4 "" H 6150 2700 50  0001 C CNN "Price"
-F 5 "C23058" H 6150 2700 50  0001 C CNN "LCSC"
+F 5 "" H 6150 2700 50  0001 C CNN "LCSC"
 F 6 "-" H 6150 2700 50  0001 C CNN "Mouser"
 F 7 "N" H 6150 2700 50  0001 C CNN "Sponsored"
@@
 F 0 "C24" H 2665 3796 50  0000 L CNN
 F 1 "100n" H 2665 3705 50  0000 L CNN
-F 2 "Capacitor_SMD:C_0603_1608Metric" H 2588 3600 50  0001 C CNN
-F 3 "~" H 2550 3750 50  0001 C CNN
-F 4 "C14663" H 2550 3750 50  0001 C CNN "LCSC"
+F 2 "Capacitor_SMD:C_0402_1005Metric" H 2588 3600 50  0001 C CNN
+F 3 "" H 2550 3750 50  0001 C CNN
+F 4 "C83056 " H 2550 3750 50  0001 C CNN "LCSC"
 F 5 "" H 2550 3750 50  0001 C CNN "Price"
 F 6 "-" H 2550 3750 50  0001 C CNN "Mouser"

Commit message: Some more work
Parts:
- removed TP12: ESP EN, TestPoint:TestPoint_Pad_1.0x1.0mm, symbol Connector:TestPoint_Small
- removed TP13: IRQ SENSOR, TestPoint:TestPoint_Pad_1.0x1.0mm, symbol Connector:TestPoint_Small
- removed TP14: IRQ FPGA, TestPoint:TestPoint_Pad_1.0x1.0mm, symbol Connector:TestPoint_Small
- removed TP15: ESP32 BL, TestPoint:TestPoint_Pad_1.0x1.0mm, symbol Connector:TestPoint_Small
- removed TP16: ESP32 TX, TestPoint:TestPoint_Pad_1.0x1.0mm, symbol Connector:TestPoint_Small
- removed TP17: ESP32 RX, TestPoint:TestPoint_Pad_1.0x1.0mm, symbol Connector:TestPoint_Small
- removed TP18, TP19, TP20: ESP32 TDI, TestPoint:TestPoint_Pad_1.0x1.0mm, symbol Connector:TestPoint_Small
- removed TP21: ESP32 TCK, TestPoint:TestPoint_Pad_1.0x1.0mm, symbol Connector:TestPoint_Small
- removed TP22: ESP32 TMS, TestPoint:TestPoint_Pad_1.0x1.0mm, symbol Connector:TestPoint_Small
- removed TP23: ESP32 TDO, TestPoint:TestPoint_Pad_1.0x1.0mm, symbol Connector:TestPoint_Small
- removed TP24: SPI CLK, TestPoint:TestPoint_Pad_1.0x1.0mm, symbol Connector:TestPoint_Small
- removed TP25: SPI CS STM32, TestPoint:TestPoint_Pad_1.0x1.0mm, symbol Connector:TestPoint_Small
- removed TP26: SPI MOSI, TestPoint:TestPoint_Pad_1.0x1.0mm, symbol Connector:TestPoint_Small
- removed TP29: SPI CS FPGA, TestPoint:TestPoint_Pad_1.0x1.0mm, symbol Connector:TestPoint_Small
- removed TP30: SPI CS LCD, TestPoint:TestPoint_Pad_1.0x1.0mm, symbol Connector:TestPoint_Small
- removed TP31: LCD DC, TestPoint:TestPoint_Pad_1.0x1.0mm, symbol Connector:TestPoint_Small
- removed TP32: IRQ BTN, TestPoint:TestPoint_Pad_1.0x1.0mm, symbol Connector:TestPoint_Small
- removed TP33: SPI MISO, TestPoint:TestPoint_Pad_1.0x1.0mm, symbol Connector:TestPoint_Small
- renumbered C24 to C23, C43 to C24, C44 to C25, R47 to R37, R48 to R38, R46 to R39, R49 to R40, R59 to R41, R60 to R42, R51 to R43, R52 to R44, R69 to R45, R73 to R46, U13 to U7

Commit message: Fix most of the bugs found on prototype 2 board
Parts:
- added J5: Micro SD card, custom:MicroSD-SOFNG-TF-002-H18, symbol Connector:Micro_SD_Card
- added R10, R11, R50, R77, R8, R9: 10k, Resistor_SMD:R_0402_1005Metric, symbol Device:R
Connections:
- net GND: now also J5.6 (VSS), J5.9 (SHIELD)
- net SD_CLK: now also J5.5 (CLK), R10.2
- net SD_CMD: now also J5.3 (CMD), R11.2
- net SD_D0: now also J5.7 (DAT0), R9.2
- net LED_DATA renamed SD_POWER
- new net: J5.1 (DAT2), R77.2
- new net: J5.2 (DAT3/CD), R50.2
- new net: J5.8 (DAT1), R8.2
- new net PWR_SDCARD: J5.4 (VDD), R10.1, R11.1, R50.1, R77.1, R8.1, R9.1

Commit message: Change pinout of expansion header close to board edge to be fully ground instead of gnd + 3.3v (& update component references)
Parts:
- C23, C24, C25: symbol Device:C -> mch2021-rescue:C-Device
- J5: symbol Connector:Micro_SD_Card -> mch2021-rescue:Micro_SD_Card-Connector
- R10, R11, R37, R38, R39, R40, R41, R42, R43, R44, R45, R46, R50, R77, R8, R9: symbol Device:R -> mch2021-rescue:R-Device
Changed lines of the file:
@@
 $EndDescr
 $Comp
-L power:+3.3V #PWR0103
+L mch2021-rescue:+3.3V-power #PWR0103
 U 1 1 605756DE
 P 3650 2550
@@
 NoConn ~ 3050 4200
 $Comp
-L power:GND #PWR0104
+L mch2021-rescue:GND-power #PWR0104
 U 1 1 60721513
 P 3650 5700
@@
 $EndComp
 $Comp
-L power:+3.3V #PWR0116
+L mch2021-rescue:+3.3V-power #PWR0116
 U 1 1 60AFAF9F
 P 6600 7150
@@
 $EndComp
 $Comp
-L power:+3.3V #PWR0114
+L mch2021-rescue:+3.3V-power #PWR0114
 U 1 1 60575709
 P 6150 7150
@@
 $EndComp
 $Comp
-L power:GND #PWR0117
+L mch2021-rescue:GND-power #PWR0117
 U 1 1 605756D0
 P 6600 7450
@@
 $EndComp
 $Comp
-L power:GND #PWR0115
+L mch2021-rescue:GND-power #PWR0115
 U 1 1 5F61964A
 P 6150 7450
@@
 $EndComp
 $Comp
-L Device:C C24
+L mch2021-rescue:C-Device C24
 U 1 1 605756E3
 P 6150 7300
@@
 $EndComp
 $Comp
-L Device:C C25
+L mch2021-rescue:C-Device C25
 U 1 1 5F619647
 P 6600 7300
@@
 $EndComp
 $Comp
-L power:GND #PWR0109
+L mch2021-rescue:GND-power #PWR0109
 U 1 1 605756F0
 P 4950 5700
@@
 $EndComp
 $Comp
-L Device:R R42
+L mch2021-rescue:R-Device R42
 U 1 1 605756E5
 P 4950 5550
@@
 * Bootstrapping pins\nIO 0:Low for UART DL mode, pull high for normal boot\nIO 2: Pull down to select UART DL mode when GPIO 0 is LOW\nIO 12: Selects internal flash/ram voltage. Pull-up for 1.8v, pull-down for 3.3v\nIO 15: Pull down for silent bootloader
 $Comp
-L Device:R R39
+L mch2021-rescue:R-Device R39
 U 1 1 6072151D
 P 4350 5550
@@
 $EndComp
 $Comp
-L power:GND #PWR0106
+L mch2021-rescue:GND-power #PWR0106
 U 1 1 6072151E
 P 4350 5700
@@
 $EndComp
 $Comp
-L Device:R R40
+L mch2021-rescue:R-Device R40
 U 1 1 60721539
 P 4650 5550
@@
 	3600 3350 3150 3350
 $Comp
-L Device:R R44
+L mch2021-rescue:R-Device R44
 U 1 1 5F472114
 P 5550 2700
@@
 $EndComp
 $Comp
-L Device:R R43
+L mch2021-rescue:R-Device R43
 U 1 1 5F47253D
 P 5250 2700
@@
 $EndComp
 $Comp
-L Device:R R38
+L mch2021-rescue:R-Device R38
 U 1 1 5F472778
 P 4350 2700
@@
 $EndComp
 $Comp
-L Device:R R37
+L mch2021-rescue:R-Device R37
 U 1 1 5F47298B
 P 2950 2650
@@
 	3050 5100 2950 5100
 $Comp
-L power:GND #PWR0102
+L mch2021-rescue:GND-power #PWR0102
 U 1 1 5F69C61B
 P 2950 5700
@@
 Connection ~ 4950 3900
 $Comp
-L power:+3.3V #PWR0105
+L mch2021-rescue:+3.3V-power #PWR0105
 U 1 1 5FDBC3D5
 P 4350 2550
@@
 	4350 3000 4250 3000
 $Comp
-L power:+3.3V #PWR0101
+L mch2021-rescue:+3.3V-power #PWR0101
 U 1 1 5FDCAB36
 P 2950 2500
@@
 Connection ~ 5550 4500
 $Comp
-L power:+3.3V #PWR0110
+L mch2021-rescue:+3.3V-power #PWR0110
 U 1 1 5FE09909
 P 5250 2550
@@
 $EndComp
 $Comp
-L power:+3.3V #PWR0111
+L mch2021-rescue:+3.3V-power #PWR0111
 U 1 1 5FE09C3A
 P 5550 2550
@@
 	4950 3900 4950 2850
 $Comp
-L power:+3.3V #PWR0108
+L mch2021-rescue:+3.3V-power #PWR0108
 U 1 1 605756EE
 P 4950 2550
@@
 $EndComp
 $Comp
-L Device:R R41
+L mch2021-rescue:R-Device R41
 U 1 1 60534310
 P 4950 2700
@@
 $EndComp
 $Comp
-L Device:R R45
+L mch2021-rescue:R-Device R45
 U 1 1 6040FC0D
 P 5850 2700
@@
 $EndComp
 $Comp
-L power:+3.3V #PWR0112
+L mch2021-rescue:+3.3V-power #PWR0112
 U 1 1 60432E08
 P 5850 2550
@@
 EXT_I2C_SCL
 $Comp
-L power:GND #PWR0107
+L mch2021-rescue:GND-power #PWR0107
 U 1 1 5FDD9C6F
 P 4650 5700
@@
 Connection ~ 5850 4700
 $Comp
-L Device:R R46
+L mch2021-rescue:R-Device R46
 U 1 1 5FDFAB98
 P 6150 2700
@@
 $EndComp
 $Comp
-L power:+3.3V #PWR0113
+L mch2021-rescue:+3.3V-power #PWR0113
 U 1 1 5FDFB48F
 P 6150 2550
@@
 	5850 4700 6700 4700
 $Comp
-L Device:C C23
+L mch2021-rescue:C-Device C23
 U 1 1 5FE0AEBE
 P 2550 3750
@@
 	2550 3000 2950 3000
 $Comp
-L power:GND #PWR0100
+L mch2021-rescue:GND-power #PWR0100
 U 1 1 5FE22DD7
 P 2550 5700
@@
 	8750 1700 8750 2100
 $Comp
-L power:GND #PWR?
+L mch2021-rescue:GND-power #PWR?
 U 1 1 61828AAB
 P 8750 2100
@@
 PWR_SDCARD
 $Comp
-L Connector:Micro_SD_Card J?
+L mch2021-rescue:Micro_SD_Card-Connector J?
 U 1 1 61828AB6
 P 9850 1500
@@
 	10700 2100 10650 2100
 $Comp
-L power:GND #PWR?
+L mch2021-rescue:GND-power #PWR?
 U 1 1 61828ABE
 P 10700 2150
@@
 $EndComp
 $Comp
-L Device:R R77
+L mch2021-rescue:R-Device R77
 U 1 1 61828AC8
 P 8800 1000
@@
 $EndComp
 $Comp
-L Device:R R50
+L mch2021-rescue:R-Device R50
 U 1 1 61828AD2
 P 8700 1000
@@
 $EndComp
 $Comp
-L Device:R R11
+L mch2021-rescue:R-Device R11
 U 1 1 61828ADC
 P 8600 1000
@@
 	8700 800  8600 800
 $Comp
-L Device:R R9
+L mch2021-rescue:R-Device R9
 U 1 1 61828AF2
 P 8400 1000
@@
 $EndComp
 $Comp
-L Device:R R10
+L mch2021-rescue:R-Device R10
 U 1 1 61828AFC
 P 8500 1000
@@
 	8500 800  8400 800
 $Comp
-L Device:R R8
+L mch2021-rescue:R-Device R8
 U 1 1 61828B09
 P 8300 1000
