File: lcd.sch (KiCad schematic (older format))
At the start: 12 parts, among them J8 LCD, Q1 Q_NMOS_GSD, Q2 Q_NMOS_GSD, U13 74LVC1G125

Commit message: Dump.
Parts:
- J7: renamed from J8; LCSC (none) -> C202114; Mouser (none) -> -; Price (none) -> 0.37; Sponsored (none) -> N
- Q1, Q2: footprint (none) -> Package_TO_SOT_SMD:SOT-23; LCSC (none) -> C406812; Mouser (none) -> -; Price (none) -> 0.0077; Sponsored (none) -> N
- R23: renamed from R34; footprint (none) -> Resistor_SMD:R_0603_1608Metric; LCSC (none) -> -; Mouser (none) -> -; Price (none) -> 0.0005; Sponsored (none) -> N
- R24: renamed from R35; footprint (none) -> Resistor_SMD:R_0603_1608Metric; LCSC (none) -> -; Mouser (none) -> -; Price (none) -> 0.0005; Sponsored (none) -> N
- RN10: renamed from RN9; footprint (none) -> Resistor_SMD:R_Array_Convex_4x0603; LCSC (none) -> C173315; Mouser (none) -> -; Price (none) -> 0.0042; Sponsored (none) -> N
- RN11: renamed from RN10; footprint (none) -> Resistor_SMD:R_Array_Convex_4x0603; LCSC (none) -> C173315; Mouser (none) -> -; Price (none) -> 0.0042; Sponsored (none) -> N
- RN12: renamed from RN11; footprint (none) -> Resistor_SMD:R_Array_Convex_4x0603; LCSC (none) -> C173315; Mouser (none) -> -; Price (none) -> 0.0042; Sponsored (none) -> N
- RN7: renamed from RN6; footprint (none) -> Resistor_SMD:R_Array_Convex_4x0603; LCSC (none) -> -; Mouser (none) -> -; Price (none) -> 0.0042; Sponsored (none) -> N
- RN8: renamed from RN7; footprint (none) -> Resistor_SMD:R_Array_Convex_4x0603; LCSC (none) -> -; Mouser (none) -> -; Price (none) -> 0.0042; Sponsored (none) -> N
- RN9: renamed from RN8; footprint (none) -> Resistor_SMD:R_Array_Convex_4x0603; LCSC (none) -> C173315; Mouser (none) -> -; Price (none) -> 0.0042; Sponsored (none) -> N
- U10: renamed from U13; footprint (none) -> Package_TO_SOT_SMD:SOT-353_SC-70-5; LCSC (none) -> C703585; Mouser (none) -> -; Price (none) -> 0.020; Sponsored (none) -> N
Connections:
- net labels added: CS, LCD_IM0, LCD_K0, LCD_K1, LCD_K2, LCD_RS_SCK, LCD_RS_SCK_SWITCH, LCD_WR_RS, SPI_DC
- net labels removed: PAR_CS, SPI_CS, SPI_RS
- wire segments 161 -> 159

Commit message: Dump.
Parts:
- renumbered Q1 to Q2, Q2 to Q3, R23 to R19, R24 to R20, RN7 to RN3, RN8 to RN4, RN9 to RN5, RN10 to RN6, RN11 to RN7, RN12 to RN8, U10 to U7
Changed lines of the file:
@@
 NoConn ~ 6850 1850
 $Comp
-L power:GND #PWR0119
+L power:GND #PWR095
 U 1 1 5FE093AF
 P 6750 6050
-F 0 "#PWR0119" H 6750 5800 50  0001 C CNN
+F 0 "#PWR095" H 6750 5800 50  0001 C CNN
 F 1 "GND" H 6755 5877 50  0000 C CNN
 F 2 "" H 6750 6050 50  0001 C CNN
@@
 	6750 1950 6850 1950
 $Comp
-L power:+3.3V #PWR0118
+L power:+3.3V #PWR094
 U 1 1 5FE0C2BF
 P 6650 1250
-F 0 "#PWR0118" H 6650 1100 50  0001 C CNN
+F 0 "#PWR094" H 6650 1100 50  0001 C CNN
 F 1 "+3.3V" H 6665 1423 50  0000 C CNN
 F 2 "" H 6650 1250 50  0001 C CNN
@@
 Connection ~ 6650 2050
 $Comp
-L 74xGxx:74LVC1G125 U10
+L 74xGxx:74LVC1G125 U7
 U 1 1 5FE0FF4D
 P 5800 2350
-F 0 "U10" H 6100 2550 50  0000 C CNN
+F 0 "U7" H 6100 2550 50  0000 C CNN
 F 1 "74LVC1G125" H 6100 2450 50  0000 C CNN
 F 2 "Package_TO_SOT_SMD:SOT-353_SC-70-5" H 5800 2350 50  0001 C CNN
@@
 $EndComp
 $Comp
-L power:+3.3V #PWR0115
+L power:+3.3V #PWR091
 U 1 1 5FE23AF8
 P 5850 1250
-F 0 "#PWR0115" H 5850 1100 50  0001 C CNN
+F 0 "#PWR091" H 5850 1100 50  0001 C CNN
 F 1 "+3.3V" H 5865 1423 50  0000 C CNN
 F 2 "" H 5850 1250 50  0001 C CNN
@@
 	6750 3850 6750 5150
 $Comp
-L power:GND #PWR0117
+L power:GND #PWR093
 U 1 1 5FEDB6BC
 P 6250 6050
-F 0 "#PWR0117" H 6250 5800 50  0001 C CNN
+F 0 "#PWR093" H 6250 5800 50  0001 C CNN
 F 1 "GND" H 6255 5877 50  0000 C CNN
 F 2 "" H 6250 6050 50  0001 C CNN
@@
 $EndComp
 $Comp
-L power:GND #PWR0116
+L power:GND #PWR092
 U 1 1 5FEDBAA4
 P 5850 6050
-F 0 "#PWR0116" H 5850 5800 50  0001 C CNN
+F 0 "#PWR092" H 5850 5800 50  0001 C CNN
 F 1 "GND" H 5855 5877 50  0000 C CNN
 F 2 "" H 5850 6050 50  0001 C CNN
@@
 $EndComp
 $Comp
-L power:GND #PWR0113
+L power:GND #PWR089
 U 1 1 5FEDBDD6
 P 4750 6050
-F 0 "#PWR0113" H 4750 5800 50  0001 C CNN
+F 0 "#PWR089" H 4750 5800 50  0001 C CNN
 F 1 "GND" H 4755 5877 50  0000 C CNN
 F 2 "" H 4750 6050 50  0001 C CNN
@@
 	6100 4350 6850 4350
 $Comp
-L power:GND #PWR0114
+L power:GND #PWR090
 U 1 1 5FEF458A
 P 5350 6050
-F 0 "#PWR0114" H 5350 5800 50  0001 C CNN
+F 0 "#PWR090" H 5350 5800 50  0001 C CNN
 F 1 "GND" H 5355 5877 50  0000 C CNN
 F 2 "" H 5350 6050 50  0001 C CNN
@@
 PAR_RS
 $Comp
-L Device:R_Small R23
+L Device:R_Small R19
 U 1 1 5FE5D02B
 P 3700 2350
-F 0 "R23" V 3750 2500 50  0000 C CNN
+F 0 "R19" V 3750 2500 50  0000 C CNN
 F 1 "47" V 3700 2350 50  0000 C CNN
 F 2 "Resistor_SMD:R_0603_1608Metric" H 3700 2350 50  0001 C CNN
@@
 	3500 4950 3500 5050
 $Comp
-L power:GND #PWR0110
+L power:GND #PWR086
 U 1 1 6016D996
 P 3050 6050
-F 0 "#PWR0110" H 3050 5800 50  0001 C CNN
+F 0 "#PWR086" H 3050 5800 50  0001 C CNN
 F 1 "GND" H 3055 5877 50  0000 C CNN
 F 2 "" H 3050 6050 50  0001 C CNN
@@
 	4400 5400 6800 5400
 $Comp
-L power:GND #PWR0112
+L power:GND #PWR088
 U 1 1 6021B8D1
 P 4400 6050
-F 0 "#PWR0112" H 4400 5800 50  0001 C CNN
+F 0 "#PWR088" H 4400 5800 50  0001 C CNN
 F 1 "GND" H 4405 5877 50  0000 C CNN
 F 2 "" H 4400 6050 50  0001 C CNN
@@
 	3050 4850 3050 6050
 $Comp
-L Device:Q_NMOS_GSD Q1
+L Device:Q_NMOS_GSD Q2
 U 1 1 6005561C
 P 3250 4950
-F 0 "Q1" V 3150 5100 50  0000 C CNN
+F 0 "Q2" V 3150 5100 50  0000 C CNN
 F 1 "Q_NMOS_GSD" V 3000 5000 50  0000 C CNN
 F 2 "Package_TO_SOT_SMD:SOT-23" H 3450 5050 50  0001 C CNN
@@
 Connection ~ 4400 5400
 $Comp
-L Device:Q_NMOS_GSD Q2
+L Device:Q_NMOS_GSD Q3
 U 1 1 601EC337
 P 4300 5600
-F 0 "Q2" H 4350 5400 50  0000 C CNN
+F 0 "Q3" H 4350 5400 50  0000 C CNN
 F 1 "Q_NMOS_GSD" H 4150 5300 50  0000 C CNN
 F 2 "Package_TO_SOT_SMD:SOT-23" H 4500 5700 50  0001 C CNN
@@
 	4100 5250 4100 5600
 $Comp
-L Device:R_Small R24
+L Device:R_Small R20
 U 1 1 6027CDDC
 P 3750 5600
-F 0 "R24" V 3554 5600 50  0000 C CNN
+F 0 "R20" V 3554 5600 50  0000 C CNN
 F 1 "47" V 3645 5600 50  0000 C CNN
 F 2 "Resistor_SMD:R_0603_1608Metric" H 3750 5600 50  0001 C CNN
@@
 	3650 5600 3600 5600
 $Comp
-L power:+3.3V #PWR0111
+L power:+3.3V #PWR087
 U 1 1 602901D6
 P 4250 1250
-F 0 "#PWR0111" H 4250 1100 50  0001 C CNN
+F 0 "#PWR087" H 4250 1100 50  0001 C CNN
 F 1 "+3.3V" H 4265 1423 50  0000 C CNN
 F 2 "" H 4250 1250 50  0001 C CNN
@@
 	3900 2550 4900 2550
 $Comp
-L Device:R_Pack04_Split RN7
+L Device:R_Pack04_Split RN3
 U 3 1 603477D3
 P 3700 2450
-F 0 "RN7" V 3750 2650 50  0000 L CNN
+F 0 "RN3" V 3750 2650 50  0000 L CNN
 F 1 "47" V 3700 2400 50  0000 L CNN
 F 2 "Resistor_SMD:R_Array_Convex_4x0603" V 3620 2450 50  0001 C CNN
@@
 $EndComp
 $Comp
-L Device:R_Pack04_Split RN7
+L Device:R_Pack04_Split RN3
 U 1 1 60346000
 P 2000 2050
-F 0 "RN7" V 2050 2250 50  0000 L CNN
+F 0 "RN3" V 2050 2250 50  0000 L CNN
 F 1 "47" V 2000 2000 50  0000 L CNN
 F 2 "Resistor_SMD:R_Array_Convex_4x0603" V 1920 2050 50  0001 C CNN
@@
 $EndComp
 $Comp
-L Device:R_Pack04 RN10
+L Device:R_Pack04 RN6
 U 1 1 6002B54B
 P 4800 5750
-F 0 "RN10" H 4950 5800 50  0000 L CNN
+F 0 "RN6" H 4950 5800 50  0000 L CNN
 F 1 "100k" H 4950 5700 50  0000 L CNN
 F 2 "Resistor_SMD:R_Array_Convex_4x0603" V 5075 5750 50  0001 C CNN
@@
 $EndComp
 $Comp
-L Device:R_Pack04 RN8
+L Device:R_Pack04 RN4
 U 1 1 5FE031D6
 P 3750 5050
-F 0 "RN8" V 3450 5050 50  0000 C CNN
+F 0 "RN4" V 3450 5050 50  0000 C CNN
 F 1 "47" V 3450 5200 50  0000 C CNN
 F 2 "Resistor_SMD:R_Array_Convex_4x0603" V 4025 5050 50  0001 C CNN
@@
 $EndComp
 $Comp
-L Device:R_Pack04 RN11
+L Device:R_Pack04 RN7
 U 1 1 5FEF4584
 P 5400 5750
-F 0 "RN11" H 5588 5796 50  0000 L CNN
+F 0 "RN7" H 5588 5796 50  0000 L CNN
 F 1 "100k" H 5588 5705 50  0000 L CNN
 F 2 "Resistor_SMD:R_Array_Convex_4x0603" V 5675 5750 50  0001 C CNN
@@
 $EndComp
 $Comp
-L Device:R_Pack04 RN12
+L Device:R_Pack04 RN8
 U 1 1 5FEC659D
 P 6300 5750
-F 0 "RN12" H 6488 5796 50  0000 L CNN
+F 0 "RN8" H 6488 5796 50  0000 L CNN
 F 1 "100k" H 6488 5705 50  0000 L CNN
 F 2 "Resistor_SMD:R_Array_Convex_4x0603" V 6575 5750 50  0001 C CNN
@@
 $EndComp
 $Comp
-L Device:R_Pack04_Split RN7
+L Device:R_Pack04_Split RN3
 U 4 1 60347C63
 P 3700 2550
-F 0 "RN7" V 3750 2750 50  0000 L CNN
+F 0 "RN3" V 3750 2750 50  0000 L CNN
 F 1 "47" V 3700 2500 50  0000 L CNN
 F 2 "Resistor_SMD:R_Array_Convex_4x0603" V 3620 2550 50  0001 C CNN
@@
 LCD\nType: Z240IT008\nController: ILI9341\nSize: 2.4 inch
 $Comp
-L Device:R_Pack04_Split RN7
+L Device:R_Pack04_Split RN3
 U 2 1 60347281
 P 2000 2250
-F 0 "RN7" V 2050 2450 50  0000 L CNN
+F 0 "RN3" V 2050 2450 50  0000 L CNN
 F 1 "47" V 2000 2200 50  0000 L CNN
 F 2 "Resistor_SMD:R_Array_Convex_4x0603" V 1920 2250 50  0001 C CNN
@@
 SPI: IM0 = 0, IM1 = 1, IM2 = 1\nPAR: IM0 = 1, IM1 = 0, IM2 = 0
 $Comp
-L Device:R_Pack04 RN9
+L Device:R_Pack04 RN5
 U 1 1 60444DB2
 P 4300 1550
-F 0 "RN9" H 4450 1600 50  0000 L CNN
+F 0 "RN5" H 4450 1600 50  0000 L CNN
 F 1 "100k" H 4450 1500 50  0000 L CNN
 F 2 "Resistor_SMD:R_Array_Convex_4x0603" V 4575 1550 50  0001 C CNN

Commit message: Dump.
Parts:
- removed R19, R20: 47, Resistor_SMD:R_0603_1608Metric, symbol Device:R_Small
- removed RN3: 47, Resistor_SMD:R_Array_Convex_4x0603, symbol Device:R_Pack04_Split
- removed RN4: 47, Resistor_SMD:R_Array_Convex_4x0603, symbol Device:R_Pack04
- removed RN5, RN6: 100k, Resistor_SMD:R_Array_Convex_4x0603, symbol Device:R_Pack04
- added R18, R19, R20, R21, R22, R23, R24, R25: 47, Resistor_SMD:R_0603_1608Metric, symbol Device:R
- added R26, R27, R28, R29, R30, R31, R32: 100k, Resistor_SMD:R_0603_1608Metric, symbol Device:R
- renumbered RN7 to RN3, RN8 to RN4
Connections:
- wire segments 159 -> 154

Commit message: Dump.
Parts:
- J7: Price 0.37 -> (none)
- Q2, Q3: Price 0.0077 -> (none)
- R18, R19, R20, R21, R22, R23, R24, R25: LCSC - -> C1211; Price 0.0005 -> (none)
- R26, R27, R28, R29, R30, R31, R32: LCSC - -> C15458; Price 0.0005 -> (none)
- RN3, RN4: Price 0.0042 -> (none)
- U7: Price 0.020 -> (none)
Changed lines of the file:
@@
 F 4 "C202114" H 7050 3450 50  0001 C CNN "LCSC"
 F 5 "-" H 7050 3450 50  0001 C CNN "Mouser"
-F 6 "0.37" H 7050 3450 50  0001 C CNN "Price"
+F 6 "" H 7050 3450 50  0001 C CNN "Price"
 F 7 "N" H 7050 3450 50  0001 C CNN "Sponsored"
 	1    7050 3450
@@
 F 3 "http://www.ti.com/lit/sg/scyt129e/scyt129e.pdf" H 5800 2350 50  0001 C CNN
 F 4 "C703585" H 5800 2350 50  0001 C CNN "LCSC"
-F 5 "0.020" H 5800 2350 50  0001 C CNN "Price"
+F 5 "" H 5800 2350 50  0001 C CNN "Price"
 F 6 "-" H 5800 2350 50  0001 C CNN "Mouser"
 F 7 "N" H 5800 2350 50  0001 C CNN "Sponsored"
@@
 F 4 "C406812" H 3250 4950 50  0001 C CNN "LCSC"
 F 5 "-" H 3250 4950 50  0001 C CNN "Mouser"
-F 6 "0.0077" H 3250 4950 50  0001 C CNN "Price"
+F 6 "" H 3250 4950 50  0001 C CNN "Price"
 F 7 "N" H 3250 4950 50  0001 C CNN "Sponsored"
 	1    3250 4950
@@
 F 4 "C406812" H 4300 5600 50  0001 C CNN "LCSC"
 F 5 "-" H 4300 5600 50  0001 C CNN "Mouser"
-F 6 "0.0077" H 4300 5600 50  0001 C CNN "Price"
+F 6 "" H 4300 5600 50  0001 C CNN "Price"
 F 7 "N" H 4300 5600 50  0001 C CNN "Sponsored"
 	1    4300 5600
@@
 F 4 "C173315" H 5400 5750 50  0001 C CNN "LCSC"
 F 5 "-" H 5400 5750 50  0001 C CNN "Mouser"
-F 6 "0.0042" H 5400 5750 50  0001 C CNN "Price"
+F 6 "" H 5400 5750 50  0001 C CNN "Price"
 F 7 "N" H 5400 5750 50  0001 C CNN "Sponsored"
 	1    5400 5750
@@
 F 4 "C173315" H 6300 5750 50  0001 C CNN "LCSC"
 F 5 "-" H 6300 5750 50  0001 C CNN "Mouser"
-F 6 "0.0042" H 6300 5750 50  0001 C CNN "Price"
+F 6 "" H 6300 5750 50  0001 C CNN "Price"
 F 7 "N" H 6300 5750 50  0001 C CNN "Sponsored"
 	1    6300 5750
@@
 F 2 "Resistor_SMD:R_0603_1608Metric" V 4330 1550 50  0001 C CNN
 F 3 "~" H 4400 1550 50  0001 C CNN
-F 4 "-" H 4400 1550 50  0001 C CNN "LCSC"
-F 5 "0.0005" H 4400 1550 50  0001 C CNN "Price"
+F 4 "C15458" H 4400 1550 50  0001 C CNN "LCSC"
+F 5 "" H 4400 1550 50  0001 C CNN "Price"
 F 6 "-" H 4400 1550 50  0001 C CNN "Mouser"
 F 7 "N" H 4400 1550 50  0001 C CNN "Sponsored"
@@
 F 2 "Resistor_SMD:R_0603_1608Metric" V 4130 1550 50  0001 C CNN
 F 3 "~" H 4200 1550 50  0001 C CNN
-F 4 "-" H 4200 1550 50  0001 C CNN "LCSC"
-F 5 "0.0005" H 4200 1550 50  0001 C CNN "Price"
+F 4 "C15458" H 4200 1550 50  0001 C CNN "LCSC"
+F 5 "" H 4200 1550 50  0001 C CNN "Price"
 F 6 "-" H 4200 1550 50  0001 C CNN "Mouser"
 F 7 "N" H 4200 1550 50  0001 C CNN "Sponsored"
@@
 F 2 "Resistor_SMD:R_0603_1608Metric" V 4030 1550 50  0001 C CNN
 F 3 "~" H 4100 1550 50  0001 C CNN
-F 4 "-" H 4100 1550 50  0001 C CNN "LCSC"
-F 5 "0.0005" H 4100 1550 50  0001 C CNN "Price"
+F 4 "C15458" H 4100 1550 50  0001 C CNN "LCSC"
+F 5 "" H 4100 1550 50  0001 C CNN "Price"
 F 6 "-" H 4100 1550 50  0001 C CNN "Mouser"
 F 7 "N" H 4100 1550 50  0001 C CNN "Sponsored"
@@
 F 2 "Resistor_SMD:R_0603_1608Metric" V 4230 1550 50  0001 C CNN
 F 3 "~" H 4300 1550 50  0001 C CNN
-F 4 "-" H 4300 1550 50  0001 C CNN "LCSC"
-F 5 "0.0005" H 4300 1550 50  0001 C CNN "Price"
+F 4 "C15458" H 4300 1550 50  0001 C CNN "LCSC"
+F 5 "" H 4300 1550 50  0001 C CNN "Price"
 F 6 "-" H 4300 1550 50  0001 C CNN "Mouser"
 F 7 "N" H 4300 1550 50  0001 C CNN "Sponsored"
@@
 F 2 "Resistor_SMD:R_0603_1608Metric" V 3630 2350 50  0001 C CNN
 F 3 "~" H 3700 2350 50  0001 C CNN
-F 4 "-" H 3700 2350 50  0001 C CNN "LCSC"
-F 5 "0.0005" H 3700 2350 50  0001 C CNN "Price"
+F 4 "C1211" H 3700 2350 50  0001 C CNN "LCSC"
+F 5 "" H 3700 2350 50  0001 C CNN "Price"
 F 6 "-" H 3700 2350 50  0001 C CNN "Mouser"
 F 7 "N" H 3700 2350 50  0001 C CNN "Sponsored"
@@
 F 2 "Resistor_SMD:R_0603_1608Metric" V 3630 2450 50  0001 C CNN
 F 3 "~" H 3700 2450 50  0001 C CNN
-F 4 "-" H 3700 2450 50  0001 C CNN "LCSC"
-F 5 "0.0005" H 3700 2450 50  0001 C CNN "Price"
+F 4 "C1211" H 3700 2450 50  0001 C CNN "LCSC"
+F 5 "" H 3700 2450 50  0001 C CNN "Price"
 F 6 "-" H 3700 2450 50  0001 C CNN "Mouser"
 F 7 "N" H 3700 2450 50  0001 C CNN "Sponsored"
@@
 F 2 "Resistor_SMD:R_0603_1608Metric" V 3630 2550 50  0001 C CNN
 F 3 "~" H 3700 2550 50  0001 C CNN
-F 4 "-" H 3700 2550 50  0001 C CNN "LCSC"
-F 5 "0.0005" H 3700 2550 50  0001 C CNN "Price"
+F 4 "C1211" H 3700 2550 50  0001 C CNN "LCSC"
+F 5 "" H 3700 2550 50  0001 C CNN "Price"
 F 6 "-" H 3700 2550 50  0001 C CNN "Mouser"
 F 7 "N" H 3700 2550 50  0001 C CNN "Sponsored"
@@
 F 2 "Resistor_SMD:R_0603_1608Metric" V 3680 4850 50  0001 C CNN
 F 3 "~" H 3750 4850 50  0001 C CNN
-F 4 "-" H 3750 4850 50  0001 C CNN "LCSC"
-F 5 "0.0005" H 3750 4850 50  0001 C CNN "Price"
+F 4 "C1211" H 3750 4850 50  0001 C CNN "LCSC"
+F 5 "" H 3750 4850 50  0001 C CNN "Price"
 F 6 "-" H 3750 4850 50  0001 C CNN "Mouser"
 F 7 "N" H 3750 4850 50  0001 C CNN "Sponsored"
@@
 F 2 "Resistor_SMD:R_0603_1608Metric" V 3680 4950 50  0001 C CNN
 F 3 "~" H 3750 4950 50  0001 C CNN
-F 4 "-" H 3750 4950 50  0001 C CNN "LCSC"
-F 5 "0.0005" H 3750 4950 50  0001 C CNN "Price"
+F 4 "C1211" H 3750 4950 50  0001 C CNN "LCSC"
+F 5 "" H 3750 4950 50  0001 C CNN "Price"
 F 6 "-" H 3750 4950 50  0001 C CNN "Mouser"
 F 7 "N" H 3750 4950 50  0001 C CNN "Sponsored"
@@
 F 2 "Resistor_SMD:R_0603_1608Metric" V 3680 5050 50  0001 C CNN
 F 3 "~" H 3750 5050 50  0001 C CNN
-F 4 "-" H 3750 5050 50  0001 C CNN "LCSC"
-F 5 "0.0005" H 3750 5050 50  0001 C CNN "Price"
+F 4 "C1211" H 3750 5050 50  0001 C CNN "LCSC"
+F 5 "" H 3750 5050 50  0001 C CNN "Price"
 F 6 "-" H 3750 5050 50  0001 C CNN "Mouser"
 F 7 "N" H 3750 5050 50  0001 C CNN "Sponsored"
@@
 F 2 "Resistor_SMD:R_0603_1608Metric" V 3680 5150 50  0001 C CNN
 F 3 "~" H 3750 5150 50  0001 C CNN
-F 4 "-" H 3750 5150 50  0001 C CNN "LCSC"
-F 5 "0.0005" H 3750 5150 50  0001 C CNN "Price"
+F 4 "C1211" H 3750 5150 50  0001 C CNN "LCSC"
+F 5 "" H 3750 5150 50  0001 C CNN "Price"
 F 6 "-" H 3750 5150 50  0001 C CNN "Mouser"
 F 7 "N" H 3750 5150 50  0001 C CNN "Sponsored"
@@
 F 2 "Resistor_SMD:R_0603_1608Metric" V 3730 5600 50  0001 C CNN
 F 3 "~" H 3800 5600 50  0001 C CNN
-F 4 "-" H 3800 5600 50  0001 C CNN "LCSC"
-F 5 "0.0005" H 3800 5600 50  0001 C CNN "Price"
+F 4 "C1211" H 3800 5600 50  0001 C CNN "LCSC"
+F 5 "" H 3800 5600 50  0001 C CNN "Price"
 F 6 "-" H 3800 5600 50  0001 C CNN "Mouser"
 F 7 "N" H 3800 5600 50  0001 C CNN "Sponsored"
@@
 F 2 "Resistor_SMD:R_0603_1608Metric" V 4830 5750 50  0001 C CNN
 F 3 "~" H 4900 5750 50  0001 C CNN
-F 4 "-" H 4900 5750 50  0001 C CNN "LCSC"
-F 5 "0.0005" H 4900 5750 50  0001 C CNN "Price"
+F 4 "C15458" H 4900 5750 50  0001 C CNN "LCSC"
+F 5 "" H 4900 5750 50  0001 C CNN "Price"
 F 6 "-" H 4900 5750 50  0001 C CNN "Mouser"
 F 7 "N" H 4900 5750 50  0001 C CNN "Sponsored"
@@
 F 2 "Resistor_SMD:R_0603_1608Metric" V 4730 5750 50  0001 C CNN
 F 3 "~" H 4800 5750 50  0001 C CNN
-F 4 "-" H 4800 5750 50  0001 C CNN "LCSC"
-F 5 "0.0005" H 4800 5750 50  0001 C CNN "Price"
+F 4 "C15458" H 4800 5750 50  0001 C CNN "LCSC"
+F 5 "" H 4800 5750 50  0001 C CNN "Price"
 F 6 "-" H 4800 5750 50  0001 C CNN "Mouser"
 F 7 "N" H 4800 5750 50  0001 C CNN "Sponsored"
@@
 F 2 "Resistor_SMD:R_0603_1608Metric" V 4530 5750 50  0001 C CNN
 F 3 "~" H 4600 5750 50  0001 C CNN
-F 4 "-" H 4600 5750 50  0001 C CNN "LCSC"
-F 5 "0.0005" H 4600 5750 50  0001 C CNN "Price"
+F 4 "C15458" H 4600 5750 50  0001 C CNN "LCSC"
+F 5 "" H 4600 5750 50  0001 C CNN "Price"
 F 6 "-" H 4600 5750 50  0001 C CNN "Mouser"
 F 7 "N" H 4600 5750 50  0001 C CNN "Sponsored"

Commit message: Work in progress: prototype 2
Parts:
- removed R30: 100k, Resistor_SMD:R_0603_1608Metric, symbol Device:R
Connections:
- net LCD_IM0: now also U7.1
- net LCD_RS_SCK_SWITCH: no longer names the net of J7.39 (Pin_39), J7.40 (Pin_40), Q3.3 (D), R27.2
- net LCD_RS_SCK_SWITCH: no longer U7.1
Changed lines of the file:
@@
 L power:GND #PWR088
 U 1 1 5FEDBDD6
-P 4750 6050
-F 0 "#PWR088" H 4750 5800 50  0001 C CNN
-F 1 "GND" H 4755 5877 50  0000 C CNN
-F 2 "" H 4750 6050 50  0001 C CNN
-F 3 "" H 4750 6050 50  0001 C CNN
-	1    4750 6050
+P 4850 6050
+F 0 "#PWR088" H 4850 5800 50  0001 C CNN
+F 1 "GND" H 4855 5877 50  0000 C CNN
+F 2 "" H 4850 6050 50  0001 C CNN
+F 3 "" H 4850 6050 50  0001 C CNN
+	1    4850 6050
 	1    0    0    -1
 $EndComp
@@
 Connection ~ 5500 4250
 Wire Wire Line
-	4750 6050 4750 6000
-Connection ~ 4750 6000
-Wire Wire Line
-	4750 6000 4800 6000
-Connection ~ 4800 6000
-Wire Wire Line
-	4800 6000 4900 6000
+	4800 6000 4850 6000
 Wire Wire Line
 	4800 5250 6850 5250
@@
 	0    1    -1   0
 $EndComp
-Wire Wire Line
-	4100 5250 4800 5250
 Connection ~ 4400 5400
 $Comp
@@
 	4100 5600 3950 5600
 Connection ~ 4100 5600
-Wire Wire Line
-	3650 5600 3600 5600
 $Comp
 L power:+3.3V #PWR086
@@
 Wire Wire Line
 	4200 5400 4400 5400
-Connection ~ 4200 2150
-Wire Wire Line
-	4200 2150 4200 5400
-Wire Wire Line
-	4200 2150 5800 2150
 Connection ~ 4300 2000
 Connection ~ 4400 2950
@@
 Wire Wire Line
 	2950 2350 3550 2350
-Wire Wire Line
-	4600 5350 3600 5350
-Wire Wire Line
-	3600 5350 3600 5600
-Connection ~ 3600 5600
-Wire Wire Line
-	3600 5600 2950 5600
 Wire Wire Line
 	2950 2000 4300 2000
@@
 Wire Wire Line
 	4300 1700 4300 2000
-Wire Wire Line
-	4200 1700 4200 2150
 Wire Wire Line
 	4100 1700 4100 5150
@@
 	-1   0    0    1
 $EndComp
-$Comp
-L Device:R R?
-U 1 1 5F8D60B6
-P 4600 5750
-AR Path="/5DC753C3/5F8D60B6" Ref="R?"  Part="1"
-AR Path="/5F8D60B6" Ref="R?"  Part="1"
-AR Path="/5E3BA64A/5F8D60B6" Ref="R?"  Part="1"
-AR Path="/5F51E414/5F8D60B6" Ref="R?"  Part="1"
-AR Path="/5FDC6C76/5F8D60B6" Ref="R30"  Part="1"
-F 0 "R30" V 4650 5950 50  0000 C CNN
-F 1 "100k" V 4600 5750 50  0000 C CNN
-F 2 "Resistor_SMD:R_0603_1608Metric" V 4530 5750 50  0001 C CNN
-F 3 "~" H 4600 5750 50  0001 C CNN
-F 4 "C15458" H 4600 5750 50  0001 C CNN "LCSC"
-F 5 "" H 4600 5750 50  0001 C CNN "Price"
-F 6 "-" H 4600 5750 50  0001 C CNN "Mouser"
-F 7 "N" H 4600 5750 50  0001 C CNN "Sponsored"
-	1    4600 5750
-	-1   0    0    1
-$EndComp
 Wire Wire Line
 	4900 5900 4900 6000
@@
 	4800 5900 4800 6000
 Wire Wire Line
-	4600 6000 4750 6000
-Wire Wire Line
-	4600 5900 4600 6000
-Wire Wire Line
-	4600 5350 4600 5600
-Wire Wire Line
 	4800 5250 4800 5600
 Wire Wire Line
 	4900 2550 4900 5600
+Wire Wire Line
+	4200 1700 4200 5400
+Wire Wire Line
+	2950 5600 3650 5600
+Wire Wire Line
+	4800 5250 4800 2150
+Wire Wire Line
+	4800 2150 5800 2150
+Wire Wire Line
+	4100 5250 4800 5250
+Wire Wire Line
+	4850 6050 4850 6000
+Connection ~ 4850 6000
+Wire Wire Line
+	4850 6000 4900 6000
 $EndSCHEMATC
