File: lcd.sch (KiCad schematic (older format))
At the start: 20 parts, among them J7 LCD, Q2 Q_NMOS_GSD, Q3 Q_NMOS_GSD, U7 74LVC1G125

Commit message: First steps of routing prototype 2, switch to 0402 for most passives
Parts:
- removed R21, R22, R23, R24: 47, Resistor_SMD:R_0603_1608Metric, symbol Device:R
- added RN1: 47, Resistor_SMD:R_Array_Convex_4x0603, symbol Device:R_Pack04
- R18, R19, R20, R25: footprint Resistor_SMD:R_0603_1608Metric -> Resistor_SMD:R_0402_1005Metric; LCSC C1211 -> (none)
- R26, R27, R28, R29, R31, R32: footprint Resistor_SMD:R_0603_1608Metric -> Resistor_SMD:R_0402_1005Metric; LCSC C15458 -> (none)
Connections:
- wire segments 148 -> 149

Commit message: Some more work
Parts:
- renumbered Q2 to Q1, Q3 to Q2, R18 to R12, R19 to R13, R20 to R14, R25 to R15, R26 to R16, R27 to R17, R28 to R18, R29 to R19, R31 to R20, R32 to R21, RN3 to RN2, RN4 to RN3, U7 to U2
Changed lines of the file:
@@
 NoConn ~ 6850 1850
 $Comp
-L power:GND #PWR094
+L power:GND #PWR043
 U 1 1 5FE093AF
 P 6750 6050
-F 0 "#PWR094" H 6750 5800 50  0001 C CNN
+F 0 "#PWR043" H 6750 5800 50  0001 C CNN
 F 1 "GND" H 6755 5877 50  0000 C CNN
 F 2 "" H 6750 6050 50  0001 C CNN
@@
 	6750 1950 6850 1950
 $Comp
-L power:+3.3V #PWR093
+L power:+3.3V #PWR042
 U 1 1 5FE0C2BF
 P 6650 1250
-F 0 "#PWR093" H 6650 1100 50  0001 C CNN
+F 0 "#PWR042" H 6650 1100 50  0001 C CNN
 F 1 "+3.3V" H 6665 1423 50  0000 C CNN
 F 2 "" H 6650 1250 50  0001 C CNN
@@
 Connection ~ 6650 2050
 $Comp
-L 74xGxx:74LVC1G125 U7
+L 74xGxx:74LVC1G125 U2
 U 1 1 5FE0FF4D
 P 5800 2350
-F 0 "U7" H 6100 2550 50  0000 C CNN
+F 0 "U2" H 6100 2550 50  0000 C CNN
 F 1 "74LVC1G125" H 6100 2450 50  0000 C CNN
 F 2 "Package_TO_SOT_SMD:SOT-353_SC-70-5" H 5800 2350 50  0001 C CNN
@@
 $EndComp
 $Comp
-L power:+3.3V #PWR090
+L power:+3.3V #PWR039
 U 1 1 5FE23AF8
 P 5850 1250
-F 0 "#PWR090" H 5850 1100 50  0001 C CNN
+F 0 "#PWR039" H 5850 1100 50  0001 C CNN
 F 1 "+3.3V" H 5865 1423 50  0000 C CNN
 F 2 "" H 5850 1250 50  0001 C CNN
@@
 	6750 3850 6750 5150
 $Comp
-L power:GND #PWR092
+L power:GND #PWR041
 U 1 1 5FEDB6BC
 P 6250 6050
-F 0 "#PWR092" H 6250 5800 50  0001 C CNN
+F 0 "#PWR041" H 6250 5800 50  0001 C CNN
 F 1 "GND" H 6255 5877 50  0000 C CNN
 F 2 "" H 6250 6050 50  0001 C CNN
@@
 $EndComp
 $Comp
-L power:GND #PWR091
+L power:GND #PWR040
 U 1 1 5FEDBAA4
 P 5850 6050
-F 0 "#PWR091" H 5850 5800 50  0001 C CNN
+F 0 "#PWR040" H 5850 5800 50  0001 C CNN
 F 1 "GND" H 5855 5877 50  0000 C CNN
 F 2 "" H 5850 6050 50  0001 C CNN
@@
 $EndComp
 $Comp
-L power:GND #PWR088
+L power:GND #PWR037
 U 1 1 5FEDBDD6
 P 4850 6050
-F 0 "#PWR088" H 4850 5800 50  0001 C CNN
+F 0 "#PWR037" H 4850 5800 50  0001 C CNN
 F 1 "GND" H 4855 5877 50  0000 C CNN
 F 2 "" H 4850 6050 50  0001 C CNN
@@
 	6100 4350 6850 4350
 $Comp
-L power:GND #PWR089
+L power:GND #PWR038
 U 1 1 5FEF458A
 P 5350 6050
-F 0 "#PWR089" H 5350 5800 50  0001 C CNN
+F 0 "#PWR038" H 5350 5800 50  0001 C CNN
 F 1 "GND" H 5355 5877 50  0000 C CNN
 F 2 "" H 5350 6050 50  0001 C CNN
@@
 	6800 5400 6800 5450
 $Comp
-L power:GND #PWR085
+L power:GND #PWR034
 U 1 1 6016D996
 P 2150 6050
-F 0 "#PWR085" H 2150 5800 50  0001 C CNN
+F 0 "#PWR034" H 2150 5800 50  0001 C CNN
 F 1 "GND" H 2155 5877 50  0000 C CNN
 F 2 "" H 2150 6050 50  0001 C CNN
@@
 	4400 5400 6800 5400
 $Comp
-L power:GND #PWR087
+L power:GND #PWR036
 U 1 1 6021B8D1
 P 4400 6050
-F 0 "#PWR087" H 4400 5800 50  0001 C CNN
+F 0 "#PWR036" H 4400 5800 50  0001 C CNN
 F 1 "GND" H 4405 5877 50  0000 C CNN
 F 2 "" H 4400 6050 50  0001 C CNN
@@
 Connection ~ 4400 5400
 $Comp
-L Device:Q_NMOS_GSD Q3
+L Device:Q_NMOS_GSD Q2
 U 1 1 601EC337
 P 4300 5600
-F 0 "Q3" H 4350 5400 50  0000 C CNN
+F 0 "Q2" H 4350 5400 50  0000 C CNN
 F 1 "Q_NMOS_GSD" H 4150 5300 50  0000 C CNN
 F 2 "Package_TO_SOT_SMD:SOT-23" H 4500 5700 50  0001 C CNN
@@
 Connection ~ 4100 5600
 $Comp
-L power:+3.3V #PWR086
+L power:+3.3V #PWR035
 U 1 1 602901D6
 P 4250 1250
-F 0 "#PWR086" H 4250 1100 50  0001 C CNN
+F 0 "#PWR035" H 4250 1100 50  0001 C CNN
 F 1 "+3.3V" H 4265 1423 50  0000 C CNN
 F 2 "" H 4250 1250 50  0001 C CNN
@@
 	3900 2550 4900 2550
 $Comp
-L Device:R_Pack04 RN3
+L Device:R_Pack04 RN2
 U 1 1 5FEF4584
 P 5400 5750
-F 0 "RN3" H 5588 5796 50  0000 L CNN
+F 0 "RN2" H 5588 5796 50  0000 L CNN
 F 1 "100k" H 5588 5705 50  0000 L CNN
 F 2 "Resistor_SMD:R_Array_Convex_4x0603" V 5675 5750 50  0001 C CNN
@@
 $EndComp
 $Comp
-L Device:R_Pack04 RN4
+L Device:R_Pack04 RN3
 U 1 1 5FEC659D
 P 6300 5750
-F 0 "RN4" H 6488 5796 50  0000 L CNN
+F 0 "RN3" H 6488 5796 50  0000 L CNN
 F 1 "100k" H 6488 5705 50  0000 L CNN
 F 2 "Resistor_SMD:R_Array_Convex_4x0603" V 6575 5750 50  0001 C CNN
@@
 AR Path="/5E3BA64A/5F816B28" Ref="R?"  Part="1"
 AR Path="/5F51E414/5F816B28" Ref="R?"  Part="1"
-AR Path="/5FDC6C76/5F816B28" Ref="R29"  Part="1"
-F 0 "R29" V 4350 1350 50  0000 C CNN
+AR Path="/5FDC6C76/5F816B28" Ref="R19"  Part="1"
+F 0 "R19" V 4350 1350 50  0000 C CNN
 F 1 "100k" V 4400 1550 50  0000 C CNN
 F 2 "Resistor_SMD:R_0402_1005Metric" V 4330 1550 50  0001 C CNN
@@
 AR Path="/5E3BA64A/5F81FE16" Ref="R?"  Part="1"
 AR Path="/5F51E414/5F81FE16" Ref="R?"  Part="1"
-AR Path="/5FDC6C76/5F81FE16" Ref="R27"  Part="1"
-F 0 "R27" V 4150 1350 50  0000 C CNN
+AR Path="/5FDC6C76/5F81FE16" Ref="R17"  Part="1"
+F 0 "R17" V 4150 1350 50  0000 C CNN
 F 1 "100k" V 4200 1550 50  0000 C CNN
 F 2 "Resistor_SMD:R_0402_1005Metric" V 4130 1550 50  0001 C CNN
@@
 AR Path="/5E3BA64A/5F81FFF6" Ref="R?"  Part="1"
 AR Path="/5F51E414/5F81FFF6" Ref="R?"  Part="1"
-AR Path="/5FDC6C76/5F81FFF6" Ref="R26"  Part="1"
-F 0 "R26" V 4050 1350 50  0000 C CNN
+AR Path="/5FDC6C76/5F81FFF6" Ref="R16"  Part="1"
+F 0 "R16" V 4050 1350 50  0000 C CNN
 F 1 "100k" V 4100 1550 50  0000 C CNN
 F 2 "Resistor_SMD:R_0402_1005Metric" V 4030 1550 50  0001 C CNN
@@
 AR Path="/5E3BA64A/5F81FC54" Ref="R?"  Part="1"
 AR Path="/5F51E414/5F81FC54" Ref="R?"  Part="1"
-AR Path="/5FDC6C76/5F81FC54" Ref="R28"  Part="1"
-F 0 "R28" V 4250 1350 50  0000 C CNN
+AR Path="/5FDC6C76/5F81FC54" Ref="R18"  Part="1"
+F 0 "R18" V 4250 1350 50  0000 C CNN
 F 1 "100k" V 4300 1550 50  0000 C CNN
 F 2 "Resistor_SMD:R_0402_1005Metric" V 4230 1550 50  0001 C CNN
@@
 AR Path="/5E3BA64A/5F866853" Ref="R?"  Part="1"
 AR Path="/5F51E414/5F866853" Ref="R?"  Part="1"
-AR Path="/5FDC6C76/5F866853" Ref="R18"  Part="1"
-F 0 "R18" V 3650 2150 50  0000 C CNN
+AR Path="/5FDC6C76/5F866853" Ref="R12"  Part="1"
+F 0 "R12" V 3650 2150 50  0000 C CNN
 F 1 "47" V 3700 2350 50  0000 C CNN
 F 2 "Resistor_SMD:R_0402_1005Metric" V 3630 2350 50  0001 C CNN
@@
 AR Path="/5E3BA64A/5F869130" Ref="R?"  Part="1"
 AR Path="/5F51E414/5F869130" Ref="R?"  Part="1"
-AR Path="/5FDC6C76/5F869130" Ref="R19"  Part="1"
-F 0 "R19" V 3650 2250 50  0000 C CNN
+AR Path="/5FDC6C76/5F869130" Ref="R13"  Part="1"
+F 0 "R13" V 3650 2250 50  0000 C CNN
 F 1 "47" V 3700 2450 50  0000 C CNN
 F 2 "Resistor_SMD:R_0402_1005Metric" V 3630 2450 50  0001 C CNN
@@
 AR Path="/5E3BA64A/5F869489" Ref="R?"  Part="1"
 AR Path="/5F51E414/5F869489" Ref="R?"  Part="1"
-AR Path="/5FDC6C76/5F869489" Ref="R20"  Part="1"
-F 0 "R20" V 3650 2350 50  0000 C CNN
+AR Path="/5FDC6C76/5F869489" Ref="R14"  Part="1"
+F 0 "R14" V 3650 2350 50  0000 C CNN
 F 1 "47" V 3700 2550 50  0000 C CNN
 F 2 "Resistor_SMD:R_0402_1005Metric" V 3630 2550 50  0001 C CNN
@@
 AR Path="/5E3BA64A/5F8C896D" Ref="R?"  Part="1"
 AR Path="/5F51E414/5F8C896D" Ref="R?"  Part="1"
-AR Path="/5FDC6C76/5F8C896D" Ref="R25"  Part="1"
-F 0 "R25" V 3700 5600 50  0000 C CNN
+AR Path="/5FDC6C76/5F8C896D" Ref="R15"  Part="1"
+F 0 "R15" V 3700 5600 50  0000 C CNN
 F 1 "47" V 3800 5600 50  0000 C CNN
 F 2 "Resistor_SMD:R_0402_1005Metric" V 3730 5600 50  0001 C CNN
@@
 AR Path="/5E3BA64A/5F8D0A10" Ref="R?"  Part="1"
 AR Path="/5F51E414/5F8D0A10" Ref="R?"  Part="1"
-AR Path="/5FDC6C76/5F8D0A10" Ref="R32"  Part="1"
-F 0 "R32" V 4950 5950 50  0000 C CNN
+AR Path="/5FDC6C76/5F8D0A10" Ref="R21"  Part="1"
+F 0 "R21" V 4950 5950 50  0000 C CNN
 F 1 "100k" V 4900 5750 50  0000 C CNN
 F 2 "Resistor_SMD:R_0402_1005Metric" V 4830 5750 50  0001 C CNN
@@
 AR Path="/5E3BA64A/5F8D5CA4" Ref="R?"  Part="1"
 AR Path="/5F51E414/5F8D5CA4" Ref="R?"  Part="1"
-AR Path="/5FDC6C76/5F8D5CA4" Ref="R31"  Part="1"
-F 0 "R31" V 4850 5950 50  0000 C CNN
+AR Path="/5FDC6C76/5F8D5CA4" Ref="R20"  Part="1"
+F 0 "R20" V 4850 5950 50  0000 C CNN
 F 1 "100k" V 4800 5750 50  0000 C CNN
 F 2 "Resistor_SMD:R_0402_1005Metric" V 4730 5750 50  0001 C CNN
@@
 	2150 4850 2150 6050
 $Comp
-L Device:Q_NMOS_GSD Q2
+L Device:Q_NMOS_GSD Q1
 U 1 1 6005561C
 P 3150 4950
-F 0 "Q2" V 3050 5100 50  0000 C CNN
+F 0 "Q1" V 3050 5100 50  0000 C CNN
 F 1 "Q_NMOS_GSD" V 2900 5000 50  0000 C CNN
 F 2 "Package_TO_SOT_SMD:SOT-23" H 3350 5050 50  0001 C CNN

Commit message: Change pinout of expansion header close to board edge to be fully ground instead of gnd + 3.3v (& update component references)
Parts:
- J7: symbol Connector_Generic:Conn_01x40 -> mch2021-rescue:Conn_01x40-Connector_Generic
- Q1, Q2: symbol Device:Q_NMOS_GSD -> mch2021-rescue:Q_NMOS_GSD-Device
- R12, R13, R14, R15, R16, R17, R18, R19, R20, R21: symbol Device:R -> mch2021-rescue:R-Device
- RN1, RN2, RN3: symbol Device:R_Pack04 -> mch2021-rescue:R_Pack04-Device
- U2: symbol 74xGxx:74LVC1G125 -> mch2021-rescue:74LVC1G125-74xGxx
Changed lines of the file:
@@
 $EndDescr
 $Comp
-L Connector_Generic:Conn_01x40 J7
+L mch2021-rescue:Conn_01x40-Connector_Generic J7
 U 1 1 5FDC876E
 P 7050 3450
@@
 NoConn ~ 6850 1850
 $Comp
-L power:GND #PWR043
+L mch2021-rescue:GND-power #PWR043
 U 1 1 5FE093AF
 P 6750 6050
@@
 	6750 1950 6850 1950
 $Comp
-L power:+3.3V #PWR042
+L mch2021-rescue:+3.3V-power #PWR042
 U 1 1 5FE0C2BF
 P 6650 1250
@@
 Connection ~ 6650 2050
 $Comp
-L 74xGxx:74LVC1G125 U2
+L mch2021-rescue:74LVC1G125-74xGxx U2
 U 1 1 5FE0FF4D
 P 5800 2350
+AR Path="/5FE0FF4D" Ref="U2"  Part="1"
+AR Path="/5FDC6C76/5FE0FF4D" Ref="U2"  Part="1"
 F 0 "U2" H 6100 2550 50  0000 C CNN
 F 1 "74LVC1G125" H 6100 2450 50  0000 C CNN
@@
 $EndComp
 $Comp
-L power:+3.3V #PWR039
+L mch2021-rescue:+3.3V-power #PWR039
 U 1 1 5FE23AF8
 P 5850 1250
@@
 	6750 3850 6750 5150
 $Comp
-L power:GND #PWR041
+L mch2021-rescue:GND-power #PWR041
 U 1 1 5FEDB6BC
 P 6250 6050
@@
 $EndComp
 $Comp
-L power:GND #PWR040
+L mch2021-rescue:GND-power #PWR040
 U 1 1 5FEDBAA4
 P 5850 6050
@@
 $EndComp
 $Comp
-L power:GND #PWR037
+L mch2021-rescue:GND-power #PWR037
 U 1 1 5FEDBDD6
 P 4850 6050
@@
 	6100 4350 6850 4350
 $Comp
-L power:GND #PWR038
+L mch2021-rescue:GND-power #PWR038
 U 1 1 5FEF458A
 P 5350 6050
@@
 	6800 5400 6800 5450
 $Comp
-L power:GND #PWR034
+L mch2021-rescue:GND-power #PWR034
 U 1 1 6016D996
 P 2150 6050
@@
 	4400 5400 6800 5400
 $Comp
-L power:GND #PWR036
+L mch2021-rescue:GND-power #PWR036
 U 1 1 6021B8D1
 P 4400 6050
@@
 Connection ~ 4400 5400
 $Comp
-L Device:Q_NMOS_GSD Q2
+L mch2021-rescue:Q_NMOS_GSD-Device Q2
 U 1 1 601EC337
 P 4300 5600
@@
 Connection ~ 4100 5600
 $Comp
-L power:+3.3V #PWR035
+L mch2021-rescue:+3.3V-power #PWR035
 U 1 1 602901D6
 P 4250 1250
@@
 	3900 2550 4900 2550
 $Comp
-L Device:R_Pack04 RN2
+L mch2021-rescue:R_Pack04-Device RN2
 U 1 1 5FEF4584
 P 5400 5750
@@
 $EndComp
 $Comp
-L Device:R_Pack04 RN3
+L mch2021-rescue:R_Pack04-Device RN3
 U 1 1 5FEC659D
 P 6300 5750
@@
 LCD_K2
 $Comp
-L Device:R R?
+L mch2021-rescue:R-Device R?
 U 1 1 5F816B28
 P 4400 1550
@@
 $EndComp
 $Comp
-L Device:R R?
+L mch2021-rescue:R-Device R?
 U 1 1 5F81FE16
 P 4200 1550
@@
 $EndComp
 $Comp
-L Device:R R?
+L mch2021-rescue:R-Device R?
 U 1 1 5F81FFF6
 P 4100 1550
@@
 	4300 1300 4300 1400
 $Comp
-L Device:R R?
+L mch2021-rescue:R-Device R?
 U 1 1 5F81FC54
 P 4300 1550
@@
 $EndComp
 $Comp
-L Device:R R?
+L mch2021-rescue:R-Device R?
 U 1 1 5F866853
 P 3700 2350
@@
 	3850 2350 5400 2350
 $Comp
-L Device:R R?
+L mch2021-rescue:R-Device R?
 U 1 1 5F869130
 P 3700 2450
@@
 $EndComp
 $Comp
-L Device:R R?
+L mch2021-rescue:R-Device R?
 U 1 1 5F869489
 P 3700 2550
@@
 	3900 5050 6850 5050
 $Comp
-L Device:R R?
+L mch2021-rescue:R-Device R?
 U 1 1 5F8C896D
 P 3800 5600
@@
 $EndComp
 $Comp
-L Device:R R?
+L mch2021-rescue:R-Device R?
 U 1 1 5F8D0A10
 P 4900 5750
@@
 $EndComp
 $Comp
-L Device:R R?
+L mch2021-rescue:R-Device R?
 U 1 1 5F8D5CA4
 P 4800 5750
@@
 	2150 4850 2150 6050
 $Comp
-L Device:Q_NMOS_GSD Q1
+L mch2021-rescue:Q_NMOS_GSD-Device Q1
 U 1 1 6005561C
 P 3150 4950
@@
 	3400 4850 3500 4850
 $Comp
-L Device:R_Pack04 RN1
+L mch2021-rescue:R_Pack04-Device RN1
 U 1 1 6005D825
 P 3700 5050
