File: lcd.sch (KiCad schematic (older format))
At the start: 17 parts, among them J7 LCD, Q1 Q_NMOS_GSD, Q2 Q_NMOS_GSD, U2 74LVC1G125

Commit message: Last fixes before ordering
Parts:
- J7: LCSC C202114 -> C2856812; MANUFACTURER (none) -> XUNPU; MPN (none) -> FPC-05F-40PH20; Mouser - -> (none); Price (none) -> 0.757
- Q1, Q2: MANUFACTURER (none) -> ALLPOWER; MPN (none) -> AP2302B
- R12, R13, R14, R15: LCSC (none) -> C25168; MANUFACTURER (none) -> UNI-ROYAL; MPN (none) -> 0402WGJ0470TCE
- R16, R17, R18, R19, R20, R21: LCSC (none) -> C258090; MANUFACTURER (none) -> FH; MPN (none) -> RC-02W1003FT
- RN1: LCSC (none) -> C425204; MANUFACTURER (none) -> UNI-ROYAL; MPN (none) -> 4D03WGF470JT5E
- RN2, RN3: MANUFACTURER (none) -> UNI-ROYAL; MPN (none) -> 4D03WGF1003T5E
- U2: MPN (none) -> 74LVC1G125GW; Manufacturer (none) -> Nexperia; Mouser - -> (none)
Changed lines of the file:
@@
 F 1 "LCD" H 6968 1316 50  0000 C CNN
 F 2 "Connector_FFC-FPC:Hirose_FH12-40S-0.5SH_1x40-1MP_P0.50mm_Horizontal" H 7050 3450 50  0001 C CNN
-F 3 "~" H 7050 3450 50  0001 C CNN
-F 4 "C202114" H 7050 3450 50  0001 C CNN "LCSC"
-F 5 "-" H 7050 3450 50  0001 C CNN "Mouser"
-F 6 "" H 7050 3450 50  0001 C CNN "Price"
+F 3 "https://datasheet.lcsc.com/lcsc/2109221430_XUNPU-FPC-05F-40PH20_C2856812.pdf" H 7050 3450 50  0001 C CNN
+F 4 "C2856812" H 7050 3450 50  0001 C CNN "LCSC"
+F 5 "" H 7050 3450 50  0001 C CNN "Mouser"
+F 6 "0.757" H 7050 3450 50  0001 C CNN "Price"
 F 7 "N" H 7050 3450 50  0001 C CNN "Sponsored"
+F 8 "XUNPU" H 7050 3450 50  0001 C CNN "MANUFACTURER"
+F 9 "FPC-05F-40PH20" H 7050 3450 50  0001 C CNN "MPN"
 	1    7050 3450
 	1    0    0    -1
@@
 F 4 "C703585" H 5800 2350 50  0001 C CNN "LCSC"
 F 5 "" H 5800 2350 50  0001 C CNN "Price"
-F 6 "-" H 5800 2350 50  0001 C CNN "Mouser"
+F 6 "" H 5800 2350 50  0001 C CNN "Mouser"
 F 7 "N" H 5800 2350 50  0001 C CNN "Sponsored"
+F 8 "74LVC1G125GW" H 5800 2350 50  0001 C CNN "MPN"
+F 9 "Nexperia" H 5800 2350 50  0001 C CNN "Manufacturer"
 	1    5800 2350
 	1    0    0    -1
@@
 F 6 "" H 4300 5600 50  0001 C CNN "Price"
 F 7 "N" H 4300 5600 50  0001 C CNN "Sponsored"
+F 8 "ALLPOWER" H 4300 5600 50  0001 C CNN "MANUFACTURER"
+F 9 "AP2302B" H 4300 5600 50  0001 C CNN "MPN"
 	1    4300 5600
 	1    0    0    -1
@@
 F 6 "" H 5400 5750 50  0001 C CNN "Price"
 F 7 "N" H 5400 5750 50  0001 C CNN "Sponsored"
+F 8 "UNI-ROYAL" H 5400 5750 50  0001 C CNN "MANUFACTURER"
+F 9 "4D03WGF1003T5E" H 5400 5750 50  0001 C CNN "MPN"
 	1    5400 5750
 	1    0    0    -1
@@
 F 6 "" H 6300 5750 50  0001 C CNN "Price"
 F 7 "N" H 6300 5750 50  0001 C CNN "Sponsored"
+F 8 "UNI-ROYAL" H 6300 5750 50  0001 C CNN "MANUFACTURER"
+F 9 "4D03WGF1003T5E" H 6300 5750 50  0001 C CNN "MPN"
 	1    6300 5750
 	1    0    0    -1
@@
 F 2 "Resistor_SMD:R_0402_1005Metric" V 4330 1550 50  0001 C CNN
 F 3 "~" H 4400 1550 50  0001 C CNN
-F 4 "" H 4400 1550 50  0001 C CNN "LCSC"
+F 4 "C258090" H 4400 1550 50  0001 C CNN "LCSC"
 F 5 "" H 4400 1550 50  0001 C CNN "Price"
 F 6 "-" H 4400 1550 50  0001 C CNN "Mouser"
 F 7 "N" H 4400 1550 50  0001 C CNN "Sponsored"
+F 8 "FH" H 4400 1550 50  0001 C CNN "MANUFACTURER"
+F 9 "RC-02W1003FT" H 4400 1550 50  0001 C CNN "MPN"
 	1    4400 1550
 	1    0    0    -1
@@
 F 2 "Resistor_SMD:R_0402_1005Metric" V 4130 1550 50  0001 C CNN
 F 3 "~" H 4200 1550 50  0001 C CNN
-F 4 "" H 4200 1550 50  0001 C CNN "LCSC"
+F 4 "C258090" H 4200 1550 50  0001 C CNN "LCSC"
 F 5 "" H 4200 1550 50  0001 C CNN "Price"
 F 6 "-" H 4200 1550 50  0001 C CNN "Mouser"
 F 7 "N" H 4200 1550 50  0001 C CNN "Sponsored"
+F 8 "FH" H 4200 1550 50  0001 C CNN "MANUFACTURER"
+F 9 "RC-02W1003FT" H 4200 1550 50  0001 C CNN "MPN"
 	1    4200 1550
 	1    0    0    -1
@@
 F 2 "Resistor_SMD:R_0402_1005Metric" V 4030 1550 50  0001 C CNN
 F 3 "~" H 4100 1550 50  0001 C CNN
-F 4 "" H 4100 1550 50  0001 C CNN "LCSC"
+F 4 "C258090" H 4100 1550 50  0001 C CNN "LCSC"
 F 5 "" H 4100 1550 50  0001 C CNN "Price"
 F 6 "-" H 4100 1550 50  0001 C CNN "Mouser"
 F 7 "N" H 4100 1550 50  0001 C CNN "Sponsored"
+F 8 "FH" H 4100 1550 50  0001 C CNN "MANUFACTURER"
+F 9 "RC-02W1003FT" H 4100 1550 50  0001 C CNN "MPN"
 	1    4100 1550
 	1    0    0    -1
@@
 F 2 "Resistor_SMD:R_0402_1005Metric" V 4230 1550 50  0001 C CNN
 F 3 "~" H 4300 1550 50  0001 C CNN
-F 4 "" H 4300 1550 50  0001 C CNN "LCSC"
+F 4 "C258090" H 4300 1550 50  0001 C CNN "LCSC"
 F 5 "" H 4300 1550 50  0001 C CNN "Price"
 F 6 "-" H 4300 1550 50  0001 C CNN "Mouser"
 F 7 "N" H 4300 1550 50  0001 C CNN "Sponsored"
+F 8 "FH" H 4300 1550 50  0001 C CNN "MANUFACTURER"
+F 9 "RC-02W1003FT" H 4300 1550 50  0001 C CNN "MPN"
 	1    4300 1550
 	1    0    0    -1
@@
 F 2 "Resistor_SMD:R_0402_1005Metric" V 3630 2350 50  0001 C CNN
 F 3 "~" H 3700 2350 50  0001 C CNN
-F 4 "" H 3700 2350 50  0001 C CNN "LCSC"
+F 4 "C25168" H 3700 2350 50  0001 C CNN "LCSC"
 F 5 "" H 3700 2350 50  0001 C CNN "Price"
 F 6 "-" H 3700 2350 50  0001 C CNN "Mouser"
 F 7 "N" H 3700 2350 50  0001 C CNN "Sponsored"
+F 8 "UNI-ROYAL" H 3700 2350 50  0001 C CNN "MANUFACTURER"
+F 9 "0402WGJ0470TCE" H 3700 2350 50  0001 C CNN "MPN"
 	1    3700 2350
 	0    1    1    0
@@
 F 2 "Resistor_SMD:R_0402_1005Metric" V 3630 2450 50  0001 C CNN
 F 3 "~" H 3700 2450 50  0001 C CNN
-F 4 "" H 3700 2450 50  0001 C CNN "LCSC"
+F 4 "C25168" H 3700 2450 50  0001 C CNN "LCSC"
 F 5 "" H 3700 2450 50  0001 C CNN "Price"
 F 6 "-" H 3700 2450 50  0001 C CNN "Mouser"
 F 7 "N" H 3700 2450 50  0001 C CNN "Sponsored"
+F 8 "UNI-ROYAL" H 3700 2450 50  0001 C CNN "MANUFACTURER"
+F 9 "0402WGJ0470TCE" H 3700 2450 50  0001 C CNN "MPN"
 	1    3700 2450
 	0    1    1    0
@@
 F 2 "Resistor_SMD:R_0402_1005Metric" V 3630 2550 50  0001 C CNN
 F 3 "~" H 3700 2550 50  0001 C CNN
-F 4 "" H 3700 2550 50  0001 C CNN "LCSC"
+F 4 "C25168" H 3700 2550 50  0001 C CNN "LCSC"
 F 5 "" H 3700 2550 50  0001 C CNN "Price"
 F 6 "-" H 3700 2550 50  0001 C CNN "Mouser"
 F 7 "N" H 3700 2550 50  0001 C CNN "Sponsored"
+F 8 "UNI-ROYAL" H 3700 2550 50  0001 C CNN "MANUFACTURER"
+F 9 "0402WGJ0470TCE" H 3700 2550 50  0001 C CNN "MPN"
 	1    3700 2550
 	0    1    1    0
@@
 F 2 "Resistor_SMD:R_0402_1005Metric" V 3730 5600 50  0001 C CNN
 F 3 "~" H 3800 5600 50  0001 C CNN
-F 4 "" H 3800 5600 50  0001 C CNN "LCSC"
+F 4 "C25168" H 3800 5600 50  0001 C CNN "LCSC"
 F 5 "" H 3800 5600 50  0001 C CNN "Price"
 F 6 "-" H 3800 5600 50  0001 C CNN "Mouser"
 F 7 "N" H 3800 5600 50  0001 C CNN "Sponsored"
+F 8 "UNI-ROYAL" H 3800 5600 50  0001 C CNN "MANUFACTURER"
+F 9 "0402WGJ0470TCE" H 3800 5600 50  0001 C CNN "MPN"
 	1    3800 5600
 	0    1    1    0
@@
 F 2 "Resistor_SMD:R_0402_1005Metric" V 4830 5750 50  0001 C CNN
 F 3 "~" H 4900 5750 50  0001 C CNN
-F 4 "" H 4900 5750 50  0001 C CNN "LCSC"
+F 4 "C258090" H 4900 5750 50  0001 C CNN "LCSC"
 F 5 "" H 4900 5750 50  0001 C CNN "Price"
 F 6 "-" H 4900 5750 50  0001 C CNN "Mouser"
 F 7 "N" H 4900 5750 50  0001 C CNN "Sponsored"
+F 8 "FH" H 4900 5750 50  0001 C CNN "MANUFACTURER"
+F 9 "RC-02W1003FT" H 4900 5750 50  0001 C CNN "MPN"
 	1    4900 5750
 	-1   0    0    1
@@
 F 2 "Resistor_SMD:R_0402_1005Metric" V 4730 5750 50  0001 C CNN
 F 3 "~" H 4800 5750 50  0001 C CNN
-F 4 "" H 4800 5750 50  0001 C CNN "LCSC"
+F 4 "C258090" H 4800 5750 50  0001 C CNN "LCSC"
 F 5 "" H 4800 5750 50  0001 C CNN "Price"
 F 6 "-" H 4800 5750 50  0001 C CNN "Mouser"
 F 7 "N" H 4800 5750 50  0001 C CNN "Sponsored"
+F 8 "FH" H 4800 5750 50  0001 C CNN "MANUFACTURER"
+F 9 "RC-02W1003FT" H 4800 5750 50  0001 C CNN "MPN"
 	1    4800 5750
 	-1   0    0    1
@@
 F 6 "" H 3150 4950 50  0001 C CNN "Price"
 F 7 "N" H 3150 4950 50  0001 C CNN "Sponsored"
+F 8 "ALLPOWER" H 3150 4950 50  0001 C CNN "MANUFACTURER"
+F 9 "AP2302B" H 3150 4950 50  0001 C CNN "MPN"
 	1    3150 4950
 	0    1    -1   0
@@
 F 2 "Resistor_SMD:R_Array_Convex_4x0603" V 3975 5050 50  0001 C CNN
 F 3 "~" H 3700 5050 50  0001 C CNN
-F 4 "" H 3700 5050 50  0001 C CNN "LCSC"
+F 4 "C425204" H 3700 5050 50  0001 C CNN "LCSC"
 F 5 "-" H 3700 5050 50  0001 C CNN "Mouser"
 F 6 "" H 3700 5050 50  0001 C CNN "Price"
 F 7 "N" H 3700 5050 50  0001 C CNN "Sponsored"
+F 8 "UNI-ROYAL" H 3700 5050 50  0001 C CNN "MANUFACTURER"
+F 9 "4D03WGF470JT5E" H 3700 5050 50  0001 C CNN "MPN"
 	1    3700 5050
 	0    -1   1    0
