File: buttons.sch (KiCad schematic (older format))
At the start: 10 parts, among them SW2 Start, SW3 Select, SW4 Menu, SW5 Home, SW6 Back, SW7 Accept, U12 PCA9555PW

Commit message: First steps of routing prototype 2, switch to 0402 for most passives
Parts:
- C42: footprint Capacitor_SMD:C_0603_1608Metric -> Capacitor_SMD:C_0402_1005Metric; LCSC C14663 -> C83056
- R45: footprint Resistor_SMD:R_0603_1608Metric -> Resistor_SMD:R_0402_1005Metric; LCSC C269694 -> (none)
Other:
- note added: "I2C I/O expander"
- note removed: "MPR121 touch button interface"
Changed lines of the file:
@@
 $EndDescr
 Text Notes 550  700  0    79   ~ 0
-MPR121 touch button interface
+I2C I/O expander
 Text HLabel 4850 2100 2    50   Output ~ 0
 STM32_BOOT0
@@
 F 0 "C42" H 10992 6246 50  0000 L CNN
 F 1 "100n" H 10992 6155 50  0000 L CNN
-F 2 "Capacitor_SMD:C_0603_1608Metric" H 10900 6200 50  0001 C CNN
-F 3 "~" H 10900 6200 50  0001 C CNN
-F 4 "C14663" H 10900 6200 50  0001 C CNN "LCSC"
+F 2 "Capacitor_SMD:C_0402_1005Metric" H 10900 6200 50  0001 C CNN
+F 3 "" H 10900 6200 50  0001 C CNN
+F 4 "C83056 " H 10900 6200 50  0001 C CNN "LCSC"
 F 5 "" H 10900 6200 50  0001 C CNN "Price"
 F 6 "-" H 10900 6200 50  0001 C CNN "Mouser"
@@
 F 0 "R45" H 3859 1846 50  0000 L CNN
 F 1 "4k7" H 3859 1755 50  0000 L CNN
-F 2 "Resistor_SMD:R_0603_1608Metric" H 3800 1800 50  0001 C CNN
+F 2 "Resistor_SMD:R_0402_1005Metric" H 3800 1800 50  0001 C CNN
 F 3 "~" H 3800 1800 50  0001 C CNN
-F 4 "C269694" H 3800 1800 50  0001 C CNN "LCSC"
+F 4 "" H 3800 1800 50  0001 C CNN "LCSC"
 F 5 "N" H 3800 1800 50  0001 C CNN "Sponsored"
 	1    3800 1800

Commit message: Some more work
Parts:
- renumbered C42 to C14, R45 to R30, SW2 to SW1, SW3 to SW2, SW4 to SW3, SW5 to SW4, SW6 to SW5, SW7 to SW6, U12 to U4
Changed lines of the file:
@@
 STM32_BOOT0
 $Comp
-L Device:C_Small C42
+L Device:C_Small C14
 U 1 1 5F33C3B2
 P 10900 6200
-F 0 "C42" H 10992 6246 50  0000 L CNN
+F 0 "C14" H 10992 6246 50  0000 L CNN
 F 1 "100n" H 10992 6155 50  0000 L CNN
 F 2 "Capacitor_SMD:C_0402_1005Metric" H 10900 6200 50  0001 C CNN
@@
 $EndComp
 $Comp
-L power:GND #PWR0162
+L power:GND #PWR074
 U 1 1 5F33C3B8
 P 10900 6300
-F 0 "#PWR0162" H 10900 6050 50  0001 C CNN
+F 0 "#PWR074" H 10900 6050 50  0001 C CNN
 F 1 "GND" H 10905 6127 50  0000 C CNN
 F 2 "" H 10900 6300 50  0001 C CNN
@@
 $EndComp
 $Comp
-L power:+3.3V #PWR0161
+L power:+3.3V #PWR073
 U 1 1 5F33C3BE
 P 10900 6100
-F 0 "#PWR0161" H 10900 5950 50  0001 C CNN
+F 0 "#PWR073" H 10900 5950 50  0001 C CNN
 F 1 "+3.3V" H 10900 6250 50  0000 C CNN
 F 2 "" H 10900 6100 50  0001 C CNN
@@
 $EndComp
 $Comp
-L Interface_Expansion:PCA9555PW U12
+L Interface_Expansion:PCA9555PW U4
 U 1 1 5F5BEEA4
 P 4350 2800
-F 0 "U12" H 4000 1850 50  0000 C CNN
+F 0 "U4" H 4000 1850 50  0000 C CNN
 F 1 "PCA9555PW" H 4350 2800 50  0000 C CNN
 F 2 "Package_SO:TSSOP-24_4.4x7.8mm_P0.65mm" H 4350 2800 50  0001 C CNN
@@
 	3850 3400 3750 3400
 $Comp
-L power:GND #PWR0155
+L power:GND #PWR066
 U 1 1 5F5EA80A
 P 3750 3800
-F 0 "#PWR0155" H 3750 3550 50  0001 C CNN
+F 0 "#PWR066" H 3750 3550 50  0001 C CNN
 F 1 "GND" H 3755 3627 50  0000 C CNN
 F 2 "" H 3750 3800 50  0001 C CNN
@@
 $EndComp
 $Comp
-L power:GND #PWR0158
+L power:GND #PWR070
 U 1 1 5F5EABC3
 P 4350 3800
-F 0 "#PWR0158" H 4350 3550 50  0001 C CNN
+F 0 "#PWR070" H 4350 3550 50  0001 C CNN
 F 1 "GND" H 4355 3627 50  0000 C CNN
 F 2 "" H 4350 3800 50  0001 C CNN
@@
 $EndComp
 $Comp
-L power:GND #PWR0159
+L power:GND #PWR071
 U 1 1 5F61B54E
 P 5150 5800
-F 0 "#PWR0159" H 5150 5550 50  0001 C CNN
+F 0 "#PWR071" H 5150 5550 50  0001 C CNN
 F 1 "GND" H 5155 5627 50  0000 C CNN
 F 2 "" H 5150 5800 50  0001 C CNN
@@
 $EndComp
 $Comp
-L power:+3.3V #PWR0157
+L power:+3.3V #PWR069
 U 1 1 5F48E130
 P 4350 1700
-F 0 "#PWR0157" H 4350 1550 50  0001 C CNN
+F 0 "#PWR069" H 4350 1550 50  0001 C CNN
 F 1 "+3.3V" H 4365 1873 50  0000 C CNN
 F 2 "" H 4350 1700 50  0001 C CNN
@@
 $EndComp
 $Comp
-L power:+3.3V #PWR0156
+L power:+3.3V #PWR067
 U 1 1 5F48EC4C
 P 3800 1700
-F 0 "#PWR0156" H 3800 1550 50  0001 C CNN
+F 0 "#PWR067" H 3800 1550 50  0001 C CNN
 F 1 "+3.3V" H 3815 1873 50  0000 C CNN
 F 2 "" H 3800 1700 50  0001 C CNN
@@
 $EndComp
 $Comp
-L Device:R_Small R45
+L Device:R_Small R30
 U 1 1 5F4989F8
 P 3800 1800
-F 0 "R45" H 3859 1846 50  0000 L CNN
+F 0 "R30" H 3859 1846 50  0000 L CNN
 F 1 "4k7" H 3859 1755 50  0000 L CNN
 F 2 "Resistor_SMD:R_0402_1005Metric" H 3800 1800 50  0001 C CNN
@@
 	4850 2700 5600 2700
 $Comp
-L Switch:SW_Push SW5
+L Switch:SW_Push SW4
 U 1 1 5F5F70AF
 P 9050 4150
-F 0 "SW5" H 9050 4435 50  0000 C CNN
+F 0 "SW4" H 9050 4435 50  0000 C CNN
 F 1 "Home" H 9050 4344 50  0000 C CNN
 F 2 "custom:1TS009" H 9050 4350 50  0001 C CNN
@@
 $EndComp
 $Comp
-L Switch:SW_Push SW2
+L Switch:SW_Push SW1
 U 1 1 5F601049
 P 9050 2950
-F 0 "SW2" H 9050 3235 50  0000 C CNN
+F 0 "SW1" H 9050 3235 50  0000 C CNN
 F 1 "Start" H 9050 3144 50  0000 C CNN
 F 2 "custom:1TS009" H 9050 3150 50  0001 C CNN
@@
 $EndComp
 $Comp
-L Switch:SW_Push SW6
+L Switch:SW_Push SW5
 U 1 1 5F5F70A3
 P 9050 4550
-F 0 "SW6" H 9050 4835 50  0000 C CNN
+F 0 "SW5" H 9050 4835 50  0000 C CNN
 F 1 "Back" H 9050 4744 50  0000 C CNN
 F 2 "custom:1TS009" H 9050 4750 50  0001 C CNN
@@
 $EndComp
 $Comp
-L Switch:SW_Push SW7
+L Switch:SW_Push SW6
 U 1 1 5F5F709D
 P 9050 4950
-F 0 "SW7" H 9050 5235 50  0000 C CNN
+F 0 "SW6" H 9050 5235 50  0000 C CNN
 F 1 "Accept" H 9050 5144 50  0000 C CNN
 F 2 "custom:1TS009" H 9050 5150 50  0001 C CNN
@@
 $EndComp
 $Comp
-L Switch:SW_Push SW3
+L Switch:SW_Push SW2
 U 1 1 5F60575E
 P 9050 3350
-F 0 "SW3" H 9050 3635 50  0000 C CNN
+F 0 "SW2" H 9050 3635 50  0000 C CNN
 F 1 "Select" H 9050 3544 50  0000 C CNN
 F 2 "custom:1TS009" H 9050 3550 50  0001 C CNN
@@
 Connection ~ 9350 4950
 $Comp
-L power:GND #PWR0160
+L power:GND #PWR072
 U 1 1 5F64058E
 P 9350 5000
-F 0 "#PWR0160" H 9350 4750 50  0001 C CNN
+F 0 "#PWR072" H 9350 4750 50  0001 C CNN
 F 1 "GND" H 9355 4827 50  0000 C CNN
 F 2 "" H 9350 5000 50  0001 C CNN
@@
 	9250 3750 9350 3750
 $Comp
-L Switch:SW_Push SW4
+L Switch:SW_Push SW3
 U 1 1 5F5F70A9
 P 9050 3750
-F 0 "SW4" H 9050 4035 50  0000 C CNN
+F 0 "SW3" H 9050 4035 50  0000 C CNN
 F 1 "Menu" H 9050 3944 50  0000 C CNN
 F 2 "custom:1TS009" H 9050 3950 50  0001 C CNN
@@
 	3650 3500 3650 3300
 $Comp
-L power:+3.3V #PWR0175
+L power:+3.3V #PWR065
 U 1 1 5FA973E7
 P 3650 3300
-F 0 "#PWR0175" H 3650 3150 50  0001 C CNN
+F 0 "#PWR065" H 3650 3150 50  0001 C CNN
 F 1 "+3.3V" H 3665 3473 50  0000 C CNN
 F 2 "" H 3650 3300 50  0001 C CNN
@@
 $EndComp
 $Comp
-L power:GND #PWR0176
+L power:GND #PWR068
 U 1 1 5FBEF4DF
 P 4050 5800
-F 0 "#PWR0176" H 4050 5550 50  0001 C CNN
+F 0 "#PWR068" H 4050 5550 50  0001 C CNN
 F 1 "GND" H 4055 5627 50  0000 C CNN
 F 2 "" H 4050 5800 50  0001 C CNN

Commit message: Moar fixes
Parts:
- SW5: value Back -> B
- SW6: value Accept -> A
Connections:
- net BTN_BACK: now reaches SW5.1, U4.19 (IO1_6)
- net BTN_ACCEPT: now reaches SW6.1, U4.20 (IO1_7)
Changed lines of the file:
@@
 P 9050 4550
 F 0 "SW5" H 9050 4835 50  0000 C CNN
-F 1 "Back" H 9050 4744 50  0000 C CNN
+F 1 "B" H 9050 4744 50  0000 C CNN
 F 2 "custom:1TS009" H 9050 4750 50  0001 C CNN
 F 3 "~" H 9050 4750 50  0001 C CNN
@@
 P 9050 4950
 F 0 "SW6" H 9050 5235 50  0000 C CNN
-F 1 "Accept" H 9050 5144 50  0000 C CNN
+F 1 "A" H 9050 5144 50  0000 C CNN
 F 2 "custom:1TS009" H 9050 5150 50  0001 C CNN
 F 3 "~" H 9050 5150 50  0001 C CNN
@@
 Text HLabel 4850 2400 2    50   Output ~ 0
 BNO055_RESET
+Text Label 8250 4550 0    50   ~ 0
+BTN_BACK
+Text Label 8250 4950 0    50   ~ 0
+BTN_ACCEPT
 $EndSCHEMATC

Commit message: Change button LCSC id (and 3d stuff)
Parts:
- SW1, SW2, SW3, SW4, SW5, SW6: LCSC C255817 -> C115348
Changed lines of the file:
@@
 F 3 "~" H 9050 4350 50  0001 C CNN
 F 4 "N" H 9050 4150 50  0001 C CNN "Sponsored"
-F 5 "C255817" H 9050 4150 50  0001 C CNN "LCSC"
+F 5 "C115348" H 9050 4150 50  0001 C CNN "LCSC"
 F 6 "" H 9050 4150 50  0001 C CNN "Price"
 	1    9050 4150
@@
 F 3 "~" H 9050 3150 50  0001 C CNN
 F 4 "N" H 9050 2950 50  0001 C CNN "Sponsored"
-F 5 "C255817" H 9050 2950 50  0001 C CNN "LCSC"
+F 5 "C115348" H 9050 2950 50  0001 C CNN "LCSC"
 F 6 "" H 9050 2950 50  0001 C CNN "Price"
 	1    9050 2950
@@
 F 3 "~" H 9050 4750 50  0001 C CNN
 F 4 "N" H 9050 4550 50  0001 C CNN "Sponsored"
-F 5 "C255817" H 9050 4550 50  0001 C CNN "LCSC"
+F 5 "C115348" H 9050 4550 50  0001 C CNN "LCSC"
 F 6 "" H 9050 4550 50  0001 C CNN "Price"
 	1    9050 4550
@@
 F 3 "~" H 9050 5150 50  0001 C CNN
 F 4 "N" H 9050 4950 50  0001 C CNN "Sponsored"
-F 5 "C255817" H 9050 4950 50  0001 C CNN "LCSC"
+F 5 "C115348" H 9050 4950 50  0001 C CNN "LCSC"
 F 6 "" H 9050 4950 50  0001 C CNN "Price"
 	1    9050 4950
@@
 F 3 "~" H 9050 3550 50  0001 C CNN
 F 4 "N" H 9050 3350 50  0001 C CNN "Sponsored"
-F 5 "C255817" H 9050 3350 50  0001 C CNN "LCSC"
+F 5 "C115348" H 9050 3350 50  0001 C CNN "LCSC"
 F 6 "" H 9050 3350 50  0001 C CNN "Price"
 	1    9050 3350
@@
 F 3 "~" H 9050 3950 50  0001 C CNN
 F 4 "N" H 9050 3750 50  0001 C CNN "Sponsored"
-F 5 "C255817" H 9050 3750 50  0001 C CNN "LCSC"
+F 5 "C115348" H 9050 3750 50  0001 C CNN "LCSC"
 F 6 "" H 9050 3750 50  0001 C CNN "Price"
 	1    9050 3750

Commit message: Change pinout of expansion header close to board edge to be fully ground instead of gnd + 3.3v (& update component references)
Parts:
- C14: symbol Device:C_Small -> mch2021-rescue:C_Small-Device
- R30: symbol Device:R_Small -> mch2021-rescue:R_Small-Device
- SW1, SW2, SW3, SW4, SW5, SW6: symbol Switch:SW_Push -> mch2021-rescue:SW_Push-Switch
- U4: symbol Interface_Expansion:PCA9555PW -> mch2021-rescue:PCA9555PW-Interface_Expansion
Changed lines of the file:
@@
 STM32_BOOT0
 $Comp
-L Device:C_Small C14
+L mch2021-rescue:C_Small-Device C14
 U 1 1 5F33C3B2
 P 10900 6200
@@
 $EndComp
 $Comp
-L power:GND #PWR074
+L mch2021-rescue:GND-power #PWR074
 U 1 1 5F33C3B8
 P 10900 6300
@@
 $EndComp
 $Comp
-L power:+3.3V #PWR073
+L mch2021-rescue:+3.3V-power #PWR073
 U 1 1 5F33C3BE
 P 10900 6100
@@
 $EndComp
 $Comp
-L Interface_Expansion:PCA9555PW U4
+L mch2021-rescue:PCA9555PW-Interface_Expansion U4
 U 1 1 5F5BEEA4
 P 4350 2800
@@
 	3850 3400 3750 3400
 $Comp
-L power:GND #PWR066
+L mch2021-rescue:GND-power #PWR066
 U 1 1 5F5EA80A
 P 3750 3800
@@
 $EndComp
 $Comp
-L power:GND #PWR070
+L mch2021-rescue:GND-power #PWR070
 U 1 1 5F5EABC3
 P 4350 3800
@@
 $EndComp
 $Comp
-L power:GND #PWR071
+L mch2021-rescue:GND-power #PWR071
 U 1 1 5F61B54E
 P 5150 5800
@@
 $EndComp
 $Comp
-L power:+3.3V #PWR069
+L mch2021-rescue:+3.3V-power #PWR069
 U 1 1 5F48E130
 P 4350 1700
@@
 $EndComp
 $Comp
-L power:+3.3V #PWR067
+L mch2021-rescue:+3.3V-power #PWR067
 U 1 1 5F48EC4C
 P 3800 1700
@@
 $EndComp
 $Comp
-L Device:R_Small R30
+L mch2021-rescue:R_Small-Device R30
 U 1 1 5F4989F8
 P 3800 1800
@@
 	4850 2700 5600 2700
 $Comp
-L Switch:SW_Push SW4
+L mch2021-rescue:SW_Push-Switch SW4
 U 1 1 5F5F70AF
 P 9050 4150
@@
 $EndComp
 $Comp
-L Switch:SW_Push SW1
+L mch2021-rescue:SW_Push-Switch SW1
 U 1 1 5F601049
 P 9050 2950
@@
 $EndComp
 $Comp
-L Switch:SW_Push SW5
+L mch2021-rescue:SW_Push-Switch SW5
 U 1 1 5F5F70A3
 P 9050 4550
@@
 $EndComp
 $Comp
-L Switch:SW_Push SW6
+L mch2021-rescue:SW_Push-Switch SW6
 U 1 1 5F5F709D
 P 9050 4950
@@
 $EndComp
 $Comp
-L Switch:SW_Push SW2
+L mch2021-rescue:SW_Push-Switch SW2
 U 1 1 5F60575E
 P 9050 3350
@@
 Connection ~ 9350 4950
 $Comp
-L power:GND #PWR072
+L mch2021-rescue:GND-power #PWR072
 U 1 1 5F64058E
 P 9350 5000
@@
 	9250 3750 9350 3750
 $Comp
-L Switch:SW_Push SW3
+L mch2021-rescue:SW_Push-Switch SW3
 U 1 1 5F5F70A9
 P 9050 3750
@@
 	3650 3500 3650 3300
 $Comp
-L power:+3.3V #PWR065
+L mch2021-rescue:+3.3V-power #PWR065
 U 1 1 5FA973E7
 P 3650 3300
@@
 $EndComp
 $Comp
-L power:GND #PWR068
+L mch2021-rescue:GND-power #PWR068
 U 1 1 5FBEF4DF
 P 4050 5800
