File: buttons.sch (KiCad schematic (older format))
At the start: 10 parts, among them SW1 Start, SW2 Select, SW3 Menu, SW4 Home, SW5 B, SW6 A, U4 PCA9555PW

Commit message: More work on RP2040 integration
Connections:
- net STM32_BOOT0 renamed RP2040_BOOT
- net STM32_RESET renamed RP2040_RESET
Changed lines of the file:
@@
 I2C I/O expander
 Text HLabel 4850 2100 2    50   Output ~ 0
-STM32_BOOT0
+RP2040_BOOT
 $Comp
 L mch2021-rescue:C_Small-Device C14
@@
 	5550 4150 8850 4150
 Text HLabel 4850 2000 2    50   Output ~ 0
-STM32_RESET
+RP2040_RESET
 Wire Wire Line
 	8850 3350 5650 3350

Commit message: Last fixes before ordering
Parts:
- R30: value 4k7 -> 4.7k; LCSC (none) -> C25940; MANUFACTURER (none) -> UNI-ROYAL; MPN (none) -> 0402WGJ0472TCE
Changed lines of the file:
@@
 P 3800 1800
 F 0 "R30" H 3859 1846 50  0000 L CNN
-F 1 "4k7" H 3859 1755 50  0000 L CNN
+F 1 "4.7k" H 3859 1755 50  0000 L CNN
 F 2 "Resistor_SMD:R_0402_1005Metric" H 3800 1800 50  0001 C CNN
 F 3 "~" H 3800 1800 50  0001 C CNN
-F 4 "" H 3800 1800 50  0001 C CNN "LCSC"
+F 4 "C25940" H 3800 1800 50  0001 C CNN "LCSC"
 F 5 "N" H 3800 1800 50  0001 C CNN "Sponsored"
+F 6 "UNI-ROYAL" H 3800 1800 50  0001 C CNN "MANUFACTURER"
+F 7 "0402WGJ0472TCE" H 3800 1800 50  0001 C CNN "MPN"
 	1    3800 1800
 	1    0    0    -1
