File: led.sch (KiCad schematic (older format))
At the start: 12 parts

Commit message: Dump.
Parts:
- removed D3: WS2812B, corelib:SK6212SIDE, symbol LED:WS2812B
- added D4: WS2812B, LED_SMD:LED_WS2812B_PLCC4_5.0x5.0mm_P3.2mm, symbol LED:WS2812B
- C27: renamed from C34; footprint Capacitor_SMD:C_0402_1005Metric -> Capacitor_SMD:C_0603_1608Metric; Price (none) -> 0.0020; Sponsored (none) -> N
- C28: renamed from C35; footprint Capacitor_SMD:C_0402_1005Metric -> Capacitor_SMD:C_0603_1608Metric; Price (none) -> 0.0020; Sponsored (none) -> N
- C29: renamed from C36; footprint Capacitor_SMD:C_0402_1005Metric -> Capacitor_SMD:C_0603_1608Metric; Price (none) -> 0.0020; Sponsored (none) -> N
- C30: renamed from C37; footprint Capacitor_SMD:C_0402_1005Metric -> Capacitor_SMD:C_0603_1608Metric; Price (none) -> 0.0020; Sponsored (none) -> N
- C31: renamed from C38; footprint Capacitor_SMD:C_0402_1005Metric -> Capacitor_SMD:C_0603_1608Metric; Price (none) -> 0.0020; Sponsored (none) -> N
- C32: renamed from C39; footprint Capacitor_SMD:C_0402_1005Metric -> Capacitor_SMD:C_0603_1608Metric; Price (none) -> 0.0020; Sponsored (none) -> N
- D5: renamed from D4; footprint corelib:SK6212SIDE -> LED_SMD:LED_WS2812B_PLCC4_5.0x5.0mm_P3.2mm; LCSC (none) -> C139127; Mouser (none) -> -; Price (none) -> 0.037; Sponsored (none) -> N
- D6: renamed from D5; footprint corelib:SK6212SIDE -> LED_SMD:LED_WS2812B_PLCC4_5.0x5.0mm_P3.2mm; LCSC (none) -> C139127; Mouser (none) -> -; Price (none) -> 0.037; Sponsored (none) -> N
- D7: renamed from D6; footprint corelib:SK6212SIDE -> LED_SMD:LED_WS2812B_PLCC4_5.0x5.0mm_P3.2mm; LCSC (none) -> C139127; Mouser (none) -> -; Price (none) -> 0.037; Sponsored (none) -> N
- D8: renamed from D7; footprint corelib:SK6212SIDE -> LED_SMD:LED_WS2812B_PLCC4_5.0x5.0mm_P3.2mm; LCSC (none) -> C139127; Mouser (none) -> -; Price (none) -> 0.037; Sponsored (none) -> N
- D9: renamed from D8; footprint corelib:SK6212SIDE -> LED_SMD:LED_WS2812B_PLCC4_5.0x5.0mm_P3.2mm; LCSC (none) -> C139127; Mouser (none) -> -; Price (none) -> 0.037; Sponsored (none) -> N
Connections:
- net DATA_IN: now also D4.4 (DIN)
- net GND: now also D4.3 (VSS)
- net PWR_LED: now also D4.1 (VDD)
- net at D5.4 (DIN): now also D4.2 (DOUT)
Changed lines of the file:
@@
 $Descr A4 11693 8268
 encoding utf-8
-Sheet 8 9
+Sheet 5 9
 Title ""
 Date ""
@@
 $EndDescr
 $Comp
-L LED:WS2812B D3
-U 1 1 60C79CD3
+L LED:WS2812B D4
+U 1 1 5F7D8169
 P 4300 4050
-F 0 "D3" H 4100 4300 50  0000 L CNN
+F 0 "D4" H 4100 4300 50  0000 L CNN
 F 1 "WS2812B" V 4450 4300 50  0000 L CNN
-F 2 "corelib:SK6212SIDE" H 4350 3750 50  0001 L TNN
+F 2 "LED_SMD:LED_WS2812B_PLCC4_5.0x5.0mm_P3.2mm" H 4350 3750 50  0001 L TNN
 F 3 "https://cdn-shop.adafruit.com/datasheets/WS2812B.pdf" H 4400 3675 50  0001 L TNN
+F 4 "C139127" H 4300 4050 50  0001 C CNN "LCSC"
+F 5 "-" H 4300 4050 50  0001 C CNN "Mouser"
+F 6 "0.037" H 4300 4050 50  0001 C CNN "Price"
+F 7 "N" H 4300 4050 50  0001 C CNN "Sponsored"
 	1    4300 4050
 	1    0    0    -1
 $EndComp
 $Comp
-L power:GND #PWR0147
+L power:GND #PWR0120
 U 1 1 612C7A49
 P 4300 4350
-F 0 "#PWR0147" H 4300 4100 50  0001 C CNN
+F 0 "#PWR0120" H 4300 4100 50  0001 C CNN
 F 1 "GND" H 4305 4177 50  0000 C CNN
 F 2 "" H 4300 4350 50  0001 C CNN
@@
 PWR_LED
 $Comp
-L LED:WS2812B D4
+L LED:WS2812B D5
 U 1 1 612CEAF2
 P 4900 4050
-F 0 "D4" H 4700 4300 50  0000 L CNN
+F 0 "D5" H 4700 4300 50  0000 L CNN
 F 1 "WS2812B" V 5050 4300 50  0000 L CNN
-F 2 "corelib:SK6212SIDE" H 4950 3750 50  0001 L TNN
+F 2 "LED_SMD:LED_WS2812B_PLCC4_5.0x5.0mm_P3.2mm" H 4950 3750 50  0001 L TNN
 F 3 "https://cdn-shop.adafruit.com/datasheets/WS2812B.pdf" H 5000 3675 50  0001 L TNN
+F 4 "C139127" H 4900 4050 50  0001 C CNN "LCSC"
+F 5 "-" H 4900 4050 50  0001 C CNN "Mouser"
+F 6 "0.037" H 4900 4050 50  0001 C CNN "Price"
+F 7 "N" H 4900 4050 50  0001 C CNN "Sponsored"
 	1    4900 4050
 	1    0    0    -1
 $EndComp
 $Comp
-L power:GND #PWR0148
+L power:GND #PWR0121
 U 1 1 612CEAF8
 P 4900 4350
-F 0 "#PWR0148" H 4900 4100 50  0001 C CNN
+F 0 "#PWR0121" H 4900 4100 50  0001 C CNN
 F 1 "GND" H 4905 4177 50  0000 C CNN
 F 2 "" H 4900 4350 50  0001 C CNN
@@
 PWR_LED
 $Comp
-L LED:WS2812B D5
+L LED:WS2812B D6
 U 1 1 612CEE91
 P 5500 4050
-F 0 "D5" H 5300 4300 50  0000 L CNN
+F 0 "D6" H 5300 4300 50  0000 L CNN
 F 1 "WS2812B" V 5650 4300 50  0000 L CNN
-F 2 "corelib:SK6212SIDE" H 5550 3750 50  0001 L TNN
+F 2 "LED_SMD:LED_WS2812B_PLCC4_5.0x5.0mm_P3.2mm" H 5550 3750 50  0001 L TNN
 F 3 "https://cdn-shop.adafruit.com/datasheets/WS2812B.pdf" H 5600 3675 50  0001 L TNN
+F 4 "C139127" H 5500 4050 50  0001 C CNN "LCSC"
+F 5 "-" H 5500 4050 50  0001 C CNN "Mouser"
+F 6 "0.037" H 5500 4050 50  0001 C CNN "Price"
+F 7 "N" H 5500 4050 50  0001 C CNN "Sponsored"
 	1    5500 4050
 	1    0    0    -1
 $EndComp
 $Comp
-L power:GND #PWR0149
+L power:GND #PWR0122
 U 1 1 612CEE97
 P 5500 4350
-F 0 "#PWR0149" H 5500 4100 50  0001 C CNN
+F 0 "#PWR0122" H 5500 4100 50  0001 C CNN
 F 1 "GND" H 5505 4177 50  0000 C CNN
 F 2 "" H 5500 4350 50  0001 C CNN
@@
 PWR_LED
 $Comp
-L LED:WS2812B D6
+L LED:WS2812B D7
 U 1 1 612CF6E4
 P 6100 4050
-F 0 "D6" H 5900 4300 50  0000 L CNN
+F 0 "D7" H 5900 4300 50  0000 L CNN
 F 1 "WS2812B" V 6250 4300 50  0000 L CNN
-F 2 "corelib:SK6212SIDE" H 6150 3750 50  0001 L TNN
+F 2 "LED_SMD:LED_WS2812B_PLCC4_5.0x5.0mm_P3.2mm" H 6150 3750 50  0001 L TNN
 F 3 "https://cdn-shop.adafruit.com/datasheets/WS2812B.pdf" H 6200 3675 50  0001 L TNN
+F 4 "C139127" H 6100 4050 50  0001 C CNN "LCSC"
+F 5 "-" H 6100 4050 50  0001 C CNN "Mouser"
+F 6 "0.037" H 6100 4050 50  0001 C CNN "Price"
+F 7 "N" H 6100 4050 50  0001 C CNN "Sponsored"
 	1    6100 4050
 	1    0    0    -1
 $EndComp
 $Comp
-L power:GND #PWR0150
+L power:GND #PWR0123
 U 1 1 612CF6EA
 P 6100 4350
-F 0 "#PWR0150" H 6100 4100 50  0001 C CNN
+F 0 "#PWR0123" H 6100 4100 50  0001 C CNN
 F 1 "GND" H 6105 4177 50  0000 C CNN
 F 2 "" H 6100 4350 50  0001 C CNN
@@
 PWR_LED
 $Comp
-L LED:WS2812B D7
+L LED:WS2812B D8
 U 1 1 612CFE55
 P 6700 4050
-F 0 "D7" H 6500 4300 50  0000 L CNN
+F 0 "D8" H 6500 4300 50  0000 L CNN
 F 1 "WS2812B" V 6850 4300 50  0000 L CNN
-F 2 "corelib:SK6212SIDE" H 6750 3750 50  0001 L TNN
+F 2 "LED_SMD:LED_WS2812B_PLCC4_5.0x5.0mm_P3.2mm" H 6750 3750 50  0001 L TNN
 F 3 "https://cdn-shop.adafruit.com/datasheets/WS2812B.pdf" H 6800 3675 50  0001 L TNN
+F 4 "C139127" H 6700 4050 50  0001 C CNN "LCSC"
+F 5 "-" H 6700 4050 50  0001 C CNN "Mouser"
+F 6 "0.037" H 6700 4050 50  0001 C CNN "Price"
+F 7 "N" H 6700 4050 50  0001 C CNN "Sponsored"
 	1    6700 4050
 	1    0    0    -1
 $EndComp
 $Comp
-L power:GND #PWR0151
+L power:GND #PWR0124
 U 1 1 612CFE5B
 P 6700 4350
-F 0 "#PWR0151" H 6700 4100 50  0001 C CNN
+F 0 "#PWR0124" H 6700 4100 50  0001 C CNN
 F 1 "GND" H 6705 4177 50  0000 C CNN
 F 2 "" H 6700 4350 50  0001 C CNN
@@
 PWR_LED
 $Comp
-L LED:WS2812B D8
+L LED:WS2812B D9
 U 1 1 612D0799
 P 7300 4050
-F 0 "D8" H 7100 4300 50  0000 L CNN
+F 0 "D9" H 7100 4300 50  0000 L CNN
 F 1 "WS2812B" V 7450 4300 50  0000 L CNN
-F 2 "corelib:SK6212SIDE" H 7350 3750 50  0001 L TNN
+F 2 "LED_SMD:LED_WS2812B_PLCC4_5.0x5.0mm_P3.2mm" H 7350 3750 50  0001 L TNN
 F 3 "https://cdn-shop.adafruit.com/datasheets/WS2812B.pdf" H 7400 3675 50  0001 L TNN
+F 4 "C139127" H 7300 4050 50  0001 C CNN "LCSC"
+F 5 "-" H 7300 4050 50  0001 C CNN "Mouser"
+F 6 "0.037" H 7300 4050 50  0001 C CNN "Price"
+F 7 "N" H 7300 4050 50  0001 C CNN "Sponsored"
 	1    7300 4050
 	1    0    0    -1
 $EndComp
 $Comp
-L power:GND #PWR0152
+L power:GND #PWR0125
 U 1 1 612D079F
 P 7300 4350
-F 0 "#PWR0152" H 7300 4100 50  0001 C CNN
+F 0 "#PWR0125" H 7300 4100 50  0001 C CNN
 F 1 "GND" H 7305 4177 50  0000 C CNN
 F 2 "" H 7300 4350 50  0001 C CNN
@@
 PWR_LED
 $Comp
-L Device:C C34
+L Device:C C27
 U 1 1 612D0DFB
 P 9150 6050
-F 0 "C34" H 9265 6096 50  0000 L CNN
+F 0 "C27" H 9265 6096 50  0000 L CNN
 F 1 "1u" H 9265 6005 50  0000 L CNN
-F 2 "Capacitor_SMD:C_0402_1005Metric" H 9188 5900 50  0001 C CNN
+F 2 "Capacitor_SMD:C_0603_1608Metric" H 9188 5900 50  0001 C CNN
 F 3 "~" H 9150 6050 50  0001 C CNN
+F 4 "0.0020" H 9150 6050 50  0001 C CNN "Price"
+F 5 "N" H 9150 6050 50  0001 C CNN "Sponsored"
 	1    9150 6050
 	-1   0    0    -1
 $EndComp
 $Comp
-L power:GND #PWR0153
+L power:GND #PWR0126
 U 1 1 612D0F05
 P 9150 6200
-F 0 "#PWR0153" H 9150 5950 50  0001 C CNN
+F 0 "#PWR0126" H 9150 5950 50  0001 C CNN
 F 1 "GND" H 9155 6027 50  0000 C CNN
 F 2 "" H 9150 6200 50  0001 C CNN
@@
 PWR_LED
 $Comp
-L Device:C C35
+L Device:C C28
 U 1 1 612D2985
 P 9500 6050
-F 0 "C35" H 9615 6096 50  0000 L CNN
+F 0 "C28" H 9615 6096 50  0000 L CNN
 F 1 "1u" H 9615 6005 50  0000 L CNN
-F 2 "Capacitor_SMD:C_0402_1005Metric" H 9538 5900 50  0001 C CNN
+F 2 "Capacitor_SMD:C_0603_1608Metric" H 9538 5900 50  0001 C CNN
 F 3 "~" H 9500 6050 50  0001 C CNN
+F 4 "0.0020" H 9500 6050 50  0001 C CNN "Price"
+F 5 "N" H 9500 6050 50  0001 C CNN "Sponsored"
 	1    9500 6050
 	-1   0    0    -1
 $EndComp
 $Comp
-L power:GND #PWR0154
+L power:GND #PWR0127
 U 1 1 612D298B
 P 9500 6200
-F 0 "#PWR0154" H 9500 5950 50  0001 C CNN
+F 0 "#PWR0127" H 9500 5950 50  0001 C CNN
 F 1 "GND" H 9505 6027 50  0000 C CNN
 F 2 "" H 9500 6200 50  0001 C CNN
@@
 PWR_LED
 $Comp
-L Device:C C36
+L Device:C C29
 U 1 1 612D3CA5
 P 9850 6050
-F 0 "C36" H 9965 6096 50  0000 L CNN
+F 0 "C29" H 9965 6096 50  0000 L CNN
 F 1 "1u" H 9965 6005 50  0000 L CNN
-F 2 "Capacitor_SMD:C_0402_1005Metric" H 9888 5900 50  0001 C CNN
+F 2 "Capacitor_SMD:C_0603_1608Metric" H 9888 5900 50  0001 C CNN
 F 3 "~" H 9850 6050 50  0001 C CNN
+F 4 "0.0020" H 9850 6050 50  0001 C CNN "Price"
+F 5 "N" H 9850 6050 50  0001 C CNN "Sponsored"
 	1    9850 6050
 	-1   0    0    -1
 $EndComp
 $Comp
-L power:GND #PWR0155
+L power:GND #PWR0128
 U 1 1 612D3CAB
 P 9850 6200
-F 0 "#PWR0155" H 9850 5950 50  0001 C CNN
+F 0 "#PWR0128" H 9850 5950 50  0001 C CNN
 F 1 "GND" H 9855 6027 50  0000 C CNN
 F 2 "" H 9850 6200 50  0001 C CNN
@@
 PWR_LED
 $Comp
-L Device:C C37
+L Device:C C30
 U 1 1 612D4333
 P 10200 6050
-F 0 "C37" H 10315 6096 50  0000 L CNN
+F 0 "C30" H 10315 6096 50  0000 L CNN
 F 1 "1u" H 10315 6005 50  0000 L CNN
-F 2 "Capacitor_SMD:C_0402_1005Metric" H 10238 5900 50  0001 C CNN
+F 2 "Capacitor_SMD:C_0603_1608Metric" H 10238 5900 50  0001 C CNN
 F 3 "~" H 10200 6050 50  0001 C CNN
+F 4 "0.0020" H 10200 6050 50  0001 C CNN "Price"
+F 5 "N" H 10200 6050 50  0001 C CNN "Sponsored"
 	1    10200 6050
 	-1   0    0    -1
 $EndComp
 $Comp
-L power:GND #PWR0156
+L power:GND #PWR0129
 U 1 1 612D4339
 P 10200 6200
-F 0 "#PWR0156" H 10200 5950 50  0001 C CNN
+F 0 "#PWR0129" H 10200 5950 50  0001 C CNN
 F 1 "GND" H 10205 6027 50  0000 C CNN
 F 2 "" H 10200 6200 50  0001 C CNN
@@
 PWR_LED
 $Comp
-L Device:C C38
+L Device:C C31
 U 1 1 612D45EF
 P 10550 6050
-F 0 "C38" H 10665 6096 50  0000 L CNN
+F 0 "C31" H 10665 6096 50  0000 L CNN
 F 1 "1u" H 10665 6005 50  0000 L CNN
-F 2 "Capacitor_SMD:C_0402_1005Metric" H 10588 5900 50  0001 C CNN
+F 2 "Capacitor_SMD:C_0603_1608Metric" H 10588 5900 50  0001 C CNN
 F 3 "~" H 10550 6050 50  0001 C CNN
+F 4 "0.0020" H 10550 6050 50  0001 C CNN "Price"
+F 5 "N" H 10550 6050 50  0001 C CNN "Sponsored"
 	1    10550 6050
 	-1   0    0    -1
 $EndComp
 $Comp
-L power:GND #PWR0157
+L power:GND #PWR0130
 U 1 1 612D45F5
 P 10550 6200
-F 0 "#PWR0157" H 10550 5950 50  0001 C CNN
+F 0 "#PWR0130" H 10550 5950 50  0001 C CNN
 F 1 "GND" H 10555 6027 50  0000 C CNN
 F 2 "" H 10550 6200 50  0001 C CNN
@@
 PWR_LED
 $Comp
-L Device:C C39
+L Device:C C32
 U 1 1 612DE7A2
 P 10900 6050
-F 0 "C39" H 11015 6096 50  0000 L CNN
+F 0 "C32" H 11015 6096 50  0000 L CNN
 F 1 "1u" H 11015 6005 50  0000 L CNN
-F 2 "Capacitor_SMD:C_0402_1005Metric" H 10938 5900 50  0001 C CNN
+F 2 "Capacitor_SMD:C_0603_1608Metric" H 10938 5900 50  0001 C CNN
 F 3 "~" H 10900 6050 50  0001 C CNN
+F 4 "0.0020" H 10900 6050 50  0001 C CNN "Price"
+F 5 "N" H 10900 6050 50  0001 C CNN "Sponsored"
 	1    10900 6050
 	-1   0    0    -1
 $EndComp
 $Comp
-L power:GND #PWR0158
+L power:GND #PWR0131
 U 1 1 612DE7A8
 P 10900 6200
-F 0 "#PWR0158" H 10900 5950 50  0001 C CNN
+F 0 "#PWR0131" H 10900 5950 50  0001 C CNN
 F 1 "GND" H 10905 6027 50  0000 C CNN
 F 2 "" H 10900 6200 50  0001 C CNN

Commit message: Dump.
Parts:
- renumbered C27 to C21, C28 to C22, C29 to C23, C30 to C24, C31 to C25, C32 to C26, D9 to D10, D4 to D5, D5 to D6, D6 to D7, D7 to D8, D8 to D9
Changed lines of the file:
@@
 $EndDescr
 $Comp
-L LED:WS2812B D4
+L LED:WS2812B D5
 U 1 1 5F7D8169
 P 4300 4050
-F 0 "D4" H 4100 4300 50  0000 L CNN
+F 0 "D5" H 4100 4300 50  0000 L CNN
 F 1 "WS2812B" V 4450 4300 50  0000 L CNN
 F 2 "LED_SMD:LED_WS2812B_PLCC4_5.0x5.0mm_P3.2mm" H 4350 3750 50  0001 L TNN
@@
 $EndComp
 $Comp
-L power:GND #PWR0120
+L power:GND #PWR096
 U 1 1 612C7A49
 P 4300 4350
-F 0 "#PWR0120" H 4300 4100 50  0001 C CNN
+F 0 "#PWR096" H 4300 4100 50  0001 C CNN
 F 1 "GND" H 4305 4177 50  0000 C CNN
 F 2 "" H 4300 4350 50  0001 C CNN
@@
 PWR_LED
 $Comp
-L LED:WS2812B D5
+L LED:WS2812B D6
 U 1 1 612CEAF2
 P 4900 4050
-F 0 "D5" H 4700 4300 50  0000 L CNN
+F 0 "D6" H 4700 4300 50  0000 L CNN
 F 1 "WS2812B" V 5050 4300 50  0000 L CNN
 F 2 "LED_SMD:LED_WS2812B_PLCC4_5.0x5.0mm_P3.2mm" H 4950 3750 50  0001 L TNN
@@
 $EndComp
 $Comp
-L power:GND #PWR0121
+L power:GND #PWR097
 U 1 1 612CEAF8
 P 4900 4350
-F 0 "#PWR0121" H 4900 4100 50  0001 C CNN
+F 0 "#PWR097" H 4900 4100 50  0001 C CNN
 F 1 "GND" H 4905 4177 50  0000 C CNN
 F 2 "" H 4900 4350 50  0001 C CNN
@@
 PWR_LED
 $Comp
-L LED:WS2812B D6
+L LED:WS2812B D7
 U 1 1 612CEE91
 P 5500 4050
-F 0 "D6" H 5300 4300 50  0000 L CNN
+F 0 "D7" H 5300 4300 50  0000 L CNN
 F 1 "WS2812B" V 5650 4300 50  0000 L CNN
 F 2 "LED_SMD:LED_WS2812B_PLCC4_5.0x5.0mm_P3.2mm" H 5550 3750 50  0001 L TNN
@@
 $EndComp
 $Comp
-L power:GND #PWR0122
+L power:GND #PWR098
 U 1 1 612CEE97
 P 5500 4350
-F 0 "#PWR0122" H 5500 4100 50  0001 C CNN
+F 0 "#PWR098" H 5500 4100 50  0001 C CNN
 F 1 "GND" H 5505 4177 50  0000 C CNN
 F 2 "" H 5500 4350 50  0001 C CNN
@@
 PWR_LED
 $Comp
-L LED:WS2812B D7
+L LED:WS2812B D8
 U 1 1 612CF6E4
 P 6100 4050
-F 0 "D7" H 5900 4300 50  0000 L CNN
+F 0 "D8" H 5900 4300 50  0000 L CNN
 F 1 "WS2812B" V 6250 4300 50  0000 L CNN
 F 2 "LED_SMD:LED_WS2812B_PLCC4_5.0x5.0mm_P3.2mm" H 6150 3750 50  0001 L TNN
@@
 $EndComp
 $Comp
-L power:GND #PWR0123
+L power:GND #PWR099
 U 1 1 612CF6EA
 P 6100 4350
-F 0 "#PWR0123" H 6100 4100 50  0001 C CNN
+F 0 "#PWR099" H 6100 4100 50  0001 C CNN
 F 1 "GND" H 6105 4177 50  0000 C CNN
 F 2 "" H 6100 4350 50  0001 C CNN
@@
 PWR_LED
 $Comp
-L LED:WS2812B D8
+L LED:WS2812B D9
 U 1 1 612CFE55
 P 6700 4050
-F 0 "D8" H 6500 4300 50  0000 L CNN
+F 0 "D9" H 6500 4300 50  0000 L CNN
 F 1 "WS2812B" V 6850 4300 50  0000 L CNN
 F 2 "LED_SMD:LED_WS2812B_PLCC4_5.0x5.0mm_P3.2mm" H 6750 3750 50  0001 L TNN
@@
 $EndComp
 $Comp
-L power:GND #PWR0124
+L power:GND #PWR0100
 U 1 1 612CFE5B
 P 6700 4350
-F 0 "#PWR0124" H 6700 4100 50  0001 C CNN
+F 0 "#PWR0100" H 6700 4100 50  0001 C CNN
 F 1 "GND" H 6705 4177 50  0000 C CNN
 F 2 "" H 6700 4350 50  0001 C CNN
@@
 PWR_LED
 $Comp
-L LED:WS2812B D9
+L LED:WS2812B D10
 U 1 1 612D0799
 P 7300 4050
-F 0 "D9" H 7100 4300 50  0000 L CNN
+F 0 "D10" H 7100 4300 50  0000 L CNN
 F 1 "WS2812B" V 7450 4300 50  0000 L CNN
 F 2 "LED_SMD:LED_WS2812B_PLCC4_5.0x5.0mm_P3.2mm" H 7350 3750 50  0001 L TNN
@@
 $EndComp
 $Comp
-L power:GND #PWR0125
+L power:GND #PWR0101
 U 1 1 612D079F
 P 7300 4350
-F 0 "#PWR0125" H 7300 4100 50  0001 C CNN
+F 0 "#PWR0101" H 7300 4100 50  0001 C CNN
 F 1 "GND" H 7305 4177 50  0000 C CNN
 F 2 "" H 7300 4350 50  0001 C CNN
@@
 PWR_LED
 $Comp
-L Device:C C27
+L Device:C C21
 U 1 1 612D0DFB
 P 9150 6050
-F 0 "C27" H 9265 6096 50  0000 L CNN
+F 0 "C21" H 9265 6096 50  0000 L CNN
 F 1 "1u" H 9265 6005 50  0000 L CNN
 F 2 "Capacitor_SMD:C_0603_1608Metric" H 9188 5900 50  0001 C CNN
@@
 $EndComp
 $Comp
-L power:GND #PWR0126
+L power:GND #PWR0102
 U 1 1 612D0F05
 P 9150 6200
-F 0 "#PWR0126" H 9150 5950 50  0001 C CNN
+F 0 "#PWR0102" H 9150 5950 50  0001 C CNN
 F 1 "GND" H 9155 6027 50  0000 C CNN
 F 2 "" H 9150 6200 50  0001 C CNN
@@
 PWR_LED
 $Comp
-L Device:C C28
+L Device:C C22
 U 1 1 612D2985
 P 9500 6050
-F 0 "C28" H 9615 6096 50  0000 L CNN
+F 0 "C22" H 9615 6096 50  0000 L CNN
 F 1 "1u" H 9615 6005 50  0000 L CNN
 F 2 "Capacitor_SMD:C_0603_1608Metric" H 9538 5900 50  0001 C CNN
@@
 $EndComp
 $Comp
-L power:GND #PWR0127
+L power:GND #PWR0103
 U 1 1 612D298B
 P 9500 6200
-F 0 "#PWR0127" H 9500 5950 50  0001 C CNN
+F 0 "#PWR0103" H 9500 5950 50  0001 C CNN
 F 1 "GND" H 9505 6027 50  0000 C CNN
 F 2 "" H 9500 6200 50  0001 C CNN
@@
 PWR_LED
 $Comp
-L Device:C C29
+L Device:C C23
 U 1 1 612D3CA5
 P 9850 6050
-F 0 "C29" H 9965 6096 50  0000 L CNN
+F 0 "C23" H 9965 6096 50  0000 L CNN
 F 1 "1u" H 9965 6005 50  0000 L CNN
 F 2 "Capacitor_SMD:C_0603_1608Metric" H 9888 5900 50  0001 C CNN
@@
 $EndComp
 $Comp
-L power:GND #PWR0128
+L power:GND #PWR0104
 U 1 1 612D3CAB
 P 9850 6200
-F 0 "#PWR0128" H 9850 5950 50  0001 C CNN
+F 0 "#PWR0104" H 9850 5950 50  0001 C CNN
 F 1 "GND" H 9855 6027 50  0000 C CNN
 F 2 "" H 9850 6200 50  0001 C CNN
@@
 PWR_LED
 $Comp
-L Device:C C30
+L Device:C C24
 U 1 1 612D4333
 P 10200 6050
-F 0 "C30" H 10315 6096 50  0000 L CNN
+F 0 "C24" H 10315 6096 50  0000 L CNN
 F 1 "1u" H 10315 6005 50  0000 L CNN
 F 2 "Capacitor_SMD:C_0603_1608Metric" H 10238 5900 50  0001 C CNN
@@
 $EndComp
 $Comp
-L power:GND #PWR0129
+L power:GND #PWR0105
 U 1 1 612D4339
 P 10200 6200
-F 0 "#PWR0129" H 10200 5950 50  0001 C CNN
+F 0 "#PWR0105" H 10200 5950 50  0001 C CNN
 F 1 "GND" H 10205 6027 50  0000 C CNN
 F 2 "" H 10200 6200 50  0001 C CNN
@@
 PWR_LED
 $Comp
-L Device:C C31
+L Device:C C25
 U 1 1 612D45EF
 P 10550 6050
-F 0 "C31" H 10665 6096 50  0000 L CNN
+F 0 "C25" H 10665 6096 50  0000 L CNN
 F 1 "1u" H 10665 6005 50  0000 L CNN
 F 2 "Capacitor_SMD:C_0603_1608Metric" H 10588 5900 50  0001 C CNN
@@
 $EndComp
 $Comp
-L power:GND #PWR0130
+L power:GND #PWR0106
 U 1 1 612D45F5
 P 10550 6200
-F 0 "#PWR0130" H 10550 5950 50  0001 C CNN
+F 0 "#PWR0106" H 10550 5950 50  0001 C CNN
 F 1 "GND" H 10555 6027 50  0000 C CNN
 F 2 "" H 10550 6200 50  0001 C CNN
@@
 PWR_LED
 $Comp
-L Device:C C32
+L Device:C C26
 U 1 1 612DE7A2
 P 10900 6050
-F 0 "C32" H 11015 6096 50  0000 L CNN
+F 0 "C26" H 11015 6096 50  0000 L CNN
 F 1 "1u" H 11015 6005 50  0000 L CNN
 F 2 "Capacitor_SMD:C_0603_1608Metric" H 10938 5900 50  0001 C CNN
@@
 $EndComp
 $Comp
-L power:GND #PWR0131
+L power:GND #PWR0107
 U 1 1 612DE7A8
 P 10900 6200
-F 0 "#PWR0131" H 10900 5950 50  0001 C CNN
+F 0 "#PWR0107" H 10900 5950 50  0001 C CNN
 F 1 "GND" H 10905 6027 50  0000 C CNN
 F 2 "" H 10900 6200 50  0001 C CNN
