File: led.sch (KiCad schematic (older format))
At the start: 12 parts

Commit message: Dump.
Parts:
- renumbered D5 to D4, D6 to D5, D7 to D6, D8 to D7, D9 to D8, D10 to D9
Changed lines of the file:
@@
 $EndDescr
 $Comp
-L LED:WS2812B D5
+L LED:WS2812B D4
 U 1 1 5F7D8169
 P 4300 4050
-F 0 "D5" H 4100 4300 50  0000 L CNN
+F 0 "D4" H 4100 4300 50  0000 L CNN
 F 1 "WS2812B" V 4450 4300 50  0000 L CNN
 F 2 "LED_SMD:LED_WS2812B_PLCC4_5.0x5.0mm_P3.2mm" H 4350 3750 50  0001 L TNN
@@
 $EndComp
 $Comp
-L power:GND #PWR096
+L power:GND #PWR095
 U 1 1 612C7A49
 P 4300 4350
-F 0 "#PWR096" H 4300 4100 50  0001 C CNN
+F 0 "#PWR095" H 4300 4100 50  0001 C CNN
 F 1 "GND" H 4305 4177 50  0000 C CNN
 F 2 "" H 4300 4350 50  0001 C CNN
@@
 PWR_LED
 $Comp
-L LED:WS2812B D6
+L LED:WS2812B D5
 U 1 1 612CEAF2
 P 4900 4050
-F 0 "D6" H 4700 4300 50  0000 L CNN
+F 0 "D5" H 4700 4300 50  0000 L CNN
 F 1 "WS2812B" V 5050 4300 50  0000 L CNN
 F 2 "LED_SMD:LED_WS2812B_PLCC4_5.0x5.0mm_P3.2mm" H 4950 3750 50  0001 L TNN
@@
 $EndComp
 $Comp
-L power:GND #PWR097
+L power:GND #PWR096
 U 1 1 612CEAF8
 P 4900 4350
-F 0 "#PWR097" H 4900 4100 50  0001 C CNN
+F 0 "#PWR096" H 4900 4100 50  0001 C CNN
 F 1 "GND" H 4905 4177 50  0000 C CNN
 F 2 "" H 4900 4350 50  0001 C CNN
@@
 PWR_LED
 $Comp
-L LED:WS2812B D7
+L LED:WS2812B D6
 U 1 1 612CEE91
 P 5500 4050
-F 0 "D7" H 5300 4300 50  0000 L CNN
+F 0 "D6" H 5300 4300 50  0000 L CNN
 F 1 "WS2812B" V 5650 4300 50  0000 L CNN
 F 2 "LED_SMD:LED_WS2812B_PLCC4_5.0x5.0mm_P3.2mm" H 5550 3750 50  0001 L TNN
@@
 $EndComp
 $Comp
-L power:GND #PWR098
+L power:GND #PWR097
 U 1 1 612CEE97
 P 5500 4350
-F 0 "#PWR098" H 5500 4100 50  0001 C CNN
+F 0 "#PWR097" H 5500 4100 50  0001 C CNN
 F 1 "GND" H 5505 4177 50  0000 C CNN
 F 2 "" H 5500 4350 50  0001 C CNN
@@
 PWR_LED
 $Comp
-L LED:WS2812B D8
+L LED:WS2812B D7
 U 1 1 612CF6E4
 P 6100 4050
-F 0 "D8" H 5900 4300 50  0000 L CNN
+F 0 "D7" H 5900 4300 50  0000 L CNN
 F 1 "WS2812B" V 6250 4300 50  0000 L CNN
 F 2 "LED_SMD:LED_WS2812B_PLCC4_5.0x5.0mm_P3.2mm" H 6150 3750 50  0001 L TNN
@@
 $EndComp
 $Comp
-L power:GND #PWR099
+L power:GND #PWR098
 U 1 1 612CF6EA
 P 6100 4350
-F 0 "#PWR099" H 6100 4100 50  0001 C CNN
+F 0 "#PWR098" H 6100 4100 50  0001 C CNN
 F 1 "GND" H 6105 4177 50  0000 C CNN
 F 2 "" H 6100 4350 50  0001 C CNN
@@
 PWR_LED
 $Comp
-L LED:WS2812B D9
+L LED:WS2812B D8
 U 1 1 612CFE55
 P 6700 4050
-F 0 "D9" H 6500 4300 50  0000 L CNN
+F 0 "D8" H 6500 4300 50  0000 L CNN
 F 1 "WS2812B" V 6850 4300 50  0000 L CNN
 F 2 "LED_SMD:LED_WS2812B_PLCC4_5.0x5.0mm_P3.2mm" H 6750 3750 50  0001 L TNN
@@
 $EndComp
 $Comp
-L power:GND #PWR0100
+L power:GND #PWR099
 U 1 1 612CFE5B
 P 6700 4350
-F 0 "#PWR0100" H 6700 4100 50  0001 C CNN
+F 0 "#PWR099" H 6700 4100 50  0001 C CNN
 F 1 "GND" H 6705 4177 50  0000 C CNN
 F 2 "" H 6700 4350 50  0001 C CNN
@@
 PWR_LED
 $Comp
-L LED:WS2812B D10
+L LED:WS2812B D9
 U 1 1 612D0799
 P 7300 4050
-F 0 "D10" H 7100 4300 50  0000 L CNN
+F 0 "D9" H 7100 4300 50  0000 L CNN
 F 1 "WS2812B" V 7450 4300 50  0000 L CNN
 F 2 "LED_SMD:LED_WS2812B_PLCC4_5.0x5.0mm_P3.2mm" H 7350 3750 50  0001 L TNN
@@
 $EndComp
 $Comp
-L power:GND #PWR0101
+L power:GND #PWR0100
 U 1 1 612D079F
 P 7300 4350
-F 0 "#PWR0101" H 7300 4100 50  0001 C CNN
+F 0 "#PWR0100" H 7300 4100 50  0001 C CNN
 F 1 "GND" H 7305 4177 50  0000 C CNN
 F 2 "" H 7300 4350 50  0001 C CNN
@@
 $EndComp
 $Comp
-L power:GND #PWR0102
+L power:GND #PWR0101
 U 1 1 612D0F05
 P 9150 6200
-F 0 "#PWR0102" H 9150 5950 50  0001 C CNN
+F 0 "#PWR0101" H 9150 5950 50  0001 C CNN
 F 1 "GND" H 9155 6027 50  0000 C CNN
 F 2 "" H 9150 6200 50  0001 C CNN
@@
 $EndComp
 $Comp
-L power:GND #PWR0103
+L power:GND #PWR0102
 U 1 1 612D298B
 P 9500 6200
-F 0 "#PWR0103" H 9500 5950 50  0001 C CNN
+F 0 "#PWR0102" H 9500 5950 50  0001 C CNN
 F 1 "GND" H 9505 6027 50  0000 C CNN
 F 2 "" H 9500 6200 50  0001 C CNN
@@
 $EndComp
 $Comp
-L power:GND #PWR0104
+L power:GND #PWR0103
 U 1 1 612D3CAB
 P 9850 6200
-F 0 "#PWR0104" H 9850 5950 50  0001 C CNN
+F 0 "#PWR0103" H 9850 5950 50  0001 C CNN
 F 1 "GND" H 9855 6027 50  0000 C CNN
 F 2 "" H 9850 6200 50  0001 C CNN
@@
 $EndComp
 $Comp
-L power:GND #PWR0105
+L power:GND #PWR0104
 U 1 1 612D4339
 P 10200 6200
-F 0 "#PWR0105" H 10200 5950 50  0001 C CNN
+F 0 "#PWR0104" H 10200 5950 50  0001 C CNN
 F 1 "GND" H 10205 6027 50  0000 C CNN
 F 2 "" H 10200 6200 50  0001 C CNN
@@
 $EndComp
 $Comp
-L power:GND #PWR0106
+L power:GND #PWR0105
 U 1 1 612D45F5
 P 10550 6200
-F 0 "#PWR0106" H 10550 5950 50  0001 C CNN
+F 0 "#PWR0105" H 10550 5950 50  0001 C CNN
 F 1 "GND" H 10555 6027 50  0000 C CNN
 F 2 "" H 10550 6200 50  0001 C CNN
@@
 $EndComp
 $Comp
-L power:GND #PWR0107
+L power:GND #PWR0106
 U 1 1 612DE7A8
 P 10900 6200
-F 0 "#PWR0107" H 10900 5950 50  0001 C CNN
+F 0 "#PWR0106" H 10900 5950 50  0001 C CNN
 F 1 "GND" H 10905 6027 50  0000 C CNN
 F 2 "" H 10900 6200 50  0001 C CNN

Commit message: Dump.
Parts:
- C21, C22, C23, C24, C25, C26: LCSC (none) -> C26413; Price 0.0020 -> (none)
- D4, D5, D6, D7, D8, D9: Price 0.037 -> (none)
Changed lines of the file:
@@
 F 4 "C139127" H 4300 4050 50  0001 C CNN "LCSC"
 F 5 "-" H 4300 4050 50  0001 C CNN "Mouser"
-F 6 "0.037" H 4300 4050 50  0001 C CNN "Price"
+F 6 "" H 4300 4050 50  0001 C CNN "Price"
 F 7 "N" H 4300 4050 50  0001 C CNN "Sponsored"
 	1    4300 4050
@@
 F 4 "C139127" H 4900 4050 50  0001 C CNN "LCSC"
 F 5 "-" H 4900 4050 50  0001 C CNN "Mouser"
-F 6 "0.037" H 4900 4050 50  0001 C CNN "Price"
+F 6 "" H 4900 4050 50  0001 C CNN "Price"
 F 7 "N" H 4900 4050 50  0001 C CNN "Sponsored"
 	1    4900 4050
@@
 F 4 "C139127" H 5500 4050 50  0001 C CNN "LCSC"
 F 5 "-" H 5500 4050 50  0001 C CNN "Mouser"
-F 6 "0.037" H 5500 4050 50  0001 C CNN "Price"
+F 6 "" H 5500 4050 50  0001 C CNN "Price"
 F 7 "N" H 5500 4050 50  0001 C CNN "Sponsored"
 	1    5500 4050
@@
 F 4 "C139127" H 6100 4050 50  0001 C CNN "LCSC"
 F 5 "-" H 6100 4050 50  0001 C CNN "Mouser"
-F 6 "0.037" H 6100 4050 50  0001 C CNN "Price"
+F 6 "" H 6100 4050 50  0001 C CNN "Price"
 F 7 "N" H 6100 4050 50  0001 C CNN "Sponsored"
 	1    6100 4050
@@
 F 4 "C139127" H 6700 4050 50  0001 C CNN "LCSC"
 F 5 "-" H 6700 4050 50  0001 C CNN "Mouser"
-F 6 "0.037" H 6700 4050 50  0001 C CNN "Price"
+F 6 "" H 6700 4050 50  0001 C CNN "Price"
 F 7 "N" H 6700 4050 50  0001 C CNN "Sponsored"
 	1    6700 4050
@@
 F 4 "C139127" H 7300 4050 50  0001 C CNN "LCSC"
 F 5 "-" H 7300 4050 50  0001 C CNN "Mouser"
-F 6 "0.037" H 7300 4050 50  0001 C CNN "Price"
+F 6 "" H 7300 4050 50  0001 C CNN "Price"
 F 7 "N" H 7300 4050 50  0001 C CNN "Sponsored"
 	1    7300 4050
@@
 F 2 "Capacitor_SMD:C_0603_1608Metric" H 9188 5900 50  0001 C CNN
 F 3 "~" H 9150 6050 50  0001 C CNN
-F 4 "0.0020" H 9150 6050 50  0001 C CNN "Price"
+F 4 "" H 9150 6050 50  0001 C CNN "Price"
 F 5 "N" H 9150 6050 50  0001 C CNN "Sponsored"
+F 6 "C26413" H 9150 6050 50  0001 C CNN "LCSC"
 	1    9150 6050
 	-1   0    0    -1
@@
 F 2 "Capacitor_SMD:C_0603_1608Metric" H 9538 5900 50  0001 C CNN
 F 3 "~" H 9500 6050 50  0001 C CNN
-F 4 "0.0020" H 9500 6050 50  0001 C CNN "Price"
+F 4 "" H 9500 6050 50  0001 C CNN "Price"
 F 5 "N" H 9500 6050 50  0001 C CNN "Sponsored"
+F 6 "C26413" H 9500 6050 50  0001 C CNN "LCSC"
 	1    9500 6050
 	-1   0    0    -1
@@
 F 2 "Capacitor_SMD:C_0603_1608Metric" H 9888 5900 50  0001 C CNN
 F 3 "~" H 9850 6050 50  0001 C CNN
-F 4 "0.0020" H 9850 6050 50  0001 C CNN "Price"
+F 4 "" H 9850 6050 50  0001 C CNN "Price"
 F 5 "N" H 9850 6050 50  0001 C CNN "Sponsored"
+F 6 "C26413" H 9850 6050 50  0001 C CNN "LCSC"
 	1    9850 6050
 	-1   0    0    -1
@@
 F 2 "Capacitor_SMD:C_0603_1608Metric" H 10238 5900 50  0001 C CNN
 F 3 "~" H 10200 6050 50  0001 C CNN
-F 4 "0.0020" H 10200 6050 50  0001 C CNN "Price"
+F 4 "" H 10200 6050 50  0001 C CNN "Price"
 F 5 "N" H 10200 6050 50  0001 C CNN "Sponsored"
+F 6 "C26413" H 10200 6050 50  0001 C CNN "LCSC"
 	1    10200 6050
 	-1   0    0    -1
@@
 F 2 "Capacitor_SMD:C_0603_1608Metric" H 10588 5900 50  0001 C CNN
 F 3 "~" H 10550 6050 50  0001 C CNN
-F 4 "0.0020" H 10550 6050 50  0001 C CNN "Price"
+F 4 "" H 10550 6050 50  0001 C CNN "Price"
 F 5 "N" H 10550 6050 50  0001 C CNN "Sponsored"
+F 6 "C26413" H 10550 6050 50  0001 C CNN "LCSC"
 	1    10550 6050
 	-1   0    0    -1
@@
 F 2 "Capacitor_SMD:C_0603_1608Metric" H 10938 5900 50  0001 C CNN
 F 3 "~" H 10900 6050 50  0001 C CNN
-F 4 "0.0020" H 10900 6050 50  0001 C CNN "Price"
+F 4 "" H 10900 6050 50  0001 C CNN "Price"
 F 5 "N" H 10900 6050 50  0001 C CNN "Sponsored"
+F 6 "C26413" H 10900 6050 50  0001 C CNN "LCSC"
 	1    10900 6050
 	-1   0    0    -1
