File: led.sch (KiCad schematic (older format))
At the start: 11 parts, among them U10 74LVC1G125

Commit message: Moar fixes
Parts:
- removed D8: SK6812-EC15, LED_SMD:LED_SK6812_EC15_1.5x1.5mm, symbol LED:WS2812B
- added C55, C56: 1u, Capacitor_SMD:C_0402_1005Metric, symbol Device:C
Connections:
- net DATA_IN1: now also R50.1, U10.2 (A); no longer R50.2
- net DATA_IN2: now also R50.2; no longer R50.1, U10.2 (A)
- net DATA_OUT: now also D7.2 (DOUT)
- net GND: now also C55.2, C56.2
- net PWR_LED: now also C55.1, C56.1
- net LED2_DATA: now reaches D3.2 (DOUT), D4.4 (DIN)
- net LED1_DATA: now reaches D3.4 (DIN), U10.4 (Y)
- net LED3_DATA: now reaches D4.2 (DOUT), D5.4 (DIN)
- net LED4_DATA: now reaches D5.2 (DOUT), D6.4 (DIN)
- net LED5_DATA: now reaches D6.2 (DOUT), D7.4 (DIN)
Other:
- moved on the sheet: C31, C32, C33, R50
Changed lines of the file:
@@
-PWR_LED
-$Comp
-L LED:WS2812B D8
-U 1 1 612D0799
-P 7300 4050
-F 0 "D8" H 7100 4300 50  0000 L CNN
-F 1 "SK6812-EC15" V 7450 4300 50  0000 L CNN
-F 2 "LED_SMD:LED_SK6812_EC15_1.5x1.5mm" H 7350 3750 50  0001 L TNN
-F 3 "http://www.normandled.com/Product/view/id/842.html" H 7400 3675 50  0001 L TNN
-F 4 "" H 7300 4050 50  0001 C CNN "LCSC"
-F 5 "-" H 7300 4050 50  0001 C CNN "Mouser"
-F 6 "" H 7300 4050 50  0001 C CNN "Price"
-F 7 "N" H 7300 4050 50  0001 C CNN "Sponsored"
-	1    7300 4050
-	1    0    0    -1
-$EndComp
-$Comp
-L power:GND #PWR0149
-U 1 1 612D079F
-P 7300 4350
-F 0 "#PWR0149" H 7300 4100 50  0001 C CNN
-F 1 "GND" H 7305 4177 50  0000 C CNN
-F 2 "" H 7300 4350 50  0001 C CNN
-F 3 "" H 7300 4350 50  0001 C CNN
-	1    7300 4350
-	1    0    0    -1
-$EndComp
-Text GLabel 7300 3750 1    39   Input ~ 0
 PWR_LED
 $Comp
 L Device:C C31
 U 1 1 612D0DFB
-P 10250 6100
-F 0 "C31" H 10365 6146 50  0000 L CNN
-F 1 "1u" H 10365 6055 50  0000 L CNN
-F 2 "Capacitor_SMD:C_0402_1005Metric" H 10288 5950 50  0001 C CNN
-F 3 "" H 10250 6100 50  0001 C CNN
-F 4 "" H 10250 6100 50  0001 C CNN "Price"
-F 5 "N" H 10250 6100 50  0001 C CNN "Sponsored"
-F 6 "C107372" H 10250 6100 50  0001 C CNN "LCSC"
-	1    10250 6100
+P 4300 5100
+F 0 "C31" H 4415 5146 50  0000 L CNN
+F 1 "1u" H 4415 5055 50  0000 L CNN
+F 2 "Capacitor_SMD:C_0402_1005Metric" H 4338 4950 50  0001 C CNN
+F 3 "" H 4300 5100 50  0001 C CNN
+F 4 "" H 4300 5100 50  0001 C CNN "Price"
+F 5 "N" H 4300 5100 50  0001 C CNN "Sponsored"
+F 6 "C107372" H 4300 5100 50  0001 C CNN "LCSC"
+	1    4300 5100
 	-1   0    0    -1
 $EndComp
@@
 L power:GND #PWR0150
 U 1 1 612D0F05
-P 10250 6250
-F 0 "#PWR0150" H 10250 6000 50  0001 C CNN
-F 1 "GND" H 10255 6077 50  0000 C CNN
-F 2 "" H 10250 6250 50  0001 C CNN
-F 3 "" H 10250 6250 50  0001 C CNN
-	1    10250 6250
-	1    0    0    -1
-$EndComp
-Text GLabel 10250 5950 1    39   Input ~ 0
+P 4300 5250
+F 0 "#PWR0150" H 4300 5000 50  0001 C CNN
+F 1 "GND" H 4305 5077 50  0000 C CNN
+F 2 "" H 4300 5250 50  0001 C CNN
+F 3 "" H 4300 5250 50  0001 C CNN
+	1    4300 5250
+	1    0    0    -1
+$EndComp
+Text GLabel 4300 4950 1    39   Input ~ 0
 PWR_LED
 $Comp
 L Device:C C32
 U 1 1 612D2985
-P 10600 6100
-F 0 "C32" H 10715 6146 50  0000 L CNN
-F 1 "1u" H 10715 6055 50  0000 L CNN
-F 2 "Capacitor_SMD:C_0402_1005Metric" H 10638 5950 50  0001 C CNN
-F 3 "" H 10600 6100 50  0001 C CNN
-F 4 "" H 10600 6100 50  0001 C CNN "Price"
-F 5 "N" H 10600 6100 50  0001 C CNN "Sponsored"
-F 6 "C107372" H 10600 6100 50  0001 C CNN "LCSC"
-	1    10600 6100
+P 4900 5100
+F 0 "C32" H 5015 5146 50  0000 L CNN
+F 1 "1u" H 5015 5055 50  0000 L CNN
+F 2 "Capacitor_SMD:C_0402_1005Metric" H 4938 4950 50  0001 C CNN
+F 3 "" H 4900 5100 50  0001 C CNN
+F 4 "" H 4900 5100 50  0001 C CNN "Price"
+F 5 "N" H 4900 5100 50  0001 C CNN "Sponsored"
+F 6 "C107372" H 4900 5100 50  0001 C CNN "LCSC"
+	1    4900 5100
 	-1   0    0    -1
 $EndComp
@@
 L power:GND #PWR0151
 U 1 1 612D298B
-P 10600 6250
-F 0 "#PWR0151" H 10600 6000 50  0001 C CNN
-F 1 "GND" H 10605 6077 50  0000 C CNN
-F 2 "" H 10600 6250 50  0001 C CNN
-F 3 "" H 10600 6250 50  0001 C CNN
-	1    10600 6250
-	1    0    0    -1
-$EndComp
-Text GLabel 10600 5950 1    39   Input ~ 0
+P 4900 5250
+F 0 "#PWR0151" H 4900 5000 50  0001 C CNN
+F 1 "GND" H 4905 5077 50  0000 C CNN
+F 2 "" H 4900 5250 50  0001 C CNN
+F 3 "" H 4900 5250 50  0001 C CNN
+	1    4900 5250
+	1    0    0    -1
+$EndComp
+Text GLabel 4900 4950 1    39   Input ~ 0
 PWR_LED
 $Comp
 L Device:C C33
 U 1 1 612D3CA5
-P 10950 6100
-F 0 "C33" H 11065 6146 50  0000 L CNN
-F 1 "1u" H 11065 6055 50  0000 L CNN
-F 2 "Capacitor_SMD:C_0402_1005Metric" H 10988 5950 50  0001 C CNN
-F 3 "" H 10950 6100 50  0001 C CNN
-F 4 "" H 10950 6100 50  0001 C CNN "Price"
-F 5 "N" H 10950 6100 50  0001 C CNN "Sponsored"
-F 6 "C107372" H 10950 6100 50  0001 C CNN "LCSC"
-	1    10950 6100
+P 5500 5100
+F 0 "C33" H 5615 5146 50  0000 L CNN
+F 1 "1u" H 5615 5055 50  0000 L CNN
+F 2 "Capacitor_SMD:C_0402_1005Metric" H 5538 4950 50  0001 C CNN
+F 3 "" H 5500 5100 50  0001 C CNN
+F 4 "" H 5500 5100 50  0001 C CNN "Price"
+F 5 "N" H 5500 5100 50  0001 C CNN "Sponsored"
+F 6 "C107372" H 5500 5100 50  0001 C CNN "LCSC"
+	1    5500 5100
 	-1   0    0    -1
 $EndComp
@@
 L power:GND #PWR0152
 U 1 1 612D3CAB
-P 10950 6250
-F 0 "#PWR0152" H 10950 6000 50  0001 C CNN
-F 1 "GND" H 10955 6077 50  0000 C CNN
-F 2 "" H 10950 6250 50  0001 C CNN
-F 3 "" H 10950 6250 50  0001 C CNN
-	1    10950 6250
-	1    0    0    -1
-$EndComp
-Text GLabel 10950 5950 1    39   Input ~ 0
+P 5500 5250
+F 0 "#PWR0152" H 5500 5000 50  0001 C CNN
+F 1 "GND" H 5505 5077 50  0000 C CNN
+F 2 "" H 5500 5250 50  0001 C CNN
+F 3 "" H 5500 5250 50  0001 C CNN
+	1    5500 5250
+	1    0    0    -1
+$EndComp
+Text GLabel 5500 4950 1    39   Input ~ 0
 PWR_LED
 Text Notes 1400 650  2    79   ~ 0
@@
 Text HLabel 2000 3950 0    79   Input ~ 0
 DATA_IN1
-Text HLabel 7600 4050 2    79   Output ~ 0
+Text HLabel 7000 4050 2    79   Output ~ 0
 DATA_OUT
 $Comp
@@
 L Device:R_Small R?
 U 1 1 6035A383
-P 2100 3950
+P 2100 4150
 AR Path="/6035A383" Ref="R?"  Part="1"
 AR Path="/612408B6/6035A383" Ref="R50"  Part="1"
-F 0 "R50" V 2000 3950 50  0000 C CNN
-F 1 "470" V 2200 3950 50  0000 C CNN
-F 2 "Resistor_SMD:R_0402_1005Metric" H 2100 3950 50  0001 C CNN
-F 3 "~" H 2100 3950 50  0001 C CNN
-F 4 "" H 2100 3950 50  0001 C CNN "Price"
-F 5 "" H 2100 3950 50  0001 C CNN "LCSC"
-F 6 "-" H 2100 3950 50  0001 C CNN "Mouser"
-F 7 "N" H 2100 3950 50  0001 C CNN "Sponsored"
-	1    2100 3950
+F 0 "R50" V 2000 4150 50  0000 C CNN
+F 1 "470" V 2200 4150 50  0000 C CNN
+F 2 "Resistor_SMD:R_0402_1005Metric" H 2100 4150 50  0001 C CNN
+F 3 "~" H 2100 4150 50  0001 C CNN
+F 4 "" H 2100 4150 50  0001 C CNN "Price"
+F 5 "" H 2100 4150 50  0001 C CNN "LCSC"
+F 6 "-" H 2100 4150 50  0001 C CNN "Mouser"
+F 7 "N" H 2100 4150 50  0001 C CNN "Sponsored"
+	1    2100 4150
 	0    1    1    0
 $EndComp
-Wire Wire Line
-	2200 3950 2250 3950
 Wire Wire Line
 	2250 3950 2250 4050
@@
 PWR_LED
 Wire Wire Line
-	2000 4150 2250 4150
-Wire Wire Line
 	2250 4150 2250 4050
 Connection ~ 2250 4050
+Wire Wire Line
+	2000 3950 2250 3950
+Wire Wire Line
+	2200 4150 2250 4150
+$Comp
+L Device:C C55
+U 1 1 60027D12
+P 6100 5100
+F 0 "C55" H 6215 5146 50  0000 L CNN
+F 1 "1u" H 6215 5055 50  0000 L CNN
+F 2 "Capacitor_SMD:C_0402_1005Metric" H 6138 4950 50  0001 C CNN
+F 3 "" H 6100 5100 50  0001 C CNN
+F 4 "" H 6100 5100 50  0001 C CNN "Price"
+F 5 "N" H 6100 5100 50  0001 C CNN "Sponsored"
+F 6 "C107372" H 6100 5100 50  0001 C CNN "LCSC"
+	1    6100 5100
+	-1   0    0    -1
+$EndComp
+$Comp
+L power:GND #PWR0149
+U 1 1 60027D18
+P 6100 5250
+F 0 "#PWR0149" H 6100 5000 50  0001 C CNN
+F 1 "GND" H 6105 5077 50  0000 C CNN
+F 2 "" H 6100 5250 50  0001 C CNN
+F 3 "" H 6100 5250 50  0001 C CNN
+	1    6100 5250
+	1    0    0    -1
+$EndComp
+Text GLabel 6100 4950 1    39   Input ~ 0
+PWR_LED
+$Comp
+L Device:C C56
+U 1 1 6002876A
+P 6700 5100
+F 0 "C56" H 6815 5146 50  0000 L CNN
+F 1 "1u" H 6815 5055 50  0000 L CNN
+F 2 "Capacitor_SMD:C_0402_1005Metric" H 6738 4950 50  0001 C CNN
+F 3 "" H 6700 5100 50  0001 C CNN
+F 4 "" H 6700 5100 50  0001 C CNN "Price"
+F 5 "N" H 6700 5100 50  0001 C CNN "Sponsored"
+F 6 "C107372" H 6700 5100 50  0001 C CNN "LCSC"
+	1    6700 5100
+	-1   0    0    -1
+$EndComp
+$Comp
+L power:GND #PWR0219
+U 1 1 60028770
+P 6700 5250
+F 0 "#PWR0219" H 6700 5000 50  0001 C CNN
+F 1 "GND" H 6705 5077 50  0000 C CNN
+F 2 "" H 6700 5250 50  0001 C CNN
+F 3 "" H 6700 5250 50  0001 C CNN
+	1    6700 5250
+	1    0    0    -1
+$EndComp
+Text GLabel 6700 4950 1    39   Input ~ 0
+PWR_LED
+Text Label 3550 4050 0    50   ~ 0
+LED1_DATA
+Text Label 4600 4050 3    20   ~ 0
+LED2_DATA
+Text Label 5200 4050 3    20   ~ 0
+LED3_DATA
+Text Label 5800 4050 3    20   ~ 0
+LED4_DATA
+Text Label 6400 4050 3    20   ~ 0
+LED5_DATA
 $EndSCHEMATC
