File: led.sch (KiCad schematic (older format))
At the start: 12 parts, among them U10 74LVC1G125

Commit message: Fix most of the bugs found on prototype 2 board
Parts:
- removed R50: 470, Resistor_SMD:R_0402_1005Metric, symbol Device:R_Small
- added TP2: LED_DATA_BUFF, TestPoint:TestPoint_Pad_1.0x1.0mm, symbol Connector:TestPoint
- added TP3: LED_DATA, TestPoint:TestPoint_Pad_1.0x1.0mm, symbol Connector:TestPoint
- D3, D4, D5, D6, D7: value SK6812-EC15 -> SK6805-EC15
Connections:
- net labels added: DATA_IN
- net labels removed: DATA_IN1, DATA_IN2
- wire segments 9 -> 7
Changed lines of the file:
@@
 Sheet 7 9
 Title ""
-Date "2021-01-14"
-Rev "2"
+Date "2021-10-09"
+Rev "3"
 Comp "BADGE.TEAM"
 Comment1 ""
@@
 P 4300 4050
 F 0 "D3" H 4100 4300 50  0000 L CNN
-F 1 "SK6812-EC15" V 4450 4300 50  0000 L CNN
+F 1 "SK6805-EC15" V 4450 4300 50  0000 L CNN
 F 2 "LED_SMD:LED_SK6812_EC15_1.5x1.5mm" H 4350 3750 50  0001 L TNN
 F 3 "http://www.normandled.com/Product/view/id/842.html" H 4400 3675 50  0001 L TNN
@@
 P 4900 4050
 F 0 "D4" H 4700 4300 50  0000 L CNN
-F 1 "SK6812-EC15" V 5050 4300 50  0000 L CNN
+F 1 "SK6805-EC15" V 5050 4300 50  0000 L CNN
 F 2 "LED_SMD:LED_SK6812_EC15_1.5x1.5mm" H 4950 3750 50  0001 L TNN
 F 3 "http://www.normandled.com/Product/view/id/842.html" H 5000 3675 50  0001 L TNN
@@
 P 5500 4050
 F 0 "D5" H 5300 4300 50  0000 L CNN
-F 1 "SK6812-EC15" V 5650 4300 50  0000 L CNN
+F 1 "SK6805-EC15" V 5650 4300 50  0000 L CNN
 F 2 "LED_SMD:LED_SK6812_EC15_1.5x1.5mm" H 5550 3750 50  0001 L TNN
 F 3 "http://www.normandled.com/Product/view/id/842.html" H 5600 3675 50  0001 L TNN
@@
 P 6100 4050
 F 0 "D6" H 5900 4300 50  0000 L CNN
-F 1 "SK6812-EC15" V 6250 4300 50  0000 L CNN
+F 1 "SK6805-EC15" V 6250 4300 50  0000 L CNN
 F 2 "LED_SMD:LED_SK6812_EC15_1.5x1.5mm" H 6150 3750 50  0001 L TNN
 F 3 "http://www.normandled.com/Product/view/id/842.html" H 6200 3675 50  0001 L TNN
@@
 P 6700 4050
 F 0 "D7" H 6500 4300 50  0000 L CNN
-F 1 "SK6812-EC15" V 6850 4300 50  0000 L CNN
+F 1 "SK6805-EC15" V 6850 4300 50  0000 L CNN
 F 2 "LED_SMD:LED_SK6812_EC15_1.5x1.5mm" H 6750 3750 50  0001 L TNN
 F 3 "http://www.normandled.com/Product/view/id/842.html" H 6800 3675 50  0001 L TNN
@@
 Text Notes 1400 650  2    79   ~ 0
 WS2812B LEDs
-Text HLabel 2000 3950 0    79   Input ~ 0
-DATA_IN1
 Text HLabel 7000 4050 2    79   Output ~ 0
 DATA_OUT
@@
 	3150 4250 3150 4350
 Wire Wire Line
-	3350 4050 4000 4050
-Wire Wire Line
-	2850 4050 2250 4050
-$Comp
-L Device:R_Small R?
-U 1 1 6035A383
-P 2100 4150
-AR Path="/6035A383" Ref="R?"  Part="1"
-AR Path="/612408B6/6035A383" Ref="R50"  Part="1"
-F 0 "R50" V 2000 4150 50  0000 C CNN
-F 1 "470" V 2200 4150 50  0000 C CNN
-F 2 "Resistor_SMD:R_0402_1005Metric" H 2100 4150 50  0001 C CNN
-F 3 "~" H 2100 4150 50  0001 C CNN
-F 4 "" H 2100 4150 50  0001 C CNN "Price"
-F 5 "" H 2100 4150 50  0001 C CNN "LCSC"
-F 6 "-" H 2100 4150 50  0001 C CNN "Mouser"
-F 7 "N" H 2100 4150 50  0001 C CNN "Sponsored"
-	1    2100 4150
-	0    1    1    0
-$EndComp
-Wire Wire Line
-	2250 3950 2250 4050
-Text HLabel 2000 4150 0    79   Input ~ 0
-DATA_IN2
+	3350 4050 3450 4050
+Wire Wire Line
+	2850 4050 2350 4050
+Text HLabel 2250 4050 0    79   Input ~ 0
+DATA_IN
 Text GLabel 3150 3650 1    39   Input ~ 0
 PWR_LED
-Wire Wire Line
-	2250 4150 2250 4050
-Connection ~ 2250 4050
-Wire Wire Line
-	2000 3950 2250 3950
-Wire Wire Line
-	2200 4150 2250 4150
 $Comp
 L Device:C C55
@@
 	-1   0    0    -1
 $EndComp
+$Comp
+L Connector:TestPoint TP2
+U 1 1 6165A2F6
+P 3450 4050
+F 0 "TP2" H 3400 4100 50  0000 R CNN
+F 1 "LED_DATA_BUFF" H 3400 4200 50  0000 R CNN
+F 2 "TestPoint:TestPoint_Pad_1.0x1.0mm" H 3650 4050 50  0001 C CNN
+F 3 "~" H 3650 4050 50  0001 C CNN
+	1    3450 4050
+	-1   0    0    1
+$EndComp
+Connection ~ 3450 4050
+Wire Wire Line
+	3450 4050 4000 4050
+$Comp
+L Connector:TestPoint TP3
+U 1 1 6168BD17
+P 2350 4050
+F 0 "TP3" H 2300 4100 50  0000 R CNN
+F 1 "LED_DATA" H 2300 4200 50  0000 R CNN
+F 2 "TestPoint:TestPoint_Pad_1.0x1.0mm" H 2550 4050 50  0001 C CNN
+F 3 "~" H 2550 4050 50  0001 C CNN
+	1    2350 4050
+	-1   0    0    1
+$EndComp
+Connection ~ 2350 4050
+Wire Wire Line
+	2350 4050 2250 4050
 $EndSCHEMATC

Commit message: Change pinout of expansion header close to board edge to be fully ground instead of gnd + 3.3v (& update component references)
Parts:
- C31, C32, C33, C55, C56: symbol Device:C -> mch2021-rescue:C-Device
- D3, D4, D5, D6, D7: symbol LED:WS2812B -> mch2021-rescue:WS2812B-LED
- TP2, TP3: symbol Connector:TestPoint -> mch2021-rescue:TestPoint-Connector
- U10: symbol dk_Logic-Buffers-Drivers-Receivers-Transceivers:SN74LVC1G125DCKR -> mch2021-rescue:SN74LVC1G125DCKR-dk_Logic-Buffers-Drivers-Receivers-Transceivers
Changed lines of the file:
@@
 $EndDescr
 $Comp
-L LED:WS2812B D3
+L mch2021-rescue:WS2812B-LED D3
 U 1 1 5F7D8169
 P 4300 4050
@@
 $EndComp
 $Comp
-L power:GND #PWR0144
+L mch2021-rescue:GND-power #PWR0144
 U 1 1 612C7A49
 P 4300 4350
@@
 PWR_LED
 $Comp
-L LED:WS2812B D4
+L mch2021-rescue:WS2812B-LED D4
 U 1 1 612CEAF2
 P 4900 4050
@@
 $EndComp
 $Comp
-L power:GND #PWR0145
+L mch2021-rescue:GND-power #PWR0145
 U 1 1 612CEAF8
 P 4900 4350
@@
 PWR_LED
 $Comp
-L LED:WS2812B D5
+L mch2021-rescue:WS2812B-LED D5
 U 1 1 612CEE91
 P 5500 4050
@@
 $EndComp
 $Comp
-L power:GND #PWR0146
+L mch2021-rescue:GND-power #PWR0146
 U 1 1 612CEE97
 P 5500 4350
@@
 PWR_LED
 $Comp
-L LED:WS2812B D6
+L mch2021-rescue:WS2812B-LED D6
 U 1 1 612CF6E4
 P 6100 4050
@@
 $EndComp
 $Comp
-L power:GND #PWR0147
+L mch2021-rescue:GND-power #PWR0147
 U 1 1 612CF6EA
 P 6100 4350
@@
 PWR_LED
 $Comp
-L LED:WS2812B D7
+L mch2021-rescue:WS2812B-LED D7
 U 1 1 612CFE55
 P 6700 4050
@@
 $EndComp
 $Comp
-L power:GND #PWR0148
+L mch2021-rescue:GND-power #PWR0148
 U 1 1 612CFE5B
 P 6700 4350
@@
 PWR_LED
 $Comp
-L Device:C C31
+L mch2021-rescue:C-Device C31
 U 1 1 612D0DFB
 P 4300 5100
@@
 $EndComp
 $Comp
-L power:GND #PWR0150
+L mch2021-rescue:GND-power #PWR0150
 U 1 1 612D0F05
 P 4300 5250
@@
 PWR_LED
 $Comp
-L Device:C C32
+L mch2021-rescue:C-Device C32
 U 1 1 612D2985
 P 4900 5100
@@
 $EndComp
 $Comp
-L power:GND #PWR0151
+L mch2021-rescue:GND-power #PWR0151
 U 1 1 612D298B
 P 4900 5250
@@
 PWR_LED
 $Comp
-L Device:C C33
+L mch2021-rescue:C-Device C33
 U 1 1 612D3CA5
 P 5500 5100
@@
 $EndComp
 $Comp
-L power:GND #PWR0152
+L mch2021-rescue:GND-power #PWR0152
 U 1 1 612D3CAB
 P 5500 5250
@@
 DATA_OUT
 $Comp
-L power:GND #PWR?
+L mch2021-rescue:GND-power #PWR?
 U 1 1 60345F64
 P 2800 4350
@@
 	2850 3850 2800 3850
 $Comp
-L dk_Logic-Buffers-Drivers-Receivers-Transceivers:SN74LVC1G125DCKR U?
+L mch2021-rescue:SN74LVC1G125DCKR-dk_Logic-Buffers-Drivers-Receivers-Transceivers U?
 U 1 1 60345F5C
 P 3150 3950
@@
 $EndComp
 $Comp
-L power:GND #PWR?
+L mch2021-rescue:GND-power #PWR?
 U 1 1 60345F44
 P 3150 4350
@@
 PWR_LED
 $Comp
-L Device:C C55
+L mch2021-rescue:C-Device C55
 U 1 1 60027D12
 P 6100 5100
@@
 $EndComp
 $Comp
-L power:GND #PWR0149
+L mch2021-rescue:GND-power #PWR0149
 U 1 1 60027D18
 P 6100 5250
@@
 PWR_LED
 $Comp
-L power:GND #PWR0219
+L mch2021-rescue:GND-power #PWR0219
 U 1 1 60028770
 P 6700 5250
@@
 $EndComp
 $Comp
-L Device:C C56
+L mch2021-rescue:C-Device C56
 U 1 1 6002876A
 P 6700 5100
@@
 $EndComp
 $Comp
-L Connector:TestPoint TP2
+L mch2021-rescue:TestPoint-Connector TP2
 U 1 1 6165A2F6
 P 3450 4050
@@
 	3450 4050 4000 4050
 $Comp
-L Connector:TestPoint TP3
+L mch2021-rescue:TestPoint-Connector TP3
 U 1 1 6168BD17
 P 2350 4050

Commit message: Fix SK6805-EC15 footprint and symbol
Parts:
- D3, D4, D5, D6, D7: footprint LED_SMD:LED_SK6812_EC15_1.5x1.5mm -> custom:LED_SK6805_EC15_1.5x1.5mm; symbol mch2021-rescue:WS2812B-LED -> custom:SK6805-EC15
Connections:
- net DATA_OUT: now also D7.3 (DOUT); no longer D7.2 (DOUT)
- net GND: now also D3.4 (GND), D4.4 (GND), D5.4 (GND), D6.4 (GND), D7.4 (GND); no longer D3.3 (VSS), D4.3 (VSS), D5.3 (VSS), D6.3 (VSS), D7.3 (VSS)
- net LED1_DATA: now also D3.1 (DIN); no longer D3.4 (DIN)
- net LED2_DATA: now also D3.3 (DOUT), D4.1 (DIN); no longer D3.2 (DOUT), D4.4 (DIN)
- net LED3_DATA: now also D4.3 (DOUT), D5.1 (DIN); no longer D4.2 (DOUT), D5.4 (DIN)
- net LED4_DATA: now also D5.3 (DOUT), D6.1 (DIN); no longer D5.2 (DOUT), D6.4 (DIN)
- net LED5_DATA: now also D6.3 (DOUT), D7.1 (DIN); no longer D6.2 (DOUT), D7.4 (DIN)
- net PWR_LED: now also D3.2 (VDD), D4.2 (VDD), D5.2 (VDD), D6.2 (VDD), D7.2 (VDD); no longer D3.1 (VDD), D4.1 (VDD), D5.1 (VDD), D6.1 (VDD), D7.1 (VDD)
Changed lines of the file:
@@
 $EndDescr
 $Comp
-L mch2021-rescue:WS2812B-LED D3
+L custom:SK6805-EC15 D3
 U 1 1 5F7D8169
 P 4300 4050
 F 0 "D3" H 4100 4300 50  0000 L CNN
 F 1 "SK6805-EC15" V 4450 4300 50  0000 L CNN
-F 2 "LED_SMD:LED_SK6812_EC15_1.5x1.5mm" H 4350 3750 50  0001 L TNN
+F 2 "custom:LED_SK6805_EC15_1.5x1.5mm" H 4350 3750 50  0001 L TNN
 F 3 "http://www.normandled.com/Product/view/id/842.html" H 4400 3675 50  0001 L TNN
 F 4 "" H 4300 4050 50  0001 C CNN "LCSC"
@@
 PWR_LED
 $Comp
-L mch2021-rescue:WS2812B-LED D4
+L custom:SK6805-EC15 D4
 U 1 1 612CEAF2
 P 4900 4050
 F 0 "D4" H 4700 4300 50  0000 L CNN
 F 1 "SK6805-EC15" V 5050 4300 50  0000 L CNN
-F 2 "LED_SMD:LED_SK6812_EC15_1.5x1.5mm" H 4950 3750 50  0001 L TNN
+F 2 "custom:LED_SK6805_EC15_1.5x1.5mm" H 4950 3750 50  0001 L TNN
 F 3 "http://www.normandled.com/Product/view/id/842.html" H 5000 3675 50  0001 L TNN
 F 4 "" H 4900 4050 50  0001 C CNN "LCSC"
@@
 PWR_LED
 $Comp
-L mch2021-rescue:WS2812B-LED D5
+L custom:SK6805-EC15 D5
 U 1 1 612CEE91
 P 5500 4050
 F 0 "D5" H 5300 4300 50  0000 L CNN
 F 1 "SK6805-EC15" V 5650 4300 50  0000 L CNN
-F 2 "LED_SMD:LED_SK6812_EC15_1.5x1.5mm" H 5550 3750 50  0001 L TNN
+F 2 "custom:LED_SK6805_EC15_1.5x1.5mm" H 5550 3750 50  0001 L TNN
 F 3 "http://www.normandled.com/Product/view/id/842.html" H 5600 3675 50  0001 L TNN
 F 4 "" H 5500 4050 50  0001 C CNN "LCSC"
@@
 PWR_LED
 $Comp
-L mch2021-rescue:WS2812B-LED D6
+L custom:SK6805-EC15 D6
 U 1 1 612CF6E4
 P 6100 4050
 F 0 "D6" H 5900 4300 50  0000 L CNN
 F 1 "SK6805-EC15" V 6250 4300 50  0000 L CNN
-F 2 "LED_SMD:LED_SK6812_EC15_1.5x1.5mm" H 6150 3750 50  0001 L TNN
+F 2 "custom:LED_SK6805_EC15_1.5x1.5mm" H 6150 3750 50  0001 L TNN
 F 3 "http://www.normandled.com/Product/view/id/842.html" H 6200 3675 50  0001 L TNN
 F 4 "" H 6100 4050 50  0001 C CNN "LCSC"
@@
 PWR_LED
 $Comp
-L mch2021-rescue:WS2812B-LED D7
+L custom:SK6805-EC15 D7
 U 1 1 612CFE55
 P 6700 4050
 F 0 "D7" H 6500 4300 50  0000 L CNN
 F 1 "SK6805-EC15" V 6850 4300 50  0000 L CNN
-F 2 "LED_SMD:LED_SK6812_EC15_1.5x1.5mm" H 6750 3750 50  0001 L TNN
+F 2 "custom:LED_SK6805_EC15_1.5x1.5mm" H 6750 3750 50  0001 L TNN
 F 3 "http://www.normandled.com/Product/view/id/842.html" H 6800 3675 50  0001 L TNN
 F 4 "" H 6700 4050 50  0001 C CNN "LCSC"

Commit message: Last fixes before ordering
Parts:
- U10: LCSC C7833 -> C703585; MPN SN74LVC1G125DCKR -> 74LVC1G125GW; Manufacturer Texas Instruments -> Nexperia
Changed lines of the file:
@@
 F 3 "http://www.ti.com/general/docs/suppproductinfo.tsp?distId=10&gotoUrl=http%3A%2F%2Fwww.ti.com%2Flit%2Fgpn%2Fsn74lvc1g125" H 3350 4250 60  0001 L CNN
 F 4 "296-11604-1-ND" H 3350 4350 60  0001 L CNN "Digi-Key_PN"
-F 5 "SN74LVC1G125DCKR" H 3350 4450 60  0001 L CNN "MPN"
+F 5 "74LVC1G125GW" H 3350 4450 60  0001 L CNN "MPN"
 F 6 "Integrated Circuits (ICs)" H 3350 4550 60  0001 L CNN "Category"
 F 7 "Logic - Buffers, Drivers, Receivers, Transceivers" H 3350 4650 60  0001 L CNN "Family"
@@
 F 9 "/product-detail/en/texas-instruments/SN74LVC1G125DCKR/296-11604-1-ND/385743" H 3350 4850 60  0001 L CNN "DK_Detail_Page"
 F 10 "IC BUF NON-INVERT 5.5V SC70-5" H 3350 4950 60  0001 L CNN "Description"
-F 11 "Texas Instruments" H 3350 5050 60  0001 L CNN "Manufacturer"
+F 11 "Nexperia" H 3350 5050 60  0001 L CNN "Manufacturer"
 F 12 "Active" H 3350 5150 60  0001 L CNN "Status"
 F 13 "N" H 3150 3950 50  0001 C CNN "Sponsored"
-F 14 "C7833" H 3150 3950 50  0001 C CNN "LCSC"
+F 14 "C703585" H 3150 3950 50  0001 C CNN "LCSC"
 F 15 "" H 3150 3950 50  0001 C CNN "Price"
 	1    3150 3950
