File: power.sch (KiCad schematic (older format))
At the start: 33 parts

Commit message: Finished work on initial schematic
Parts:
- added C13: 22u, Capacitor_SMD:C_0603_1608Metric, symbol Device:C
- gave numbers to parts that had none: 33
Connections:
- wire segments 92 -> 95

Commit message: Dump.
Parts:
- removed BT1: LiPo, corelib:S2B-ZR, symbol Device:Battery_Cell
- added BT1: LiPo, Connector_JST:JST_PH_S3B-PH-SM4-TB_1x03-1MP_P2.00mm_Horizontal, symbol Connector:Conn_01x03_Male
- C10: renamed from C7; Price (none) -> 0.0020; Sponsored (none) -> N
- C11: renamed from C8; Price (none) -> 0.0020; Sponsored (none) -> N
- C12: renamed from C9; Price (none) -> 0.0020; Sponsored (none) -> N
- C13: renamed from C10; Price (none) -> 0.0020; Sponsored (none) -> N
- C14: renamed from C11; Price (none) -> 0.0020; Sponsored (none) -> N
- C15: renamed from C12; value 0.1u -> 100n; LCSC (none) -> C14663; Mouser (none) -> -; Price (none) -> 0.0020; Sponsored (none) -> N
- C16: renamed from C13; Price (none) -> 0.0020; Sponsored (none) -> N
- C4: renamed from C1; Price (none) -> 0.0020; Sponsored (none) -> N
- C5: renamed from C2; Price (none) -> 0.0020; Sponsored (none) -> N
- C6: renamed from C3; Price (none) -> 0.0020; Sponsored (none) -> N
- C7: renamed from C4; footprint Capacitor_SMD:C_0402_1005Metric -> Capacitor_SMD:C_0603_1608Metric; LCSC (none) -> C14663; Mouser (none) -> -; Price (none) -> 0.0020; Sponsored (none) -> N
- C8: renamed from C5; Price (none) -> 0.0020; Sponsored (none) -> N
- C9: renamed from C6; Price (none) -> 0.0020; Sponsored (none) -> N
- D3: renamed from D2; footprint (none) -> Diode_SMD:D_0603_1608Metric; symbol schottky:SCHOTTKY -> Device:D_Schottky_Small; LCSC (none) -> -; Mouser (none) -> 750-CDBU0130R; Price (none) -> 0.053; Sponsored (none) -> N
- L1, L2: footprint corelib:Inductor_MSC20FC -> custom:Inductor_MSC20FC; LCSC (none) -> C375944; Mouser (none) -> -; Price (none) -> 0.026; Sponsored (none) -> N
- R10: renamed from R9; LCSC (none) -> -; Mouser (none) -> -; Price (none) -> 0.0005; Sponsored (none) -> N
- R11: renamed from R10; LCSC (none) -> -; Mouser (none) -> -; Price (none) -> 0.0005; Sponsored (none) -> N
- R12: renamed from R11; LCSC (none) -> -; Mouser (none) -> -; Price (none) -> 0.0005; Sponsored (none) -> N
- R13: renamed from R12; LCSC (none) -> -; Mouser (none) -> -; Price (none) -> 0.0005; Sponsored (none) -> N
- R14: renamed from R13; LCSC (none) -> C325685; Mouser (none) -> -; Price (none) -> 0.0016; Sponsored (none) -> N
- R5: renamed from R4; LCSC (none) -> -; Mouser (none) -> -; Price (none) -> 0.0005; Sponsored (none) -> N
- R6: renamed from R5; LCSC (none) -> -; Mouser (none) -> -; Price (none) -> 0.0005; Sponsored (none) -> N
- R7: renamed from R6; LCSC (none) -> -; Mouser (none) -> -; Price (none) -> 0.0005; Sponsored (none) -> N
- R8: renamed from R7; LCSC (none) -> -; Mouser (none) -> -; Price (none) -> 0.0005; Sponsored (none) -> N
- R9: renamed from R8; LCSC (none) -> -; Mouser (none) -> -; Price (none) -> 0.0005; Sponsored (none) -> N
- RN2: renamed from RN1; LCSC (none) -> C173315; Mouser (none) -> -; Price (none) -> 0.0042; Sponsored (none) -> N
- SW1: LCSC (none) -> C319020; Mouser (none) -> -; Price (none) -> 0.023; Sponsored (none) -> N
- U2: renamed from U1; value SY8079 -> SY8079AAC; LCSC (none) -> C133751; Mouser (none) -> -; Price (none) -> 0.067; Sponsored (none) -> N
- U3: renamed from U2; value SY8079 -> SY8079AAC; LCSC (none) -> C133751; Mouser (none) -> -; Price (none) -> 0.067; Sponsored (none) -> N
- U4: renamed from U3; LCSC (none) -> C141405; Mouser (none) -> -; Price (none) -> 0.028; Sponsored (none) -> N
- U5: renamed from U4; LCSC (none) -> C55136; Mouser (none) -> -; Price (none) -> 0.061; Sponsored (none) -> N
- U6: renamed from U5; LCSC (none) -> C55136; Mouser (none) -> -; Price (none) -> 0.061; Sponsored (none) -> N
Connections:
- net labels added: FB12, FB33, SW12, SW33
- wire segments 95 -> 98
- no-connect marks 0 -> 1

Commit message: Dump.
Parts:
- added D3: NSVR0320MW2T1G, Diode_SMD:D_SOD-323, symbol Device:D_Schottky
- added Q1: Q_PMOS_GSD, Package_TO_SOT_SMD:SOT-23, symbol Device:Q_PMOS_GSD
- added R8: 2k, Resistor_SMD:R_0603_1608Metric, symbol Device:R
- renumbered C11 to C10, C12 to C11, C13 to C12, C14 to C13, C15 to C14, C16 to C15, C4 to C3, C5 to C4, C6 to C5, C7 to C6, C8 to C7, C9 to C8, C10 to C9, D3 to D4, R9 to R10, R10 to R11, R11 to R12, R12 to R13, R13 to R14, R14 to R15, R8 to R9, U2 to U1, U3 to U2, U4 to U3, U5 to U4, U6 to U5
Connections:
- net GND: now also R8.2
- net VBAT: now also Q1.3 (D); no longer SW1.1 (A), U5.5 (IN)
- net VIN: now also U5.5 (IN)
- net VUSB: now also D3.2 (A), Q1.1 (G), R8.1
- new net: D3.1 (K), Q1.2 (S), SW1.1 (A)
Other:
- note added: "This "ideal diode" circuit\nprevents the user from\naccidently powering\nthe badge through\nthe battery charing circuit.\n\nWhen the power switch\nis set to battery mode\nand USB power is available\nthen the PMOSFET will\nbypass the battery and\ncharger and instead power\nthe badge using USB power"
- moved on the sheet: SW1

Commit message: Dump.
Parts:
- renumbered D3 to D2, D4 to D3, R11 to R10, R12 to R11, R13 to R12, R14 to R13, R15 to R14, R5 to R4, R6 to R5, R7 to R6, R8 to R7, R9 to R8, R10 to R9

Commit message: Dump.
Parts:
- added C45, C46: 100n, Capacitor_SMD:C_0603_1608Metric, symbol Device:C
- BT1: Price 0.12 -> (none)
- C10, C11, C12, C15, C4, C5, C9: footprint Capacitor_SMD:C_0603_1608Metric -> Capacitor_SMD:C_0805_2012Metric; LCSC (none) -> C5674; Price 0.0020 -> (none)
- C13, C3: LCSC (none) -> C307461; Price 0.0020 -> (none)
- C14, C6: Price 0.0020 -> (none)
- C7, C8: LCSC (none) -> C388041; Price 0.0020 -> (none)
- D2: LCSC (none) -> C232573; Sponsored (none) -> N
- D3: LCSC - -> C383224; Price 0.053 -> (none)
- L1, L2: Price 0.026 -> (none)
- Q1: LCSC (none) -> C180952; Sponsored (none) -> N
- R10, R4, R7: LCSC - -> C269690; Price 0.0005 -> (none)
- R11, R12, R13, R5, R6, R9: LCSC - -> C115324; Price 0.0005 -> (none)
- R14: Price 0.0016 -> (none)
- R8: LCSC - -> C23058; Price 0.0005 -> (none)
- RN2: Price 0.0042 -> (none)
- SW1: Price 0.023 -> (none)
- U1, U2: Price 0.067 -> (none)
- U3: Price 0.028 -> (none)
- U4, U5: Price 0.061 -> (none)
Connections:
- net GND: now also C45.2, C46.2
- net SENSE_VBAT: now also C46.1
- net SENSE_VUSB: now also C45.1
Other:
- moved on the sheet: RN2

Commit message: Work in progress: prototype 2
Parts:
- removed C14: 100n, Capacitor_SMD:C_0603_1608Metric, symbol Device:C
- removed D2: NSVR0320MW2T1G, Diode_SMD:D_SOD-323, symbol Device:D_Schottky
- removed D3: CDBU0130R, Diode_SMD:D_0603_1608Metric, symbol Device:D_Schottky_Small
- removed Q1: Q_PMOS_GSD, Package_TO_SOT_SMD:SOT-23, symbol Device:Q_PMOS_GSD
- removed R7: 2k, Resistor_SMD:R_0603_1608Metric, symbol Device:R
- added D?: NSVR0320MW2T1G, Diode_SMD:D_SOD-323, symbol Device:D_Schottky
- added Q?: Q_NMOS_GSD, Package_TO_SOT_SMD:SOT-23, symbol Device:Q_NMOS_GSD
- added R? (x4): 10k, Resistor_SMD:R_0603_1608Metric, symbol Device:R
- added R?: 100k, Resistor_SMD:R_0603_1608Metric, symbol Device:R
- added U?: SY6280AAC, Package_TO_SOT_SMD:SOT-23-5, symbol Power_Management:AAT4610BIGV-1-T1
Connections:
- net GND: now also Q?.2 (S), R?.1, R?.1, R?.2, U?.2 (GND)
- net VBAT: now also BT1.3 (Pin_3), SW1.2 (B), U?.5 (IN); no longer BT1.1 (Pin_1)
- net VIN: now also D?.1 (K), U?.1 (OUT); no longer SW1.2 (B)
- net VUSB: now also D?.2 (A), R?.1, R?.1; no longer SW1.3 (C)
- net at SW1.1 (A): now also R?.1
- new net: R?.2, U?.3 (SET)
- new net: Q?.3 (D), R?.2, R?.2, U?.4 (ON)
- new net: Q?.1 (G), R?.2
Other:
- note removed: "2.5v voltage regulator"
- note removed: "The power switch never really\nturns the badge off. Instead\nit lets you choose to bypass\nthe battery when powering\nthe badge from USB. This\nincreases charging speed and\nturns the badge off completely\nwhen USB is not connected"
- note removed: "This "ideal diode" circuit\nprevents the user from\naccidently powering\nthe badge through\nthe battery charing circuit.\n\nWhen the power switch\nis set to battery mode\nand USB power is available\nthen the PMOSFET will\nbypass the battery and\ncharger and instead power\nthe badge using USB power"
- moved on the sheet: SW1

Commit message: More work on prototype 2
Parts:
- added C1: 100n, Capacitor_SMD:C_0603_1608Metric, symbol Device:C
- added U15: AMS1117-3.3, Package_TO_SOT_SMD:SOT-223-3_TabPin2, symbol Regulator_Linear:AMS1117-3.3
- gave numbers to parts that had none: 8
Connections:
- net GND: now also C1.2, U15.1 (GND)
- net VBAT: now also U15.3 (VI)
- new net BAT_3.3: C1.1, U15.2 (VO)
Other:
- note added: "3.3v voltage regulator for RTC backup"
Changed lines of the file:
@@
 Sheet 2 9
 Title "MCH2021 badge - Power management"
-Date "2020-08-08"
-Rev "1"
+Date "2020-11-22"
+Rev "2"
 Comp "BADGE.TEAM"
 Comment1 ""
@@
 $EndComp
 $Comp
-L power:GND #PWR?
+L power:GND #PWR0119
 U 1 1 5FC2721B
 P 2950 4100
-F 0 "#PWR?" H 2950 3850 50  0001 C CNN
+F 0 "#PWR0119" H 2950 3850 50  0001 C CNN
 F 1 "GND" H 2955 3927 50  0000 C CNN
 F 2 "" H 2950 4100 50  0001 C CNN
@@
 $EndComp
 $Comp
-L power:GND #PWR?
+L power:GND #PWR0140
 U 1 1 5FC35B7C
 P 3400 4100
-F 0 "#PWR?" H 3400 3850 50  0001 C CNN
+F 0 "#PWR0140" H 3400 3850 50  0001 C CNN
 F 1 "GND" H 3405 3927 50  0000 C CNN
 F 2 "" H 3400 4100 50  0001 C CNN
@@
 $EndComp
 $Comp
-L Device:R R?
+L Device:R R58
 U 1 1 5FC35B86
 P 3400 3600
-F 0 "R?" H 3250 3550 50  0000 C CNN
+F 0 "R58" H 3250 3550 50  0000 C CNN
 F 1 "10k" H 3250 3650 50  0000 C CNN
 F 2 "Resistor_SMD:R_0603_1608Metric" V 3330 3600 50  0001 C CNN
@@
 	3400 3400 3350 3400
 $Comp
-L vin:VIN #PWR?
+L vin:VIN #PWR0172
 U 1 1 5FC4F90F
 P 3450 2700
-F 0 "#PWR?" H 3460 2700 20  0001 C CNN
+F 0 "#PWR0172" H 3460 2700 20  0001 C CNN
 F 1 "VIN" H 3450 2796 40  0000 C CNN
 F 2 "" H 3450 2700 60  0001 C CNN
@@
 	3350 3200 3450 3200
 $Comp
-L Device:D_Schottky D?
+L Device:D_Schottky D2
 U 1 1 5FC55914
 P 2950 2750
-F 0 "D?" H 2900 2850 50  0000 L CNN
+F 0 "D2" H 2900 2850 50  0000 L CNN
 F 1 "NSVR0320MW2T1G" H 2600 2650 50  0000 L CNN
 F 2 "Diode_SMD:D_SOD-323" H 2950 2750 50  0001 C CNN
@@
 Connection ~ 3450 2750
 $Comp
-L Device:R R?
+L Device:R R57
 U 1 1 5FD40AE5
 P 2450 3800
-F 0 "R?" H 2300 3750 50  0000 C CNN
+F 0 "R57" H 2300 3750 50  0000 C CNN
 F 1 "100k" H 2300 3850 50  0000 C CNN
 F 2 "Resistor_SMD:R_0603_1608Metric" V 2380 3800 50  0001 C CNN
@@
 	1700 3400 2000 3400
 $Comp
-L Device:R R?
+L Device:R R55
 U 1 1 5FC6C186
 P 1550 3400
-F 0 "R?" H 1400 3350 50  0000 C CNN
+F 0 "R55" H 1400 3350 50  0000 C CNN
 F 1 "10k" H 1400 3450 50  0000 C CNN
 F 2 "Resistor_SMD:R_0603_1608Metric" V 1480 3400 50  0001 C CNN
@@
 $EndComp
 $Comp
-L powersyms:VBAT #PWR?
+L powersyms:VBAT #PWR0183
 U 1 1 5FC464F4
 P 650 2700
-F 0 "#PWR?" H 660 2700 20  0001 C CNN
+F 0 "#PWR0183" H 660 2700 20  0001 C CNN
 F 1 "VBAT" H 650 2796 40  0000 C CNN
 F 2 "" H 650 2700 60  0001 C CNN
@@
 Connection ~ 1300 3800
 $Comp
-L Device:R R?
+L Device:R R54
 U 1 1 5FCE7654
 P 1300 3950
-F 0 "R?" H 1150 3900 50  0000 C CNN
+F 0 "R54" H 1150 3900 50  0000 C CNN
 F 1 "10k" H 1150 4000 50  0000 C CNN
 F 2 "Resistor_SMD:R_0603_1608Metric" V 1230 3950 50  0001 C CNN
@@
 	1300 2750 1300 2700
 $Comp
-L power:GND #PWR?
+L power:GND #PWR0184
 U 1 1 5FCC13F7
 P 1300 4100
-F 0 "#PWR?" H 1300 3850 50  0001 C CNN
+F 0 "#PWR0184" H 1300 3850 50  0001 C CNN
 F 1 "GND" H 1305 3927 50  0000 C CNN
 F 2 "" H 1300 4100 50  0001 C CNN
@@
 $EndComp
 $Comp
-L Device:R R?
+L Device:R R56
 U 1 1 5FCB5BEC
 P 1550 3800
-F 0 "R?" H 1400 3750 50  0000 C CNN
+F 0 "R56" H 1400 3750 50  0000 C CNN
 F 1 "10k" H 1400 3850 50  0000 C CNN
 F 2 "Resistor_SMD:R_0603_1608Metric" V 1480 3800 50  0001 C CNN
@@
 $EndComp
 $Comp
-L power:GND #PWR?
+L power:GND #PWR0185
 U 1 1 5FCA3FDA
 P 2000 4100
-F 0 "#PWR?" H 2000 3850 50  0001 C CNN
+F 0 "#PWR0185" H 2000 3850 50  0001 C CNN
 F 1 "GND" H 2005 3927 50  0000 C CNN
 F 2 "" H 2000 4100 50  0001 C CNN
@@
 P 1900 3800
 AR Path="/5FDC6C76/5FC8BD8A" Ref="Q?"  Part="1"
-AR Path="/60C789DE/5FC8BD8A" Ref="Q?"  Part="1"
-F 0 "Q?" V 2150 3800 50  0000 C CNN
+AR Path="/60C789DE/5FC8BD8A" Ref="Q1"  Part="1"
+F 0 "Q1" V 2150 3800 50  0000 C CNN
 F 1 "Q_NMOS_GSD" V 2250 3800 50  0000 C CNN
 F 2 "Package_TO_SOT_SMD:SOT-23" H 2100 3900 50  0001 C CNN
@@
 $EndComp
 $Comp
-L vusb:VUSB #PWR?
+L vusb:VUSB #PWR0186
 U 1 1 5FC5FBC2
 P 1300 2700
-F 0 "#PWR?" H 1310 2700 20  0001 C CNN
+F 0 "#PWR0186" H 1310 2700 20  0001 C CNN
 F 1 "VUSB" H 1300 2796 40  0000 C CNN
 F 2 "" H 1300 2700 60  0001 C CNN
@@
 $EndComp
 $Comp
-L Power_Management:AAT4610BIGV-1-T1 U?
+L Power_Management:AAT4610BIGV-1-T1 U14
 U 1 1 5FC24F91
 P 2950 3300
-F 0 "U?" H 2950 3650 50  0000 C CNN
+F 0 "U14" H 2950 3650 50  0000 C CNN
 F 1 "SY6280AAC" H 2950 3550 50  0000 C CNN
 F 2 "Package_TO_SOT_SMD:SOT-23-5" H 2950 3650 50  0001 C CNN
@@
 	2450 3400 2550 3400
 $Comp
-L power:GND #PWR?
+L power:GND #PWR0187
 U 1 1 5FD7F71E
 P 2450 4100
-F 0 "#PWR?" H 2450 3850 50  0001 C CNN
+F 0 "#PWR0187" H 2450 3850 50  0001 C CNN
 F 1 "GND" H 2455 3927 50  0000 C CNN
 F 2 "" H 2450 4100 50  0001 C CNN
@@
 Wire Wire Line
 	1400 3800 1300 3800
+Text Notes 6700 4600 2    98   ~ 0
+3.3v voltage regulator for RTC backup
+$Comp
+L powersyms:VBAT #PWR0188
+U 1 1 5FC609DB
+P 4700 4900
+F 0 "#PWR0188" H 4710 4900 20  0001 C CNN
+F 1 "VBAT" H 4700 4996 40  0000 C CNN
+F 2 "" H 4700 4900 60  0001 C CNN
+F 3 "" H 4700 4900 60  0001 C CNN
+	1    4700 4900
+	1    0    0    -1
+$EndComp
+$Comp
+L power:GND #PWR0189
+U 1 1 5FC62772
+P 5100 5850
+F 0 "#PWR0189" H 5100 5600 50  0001 C CNN
+F 1 "GND" H 5105 5677 50  0000 C CNN
+F 2 "" H 5100 5850 50  0001 C CNN
+F 3 "" H 5100 5850 50  0001 C CNN
+	1    5100 5850
+	1    0    0    -1
+$EndComp
+Text GLabel 5800 5000 2    50   Output ~ 0
+BAT_3.3
+$Comp
+L Regulator_Linear:AMS1117-3.3 U15
+U 1 1 5FBC430F
+P 5100 5000
+F 0 "U15" H 5100 5242 50  0000 C CNN
+F 1 "AMS1117-3.3" H 5100 5151 50  0000 C CNN
+F 2 "Package_TO_SOT_SMD:SOT-223-3_TabPin2" H 5100 5200 50  0001 C CNN
+F 3 "http://www.advanced-monolithic.com/pdf/ds1117.pdf" H 5200 4750 50  0001 C CNN
+	1    5100 5000
+	1    0    0    -1
+$EndComp
+Wire Wire Line
+	5100 5850 5100 5300
+Wire Wire Line
+	4800 5000 4700 5000
+Wire Wire Line
+	4700 5000 4700 4900
+Wire Wire Line
+	5800 5000 5600 5000
+$Comp
+L power:GND #PWR0190
+U 1 1 5FBF5265
+P 5600 5850
+F 0 "#PWR0190" H 5600 5600 50  0001 C CNN
+F 1 "GND" H 5605 5677 50  0000 C CNN
+F 2 "" H 5600 5850 50  0001 C CNN
+F 3 "" H 5600 5850 50  0001 C CNN
+	1    5600 5850
+	1    0    0    -1
+$EndComp
+$Comp
+L Device:C C1
+U 1 1 5FBF526F
+P 5600 5450
+F 0 "C1" H 5650 5650 50  0000 L CNN
+F 1 "100n" H 5650 5550 50  0000 L CNN
+F 2 "Capacitor_SMD:C_0603_1608Metric" H 5638 5300 50  0001 C CNN
+F 3 "~" H 5600 5450 50  0001 C CNN
+F 4 "C14663" H 5600 5450 50  0001 C CNN "LCSC"
+F 5 "" H 5600 5450 50  0001 C CNN "Price"
+F 6 "-" H 5600 5450 50  0001 C CNN "Mouser"
+F 7 "N" H 5600 5450 50  0001 C CNN "Sponsored"
+	1    5600 5450
+	1    0    0    -1
+$EndComp
+Wire Wire Line
+	5600 5300 5600 5000
+Connection ~ 5600 5000
+Wire Wire Line
+	5600 5000 5400 5000
+Wire Wire Line
+	5600 5600 5600 5850
 $EndSCHEMATC
