File: power.sch (KiCad schematic (older format))
At the start: 46 parts, among them Q1 Q_NMOS_GSD, SW1 Power switch, U1 SY8079AAC, U14 SY6280AAC, U2 SY8079AAC, U3 XT4054K421MR-G, U4 SY6280AAC, U5 SY6280AAC

Commit message: Updated schematic, add design file
Parts:
- added C25, C26: DNP, Capacitor_SMD:C_0603_1608Metric, symbol Device:C
- added R15, R17: 0, Resistor_SMD:R_0603_1608Metric, symbol Device:R
- D11: renamed from D?; footprint (none) -> Diode_SMD:D_SOD-323; LCSC (none) -> C123917
- R74: renamed from R?; footprint (none) -> Resistor_SMD:R_0603_1608Metric
- gave numbers to parts that had none: 1
Connections:
- net GND: now also C25.2, C26.2
- net VIN: now also R15.2, R17.2; no longer C4.1, C5.1, U1.1 (EN), U1.4 (VIN), U2.1 (EN), U2.4 (VIN)
- new net: C26.1, C5.1, R17.1, U2.1 (EN), U2.4 (VIN)
- new net: C25.1, C4.1, R15.1, U1.1 (EN), U1.4 (VIN)
Other:
- moved on the sheet: C10, C11, C12, C4, C5, C7, C8, C9, L1, L2, R5, R6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

Commit message: First steps of routing prototype 2, switch to 0402 for most passives
Parts:
- C1, C45, C46, C6: footprint Capacitor_SMD:C_0603_1608Metric -> Capacitor_SMD:C_0402_1005Metric; LCSC C14663 -> C83056
- C10, C11, C12, C15, C4, C5, C9: LCSC C5674 -> C159801
- C13, C3: footprint Capacitor_SMD:C_0603_1608Metric -> Capacitor_SMD:C_0402_1005Metric; LCSC C307461 -> C15525
- C25, C26: footprint Capacitor_SMD:C_0603_1608Metric -> Capacitor_SMD:C_0402_1005Metric
- C7, C8: footprint Capacitor_SMD:C_0603_1608Metric -> Capacitor_SMD:C_0402_1005Metric; LCSC C388041 -> C696906
- D3: LCSC (none) -> C402213
- R10, R4: footprint Resistor_SMD:R_0603_1608Metric -> Resistor_SMD:R_0402_1005Metric; LCSC C269690 -> C258126
- R11, R12, R13, R15, R17, R5, R55, R56, R57, R58, R6, R9: footprint Resistor_SMD:R_0603_1608Metric -> Resistor_SMD:R_0402_1005Metric; LCSC C115324 -> (none)
- R14: footprint Resistor_SMD:R_0603_1608Metric -> Resistor_SMD:R_0402_1005Metric; LCSC C325685 -> (none)
- R54: value 10k -> 100k; footprint Resistor_SMD:R_0603_1608Metric -> Resistor_SMD:R_0402_1005Metric; LCSC C115324 -> (none)
- R74: footprint Resistor_SMD:R_0603_1608Metric -> Resistor_SMD:R_0402_1005Metric
- R8: footprint Resistor_SMD:R_0603_1608Metric -> Resistor_SMD:R_0402_1005Metric; LCSC C23058 -> (none)

Commit message: More routing...
Connections:
- net 1V2REG_VIN: now reaches C26.1, C5.1, R17.1, U2.1 (EN), U2.4 (VIN)
Changed lines of the file:
@@
 	1150 6900 1500 6900
 Connection ~ 1150 6900
+Text Label 1200 6900 0    20   ~ 0
+1V2REG_VIN
 $EndSCHEMATC

Commit message: dump.
Connections:
- net 3V3REG_VIN: now reaches C25.1, C4.1, R15.1, U1.1 (EN), U1.4 (VIN)
Changed lines of the file:
@@
 Text Label 1200 6900 0    20   ~ 0
 1V2REG_VIN
+Text Label 1200 5150 0    20   ~ 0
+3V3REG_VIN
 $EndSCHEMATC

Commit message: Some more work
Parts:
- renumbered C3 to C34, C25 to C35, C26 to C36, C6 to C37, C4 to C38, C5 to C39, C7 to C40, C8 to C41, C13 to C42, C9 to C43, C10 to C44, C11 to C45, C12 to C46, C1 to C47, C45 to C48, C15 to C49, C46 to C50, D3 to D10, D2 to D9, L1 to L3, L2 to L4, Q1 to Q4, R15 to R51, R17 to R52, R54 to R53, R55 to R54, R56 to R55, R4 to R56, R5 to R57, R6 to R58, R57 to R59, R8 to R60, R9 to R61, R10 to R62, R58 to R63, R11 to R64, R12 to R65, R74 to R66, R13 to R67, R14 to R68, RN2 to RN6, SW1 to SW7, U1 to U11, U2 to U12, U3 to U13, U4 to U15, U5 to U16

Commit message: Add extra IO header, add battery NTC connection
Parts:
- added R76: 10k, Resistor_SMD:R_0402_1005Metric, symbol Device:R
Connections:
- net +3V3: now also R76.1
- net BATT_TEMP: now reaches BT1.1 (Pin_1)
- net BATT_TEMP: now also R76.2
- no-connect marks 1 -> 0
Changed lines of the file:
@@
 Wire Wire Line
 	3350 1650 3350 1800
-NoConn ~ 3400 1750
 Connection ~ 3000 1250
 Wire Wire Line
@@
 P 2050 1350
 F 0 "U13" H 1750 1600 50  0000 L CNN
-F 1 "XT4054K421MR-G" H 2100 1100 50  0000 L CNN
+F 1 "XT4054K421MR-G" H 1700 1850 50  0000 L CNN
 F 2 "Package_TO_SOT_SMD:SOT-23-5" H 2100 1100 50  0001 L CIN
 F 3 "" H 1900 1300 50  0001 C CNN
@@
 Text Label 1200 5150 0    20   ~ 0
 3V3REG_VIN
+Wire Wire Line
+	3400 1750 3200 1750
+Wire Wire Line
+	3200 1750 3200 2050
+Wire Wire Line
+	3200 2050 2700 2050
+$Comp
+L power:+3.3V #PWR0228
+U 1 1 601216C2
+P 2700 1750
+F 0 "#PWR0228" H 2700 1600 50  0001 C CNN
+F 1 "+3.3V" H 2700 1900 50  0000 C CNN
+F 2 "" H 2700 1750 50  0001 C CNN
+F 3 "" H 2700 1750 50  0001 C CNN
+	1    2700 1750
+	1    0    0    -1
+$EndComp
+$Comp
+L Device:R R76
+U 1 1 60121C9F
+P 2700 1900
+F 0 "R76" H 2770 1946 50  0000 L CNN
+F 1 "10k" H 2770 1855 50  0000 L CNN
+F 2 "Resistor_SMD:R_0402_1005Metric" V 2630 1900 50  0001 C CNN
+F 3 "~" H 2700 1900 50  0001 C CNN
+F 4 "" H 2700 1900 50  0001 C CNN "Price"
+F 5 "C258126 " H 2700 1900 50  0001 C CNN "LCSC"
+F 6 "-" H 2700 1900 50  0001 C CNN "Mouser"
+F 7 "N" H 2700 1900 50  0001 C CNN "Sponsored"
+	1    2700 1900
+	1    0    0    -1
+$EndComp
+Wire Wire Line
+	2700 2050 2600 2050
+Connection ~ 2700 2050
+Text HLabel 2600 2050 0    50   Output ~ 0
+BATT_TEMP
 $EndSCHEMATC
