File: power.sch (KiCad schematic (older format))
At the start: 51 parts, among them Q4 Q_NMOS_GSD, SW7 Power switch, U11 SY8079AAC, U12 SY8079AAC, U13 XT4054K421MR-G, U14 SY6280AAC, U15 SY6280AAC, U16 SY6280AAC

Commit message: Change pinout of expansion header close to board edge to be fully ground instead of gnd + 3.3v (& update component references)
Parts:
- BT1: symbol Connector:Conn_01x03_Male -> mch2021-rescue:Conn_01x03_Male-Connector
- C34, C35, C36, C37, C38, C39, C40, C41, C42, C43, C44, C45, C46, C47, C48, C49, C50: symbol Device:C -> mch2021-rescue:C-Device
- D10: symbol Diode:1N4148W -> mch2021-rescue:1N4148W-Diode
- D11: symbol Device:D_Zener -> mch2021-rescue:D_Zener-Device
- D9: symbol Device:D_Schottky -> mch2021-rescue:D_Schottky-Device
- L3, L4: symbol Device:L -> mch2021-rescue:L-Device
- Q4: symbol Device:Q_NMOS_GSD -> mch2021-rescue:Q_NMOS_GSD-Device
- R51, R52, R53, R54, R55, R56, R57, R58, R59, R60, R61, R62, R63, R64, R65, R67, R68, R76: symbol Device:R -> mch2021-rescue:R-Device
- R66: symbol Device:R_Small -> mch2021-rescue:R_Small-Device
- RN6: symbol Device:R_Pack04 -> mch2021-rescue:R_Pack04-Device
- SW7: symbol Switch:SW_SPDT -> mch2021-rescue:SW_SPDT-Switch
- U11, U12: symbol Regulator_Switching:TLV62568DBV -> mch2021-rescue:TLV62568DBV-Regulator_Switching
- U13: symbol Battery_Management:MCP73831-2-OT -> mch2021-rescue:MCP73831-2-OT-Battery_Management
- U14, U15, U16: symbol Power_Management:AAT4610BIGV-1-T1 -> mch2021-rescue:AAT4610BIGV-1-T1-Power_Management

Commit message: More work on RP2040 integration
Parts:
- removed C47: 100n, Capacitor_SMD:C_0402_1005Metric, symbol mch2021-rescue:C-Device
- removed D10: 1N4148W, Diode_SMD:D_SOD-123, symbol mch2021-rescue:1N4148W-Diode
- removed D11: 3V3, Diode_SMD:D_SOD-323, symbol mch2021-rescue:D_Zener-Device
- removed R66: 100k, Resistor_SMD:R_0402_1005Metric, symbol mch2021-rescue:R_Small-Device
Other:
- note removed: "3.3v voltage regulator for RTC backup"
Changed lines of the file:
@@
 Wire Wire Line
 	1400 3800 1300 3800
-Text Notes 6700 4600 2    98   ~ 0
-3.3v voltage regulator for RTC backup
-$Comp
-L mch2021-rescue:VBAT-powersyms #PWR0192
-U 1 1 5FC609DB
-P 4400 4900
-F 0 "#PWR0192" H 4410 4900 20  0001 C CNN
-F 1 "VBAT" H 4400 4996 40  0000 C CNN
-F 2 "" H 4400 4900 60  0001 C CNN
-F 3 "" H 4400 4900 60  0001 C CNN
-	1    4400 4900
-	1    0    0    -1
-$EndComp
-$Comp
-L mch2021-rescue:GND-power #PWR0200
-U 1 1 5FC62772
-P 5200 5850
-F 0 "#PWR0200" H 5200 5600 50  0001 C CNN
-F 1 "GND" H 5205 5677 50  0000 C CNN
-F 2 "" H 5200 5850 50  0001 C CNN
-F 3 "" H 5200 5850 50  0001 C CNN
-	1    5200 5850
-	1    0    0    -1
-$EndComp
-Text GLabel 5800 5000 2    50   Output ~ 0
-BAT_3.3
-Wire Wire Line
-	5200 5850 5200 5600
-Wire Wire Line
-	4500 5000 4400 5000
-Wire Wire Line
-	4400 5000 4400 4900
-Wire Wire Line
-	5800 5000 5600 5000
-$Comp
-L mch2021-rescue:GND-power #PWR0203
-U 1 1 5FBF5265
-P 5600 5850
-F 0 "#PWR0203" H 5600 5600 50  0001 C CNN
-F 1 "GND" H 5605 5677 50  0000 C CNN
-F 2 "" H 5600 5850 50  0001 C CNN
-F 3 "" H 5600 5850 50  0001 C CNN
-	1    5600 5850
-	1    0    0    -1
-$EndComp
-$Comp
-L mch2021-rescue:C-Device C47
-U 1 1 5FBF526F
-P 5600 5450
-F 0 "C47" H 5650 5650 50  0000 L CNN
-F 1 "100n" H 5650 5550 50  0000 L CNN
-F 2 "Capacitor_SMD:C_0402_1005Metric" H 5638 5300 50  0001 C CNN
-F 3 "" H 5600 5450 50  0001 C CNN
-F 4 "C83056 " H 5600 5450 50  0001 C CNN "LCSC"
-F 5 "" H 5600 5450 50  0001 C CNN "Price"
-F 6 "-" H 5600 5450 50  0001 C CNN "Mouser"
-F 7 "N" H 5600 5450 50  0001 C CNN "Sponsored"
-	1    5600 5450
-	1    0    0    -1
-$EndComp
-Wire Wire Line
-	5600 5300 5600 5000
-Connection ~ 5600 5000
-Wire Wire Line
-	5600 5600 5600 5850
-$Comp
-L mch2021-rescue:1N4148W-Diode D10
-U 1 1 5FD89C96
-P 4650 5000
-F 0 "D10" H 4650 4783 50  0000 C CNN
-F 1 "1N4148W" H 4650 4874 50  0000 C CNN
-F 2 "Diode_SMD:D_SOD-123" H 4650 4825 50  0001 C CNN
-F 3 "" H 4650 5000 50  0001 C CNN
-F 4 "C402213 " H 4650 5000 50  0001 C CNN "LCSC"
-	1    4650 5000
-	-1   0    0    1
-$EndComp
-$Comp
-L mch2021-rescue:R_Small-Device R66
-U 1 1 5FD8ABC7
-P 5000 5000
-F 0 "R66" V 4804 5000 50  0000 C CNN
-F 1 "100k" V 4895 5000 50  0000 C CNN
-F 2 "Resistor_SMD:R_0402_1005Metric" H 5000 5000 50  0001 C CNN
-F 3 "~" H 5000 5000 50  0001 C CNN
-	1    5000 5000
-	0    1    1    0
-$EndComp
-Wire Wire Line
-	4800 5000 4900 5000
-$Comp
-L mch2021-rescue:D_Zener-Device D11
-U 1 1 5FD972D4
-P 5200 5450
-F 0 "D11" V 5154 5530 50  0000 L CNN
-F 1 "3V3" V 5245 5530 50  0000 L CNN
-F 2 "Diode_SMD:D_SOD-323" H 5200 5450 50  0001 C CNN
-F 3 "https://datasheet.lcsc.com/szlcsc/1808062134_Shandong-Jingdao-Microelectronics-MM3Z3V3_C123917.pdf" H 5200 5450 50  0001 C CNN
-F 4 "C123917" V 5200 5450 50  0001 C CNN "LCSC"
-	1    5200 5450
-	0    1    1    0
-$EndComp
-Wire Wire Line
-	5100 5000 5200 5000
-Wire Wire Line
-	5200 5000 5200 5300
-Wire Wire Line
-	5200 5000 5600 5000
-Connection ~ 5200 5000
 $Comp
 L mch2021-rescue:C-Device C35

Commit message: Last fixes before ordering
Parts:
- C40, C41: LCSC C696906 -> C106203; MANUFACTURER (none) -> YAGEO; MPN (none) -> CC0402JRNPO9BN220
- D9: value NSVR0320MW2T1G -> PSBD3D40V1H; LCSC C232573 -> C110733
- Q4: MANUFACTURER (none) -> ALLPOWER; MPN (none) -> AP2302B
- R51, R52: LCSC (none) -> C60485; MANUFACTURER (none) -> YAGEO; MPN (none) -> RC0402JR-070RL
- R53, R59: LCSC (none) -> C258090; MANUFACTURER (none) -> FH; MPN (none) -> RC-02W1003FT
- R54, R55, R57, R58, R61, R63, R64, R65, R67: LCSC (none) -> C144807; MANUFACTURER (none) -> YAGEO; MPN (none) -> AC0402FR-0710KL
- R56, R62: LCSC C258126 -> C4109; MANUFACTURER (none) -> UNI-ROYAL; MPN (none) -> 0402WGF2001TCE
- R60: LCSC (none) -> C26980; MANUFACTURER (none) -> UNI-ROYAL; MPN (none) -> 0402WGF4532TCE
- R68: LCSC (none) -> C4940; MANUFACTURER (none) -> UNI-ROYAL; MPN (none) -> 0402WGF3401TCE
- R76: LCSC C258126 -> C144807; MANUFACTURER (none) -> YAGEO; MPN (none) -> AC0402FR-0710KL
- RN6: MANUFACTURER (none) -> UNI-ROYAL; MPN (none) -> 4D03WGF1003T5E
Changed lines of the file:
@@
 F 3 "~" H 1600 1650 50  0001 C CNN
 F 4 "" H 1600 1650 50  0001 C CNN "Price"
-F 5 "C258126 " H 1600 1650 50  0001 C CNN "LCSC"
+F 5 "C4109" H 1600 1650 50  0001 C CNN "LCSC"
 F 6 "-" H 1600 1650 50  0001 C CNN "Mouser"
 F 7 "N" H 1600 1650 50  0001 C CNN "Sponsored"
+F 8 "UNI-ROYAL" H 1600 1650 50  0001 C CNN "MANUFACTURER"
+F 9 "0402WGF2001TCE" H 1600 1650 50  0001 C CNN "MPN"
 	1    1600 1650
 	1    0    0    -1
@@
 F 6 "" H 5350 7050 50  0001 C CNN "Price"
 F 7 "N" H 5350 7050 50  0001 C CNN "Sponsored"
+F 8 "UNI-ROYAL" H 5350 7050 50  0001 C CNN "MANUFACTURER"
+F 9 "4D03WGF1003T5E" H 5350 7050 50  0001 C CNN "MPN"
 	1    5350 7050
 	0    1    1    0
@@
 F 3 "~" H 5800 3550 50  0001 C CNN
 F 4 "" H 5800 3550 50  0001 C CNN "Price"
-F 5 "" H 5800 3550 50  0001 C CNN "LCSC"
+F 5 "C4940" H 5800 3550 50  0001 C CNN "LCSC"
 F 6 "-" H 5800 3550 50  0001 C CNN "Mouser"
 F 7 "N" H 5800 3550 50  0001 C CNN "Sponsored"
+F 8 "UNI-ROYAL" H 5800 3550 50  0001 C CNN "MANUFACTURER"
+F 9 "0402WGF3401TCE" H 5800 3550 50  0001 C CNN "MPN"
 	1    5800 3550
 	1    0    0    -1
@@
 F 3 "~" H 4900 3550 50  0001 C CNN
 F 4 "" H 4900 3550 50  0001 C CNN "Price"
-F 5 "" H 4900 3550 50  0001 C CNN "LCSC"
+F 5 "C144807" H 4900 3550 50  0001 C CNN "LCSC"
 F 6 "-" H 4900 3550 50  0001 C CNN "Mouser"
 F 7 "N" H 4900 3550 50  0001 C CNN "Sponsored"
+F 8 "YAGEO" H 4900 3550 50  0001 C CNN "MANUFACTURER"
+F 9 "AC0402FR-0710KL" H 4900 3550 50  0001 C CNN "MPN"
 	1    4900 3550
 	-1   0    0    1
@@
 F 1 "22p" V 2450 5350 50  0000 C CNN
 F 2 "Capacitor_SMD:C_0402_1005Metric" H 2538 5300 50  0001 C CNN
-F 3 "" H 2500 5450 50  0001 C CNN
+F 3 "https://datasheet.lcsc.com/lcsc/1809301912_YAGEO-CC0402JRNPO9BN220_C106203.pdf" H 2500 5450 50  0001 C CNN
 F 4 "" H 2500 5450 50  0001 C CNN "Price"
 F 5 "N" H 2500 5450 50  0001 C CNN "Sponsored"
-F 6 "C696906" H 2500 5450 50  0001 C CNN "LCSC"
+F 6 "C106203" H 2500 5450 50  0001 C CNN "LCSC"
+F 7 "YAGEO" H 2500 5450 50  0001 C CNN "MANUFACTURER"
+F 8 "CC0402JRNPO9BN220" H 2500 5450 50  0001 C CNN "MPN"
 	1    2500 5450
 	0    1    1    0
@@
 F 3 "~" H 2500 5250 50  0001 C CNN
 F 4 "" H 2500 5250 50  0001 C CNN "Price"
-F 5 "" H 2500 5250 50  0001 C CNN "LCSC"
+F 5 "C26980" H 2500 5250 50  0001 C CNN "LCSC"
 F 6 "-" H 2500 5250 50  0001 C CNN "Mouser"
 F 7 "N" H 2500 5250 50  0001 C CNN "Sponsored"
+F 8 "UNI-ROYAL" H 2500 5250 50  0001 C CNN "MANUFACTURER"
+F 9 "0402WGF4532TCE" H 2500 5250 50  0001 C CNN "MPN"
 	1    2500 5250
 	0    1    1    0
@@
 F 3 "~" H 2300 5650 50  0001 C CNN
 F 4 "" H 2300 5650 50  0001 C CNN "Price"
-F 5 "" H 2300 5650 50  0001 C CNN "LCSC"
+F 5 "C144807" H 2300 5650 50  0001 C CNN "LCSC"
 F 6 "-" H 2300 5650 50  0001 C CNN "Mouser"
 F 7 "N" H 2300 5650 50  0001 C CNN "Sponsored"
+F 8 "YAGEO" H 2300 5650 50  0001 C CNN "MANUFACTURER"
+F 9 "AC0402FR-0710KL" H 2300 5650 50  0001 C CNN "MPN"
 	1    2300 5650
 	1    0    0    -1
@@
 F 3 "~" H 4900 1750 50  0001 C CNN
 F 4 "" H 4900 1750 50  0001 C CNN "Price"
-F 5 "" H 4900 1750 50  0001 C CNN "LCSC"
+F 5 "C144807" H 4900 1750 50  0001 C CNN "LCSC"
 F 6 "-" H 4900 1750 50  0001 C CNN "Mouser"
 F 7 "N" H 4900 1750 50  0001 C CNN "Sponsored"
+F 8 "YAGEO" H 4900 1750 50  0001 C CNN "MANUFACTURER"
+F 9 "AC0402FR-0710KL" H 4900 1750 50  0001 C CNN "MPN"
 	1    4900 1750
 	-1   0    0    1
@@
 F 3 "~" H 5800 1750 50  0001 C CNN
 F 4 "" H 5800 1750 50  0001 C CNN "Price"
-F 5 "" H 5800 1750 50  0001 C CNN "LCSC"
+F 5 "C144807" H 5800 1750 50  0001 C CNN "LCSC"
 F 6 "-" H 5800 1750 50  0001 C CNN "Mouser"
 F 7 "N" H 5800 1750 50  0001 C CNN "Sponsored"
+F 8 "YAGEO" H 5800 1750 50  0001 C CNN "MANUFACTURER"
+F 9 "AC0402FR-0710KL" H 5800 1750 50  0001 C CNN "MPN"
 	1    5800 1750
 	-1   0    0    1
@@
 F 1 "22p" V 2450 7100 50  0000 C CNN
 F 2 "Capacitor_SMD:C_0402_1005Metric" H 2538 7050 50  0001 C CNN
-F 3 "" H 2500 7200 50  0001 C CNN
+F 3 "https://datasheet.lcsc.com/lcsc/1809301912_YAGEO-CC0402JRNPO9BN220_C106203.pdf" H 2500 7200 50  0001 C CNN
 F 4 "" H 2500 7200 50  0001 C CNN "Price"
 F 5 "N" H 2500 7200 50  0001 C CNN "Sponsored"
-F 6 "C696906" H 2500 7200 50  0001 C CNN "LCSC"
+F 6 "C106203" H 2500 7200 50  0001 C CNN "LCSC"
+F 7 "YAGEO" H 2500 7200 50  0001 C CNN "MANUFACTURER"
+F 8 "CC0402JRNPO9BN220" H 2500 7200 50  0001 C CNN "MPN"
 	1    2500 7200
 	0    1    1    0
@@
 F 3 "~" H 2500 7000 50  0001 C CNN
 F 4 "" H 2500 7000 50  0001 C CNN "Price"
-F 5 "" H 2500 7000 50  0001 C CNN "LCSC"
+F 5 "C144807" H 2500 7000 50  0001 C CNN "LCSC"
 F 6 "-" H 2500 7000 50  0001 C CNN "Mouser"
 F 7 "N" H 2500 7000 50  0001 C CNN "Sponsored"
+F 8 "YAGEO" H 2500 7000 50  0001 C CNN "MANUFACTURER"
+F 9 "AC0402FR-0710KL" H 2500 7000 50  0001 C CNN "MPN"
 	1    2500 7000
 	0    1    1    0
@@
 F 3 "~" H 2300 7400 50  0001 C CNN
 F 4 "" H 2300 7400 50  0001 C CNN "Price"
-F 5 "" H 2300 7400 50  0001 C CNN "LCSC"
+F 5 "C144807" H 2300 7400 50  0001 C CNN "LCSC"
 F 6 "-" H 2300 7400 50  0001 C CNN "Mouser"
 F 7 "N" H 2300 7400 50  0001 C CNN "Sponsored"
+F 8 "YAGEO" H 2300 7400 50  0001 C CNN "MANUFACTURER"
+F 9 "AC0402FR-0710KL" H 2300 7400 50  0001 C CNN "MPN"
 	1    2300 7400
 	1    0    0    -1
@@
 F 3 "~" H 2750 1150 50  0001 C CNN
 F 4 "" H 2750 1150 50  0001 C CNN "Price"
-F 5 "C258126 " H 2750 1150 50  0001 C CNN "LCSC"
+F 5 "C4109" H 2750 1150 50  0001 C CNN "LCSC"
 F 6 "-" H 2750 1150 50  0001 C CNN "Mouser"
 F 7 "N" H 2750 1150 50  0001 C CNN "Sponsored"
+F 8 "UNI-ROYAL" H 2750 1150 50  0001 C CNN "MANUFACTURER"
+F 9 "0402WGF2001TCE" H 2750 1150 50  0001 C CNN "MPN"
 	1    2750 1150
 	0    -1   -1   0
@@
 F 3 "~" H 3400 3600 50  0001 C CNN
 F 4 "" H 3400 3600 50  0001 C CNN "Price"
-F 5 "" H 3400 3600 50  0001 C CNN "LCSC"
+F 5 "C144807" H 3400 3600 50  0001 C CNN "LCSC"
 F 6 "-" H 3400 3600 50  0001 C CNN "Mouser"
 F 7 "N" H 3400 3600 50  0001 C CNN "Sponsored"
+F 8 "YAGEO" H 3400 3600 50  0001 C CNN "MANUFACTURER"
+F 9 "AC0402FR-0710KL" H 3400 3600 50  0001 C CNN "MPN"
 	1    3400 3600
 	-1   0    0    1
@@
 P 2950 2750
 F 0 "D9" H 2900 2850 50  0000 L CNN
-F 1 "NSVR0320MW2T1G" H 2600 2650 50  0000 L CNN
+F 1 "PSBD3D40V1H" H 2700 2650 50  0000 L CNN
 F 2 "Diode_SMD:D_SOD-323" H 2950 2750 50  0001 C CNN
-F 3 "" H 2950 2750 50  0001 C CNN
+F 3 "https://datasheet.lcsc.com/lcsc/1810251323_Shanghai-Prisemi-Elec-PSBD3D40V1H_C110733.pdf" H 2950 2750 50  0001 C CNN
 F 4 "N" H 2950 2750 50  0001 C CNN "Sponsored"
-F 5 "C232573" H 2950 2750 50  0001 C CNN "LCSC"
+F 5 "C110733" H 2950 2750 50  0001 C CNN "LCSC"
 	1    2950 2750
 	-1   0    0    1
@@
 F 3 "~" H 2450 3800 50  0001 C CNN
 F 4 "" H 2450 3800 50  0001 C CNN "Price"
-F 5 "" H 2450 3800 50  0001 C CNN "LCSC"
+F 5 "C258090" H 2450 3800 50  0001 C CNN "LCSC"
 F 6 "-" H 2450 3800 50  0001 C CNN "Mouser"
 F 7 "N" H 2450 3800 50  0001 C CNN "Sponsored"
+F 8 "FH" H 2450 3800 50  0001 C CNN "MANUFACTURER"
+F 9 "RC-02W1003FT" H 2450 3800 50  0001 C CNN "MPN"
 	1    2450 3800
 	-1   0    0    1
@@
 F 3 "~" H 1550 3400 50  0001 C CNN
 F 4 "" H 1550 3400 50  0001 C CNN "Price"
-F 5 "" H 1550 3400 50  0001 C CNN "LCSC"
+F 5 "C144807" H 1550 3400 50  0001 C CNN "LCSC"
 F 6 "-" H 1550 3400 50  0001 C CNN "Mouser"
 F 7 "N" H 1550 3400 50  0001 C CNN "Sponsored"
+F 8 "YAGEO" H 1550 3400 50  0001 C CNN "MANUFACTURER"
+F 9 "AC0402FR-0710KL" H 1550 3400 50  0001 C CNN "MPN"
 	1    1550 3400
 	0    -1   -1   0
@@
 F 3 "~" H 1300 3950 50  0001 C CNN
 F 4 "" H 1300 3950 50  0001 C CNN "Price"
-F 5 "" H 1300 3950 50  0001 C CNN "LCSC"
+F 5 "C258090" H 1300 3950 50  0001 C CNN "LCSC"
 F 6 "-" H 1300 3950 50  0001 C CNN "Mouser"
 F 7 "N" H 1300 3950 50  0001 C CNN "Sponsored"
+F 8 "FH" H 1300 3950 50  0001 C CNN "MANUFACTURER"
+F 9 "RC-02W1003FT" H 1300 3950 50  0001 C CNN "MPN"
 	1    1300 3950
 	1    0    0    -1
@@
 F 3 "~" H 1550 3800 50  0001 C CNN
 F 4 "" H 1550 3800 50  0001 C CNN "Price"
-F 5 "" H 1550 3800 50  0001 C CNN "LCSC"
+F 5 "C144807" H 1550 3800 50  0001 C CNN "LCSC"
 F 6 "-" H 1550 3800 50  0001 C CNN "Mouser"
 F 7 "N" H 1550 3800 50  0001 C CNN "Sponsored"
+F 8 "YAGEO" H 1550 3800 50  0001 C CNN "MANUFACTURER"
+F 9 "AC0402FR-0710KL" H 1550 3800 50  0001 C CNN "MPN"
 	1    1550 3800
 	0    -1   -1   0
@@
 F 6 "" H 1900 3800 50  0001 C CNN "Price"
 F 7 "N" H 1900 3800 50  0001 C CNN "Sponsored"
+F 8 "ALLPOWER" H 1900 3800 50  0001 C CNN "MANUFACTURER"
+F 9 "AP2302B" H 1900 3800 50  0001 C CNN "MPN"
 	1    1900 3800
 	1    0    0    -1
@@
 F 3 "~" H 900 5150 50  0001 C CNN
 F 4 "" H 900 5150 50  0001 C CNN "Price"
-F 5 "" H 900 5150 50  0001 C CNN "LCSC"
+F 5 "C60485" H 900 5150 50  0001 C CNN "LCSC"
 F 6 "-" H 900 5150 50  0001 C CNN "Mouser"
 F 7 "N" H 900 5150 50  0001 C CNN "Sponsored"
+F 8 "YAGEO" H 900 5150 50  0001 C CNN "MANUFACTURER"
+F 9 "RC0402JR-070RL" H 900 5150 50  0001 C CNN "MPN"
 	1    900  5150
 	0    1    1    0
@@
 F 3 "~" H 900 6900 50  0001 C CNN
 F 4 "" H 900 6900 50  0001 C CNN "Price"
-F 5 "" H 900 6900 50  0001 C CNN "LCSC"
+F 5 "C60485" H 900 6900 50  0001 C CNN "LCSC"
 F 6 "-" H 900 6900 50  0001 C CNN "Mouser"
 F 7 "N" H 900 6900 50  0001 C CNN "Sponsored"
+F 8 "YAGEO" H 900 6900 50  0001 C CNN "MANUFACTURER"
+F 9 "RC0402JR-070RL" H 900 6900 50  0001 C CNN "MPN"
 	1    900  6900
 	0    1    1    0
@@
 F 3 "~" H 2700 1900 50  0001 C CNN
 F 4 "" H 2700 1900 50  0001 C CNN "Price"
-F 5 "C258126 " H 2700 1900 50  0001 C CNN "LCSC"
+F 5 "C144807" H 2700 1900 50  0001 C CNN "LCSC"
 F 6 "-" H 2700 1900 50  0001 C CNN "Mouser"
 F 7 "N" H 2700 1900 50  0001 C CNN "Sponsored"
+F 8 "YAGEO" H 2700 1900 50  0001 C CNN "MANUFACTURER"
+F 9 "AC0402FR-0710KL" H 2700 1900 50  0001 C CNN "MPN"
 	1    2700 1900
 	1    0    0    -1
