File: bosch.sch (KiCad schematic (older format))
At the start: 11 parts

Commit message: Schematic for prototype 2 is now complete, time for review! :D
Parts:
- gave numbers to parts that had none: 11
