File: bosch.sch (KiCad schematic (older format))
At the start: 11 parts, among them U16 BNO055, U17 BME680, Y3 32kHz

Commit message: Updated schematic, add design file
Parts:
- Y3: footprint (none) -> Crystal:Crystal_SMD_3215-2Pin_3.2x1.5mm
Changed lines of the file:
@@
 F 0 "Y3" V 5654 4138 50  0000 L CNN
 F 1 "32kHz" V 5745 4138 50  0000 L CNN
-F 2 "" H 5700 4050 50  0001 C CNN
+F 2 "Crystal:Crystal_SMD_3215-2Pin_3.2x1.5mm" H 5700 4050 50  0001 C CNN
 F 3 "~" H 5700 4050 50  0001 C CNN
 	1    5700 4050

Commit message: First steps of routing prototype 2, switch to 0402 for most passives
Parts:
- C31, C47, C50: footprint Capacitor_SMD:C_0603_1608Metric -> Capacitor_SMD:C_0402_1005Metric; LCSC C14663 -> C83056
- C48, C49: footprint Capacitor_SMD:C_0603_1608Metric -> Capacitor_SMD:C_0402_1005Metric; LCSC C388041 -> C696906
- R70, R71, R72: footprint Resistor_SMD:R_0603_1608Metric -> Resistor_SMD:R_0402_1005Metric; LCSC C269694 -> (none)
Changed lines of the file:
@@
 F 0 "C47" V 4900 4650 50  0000 L CNN
 F 1 "100n" V 5200 4600 50  0000 L CNN
-F 2 "Capacitor_SMD:C_0603_1608Metric" H 5088 4550 50  0001 C CNN
-F 3 "~" H 5050 4700 50  0001 C CNN
-F 4 "C14663" H 5050 4700 50  0001 C CNN "LCSC"
+F 2 "Capacitor_SMD:C_0402_1005Metric" H 5088 4550 50  0001 C CNN
+F 3 "" H 5050 4700 50  0001 C CNN
+F 4 "C83056 " H 5050 4700 50  0001 C CNN "LCSC"
 F 5 "" H 5050 4700 50  0001 C CNN "Price"
 F 6 "-" H 5050 4700 50  0001 C CNN "Mouser"
@@
 F 0 "R72" H 5459 3496 50  0000 L CNN
 F 1 "4k7" H 5459 3405 50  0000 L CNN
-F 2 "Resistor_SMD:R_0603_1608Metric" H 5400 3450 50  0001 C CNN
+F 2 "Resistor_SMD:R_0402_1005Metric" H 5400 3450 50  0001 C CNN
 F 3 "~" H 5400 3450 50  0001 C CNN
 F 4 "" H 5400 3450 50  0001 C CNN "Price"
-F 5 "C269694" H 5400 3450 50  0001 C CNN "LCSC"
+F 5 "" H 5400 3450 50  0001 C CNN "LCSC"
 F 6 "-" H 5400 3450 50  0001 C CNN "Mouser"
 F 7 "N" H 5400 3450 50  0001 C CNN "Sponsored"
@@
 F 0 "R71" H 3409 3496 50  0000 L CNN
 F 1 "4k7" H 3409 3405 50  0000 L CNN
-F 2 "Resistor_SMD:R_0603_1608Metric" H 3350 3450 50  0001 C CNN
+F 2 "Resistor_SMD:R_0402_1005Metric" H 3350 3450 50  0001 C CNN
 F 3 "~" H 3350 3450 50  0001 C CNN
 F 4 "" H 3350 3450 50  0001 C CNN "Price"
-F 5 "C269694" H 3350 3450 50  0001 C CNN "LCSC"
+F 5 "" H 3350 3450 50  0001 C CNN "LCSC"
 F 6 "-" H 3350 3450 50  0001 C CNN "Mouser"
 F 7 "N" H 3350 3450 50  0001 C CNN "Sponsored"
@@
 F 0 "C48" H 5350 4800 50  0000 L CNN
 F 1 "22p" H 5300 4600 50  0000 L CNN
-F 2 "Capacitor_SMD:C_0603_1608Metric" H 5538 4550 50  0001 C CNN
-F 3 "~" H 5500 4700 50  0001 C CNN
-F 4 "C388041" H 5500 4700 50  0001 C CNN "LCSC"
+F 2 "Capacitor_SMD:C_0402_1005Metric" H 5538 4550 50  0001 C CNN
+F 3 "" H 5500 4700 50  0001 C CNN
+F 4 "C696906" H 5500 4700 50  0001 C CNN "LCSC"
 F 5 "" H 5500 4700 50  0001 C CNN "Price"
 F 6 "N" H 5500 4700 50  0001 C CNN "Sponsored"
@@
 F 0 "C49" H 5750 4800 50  0000 L CNN
 F 1 "22p" H 5700 4600 50  0000 L CNN
-F 2 "Capacitor_SMD:C_0603_1608Metric" H 5938 4550 50  0001 C CNN
-F 3 "~" H 5900 4700 50  0001 C CNN
-F 4 "C388041" H 5900 4700 50  0001 C CNN "LCSC"
+F 2 "Capacitor_SMD:C_0402_1005Metric" H 5938 4550 50  0001 C CNN
+F 3 "" H 5900 4700 50  0001 C CNN
+F 4 "C696906" H 5900 4700 50  0001 C CNN "LCSC"
 F 5 "" H 5900 4700 50  0001 C CNN "Price"
 F 6 "N" H 5900 4700 50  0001 C CNN "Sponsored"
@@
 F 0 "R70" H 3109 3496 50  0000 L CNN
 F 1 "4k7" H 3109 3405 50  0000 L CNN
-F 2 "Resistor_SMD:R_0603_1608Metric" H 3050 3450 50  0001 C CNN
+F 2 "Resistor_SMD:R_0402_1005Metric" H 3050 3450 50  0001 C CNN
 F 3 "~" H 3050 3450 50  0001 C CNN
 F 4 "" H 3050 3450 50  0001 C CNN "Price"
-F 5 "C269694" H 3050 3450 50  0001 C CNN "LCSC"
+F 5 "" H 3050 3450 50  0001 C CNN "LCSC"
 F 6 "-" H 3050 3450 50  0001 C CNN "Mouser"
 F 7 "N" H 3050 3450 50  0001 C CNN "Sponsored"
@@
 F 0 "C50" V 6850 4650 50  0000 L CNN
 F 1 "100n" V 7150 4600 50  0000 L CNN
-F 2 "Capacitor_SMD:C_0603_1608Metric" H 7038 4550 50  0001 C CNN
-F 3 "~" H 7000 4700 50  0001 C CNN
-F 4 "C14663" H 7000 4700 50  0001 C CNN "LCSC"
+F 2 "Capacitor_SMD:C_0402_1005Metric" H 7038 4550 50  0001 C CNN
+F 3 "" H 7000 4700 50  0001 C CNN
+F 4 "C83056 " H 7000 4700 50  0001 C CNN "LCSC"
 F 5 "" H 7000 4700 50  0001 C CNN "Price"
 F 6 "-" H 7000 4700 50  0001 C CNN "Mouser"
@@
 F 0 "C31" V 2250 4650 50  0000 L CNN
 F 1 "100n" V 2550 4600 50  0000 L CNN
-F 2 "Capacitor_SMD:C_0603_1608Metric" H 2438 4550 50  0001 C CNN
-F 3 "~" H 2400 4700 50  0001 C CNN
-F 4 "C14663" H 2400 4700 50  0001 C CNN "LCSC"
+F 2 "Capacitor_SMD:C_0402_1005Metric" H 2438 4550 50  0001 C CNN
+F 3 "" H 2400 4700 50  0001 C CNN
+F 4 "C83056 " H 2400 4700 50  0001 C CNN "LCSC"
 F 5 "" H 2400 4700 50  0001 C CNN "Price"
 F 6 "-" H 2400 4700 50  0001 C CNN "Mouser"

Commit message: More routing...
Connections:
- net BNO055_XOUT32: now reaches C49.1, U16.26 (XOUT32), Y3.1
- net BNO055_XIN32: now reaches C48.1, U16.27 (XIN32), Y3.2
- net BNO055_CAP: now reaches C47.1, U16.9 (CAP)
Changed lines of the file:
@@
 Text Notes 550  850  0    197  ~ 0
 BOSCH BNO055 & BME680 SENSORS
+Text Label 5050 4300 1    20   ~ 0
+BNO055_CAP
+Text Label 5000 3950 0    20   ~ 0
+BNO055_XIN32
+Text Label 5000 3850 0    20   ~ 0
+BNO055_XOUT32
 $EndSCHEMATC

Commit message: Some more work
Parts:
- renumbered C31 to C26, C47 to C27, C48 to C28, C49 to C29, C50 to C30, R70 to R47, R71 to R48, R72 to R49, U16 to U8, U17 to U9
Changed lines of the file:
@@
 $EndDescr
 $Comp
-L Sensor:BME680 U17
+L Sensor:BME680 U9
 U 1 1 5FDA6CD0
 P 7700 4250
-F 0 "U17" H 7300 4800 50  0000 R CNN
+F 0 "U9" H 7300 4800 50  0000 R CNN
 F 1 "BME680" H 7500 4700 50  0000 R CNN
 F 2 "Package_LGA:Bosch_LGA-8_3x3mm_P0.8mm_ClockwisePinNumbering" H 9150 3800 50  0001 C CNN
@@
 	8400 3950 8400 3650
 $Comp
-L power:+3.3V #PWR0215
+L power:+3.3V #PWR0136
 U 1 1 5FDAD653
 P 7600 3650
-F 0 "#PWR0215" H 7600 3500 50  0001 C CNN
+F 0 "#PWR0136" H 7600 3500 50  0001 C CNN
 F 1 "+3.3V" V 7600 3900 50  0000 C CNN
 F 2 "" H 7600 3650 50  0001 C CNN
@@
 $EndComp
 $Comp
-L power:+3.3V #PWR0216
+L power:+3.3V #PWR0138
 U 1 1 5FDADA74
 P 7800 3650
-F 0 "#PWR0216" H 7800 3500 50  0001 C CNN
+F 0 "#PWR0138" H 7800 3500 50  0001 C CNN
 F 1 "+3.3V" V 7800 3900 50  0000 C CNN
 F 2 "" H 7800 3650 50  0001 C CNN
@@
 $EndComp
 $Comp
-L power:+3.3V #PWR0217
+L power:+3.3V #PWR0140
 U 1 1 5FDADCA9
 P 8400 3650
-F 0 "#PWR0217" H 8400 3500 50  0001 C CNN
+F 0 "#PWR0140" H 8400 3500 50  0001 C CNN
 F 1 "+3.3V" V 8400 3900 50  0000 C CNN
 F 2 "" H 8400 3650 50  0001 C CNN
@@
 $EndComp
 $Comp
-L power:+3.3V #PWR0218
+L power:+3.3V #PWR0141
 U 1 1 5FDAE00D
 P 8700 3650
-F 0 "#PWR0218" H 8700 3500 50  0001 C CNN
+F 0 "#PWR0141" H 8700 3500 50  0001 C CNN
 F 1 "+3.3V" V 8700 3900 50  0000 C CNN
 F 2 "" H 8700 3650 50  0001 C CNN
@@
 SDA
 $Comp
-L power:GND #PWR0219
+L power:GND #PWR0137
 U 1 1 5FDB054C
 P 7600 4850
-F 0 "#PWR0219" H 7600 4600 50  0001 C CNN
+F 0 "#PWR0137" H 7600 4600 50  0001 C CNN
 F 1 "GND" V 7600 4650 50  0000 C CNN
 F 2 "" H 7600 4850 50  0001 C CNN
@@
 $EndComp
 $Comp
-L power:GND #PWR0220
+L power:GND #PWR0139
 U 1 1 5FDB0857
 P 7800 4850
-F 0 "#PWR0220" H 7800 4600 50  0001 C CNN
+F 0 "#PWR0139" H 7800 4600 50  0001 C CNN
 F 1 "GND" V 7800 4650 50  0000 C CNN
 F 2 "" H 7800 4850 50  0001 C CNN
@@
 $EndComp
 $Comp
-L power:+3.3V #PWR0221
+L power:+3.3V #PWR0128
 U 1 1 5FDB4B11
 P 4450 3350
-F 0 "#PWR0221" H 4450 3200 50  0001 C CNN
+F 0 "#PWR0128" H 4450 3200 50  0001 C CNN
 F 1 "+3.3V" V 4450 3600 50  0000 C CNN
 F 2 "" H 4450 3350 50  0001 C CNN
@@
 $EndComp
 $Comp
-L power:+3.3V #PWR0222
+L power:+3.3V #PWR0126
 U 1 1 5FDB5755
 P 4350 3350
-F 0 "#PWR0222" H 4350 3200 50  0001 C CNN
+F 0 "#PWR0126" H 4350 3200 50  0001 C CNN
 F 1 "+3.3V" V 4350 3600 50  0000 C CNN
 F 2 "" H 4350 3350 50  0001 C CNN
@@
 SDA
 $Comp
-L dk_Motion-Sensors-IMUs-Inertial-Measurement-Units:BNO055 U16
+L dk_Motion-Sensors-IMUs-Inertial-Measurement-Units:BNO055 U8
 U 1 1 5FDBA21A
 P 4250 4050
-F 0 "U16" H 3700 4600 50  0000 C CNN
+F 0 "U8" H 3700 4600 50  0000 C CNN
 F 1 "BNO055" H 4700 4600 50  0000 C CNN
 F 2 "digikey-footprints:LGA-28_5.2x3.8mm_BNO0055" H 4450 4250 60  0001 L CNN
@@
 $EndComp
 $Comp
-L power:GND #PWR0223
+L power:GND #PWR0127
 U 1 1 5FDC2D52
 P 4350 4850
-F 0 "#PWR0223" H 4350 4600 50  0001 C CNN
+F 0 "#PWR0127" H 4350 4600 50  0001 C CNN
 F 1 "GND" V 4350 4650 50  0000 C CNN
 F 2 "" H 4350 4850 50  0001 C CNN
@@
 $EndComp
 $Comp
-L power:GND #PWR0224
+L power:GND #PWR0123
 U 1 1 5FDC3E74
 P 4050 4850
-F 0 "#PWR0224" H 4050 4600 50  0001 C CNN
+F 0 "#PWR0123" H 4050 4600 50  0001 C CNN
 F 1 "GND" V 4050 4650 50  0000 C CNN
 F 2 "" H 4050 4850 50  0001 C CNN
@@
 $EndComp
 $Comp
-L power:GND #PWR0225
+L power:GND #PWR0124
 U 1 1 5FDC40F7
 P 4150 4850
-F 0 "#PWR0225" H 4150 4600 50  0001 C CNN
+F 0 "#PWR0124" H 4150 4600 50  0001 C CNN
 F 1 "GND" V 4150 4650 50  0000 C CNN
 F 2 "" H 4150 4850 50  0001 C CNN
@@
 $EndComp
 $Comp
-L power:GND #PWR0226
+L power:GND #PWR0125
 U 1 1 5FDC4313
 P 4250 4850
-F 0 "#PWR0226" H 4250 4600 50  0001 C CNN
+F 0 "#PWR0125" H 4250 4600 50  0001 C CNN
 F 1 "GND" V 4250 4650 50  0000 C CNN
 F 2 "" H 4250 4850 50  0001 C CNN
@@
 	3450 4050 3450 4850
 $Comp
-L power:GND #PWR0227
+L power:GND #PWR0122
 U 1 1 5FDC69E0
 P 3450 4850
-F 0 "#PWR0227" H 3450 4600 50  0001 C CNN
+F 0 "#PWR0122" H 3450 4600 50  0001 C CNN
 F 1 "GND" V 3450 4650 50  0000 C CNN
 F 2 "" H 3450 4850 50  0001 C CNN
@@
 P 5050 4700
 AR Path="/60C789DE/5FDD510F" Ref="C?"  Part="1"
-AR Path="/5FDA4DDF/5FDD510F" Ref="C47"  Part="1"
-F 0 "C47" V 4900 4650 50  0000 L CNN
+AR Path="/5FDA4DDF/5FDD510F" Ref="C27"  Part="1"
+F 0 "C27" V 4900 4650 50  0000 L CNN
 F 1 "100n" V 5200 4600 50  0000 L CNN
 F 2 "Capacitor_SMD:C_0402_1005Metric" H 5088 4550 50  0001 C CNN
@@
 $EndComp
 $Comp
-L power:GND #PWR0228
+L power:GND #PWR0129
 U 1 1 5FDD53C2
 P 5050 4850
-F 0 "#PWR0228" H 5050 4600 50  0001 C CNN
+F 0 "#PWR0129" H 5050 4600 50  0001 C CNN
 F 1 "GND" V 5050 4650 50  0000 C CNN
 F 2 "" H 5050 4850 50  0001 C CNN
@@
 P 5400 3450
 AR Path="/6057522A/5FDDF192" Ref="R?"  Part="1"
-AR Path="/5FDA4DDF/5FDDF192" Ref="R72"  Part="1"
-F 0 "R72" H 5459 3496 50  0000 L CNN
+AR Path="/5FDA4DDF/5FDDF192" Ref="R49"  Part="1"
+F 0 "R49" H 5459 3496 50  0000 L CNN
 F 1 "4k7" H 5459 3405 50  0000 L CNN
 F 2 "Resistor_SMD:R_0402_1005Metric" H 5400 3450 50  0001 C CNN
@@
 P 5400 3350
 AR Path="/6057522A/5FDDF199" Ref="#PWR?"  Part="1"
-AR Path="/5FDA4DDF/5FDDF199" Ref="#PWR0229"  Part="1"
-F 0 "#PWR0229" H 5400 3200 50  0001 C CNN
+AR Path="/5FDA4DDF/5FDDF199" Ref="#PWR0131"  Part="1"
+F 0 "#PWR0131" H 5400 3200 50  0001 C CNN
 F 1 "+3.3V" V 5415 3478 50  0000 L CNN
 F 2 "" H 5400 3350 50  0001 C CNN
@@
 P 3350 3450
 AR Path="/6057522A/5FDE4845" Ref="R?"  Part="1"
-AR Path="/5FDA4DDF/5FDE4845" Ref="R71"  Part="1"
-F 0 "R71" H 3409 3496 50  0000 L CNN
+AR Path="/5FDA4DDF/5FDE4845" Ref="R48"  Part="1"
+F 0 "R48" H 3409 3496 50  0000 L CNN
 F 1 "4k7" H 3409 3405 50  0000 L CNN
 F 2 "Resistor_SMD:R_0402_1005Metric" H 3350 3450 50  0001 C CNN
@@
 P 3350 3350
 AR Path="/6057522A/5FDE484C" Ref="#PWR?"  Part="1"
-AR Path="/5FDA4DDF/5FDE484C" Ref="#PWR0230"  Part="1"
-F 0 "#PWR0230" H 3350 3200 50  0001 C CNN
+AR Path="/5FDA4DDF/5FDE484C" Ref="#PWR0121"  Part="1"
+F 0 "#PWR0121" H 3350 3200 50  0001 C CNN
 F 1 "+3.3V" V 3365 3478 50  0000 L CNN
 F 2 "" H 3350 3350 50  0001 C CNN
@@
 	5300 3650 5300 4850
 $Comp
-L power:GND #PWR0231
+L power:GND #PWR0130
 U 1 1 5FDF8481
 P 5300 4850
-F 0 "#PWR0231" H 5300 4600 50  0001 C CNN
+F 0 "#PWR0130" H 5300 4600 50  0001 C CNN
 F 1 "GND" V 5300 4650 50  0000 C CNN
 F 2 "" H 5300 4850 50  0001 C CNN
@@
 AR Path="/5E3BA64A/5FDFF3EC" Ref="C?"  Part="1"
 AR Path="/5F51E414/5FDFF3EC" Ref="C?"  Part="1"
-AR Path="/5FDA4DDF/5FDFF3EC" Ref="C48"  Part="1"
-F 0 "C48" H 5350 4800 50  0000 L CNN
+AR Path="/5FDA4DDF/5FDFF3EC" Ref="C28"  Part="1"
+F 0 "C28" H 5350 4800 50  0000 L CNN
 F 1 "22p" H 5300 4600 50  0000 L CNN
 F 2 "Capacitor_SMD:C_0402_1005Metric" H 5538 4550 50  0001 C CNN
@@
 AR Path="/5E3BA64A/5FDFF81E" Ref="C?"  Part="1"
 AR Path="/5F51E414/5FDFF81E" Ref="C?"  Part="1"
-AR Path="/5FDA4DDF/5FDFF81E" Ref="C49"  Part="1"
-F 0 "C49" H 5750 4800 50  0000 L CNN
+AR Path="/5FDA4DDF/5FDFF81E" Ref="C29"  Part="1"
+F 0 "C29" H 5750 4800 50  0000 L CNN
 F 1 "22p" H 5700 4600 50  0000 L CNN
 F 2 "Capacitor_SMD:C_0402_1005Metric" H 5938 4550 50  0001 C CNN
@@
 $EndComp
 $Comp
-L power:GND #PWR0232
+L power:GND #PWR0132
 U 1 1 5FE114D2
 P 5500 4850
-F 0 "#PWR0232" H 5500 4600 50  0001 C CNN
+F 0 "#PWR0132" H 5500 4600 50  0001 C CNN
 F 1 "GND" V 5500 4650 50  0000 C CNN
 F 2 "" H 5500 4850 50  0001 C CNN
@@
 $EndComp
 $Comp
-L power:GND #PWR0233
+L power:GND #PWR0133
 U 1 1 5FE1191E
 P 5900 4850
-F 0 "#PWR0233" H 5900 4600 50  0001 C CNN
+F 0 "#PWR0133" H 5900 4600 50  0001 C CNN
 F 1 "GND" V 5900 4650 50  0000 C CNN
 F 2 "" H 5900 4850 50  0001 C CNN
@@
 P 3050 3450
 AR Path="/6057522A/5FE17C0C" Ref="R?"  Part="1"
-AR Path="/5FDA4DDF/5FE17C0C" Ref="R70"  Part="1"
-F 0 "R70" H 3109 3496 50  0000 L CNN
+AR Path="/5FDA4DDF/5FE17C0C" Ref="R47"  Part="1"
+F 0 "R47" H 3109 3496 50  0000 L CNN
 F 1 "4k7" H 3109 3405 50  0000 L CNN
 F 2 "Resistor_SMD:R_0402_1005Metric" H 3050 3450 50  0001 C CNN
@@
 P 3050 3350
 AR Path="/6057522A/5FE17C12" Ref="#PWR?"  Part="1"
-AR Path="/5FDA4DDF/5FE17C12" Ref="#PWR0234"  Part="1"
-F 0 "#PWR0234" H 3050 3200 50  0001 C CNN
+AR Path="/5FDA4DDF/5FE17C12" Ref="#PWR0120"  Part="1"
+F 0 "#PWR0120" H 3050 3200 50  0001 C CNN
 F 1 "+3.3V" V 3065 3478 50  0000 L CNN
 F 2 "" H 3050 3350 50  0001 C CNN
@@
 P 7000 4700
 AR Path="/60C789DE/5FE44369" Ref="C?"  Part="1"
-AR Path="/5FDA4DDF/5FE44369" Ref="C50"  Part="1"
-F 0 "C50" V 6850 4650 50  0000 L CNN
+AR Path="/5FDA4DDF/5FE44369" Ref="C30"  Part="1"
+F 0 "C30" V 6850 4650 50  0000 L CNN
 F 1 "100n" V 7150 4600 50  0000 L CNN
 F 2 "Capacitor_SMD:C_0402_1005Metric" H 7038 4550 50  0001 C CNN
@@
 $EndComp
 $Comp
-L power:GND #PWR0235
+L power:GND #PWR0135
 U 1 1 5FE4436F
 P 7000 4850
-F 0 "#PWR0235" H 7000 4600 50  0001 C CNN
+F 0 "#PWR0135" H 7000 4600 50  0001 C CNN
 F 1 "GND" V 7000 4650 50  0000 C CNN
 F 2 "" H 7000 4850 50  0001 C CNN
@@
 $EndComp
 $Comp
-L power:+3.3V #PWR0236
+L power:+3.3V #PWR0134
 U 1 1 5FE4A185
 P 7000 4550
-F 0 "#PWR0236" H 7000 4400 50  0001 C CNN
+F 0 "#PWR0134" H 7000 4400 50  0001 C CNN
 F 1 "+3.3V" V 7000 4800 50  0000 C CNN
 F 2 "" H 7000 4550 50  0001 C CNN
@@
 P 2400 4700
 AR Path="/60C789DE/5FE5AFEB" Ref="C?"  Part="1"
-AR Path="/5FDA4DDF/5FE5AFEB" Ref="C31"  Part="1"
-F 0 "C31" V 2250 4650 50  0000 L CNN
+AR Path="/5FDA4DDF/5FE5AFEB" Ref="C26"  Part="1"
+F 0 "C26" V 2250 4650 50  0000 L CNN
 F 1 "100n" V 2550 4600 50  0000 L CNN
 F 2 "Capacitor_SMD:C_0402_1005Metric" H 2438 4550 50  0001 C CNN
@@
 $EndComp
 $Comp
-L power:GND #PWR0237
+L power:GND #PWR0119
 U 1 1 5FE5AFF1
 P 2400 4850
-F 0 "#PWR0237" H 2400 4600 50  0001 C CNN
+F 0 "#PWR0119" H 2400 4600 50  0001 C CNN
 F 1 "GND" V 2400 4650 50  0000 C CNN
 F 2 "" H 2400 4850 50  0001 C CNN
@@
 $EndComp
 $Comp
-L power:+3.3V #PWR0238
+L power:+3.3V #PWR0118
 U 1 1 5FE5AFF7
 P 2400 4550
-F 0 "#PWR0238" H 2400 4400 50  0001 C CNN
+F 0 "#PWR0118" H 2400 4400 50  0001 C CNN
 F 1 "+3.3V" V 2400 4800 50  0000 C CNN
 F 2 "" H 2400 4550 50  0001 C CNN

Commit message: Update LCSC code for the 32kHz crystals
Parts:
- Y3: LCSC (none) -> C271654
Changed lines of the file:
@@
 F 2 "Crystal:Crystal_SMD_3215-2Pin_3.2x1.5mm" H 5700 4050 50  0001 C CNN
 F 3 "~" H 5700 4050 50  0001 C CNN
+F 4 "C271654" H 5700 4050 50  0001 C CNN "LCSC"
 	1    5700 4050
 	-1   0    0    1
