File: bosch.sch (KiCad schematic (older format))
At the start: 11 parts, among them U8 BNO055, U9 BME680, Y3 32kHz

Commit message: Fix most of the bugs found on prototype 2 board
Parts:
- added TP15: BL, TestPoint:TestPoint_Pad_1.0x1.0mm, symbol Connector:TestPoint
Connections:
- net labels removed: BOOT
Changed lines of the file:
@@
 Sheet 6 9
 Title "MCH2021 badge - BOSCH"
-Date "2021-01-14"
-Rev "2"
+Date "2021-10-09"
+Rev "3"
 Comp "BADGE.TEAM"
 Comment1 ""
@@
 Wire Wire Line
 	3050 3750 3050 4350
-Text HLabel 2850 3650 0    50   Input ~ 0
-BOOT
 Text HLabel 2850 3750 0    50   Input ~ 0
 RESET
@@
 Text Label 5000 3850 0    20   ~ 0
 BNO055_XOUT32
+$Comp
+L Connector:TestPoint TP15
+U 1 1 61C1AC47
+P 2850 3650
+F 0 "TP15" V 3045 3722 50  0000 C CNN
+F 1 "BL" V 2954 3722 50  0000 C CNN
+F 2 "TestPoint:TestPoint_Pad_1.0x1.0mm" H 3050 3650 50  0001 C CNN
+F 3 "~" H 3050 3650 50  0001 C CNN
+	1    2850 3650
+	0    -1   -1   0
+$EndComp
 $EndSCHEMATC

Commit message: Change pinout of expansion header close to board edge to be fully ground instead of gnd + 3.3v (& update component references)
Parts:
- C26, C27, C28, C29, C30: symbol Device:C -> mch2021-rescue:C-Device
- R47, R48, R49: symbol Device:R_Small -> mch2021-rescue:R_Small-Device
- TP15: symbol Connector:TestPoint -> mch2021-rescue:TestPoint-Connector
- U8: symbol dk_Motion-Sensors-IMUs-Inertial-Measurement-Units:BNO055 -> mch2021-rescue:BNO055-dk_Motion-Sensors-IMUs-Inertial-Measurement-Units
- U9: symbol Sensor:BME680 -> mch2021-rescue:BME680-Sensor
- Y3: symbol Device:Crystal_Small -> mch2021-rescue:Crystal_Small-Device
Changed lines of the file:
@@
 $EndDescr
 $Comp
-L Sensor:BME680 U9
+L mch2021-rescue:BME680-Sensor U9
 U 1 1 5FDA6CD0
 P 7700 4250
@@
 	8400 3950 8400 3650
 $Comp
-L power:+3.3V #PWR0136
+L mch2021-rescue:+3.3V-power #PWR0136
 U 1 1 5FDAD653
 P 7600 3650
@@
 $EndComp
 $Comp
-L power:+3.3V #PWR0138
+L mch2021-rescue:+3.3V-power #PWR0138
 U 1 1 5FDADA74
 P 7800 3650
@@
 $EndComp
 $Comp
-L power:+3.3V #PWR0140
+L mch2021-rescue:+3.3V-power #PWR0140
 U 1 1 5FDADCA9
 P 8400 3650
@@
 $EndComp
 $Comp
-L power:+3.3V #PWR0141
+L mch2021-rescue:+3.3V-power #PWR0141
 U 1 1 5FDAE00D
 P 8700 3650
@@
 SDA
 $Comp
-L power:GND #PWR0137
+L mch2021-rescue:GND-power #PWR0137
 U 1 1 5FDB054C
 P 7600 4850
@@
 $EndComp
 $Comp
-L power:GND #PWR0139
+L mch2021-rescue:GND-power #PWR0139
 U 1 1 5FDB0857
 P 7800 4850
@@
 $EndComp
 $Comp
-L power:+3.3V #PWR0128
+L mch2021-rescue:+3.3V-power #PWR0128
 U 1 1 5FDB4B11
 P 4450 3350
@@
 $EndComp
 $Comp
-L power:+3.3V #PWR0126
+L mch2021-rescue:+3.3V-power #PWR0126
 U 1 1 5FDB5755
 P 4350 3350
@@
 SDA
 $Comp
-L dk_Motion-Sensors-IMUs-Inertial-Measurement-Units:BNO055 U8
+L mch2021-rescue:BNO055-dk_Motion-Sensors-IMUs-Inertial-Measurement-Units U8
 U 1 1 5FDBA21A
 P 4250 4050
@@
 $EndComp
 $Comp
-L power:GND #PWR0127
+L mch2021-rescue:GND-power #PWR0127
 U 1 1 5FDC2D52
 P 4350 4850
@@
 $EndComp
 $Comp
-L power:GND #PWR0123
+L mch2021-rescue:GND-power #PWR0123
 U 1 1 5FDC3E74
 P 4050 4850
@@
 $EndComp
 $Comp
-L power:GND #PWR0124
+L mch2021-rescue:GND-power #PWR0124
 U 1 1 5FDC40F7
 P 4150 4850
@@
 $EndComp
 $Comp
-L power:GND #PWR0125
+L mch2021-rescue:GND-power #PWR0125
 U 1 1 5FDC4313
 P 4250 4850
@@
 	3450 4050 3450 4850
 $Comp
-L power:GND #PWR0122
+L mch2021-rescue:GND-power #PWR0122
 U 1 1 5FDC69E0
 P 3450 4850
@@
 INT
 $Comp
-L Device:C C?
+L mch2021-rescue:C-Device C?
 U 1 1 5FDD510F
 P 5050 4700
@@
 $EndComp
 $Comp
-L power:GND #PWR0129
+L mch2021-rescue:GND-power #PWR0129
 U 1 1 5FDD53C2
 P 5050 4850
@@
 	5550 3750 5400 3750
 $Comp
-L Device:R_Small R?
+L mch2021-rescue:R_Small-Device R?
 U 1 1 5FDDF192
 P 5400 3450
@@
 	5400 3550 5400 3750
 $Comp
-L power:+3.3V #PWR?
+L mch2021-rescue:+3.3V-power #PWR?
 U 1 1 5FDDF199
 P 5400 3350
@@
 	3450 3950 3450 4050
 $Comp
-L Device:R_Small R?
+L mch2021-rescue:R_Small-Device R?
 U 1 1 5FDE4845
 P 3350 3450
@@
 $EndComp
 $Comp
-L power:+3.3V #PWR?
+L mch2021-rescue:+3.3V-power #PWR?
 U 1 1 5FDE484C
 P 3350 3350
@@
 	5300 3650 5300 4850
 $Comp
-L power:GND #PWR0130
+L mch2021-rescue:GND-power #PWR0130
 U 1 1 5FDF8481
 P 5300 4850
@@
 $EndComp
 $Comp
-L Device:C C?
+L mch2021-rescue:C-Device C?
 U 1 1 5FDFF3EC
 P 5500 4700
@@
 $EndComp
 $Comp
-L Device:C C?
+L mch2021-rescue:C-Device C?
 U 1 1 5FDFF81E
 P 5900 4700
@@
 $EndComp
 $Comp
-L Device:Crystal_Small Y?
+L mch2021-rescue:Crystal_Small-Device Y?
 U 1 1 5FE05137
 P 5700 4050
@@
 $EndComp
 $Comp
-L power:GND #PWR0132
+L mch2021-rescue:GND-power #PWR0132
 U 1 1 5FE114D2
 P 5500 4850
@@
 $EndComp
 $Comp
-L power:GND #PWR0133
+L mch2021-rescue:GND-power #PWR0133
 U 1 1 5FE1191E
 P 5900 4850
@@
 Connection ~ 5900 4050
 $Comp
-L Device:R_Small R?
+L mch2021-rescue:R_Small-Device R?
 U 1 1 5FE17C0C
 P 3050 3450
@@
 $EndComp
 $Comp
-L power:+3.3V #PWR?
+L mch2021-rescue:+3.3V-power #PWR?
 U 1 1 5FE17C12
 P 3050 3350
@@
 RESET
 $Comp
-L Device:C C?
+L mch2021-rescue:C-Device C?
 U 1 1 5FE44369
 P 7000 4700
@@
 $EndComp
 $Comp
-L power:GND #PWR0135
+L mch2021-rescue:GND-power #PWR0135
 U 1 1 5FE4436F
 P 7000 4850
@@
 $EndComp
 $Comp
-L power:+3.3V #PWR0134
+L mch2021-rescue:+3.3V-power #PWR0134
 U 1 1 5FE4A185
 P 7000 4550
@@
 $EndComp
 $Comp
-L Device:C C?
+L mch2021-rescue:C-Device C?
 U 1 1 5FE5AFEB
 P 2400 4700
@@
 $EndComp
 $Comp
-L power:GND #PWR0119
+L mch2021-rescue:GND-power #PWR0119
 U 1 1 5FE5AFF1
 P 2400 4850
@@
 $EndComp
 $Comp
-L power:+3.3V #PWR0118
+L mch2021-rescue:+3.3V-power #PWR0118
 U 1 1 5FE5AFF7
 P 2400 4550
@@
 BNO055_XOUT32
 $Comp
-L Connector:TestPoint TP15
+L mch2021-rescue:TestPoint-Connector TP15
 U 1 1 61C1AC47
 P 2850 3650

Commit message: Last fixes before ordering
Parts:
- C28, C29: LCSC C696906 -> C106203; MANUFACTURER (none) -> YAGEO; MPN (none) -> CC0402JRNPO9BN220
- R47, R48, R49: value 4k7 -> 4.7k; LCSC (none) -> C25940; MANUFACTURER (none) -> UNI-ROYAL; MPN (none) -> 0402WGJ0472TCE
- U8: LCSC (none) -> C93216; Sponsored (none) -> Y; Status Active -> (none)
- U9: LCSC (none) -> C125972; MPN (none) -> BME680; Manufacturer (none) -> Bosch Sensortec
Changed lines of the file:
@@
 F 2 "Package_LGA:Bosch_LGA-8_3x3mm_P0.8mm_ClockwisePinNumbering" H 9150 3800 50  0001 C CNN
 F 3 "https://ae-bst.resource.bosch.com/media/_tech/media/datasheets/BST-BME680-DS001.pdf" H 7700 4050 50  0001 C CNN
+F 4 "C125972" H 7700 4250 50  0001 C CNN "LCSC"
+F 5 "BME680" H 7700 4250 50  0001 C CNN "MPN"
+F 6 "Bosch Sensortec" H 7700 4250 50  0001 C CNN "Manufacturer"
 	1    7700 4250
 	1    0    0    -1
@@
 F 10 "IMU ACCEL/GYRO/MAG I2C 28LGA" H 4450 5050 60  0001 L CNN "Description"
 F 11 "Bosch Sensortec" H 4450 5150 60  0001 L CNN "Manufacturer"
-F 12 "Active" H 4450 5250 60  0001 L CNN "Status"
+F 12 "" H 4450 5250 60  0001 L CNN "Status"
+F 13 "C93216" H 4250 4050 50  0001 C CNN "LCSC"
+F 14 "Y" H 4250 4050 50  0001 C CNN "Sponsored"
 	1    4250 4050
 	1    0    0    -1
@@
 AR Path="/5FDA4DDF/5FDDF192" Ref="R49"  Part="1"
 F 0 "R49" H 5459 3496 50  0000 L CNN
-F 1 "4k7" H 5459 3405 50  0000 L CNN
+F 1 "4.7k" H 5459 3405 50  0000 L CNN
 F 2 "Resistor_SMD:R_0402_1005Metric" H 5400 3450 50  0001 C CNN
 F 3 "~" H 5400 3450 50  0001 C CNN
 F 4 "" H 5400 3450 50  0001 C CNN "Price"
-F 5 "" H 5400 3450 50  0001 C CNN "LCSC"
+F 5 "C25940" H 5400 3450 50  0001 C CNN "LCSC"
 F 6 "-" H 5400 3450 50  0001 C CNN "Mouser"
 F 7 "N" H 5400 3450 50  0001 C CNN "Sponsored"
+F 8 "UNI-ROYAL" H 5400 3450 50  0001 C CNN "MANUFACTURER"
+F 9 "0402WGJ0472TCE" H 5400 3450 50  0001 C CNN "MPN"
 	1    5400 3450
 	1    0    0    -1
@@
 AR Path="/5FDA4DDF/5FDE4845" Ref="R48"  Part="1"
 F 0 "R48" H 3409 3496 50  0000 L CNN
-F 1 "4k7" H 3409 3405 50  0000 L CNN
+F 1 "4.7k" H 3409 3405 50  0000 L CNN
 F 2 "Resistor_SMD:R_0402_1005Metric" H 3350 3450 50  0001 C CNN
 F 3 "~" H 3350 3450 50  0001 C CNN
 F 4 "" H 3350 3450 50  0001 C CNN "Price"
-F 5 "" H 3350 3450 50  0001 C CNN "LCSC"
+F 5 "C25940" H 3350 3450 50  0001 C CNN "LCSC"
 F 6 "-" H 3350 3450 50  0001 C CNN "Mouser"
 F 7 "N" H 3350 3450 50  0001 C CNN "Sponsored"
+F 8 "UNI-ROYAL" H 3350 3450 50  0001 C CNN "MANUFACTURER"
+F 9 "0402WGJ0472TCE" H 3350 3450 50  0001 C CNN "MPN"
 	1    3350 3450
 	1    0    0    -1
@@
 F 1 "22p" H 5300 4600 50  0000 L CNN
 F 2 "Capacitor_SMD:C_0402_1005Metric" H 5538 4550 50  0001 C CNN
-F 3 "" H 5500 4700 50  0001 C CNN
-F 4 "C696906" H 5500 4700 50  0001 C CNN "LCSC"
+F 3 "https://datasheet.lcsc.com/lcsc/1809301912_YAGEO-CC0402JRNPO9BN220_C106203.pdf" H 5500 4700 50  0001 C CNN
+F 4 "C106203" H 5500 4700 50  0001 C CNN "LCSC"
 F 5 "" H 5500 4700 50  0001 C CNN "Price"
 F 6 "N" H 5500 4700 50  0001 C CNN "Sponsored"
+F 7 "YAGEO" H 5500 4700 50  0001 C CNN "MANUFACTURER"
+F 8 "CC0402JRNPO9BN220" H 5500 4700 50  0001 C CNN "MPN"
 	1    5500 4700
 	-1   0    0    -1
@@
 F 1 "22p" H 5700 4600 50  0000 L CNN
 F 2 "Capacitor_SMD:C_0402_1005Metric" H 5938 4550 50  0001 C CNN
-F 3 "" H 5900 4700 50  0001 C CNN
-F 4 "C696906" H 5900 4700 50  0001 C CNN "LCSC"
+F 3 "https://datasheet.lcsc.com/lcsc/1809301912_YAGEO-CC0402JRNPO9BN220_C106203.pdf" H 5900 4700 50  0001 C CNN
+F 4 "C106203" H 5900 4700 50  0001 C CNN "LCSC"
 F 5 "" H 5900 4700 50  0001 C CNN "Price"
 F 6 "N" H 5900 4700 50  0001 C CNN "Sponsored"
+F 7 "YAGEO" H 5900 4700 50  0001 C CNN "MANUFACTURER"
+F 8 "CC0402JRNPO9BN220" H 5900 4700 50  0001 C CNN "MPN"
 	1    5900 4700
 	-1   0    0    -1
@@
 AR Path="/5FDA4DDF/5FE17C0C" Ref="R47"  Part="1"
 F 0 "R47" H 3109 3496 50  0000 L CNN
-F 1 "4k7" H 3109 3405 50  0000 L CNN
+F 1 "4.7k" H 3109 3405 50  0000 L CNN
 F 2 "Resistor_SMD:R_0402_1005Metric" H 3050 3450 50  0001 C CNN
 F 3 "~" H 3050 3450 50  0001 C CNN
 F 4 "" H 3050 3450 50  0001 C CNN "Price"
-F 5 "" H 3050 3450 50  0001 C CNN "LCSC"
+F 5 "C25940" H 3050 3450 50  0001 C CNN "LCSC"
 F 6 "-" H 3050 3450 50  0001 C CNN "Mouser"
 F 7 "N" H 3050 3450 50  0001 C CNN "Sponsored"
+F 8 "UNI-ROYAL" H 3050 3450 50  0001 C CNN "MANUFACTURER"
+F 9 "0402WGJ0472TCE" H 3050 3450 50  0001 C CNN "MPN"
 	1    3050 3450
 	1    0    0    -1
