File: rp2040.sch (KiCad schematic (older format))
At the start: 21 parts, among them J8 JTAG, Q3 Q_NMOS_GSD, Y2 12MHz

Commit message: More work on RP2040 integration
Parts:
- removed J8: JTAG, Connector:Tag-Connect_TC2030-IDC-FP_2x03_P1.27mm_Vertical, symbol mch2021-rescue:Conn_02x03_Odd_Even-Connector_Generic
- removed Q3, Q?: Q_NMOS_GSD, Package_TO_SOT_SMD:SOT-23, symbol mch2021-rescue:Q_NMOS_GSD-Device
- removed R24, R25: 10k, Resistor_SMD:R_0402_1005Metric, symbol mch2021-rescue:R-Device
- removed TP14: UNUSED PIN, TestPoint:TestPoint_Pad_1.0x1.0mm, symbol mch2021-rescue:TestPoint-Connector
- added C47, C58, C59, C60, C61, C62, C63, C8: 100n, Capacitor_SMD:C_0402_1005Metric, symbol mch2021-rescue:C-Device
- added C7: 1u, Capacitor_SMD:C_0402_1005Metric, symbol mch2021-rescue:C-Device
- added Q5: Q_NMOS_GSD, Package_TO_SOT_SMD:SOT-23, symbol mch2021-rescue:Q_NMOS_GSD-Device
- added R27: 47, Resistor_SMD:R_0402_1005Metric, symbol mch2021-rescue:R-Device
- added TP14, TP16, TP9: LED OUT, TestPoint:TestPoint_Pad_1.0x1.0mm, symbol mch2021-rescue:TestPoint_Small-Connector
- C11: value 100n -> 1u
- R22: value 47 -> 10k
- U3: renamed from U?; footprint QFN40P700X700X90-57N -> RP2040:QFN40P700X700X90-57N
- gave numbers to parts that had none: 2
Connections:
- net +1V1: now also C58.1, C7.1, C8.1
- net +3V3: now also R22.2, U3.43 (ADC_AVDD), C47.1, C59.1, C60.1, C61.1, C62.1, C63.1
- net GND: now also C47.2, C58.2, C59.2, C60.2, C61.2, C62.2, C63.2, C7.2, C8.2, Q5.2 (S)
- net USB_DET: now also R27.2; no longer R22.2
- net at R22.1: now also U3.35 (GPIO23), Q5.3 (D)
- net EXT_SCL: now reaches U3.28 (GPIO17)
- net SAO2: now reaches U3.18 (GPIO15)
- net EXT_SDA: now reaches U3.27 (GPIO16)
- net at U17.1 (~CS), U3.56 (QSPI_CSN): now also R24.1
- net STM32_BOOT0 renamed RP2040_BOOT
- net STM32_RESET renamed RP2040_RESET
- net RP2040_RESET: now also TP16.1
- net STM32_SWCLK renamed RP2040_SWCLK
- net RP2040_SWCLK: now also TP14.1
- net STM32_SWDIO renamed RP2040_SWDIO
- net RP2040_SWDIO: now also TP9.1
- new net: Q5.1 (G), R27.1
- no-connect marks 1 -> 0
Other:
- note added: "I2C0 SDA\nI2C0 SCL"
- note added: "Place close to chip"
- note added: "Place close\nto pin 44"
- note added: "Place close\nto pin 45"
- note added: "SPI0 SCK\nSPI0 TX\nSPI0 RX\nSPI0 CSn"
- moved on the sheet: C10, C11, C12, C13, C9, R23, R24, R26, R28, R6, R7, U17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

Commit message: More wiring for the RP2040
Parts:
- removed TP16: LED OUT, TestPoint:TestPoint_Pad_1.0x1.0mm, symbol mch2021-rescue:TestPoint_Small-Connector
Connections:
- net BATT_TEMP: now also U3.39 (GPIO27/ADC1); no longer U3.38 (GPIO26/ADC0)
- net CHARGING: now also U3.35 (GPIO23); no longer U3.37 (GPIO25)
- net EXT_SCL: now also U3.12 (GPIO9); no longer U3.28 (GPIO17)
- net EXT_SDA: now also U3.11 (GPIO8); no longer U3.27 (GPIO16)
- net FPGA_RX: now also U3.36 (GPIO24); no longer U3.6 (GPIO4)
- net FPGA_TX: now also U3.37 (GPIO25); no longer U3.7 (GPIO5)
- net LCD_BACKLIGHT: now also U3.18 (GPIO15); no longer U3.11 (GPIO8)
- net LCD_MODE: now also U3.28 (GPIO17); no longer U3.12 (GPIO9)
- net LCD_RESET: now also U3.27 (GPIO16); no longer U3.13 (GPIO10)
- net PWR_LED_ENABLE: now also U3.34 (GPIO22); no longer U3.36 (GPIO24)
- net SAO2: now also U3.13 (GPIO10); no longer U3.18 (GPIO15)
- net SENSE_VBAT: now also U3.40 (GPIO28/ADC2); no longer U3.39 (GPIO27/ADC1)
- net SENSE_VUSB: now also U3.41 (GPIO29/ADC3); no longer U3.40 (GPIO28/ADC2)
- net at Q5.3 (D), R22.1: no longer U3.35 (GPIO23)
Other:
- moved on the sheet: Q5, R22, R27
Changed lines of the file:
@@
 Text HLabel 6450 4150 2    50   Input ~ 0
 SPI_MOSI
-Text HLabel 6450 4550 2    50   Output ~ 0
+Text HLabel 6450 4350 2    50   Output ~ 0
 PWR_LED_ENABLE
-Text HLabel 6450 4850 2    50   Input ~ 0
+Text HLabel 6450 4950 2    50   Input ~ 0
 SENSE_VBAT
-Text HLabel 6450 4950 2    50   Input ~ 0
+Text HLabel 6450 5050 2    50   Input ~ 0
 SENSE_VUSB
 Text HLabel 4000 4250 0    50   BiDi ~ 0
@@
 Text HLabel 4000 4350 0    50   BiDi ~ 0
 SAO_IO1
-Text HLabel 4000 4650 0    50   Output ~ 0
+Text HLabel 6450 3750 2    50   Output ~ 0
 LCD_RESET
-Text HLabel 4000 4550 0    50   Output ~ 0
+Text HLabel 6450 3850 2    50   Output ~ 0
 LCD_MODE
-Text HLabel 4000 4450 0    50   Output ~ 0
+Text HLabel 6450 3650 2    50   Output ~ 0
 LCD_BACKLIGHT
 Wire Wire Line
@@
 	1    0    0    -1
 $EndComp
-Text HLabel 6450 4650 2    50   Input ~ 0
+Text HLabel 6450 4450 2    50   Input ~ 0
 CHARGING
 Text HLabel 4000 3650 0    50   Output ~ 0
@@
 Text HLabel 4000 3750 0    50   Input ~ 0
 ESP32_TX
-Text HLabel 4000 4050 0    50   Output ~ 0
+Text HLabel 6450 4550 2    50   Output ~ 0
 FPGA_RX
-Text HLabel 4000 4150 0    50   Input ~ 0
+Text HLabel 6450 4650 2    50   Input ~ 0
 FPGA_TX
 Text HLabel 4000 5050 0    50   Output ~ 0
@@
 Wire Wire Line
 	3800 2750 3800 2650
-Text HLabel 6450 4750 2    50   Input ~ 0
+Text HLabel 6450 4850 2    50   Input ~ 0
 BATT_TEMP
 $Comp
@@
 Text Notes 4750 3950 0    31   ~ 0
 I2C1 SDA\nI2C1 SCL
-Text Notes 4750 4150 0    31   ~ 0
+Text Notes 5400 4650 0    31   ~ 0
 UART1 TX\nUART1 RX
 Text HLabel 4000 4850 0    50   Output ~ 0
@@
 Text GLabel 1750 7100 2    31   Input ~ 0
 RP2040_SWCLK
-Text GLabel 1750 7200 2    31   Input ~ 0
-RP2040_RESET
 Text GLabel 1750 7000 2    31   Input ~ 0
 RP2040_SWDIO
 Text HLabel 7600 2100 2    50   Input ~ 0
 RP2040_BOOT
-Wire Notes Line
-	7550 2100 7500 2150
-Wire Notes Line
-	7500 2150 7500 2100
 $Comp
 L mch2021-rescue:R-Device R?
@@
 	6200 6750 6600 6750
 Connection ~ 6200 6750
-Text HLabel 8550 4650 2    50   Input ~ 0
+Text HLabel 9550 5350 2    50   Input ~ 0
 USB_DET
 $Comp
 L mch2021-rescue:GND-power #PWR049
 U 1 1 61BCE064
-P 7950 4850
-F 0 "#PWR049" H 7950 4600 50  0001 C CNN
-F 1 "GND" H 7955 4677 50  0000 C CNN
-F 2 "" H 7950 4850 50  0001 C CNN
-F 3 "" H 7950 4850 50  0001 C CNN
-	1    7950 4850
+P 8950 5550
+F 0 "#PWR049" H 8950 5300 50  0001 C CNN
+F 1 "GND" H 8955 5377 50  0000 C CNN
+F 2 "" H 8950 5550 50  0001 C CNN
+F 3 "" H 8950 5550 50  0001 C CNN
+	1    8950 5550
 	1    0    0    -1
 $EndComp
@@
 L mch2021-rescue:+3.3V-power #PWR047
 U 1 1 61BCE06A
-P 7950 4150
-F 0 "#PWR047" H 7950 4000 50  0001 C CNN
-F 1 "+3.3V" H 7965 4323 50  0000 C CNN
-F 2 "" H 7950 4150 50  0001 C CNN
-F 3 "" H 7950 4150 50  0001 C CNN
-	1    7950 4150
+P 8950 4850
+F 0 "#PWR047" H 8950 4700 50  0001 C CNN
+F 1 "+3.3V" H 8965 5023 50  0000 C CNN
+F 2 "" H 8950 4850 50  0001 C CNN
+F 3 "" H 8950 4850 50  0001 C CNN
+	1    8950 4850
 	1    0    0    -1
 $EndComp
@@
 L mch2021-rescue:R-Device R?
 U 1 1 61BCE074
-P 7950 4300
+P 8950 5000
 AR Path="/5DC753C3/61BCE074" Ref="R?"  Part="1"
 AR Path="/61BCE074" Ref="R?"  Part="1"
 AR Path="/5E3BA64A/61BCE074" Ref="R?"  Part="1"
 AR Path="/5F51E414/61BCE074" Ref="R22"  Part="1"
-F 0 "R22" V 8050 4300 50  0000 C CNN
-F 1 "10k" V 7950 4300 50  0000 C CNN
-F 2 "Resistor_SMD:R_0402_1005Metric" V 7880 4300 50  0001 C CNN
-F 3 "~" H 7950 4300 50  0001 C CNN
-F 4 "" H 7950 4300 50  0001 C CNN "LCSC"
-F 5 "" H 7950 4300 50  0001 C CNN "Price"
-F 6 "-" H 7950 4300 50  0001 C CNN "Mouser"
-F 7 "N" H 7950 4300 50  0001 C CNN "Sponsored"
-	1    7950 4300
+F 0 "R22" V 9050 5000 50  0000 C CNN
+F 1 "10k" V 8950 5000 50  0000 C CNN
+F 2 "Resistor_SMD:R_0402_1005Metric" V 8880 5000 50  0001 C CNN
+F 3 "~" H 8950 5000 50  0001 C CNN
+F 4 "" H 8950 5000 50  0001 C CNN "LCSC"
+F 5 "" H 8950 5000 50  0001 C CNN "Price"
+F 6 "-" H 8950 5000 50  0001 C CNN "Mouser"
+F 7 "N" H 8950 5000 50  0001 C CNN "Sponsored"
+	1    8950 5000
 	-1   0    0    1
 $EndComp
@@
 L mch2021-rescue:Q_NMOS_GSD-Device Q?
 U 1 1 61BCE07F
-P 8050 4650
+P 9050 5350
 AR Path="/5FDC6C76/61BCE07F" Ref="Q?"  Part="1"
 AR Path="/5F51E414/61BCE07F" Ref="Q5"  Part="1"
-F 0 "Q5" H 8000 4450 50  0000 C CNN
-F 1 "Q_NMOS_GSD" H 7800 4550 50  0000 C CNN
-F 2 "Package_TO_SOT_SMD:SOT-23" H 8250 4750 50  0001 C CNN
-F 3 "~" H 8050 4650 50  0001 C CNN
-F 4 "C406812" H 8050 4650 50  0001 C CNN "LCSC"
-F 5 "-" H 8050 4650 50  0001 C CNN "Mouser"
-F 6 "" H 8050 4650 50  0001 C CNN "Price"
-F 7 "N" H 8050 4650 50  0001 C CNN "Sponsored"
-	1    8050 4650
+F 0 "Q5" H 9000 5150 50  0000 C CNN
+F 1 "Q_NMOS_GSD" H 8800 5250 50  0000 C CNN
+F 2 "Package_TO_SOT_SMD:SOT-23" H 9250 5450 50  0001 C CNN
+F 3 "~" H 9050 5350 50  0001 C CNN
+F 4 "C406812" H 9050 5350 50  0001 C CNN "LCSC"
+F 5 "-" H 9050 5350 50  0001 C CNN "Mouser"
+F 6 "" H 9050 5350 50  0001 C CNN "Price"
+F 7 "N" H 9050 5350 50  0001 C CNN "Sponsored"
+	1    9050 5350
 	-1   0    0    -1
 $EndComp
@@
 L mch2021-rescue:R-Device R?
 U 1 1 61BCE089
-P 8400 4650
+P 9400 5350
 AR Path="/5DC753C3/61BCE089" Ref="R?"  Part="1"
 AR Path="/61BCE089" Ref="R?"  Part="1"
@@
 AR Path="/5F51E414/61BCE089" Ref="R27"  Part="1"
 AR Path="/5FDC6C76/61BCE089" Ref="R?"  Part="1"
-F 0 "R27" V 8500 4650 50  0000 C CNN
-F 1 "47" V 8400 4650 50  0000 C CNN
-F 2 "Resistor_SMD:R_0402_1005Metric" V 8330 4650 50  0001 C CNN
-F 3 "~" H 8400 4650 50  0001 C CNN
-F 4 "" H 8400 4650 50  0001 C CNN "LCSC"
-F 5 "" H 8400 4650 50  0001 C CNN "Price"
-F 6 "-" H 8400 4650 50  0001 C CNN "Mouser"
-F 7 "N" H 8400 4650 50  0001 C CNN "Sponsored"
-	1    8400 4650
+F 0 "R27" V 9500 5350 50  0000 C CNN
+F 1 "47" V 9400 5350 50  0000 C CNN
+F 2 "Resistor_SMD:R_0402_1005Metric" V 9330 5350 50  0001 C CNN
+F 3 "~" H 9400 5350 50  0001 C CNN
+F 4 "" H 9400 5350 50  0001 C CNN "LCSC"
+F 5 "" H 9400 5350 50  0001 C CNN "Price"
+F 6 "-" H 9400 5350 50  0001 C CNN "Mouser"
+F 7 "N" H 9400 5350 50  0001 C CNN "Sponsored"
+	1    9400 5350
 	0    -1   -1   0
 $EndComp
-Connection ~ 7950 4450
-Wire Wire Line
-	6100 4450 7950 4450
-Text GLabel 6450 3750 2    39   BiDi ~ 0
+Text GLabel 4000 4450 0    39   BiDi ~ 0
 EXT_SDA
-Text GLabel 6450 3850 2    39   Input ~ 0
+Text GLabel 4000 4550 0    39   Input ~ 0
 EXT_SCL
 Wire Wire Line
@@
 Text Notes 5400 4200 0    31   ~ 0
 SPI0 SCK\nSPI0 TX\nSPI0 RX\nSPI0 CSn
-Text GLabel 6450 3650 2    39   BiDi ~ 0
+Text GLabel 4000 4650 0    39   BiDi ~ 0
 SAO2
 Wire Wire Line
@@
 	1    0    0    -1
 $EndComp
-$Comp
-L mch2021-rescue:TestPoint_Small-Connector TP?
-U 1 1 61E69B38
-P 1650 7200
-AR Path="/61E69B38" Ref="TP?"  Part="1"
-AR Path="/5F51E414/61E69B38" Ref="TP16"  Part="1"
-F 0 "TP16" H 1450 7200 50  0000 L CNN
-F 1 "LED OUT" H 1698 7155 50  0001 L CNN
-F 2 "TestPoint:TestPoint_Pad_1.0x1.0mm" H 1850 7200 50  0001 C CNN
-F 3 "~" H 1850 7200 50  0001 C CNN
-	1    1650 7200
-	1    0    0    -1
-$EndComp
 Wire Wire Line
 	1750 7000 1650 7000
@@
 	1650 7100 1750 7100
 Wire Wire Line
-	1750 7200 1650 7200
+	6450 4450 6100 4450
+Wire Wire Line
+	6100 4350 6450 4350
+Wire Wire Line
+	6450 5050 6100 5050
 $EndSCHEMATC

Commit message: Add flash chip footprint, fix routing of flash chip, fix DRC errors
Parts:
- removed C12, C47: 100n, Capacitor_SMD:C_0402_1005Metric, symbol mch2021-rescue:C-Device
- U17: value SPIFLASH_QSPI-spiflash -> W25Q128JVS; footprint (none) -> Package_SO:SOIC-8_5.23x5.23mm_P1.27mm
Connections:
- net RP_XIN: now reaches C10.1, U3.20 (XIN), Y2.1
- net RP_XOUT: now reaches C9.1, U3.21 (XOUT), Y2.3
- net at U3.38 (GPIO26/ADC0): now also Q5.3 (D), R22.1
- net RP_QSPI_SD3: now reaches U17.7 (IO3), U3.51 (QSPI_SD3)
- net RP_QSPI_SCLK: now reaches U17.6 (SCK), U3.52 (QSPI_SCLK)
- net RP_QSPI_SD0: now reaches U17.5 (MOSI/IO0), U3.53 (QSPI_SD0)
- net RP_QSPI_SD2: now reaches U17.3 (IO2), U3.54 (QSPI_SD2)
- net RP_QSPI_SD1: now reaches U17.2 (MISO/IO1), U3.55 (QSPI_SD1)
- net RP_QSPI_CSN: now reaches R24.1, U17.1 (~CS), U3.56 (QSPI_CSN)
Other:
- moved on the sheet: C59, C60, C61, C62, C63, Q5, R22, R27

Commit message: Add oscillator for ICE40, add testpoints for unused RP2040 pins
Parts:
- added TP16: 4, TestPoint:TestPoint_Pad_1.0x1.0mm, symbol mch2021-rescue:TestPoint_Small-Connector
- added TP17: 5, TestPoint:TestPoint_Pad_1.0x1.0mm, symbol mch2021-rescue:TestPoint_Small-Connector
- added TP25: 10, TestPoint:TestPoint_Pad_1.0x1.0mm, symbol mch2021-rescue:TestPoint_Small-Connector
- TP14: value LED OUT -> SWDCLK
- TP9: value LED OUT -> SWDIO
Connections:
- net at U3.6 (GPIO4): now also TP16.1
- net at U3.7 (GPIO5): now also TP17.1
- net SAO2: no longer names the net of U3.13 (GPIO10)
- net SAO2: now also TP25.1
Changed lines of the file:
@@
 Text Notes 5400 4200 0    31   ~ 0
 SPI0 SCK\nSPI0 TX\nSPI0 RX\nSPI0 CSn
-Text GLabel 4000 4650 0    39   BiDi ~ 0
-SAO2
 Wire Wire Line
 	6100 3650 6450 3650
@@
 AR Path="/5F51E414/61E64B18" Ref="TP9"  Part="1"
 F 0 "TP9" H 1450 7000 50  0000 L CNN
-F 1 "LED OUT" H 1698 6955 50  0001 L CNN
+F 1 "SWDIO" H 1698 6955 50  0001 L CNN
 F 2 "TestPoint:TestPoint_Pad_1.0x1.0mm" H 1850 7000 50  0001 C CNN
 F 3 "~" H 1850 7000 50  0001 C CNN
@@
 AR Path="/5F51E414/61E6991E" Ref="TP14"  Part="1"
 F 0 "TP14" H 1450 7100 50  0000 L CNN
-F 1 "LED OUT" H 1698 7055 50  0001 L CNN
+F 1 "SWDCLK" H 1698 7055 50  0001 L CNN
 F 2 "TestPoint:TestPoint_Pad_1.0x1.0mm" H 1850 7100 50  0001 C CNN
 F 3 "~" H 1850 7100 50  0001 C CNN
@@
 Wire Wire Line
 	3800 6750 4150 6750
+Wire Wire Line
+	4300 4050 4000 4050
+$Comp
+L mch2021-rescue:TestPoint_Small-Connector TP?
+U 1 1 61D160CB
+P 4000 4050
+AR Path="/61D160CB" Ref="TP?"  Part="1"
+AR Path="/5F51E414/61D160CB" Ref="TP16"  Part="1"
+F 0 "TP16" H 3800 4050 50  0000 L CNN
+F 1 "4" H 4048 4005 50  0001 L CNN
+F 2 "TestPoint:TestPoint_Pad_1.0x1.0mm" H 4200 4050 50  0001 C CNN
+F 3 "~" H 4200 4050 50  0001 C CNN
+	1    4000 4050
+	1    0    0    -1
+$EndComp
+$Comp
+L mch2021-rescue:TestPoint_Small-Connector TP?
+U 1 1 61D17B0D
+P 4000 4150
+AR Path="/61D17B0D" Ref="TP?"  Part="1"
+AR Path="/5F51E414/61D17B0D" Ref="TP17"  Part="1"
+F 0 "TP17" H 3800 4150 50  0000 L CNN
+F 1 "5" H 4048 4105 50  0001 L CNN
+F 2 "TestPoint:TestPoint_Pad_1.0x1.0mm" H 4200 4150 50  0001 C CNN
+F 3 "~" H 4200 4150 50  0001 C CNN
+	1    4000 4150
+	1    0    0    -1
+$EndComp
+$Comp
+L mch2021-rescue:TestPoint_Small-Connector TP?
+U 1 1 61E0DD7B
+P 4000 4650
+AR Path="/61E0DD7B" Ref="TP?"  Part="1"
+AR Path="/5F51E414/61E0DD7B" Ref="TP25"  Part="1"
+F 0 "TP25" H 3800 4650 50  0000 L CNN
+F 1 "10" H 4048 4605 50  0001 L CNN
+F 2 "TestPoint:TestPoint_Pad_1.0x1.0mm" H 4200 4650 50  0001 C CNN
+F 3 "~" H 4200 4650 50  0001 C CNN
+	1    4000 4650
+	1    0    0    -1
+$EndComp
 $EndSCHEMATC

Commit message: Add 1k resistor for RP2040 crystal, add schematic PDF
Parts:
- added R?: 1k, Resistor_SMD:R_0402_1005Metric, symbol mch2021-rescue:R-Device
Connections:
- net RP_XOUT: now also R?.2; no longer C9.1, Y2.3
- new net: C9.1, R?.1, Y2.3
Other:
- moved on the sheet: C10, C9, Y2
Changed lines of the file:
@@
 encoding utf-8
 Sheet 3 9
-Title "MCH2021 badge - RP2040 microcontroller"
-Date "2021-11-14"
-Rev "3"
+Title "MCH2022 badge - RP2040 microcontroller"
+Date "2021-12-19"
+Rev "3.1415"
 Comp "BADGE.TEAM"
 Comment1 ""
@@
 L mch2021-rescue:C-Device C?
 U 1 1 5E3EFF6B
-P 3100 3200
+P 2500 3200
 AR Path="/5DC753C3/5E3EFF6B" Ref="C?"  Part="1"
 AR Path="/5E3EFF6B" Ref="C?"  Part="1"
 AR Path="/5E3BA64A/5E3EFF6B" Ref="C?"  Part="1"
 AR Path="/5F51E414/5E3EFF6B" Ref="C10"  Part="1"
-F 0 "C10" H 3100 3300 50  0000 L CNN
-F 1 "22p" H 3100 3100 50  0000 L CNN
-F 2 "Capacitor_SMD:C_0402_1005Metric" H 3138 3050 50  0001 C CNN
-F 3 "" H 3100 3200 50  0001 C CNN
-F 4 "C696906" H 3100 3200 50  0001 C CNN "LCSC"
-F 5 "" H 3100 3200 50  0001 C CNN "Price"
-F 6 "N" H 3100 3200 50  0001 C CNN "Sponsored"
-	1    3100 3200
+F 0 "C10" H 2500 3300 50  0000 L CNN
+F 1 "22p" H 2500 3100 50  0000 L CNN
+F 2 "Capacitor_SMD:C_0402_1005Metric" H 2538 3050 50  0001 C CNN
+F 3 "" H 2500 3200 50  0001 C CNN
+F 4 "C696906" H 2500 3200 50  0001 C CNN "LCSC"
+F 5 "" H 2500 3200 50  0001 C CNN "Price"
+F 6 "N" H 2500 3200 50  0001 C CNN "Sponsored"
+	1    2500 3200
 	0    1    1    0
 $EndComp
@@
 L mch2021-rescue:C-Device C?
 U 1 1 5E3F1F93
-P 3100 3400
+P 2500 3400
 AR Path="/5DC753C3/5E3F1F93" Ref="C?"  Part="1"
 AR Path="/5E3F1F93" Ref="C?"  Part="1"
 AR Path="/5E3BA64A/5E3F1F93" Ref="C?"  Part="1"
 AR Path="/5F51E414/5E3F1F93" Ref="C9"  Part="1"
-F 0 "C9" H 2950 3500 50  0000 L CNN
-F 1 "22p" H 2900 3300 50  0000 L CNN
-F 2 "Capacitor_SMD:C_0402_1005Metric" H 3138 3250 50  0001 C CNN
-F 3 "" H 3100 3400 50  0001 C CNN
-F 4 "C696906" H 3100 3400 50  0001 C CNN "LCSC"
-F 5 "" H 3100 3400 50  0001 C CNN "Price"
-F 6 "N" H 3100 3400 50  0001 C CNN "Sponsored"
-	1    3100 3400
+F 0 "C9" H 2350 3500 50  0000 L CNN
+F 1 "22p" H 2300 3300 50  0000 L CNN
+F 2 "Capacitor_SMD:C_0402_1005Metric" H 2538 3250 50  0001 C CNN
+F 3 "" H 2500 3400 50  0001 C CNN
+F 4 "C696906" H 2500 3400 50  0001 C CNN "LCSC"
+F 5 "" H 2500 3400 50  0001 C CNN "Price"
+F 6 "N" H 2500 3400 50  0001 C CNN "Sponsored"
+	1    2500 3400
 	0    1    -1   0
 $EndComp
@@
 L mch2021-rescue:Crystal_GND24_Small-Device Y2
 U 1 1 5E3ED918
-P 3450 3300
-F 0 "Y2" V 3400 3450 50  0000 L CNN
-F 1 "12MHz" V 3500 3450 50  0000 L CNN
-F 2 "Crystal:Crystal_SMD_3225-4Pin_3.2x2.5mm" H 3450 3300 50  0001 C CNN
-F 3 "~" H 3450 3300 50  0001 C CNN
-F 4 "C13738" H 3450 3300 50  0001 C CNN "LCSC"
-F 5 "" H 3450 3300 50  0001 C CNN "Price"
-F 6 "-" H 3450 3300 50  0001 C CNN "Mouser"
-F 7 "N" H 3450 3300 50  0001 C CNN "Sponsored"
-	1    3450 3300
+P 2850 3300
+F 0 "Y2" V 2800 3450 50  0000 L CNN
+F 1 "12MHz" V 2900 3450 50  0000 L CNN
+F 2 "Crystal:Crystal_SMD_3225-4Pin_3.2x2.5mm" H 2850 3300 50  0001 C CNN
+F 3 "~" H 2850 3300 50  0001 C CNN
+F 4 "C13738" H 2850 3300 50  0001 C CNN "LCSC"
+F 5 "" H 2850 3300 50  0001 C CNN "Price"
+F 6 "-" H 2850 3300 50  0001 C CNN "Mouser"
+F 7 "N" H 2850 3300 50  0001 C CNN "Sponsored"
+	1    2850 3300
 	0    1    1    0
 $EndComp
@@
 L mch2021-rescue:GND-power #PWR051
 U 1 1 5F916F4B
-P 2850 3700
-F 0 "#PWR051" H 2850 3450 50  0001 C CNN
-F 1 "GND" H 2855 3527 50  0000 C CNN
-F 2 "" H 2850 3700 50  0001 C CNN
-F 3 "" H 2850 3700 50  0001 C CNN
-	1    2850 3700
+P 2250 3700
+F 0 "#PWR051" H 2250 3450 50  0001 C CNN
+F 1 "GND" H 2255 3527 50  0000 C CNN
+F 2 "" H 2250 3700 50  0001 C CNN
+F 3 "" H 2250 3700 50  0001 C CNN
+	1    2250 3700
 	1    0    0    -1
 $EndComp
@@
 	6100 4850 6450 4850
 Wire Wire Line
-	3450 3400 3250 3400
-Connection ~ 3450 3400
-Wire Wire Line
-	3450 3200 3250 3200
-Connection ~ 3450 3200
+	2850 3400 2650 3400
+Wire Wire Line
+	2850 3200 2650 3200
+Connection ~ 2850 3200
 Wire Wire Line
 	4300 3400 4300 3350
 Wire Wire Line
-	3450 3400 4300 3400
-Wire Wire Line
 	4300 3200 4300 3250
 Wire Wire Line
-	3450 3200 4300 3200
-Wire Wire Line
-	2850 3700 2850 3650
-Wire Wire Line
-	2850 3200 2950 3200
-Wire Wire Line
-	2950 3400 2850 3400
-Connection ~ 2850 3400
-Wire Wire Line
-	2850 3400 2850 3200
-Connection ~ 2850 3650
-Wire Wire Line
-	2850 3650 2850 3400
+	2250 3700 2250 3650
+Wire Wire Line
+	2250 3200 2350 3200
+Wire Wire Line
+	2350 3400 2250 3400
+Connection ~ 2250 3400
+Wire Wire Line
+	2250 3400 2250 3200
+Connection ~ 2250 3650
+Wire Wire Line
+	2250 3650 2250 3400
 Wire Wire Line
 	7150 4250 7050 4250
@@
 $EndComp
 Wire Wire Line
-	3550 3300 3550 3650
-Wire Wire Line
-	3350 3650 3350 3300
-Connection ~ 3350 3650
-Wire Wire Line
-	3350 3650 3550 3650
-Wire Wire Line
-	2850 3650 3350 3650
+	2950 3300 2950 3650
+Wire Wire Line
+	2750 3650 2750 3300
+Connection ~ 2750 3650
+Wire Wire Line
+	2750 3650 2950 3650
+Wire Wire Line
+	2250 3650 2750 3650
 Wire Wire Line
 	4000 3650 4300 3650
@@
 	1    0    0    -1
 $EndComp
+Wire Wire Line
+	2850 3200 4300 3200
+$Comp
+L mch2021-rescue:R-Device R?
+U 1 1 61C35D5C
+P 3650 3400
+AR Path="/5DC753C3/61C35D5C" Ref="R?"  Part="1"
+AR Path="/61C35D5C" Ref="R?"  Part="1"
+AR Path="/5E3BA64A/61C35D5C" Ref="R?"  Part="1"
+AR Path="/5F51E414/61C35D5C" Ref="R?"  Part="1"
+AR Path="/5FDC6C76/61C35D5C" Ref="R?"  Part="1"
+F 0 "R?" V 3550 3400 50  0000 C CNN
+F 1 "1k" V 3650 3400 50  0000 C CNN
+F 2 "Resistor_SMD:R_0402_1005Metric" V 3580 3400 50  0001 C CNN
+F 3 "~" H 3650 3400 50  0001 C CNN
+F 4 "" H 3650 3400 50  0001 C CNN "LCSC"
+F 5 "" H 3650 3400 50  0001 C CNN "Price"
+F 6 "-" H 3650 3400 50  0001 C CNN "Mouser"
+F 7 "N" H 3650 3400 50  0001 C CNN "Sponsored"
+	1    3650 3400
+	0    -1   1    0
+$EndComp
+Wire Wire Line
+	3800 3400 4300 3400
+Wire Wire Line
+	3500 3400 2850 3400
+Connection ~ 2850 3400
 $EndSCHEMATC

Commit message: Cleanup
Parts:
- gave numbers to parts that had none: 1
Changed lines of the file:
@@
 AR Path="/61C35D5C" Ref="R?"  Part="1"
 AR Path="/5E3BA64A/61C35D5C" Ref="R?"  Part="1"
-AR Path="/5F51E414/61C35D5C" Ref="R?"  Part="1"
+AR Path="/5F51E414/61C35D5C" Ref="R25"  Part="1"
 AR Path="/5FDC6C76/61C35D5C" Ref="R?"  Part="1"
-F 0 "R?" V 3550 3400 50  0000 C CNN
+F 0 "R25" V 3550 3400 50  0000 C CNN
 F 1 "1k" V 3650 3400 50  0000 C CNN
 F 2 "Resistor_SMD:R_0402_1005Metric" V 3580 3400 50  0001 C CNN
