File: rp2040.sch (KiCad schematic (older format))
At the start: 30 parts, among them Q5 Q_NMOS_GSD, U17 W25Q128JVS, U3 RP2040, Y2 12MHz

Commit message: Last fixes before ordering
Parts:
- C10, C9: LCSC C696906 -> C106203; MANUFACTURER (none) -> YAGEO; MPN (none) -> CC0402JRNPO9BN220
- Q5: MANUFACTURER (none) -> ALLPOWER; MPN (none) -> AP2302B
- R22, R26: LCSC (none) -> C144807; MANUFACTURER (none) -> YAGEO; MPN (none) -> AC0402FR-0710KL
- R23, R24, R27: LCSC (none) -> C25168; MANUFACTURER (none) -> UNI-ROYAL; MPN (none) -> 0402WGJ0470TCE
- R25: LCSC (none) -> C226166; MANUFACTURER (none) -> FH; MPN (none) -> RC-02W1001FT
- R28: LCSC (none) -> C258090; MANUFACTURER (none) -> FH; MPN (none) -> RC-02W1003FT
- R6, R7: LCSC C103086 -> C203147; MANUFACTURER (none) -> BOURNS; MPN (none) -> CR0402-JW-270GLF
- U17: LCSC (none) -> C97521; MPN (none) -> W25Q128JVSIQ; Manufacturer (none) -> Winbond Elec
- U3: LCSC (none) -> C2040; MPN (none) -> RP2040; Manufacturer (none) -> Raspberry Pi; Sponsored (none) -> Y
Changed lines of the file:
@@
 F 1 "22p" H 2500 3100 50  0000 L CNN
 F 2 "Capacitor_SMD:C_0402_1005Metric" H 2538 3050 50  0001 C CNN
-F 3 "" H 2500 3200 50  0001 C CNN
-F 4 "C696906" H 2500 3200 50  0001 C CNN "LCSC"
+F 3 "https://datasheet.lcsc.com/lcsc/1809301912_YAGEO-CC0402JRNPO9BN220_C106203.pdf" H 2500 3200 50  0001 C CNN
+F 4 "C106203" H 2500 3200 50  0001 C CNN "LCSC"
 F 5 "" H 2500 3200 50  0001 C CNN "Price"
 F 6 "N" H 2500 3200 50  0001 C CNN "Sponsored"
+F 7 "YAGEO" H 2500 3200 50  0001 C CNN "MANUFACTURER"
+F 8 "CC0402JRNPO9BN220" H 2500 3200 50  0001 C CNN "MPN"
 	1    2500 3200
 	0    1    1    0
@@
 F 1 "22p" H 2300 3300 50  0000 L CNN
 F 2 "Capacitor_SMD:C_0402_1005Metric" H 2538 3250 50  0001 C CNN
-F 3 "" H 2500 3400 50  0001 C CNN
-F 4 "C696906" H 2500 3400 50  0001 C CNN "LCSC"
+F 3 "https://datasheet.lcsc.com/lcsc/1809301912_YAGEO-CC0402JRNPO9BN220_C106203.pdf" H 2500 3400 50  0001 C CNN
+F 4 "C106203" H 2500 3400 50  0001 C CNN "LCSC"
 F 5 "" H 2500 3400 50  0001 C CNN "Price"
 F 6 "N" H 2500 3400 50  0001 C CNN "Sponsored"
+F 7 "YAGEO" H 2500 3400 50  0001 C CNN "MANUFACTURER"
+F 8 "CC0402JRNPO9BN220" H 2500 3400 50  0001 C CNN "MPN"
 	1    2500 3400
 	0    1    -1   0
@@
 F 2 "Resistor_SMD:R_0402_1005Metric" V 3980 2450 50  0001 C CNN
 F 3 "~" H 4050 2450 50  0001 C CNN
-F 4 "" H 4050 2450 50  0001 C CNN "LCSC"
+F 4 "C144807" H 4050 2450 50  0001 C CNN "LCSC"
 F 5 "" H 4050 2450 50  0001 C CNN "Price"
 F 6 "-" H 4050 2450 50  0001 C CNN "Mouser"
 F 7 "N" H 4050 2450 50  0001 C CNN "Sponsored"
+F 8 "YAGEO" H 4050 2450 50  0001 C CNN "MANUFACTURER"
+F 9 "AC0402FR-0710KL" H 4050 2450 50  0001 C CNN "MPN"
 	1    4050 2450
 	1    0    0    -1
@@
 F 2 "Resistor_SMD:R_0402_1005Metric" V 6980 4050 50  0001 C CNN
 F 3 "~" H 7050 4050 50  0001 C CNN
-F 4 "" H 7050 4050 50  0001 C CNN "LCSC"
+F 4 "C258090" H 7050 4050 50  0001 C CNN "LCSC"
 F 5 "" H 7050 4050 50  0001 C CNN "Price"
 F 6 "-" H 7050 4050 50  0001 C CNN "Mouser"
 F 7 "N" H 7050 4050 50  0001 C CNN "Sponsored"
+F 8 "FH" H 7050 4050 50  0001 C CNN "MANUFACTURER"
+F 9 "RC-02W1003FT" H 7050 4050 50  0001 C CNN "MPN"
 	1    7050 4050
 	1    0    0    -1
@@
 F 3 "~" H 6200 3350 50  0001 C CNN
 F 4 "" H 6200 3350 50  0001 C CNN "Price"
-F 5 "C103086" H 6200 3350 50  0001 C CNN "LCSC"
+F 5 "C203147" H 6200 3350 50  0001 C CNN "LCSC"
 F 6 "-" H 6200 3350 50  0001 C CNN "Mouser"
 F 7 "N" H 6200 3350 50  0001 C CNN "Sponsored"
+F 8 "BOURNS" H 6200 3350 50  0001 C CNN "MANUFACTURER"
+F 9 "CR0402-JW-270GLF" H 6200 3350 50  0001 C CNN "MPN"
 	1    6200 3350
 	0    1    1    0
@@
 F 6 "IPC 7351B" H 5200 3750 50  0001 L BNN "STANDARD"
 F 7 "Raspberry Pi" H 5200 3750 50  0001 L BNN "MANUFACTURER"
+F 8 "C2040" H 5200 3750 50  0001 C CNN "LCSC"
+F 9 "RP2040" H 5200 3750 50  0001 C CNN "MPN"
+F 10 "Raspberry Pi" H 5200 3750 50  0001 C CNN "Manufacturer"
+F 11 "Y" H 5200 3750 50  0001 C CNN "Sponsored"
 	1    5200 3750
 	1    0    0    -1
@@
 F 3 "~" H 6200 3450 50  0001 C CNN
 F 4 "" H 6200 3450 50  0001 C CNN "Price"
-F 5 "C103086" H 6200 3450 50  0001 C CNN "LCSC"
+F 5 "C203147" H 6200 3450 50  0001 C CNN "LCSC"
 F 6 "-" H 6200 3450 50  0001 C CNN "Mouser"
 F 7 "N" H 6200 3450 50  0001 C CNN "Sponsored"
+F 8 "BOURNS" H 6200 3450 50  0001 C CNN "MANUFACTURER"
+F 9 "CR0402-JW-270GLF" H 6200 3450 50  0001 C CNN "MPN"
 	1    6200 3450
 	0    -1   -1   0
@@
 F 2 "Package_SO:SOIC-8_5.23x5.23mm_P1.27mm" H 7950 1950 60  0001 C CNN
 F 3 "" H 7950 1950 60  0001 C CNN
+F 4 "C97521" H 7900 2800 50  0001 C CNN "LCSC"
+F 5 "W25Q128JVSIQ" H 7900 2800 50  0001 C CNN "MPN"
+F 6 "Winbond Elec" H 7900 2800 50  0001 C CNN "Manufacturer"
 	1    7900 2800
 	1    0    0    -1
@@
 F 2 "Resistor_SMD:R_0402_1005Metric" V 4080 4850 50  0001 C CNN
 F 3 "~" H 4150 4850 50  0001 C CNN
-F 4 "" H 4150 4850 50  0001 C CNN "LCSC"
+F 4 "C25168" H 4150 4850 50  0001 C CNN "LCSC"
 F 5 "" H 4150 4850 50  0001 C CNN "Price"
 F 6 "-" H 4150 4850 50  0001 C CNN "Mouser"
 F 7 "N" H 4150 4850 50  0001 C CNN "Sponsored"
+F 8 "UNI-ROYAL" H 4150 4850 50  0001 C CNN "MANUFACTURER"
+F 9 "0402WGJ0470TCE" H 4150 4850 50  0001 C CNN "MPN"
 	1    4150 4850
 	0    -1   -1   0
@@
 F 2 "Resistor_SMD:R_0402_1005Metric" V 7130 2100 50  0001 C CNN
 F 3 "~" H 7200 2100 50  0001 C CNN
-F 4 "" H 7200 2100 50  0001 C CNN "LCSC"
+F 4 "C25168" H 7200 2100 50  0001 C CNN "LCSC"
 F 5 "" H 7200 2100 50  0001 C CNN "Price"
 F 6 "-" H 7200 2100 50  0001 C CNN "Mouser"
 F 7 "N" H 7200 2100 50  0001 C CNN "Sponsored"
+F 8 "UNI-ROYAL" H 7200 2100 50  0001 C CNN "MANUFACTURER"
+F 9 "0402WGJ0470TCE" H 7200 2100 50  0001 C CNN "MPN"
 	1    7200 2100
 	0    -1   1    0
@@
 F 2 "Resistor_SMD:R_0402_1005Metric" V 7980 4600 50  0001 C CNN
 F 3 "~" H 8050 4600 50  0001 C CNN
-F 4 "" H 8050 4600 50  0001 C CNN "LCSC"
+F 4 "C144807" H 8050 4600 50  0001 C CNN "LCSC"
 F 5 "" H 8050 4600 50  0001 C CNN "Price"
 F 6 "-" H 8050 4600 50  0001 C CNN "Mouser"
 F 7 "N" H 8050 4600 50  0001 C CNN "Sponsored"
+F 8 "YAGEO" H 8050 4600 50  0001 C CNN "MANUFACTURER"
+F 9 "AC0402FR-0710KL" H 8050 4600 50  0001 C CNN "MPN"
 	1    8050 4600
 	-1   0    0    1
@@
 F 6 "" H 8150 4950 50  0001 C CNN "Price"
 F 7 "N" H 8150 4950 50  0001 C CNN "Sponsored"
+F 8 "ALLPOWER" H 8150 4950 50  0001 C CNN "MANUFACTURER"
+F 9 "AP2302B" H 8150 4950 50  0001 C CNN "MPN"
 	1    8150 4950
 	-1   0    0    -1
@@
 F 2 "Resistor_SMD:R_0402_1005Metric" V 8430 4950 50  0001 C CNN
 F 3 "~" H 8500 4950 50  0001 C CNN
-F 4 "" H 8500 4950 50  0001 C CNN "LCSC"
+F 4 "C25168" H 8500 4950 50  0001 C CNN "LCSC"
 F 5 "" H 8500 4950 50  0001 C CNN "Price"
 F 6 "-" H 8500 4950 50  0001 C CNN "Mouser"
 F 7 "N" H 8500 4950 50  0001 C CNN "Sponsored"
+F 8 "UNI-ROYAL" H 8500 4950 50  0001 C CNN "MANUFACTURER"
+F 9 "0402WGJ0470TCE" H 8500 4950 50  0001 C CNN "MPN"
 	1    8500 4950
 	0    -1   -1   0
@@
 F 2 "Resistor_SMD:R_0402_1005Metric" V 3580 3400 50  0001 C CNN
 F 3 "~" H 3650 3400 50  0001 C CNN
-F 4 "" H 3650 3400 50  0001 C CNN "LCSC"
+F 4 "C226166" H 3650 3400 50  0001 C CNN "LCSC"
 F 5 "" H 3650 3400 50  0001 C CNN "Price"
 F 6 "-" H 3650 3400 50  0001 C CNN "Mouser"
 F 7 "N" H 3650 3400 50  0001 C CNN "Sponsored"
+F 8 "FH" H 3650 3400 50  0001 C CNN "MANUFACTURER"
+F 9 "RC-02W1001FT" H 3650 3400 50  0001 C CNN "MPN"
 	1    3650 3400
 	0    -1   1    0
