File: audio.kicad_sch (KiCad schematic)
At the start: 25 parts, among them J1 AudioJack3, U1 PCM5100, U18 TDA2822

Commit message: Fixed graphics and names
Other:
- company: (none) -> BADGE.TEAM
- title: (none) -> MCH2022 badge - Audio
Changed lines of the file:
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@@
 (kicad_sch (version 20211123) (generator eeschema)
   (paper "A4")
+  (title_block
+    (title "MCH2022 badge - Audio")
+    (date "2022-02-05")
+    (rev "3.1415")
+    (company "BADGE.TEAM")
+  )
   (junction (at 113.03 113.03) (diameter 0) (color 0 0 0 0)
   )
