File: audio.kicad_sch (KiCad schematic)
At the start: 33 parts, among them J1 AudioJack3, U1 CS4344-CZZ

Commit message: Finishing touches for audio circuit
Parts:
- removed C5, C6: 10u, Capacitor_SMD:C_0402_1005Metric, symbol Device:C_Polarized_Small
- added C5, C53, C55, C57, C6, C64, C67: 47u, Capacitor_SMD:C_0805_2012Metric, symbol Device:C_Small
- added C56: 100n, Capacitor_SMD:C_0603_1608Metric, symbol Device:C_Small
- added D8: 1N4148WS, Diode_SMD:D_SOD-323, symbol Diode:1N4148WS
- added R51: 100k, Resistor_SMD:R_0402_1005Metric, symbol mch2021-rescue:R-Device
- C52, C54, C65, C66: renamed from C?; value 100u -> 47u; footprint Capacitor_SMD:C_0402_1005Metric -> Capacitor_SMD:C_0805_2012Metric
- gave numbers to parts that had none: 7
Connections:
- net +3V3: now also R51.2
- net GND: now also C5.2, C53.1, C55.1, C56.1, C57.1, C6.2, D8.2 (A)
- net SPK_DISABLED: now also R51.1
- net VIN: now also C56.2, C57.2
- net at C68.2, J1.R: now also C66.1, C67.2; no longer C66.2
- net at C65.2, C69.2, J1.T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: now also C64.1
- net at LS1.1, SW8.2 (B): now also D8.1 (K)
- net at C65.1, U4.1: now also C64.2
- net at C52.2, U4.8 (-): now also C53.2
- net at C4.1, U1.5 (VQ): now also C6.1
- net at U1.6 (FILT+): now also C5.1
- net at U4.3: now also C66.2, C67.1; no longer C66.1
- net at C54.2, U4.5 (-): now also C55.2
Other:
- moved on the sheet: C1, C14, C2, C3, C33, C4, C54, C66, C68, C69, LS1, R27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

Commit message: Add some footprints
Parts:
- LS1: footprint (none) -> Connector_Molex:Molex_PicoBlade_53261-0271_1x02-1MP_P1.25mm_Horizontal
- U1: value CS4344-CZZ -> MS4344; AVAILABILITY Unavailable -> (none); DESCRIPTION D/A converter; 24bit; 192ksps; Channels: 2; 3÷5.25VDC; T -> (none); LCSC (none) -> C1509050; MF Cirrus Logic -> (none); MP CS4344-CZZ -> (none); PACKAGE TSSOP-10 Cirrus Logic -> (none); PARTREV F2 -> (none); PRICE None -> (none); STANDARD IPC-7351B -> (none)
- U4: value TDA2822 -> D2822M; footprint (none) -> Package_SO:SOP-8_3.9x4.9mm_P1.27mm
- U4: value TDA2822 -> D2822M; footprint (none) -> Package_SO:SOP-8_3.9x4.9mm_P1.27mm; LCSC (none) -> C2837292
Changed lines of the file:
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@@
     (in_bom yes) (on_board yes) (fields_autoplaced)
     (property "Reference" "U4" (id 0) (at 184.15 54.61 0))
-    (property "Value" "TDA2822" (id 1) (at 184.15 57.15 0))
-    (property "Footprint" "" (id 2) (at 184.15 64.77 0)
-      (effects (font (size 1.27 1.27)) hide)
-    )
-    (property "Datasheet" "~" (id 3) (at 184.15 64.77 0)
+    (property "Value" "D2822M" (id 1) (at 184.15 57.15 0))
+    (property "Footprint" "Package_SO:SOP-8_3.9x4.9mm_P1.27mm" (id 2) (at 184.15 64.77 0)
+      (effects (font (size 1.27 1.27)) hide)
+    )
+    (property "Datasheet" "https://datasheet.lcsc.com/lcsc/2111030930_Silicore-D2822M-SOP8_C2837292.pdf" (id 3) (at 184.15 64.77 0)
       (effects (font (size 1.27 1.27)) hide)
     )
@@
     (in_bom yes) (on_board yes) (fields_autoplaced)
     (property "Reference" "U1" (id 0) (at 71.12 77.47 0))
-    (property "Value" "CS4344-CZZ" (id 1) (at 71.12 80.01 0))
+    (property "Value" "MS4344" (id 1) (at 71.12 80.01 0))
     (property "Footprint" "CS4344-CZZ:SOP50P490X110-10N" (id 2) (at 71.12 95.25 0)
       (effects (font (size 1.27 1.27)) (justify left bottom) hide)
     )
-    (property "Datasheet" "" (id 3) (at 71.12 95.25 0)
+    (property "Datasheet" "https://datasheet.lcsc.com/lcsc/2012211837_Hangzhou-Ruimeng-Tech-MS4344_C1509050.pdf" (id 3) (at 71.12 95.25 0)
       (effects (font (size 1.27 1.27)) (justify left bottom) hide)
     )
-    (property "STANDARD" "IPC-7351B" (id 4) (at 71.12 95.25 0)
-      (effects (font (size 1.27 1.27)) (justify left bottom) hide)
-    )
-    (property "PARTREV" "F2" (id 5) (at 71.12 95.25 0)
-      (effects (font (size 1.27 1.27)) (justify left bottom) hide)
-    )
-    (property "MP" "CS4344-CZZ" (id 6) (at 71.12 95.25 0)
-      (effects (font (size 1.27 1.27)) (justify left bottom) hide)
-    )
-    (property "PACKAGE" "TSSOP-10 Cirrus Logic" (id 7) (at 71.12 95.25 0)
-      (effects (font (size 1.27 1.27)) (justify left bottom) hide)
-    )
-    (property "DESCRIPTION" "D/A converter; 24bit; 192ksps; Channels: 2; 3÷5.25VDC; T" (id 8) (at 71.12 95.25 0)
-      (effects (font (size 1.27 1.27)) (justify left bottom) hide)
-    )
-    (property "PRICE" "None" (id 9) (at 71.12 95.25 0)
-      (effects (font (size 1.27 1.27)) (justify left bottom) hide)
-    )
-    (property "AVAILABILITY" "Unavailable" (id 10) (at 71.12 95.25 0)
-      (effects (font (size 1.27 1.27)) (justify left bottom) hide)
-    )
-    (property "MF" "Cirrus Logic" (id 11) (at 71.12 95.25 0)
-      (effects (font (size 1.27 1.27)) (justify left bottom) hide)
+    (property "LCSC" "C1509050" (id 4) (at 71.12 95.25 0)
+      (effects (font (size 1.27 1.27)) hide)
     )
     (pin "1")
@@
     (in_bom yes) (on_board yes) (fields_autoplaced)
     (property "Reference" "U4" (id 0) (at 185.42 75.184 0))
-    (property "Value" "TDA2822" (id 1) (at 185.42 77.724 0))
-    (property "Footprint" "" (id 2) (at 185.42 85.09 0)
-      (effects (font (size 1.27 1.27)) hide)
-    )
-    (property "Datasheet" "~" (id 3) (at 185.42 85.09 0)
+    (property "Value" "D2822M" (id 1) (at 185.42 77.724 0))
+    (property "Footprint" "Package_SO:SOP-8_3.9x4.9mm_P1.27mm" (id 2) (at 185.42 85.09 0)
+      (effects (font (size 1.27 1.27)) hide)
+    )
+    (property "Datasheet" "https://datasheet.lcsc.com/lcsc/2111030930_Silicore-D2822M-SOP8_C2837292.pdf" (id 3) (at 185.42 85.09 0)
+      (effects (font (size 1.27 1.27)) hide)
+    )
+    (property "LCSC" "C2837292" (id 4) (at 185.42 85.09 0)
       (effects (font (size 1.27 1.27)) hide)
     )
@@
       (effects (font (size 1.27 1.27)) (justify left))
     )
-    (property "Value" "TDA2822" (id 1) (at 188.214 104.1399 0)
-      (effects (font (size 1.27 1.27)) (justify left))
-    )
-    (property "Footprint" "" (id 2) (at 189.23 102.87 0)
-      (effects (font (size 1.27 1.27)) hide)
-    )
-    (property "Datasheet" "~" (id 3) (at 189.23 102.87 0)
+    (property "Value" "D2822M" (id 1) (at 188.214 104.1399 0)
+      (effects (font (size 1.27 1.27)) (justify left))
+    )
+    (property "Footprint" "Package_SO:SOP-8_3.9x4.9mm_P1.27mm" (id 2) (at 189.23 102.87 0)
+      (effects (font (size 1.27 1.27)) hide)
+    )
+    (property "Datasheet" "https://datasheet.lcsc.com/lcsc/2111030930_Silicore-D2822M-SOP8_C2837292.pdf" (id 3) (at 189.23 102.87 0)
       (effects (font (size 1.27 1.27)) hide)
     )
@@
       (effects (font (size 1.27 1.27)) (justify left))
     )
-    (property "Footprint" "" (id 2) (at 234.95 50.8 0)
-      (effects (font (size 1.27 1.27)) hide)
-    )
+    (property "Footprint" "Connector_Molex:Molex_PicoBlade_53261-0271_1x02-1MP_P1.25mm_Horizontal" (id 2) (at 234.95 50.8 0)
+      (effects (font (size 1.27 1.27)) hide)
+    )

Commit message: Bill of materials 1/2
Parts:
- C1: value 1u -> (none); footprint Capacitor_SMD:C_0402_1005Metric -> (none); Category (none) -> Capacitors; LCSC C107372 -> (none)
- C14, C33, C4: value 100n -> (none); footprint Capacitor_SMD:C_0402_1005Metric -> (none); Category (none) -> Capacitors
- C2, C3: value 100n -> (none); footprint Capacitor_SMD:C_0402_1005Metric -> (none); Category (none) -> Capacitors; LCSC C83056 -> (none)
- C47, C51: value 39n -> (none); footprint Capacitor_SMD:C_0402_1005Metric -> (none); Category (none) -> Capacitors
- C5, C52, C53, C54, C55, C57, C6, C64, C65, C66, C67: value 47u -> (none); footprint Capacitor_SMD:C_0805_2012Metric -> (none); Category (none) -> Capacitors
- C56: value 100n -> (none); footprint Capacitor_SMD:C_0603_1608Metric -> (none); Category (none) -> Capacitors
- C68, C69: value 0.1u -> (none); footprint Capacitor_SMD:C_0402_1005Metric -> (none); Category (none) -> Capacitors
- D8: value 1N4148WS -> (none); footprint Diode_SMD:D_SOD-323 -> (none); Category (none) -> Diodes; LCSC (none) -> C181133; MPN (none) -> 1N4148WS; Manufacturer (none) -> Guangdong Hottech
- J1: value AudioJack3 -> (none); footprint custom:Boom-audiojack-PJ-320B -> (none); Category (none) -> Connectors; MPN (none) -> C18594; Manufacturer (none) -> Boomele; Sponsored N -> (none)
- LS1: value Speaker -> (none); footprint Connector_Molex:Molex_PicoBlade_53261-0271_1x02-1MP_P1.25mm_Horizontal -> (none); Category (none) -> Connectors
- R27, R28, R29, R30, R41, R45: value 10k -> (none); footprint Resistor_SMD:R_0402_1005Metric -> (none); Category (none) -> Resistors; LCSC C144807 -> (none); MPN AC0402FR-0710KL -> (none); Sponsored N -> (none)
- R46, R52: value 4.7 -> (none); footprint Resistor_SMD:R_0402_1005Metric -> (none); Category (none) -> Resistors; Sponsored N -> (none)
- R51: value 100k -> (none); footprint Resistor_SMD:R_0402_1005Metric -> (none); Category (none) -> Resistors; LCSC C144807 -> (none); MPN AC0402FR-0710KL -> (none); Sponsored N -> (none)
- RN7: value 47 -> (none); footprint Resistor_SMD:R_Array_Convex_4x0603 -> (none); Category (none) -> Resistor arrays; Sponsored N -> (none)
- RV1: value Volume -> (none); Category (none) -> Potentiometers
- SW8: value Speaker enable -> (none); footprint Button_Switch_SMD:SW_SPDT_PCM12 -> (none); Category (none) -> Buttons; Sponsored N -> (none)
- U1: value MS4344 -> (none); footprint CS4344-CZZ:SOP50P490X110-10N -> (none); Buy early (none) -> Y; Category (none) -> ICs; MPN (none) -> MS4344; Manufacturer (none) -> Hangzhou Ruimeng Tech; Sponsored (none) -> N
- U4: value D2822M -> (none); footprint Package_SO:SOP-8_3.9x4.9mm_P1.27mm -> (none); Buy early (none) -> Y; Category (none) -> ICs; LCSC (none) -> C2837292; MPN (none) -> D2822M SOP8; Manufacturer (none) -> Silicore; Sponsored (none) -> N
- U4: value D2822M -> (none); footprint Package_SO:SOP-8_3.9x4.9mm_P1.27mm -> (none); Buy early (none) -> Y; Category (none) -> ICs; MPN (none) -> D2822M SOP8; Manufacturer (none) -> Silicore; Sponsored (none) -> N

Commit message: Add more info to BOM
Parts:
- C1, C14, C2, C3, C33, C4, C47, C5, C51, C52, C53, C54, C55, C56, C57, C6, C64, C65, C66, C67, C68, C69, D8, J1, LS1, R27, R28, R29, R30, R41, R45, R46, R51, R52: Buy early (none) -> Y; Sponsored (none) -> N
- RN7: Buy early (none) -> Y; Manufacturer (none) -> Uni-royal; Sponsored (none) -> N
- RV1: Buy early (none) -> N; MPN (none) -> TO BE DETERMINED!; Manufacturer (none) -> TO BE DETERMINED!; Sponsored (none) -> N
- SW8: Buy early (none) -> Y; MPN (none) -> SK-3296S-01-L1; Manufacturer (none) -> XKB Connectivity; Sponsored (none) -> N

Commit message: Add IR transmitter, modify bill of materials
Parts:
- removed D8: (no value), symbol Diode:1N4148WS
- removed R51: (no value), symbol mch2021-rescue:R-Device
Connections:
- net SPK_DISABLED: no longer names the net of SW8.3 (C)

Commit message: Add passives to BOM
Parts:
- C1: LCSC (none) -> C107372; MPN (none) -> CL05A105KQ5NNNC; Manufacturer (none) -> Samsung Electro-Mechanics; Minimal voltage rating (none) -> 6; Voltage rating (none) -> 6.3
- C14, C2, C3, C33, C4, C56, C68, C69: LCSC (none) -> C307331; MPN (none) -> CL05B104KB54PNC; Manufacturer (none) -> Samsung Electro-Mechanics; Minimal voltage rating (none) -> 10; Voltage rating (none) -> 50
- C47, C51: LCSC (none) -> C880624; MPN (none) -> TCC0402X7R393K500AT; Manufacturer (none) -> CCTC; Minimal voltage rating (none) -> 10; Voltage rating (none) -> 50
- C5, C52, C53, C54, C55, C57, C6, C64, C65, C66, C67: LCSC (none) -> C16780; MPN (none) -> CL21A476MQYNNNE; Manufacturer (none) -> Samsung Electro-Mechanics; Minimal voltage rating (none) -> 6; Voltage rating (none) -> 6.3
- LS1: Buy early Y -> N
- R27, R28, R29, R30, R41, R45: LCSC (none) -> C25744; MPN (none) -> 0402WGF1002TCE; Manufacturer (none) -> Uni-royal
- R46, R52: LCSC C144807 -> C25121; MPN AC0402FR-0710KL -> 0402WGF470KTCE; Manufacturer (none) -> Uni-royal

Commit message: Artwork stuff
Parts:
- C1: value (none) -> 1u; footprint (none) -> Capacitor_SMD:C_0402_1005Metric
- C14, C2, C3, C33, C4, C56, C68, C69: value (none) -> 100n; footprint (none) -> Capacitor_SMD:C_0402_1005Metric
- C47, C51: value (none) -> 39n; footprint (none) -> Capacitor_SMD:C_0402_1005Metric
- C5, C52, C53, C54, C55, C57, C6, C64, C65, C66, C67: value (none) -> 47u; footprint (none) -> Capacitor_SMD:C_0805_2012Metric
- J1: value (none) -> AudioJack3; footprint (none) -> custom:Boom-audiojack-PJ-320B
- LS1: value (none) -> Speaker; footprint (none) -> Connector_Molex:Molex_PicoBlade_53261-0271_1x02-1MP_P1.25mm_Horizontal
- R27, R28, R29, R30, R41, R45: value (none) -> 10k; footprint (none) -> Resistor_SMD:R_0402_1005Metric
- R46, R52: value (none) -> 4.7; footprint (none) -> Resistor_SMD:R_0402_1005Metric
- RN7: value (none) -> 47; footprint (none) -> Resistor_SMD:R_Array_Convex_4x0603
- RV1: value (none) -> Volume
- SW8: value (none) -> Switch; footprint (none) -> Button_Switch_SMD:SW_SPDT_PCM12
- U1: value (none) -> MS4344; footprint (none) -> CS4344-CZZ:SOP50P490X110-10N
- U4: value (none) -> D2822M; footprint (none) -> Package_SO:SOP-8_3.9x4.9mm_P1.27mm

Commit message: Add lanyard holes, component placement
Parts:
- removed C2: 100n, Capacitor_SMD:C_0402_1005Metric, symbol mch2021-rescue:C-Device
- removed RV1: Volume, symbol Device:R_Potentiometer_Dual_Separate
Connections:
- net at C66.1, C67.2, C68.2: now also SW8.2 (B); no longer J1.R
- net at C64.1, C65.2, C69.2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: no longer SW8.1 (A)
- net at LS1.1: now also SW8.1 (A); no longer SW8.2 (B)
- net at SW8.3 (C): now also J1.R
- net at U4.7 (+): now also R41.2; no longer R29.1
- net at C64.2, C65.1: now also U4.3; no longer U4.1
- net at C52.2, C53.2: now also U4.5 (-); no longer U4.8 (-)
- net at C66.2, C67.1: now also U4.1; no longer U4.3
- net at C54.2, C55.2: now also U4.8 (-); no longer U4.5 (-)
- net at U4.6 (+): now also R29.1; no longer R41.2
Other:
- moved on the sheet: C1, R41, R45, SW8, U4A, U4B
