File: audio.kicad_sch (KiCad schematic)
At the start: 35 parts, among them J1 AudioJack3, SW8 Switch, U1 MS4344, U4 D2822M

Commit message: Last minute fixes
Parts:
- added TP34, TP35: Testpoint, TestPoint:TestPoint_Pad_1.0x1.0mm, symbol mch2021-rescue:TestPoint_Small-Connector
Connections:
- net GND: now also TP34.1
- net at LS1.1, SW8.1 (A): now also TP35.1
Changed lines of the file:
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@@
   (junction (at 196.85 64.77) (diameter 0) (color 0 0 0 0)
   )
+  (junction (at 223.52 54.61) (diameter 0) (color 0 0 0 0)
+  )
   (junction (at 182.88 95.25) (diameter 0) (color 0 0 0 0)
   )
@@
   (junction (at 191.77 64.77) (diameter 0) (color 0 0 0 0)
   )
+  (junction (at 223.774 45.72) (diameter 0) (color 0 0 0 0)
+  )
   (junction (at 171.45 87.63) (diameter 0) (color 0 0 0 0)
   )
@@
     (stroke (width 0) (type default) (color 0 0 0 0))
   )
+  (wire (pts (xy 223.52 54.61) (xy 223.52 110.49))
+    (stroke (width 0) (type default) (color 0 0 0 0))
+  )
   (wire (pts (xy 182.88 95.25) (xy 186.69 95.25))
     (stroke (width 0) (type default) (color 0 0 0 0))
@@
     (stroke (width 0) (type default) (color 0 0 0 0))
   )
-  (wire (pts (xy 223.52 48.26) (xy 223.52 110.49))
+  (wire (pts (xy 223.52 48.26) (xy 223.52 54.61))
     (stroke (width 0) (type default) (color 0 0 0 0))
   )
@@
     (stroke (width 0) (type default) (color 0 0 0 0))
   )
-  (wire (pts (xy 220.98 45.72) (xy 229.87 45.72))
+  (wire (pts (xy 220.98 45.72) (xy 223.774 45.72))
     (stroke (width 0) (type default) (color 0 0 0 0))
   )
@@
   )
   (wire (pts (xy 182.88 93.98) (xy 182.88 95.25))
+    (stroke (width 0) (type default) (color 0 0 0 0))
+  )
+  (wire (pts (xy 223.774 45.72) (xy 229.87 45.72))
     (stroke (width 0) (type default) (color 0 0 0 0))
   )
@@
     (pin "1")
   )
+  (symbol (lib_id "mch2021-rescue:TestPoint_Small-Connector") (at 223.774 45.72 270) (unit 1)
+    (in_bom yes) (on_board yes)
+    (property "Reference" "TP35" (id 0) (at 223.774 40.64 0)
+      (effects (font (size 1.27 1.27)) (justify left))
+    )
+    (property "Value" "Testpoint" (id 1) (at 222.631 46.9392 0)
+      (effects (font (size 1.27 1.27)) (justify left) hide)
+    )
+    (property "Footprint" "TestPoint:TestPoint_Pad_1.0x1.0mm" (id 2) (at 223.774 50.8 0)
+      (effects (font (size 1.27 1.27)) hide)
+    )
+    (property "Datasheet" "" (id 3) (at 223.774 50.8 0)
+      (effects (font (size 1.27 1.27)) hide)
+    )
+    (property "Category" "Testpoints" (id 4) (at 223.774 45.72 0)
+      (effects (font (size 1.27 1.27)) hide)
+    )
+    (property "Buy early" "N" (id 5) (at 223.774 45.72 0)
+      (effects (font (size 1.27 1.27)) hide)
+    )
+    (property "Sponsored" "N" (id 6) (at 223.774 45.72 0)
+      (effects (font (size 1.27 1.27)) hide)
+    )
+    (pin "1")
+  )
   (symbol (lib_id "mch2021-rescue:GND-power") (at 93.98 109.22 0) (mirror y) (unit 1)
     (in_bom yes) (on_board yes)
@@
     (pin "2")
   )
+  (symbol (lib_id "mch2021-rescue:TestPoint_Small-Connector") (at 223.52 54.61 0) (unit 1)
+    (in_bom yes) (on_board yes)
+    (property "Reference" "TP34" (id 0) (at 218.44 54.61 0)
+      (effects (font (size 1.27 1.27)) (justify left))
+    )
+    (property "Value" "Testpoint" (id 1) (at 224.7392 55.753 0)
+      (effects (font (size 1.27 1.27)) (justify left) hide)
+    )
+    (property "Footprint" "TestPoint:TestPoint_Pad_1.0x1.0mm" (id 2) (at 228.6 54.61 0)
+      (effects (font (size 1.27 1.27)) hide)
+    )
+    (property "Datasheet" "" (id 3) (at 228.6 54.61 0)
+      (effects (font (size 1.27 1.27)) hide)
+    )
+    (property "Category" "Testpoints" (id 4) (at 223.52 54.61 0)
+      (effects (font (size 1.27 1.27)) hide)
+    )
+    (property "Buy early" "N" (id 5) (at 223.52 54.61 0)
+      (effects (font (size 1.27 1.27)) hide)
+    )
+    (property "Sponsored" "N" (id 6) (at 223.52 54.61 0)
+      (effects (font (size 1.27 1.27)) hide)
+    )
+    (pin "1")
+  )
   (symbol (lib_id "Device:C_Small") (at 182.88 102.87 180) (unit 1)

Commit message: Final version of prototype 4
Parts:
- LS1: value Speaker -> (none); footprint Connector_Molex:Molex_PicoBlade_53261-0271_1x02-1MP_P1.25mm_Horizontal -> (none); symbol Device:Speaker -> Connector_Generic_MountingPin:Conn_01x02_MountingPin
Connections:
- net GND: now also LS1.MP (MountPin)
Changed lines of the file:
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@@
     (pin "4")
+  )
+  (symbol (lib_id "mch2021-rescue:GND-power") (at 234.95 53.34 0) (mirror y) (unit 1)
+    (in_bom yes) (on_board yes)
+    (property "Reference" "#PWR?" (id 0) (at 234.95 59.69 0)
+      (effects (font (size 1.27 1.27)) hide)
+    )
+    (property "Value" "GND" (id 1) (at 234.823 57.7342 0))
+    (property "Footprint" "" (id 2) (at 234.95 53.34 0)
+      (effects (font (size 1.27 1.27)) hide)
+    )
+    (property "Datasheet" "" (id 3) (at 234.95 53.34 0)
+      (effects (font (size 1.27 1.27)) hide)
+    )
+    (pin "1")
   )
   (symbol (lib_id "mch2021-rescue:GND-power") (at 182.88 111.76 0) (mirror y) (unit 1)
@@
     (pin "2")
   )
-  (symbol (lib_id "Device:Speaker") (at 234.95 45.72 0) (unit 1)
+  (symbol (lib_id "Connector_Generic_MountingPin:Conn_01x02_MountingPin") (at 234.95 45.72 0) (unit 1)
     (in_bom yes) (on_board yes) (fields_autoplaced)
     (property "Reference" "LS1" (id 0) (at 239.395 45.7199 0)
       (effects (font (size 1.27 1.27)) (justify left))
     )
-    (property "Value" "Speaker" (id 1) (at 239.395 48.2599 0)
+    (property "Value" "" (id 1) (at 239.395 48.2599 0)
       (effects (font (size 1.27 1.27)) (justify left))
     )
-    (property "Footprint" "Connector_Molex:Molex_PicoBlade_53261-0271_1x02-1MP_P1.25mm_Horizontal" (id 2) (at 234.95 50.8 0)
+    (property "Footprint" "" (id 2) (at 234.95 50.8 0)
       (effects (font (size 1.27 1.27)) hide)
     )
@@
     (pin "1")
     (pin "2")
+    (pin "MP")
   )
   (symbol (lib_id "Device:C_Small") (at 105.41 87.63 0) (unit 1)

Commit message: Small last minute tweaks
Parts:
- LS1: value (none) -> Speaker; footprint (none) -> Connector_Molex:Molex_PicoBlade_53261-0271_1x02-1MP_P1.25mm_Horizontal
- R27, R28: value 10k -> 330; LCSC C25744 -> (none); MANUFACTURER YAGEO -> (none); MPN 0402WGF1002TCE -> (none); Manufacturer Uni-royal -> (none)
- R29, R30, R41, R45: value 10k -> (none); footprint Resistor_SMD:R_0402_1005Metric -> (none); LCSC C25744 -> (none); MANUFACTURER YAGEO -> (none); MPN 0402WGF1002TCE -> (none); Manufacturer Uni-royal -> (none)
Connections:
- net AUDIO_L: no longer R45.2
- net AUDIO_R: now also R29.1; no longer R29.2, R30.2
- net at R41.2, U4.7 (+): now also R45.2
- net at U4.6 (+): now also R29.2, R30.2; no longer R29.1
Other:
- moved on the sheet: R29, R41

Commit message: Pre-production final design
Parts:
- C1: value 1u -> (none); footprint Capacitor_SMD:C_0402_1005Metric -> (none)
- C14, C3, C33, C4, C56, C68, C69: value 100n -> (none); footprint Capacitor_SMD:C_0402_1005Metric -> (none)
- C47, C51: value 39n -> (none); footprint Capacitor_SMD:C_0402_1005Metric -> (none)
- C5, C52, C53, C54, C55, C57, C6, C64, C65, C66, C67: value 47u -> (none); footprint Capacitor_SMD:C_0805_2012Metric -> (none)
- J1: value AudioJack3 -> (none); footprint custom:Boom-audiojack-PJ-320B -> (none)
- LS1: value Speaker -> (none); footprint Connector_Molex:Molex_PicoBlade_53261-0271_1x02-1MP_P1.25mm_Horizontal -> (none)
- R27, R28: value 330 -> (none); footprint Resistor_SMD:R_0402_1005Metric -> (none); LCSC (none) -> C423288; MANUFACTURER (none) -> UNI-ROYAL; MPN (none) -> 0402WGD3300TCE; Manufacturer (none) -> Uni-royal
- R29, R41: LCSC (none) -> C25768; MANUFACTURER (none) -> UNI-ROYAL; MPN (none) -> 0402WGF2202TCE; Manufacturer (none) -> Uni-royal
- R30, R45: LCSC (none) -> C11702; MANUFACTURER (none) -> UNI-ROYAL; MPN (none) -> 0402WGF1001TCE; Manufacturer (none) -> Uni-royal
- R46, R52: value 4.7 -> (none); footprint Resistor_SMD:R_0402_1005Metric -> (none); MANUFACTURER YAGEO -> UNI-ROYAL
- RN7: value 47 -> (none); footprint Resistor_SMD:R_Array_Convex_4x0603 -> (none)
- SW8: value Switch -> (none); footprint Button_Switch_SMD:SW_SPDT_PCM12 -> (none)
- TP34, TP35: value Testpoint -> (none); footprint TestPoint:TestPoint_Pad_1.0x1.0mm -> (none)
- U1: value MS4344 -> (none); footprint CS4344-CZZ:SOP50P490X110-10N -> (none)
- U4: value D2822M -> (none); footprint Package_SO:SOP-8_3.9x4.9mm_P1.27mm -> (none)

Commit message: Add gerbers, add schematic, finalize design
Parts:
- C1: value (none) -> 1u; footprint (none) -> Capacitor_SMD:C_0402_1005Metric
- C14, C3, C33, C4, C56, C68, C69: value (none) -> 100n; footprint (none) -> Capacitor_SMD:C_0402_1005Metric
- C47, C51: value (none) -> 39n; footprint (none) -> Capacitor_SMD:C_0402_1005Metric
- C5, C52, C53, C54, C55, C57, C6, C64, C65, C66, C67: value (none) -> 47u; footprint (none) -> Capacitor_SMD:C_0805_2012Metric
- J1: value (none) -> AudioJack3; footprint (none) -> custom:Boom-audiojack-PJ-320B
- LS1: value (none) -> Speaker; footprint (none) -> Connector_Molex:Molex_PicoBlade_53261-0271_1x02-1MP_P1.25mm_Horizontal
- R27, R28: value (none) -> 330; footprint (none) -> Resistor_SMD:R_0402_1005Metric
- R29, R41: value (none) -> 22k; footprint (none) -> Resistor_SMD:R_0402_1005Metric
- R30, R45: value (none) -> 1k; footprint (none) -> Resistor_SMD:R_0402_1005Metric
- R46, R52: value (none) -> 4.7; footprint (none) -> Resistor_SMD:R_0402_1005Metric
- RN7: value (none) -> 47; footprint (none) -> Resistor_SMD:R_Array_Convex_4x0603
- SW8: value (none) -> Switch; footprint (none) -> Button_Switch_SMD:SW_SPDT_PCM12
- TP34, TP35: value (none) -> Testpoint; footprint (none) -> TestPoint:TestPoint_Pad_1.0x1.0mm
- U1: value (none) -> MS4344; footprint (none) -> CS4344-CZZ:SOP50P490X110-10N
- U4: value (none) -> D2822M; footprint (none) -> Package_SO:SOP-8_3.9x4.9mm_P1.27mm
Other:
- company: (none) -> BADGE.TEAM
