File: mch2021.kicad_sch (KiCad schematic)
At the start: 36 parts

Commit message: Add passives to BOM
Parts:
- R1, R2: Manufacturer (none) -> Uni-royal
- R22, R4, R5: LCSC (none) -> C25118; MPN (none) -> 0402WGF470JTCE; Manufacturer (none) -> Uni-royal
Changed lines of the file:
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@@
       (effects (font (size 1.27 1.27)) hide)
     )
-    (property "Datasheet" "" (id 3) (at 45.72 35.56 0)
+    (property "Datasheet" "https://datasheet.lcsc.com/lcsc/2110260030_UNI-ROYAL-Uniroyal-Elec-0402WGF5101TCE_C25905.pdf" (id 3) (at 45.72 35.56 0)
       (effects (font (size 1.27 1.27)) hide)
     )
@@
     )
     (property "Description" "Generic part" (id 12) (at 45.72 35.56 0)
+      (effects (font (size 1.27 1.27)) hide)
+    )
+    (property "Manufacturer" "Uni-royal" (id 13) (at 45.72 35.56 0)
       (effects (font (size 1.27 1.27)) hide)
     )
@@
       (effects (font (size 1.27 1.27)) hide)
     )
-    (property "Datasheet" "" (id 3) (at 45.72 33.02 0)
+    (property "Datasheet" "https://datasheet.lcsc.com/lcsc/2110260030_UNI-ROYAL-Uniroyal-Elec-0402WGF5101TCE_C25905.pdf" (id 3) (at 45.72 33.02 0)
       (effects (font (size 1.27 1.27)) hide)
     )
@@
     )
     (property "Description" "Generic part" (id 12) (at 45.72 33.02 0)
+      (effects (font (size 1.27 1.27)) hide)
+    )
+    (property "Manufacturer" "Uni-royal" (id 13) (at 45.72 33.02 0)
       (effects (font (size 1.27 1.27)) hide)
     )
@@
       (effects (font (size 1.27 1.27)) hide)
     )
-    (property "Datasheet" "" (id 3) (at 152.4 111.76 0)
+    (property "Datasheet" "https://datasheet.lcsc.com/lcsc/2110252230_UNI-ROYAL-Uniroyal-Elec-0402WGF470JTCE_C25118.pdf" (id 3) (at 152.4 111.76 0)
       (effects (font (size 1.27 1.27)) hide)
     )
@@
       (effects (font (size 1.27 1.27)) hide)
     )
-    (property "LCSC" "" (id 5) (at 152.4 111.76 0)
+    (property "LCSC" "C25118" (id 5) (at 152.4 111.76 0)
       (effects (font (size 1.27 1.27)) hide)
     )
@@
       (effects (font (size 1.27 1.27)) hide)
     )
-    (property "MPN" "" (id 9) (at 152.4 111.76 0)
+    (property "MPN" "0402WGF470JTCE" (id 9) (at 152.4 111.76 0)
       (effects (font (size 1.27 1.27)) hide)
     )
@@
     )
     (property "Description" "Generic part" (id 12) (at 152.4 111.76 0)
+      (effects (font (size 1.27 1.27)) hide)
+    )
+    (property "Manufacturer" "Uni-royal" (id 13) (at 152.4 111.76 0)
       (effects (font (size 1.27 1.27)) hide)
     )
@@
       (effects (font (size 1.27 1.27)) hide)
     )
-    (property "Datasheet" "" (id 3) (at 148.59 111.76 0)
+    (property "Datasheet" "https://datasheet.lcsc.com/lcsc/2110252230_UNI-ROYAL-Uniroyal-Elec-0402WGF470JTCE_C25118.pdf" (id 3) (at 148.59 111.76 0)
       (effects (font (size 1.27 1.27)) hide)
     )
@@
       (effects (font (size 1.27 1.27)) hide)
     )
-    (property "LCSC" "" (id 5) (at 148.59 111.76 0)
+    (property "LCSC" "C25118" (id 5) (at 148.59 111.76 0)
       (effects (font (size 1.27 1.27)) hide)
     )
@@
       (effects (font (size 1.27 1.27)) hide)
     )
-    (property "MPN" "" (id 9) (at 148.59 111.76 0)
+    (property "MPN" "0402WGF470JTCE" (id 9) (at 148.59 111.76 0)
       (effects (font (size 1.27 1.27)) hide)
     )
@@
     )
     (property "Description" "Generic part" (id 12) (at 148.59 111.76 0)
+      (effects (font (size 1.27 1.27)) hide)
+    )
+    (property "Manufacturer" "Uni-royal" (id 13) (at 148.59 111.76 0)
       (effects (font (size 1.27 1.27)) hide)
     )
@@
       (effects (font (size 1.27 1.27)) hide)
     )
-    (property "Datasheet" "" (id 3) (at 144.78 111.76 0)
+    (property "Datasheet" "https://datasheet.lcsc.com/lcsc/2110252230_UNI-ROYAL-Uniroyal-Elec-0402WGF470JTCE_C25118.pdf" (id 3) (at 144.78 111.76 0)
       (effects (font (size 1.27 1.27)) hide)
     )
@@
       (effects (font (size 1.27 1.27)) hide)
     )
-    (property "LCSC" "" (id 5) (at 144.78 111.76 0)
+    (property "LCSC" "C25118" (id 5) (at 144.78 111.76 0)
       (effects (font (size 1.27 1.27)) hide)
     )
@@
       (effects (font (size 1.27 1.27)) hide)
     )
-    (property "MPN" "" (id 9) (at 144.78 111.76 0)
+    (property "MPN" "0402WGF470JTCE" (id 9) (at 144.78 111.76 0)
       (effects (font (size 1.27 1.27)) hide)
     )
@@
       (effects (font (size 1.27 1.27)) hide)
     )
+    (property "Manufacturer" "Uni-royal" (id 13) (at 144.78 111.76 0)
+      (effects (font (size 1.27 1.27)) hide)
+    )
