File: mch2021.kicad_sch (KiCad schematic)
At the start: 36 parts

Commit message: Artwork stuff
Parts:
- removed N4, N5: (no value), symbol mch2021-rescue:Housing-Mechanical
- D1: value (none) -> USBLC6-4SC6; footprint (none) -> digikey-footprints:SOT23-6L
- D2: value (none) -> RGB-5050; footprint (none) -> LED_SMD:LED_RGB_5050-6
- F1: value (none) -> 1A; footprint (none) -> Fuse:Fuse_0805_2012Metric
- J2: value (none) -> USB_C_Receptacle_USB2.0; footprint (none) -> Connector_USB:USB_C_Receptacle_HRO_TYPE-C-31-M-12
- J4: value (none) -> PMOD; footprint (none) -> Connector_PinSocket_2.54mm:PinSocket_2x06_P2.54mm_Horizontal
- N1: value (none) -> Logo; footprint (none) -> custom:badgeteam
- R1, R2: value (none) -> 5.1k; footprint (none) -> Resistor_SMD:R_0402_1005Metric
- R22, R4, R5: value (none) -> 47; footprint (none) -> Resistor_SMD:R_0402_1005Metric
- TP1, TP10, TP11, TP12, TP13, TP18, TP19, TP20, TP21, TP22, TP23, TP24, TP25, TP26, TP28, TP29, TP30, TP4, TP5, TP6, TP7, TP8: value (none) -> Testpoint; footprint (none) -> TestPoint:TestPoint_Pad_1.0x1.0mm

Commit message: Swap led data and sd power on ESP32, add speaker grill
Parts:
- removed TP23, TP24: Testpoint, TestPoint:TestPoint_Pad_1.0x1.0mm, symbol mch2021-rescue:TestPoint_Small-Connector
- N2: value (none) -> Artwork; footprint (none) -> custom:prototype4_no_outline
Changed lines of the file:
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@@
   (junction (at 170.18 104.14) (diameter 0) (color 0 0 0 0)
   )
-  (junction (at 148.59 83.82) (diameter 0) (color 0 0 0 0)
-  )
   (junction (at 74.93 52.07) (diameter 0) (color 0 0 0 0)
   )
@@
   (junction (at 148.59 34.29) (diameter 0) (color 0 0 0 0)
   )
-  (junction (at 146.05 81.28) (diameter 0) (color 0 0 0 0)
-  )
   (no_connect (at 40.64 58.42))
   (no_connect (at 40.64 55.88))
@@
       (effects (font (size 1.27 1.27)) (justify left))
     )
-    (property "Value" "" (id 1) (at 27.3812 191.3128 0)
+    (property "Value" "Artwork" (id 1) (at 27.3812 191.3128 0)
       (effects (font (size 1.27 1.27)) (justify left))
     )
-    (property "Footprint" "" (id 2) (at 24.765 188.595 0)
+    (property "Footprint" "custom:prototype4_no_outline" (id 2) (at 24.765 188.595 0)
       (effects (font (size 1.27 1.27)) hide)
     )
@@
     (pin "1")
   )
-  (symbol (lib_id "mch2021-rescue:TestPoint_Small-Connector") (at 146.05 81.28 180) (unit 1)
-    (in_bom yes) (on_board yes)
-    (property "Reference" "TP23" (id 0) (at 151.13 81.28 0)
-      (effects (font (size 1.27 1.27)) (justify left))
-    )
-    (property "Value" "Testpoint" (id 1) (at 144.8308 80.137 0)
-      (effects (font (size 1.27 1.27)) (justify left) hide)
-    )
-    (property "Footprint" "TestPoint:TestPoint_Pad_1.0x1.0mm" (id 2) (at 140.97 81.28 0)
-      (effects (font (size 1.27 1.27)) hide)
-    )
-    (property "Datasheet" "" (id 3) (at 140.97 81.28 0)
-      (effects (font (size 1.27 1.27)) hide)
-    )
-    (property "Category" "Testpoints" (id 4) (at 146.05 81.28 0)
-      (effects (font (size 1.27 1.27)) hide)
-    )
-    (property "Buy early" "N" (id 5) (at 146.05 81.28 0)
-      (effects (font (size 1.27 1.27)) hide)
-    )
-    (property "Sponsored" "N" (id 6) (at 146.05 81.28 0)
-      (effects (font (size 1.27 1.27)) hide)
-    )
-    (pin "1")
-  )
-  (symbol (lib_id "mch2021-rescue:TestPoint_Small-Connector") (at 148.59 83.82 180) (unit 1)
-    (in_bom yes) (on_board yes)
-    (property "Reference" "TP24" (id 0) (at 153.67 83.82 0)
-      (effects (font (size 1.27 1.27)) (justify left))
-    )
-    (property "Value" "Testpoint" (id 1) (at 147.3708 82.677 0)
-      (effects (font (size 1.27 1.27)) (justify left) hide)
-    )
-    (property "Footprint" "TestPoint:TestPoint_Pad_1.0x1.0mm" (id 2) (at 143.51 83.82 0)
-      (effects (font (size 1.27 1.27)) hide)
-    )
-    (property "Datasheet" "" (id 3) (at 143.51 83.82 0)
-      (effects (font (size 1.27 1.27)) hide)
-    )
-    (property "Category" "Testpoints" (id 4) (at 148.59 83.82 0)
-      (effects (font (size 1.27 1.27)) hide)
-    )
-    (property "Buy early" "N" (id 5) (at 148.59 83.82 0)
-      (effects (font (size 1.27 1.27)) hide)
-    )
-    (property "Sponsored" "N" (id 6) (at 148.59 83.82 0)
-      (effects (font (size 1.27 1.27)) hide)
-    )
-    (pin "1")
-  )
   (symbol (lib_id "mch2021-rescue:GND-power") (at 27.94 100.33 0) (mirror y) (unit 1)
     (in_bom yes) (on_board yes)
@@
       (reference "TP22") (unit 1) (value "Testpoint") (footprint "TestPoint:TestPoint_Pad_1.0x1.0mm")
     )
-    (path "/00000000-0000-0000-0000-000061dfa163"
-      (reference "TP23") (unit 1) (value "Testpoint") (footprint "TestPoint:TestPoint_Pad_1.0x1.0mm")
-    )
-    (path "/00000000-0000-0000-0000-000061dfa34c"
-      (reference "TP24") (unit 1) (value "Testpoint") (footprint "TestPoint:TestPoint_Pad_1.0x1.0mm")
-    )
     (path "/a99cc5cf-7b0a-4dbb-aee0-e27984886141"

Commit message: ...
Parts:
- N2: value Artwork -> (none); footprint custom:prototype4_no_outline -> (none)
Changed lines of the file:
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@@
       (effects (font (size 1.27 1.27)) (justify left))
     )
-    (property "Value" "Artwork" (id 1) (at 27.3812 191.3128 0)
-      (effects (font (size 1.27 1.27)) (justify left))
-    )
-    (property "Footprint" "custom:prototype4_no_outline" (id 2) (at 24.765 188.595 0)
+    (property "Value" "" (id 1) (at 27.3812 191.3128 0)
+      (effects (font (size 1.27 1.27)) (justify left))
+    )
+    (property "Footprint" "" (id 2) (at 24.765 188.595 0)
       (effects (font (size 1.27 1.27)) hide)
     )
@@
     )
     (path "/00000000-0000-0000-0000-00005ff5b20d"
-      (reference "N2") (unit 1) (value "Artwork") (footprint "custom:prototype4_no_outline")
+      (reference "N2") (unit 1) (value "Artwork") (footprint "custom:prototype4")
     )
     (path "/00000000-0000-0000-0000-00005fdc6c76/00000000-0000-0000-0000-00006005561c"

Commit message: Add lanyard holes, component placement
Parts:
- N2: value (none) -> Artwork; footprint (none) -> custom:prototype4
Connections:
- net AUDIO/I2S_MCLK: now also TP21.1
- net USB_D+: now also D1.3; no longer D1.6
- net USB_D-: now also D1.6; no longer D1.4
Changed lines of the file:
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@@
   (junction (at 40.64 45.72) (diameter 0) (color 0 0 0 0)
   )
-  (junction (at 57.15 43.18) (diameter 0) (color 0 0 0 0)
-  )
-  (junction (at 46.99 45.72) (diameter 0) (color 0 0 0 0)
-  )
   (junction (at 50.8 35.56) (diameter 0) (color 0 0 0 0)
   )
@@
   (junction (at 167.64 96.52) (diameter 0) (color 0 0 0 0)
   )
+  (junction (at 63.5 45.72) (diameter 0) (color 0 0 0 0)
+  )
   (junction (at 172.72 101.6) (diameter 0) (color 0 0 0 0)
   )
@@
   (junction (at 52.07 27.94) (diameter 0) (color 0 0 0 0)
   )
+  (junction (at 46.99 43.18) (diameter 0) (color 0 0 0 0)
+  )
   (junction (at 85.09 64.77) (diameter 0) (color 0 0 0 0)
   )
@@
     (stroke (width 0) (type default) (color 0 0 0 0))
   )
-  (wire (pts (xy 46.99 45.72) (xy 92.71 45.72))
+  (wire (pts (xy 40.64 45.72) (xy 63.5 45.72))
     (stroke (width 0) (type default) (color 0 0 0 0))
   )
@@
     (stroke (width 0) (type default) (color 0 0 0 0))
   )
+  (wire (pts (xy 46.99 43.18) (xy 46.99 50.8))
+    (stroke (width 0) (type default) (color 0 0 0 0))
+  )
   (wire (pts (xy 223.52 57.15) (xy 224.79 57.15))
     (stroke (width 0) (type default) (color 0 0 0 0))
@@
     (stroke (width 0) (type default) (color 0 0 0 0))
   )
+  (wire (pts (xy 63.5 45.72) (xy 92.71 45.72))
+    (stroke (width 0) (type default) (color 0 0 0 0))
+  )
   (wire (pts (xy 82.55 140.97) (xy 175.26 140.97))
     (stroke (width 0) (type default) (color 0 0 0 0))
@@
     (stroke (width 0) (type default) (color 0 0 0 0))
   )
-  (wire (pts (xy 40.64 43.18) (xy 57.15 43.18))
+  (wire (pts (xy 63.5 76.2) (xy 63.5 45.72))
+    (stroke (width 0) (type default) (color 0 0 0 0))
+  )
+  (wire (pts (xy 40.64 43.18) (xy 46.99 43.18))
     (stroke (width 0) (type default) (color 0 0 0 0))
   )
@@
     (stroke (width 0) (type default) (color 0 0 0 0))
   )
-  (wire (pts (xy 57.15 50.8) (xy 57.15 43.18))
-    (stroke (width 0) (type default) (color 0 0 0 0))
-  )
   (wire (pts (xy 218.44 151.13) (xy 250.19 151.13))
     (stroke (width 0) (type default) (color 0 0 0 0))
@@
     (stroke (width 0) (type default) (color 0 0 0 0))
   )
-  (wire (pts (xy 57.15 43.18) (xy 92.71 43.18))
+  (wire (pts (xy 46.99 43.18) (xy 92.71 43.18))
     (stroke (width 0) (type default) (color 0 0 0 0))
   )
@@
     (stroke (width 0) (type default) (color 0 0 0 0))
   )
-  (wire (pts (xy 40.64 45.72) (xy 46.99 45.72))
-    (stroke (width 0) (type default) (color 0 0 0 0))
-  )
   (wire (pts (xy 228.6 83.82) (xy 228.6 118.11))
     (stroke (width 0) (type default) (color 0 0 0 0))
@@
     (stroke (width 0) (type default) (color 0 0 0 0))
   )
+  (wire (pts (xy 57.15 76.2) (xy 63.5 76.2))
+    (stroke (width 0) (type default) (color 0 0 0 0))
+  )
   (wire (pts (xy 175.26 153.67) (xy 171.45 153.67))
     (stroke (width 0) (type default) (color 0 0 0 0))
@@
     (stroke (width 0) (type default) (color 0 0 0 0))
   )
-  (wire (pts (xy 46.99 50.8) (xy 46.99 45.72))
-    (stroke (width 0) (type default) (color 0 0 0 0))
-  )
   (wire (pts (xy 218.44 123.19) (xy 233.68 123.19))
     (stroke (width 0) (type default) (color 0 0 0 0))
@@
       (effects (font (size 1.27 1.27)) (justify left))
     )
-    (property "Value" "" (id 1) (at 27.3812 191.3128 0)
+    (property "Value" "Artwork" (id 1) (at 27.3812 191.3128 0)
       (effects (font (size 1.27 1.27)) (justify left))
     )
-    (property "Footprint" "" (id 2) (at 24.765 188.595 0)
+    (property "Footprint" "custom:prototype4" (id 2) (at 24.765 188.595 0)
       (effects (font (size 1.27 1.27)) hide)
     )
@@
       (effects (font (size 1.27 1.27)) (justify left))
     )
-    (pin "I2S_MCLK" output (at 218.44 49.784 0)
+    (pin "I2S_MCLK" output (at 218.44 49.53 0)
       (effects (font (size 1.27 1.27)) (justify right))
     )
@@
       (effects (font (size 1.27 1.27)) (justify left))
     )
-    (pin "I2S_MCLK" input (at 224.79 49.784 180)
+    (pin "I2S_MCLK" input (at 224.79 49.53 180)
       (effects (font (size 1.27 1.27)) (justify left))
     )
@@
       (reference "#PWR0112") (unit 1) (value "GND") (footprint "")
     )
-    (path "/8ec93f95-b65c-4f0d-a4f4-32395a9e162a/875c29b3-34af-424e-932a-e02bbfc5c48c"
-      (reference "#PWR0113") (unit 1) (value "+3.3V") (footprint "")
-    )
     (path "/00000000-0000-0000-0000-000060c794cb/00000000-0000-0000-0000-000060575709"
       (reference "#PWR0114") (unit 1) (value "+3.3V") (footprint "")
@@
       (reference "#PWR0166") (unit 1) (value "GND") (footprint "")
     )
-    (path "/8ec93f95-b65c-4f0d-a4f4-32395a9e162a/1ea4fcc5-ccb1-4862-b05f-bd5ed8827319"
-      (reference "#PWR0167") (unit 1) (value "GND") (footprint "")
-    )
     (path "/00000000-0000-0000-0000-000060c789de/00000000-0000-0000-0000-000060c79ccb"
       (reference "#PWR0168") (unit 1) (value "GND") (footprint "")
@@
       (reference "#PWR0208") (unit 1) (value "GND") (footprint "")
     )
-    (path "/8ec93f95-b65c-4f0d-a4f4-32395a9e162a/6f8197c0-10c3-4fa5-81df-8a1835ab5626"
-      (reference "#PWR0209") (unit 1) (value "+3.3V") (footprint "")
-    )
     (path "/8ec93f95-b65c-4f0d-a4f4-32395a9e162a/7c516d1c-50a2-44a2-8220-4d01906fc98e"
       (reference "#PWR0210") (unit 1) (value "GND") (footprint "")
@@
       (reference "C1") (unit 1) (value "1u") (footprint "Capacitor_SMD:C_0402_1005Metric")
     )
-    (path "/8ec93f95-b65c-4f0d-a4f4-32395a9e162a/4252f8ec-ac2f-46c4-8fe7-599d67a2364a"
-      (reference "C2") (unit 1) (value "100n") (footprint "Capacitor_SMD:C_0402_1005Metric")
-    )
     (path "/8ec93f95-b65c-4f0d-a4f4-32395a9e162a/dbd40e82-8eac-4561-aed1-5a215b72798b"
       (reference "C3") (unit 1) (value "100n") (footprint "Capacitor_SMD:C_0402_1005Metric")
@@
       (reference "RN7") (unit 1) (value "47") (footprint "Resistor_SMD:R_Array_Convex_4x0603")
     )
-    (path "/8ec93f95-b65c-4f0d-a4f4-32395a9e162a/2521e63a-f996-4628-b2cc-27867cf95bd6"
-      (reference "RV1") (unit 1) (value "Volume") (footprint "")
-    )
-    (path "/8ec93f95-b65c-4f0d-a4f4-32395a9e162a/cc05c568-98be-496c-8896-a7eaf339e679"
-      (reference "RV1") (unit 2) (value "Volume") (footprint "")
-    )
     (path "/00000000-0000-0000-0000-00005f51e414/f33d3773-5cbc-4cce-b0e3-b040f6c13618"
       (reference "S1") (unit 1) (value "JS1400BFQ") (footprint "custom:SW_JS1400BFQ")
@@
       (reference "TP15") (unit 1) (value "Testpoint") (footprint "TestPoint:TestPoint_Pad_1.0x1.0mm")
     )
-    (path "/00000000-0000-0000-0000-00005fda4ddf/5cf64d14-3845-4d0f-b6c3-e8284a56ee24"
-      (reference "TP16") (unit 1) (value "Testpoint") (footprint "TestPoint:TestPoint_Pad_1.0x1.0mm")
-    )
-    (path "/00000000-0000-0000-0000-00005fda4ddf/36a6b977-0122-4af4-bfad-bdc4d857e679"
-      (reference "TP17") (unit 1) (value "Testpoint") (footprint "TestPoint:TestPoint_Pad_1.0x1.0mm")
-    )
     (path "/00000000-0000-0000-0000-000061d7b76c"

Commit message: 0 DRC errors, lots of warnings left to fix
Parts:
- removed TP19, TP20, TP26: Testpoint, TestPoint:TestPoint_Pad_1.0x1.0mm, symbol mch2021-rescue:TestPoint_Small-Connector
Changed lines of the file:
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@@
     (stroke (width 0) (type default) (color 0 0 0 0))
   )
-  (wire (pts (xy 26.67 88.9) (xy 33.02 88.9))
-    (stroke (width 0) (type default) (color 0 0 0 0))
-  )
   (wire (pts (xy 146.05 31.75) (xy 146.05 81.28))
     (stroke (width 0) (type default) (color 0 0 0 0))
@@
     (stroke (width 0) (type default) (color 0 0 0 0))
   )
-  (wire (pts (xy 26.67 99.06) (xy 27.94 99.06))
-    (stroke (width 0) (type default) (color 0 0 0 0))
-  )
   (wire (pts (xy 274.32 160.02) (xy 274.32 146.05))
     (stroke (width 0) (type default) (color 0 0 0 0))
@@
     (stroke (width 0) (type default) (color 0 0 0 0))
   )
-  (wire (pts (xy 27.94 91.44) (xy 27.94 92.71))
-    (stroke (width 0) (type default) (color 0 0 0 0))
-  )
   (wire (pts (xy 220.98 161.29) (xy 220.98 158.75))
     (stroke (width 0) (type default) (color 0 0 0 0))
@@
     (stroke (width 0) (type default) (color 0 0 0 0))
   )
-  (wire (pts (xy 26.67 91.44) (xy 27.94 91.44))
-    (stroke (width 0) (type default) (color 0 0 0 0))
-  )
   (wire (pts (xy 222.25 160.02) (xy 274.32 160.02))
     (stroke (width 0) (type default) (color 0 0 0 0))
@@
     (stroke (width 0) (type default) (color 0 0 0 0))
   )
-  (wire (pts (xy 33.02 88.9) (xy 33.02 86.36))
-    (stroke (width 0) (type default) (color 0 0 0 0))
-  )
   (wire (pts (xy 74.93 99.06) (xy 74.93 52.07))
     (stroke (width 0) (type default) (color 0 0 0 0))
@@
     (stroke (width 0) (type default) (color 0 0 0 0))
   )
-  (wire (pts (xy 27.94 99.06) (xy 27.94 100.33))
-    (stroke (width 0) (type default) (color 0 0 0 0))
-  )
   (wire (pts (xy 273.05 143.51) (xy 262.89 143.51))
     (stroke (width 0) (type default) (color 0 0 0 0))
@@
     (pin "1")
   )
-  (symbol (lib_id "mch2021-rescue:+3.3V-power") (at 33.02 86.36 0) (unit 1)
-    (in_bom yes) (on_board yes)
-    (property "Reference" "#PWR0229" (id 0) (at 33.02 90.17 0)
-      (effects (font (size 1.27 1.27)) hide)
-    )
-    (property "Value" "+3.3V" (id 1) (at 33.02 82.55 0))
-    (property "Footprint" "" (id 2) (at 33.02 86.36 0)
-      (effects (font (size 1.27 1.27)) hide)
-    )
-    (property "Datasheet" "" (id 3) (at 33.02 86.36 0)
-      (effects (font (size 1.27 1.27)) hide)
-    )
-    (pin "1")
-  )
-  (symbol (lib_id "mch2021-rescue:GND-power") (at 27.94 92.71 0) (mirror y) (unit 1)
-    (in_bom yes) (on_board yes)
-    (property "Reference" "#PWR0230" (id 0) (at 27.94 99.06 0)
-      (effects (font (size 1.27 1.27)) hide)
-    )
-    (property "Value" "GND" (id 1) (at 27.813 97.1042 0))
-    (property "Footprint" "" (id 2) (at 27.94 92.71 0)
-      (effects (font (size 1.27 1.27)) hide)
-    )
-    (property "Datasheet" "" (id 3) (at 27.94 92.71 0)
-      (effects (font (size 1.27 1.27)) hide)
-    )
-    (pin "1")
-  )
   (symbol (lib_id "custom:RGB-5050-MCH") (at 165.1 156.21 90) (mirror x) (unit 1)
     (in_bom yes) (on_board yes)
@@
     (pin "1")
   )
-  (symbol (lib_id "mch2021-rescue:TestPoint_Small-Connector") (at 26.67 91.44 0) (unit 1)
-    (in_bom yes) (on_board yes)
-    (property "Reference" "TP20" (id 0) (at 21.59 91.44 0)
-      (effects (font (size 1.27 1.27)) (justify left))
-    )
-    (property "Value" "Testpoint" (id 1) (at 27.8892 92.583 0)
-      (effects (font (size 1.27 1.27)) (justify left) hide)
-    )
-    (property "Footprint" "TestPoint:TestPoint_Pad_1.0x1.0mm" (id 2) (at 31.75 91.44 0)
-      (effects (font (size 1.27 1.27)) hide)
-    )
-    (property "Datasheet" "" (id 3) (at 31.75 91.44 0)
-      (effects (font (size 1.27 1.27)) hide)
-    )
-    (property "Category" "Testpoints" (id 4) (at 26.67 91.44 0)
-      (effects (font (size 1.27 1.27)) hide)
-    )
-    (property "Buy early" "N" (id 5) (at 26.67 91.44 0)
-      (effects (font (size 1.27 1.27)) hide)
-    )
-    (property "Sponsored" "N" (id 6) (at 26.67 91.44 0)
-      (effects (font (size 1.27 1.27)) hide)
-    )
-    (pin "1")
-  )
-  (symbol (lib_id "mch2021-rescue:TestPoint_Small-Connector") (at 26.67 88.9 0) (unit 1)
-    (in_bom yes) (on_board yes)
-    (property "Reference" "TP19" (id 0) (at 21.59 88.9 0)
-      (effects (font (size 1.27 1.27)) (justify left))
-    )
-    (property "Value" "Testpoint" (id 1) (at 27.8892 90.043 0)
-      (effects (font (size 1.27 1.27)) (justify left) hide)
-    )
-    (property "Footprint" "TestPoint:TestPoint_Pad_1.0x1.0mm" (id 2) (at 31.75 88.9 0)
-      (effects (font (size 1.27 1.27)) hide)
-    )
-    (property "Datasheet" "" (id 3) (at 31.75 88.9 0)
-      (effects (font (size 1.27 1.27)) hide)
-    )
-    (property "Category" "Testpoints" (id 4) (at 26.67 88.9 0)
-      (effects (font (size 1.27 1.27)) hide)
-    )
-    (property "Buy early" "N" (id 5) (at 26.67 88.9 0)
-      (effects (font (size 1.27 1.27)) hide)
-    )
-    (property "Sponsored" "N" (id 6) (at 26.67 88.9 0)
-      (effects (font (size 1.27 1.27)) hide)
-    )
-    (pin "1")
-  )
   (symbol (lib_id "mch2021-rescue:TestPoint_Small-Connector") (at 26.67 86.36 0) (unit 1)
     (in_bom yes) (on_board yes)
@@
     (pin "1")
   )
-  (symbol (lib_id "mch2021-rescue:GND-power") (at 27.94 100.33 0) (mirror y) (unit 1)
-    (in_bom yes) (on_board yes)
-    (property "Reference" "#PWR0227" (id 0) (at 27.94 106.68 0)
-      (effects (font (size 1.27 1.27)) hide)
-    )
-    (property "Value" "GND" (id 1) (at 27.813 104.7242 0))
-    (property "Footprint" "" (id 2) (at 27.94 100.33 0)
-      (effects (font (size 1.27 1.27)) hide)
-    )
-    (property "Datasheet" "" (id 3) (at 27.94 100.33 0)
-      (effects (font (size 1.27 1.27)) hide)
-    )
-    (pin "1")
-  )
-  (symbol (lib_id "mch2021-rescue:TestPoint_Small-Connector") (at 26.67 99.06 0) (unit 1)
-    (in_bom yes) (on_board yes)
-    (property "Reference" "TP26" (id 0) (at 21.59 99.06 0)
-      (effects (font (size 1.27 1.27)) (justify left))
-    )
-    (property "Value" "Testpoint" (id 1) (at 27.8892 100.203 0)
-      (effects (font (size 1.27 1.27)) (justify left) hide)
-    )
-    (property "Footprint" "TestPoint:TestPoint_Pad_1.0x1.0mm" (id 2) (at 31.75 99.06 0)
-      (effects (font (size 1.27 1.27)) hide)
-    )
-    (property "Datasheet" "" (id 3) (at 31.75 99.06 0)
-      (effects (font (size 1.27 1.27)) hide)
-    )
-    (property "Category" "Testpoints" (id 4) (at 26.67 99.06 0)
-      (effects (font (size 1.27 1.27)) hide)
-    )
-    (property "Buy early" "N" (id 5) (at 26.67 99.06 0)
-      (effects (font (size 1.27 1.27)) hide)
-    )
-    (property "Sponsored" "N" (id 6) (at 26.67 99.06 0)
-      (effects (font (size 1.27 1.27)) hide)
-    )
-    (pin "1")
-  )
   (symbol (lib_id "mch2021-rescue:TestPoint_Small-Connector") (at 223.52 57.15 0) (unit 1)
     (in_bom yes) (on_board yes)
@@
       (reference "#PWR0220") (unit 1) (value "GND") (footprint "")
     )
-    (path "/00000000-0000-0000-0000-000061e7670e"
-      (reference "#PWR0227") (unit 1) (value "GND") (footprint "")
-    )
-    (path "/00000000-0000-0000-0000-0000601672c6"
-      (reference "#PWR0229") (unit 1) (value "+3.3V") (footprint "")
-    )
-    (path "/00000000-0000-0000-0000-000060195541"
-      (reference "#PWR0230") (unit 1) (value "GND") (footprint "")
-    )
     (path "/00000000-0000-0000-0000-000060c794cb/00000000-0000-0000-0000-000061828aab"
       (reference "#PWR0231") (unit 1) (value "GND") (footprint "")
@@
       (reference "TP18") (unit 1) (value "Testpoint") (footprint "TestPoint:TestPoint_Pad_1.0x1.0mm")
     )
-    (path "/00000000-0000-0000-0000-000061d7ae30"
-      (reference "TP19") (unit 1) (value "Testpoint") (footprint "TestPoint:TestPoint_Pad_1.0x1.0mm")
-    )
-    (path "/00000000-0000-0000-0000-000061d78c6a"
-      (reference "TP20") (unit 1) (value "Testpoint") (footprint "TestPoint:TestPoint_Pad_1.0x1.0mm")
-    )
     (path "/68ce16cf-1a8f-4aec-8bf9-6a83a11b2850"
       (reference "TP21") (unit 1) (value "Testpoint") (footprint "TestPoint:TestPoint_Pad_1.0x1.0mm")
@@
       (reference "TP25") (unit 1) (value "Testpoint") (footprint "TestPoint:TestPoint_Pad_1.0x1.0mm")
     )
-    (path "/00000000-0000-0000-0000-000061e76714"
-      (reference "TP26") (unit 1) (value "Testpoint") (footprint "TestPoint:TestPoint_Pad_1.0x1.0mm")
-    )
     (path "/00000000-0000-0000-0000-00005fda4ddf/7abfc6ee-4723-4e6d-af50-8af0f441c0a6"

Commit message: Last minute fixes
Parts:
- removed D1: USBLC6-4SC6, digikey-footprints:SOT23-6L, symbol mch2021-rescue:USBLC6-4SC6-dk_TVS-Diodes
- added N3: (no value), symbol mch2021-rescue:Housing-Mechanical
- added TP19, TP23, TP24, TP26, TP31, TP32, TP33: Testpoint, TestPoint:TestPoint_Pad_1.0x1.0mm, symbol mch2021-rescue:TestPoint_Small-Connector
Connections:
- net +3V3: now also TP26.1
- net ESP32/I2C_SCL: now also TP33.1
- net ESP32/I2C_SDA: now also TP32.1
- net GND: now also TP19.1, TP24.1, TP31.1
- net VIN: now also TP23.1

Commit message: Last minute changes part 2
Parts:
- N3: value (none) -> May Contain Hardware; footprint (none) -> custom:protoboard-squares-big
Changed lines of the file:
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@@
       (effects (font (size 1.27 1.27)) (justify left))
     )
-    (property "Value" "" (id 1) (at 28.0162 172.8978 0)
-      (effects (font (size 1.27 1.27)) (justify left))
-    )
-    (property "Footprint" "" (id 2) (at 25.4 170.18 0)
+    (property "Value" "May Contain Hardware" (id 1) (at 28.0162 172.8978 0)
+      (effects (font (size 1.27 1.27)) (justify left))
+    )
+    (property "Footprint" "custom:protoboard-squares-big" (id 2) (at 25.4 170.18 0)
       (effects (font (size 1.27 1.27)) hide)
     )
@@
       (reference "#PWR0232") (unit 1) (value "GND") (footprint "")
     )
+    (path "/00000000-0000-0000-0000-00005f51e414/06f35d79-701d-4668-99e8-c39281eb6d67"
+      (reference "#PWR?") (unit 1) (value "GND") (footprint "")
+    )
     (path "/00000000-0000-0000-0000-000060c789de/00000000-0000-0000-0000-00005fb6aee8"
       (reference "BT1") (unit 1) (value "LiPo") (footprint "Connector_JST:JST_PH_S3B-PH-SM4-TB_1x03-1MP_P2.00mm_Horizontal")
@@
       (reference "SW8") (unit 1) (value "Switch") (footprint "Button_Switch_SMD:SW_SPDT_PCM12")
     )
+    (path "/00000000-0000-0000-0000-00005f51e414/00feb6b8-cc6e-4a61-b51e-26371c307bb7"
+      (reference "SW?") (unit 1) (value "DNP") (footprint "custom:1TS009")
+    )
     (path "/00000000-0000-0000-0000-00005fca324a"
