File: buttons.kicad_sch (KiCad schematic)
At the start: 10 parts, among them SW1 Start, SW2 Select, SW3 Menu, SW4 Home, SW5 B, SW6 A, U4 PCA9555PW

Commit message: Remove IO expander, move around signals
Parts:
- removed C14: 100n, Capacitor_SMD:C_0402_1005Metric, symbol mch2021-rescue:C_Small-Device
- removed R30: 4.7k, Resistor_SMD:R_0402_1005Metric, symbol mch2021-rescue:R_Small-Device
- removed S1: JS1400BFQ, custom:SW_JS1400BFQ, symbol JS1400BFQ:JS1400BFQ
- removed SW1: Start, custom:1TS009, symbol mch2021-rescue:SW_Push-Switch
- removed SW2: Select, custom:1TS009, symbol mch2021-rescue:SW_Push-Switch
- removed SW3: Menu, custom:1TS009, symbol mch2021-rescue:SW_Push-Switch
- removed SW4: Home, custom:1TS009, symbol mch2021-rescue:SW_Push-Switch
- removed SW5: B, custom:1TS009, symbol mch2021-rescue:SW_Push-Switch
- removed SW6: A, custom:1TS009, symbol mch2021-rescue:SW_Push-Switch
- removed U4: PCA9555PW, Package_SO:TSSOP-24_4.4x7.8mm_P0.65mm, symbol mch2021-rescue:PCA9555PW-Interface_Expansion
Other:
- note removed: "I2C I/O expander"
