File: rp2040.kicad_sch (KiCad schematic)
At the start: 30 parts, among them Q5 Q_NMOS_GSD, U17 W25Q128JVS, U3 RP2040, Y2 12MHz

Commit message: Fix badge on battery power issue, change bootsel resistor value
Parts:
- R24: value 47 -> 1k
Changed lines of the file:
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@@
     (in_bom yes) (on_board yes)
     (property "Reference" "R24" (id 0) (at 182.88 50.8 90))
-    (property "Value" "47" (id 1) (at 182.88 53.34 90))
+    (property "Value" "1k" (id 1) (at 182.88 53.34 90))
     (property "Footprint" "Resistor_SMD:R_0402_1005Metric" (id 2) (at 182.88 51.562 90)
       (effects (font (size 1.27 1.27)) hide)

Commit message: Small fixes
Parts:
- C11, C7: value 1u -> 100n
- C62, C8: value 100n -> 1u
- Y2: LCSC C13738 -> C390764
Other:
- moved on the sheet: C11, C62, C7, C8

Commit message: Remove IO expander, move around signals
Parts:
- removed Q5: Q_NMOS_GSD, Package_TO_SOT_SMD:SOT-23, symbol mch2021-rescue:Q_NMOS_GSD-Device
- removed R22: 10k, Resistor_SMD:R_0402_1005Metric, symbol mch2021-rescue:R-Device
- removed R27: 47, Resistor_SMD:R_0402_1005Metric, symbol mch2021-rescue:R-Device
- removed R28: 100k, Resistor_SMD:R_0402_1005Metric, symbol mch2021-rescue:R-Device
- removed TP16: 4, TestPoint:TestPoint_Pad_1.0x1.0mm, symbol mch2021-rescue:TestPoint_Small-Connector
- removed TP17: 5, TestPoint:TestPoint_Pad_1.0x1.0mm, symbol mch2021-rescue:TestPoint_Small-Connector
- removed TP25: 10, TestPoint:TestPoint_Pad_1.0x1.0mm, symbol mch2021-rescue:TestPoint_Small-Connector
- added S1: JS1400BFQ, custom:SW_JS1400BFQ, symbol JS1400BFQ:JS1400BFQ
- added SW1: Start, custom:1TS009, symbol mch2021-rescue:SW_Push-Switch
- added SW2: Select, custom:1TS009, symbol mch2021-rescue:SW_Push-Switch
- added SW3: Menu, custom:1TS009, symbol mch2021-rescue:SW_Push-Switch
- added SW4: Home, custom:1TS009, symbol mch2021-rescue:SW_Push-Switch
- added SW5: B, custom:1TS009, symbol mch2021-rescue:SW_Push-Switch
- added SW6: A, custom:1TS009, symbol mch2021-rescue:SW_Push-Switch
Connections:
- net GND: now also S1.5, S1.SH1 (SHIELD), S1.SH2 (SHIELD), SW1.2, SW2.2, SW3.2, SW4.2, SW5.2, SW6.2
- net BTN_HOME: now reaches U3.13 (GPIO10)
- net BTN_HOME: now also SW4.1
- net BTN_BACK: now reaches U3.38 (GPIO26/ADC0)
- net BTN_BACK: now also SW5.1
- net BTN_START: now reaches U3.6 (GPIO4)
- net BTN_START: now also SW1.1
- net BTN_MENU: now reaches U3.7 (GPIO5)
- net BTN_MENU: now also SW3.1
- net BATT_TEMP renamed FPGA_CDONE
- net ESP32_WK renamed ESP32_IRQ
- net LCD_MODE renamed FPGA_RESET
- net LED_DATA renamed BTN_ACCEPT
- net BTN_ACCEPT: now also SW6.1
- net PWR_LED_ENABLE renamed JOY_E
- net JOY_E: now also S1.6
- net RP2040_BOOT renamed BTN_SELECT
- net BTN_SELECT: now also SW2.1
- net SPI_CS renamed JOY_D
- net JOY_D: now also S1.4
- net SPI_MISO renamed JOY_B
- net JOY_B: now also S1.2
- net SPI_MOSI renamed JOY_C
- net JOY_C: now also S1.3
- net SPI_SCK renamed JOY_A
- net JOY_A: now also S1.1
Other:
- note removed: "SPI0 SCK SPI0 TX SPI0 RX SPI0 CSn"
- note removed: "The ESP32 BL pin also serves as IRQ"

Commit message: Remove user I2C bus, connect LCD control signals to ESP32 directly, replace I2S dac
Connections:
- net EXT_SCL: no longer names the net of U3.12 (GPIO9)
- net EXT_SDA: no longer names the net of U3.11 (GPIO8)
Other:
- note added: "How can we use these pins? They can do I2C... >"
Changed lines of the file:
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@@
     (effects (font (size 0.7874 0.7874)) (justify left bottom))
+  )
+  (text "How can we use these pins? They can do I2C... >" (at 50.546 115.062 0)
+    (effects (font (size 1.27 1.27)) (justify left bottom))
   )
   (text "I2C1 SDA\nI2C1 SCL" (at 120.65 100.33 0)
@@
     )
   )
-  (global_label "EXT_SCL" (shape input) (at 101.6 115.57 180) (fields_autoplaced)
-    (effects (font (size 0.9906 0.9906)) (justify right))
-    (property "Intersheet References" "${INTERSHEET_REFS}" (id 0) (at 0 0 0)
-      (effects (font (size 1.27 1.27)) hide)
-    )
-  )
   (global_label "JOY_D" (shape input) (at 163.83 107.95 0) (fields_autoplaced)
     (effects (font (size 1.27 1.27)) (justify left))
@@
     )
   )
-  (global_label "EXT_SDA" (shape bidirectional) (at 101.6 113.03 180) (fields_autoplaced)
-    (effects (font (size 0.9906 0.9906)) (justify right))
-    (property "Intersheet References" "${INTERSHEET_REFS}" (id 0) (at 0 0 0)
-      (effects (font (size 1.27 1.27)) hide)
-    )
-  )

Commit message: Use correct flash chip for RP2040
Parts:
- U17: value W25Q128JVS -> W25Q16JVUXIQ; footprint Package_SO:SOIC-8_5.23x5.23mm_P1.27mm -> custom:PSON50P300X200X60-9N
Changed lines of the file:
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@@
     (in_bom yes) (on_board yes)
     (property "Reference" "U17" (id 0) (at 200.66 58.039 0))
-    (property "Value" "W25Q128JVS" (id 1) (at 200.66 60.3504 0))
-    (property "Footprint" "Package_SO:SOIC-8_5.23x5.23mm_P1.27mm" (id 2) (at 201.93 92.71 0)
+    (property "Value" "W25Q16JVUXIQ" (id 1) (at 200.66 60.3504 0))
+    (property "Footprint" "custom:PSON50P300X200X60-9N" (id 2) (at 201.93 92.71 0)
       (effects (font (size 1.524 1.524)) hide)
     )

Commit message: Finishing touches for audio circuit
Connections:
- net SAO_IO3: now reaches U3.11 (GPIO8)
- net SAO_IO2: now reaches U3.12 (GPIO9)
- net LCD_RESET renamed SPK_DISABLE
Other:
- note removed: "How can we use these pins? They can do I2C... >"
Changed lines of the file:
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@@
     (effects (font (size 0.7874 0.7874)) (justify left bottom))
-  )
-  (text "How can we use these pins? They can do I2C... >" (at 50.546 115.062 0)
-    (effects (font (size 1.27 1.27)) (justify left bottom))
   )
   (text "I2C1 SDA\nI2C1 SCL" (at 120.65 100.33 0)
@@
     (effects (font (size 1.27 1.27)) (justify left))
   )
+  (hierarchical_label "SAO_IO3" (shape bidirectional) (at 101.6 113.03 180)
+    (effects (font (size 1 1)) (justify right))
+  )
   (hierarchical_label "SAO_IO1" (shape bidirectional) (at 101.6 110.49 180)
     (effects (font (size 1.27 1.27)) (justify right))
@@
     (effects (font (size 1.27 1.27)) (justify left))
   )
-  (hierarchical_label "LCD_RESET" (shape output) (at 163.83 95.25 0)
-    (effects (font (size 1.27 1.27)) (justify left))
+  (hierarchical_label "SAO_IO2" (shape bidirectional) (at 101.6 115.57 180)
+    (effects (font (size 1 1)) (justify right))
   )
   (hierarchical_label "FPGA_TX" (shape input) (at 163.83 118.11 0)
@@
     (effects (font (size 1.27 1.27)) (justify left))
   )
+  (hierarchical_label "SPK_DISABLE" (shape input) (at 163.83 95.25 0)
+    (effects (font (size 1 1)) (justify left))
+  )
   (hierarchical_label "SENSE_VBAT" (shape input) (at 163.83 125.73 0)

Commit message: Bill of materials 1/2
Parts:
- C10, C9: value 22p -> (none); footprint Capacitor_SMD:C_0402_1005Metric -> (none); Category (none) -> Capacitors; LCSC C106203 -> (none); MPN CC0402JRNPO9BN220 -> (none); Sponsored N -> (none)
- C11, C13, C58, C59, C60, C61, C63, C7: value 100n -> (none); footprint Capacitor_SMD:C_0402_1005Metric -> (none); Category (none) -> Capacitors; LCSC C83056 -> (none); Sponsored N -> (none)
- C62, C8: value 1u -> (none); footprint Capacitor_SMD:C_0402_1005Metric -> (none); Category (none) -> Capacitors; LCSC C83056 -> (none); Sponsored N -> (none)
- R23: value 47 -> (none); footprint Resistor_SMD:R_0402_1005Metric -> (none); Category (none) -> Resistors; LCSC C25168 -> (none); MPN 0402WGJ0470TCE -> (none); Sponsored N -> (none)
- R24: value 1k -> (none); footprint Resistor_SMD:R_0402_1005Metric -> (none); Category (none) -> Resistors; LCSC C25168 -> (none); MPN 0402WGJ0470TCE -> (none); Sponsored N -> (none)
- R25: value 1k -> (none); footprint Resistor_SMD:R_0402_1005Metric -> (none); Category (none) -> Resistors; LCSC C226166 -> (none); MPN RC-02W1001FT -> (none); Sponsored N -> (none)
- R26: value 10k -> (none); footprint Resistor_SMD:R_0402_1005Metric -> (none); Category (none) -> Resistors; LCSC C144807 -> (none); MPN AC0402FR-0710KL -> (none); Sponsored N -> (none)
- R6, R7: value 27 -> (none); footprint Resistor_SMD:R_0402_1005Metric -> (none); Category (none) -> Resistors; Sponsored N -> (none)
- S1: value JS1400BFQ -> (none); footprint custom:SW_JS1400BFQ -> (none); Category (none) -> Buttons; MPN (none) -> SKRHABE010; Manufacturer (none) -> Alpsalpine; Sponsored N -> (none)
- SW1: value Start -> (none); footprint custom:1TS009 -> (none); Category (none) -> Buttons; Sponsored N -> (none)
- SW2: value Select -> (none); footprint custom:1TS009 -> (none); Category (none) -> Buttons; Sponsored N -> (none)
- SW3: value Menu -> (none); footprint custom:1TS009 -> (none); Category (none) -> Buttons; Sponsored N -> (none)
- SW4: value Home -> (none); footprint custom:1TS009 -> (none); Category (none) -> Buttons; Sponsored N -> (none)
- SW5: value B -> (none); footprint custom:1TS009 -> (none); Category (none) -> Buttons; Sponsored N -> (none)
- SW6: value A -> (none); footprint custom:1TS009 -> (none); Category (none) -> Buttons; Sponsored N -> (none)
- TP14: value SWDCLK -> (none); footprint TestPoint:TestPoint_Pad_1.0x1.0mm -> (none); Buy early (none) -> N; Category (none) -> Testpoints; Sponsored (none) -> N
- TP9: value SWDIO -> (none); footprint TestPoint:TestPoint_Pad_1.0x1.0mm -> (none); Buy early (none) -> N; Category (none) -> Testpoints; Sponsored (none) -> N
- U17: value W25Q16JVUXIQ -> (none); footprint custom:PSON50P300X200X60-9N -> (none); Buy early (none) -> Y; Category (none) -> ICs; LCSC C97521 -> (none); MPN W25Q128JVSIQ -> W25Q16JVUXIQ; Sponsored (none) -> Y
- U3: value RP2040 -> (none); footprint RP2040:QFN40P700X700X90-57N -> (none); Buy early (none) -> Y; Category (none) -> ICs
- Y2: value 12MHz -> (none); footprint Crystal:Crystal_SMD_3225-4Pin_3.2x2.5mm -> (none); Buy early (none) -> Y; Category (none) -> Oscillators; MPN (none) -> S3212000181080; Manufacturer (none) -> JGHC

Commit message: Add more info to BOM
Parts:
- C10, C11, C13, C58, C59, C60, C61, C62, C63, C7, C8, C9, R23, R26, R6, R7, S1: Buy early (none) -> Y; Sponsored (none) -> N
- R24, R25: Buy early (none) -> Y; LCSC (none) -> C25543; MPN (none) -> 0402WGJ0102TCE; Manufacturer (none) -> Uni-royal; Sponsored (none) -> N
- SW1, SW2, SW3, SW4, SW5, SW6: Buy early (none) -> Y; MPN (none) -> SKPMAME010; Manufacturer (none) -> Alpsalpine; Sponsored (none) -> N
