File: rp2040.kicad_sch (KiCad schematic)
At the start: 34 parts, among them Q3 AP2302B, SW1 SKPMAME010, SW2 SKPMAME010, SW3 SKPMAME010, SW4 SKPMAME010, SW5 SKPMAME010, SW6 SKPMAME010, U17 W25Q16JVUXIQ, U3 RP2040, Y2 12MHz

Commit message: Last minute fixes
Parts:
- added TP16, TP17, TP20: Testpoint, TestPoint:TestPoint_Pad_1.0x1.0mm, symbol mch2021-rescue:TestPoint_Small-Connector
Connections:
- net FPGA_CDONE: now also U3.31 (GPIO20); no longer U3.27 (GPIO16)
- net FPGA_RESET: now also U3.32 (GPIO21); no longer U3.28 (GPIO17)
- net GND: now also TP17.1, TP20.1
- net SAO_IO2: now also U3.28 (GPIO17); no longer U3.31 (GPIO20)
- net SAO_IO3: now also U3.27 (GPIO16); no longer U3.32 (GPIO21)
- net SENSE_VBAT: now also U3.41 (GPIO29/ADC3); no longer U3.40 (GPIO28/ADC2)
- net SENSE_VUSB: now also U3.40 (GPIO28/ADC2); no longer U3.41 (GPIO29/ADC3)
- net at R51.1, U3.39 (GPIO27/ADC1): now also TP16.1
Changed lines of the file:
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@@
   (junction (at 96.52 191.77) (diameter 0) (color 0 0 0 0)
   )
+  (junction (at 193.04 123.19) (diameter 0) (color 0 0 0 0)
+  )
   (junction (at 115.57 171.45) (diameter 0) (color 0 0 0 0)
   )
@@
     (stroke (width 0) (type default) (color 0 0 0 0))
   )
+  (wire (pts (xy 193.04 137.414) (xy 193.04 139.446))
+    (stroke (width 0) (type default) (color 0 0 0 0))
+  )
   (wire (pts (xy 160.02 87.63) (xy 163.83 87.63))
     (stroke (width 0) (type default) (color 0 0 0 0))
@@
     (stroke (width 0) (type default) (color 0 0 0 0))
   )
+  (wire (pts (xy 41.91 182.626) (xy 43.434 182.626))
+    (stroke (width 0) (type default) (color 0 0 0 0))
+  )
   (wire (pts (xy 105.41 171.45) (xy 115.57 171.45))
     (stroke (width 0) (type default) (color 0 0 0 0))
@@
   )
   (wire (pts (xy 172.72 64.77) (xy 189.23 64.77))
+    (stroke (width 0) (type default) (color 0 0 0 0))
+  )
+  (wire (pts (xy 43.434 182.626) (xy 43.434 184.658))
     (stroke (width 0) (type default) (color 0 0 0 0))
   )
@@
     )
   )
-  (hierarchical_label "FPGA_RESET" (shape output) (at 163.83 97.79 0)
+  (hierarchical_label "FPGA_RESET" (shape output) (at 163.83 107.95 0)
     (effects (font (size 1.27 1.27)) (justify left))
   )
@@
     (effects (font (size 1.27 1.27)) (justify left))
   )
-  (hierarchical_label "SAO_IO3" (shape bidirectional) (at 163.83 107.95 0)
+  (hierarchical_label "SAO_IO3" (shape bidirectional) (at 163.83 95.25 0)
     (effects (font (size 1 1)) (justify left))
   )
@@
     (effects (font (size 1.27 1.27)) (justify left))
   )
-  (hierarchical_label "SENSE_VUSB" (shape input) (at 163.83 128.27 0)
+  (hierarchical_label "SENSE_VUSB" (shape input) (at 163.83 125.73 0)
     (effects (font (size 1.27 1.27)) (justify left))
   )
-  (hierarchical_label "SAO_IO2" (shape bidirectional) (at 163.83 105.41 0)
+  (hierarchical_label "SAO_IO2" (shape bidirectional) (at 163.83 97.79 0)
     (effects (font (size 1 1)) (justify left))
   )
@@
     (effects (font (size 1.27 1.27)) (justify left))
   )
-  (hierarchical_label "FPGA_CDONE" (shape input) (at 163.83 95.25 0)
+  (hierarchical_label "FPGA_CDONE" (shape input) (at 163.83 105.41 0)
     (effects (font (size 1.27 1.27)) (justify left))
   )
-  (hierarchical_label "SENSE_VBAT" (shape input) (at 163.83 125.73 0)
+  (hierarchical_label "SENSE_VBAT" (shape input) (at 163.83 128.27 0)
     (effects (font (size 1.27 1.27)) (justify left))
   )
@@
     (pin "1")
   )
+  (symbol (lib_id "mch2021-rescue:GND-power") (at 193.04 139.446 0) (unit 1)
+    (in_bom yes) (on_board yes)
+    (property "Reference" "#PWR0113" (id 0) (at 193.04 145.796 0)
+      (effects (font (size 1.27 1.27)) hide)
+    )
+    (property "Value" "GND" (id 1) (at 193.167 143.8402 0))
+    (property "Footprint" "" (id 2) (at 193.04 139.446 0)
+      (effects (font (size 1.27 1.27)) hide)
+    )
+    (property "Datasheet" "" (id 3) (at 193.04 139.446 0)
+      (effects (font (size 1.27 1.27)) hide)
+    )
+    (pin "1")
+  )
   (symbol (lib_id "mch2021-rescue:SW_Push-Switch") (at 270.51 132.08 0) (unit 1)
     (in_bom yes) (on_board yes)
@@
     )
     (property "Datasheet" "" (id 3) (at 219.71 111.76 0)
+      (effects (font (size 1.27 1.27)) hide)
+    )
+    (pin "1")
+  )
+  (symbol (lib_id "mch2021-rescue:TestPoint_Small-Connector") (at 41.91 182.626 0) (unit 1)
+    (in_bom yes) (on_board yes)
+    (property "Reference" "TP20" (id 0) (at 36.83 182.626 0)
+      (effects (font (size 1.27 1.27)) (justify left))
+    )
+    (property "Value" "Testpoint" (id 1) (at 43.1292 183.769 0)
+      (effects (font (size 1.27 1.27)) (justify left) hide)
+    )
+    (property "Footprint" "TestPoint:TestPoint_Pad_1.0x1.0mm" (id 2) (at 46.99 182.626 0)
+      (effects (font (size 1.27 1.27)) hide)
+    )
+    (property "Datasheet" "" (id 3) (at 46.99 182.626 0)
+      (effects (font (size 1.27 1.27)) hide)
+    )
+    (property "Category" "Testpoints" (id 4) (at 41.91 182.626 0)
+      (effects (font (size 1.27 1.27)) hide)
+    )
+    (property "Buy early" "N" (id 5) (at 41.91 182.626 0)
+      (effects (font (size 1.27 1.27)) hide)
+    )
+    (property "Sponsored" "N" (id 6) (at 41.91 182.626 0)
+      (effects (font (size 1.27 1.27)) hide)
+    )
+    (pin "1")
+  )
+  (symbol (lib_id "mch2021-rescue:GND-power") (at 43.434 184.658 0) (mirror y) (unit 1)
+    (in_bom yes) (on_board yes)
+    (property "Reference" "#PWR0209" (id 0) (at 43.434 191.008 0)
+      (effects (font (size 1.27 1.27)) hide)
+    )
+    (property "Value" "GND" (id 1) (at 43.307 189.0522 0))
+    (property "Footprint" "" (id 2) (at 43.434 184.658 0)
+      (effects (font (size 1.27 1.27)) hide)
+    )
+    (property "Datasheet" "" (id 3) (at 43.434 184.658 0)
       (effects (font (size 1.27 1.27)) hide)
     )
@@
     (pin "3")
   )
+  (symbol (lib_id "mch2021-rescue:TestPoint_Small-Connector") (at 193.04 123.19 180) (unit 1)
+    (in_bom yes) (on_board yes)
+    (property "Reference" "TP16" (id 0) (at 198.12 123.19 0)
+      (effects (font (size 1.27 1.27)) (justify left))
+    )
+    (property "Value" "Testpoint" (id 1) (at 191.8208 122.047 0)
+      (effects (font (size 1.27 1.27)) (justify left) hide)
+    )
+    (property "Footprint" "TestPoint:TestPoint_Pad_1.0x1.0mm" (id 2) (at 187.96 123.19 0)
+      (effects (font (size 1.27 1.27)) hide)
+    )
+    (property "Datasheet" "" (id 3) (at 187.96 123.19 0)
+      (effects (font (size 1.27 1.27)) hide)
+    )
+    (property "Category" "Testpoints" (id 4) (at 193.04 123.19 0)
+      (effects (font (size 1.27 1.27)) hide)
+    )
+    (property "Buy early" "N" (id 5) (at 193.04 123.19 0)
+      (effects (font (size 1.27 1.27)) hide)
+    )
+    (property "Sponsored" "N" (id 6) (at 193.04 123.19 0)
+      (effects (font (size 1.27 1.27)) hide)
+    )
+    (pin "1")
+  )
   (symbol (lib_id "mch2021-rescue:SW_Push-Switch") (at 270.51 101.6 0) (unit 1)
     (in_bom yes) (on_board yes)
@@
     (pin "2")
   )
+  (symbol (lib_id "mch2021-rescue:TestPoint_Small-Connector") (at 193.04 137.414 180) (unit 1)
+    (in_bom yes) (on_board yes)
+    (property "Reference" "TP17" (id 0) (at 198.12 137.414 0)
+      (effects (font (size 1.27 1.27)) (justify left))
+    )
+    (property "Value" "Testpoint" (id 1) (at 191.8208 136.271 0)
+      (effects (font (size 1.27 1.27)) (justify left) hide)
+    )
+    (property "Footprint" "TestPoint:TestPoint_Pad_1.0x1.0mm" (id 2) (at 187.96 137.414 0)
+      (effects (font (size 1.27 1.27)) hide)
+    )
+    (property "Datasheet" "" (id 3) (at 187.96 137.414 0)
+      (effects (font (size 1.27 1.27)) hide)
+    )
+    (property "Category" "Testpoints" (id 4) (at 193.04 137.414 0)
+      (effects (font (size 1.27 1.27)) hide)
+    )
+    (property "Buy early" "N" (id 5) (at 193.04 137.414 0)
+      (effects (font (size 1.27 1.27)) hide)
+    )
+    (property "Sponsored" "N" (id 6) (at 193.04 137.414 0)
+      (effects (font (size 1.27 1.27)) hide)
+    )
+    (pin "1")
+  )
   (symbol (lib_id "mch2021-rescue:SW_Push-Switch") (at 270.51 91.44 0) (unit 1)

Commit message: Last minute changes part 2
Parts:
- added SW?: (no value), symbol mch2021-rescue:SW_Push-Switch
Connections:
- net GND: now also SW?.1
- net RP2040_RESET: now also SW?.2
Changed lines of the file:
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@@
+    )
+  )
+  (global_label "RP2040_RESET" (shape output) (at 36.068 68.58 90) (fields_autoplaced)
+    (effects (font (size 0.7874 0.7874)) (justify left))
+    (property "Intersheet References" "${INTERSHEET_REFS}" (id 0) (at 36.0188 58.4027 90)
+      (effects (font (size 0.7874 0.7874)) (justify left) hide)
     )
   )
@@
     (pin "1")
   )
+  (symbol (lib_id "mch2021-rescue:SW_Push-Switch") (at 36.068 73.66 90) (unit 1)
+    (in_bom yes) (on_board yes)
+    (property "Reference" "SW?" (id 0) (at 30.988 73.66 0))
+    (property "Value" "" (id 1) (at 31.1404 73.66 0)
+      (effects (font (size 1.27 1.27)) hide)
+    )
+    (property "Footprint" "" (id 2) (at 30.988 73.66 0)
+      (effects (font (size 1.27 1.27)) hide)
+    )
+    (property "Datasheet" "" (id 3) (at 30.988 73.66 0)
+      (effects (font (size 1.27 1.27)) hide)
+    )
+    (property "Sponsored" "N" (id 4) (at 36.068 73.66 0)
+      (effects (font (size 1.27 1.27)) hide)
+    )
+    (property "LCSC" "C115348" (id 5) (at 36.068 73.66 0)
+      (effects (font (size 1.27 1.27)) hide)
+    )
+    (property "Category" "Buttons" (id 6) (at 36.068 73.66 0)
+      (effects (font (size 1.27 1.27)) hide)
+    )
+    (property "Buy early" "N" (id 7) (at 36.068 73.66 0)
+      (effects (font (size 1.27 1.27)) hide)
+    )
+    (property "Description" "DNP" (id 8) (at 36.068 73.66 0)
+      (effects (font (size 1.27 1.27)) hide)
+    )
+    (property "MPN" "DNP" (id 9) (at 36.068 73.66 0)
+      (effects (font (size 1.27 1.27)) hide)
+    )
+    (property "Manufacturer" "DNP" (id 10) (at 36.068 73.66 0)
+      (effects (font (size 1.27 1.27)) hide)
+    )
+    (pin "1")
+    (pin "2")
+  )
   (symbol (lib_id "Device:LED") (at 219.71 123.19 90) (unit 1)
     (in_bom yes) (on_board yes) (fields_autoplaced)
@@
     (pin "2")
   )
+  (symbol (lib_id "mch2021-rescue:GND-power") (at 36.068 78.74 0) (unit 1)
+    (in_bom yes) (on_board yes)
+    (property "Reference" "#PWR?" (id 0) (at 36.068 85.09 0)
+      (effects (font (size 1.27 1.27)) hide)
+    )
+    (property "Value" "GND" (id 1) (at 36.195 83.1342 0))
+    (property "Footprint" "" (id 2) (at 36.068 78.74 0)
+      (effects (font (size 1.27 1.27)) hide)
+    )
+    (property "Datasheet" "" (id 3) (at 36.068 78.74 0)
+      (effects (font (size 1.27 1.27)) hide)
+    )
+    (pin "1")
+  )
   (symbol (lib_id "mch2021-rescue:SW_Push-Switch") (at 270.51 81.28 0) (unit 1)
