File: rp2040.kicad_sch (KiCad schematic)
At the start: 38 parts, among them Q3 AP2302B, SW1 SKPMAME010, SW2 SKPMAME010, SW3 SKPMAME010, SW4 SKPMAME010, SW5 SKPMAME010, SW6 SKPMAME010, SW9 DNP, U17 W25Q16JVUXIQ, U3 RP2040, Y2 12MHz

Commit message: Pre-production final design
Parts:
- added R55: (no value), symbol mch2021-rescue:R-Device
- C10, C9: value 22p -> (none); footprint Capacitor_SMD:C_0402_1005Metric -> (none)
- C11, C13, C58, C59, C60, C61, C63, C7: value 100n -> (none); footprint Capacitor_SMD:C_0402_1005Metric -> (none)
- C62, C8: value 1u -> (none); footprint Capacitor_SMD:C_0402_1005Metric -> (none)
- D8: value IR LED -> (none); footprint LED_SMD:LED_0805_2012Metric -> (none)
- Q3: value AP2302B -> (none); footprint Package_TO_SOT_SMD:SOT-23 -> (none)
- R23, R51: value 47 -> (none); footprint Resistor_SMD:R_0402_1005Metric -> (none)
- R24: value 1k -> (none); footprint Resistor_SMD:R_0402_1005Metric -> (none)
- R25: value 1k -> (none); footprint Resistor_SMD:R_0402_1005Metric -> (none); MANUFACTURER FH -> UNI-ROYAL
- R26: value 10k -> (none); footprint Resistor_SMD:R_0402_1005Metric -> (none); MANUFACTURER YAGEO -> UNI-ROYAL
- R54: value 22 -> (none); footprint Resistor_SMD:R_0402_1005Metric -> (none)
- R6, R7: value 27 -> (none); footprint Resistor_SMD:R_0402_1005Metric -> (none); MANUFACTURER BOURNS -> UNI-ROYAL
- S1: value JS1400BFQ -> (none); footprint custom:SW_JS1400BFQ -> (none)
- SW1, SW2, SW3, SW4, SW5, SW6: value SKPMAME010 -> (none); footprint custom:1TS009 -> (none)
- SW9: value DNP -> (none); footprint custom:1TS009 -> (none); LCSC C115348 -> (none)
- TP14, TP16, TP17, TP20, TP9: value Testpoint -> (none); footprint TestPoint:TestPoint_Pad_1.0x1.0mm -> (none)
- U17: value W25Q16JVUXIQ -> (none); footprint custom:PSON50P300X200X60-9N -> (none)
- U3: value RP2040 -> (none); footprint RP2040:QFN40P700X700X90-57N -> (none)
- Y2: value 12MHz -> (none); footprint Crystal:Crystal_SMD_3225-4Pin_3.2x2.5mm -> (none)
Connections:
- net GND: now also R55.2
- net at R51.1, TP16.1, U3.39 (GPIO27/ADC1): now also R55.1

Commit message: Add gerbers, add schematic, finalize design
Parts:
- C10, C9: value (none) -> 22p; footprint (none) -> Capacitor_SMD:C_0402_1005Metric
- C11, C13, C58, C59, C60, C61, C63, C7: value (none) -> 100n; footprint (none) -> Capacitor_SMD:C_0402_1005Metric
- C62, C8: value (none) -> 1u; footprint (none) -> Capacitor_SMD:C_0402_1005Metric
- D8: value (none) -> IR LED; footprint (none) -> LED_SMD:LED_0805_2012Metric
- Q3: value (none) -> AP2302B; footprint (none) -> Package_TO_SOT_SMD:SOT-23
- R23, R51: value (none) -> 47; footprint (none) -> Resistor_SMD:R_0402_1005Metric
- R24, R25: value (none) -> 1k; footprint (none) -> Resistor_SMD:R_0402_1005Metric
- R26, R55: value (none) -> 10k; footprint (none) -> Resistor_SMD:R_0402_1005Metric
- R54: value (none) -> 22; footprint (none) -> Resistor_SMD:R_0402_1005Metric
- R6, R7: value (none) -> 27; footprint (none) -> Resistor_SMD:R_0402_1005Metric
- S1: value (none) -> JS1400BFQ; footprint (none) -> custom:SW_JS1400BFQ
- SW1, SW2, SW3, SW4, SW5, SW6: value (none) -> SKPMAME010; footprint (none) -> custom:1TS009
- SW9: value (none) -> DNP; footprint (none) -> custom:1TS009
- TP14, TP16, TP17, TP20, TP9: value (none) -> Testpoint; footprint (none) -> TestPoint:TestPoint_Pad_1.0x1.0mm
- U17: value (none) -> W25Q16JVUXIQ; footprint (none) -> custom:PSON50P300X200X60-9N
- U3: value (none) -> RP2040; footprint (none) -> RP2040:QFN40P700X700X90-57N
- Y2: value (none) -> 12MHz; footprint (none) -> Crystal:Crystal_SMD_3225-4Pin_3.2x2.5mm

Commit message: Change value of R54 to 27 ohm
Parts:
- R54: value 22 -> 27; LCSC C25092 -> C25100; MPN 0402WGF220JTCE -> 0402WGF270JTCE
Changed lines of the file:
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@@
     (in_bom yes) (on_board yes)
     (property "Reference" "R54" (id 0) (at 217.17 115.57 90))
-    (property "Value" "22" (id 1) (at 219.71 115.57 90))
+    (property "Value" "27" (id 1) (at 219.71 115.57 90))
     (property "Footprint" "Resistor_SMD:R_0402_1005Metric" (id 2) (at 217.932 115.57 90)
       (effects (font (size 1.27 1.27)) hide)
     )
-    (property "Datasheet" "https://datasheet.lcsc.com/lcsc/2110252230_UNI-ROYAL-Uniroyal-Elec-0402WGF220JTCE_C25092.pdf" (id 3) (at 219.71 115.57 0)
+    (property "Datasheet" "https://datasheet.lcsc.com/lcsc/2110252230_UNI-ROYAL-Uniroyal-Elec-0402WGF270JTCE_C25100.pdf" (id 3) (at 219.71 115.57 0)
       (effects (font (size 1.27 1.27)) hide)
     )
-    (property "LCSC" "C25092" (id 4) (at 219.71 115.57 0)
+    (property "LCSC" "C25100" (id 4) (at 219.71 115.57 0)
       (effects (font (size 1.27 1.27)) hide)
     )
@@
       (effects (font (size 1.27 1.27)) hide)
     )
-    (property "MPN" "0402WGF220JTCE" (id 9) (at 219.71 115.57 0)
+    (property "MPN" "0402WGF270JTCE" (id 9) (at 219.71 115.57 0)
       (effects (font (size 1.27 1.27)) hide)
     )
