File: esp32.kicad_sch (KiCad schematic)
At the start: 21 parts, among them J5 Micro SD card, U7 ESP32-WROVER

Commit message: Remove IO expander, move around signals
Parts:
- removed R41: DNP, Resistor_SMD:R_0402_1005Metric, symbol mch2021-rescue:R-Device
- added R3: 4.7k, Resistor_SMD:R_0402_1005Metric, symbol mch2021-rescue:R-Device
Connections:
- net +3V3: now also R3.1
- net IRQ_TOUCH renamed IRQ_RP2040
- net IRQ_RP2040: now also R3.2
- net SPI_CS_STM32 renamed LED_DATA
Changed lines of the file:
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@@
   (title_block
     (title "MCH2022 badge - ESP32 microcontroller")
-    (date "2022-01-14")
-    (rev "3.1415")
+    (date "2022-03-11")
+    (rev "4")
     (company "BADGE.TEAM")
   )
@@
   )
   (junction (at 215.9 40.64) (diameter 0) (color 0 0 0 0)
+  )
+  (junction (at 163.83 132.08) (diameter 0) (color 0 0 0 0)
   )
   (junction (at 148.59 119.38) (diameter 0) (color 0 0 0 0)
@@
     (stroke (width 0) (type default) (color 0 0 0 0))
   )
+  (wire (pts (xy 163.83 132.08) (xy 170.18 132.08))
+    (stroke (width 0) (type default) (color 0 0 0 0))
+  )
   (wire (pts (xy 64.77 76.2) (xy 74.93 76.2))
     (stroke (width 0) (type default) (color 0 0 0 0))
@@
     (stroke (width 0) (type default) (color 0 0 0 0))
   )
-  (wire (pts (xy 107.95 132.08) (xy 170.18 132.08))
+  (wire (pts (xy 107.95 132.08) (xy 163.83 132.08))
     (stroke (width 0) (type default) (color 0 0 0 0))
   )
@@
     (stroke (width 0) (type default) (color 0 0 0 0))
   )
-  (wire (pts (xy 125.73 99.06) (xy 125.73 72.39))
-    (stroke (width 0) (type default) (color 0 0 0 0))
-  )
   (wire (pts (xy 107.95 78.74) (xy 170.18 78.74))
+    (stroke (width 0) (type default) (color 0 0 0 0))
+  )
+  (wire (pts (xy 163.83 72.39) (xy 163.83 132.08))
     (stroke (width 0) (type default) (color 0 0 0 0))
   )
@@
     (effects (font (size 0.9906 0.9906)) (justify right))
   )
-  (hierarchical_label "SPI_CS_STM32" (shape output) (at 170.18 109.22 0)
-    (effects (font (size 0.9906 0.9906)) (justify left))
-  )
   (hierarchical_label "EXT_I2C_SDA" (shape output) (at 170.18 121.92 0)
     (effects (font (size 0.9906 0.9906)) (justify left))
@@
     (effects (font (size 0.9906 0.9906)) (justify left))
   )
-  (hierarchical_label "IRQ_TOUCH" (shape input) (at 170.18 132.08 0)
+  (hierarchical_label "IRQ_RP2040" (shape input) (at 170.18 132.08 0)
     (effects (font (size 0.9906 0.9906)) (justify left))
   )
@@
   (hierarchical_label "EXT_I2C_SCL" (shape output) (at 170.18 119.38 0)
     (effects (font (size 0.9906 0.9906)) (justify left))
+  )
+  (hierarchical_label "LED_DATA" (shape output) (at 170.18 109.22 0)
+    (effects (font (size 1 1)) (justify left))
   )
   (hierarchical_label "SPI_CLK" (shape output) (at 170.18 106.68 0)
@@
     )
     (pin "1")
-  )
-  (symbol (lib_id "mch2021-rescue:R-Device") (at 125.73 68.58 0) (unit 1)
-    (in_bom yes) (on_board yes)
-    (property "Reference" "R41" (id 0) (at 123.19 68.58 90))
-    (property "Value" "DNP" (id 1) (at 128.27 68.58 90))
-    (property "Footprint" "Resistor_SMD:R_0402_1005Metric" (id 2) (at 123.952 68.58 90)
-      (effects (font (size 1.27 1.27)) hide)
-    )
-    (property "Datasheet" "~" (id 3) (at 125.73 68.58 0)
-      (effects (font (size 1.27 1.27)) hide)
-    )
-    (property "Price" "" (id 4) (at 125.73 68.58 0)
-      (effects (font (size 1.27 1.27)) hide)
-    )
-    (property "LCSC" "" (id 5) (at 125.73 68.58 0)
-      (effects (font (size 1.27 1.27)) hide)
-    )
-    (property "Mouser" "-" (id 6) (at 125.73 68.58 0)
-      (effects (font (size 1.27 1.27)) hide)
-    )
-    (property "Sponsored" "N" (id 7) (at 125.73 68.58 0)
-      (effects (font (size 1.27 1.27)) hide)
-    )
-    (pin "1")
-    (pin "2")
   )
   (symbol (lib_id "mch2021-rescue:ESP32-WROVER-corelib") (at 92.71 106.68 0) (unit 1)
@@
     (pin "2")
   )
-  (symbol (lib_id "mch2021-rescue:+3.3V-power") (at 125.73 64.77 0) (unit 1)
-    (in_bom yes) (on_board yes)
-    (property "Reference" "#PWR0108" (id 0) (at 125.73 68.58 0)
-      (effects (font (size 1.27 1.27)) hide)
-    )
-    (property "Value" "+3.3V" (id 1) (at 125.73 60.96 0))
-    (property "Footprint" "" (id 2) (at 125.73 64.77 0)
-      (effects (font (size 1.27 1.27)) hide)
-    )
-    (property "Datasheet" "" (id 3) (at 125.73 64.77 0)
-      (effects (font (size 1.27 1.27)) hide)
-    )
-    (pin "1")
-  )
   (symbol (lib_id "mch2021-rescue:GND-power") (at 125.73 144.78 0) (unit 1)
     (in_bom yes) (on_board yes)
@@
       (effects (font (size 1.27 1.27)) hide)
     )
+    (pin "1")
+    (pin "2")
+  )
+  (symbol (lib_id "mch2021-rescue:+3.3V-power") (at 163.83 64.77 0) (unit 1)
+    (in_bom yes) (on_board yes)
+    (property "Reference" "#PWR0149" (id 0) (at 163.83 68.58 0)
+      (effects (font (size 1.27 1.27)) hide)
+    )
+    (property "Value" "+3.3V" (id 1) (at 163.83 60.96 0))
+    (property "Footprint" "" (id 2) (at 163.83 64.77 0)
+      (effects (font (size 1.27 1.27)) hide)
+    )
+    (property "Datasheet" "" (id 3) (at 163.83 64.77 0)
+      (effects (font (size 1.27 1.27)) hide)
+    )
+    (pin "1")
+  )
+  (symbol (lib_id "mch2021-rescue:R-Device") (at 163.83 68.58 0) (unit 1)
+    (in_bom yes) (on_board yes)
+    (property "Reference" "R3" (id 0) (at 161.29 68.58 90))
+    (property "Value" "4.7k" (id 1) (at 166.37 68.58 90))
+    (property "Footprint" "Resistor_SMD:R_0402_1005Metric" (id 2) (at 162.052 68.58 90)
+      (effects (font (size 1.27 1.27)) hide)
+    )
+    (property "Datasheet" "~" (id 3) (at 163.83 68.58 0)
+      (effects (font (size 1.27 1.27)) hide)
+    )
+    (property "Price" "" (id 4) (at 163.83 68.58 0)
+      (effects (font (size 1.27 1.27)) hide)
+    )
+    (property "LCSC" "C25940" (id 5) (at 163.83 68.58 0)
+      (effects (font (size 1.27 1.27)) hide)
+    )
+    (property "Mouser" "-" (id 6) (at 163.83 68.58 0)
+      (effects (font (size 1.27 1.27)) hide)
+    )
+    (property "Sponsored" "N" (id 7) (at 163.83 68.58 0)
+      (effects (font (size 1.27 1.27)) hide)
+    )
+    (property "MANUFACTURER" "UNI-ROYAL" (id 8) (at 163.83 68.58 0)
+      (effects (font (size 1.27 1.27)) hide)
+    )
+    (property "MPN" "0402WGJ0472TCE" (id 9) (at 163.83 68.58 0)
+      (effects (font (size 1.27 1.27)) hide)
+    )

Commit message: Remove user I2C bus, connect LCD control signals to ESP32 directly, replace I2S dac
Parts:
- removed R45, R46: 4.7k, Resistor_SMD:R_0402_1005Metric, symbol mch2021-rescue:R-Device
- added C? (x2): 100n, Capacitor_SMD:C_0402_1005Metric, symbol mch2021-rescue:C-Device
- added C? (x2): 39n, symbol Device:C_Small
- added C? (x3): 100n, symbol Device:C_Small
- added C?: 1u, Capacitor_SMD:C_0402_1005Metric, symbol mch2021-rescue:C-Device
- added C? (x2): 10u, symbol Device:C_Polarized_Small
- added J?: AudioJack3, custom:Boom-audiojack-PJ-320B, symbol mch2021-rescue:AudioJack3-Connector
- added R? (x2): 10k, Resistor_SMD:R_0402_1005Metric, symbol mch2021-rescue:R-Device
- added RN?: 47, Resistor_SMD:R_Array_Convex_4x0603, symbol mch2021-rescue:R_Pack04-Device
- added U?: CS4344-CZZ, SOP50P490X110-10N, symbol CS4344-CZZ:CS4344-CZZ
Connections:
- net +3V3: now also C?.1, C?.1, C?.1, U?.9 (VA)
- net GND: now also C?.1, C?.1, C?.2, C?.2, C?.2, C?.2, C?.2, C?.2, J?.S, U?.8 (GND)
- net ESP32_BL renamed ESP_I2S_MCLK
- net ESP_I2S_MCLK: now also RN?.8 (R1.2)
- net EXT_I2C_SCL renamed LCD_RESET
- net EXT_I2C_SDA renamed LCD_MODE
- net SPI_CS_LCD renamed LCD_CS
- new net: RN?.4 (R4.1), U?.1 (SDIN)
- new net: C?.1, U?.10 (AOUTR)
- new net: RN?.3 (R3.1), U?.2 (~{DEM}/SCLK)
- new net: RN?.2 (R2.1), U?.3 (LRCK)
- new net: RN?.1 (R1.1), U?.4 (MCLK)
- new net: C?.1, C?.1, U?.5 (VQ)
- new net: C?.1, U?.6 (FILT+)
- new net: C?.2, U?.7 (AOUTL)
- new net: C?.1, R?.1
- new net: C?.2, R?.1
- new net AUDIO_L: C?.2, J?.T, R?.2
- new net AUDIO_R: C?.2, J?.R, R?.2
- new net ESP_I2S_CLK: RN?.6 (R3.2)
- new net ESP_I2S_DATA: RN?.5 (R4.2)
- new net ESP_I2S_LR: RN?.7 (R2.2)
Other:
- note added: "-------- To-do: I2S testpoints --------"
- note added: "-------- To-do: amplifier --------"
- note added: "ESP32 microcontroller, SD card and audio output"
- note removed: "ESP32 microcontroller"
- moved on the sheet: C23, R3, R37, R38, R39, R40, R42, R43, R44, U7

Commit message: Use correct flash chip for RP2040
Parts:
- C14, C33, C4, C47, C5, C51, C6: renamed from C?; footprint (none) -> Capacitor_SMD:C_0402_1005Metric
- U1: renamed from U?; footprint SOP50P490X110-10N -> CS4344-CZZ:SOP50P490X110-10N
- gave numbers to parts that had none: 7

Commit message: Add amplifier and spekaer, fixes
Parts:
- removed C1: 1u, Capacitor_SMD:C_0402_1005Metric, symbol mch2021-rescue:C-Device
- removed C14, C33, C4: 100n, Capacitor_SMD:C_0402_1005Metric, symbol Device:C_Small
- removed C2, C3: 100n, Capacitor_SMD:C_0402_1005Metric, symbol mch2021-rescue:C-Device
- removed C47, C51: 39n, Capacitor_SMD:C_0402_1005Metric, symbol Device:C_Small
- removed C5, C6: 10u, Capacitor_SMD:C_0402_1005Metric, symbol Device:C_Polarized_Small
- removed J1: AudioJack3, custom:Boom-audiojack-PJ-320B, symbol mch2021-rescue:AudioJack3-Connector
- removed R27, R28: 10k, Resistor_SMD:R_0402_1005Metric, symbol mch2021-rescue:R-Device
- removed RN7: 47, Resistor_SMD:R_Array_Convex_4x0603, symbol mch2021-rescue:R_Pack04-Device
- removed U1: CS4344-CZZ, CS4344-CZZ:SOP50P490X110-10N, symbol CS4344-CZZ:CS4344-CZZ
Connections:
- net ESP_I2S_MCLK renamed ESP32_BL
Other:
- note removed: "-------- To-do: I2S testpoints --------"
- note removed: "-------- To-do: amplifier --------"

Commit message: Bill of materials 1/2
Parts:
- C23, C24: value 100n -> (none); footprint Capacitor_SMD:C_0402_1005Metric -> (none); Category (none) -> Capacitors; LCSC C83056 -> (none); Sponsored N -> (none)
- C25: value 10u -> (none); footprint Capacitor_SMD:C_0402_1005Metric -> (none); Category (none) -> Capacitors; LCSC C15525 -> (none); Sponsored N -> (none)
- J5: value Micro SD card -> (none); footprint custom:MicroSD-SOFNG-TF-002-H18 -> (none); Category (none) -> Connectors; Manufacturer (none) -> SOFNG; Sponsored N -> (none)
- R10, R11, R37, R38, R50, R77, R8, R9: value 10k -> (none); footprint Resistor_SMD:R_0402_1005Metric -> (none); Category (none) -> Resistors; LCSC C144807 -> (none); MPN AC0402FR-0710KL -> (none); Sponsored N -> (none)
- R3, R40, R43, R44: value 4.7k -> (none); footprint Resistor_SMD:R_0402_1005Metric -> (none); Category (none) -> Resistors; Sponsored N -> (none)
- R39, R42: value 45.3k -> (none); footprint Resistor_SMD:R_0402_1005Metric -> (none); Category (none) -> Resistors; Sponsored N -> (none)
- U7: value ESP32-WROVER -> (none); footprint custom:ESP32-WROVER -> (none); Buy early (none) -> N; Category (none) -> ICs

Commit message: Add more info to BOM
Parts:
- C23, C24, C25, J5, R10, R11, R37, R38, R39, R42, R50, R77, R8, R9: Buy early (none) -> Y; Sponsored (none) -> N
- R3, R40, R43, R44: Buy early (none) -> Y; Manufacturer (none) -> Uni-royal; Sponsored (none) -> N

Commit message: Add passives to BOM
Parts:
- C23, C24: LCSC (none) -> C307331; MPN (none) -> CL05B104KB54PNC; Manufacturer (none) -> Samsung Electro-Mechanics; Minimal voltage rating (none) -> 10; Voltage rating (none) -> 50
- C25: LCSC (none) -> C15525; MPN (none) -> CL05A106MQ5NUNC; Manufacturer (none) -> Samsung Electro-Mechanics; Minimal voltage rating (none) -> 6; Voltage rating (none) -> 6.3
- R10, R11, R37, R38, R50, R77, R8, R9: LCSC (none) -> C25744; MPN (none) -> 0402WGF1002TCE; Manufacturer (none) -> Uni-royal
- R3, R40, R43, R44: LCSC C25940 -> C25900; MPN 0402WGJ0472TCE -> 0402WGF4701TCE
- R39, R42: Manufacturer (none) -> Uni-royal
