File: esp32.kicad_sch (KiCad schematic)
At the start: 19 parts

Commit message: Artwork stuff
Parts:
- C23, C24: value (none) -> 100n; footprint (none) -> Capacitor_SMD:C_0402_1005Metric
- C25: value (none) -> 10u; footprint (none) -> Capacitor_SMD:C_0402_1005Metric
- J5: value (none) -> Micro SD card; footprint (none) -> custom:MicroSD-SOFNG-TF-002-H18
- R10, R11, R37, R38, R50, R77, R8, R9: value (none) -> 10k; footprint (none) -> Resistor_SMD:R_0402_1005Metric
- R3, R40, R43, R44: value (none) -> 4.7k; footprint (none) -> Resistor_SMD:R_0402_1005Metric
- R39, R42: value (none) -> 45.3k; footprint (none) -> Resistor_SMD:R_0402_1005Metric
- U7: value (none) -> ESP32-WROVER; footprint (none) -> custom:ESP32-WROVER
Changed lines of the file:
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@@
     (in_bom yes) (on_board yes)
     (property "Reference" "R44" (id 0) (at 126.365 30.48 90))
-    (property "Value" "" (id 1) (at 131.445 30.48 90))
-    (property "Footprint" "" (id 2) (at 127.127 30.48 90)
+    (property "Value" "4.7k" (id 1) (at 131.445 30.48 90))
+    (property "Footprint" "Resistor_SMD:R_0402_1005Metric" (id 2) (at 127.127 30.48 90)
       (effects (font (size 1.27 1.27)) hide)
     )
@@
     (in_bom yes) (on_board yes)
     (property "Reference" "R43" (id 0) (at 118.745 30.48 90))
-    (property "Value" "" (id 1) (at 123.825 30.48 90))
-    (property "Footprint" "" (id 2) (at 119.507 30.48 90)
+    (property "Value" "4.7k" (id 1) (at 123.825 30.48 90))
+    (property "Footprint" "Resistor_SMD:R_0402_1005Metric" (id 2) (at 119.507 30.48 90)
       (effects (font (size 1.27 1.27)) hide)
     )
@@
     (in_bom yes) (on_board yes)
     (property "Reference" "R38" (id 0) (at 95.885 30.48 90))
-    (property "Value" "" (id 1) (at 100.965 30.48 90))
-    (property "Footprint" "" (id 2) (at 96.647 30.48 90)
+    (property "Value" "10k" (id 1) (at 100.965 30.48 90))
+    (property "Footprint" "Resistor_SMD:R_0402_1005Metric" (id 2) (at 96.647 30.48 90)
       (effects (font (size 1.27 1.27)) hide)
     )
@@
     (in_bom yes) (on_board yes)
     (property "Reference" "R37" (id 0) (at 60.325 29.21 90))
-    (property "Value" "" (id 1) (at 65.405 29.21 90))
-    (property "Footprint" "" (id 2) (at 61.087 29.21 90)
+    (property "Value" "10k" (id 1) (at 65.405 29.21 90))
+    (property "Footprint" "Resistor_SMD:R_0402_1005Metric" (id 2) (at 61.087 29.21 90)
       (effects (font (size 1.27 1.27)) hide)
     )
@@
       (effects (font (size 1.27 1.27)) (justify left))
     )
-    (property "Value" "" (id 1) (at 170.561 186.563 0)
+    (property "Value" "10u" (id 1) (at 170.561 186.563 0)
       (effects (font (size 1.27 1.27)) (justify left))
     )
-    (property "Footprint" "" (id 2) (at 168.6052 189.23 0)
+    (property "Footprint" "Capacitor_SMD:C_0402_1005Metric" (id 2) (at 168.6052 189.23 0)
       (effects (font (size 1.27 1.27)) hide)
     )
@@
       (effects (font (size 1.27 1.27)) (justify left))
     )
-    (property "Value" "" (id 1) (at 55.626 58.293 0)
+    (property "Value" "100n" (id 1) (at 55.626 58.293 0)
       (effects (font (size 1.27 1.27)) (justify left))
     )
-    (property "Footprint" "" (id 2) (at 53.6702 60.96 0)
+    (property "Footprint" "Capacitor_SMD:C_0402_1005Metric" (id 2) (at 53.6702 60.96 0)
       (effects (font (size 1.27 1.27)) hide)
     )
@@
     (in_bom yes) (on_board yes)
     (property "Reference" "U7" (id 0) (at 89.535 31.75 0))
-    (property "Value" "" (id 1) (at 89.535 34.29 0))
-    (property "Footprint" "" (id 2) (at 80.645 106.68 0)
+    (property "Value" "ESP32-WROVER" (id 1) (at 89.535 34.29 0))
+    (property "Footprint" "custom:ESP32-WROVER" (id 2) (at 80.645 106.68 0)
       (effects (font (size 1.27 1.27)) hide)
     )
@@
       (effects (font (size 1.27 1.27)) (justify left))
     )
-    (property "Value" "" (id 1) (at 159.131 186.563 0)
+    (property "Value" "100n" (id 1) (at 159.131 186.563 0)
       (effects (font (size 1.27 1.27)) (justify left))
     )
-    (property "Footprint" "" (id 2) (at 157.1752 189.23 0)
+    (property "Footprint" "Capacitor_SMD:C_0402_1005Metric" (id 2) (at 157.1752 189.23 0)
       (effects (font (size 1.27 1.27)) hide)
     )
@@
     (in_bom yes) (on_board yes)
     (property "Reference" "R42" (id 0) (at 111.125 102.87 90))
-    (property "Value" "" (id 1) (at 116.205 102.87 90))
-    (property "Footprint" "" (id 2) (at 111.887 102.87 90)
+    (property "Value" "45.3k" (id 1) (at 116.205 102.87 90))
+    (property "Footprint" "Resistor_SMD:R_0402_1005Metric" (id 2) (at 111.887 102.87 90)
       (effects (font (size 1.27 1.27)) hide)
     )
@@
     (in_bom yes) (on_board yes)
     (property "Reference" "R39" (id 0) (at 95.885 102.87 90))
-    (property "Value" "" (id 1) (at 100.965 102.87 90))
-    (property "Footprint" "" (id 2) (at 96.647 102.87 90)
+    (property "Value" "45.3k" (id 1) (at 100.965 102.87 90))
+    (property "Footprint" "Resistor_SMD:R_0402_1005Metric" (id 2) (at 96.647 102.87 90)
       (effects (font (size 1.27 1.27)) hide)
     )
@@
     (in_bom yes) (on_board yes)
     (property "Reference" "R40" (id 0) (at 103.505 102.87 90))
-    (property "Value" "" (id 1) (at 108.585 102.87 90))
-    (property "Footprint" "" (id 2) (at 104.267 102.87 90)
+    (property "Value" "4.7k" (id 1) (at 108.585 102.87 90))
+    (property "Footprint" "Resistor_SMD:R_0402_1005Metric" (id 2) (at 104.267 102.87 90)
       (effects (font (size 1.27 1.27)) hide)
     )
@@
     (in_bom yes) (on_board yes)
     (property "Reference" "J5" (id 0) (at 232.41 22.86 0))
-    (property "Value" "" (id 1) (at 256.54 38.1 0))
-    (property "Footprint" "" (id 2) (at 279.4 30.48 0)
+    (property "Value" "Micro SD card" (id 1) (at 256.54 38.1 0))
+    (property "Footprint" "custom:MicroSD-SOFNG-TF-002-H18" (id 2) (at 279.4 30.48 0)
       (effects (font (size 1.27 1.27)) hide)
     )
@@
     (in_bom yes) (on_board yes)
     (property "Reference" "R77" (id 0) (at 224.79 29.21 90))
-    (property "Value" "" (id 1) (at 223.52 25.4 90))
-    (property "Footprint" "" (id 2) (at 221.742 25.4 90)
+    (property "Value" "10k" (id 1) (at 223.52 25.4 90))
+    (property "Footprint" "Resistor_SMD:R_0402_1005Metric" (id 2) (at 221.742 25.4 90)
       (effects (font (size 1.27 1.27)) hide)
     )
@@
     (in_bom yes) (on_board yes)
     (property "Reference" "R50" (id 0) (at 222.25 29.21 90))
-    (property "Value" "" (id 1) (at 220.98 25.4 90))
-    (property "Footprint" "" (id 2) (at 219.202 25.4 90)
+    (property "Value" "10k" (id 1) (at 220.98 25.4 90))
+    (property "Footprint" "Resistor_SMD:R_0402_1005Metric" (id 2) (at 219.202 25.4 90)
       (effects (font (size 1.27 1.27)) hide)
     )
@@
     (in_bom yes) (on_board yes)
     (property "Reference" "R11" (id 0) (at 219.71 29.21 90))
-    (property "Value" "" (id 1) (at 218.44 25.4 90))
-    (property "Footprint" "" (id 2) (at 216.662 25.4 90)
+    (property "Value" "10k" (id 1) (at 218.44 25.4 90))
+    (property "Footprint" "Resistor_SMD:R_0402_1005Metric" (id 2) (at 216.662 25.4 90)
       (effects (font (size 1.27 1.27)) hide)
     )
@@
     (in_bom yes) (on_board yes)
     (property "Reference" "R9" (id 0) (at 214.63 29.21 90))
-    (property "Value" "" (id 1) (at 213.36 25.4 90))
-    (property "Footprint" "" (id 2) (at 211.582 25.4 90)
+    (property "Value" "10k" (id 1) (at 213.36 25.4 90))
+    (property "Footprint" "Resistor_SMD:R_0402_1005Metric" (id 2) (at 211.582 25.4 90)
       (effects (font (size 1.27 1.27)) hide)
     )
@@
     (in_bom yes) (on_board yes)
     (property "Reference" "R10" (id 0) (at 217.17 29.21 90))
-    (property "Value" "" (id 1) (at 215.9 25.4 90))
-    (property "Footprint" "" (id 2) (at 214.122 25.4 90)
+    (property "Value" "10k" (id 1) (at 215.9 25.4 90))
+    (property "Footprint" "Resistor_SMD:R_0402_1005Metric" (id 2) (at 214.122 25.4 90)
       (effects (font (size 1.27 1.27)) hide)
     )
@@
     (in_bom yes) (on_board yes)
     (property "Reference" "R8" (id 0) (at 212.09 29.21 90))
-    (property "Value" "" (id 1) (at 210.82 25.4 90))
-    (property "Footprint" "" (id 2) (at 209.042 25.4 90)
+    (property "Value" "10k" (id 1) (at 210.82 25.4 90))
+    (property "Footprint" "Resistor_SMD:R_0402_1005Metric" (id 2) (at 209.042 25.4 90)
       (effects (font (size 1.27 1.27)) hide)
     )
@@
     (in_bom yes) (on_board yes)
     (property "Reference" "R3" (id 0) (at 149.225 30.48 90))
-    (property "Value" "" (id 1) (at 154.305 30.48 90))
-    (property "Footprint" "" (id 2) (at 149.987 30.48 90)
-      (effects (font (size 1.27 1.27)) hide)
-    )
+    (property "Value" "4.7k" (id 1) (at 154.305 30.48 90))
+    (property "Footprint" "Resistor_SMD:R_0402_1005Metric" (id 2) (at 149.987 30.48 90)
+      (effects (font (size 1.27 1.27)) hide)
+    )

Commit message: Swap led data and sd power on ESP32, add speaker grill
Connections:
- net LED_DATA: now also U7.29 (IO5); no longer U7.31 (IO19)
- net SD_POWER: now also U7.31 (IO19); no longer U7.29 (IO5)
Changed lines of the file:
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@@
     (effects (font (size 0.9906 0.9906)) (justify left))
   )
-  (hierarchical_label "SD_POWER" (shape output) (at 158.115 50.8 0)
+  (hierarchical_label "SD_POWER" (shape output) (at 158.115 71.12 0)
     (effects (font (size 0.9906 0.9906)) (justify left))
   )
@@
     (effects (font (size 0.9906 0.9906)) (justify left))
   )
-  (hierarchical_label "LED_DATA" (shape output) (at 158.115 71.12 0)
+  (hierarchical_label "LED_DATA" (shape output) (at 158.115 50.8 0)
     (effects (font (size 1 1)) (justify left))
   )

Commit message: Small last minute tweaks
Connections:
- net I2S_CLK: now also U7.26 (IO4); no longer R40.1, U7.14 (IO12)
- net I2S_LR: now also R40.1, U7.14 (IO12); no longer U7.26 (IO4)

Commit message: Pre-production final design
Parts:
- C23, C24: value 100n -> (none); footprint Capacitor_SMD:C_0402_1005Metric -> (none)
- C25: value 10u -> (none); footprint Capacitor_SMD:C_0402_1005Metric -> (none)
- J5: value Micro SD card -> (none); footprint custom:MicroSD-SOFNG-TF-002-H18 -> (none)
- R10, R11, R37, R38, R50, R77, R8, R9: value 10k -> (none); footprint Resistor_SMD:R_0402_1005Metric -> (none); MANUFACTURER YAGEO -> UNI-ROYAL
- R3, R40, R43, R44: value 4.7k -> (none); footprint Resistor_SMD:R_0402_1005Metric -> (none)
- R39, R42: value 45.3k -> (none); footprint Resistor_SMD:R_0402_1005Metric -> (none)
- U7: value ESP32-WROVER -> (none); footprint custom:ESP32-WROVER -> (none)

Commit message: Add gerbers, add schematic, finalize design
Parts:
- C23, C24: value (none) -> 100n; footprint (none) -> Capacitor_SMD:C_0402_1005Metric
- C25: value (none) -> 10u; footprint (none) -> Capacitor_SMD:C_0402_1005Metric
- J5: value (none) -> Micro SD card; footprint (none) -> custom:MicroSD-SOFNG-TF-002-H18
- R10, R11, R37, R38, R50, R77, R8, R9: value (none) -> 10k; footprint (none) -> Resistor_SMD:R_0402_1005Metric
- R3, R40, R43, R44: value (none) -> 4.7k; footprint (none) -> Resistor_SMD:R_0402_1005Metric
- R39, R42: value (none) -> 45.3k; footprint (none) -> Resistor_SMD:R_0402_1005Metric
- U7: value (none) -> ESP32-WROVER; footprint (none) -> custom:ESP32-WROVER
Changed lines of the file:
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@@
     (title "MCH2022 badge - ESP32 microcontroller")
     (date "2022-04-24")
-    (rev "Pre-production final")
+    (rev "Final")
     (company "BADGE.TEAM")
+    (comment 1 "License: CERN Open Hardware Licence Version 2 - Permissive")
+    (comment 2 "Contact: renze@badge.team")
+    (comment 3 "Website: mch2022.org / badge.team")
+    (comment 4 "Event badge for May Contain Hackers 2022")
   )
   (junction (at 218.44 35.56) (diameter 0) (color 0 0 0 0)
@@
     (in_bom yes) (on_board yes)
     (property "Reference" "R44" (id 0) (at 126.492 30.48 90))
-    (property "Value" "" (id 1) (at 131.572 30.48 90))
-    (property "Footprint" "" (id 2) (at 127.254 30.48 90)
+    (property "Value" "4.7k" (id 1) (at 131.572 30.48 90))
+    (property "Footprint" "Resistor_SMD:R_0402_1005Metric" (id 2) (at 127.254 30.48 90)
       (effects (font (size 1.27 1.27)) hide)
     )
@@
     (in_bom yes) (on_board yes)
     (property "Reference" "R43" (id 0) (at 118.872 30.48 90))
-    (property "Value" "" (id 1) (at 123.952 30.48 90))
-    (property "Footprint" "" (id 2) (at 119.634 30.48 90)
+    (property "Value" "4.7k" (id 1) (at 123.952 30.48 90))
+    (property "Footprint" "Resistor_SMD:R_0402_1005Metric" (id 2) (at 119.634 30.48 90)
       (effects (font (size 1.27 1.27)) hide)
     )
@@
     (in_bom yes) (on_board yes)
     (property "Reference" "R38" (id 0) (at 96.012 30.48 90))
-    (property "Value" "" (id 1) (at 101.092 30.48 90))
-    (property "Footprint" "" (id 2) (at 96.774 30.48 90)
+    (property "Value" "10k" (id 1) (at 101.092 30.48 90))
+    (property "Footprint" "Resistor_SMD:R_0402_1005Metric" (id 2) (at 96.774 30.48 90)
       (effects (font (size 1.27 1.27)) hide)
     )
@@
     (in_bom yes) (on_board yes)
     (property "Reference" "R37" (id 0) (at 60.452 29.21 90))
-    (property "Value" "" (id 1) (at 65.532 29.21 90))
-    (property "Footprint" "" (id 2) (at 61.214 29.21 90)
+    (property "Value" "10k" (id 1) (at 65.532 29.21 90))
+    (property "Footprint" "Resistor_SMD:R_0402_1005Metric" (id 2) (at 61.214 29.21 90)
       (effects (font (size 1.27 1.27)) hide)
     )
@@
       (effects (font (size 1.27 1.27)) (justify left))
     )
-    (property "Value" "" (id 1) (at 170.561 186.563 0)
+    (property "Value" "10u" (id 1) (at 170.561 186.563 0)
       (effects (font (size 1.27 1.27)) (justify left))
     )
-    (property "Footprint" "" (id 2) (at 168.6052 189.23 0)
+    (property "Footprint" "Capacitor_SMD:C_0402_1005Metric" (id 2) (at 168.6052 189.23 0)
       (effects (font (size 1.27 1.27)) hide)
     )
@@
       (effects (font (size 1.27 1.27)) (justify left))
     )
-    (property "Value" "" (id 1) (at 55.753 58.293 0)
+    (property "Value" "100n" (id 1) (at 55.753 58.293 0)
       (effects (font (size 1.27 1.27)) (justify left))
     )
-    (property "Footprint" "" (id 2) (at 53.7972 60.96 0)
+    (property "Footprint" "Capacitor_SMD:C_0402_1005Metric" (id 2) (at 53.7972 60.96 0)
       (effects (font (size 1.27 1.27)) hide)
     )
@@
     (in_bom yes) (on_board yes)
     (property "Reference" "U7" (id 0) (at 89.662 31.75 0))
-    (property "Value" "" (id 1) (at 89.662 34.29 0))
-    (property "Footprint" "" (id 2) (at 80.772 106.68 0)
+    (property "Value" "ESP32-WROVER" (id 1) (at 89.662 34.29 0))
+    (property "Footprint" "custom:ESP32-WROVER" (id 2) (at 80.772 106.68 0)
       (effects (font (size 1.27 1.27)) hide)
     )
@@
       (effects (font (size 1.27 1.27)) (justify left))
     )
-    (property "Value" "" (id 1) (at 159.131 186.563 0)
+    (property "Value" "100n" (id 1) (at 159.131 186.563 0)
       (effects (font (size 1.27 1.27)) (justify left))
     )
-    (property "Footprint" "" (id 2) (at 157.1752 189.23 0)
+    (property "Footprint" "Capacitor_SMD:C_0402_1005Metric" (id 2) (at 157.1752 189.23 0)
       (effects (font (size 1.27 1.27)) hide)
     )
@@
     (in_bom yes) (on_board yes)
     (property "Reference" "R42" (id 0) (at 111.252 102.87 90))
-    (property "Value" "" (id 1) (at 116.332 102.87 90))
-    (property "Footprint" "" (id 2) (at 112.014 102.87 90)
+    (property "Value" "45.3k" (id 1) (at 116.332 102.87 90))
+    (property "Footprint" "Resistor_SMD:R_0402_1005Metric" (id 2) (at 112.014 102.87 90)
       (effects (font (size 1.27 1.27)) hide)
     )
@@
     (in_bom yes) (on_board yes)
     (property "Reference" "R39" (id 0) (at 96.012 102.87 90))
-    (property "Value" "" (id 1) (at 101.092 102.87 90))
-    (property "Footprint" "" (id 2) (at 96.774 102.87 90)
+    (property "Value" "45.3k" (id 1) (at 101.092 102.87 90))
+    (property "Footprint" "Resistor_SMD:R_0402_1005Metric" (id 2) (at 96.774 102.87 90)
       (effects (font (size 1.27 1.27)) hide)
     )
@@
     (in_bom yes) (on_board yes)
     (property "Reference" "R40" (id 0) (at 103.632 102.87 90))
-    (property "Value" "" (id 1) (at 108.712 102.87 90))
-    (property "Footprint" "" (id 2) (at 104.394 102.87 90)
+    (property "Value" "4.7k" (id 1) (at 108.712 102.87 90))
+    (property "Footprint" "Resistor_SMD:R_0402_1005Metric" (id 2) (at 104.394 102.87 90)
       (effects (font (size 1.27 1.27)) hide)
     )
@@
     (in_bom yes) (on_board yes)
     (property "Reference" "J5" (id 0) (at 232.41 22.86 0))
-    (property "Value" "" (id 1) (at 256.54 38.1 0))
-    (property "Footprint" "" (id 2) (at 279.4 30.48 0)
+    (property "Value" "Micro SD card" (id 1) (at 256.54 38.1 0))
+    (property "Footprint" "custom:MicroSD-SOFNG-TF-002-H18" (id 2) (at 279.4 30.48 0)
       (effects (font (size 1.27 1.27)) hide)
     )
@@
     (in_bom yes) (on_board yes)
     (property "Reference" "R77" (id 0) (at 224.79 29.21 90))
-    (property "Value" "" (id 1) (at 223.52 25.4 90))
-    (property "Footprint" "" (id 2) (at 221.742 25.4 90)
+    (property "Value" "10k" (id 1) (at 223.52 25.4 90))
+    (property "Footprint" "Resistor_SMD:R_0402_1005Metric" (id 2) (at 221.742 25.4 90)
       (effects (font (size 1.27 1.27)) hide)
     )
@@
     (in_bom yes) (on_board yes)
     (property "Reference" "R50" (id 0) (at 222.25 29.21 90))
-    (property "Value" "" (id 1) (at 220.98 25.4 90))
-    (property "Footprint" "" (id 2) (at 219.202 25.4 90)
+    (property "Value" "10k" (id 1) (at 220.98 25.4 90))
+    (property "Footprint" "Resistor_SMD:R_0402_1005Metric" (id 2) (at 219.202 25.4 90)
       (effects (font (size 1.27 1.27)) hide)
     )
@@
     (in_bom yes) (on_board yes)
     (property "Reference" "R11" (id 0) (at 219.71 29.21 90))
-    (property "Value" "" (id 1) (at 218.44 25.4 90))
-    (property "Footprint" "" (id 2) (at 216.662 25.4 90)
+    (property "Value" "10k" (id 1) (at 218.44 25.4 90))
+    (property "Footprint" "Resistor_SMD:R_0402_1005Metric" (id 2) (at 216.662 25.4 90)
       (effects (font (size 1.27 1.27)) hide)
     )
@@
     (in_bom yes) (on_board yes)
     (property "Reference" "R9" (id 0) (at 214.63 29.21 90))
-    (property "Value" "" (id 1) (at 213.36 25.4 90))
-    (property "Footprint" "" (id 2) (at 211.582 25.4 90)
+    (property "Value" "10k" (id 1) (at 213.36 25.4 90))
+    (property "Footprint" "Resistor_SMD:R_0402_1005Metric" (id 2) (at 211.582 25.4 90)
       (effects (font (size 1.27 1.27)) hide)
     )
@@
     (in_bom yes) (on_board yes)
     (property "Reference" "R10" (id 0) (at 217.17 29.21 90))
-    (property "Value" "" (id 1) (at 215.9 25.4 90))
-    (property "Footprint" "" (id 2) (at 214.122 25.4 90)
+    (property "Value" "10k" (id 1) (at 215.9 25.4 90))
+    (property "Footprint" "Resistor_SMD:R_0402_1005Metric" (id 2) (at 214.122 25.4 90)
       (effects (font (size 1.27 1.27)) hide)
     )
@@
     (in_bom yes) (on_board yes)
     (property "Reference" "R8" (id 0) (at 212.09 29.21 90))
-    (property "Value" "" (id 1) (at 210.82 25.4 90))
-    (property "Footprint" "" (id 2) (at 209.042 25.4 90)
+    (property "Value" "10k" (id 1) (at 210.82 25.4 90))
+    (property "Footprint" "Resistor_SMD:R_0402_1005Metric" (id 2) (at 209.042 25.4 90)
       (effects (font (size 1.27 1.27)) hide)
     )
@@
     (in_bom yes) (on_board yes)
     (property "Reference" "R3" (id 0) (at 149.352 30.48 90))
-    (property "Value" "" (id 1) (at 154.432 30.48 90))
-    (property "Footprint" "" (id 2) (at 150.114 30.48 90)
-      (effects (font (size 1.27 1.27)) hide)
-    )
+    (property "Value" "4.7k" (id 1) (at 154.432 30.48 90))
+    (property "Footprint" "Resistor_SMD:R_0402_1005Metric" (id 2) (at 150.114 30.48 90)
+      (effects (font (size 1.27 1.27)) hide)
+    )
