File: power.kicad_sch (KiCad schematic)
At the start: 47 parts, among them Q4 Q_NMOS_GSD, SW7 Power switch, U11 SY8079AAC, U12 SY8079AAC, U13 XT4054K421MR-G, U14 SY6280AAC, U15 SY6280AAC, U16 SY6280AAC

Commit message: Small DRC fixes
Parts:
- removed Q4: Q_NMOS_GSD, Package_TO_SOT_SMD:SOT-23, symbol mch2021-rescue:Q_NMOS_GSD-Device
- removed R53: 100k, Resistor_SMD:R_0402_1005Metric, symbol mch2021-rescue:R-Device
- removed R54, R55: 10k, Resistor_SMD:R_0402_1005Metric, symbol mch2021-rescue:R-Device
Connections:
- net at R59.2, U14.4 (ON): now also SW7.1 (A)
Changed lines of the file:
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@@
   (junction (at 38.1 175.26) (diameter 0) (color 0 0 0 0)
   )
-  (junction (at 33.02 69.85) (diameter 0) (color 0 0 0 0)
-  )
   (junction (at 64.77 36.83) (diameter 0) (color 0 0 0 0)
   )
   (junction (at 156.21 175.26) (diameter 0) (color 0 0 0 0)
   )
-  (junction (at 33.02 96.52) (diameter 0) (color 0 0 0 0)
-  )
   (junction (at 68.58 133.35) (diameter 0) (color 0 0 0 0)
   )
@@
   (junction (at 76.2 31.75) (diameter 0) (color 0 0 0 0)
   )
-  (junction (at 50.8 86.36) (diameter 0) (color 0 0 0 0)
-  )
   (junction (at 43.18 175.26) (diameter 0) (color 0 0 0 0)
   )
@@
     (stroke (width 0) (type default) (color 0 0 0 0))
   )
-  (wire (pts (xy 50.8 91.44) (xy 50.8 86.36))
-    (stroke (width 0) (type default) (color 0 0 0 0))
-  )
   (wire (pts (xy 124.46 179.07) (xy 124.46 172.72))
     (stroke (width 0) (type default) (color 0 0 0 0))
   )
-  (wire (pts (xy 50.8 86.36) (xy 62.23 86.36))
+  (wire (pts (xy 30.48 86.36) (xy 62.23 86.36))
     (stroke (width 0) (type default) (color 0 0 0 0))
   )
@@
     (stroke (width 0) (type default) (color 0 0 0 0))
   )
-  (wire (pts (xy 43.18 86.36) (xy 50.8 86.36))
-    (stroke (width 0) (type default) (color 0 0 0 0))
-  )
   (wire (pts (xy 76.2 175.26) (xy 76.2 184.15))
     (stroke (width 0) (type default) (color 0 0 0 0))
@@
     (stroke (width 0) (type default) (color 0 0 0 0))
   )
-  (wire (pts (xy 50.8 104.14) (xy 50.8 101.6))
-    (stroke (width 0) (type default) (color 0 0 0 0))
-  )
   (wire (pts (xy 74.93 26.67) (xy 74.93 29.21))
     (stroke (width 0) (type default) (color 0 0 0 0))
@@
     (stroke (width 0) (type default) (color 0 0 0 0))
   )
-  (wire (pts (xy 35.56 96.52) (xy 33.02 96.52))
-    (stroke (width 0) (type default) (color 0 0 0 0))
-  )
   (wire (pts (xy 162.56 34.29) (xy 156.21 34.29))
     (stroke (width 0) (type default) (color 0 0 0 0))
   )
-  (wire (pts (xy 30.48 86.36) (xy 35.56 86.36))
-    (stroke (width 0) (type default) (color 0 0 0 0))
-  )
   (wire (pts (xy 19.05 175.26) (xy 16.51 175.26))
     (stroke (width 0) (type default) (color 0 0 0 0))
@@
   )
   (wire (pts (xy 129.54 176.53) (xy 129.54 181.61))
-    (stroke (width 0) (type default) (color 0 0 0 0))
-  )
-  (wire (pts (xy 33.02 69.85) (xy 33.02 96.52))
     (stroke (width 0) (type default) (color 0 0 0 0))
   )
@@
     (pin "1")
   )
-  (symbol (lib_id "mch2021-rescue:R-Device") (at 39.37 86.36 90) (unit 1)
-    (in_bom yes) (on_board yes)
-    (property "Reference" "R54" (id 0) (at 40.64 90.17 0))
-    (property "Value" "10k" (id 1) (at 38.1 90.17 0))
-    (property "Footprint" "Resistor_SMD:R_0402_1005Metric" (id 2) (at 39.37 88.138 90)
-      (effects (font (size 1.27 1.27)) hide)
-    )
-    (property "Datasheet" "~" (id 3) (at 39.37 86.36 0)
-      (effects (font (size 1.27 1.27)) hide)
-    )
-    (property "Price" "" (id 4) (at 39.37 86.36 0)
-      (effects (font (size 1.27 1.27)) hide)
-    )
-    (property "LCSC" "C144807" (id 5) (at 39.37 86.36 0)
-      (effects (font (size 1.27 1.27)) hide)
-    )
-    (property "Mouser" "-" (id 6) (at 39.37 86.36 0)
-      (effects (font (size 1.27 1.27)) hide)
-    )
-    (property "Sponsored" "N" (id 7) (at 39.37 86.36 0)
-      (effects (font (size 1.27 1.27)) hide)
-    )
-    (property "MANUFACTURER" "YAGEO" (id 8) (at 39.37 86.36 0)
-      (effects (font (size 1.27 1.27)) hide)
-    )
-    (property "MPN" "AC0402FR-0710KL" (id 9) (at 39.37 86.36 0)
-      (effects (font (size 1.27 1.27)) hide)
-    )
-    (pin "1")
-    (pin "2")
-  )
-  (symbol (lib_id "mch2021-rescue:Q_NMOS_GSD-Device") (at 48.26 96.52 0) (unit 1)
-    (in_bom yes) (on_board yes)
-    (property "Reference" "Q4" (id 0) (at 54.61 96.52 90))
-    (property "Value" "Q_NMOS_GSD" (id 1) (at 57.15 96.52 90))
-    (property "Footprint" "Package_TO_SOT_SMD:SOT-23" (id 2) (at 53.34 93.98 0)
-      (effects (font (size 1.27 1.27)) hide)
-    )
-    (property "Datasheet" "~" (id 3) (at 48.26 96.52 0)
-      (effects (font (size 1.27 1.27)) hide)
-    )
-    (property "LCSC" "C406812" (id 4) (at 48.26 96.52 0)
-      (effects (font (size 1.27 1.27)) hide)
-    )
-    (property "Mouser" "-" (id 5) (at 48.26 96.52 0)
-      (effects (font (size 1.27 1.27)) hide)
-    )
-    (property "Price" "" (id 6) (at 48.26 96.52 0)
-      (effects (font (size 1.27 1.27)) hide)
-    )
-    (property "Sponsored" "N" (id 7) (at 48.26 96.52 0)
-      (effects (font (size 1.27 1.27)) hide)
-    )
-    (property "MANUFACTURER" "ALLPOWER" (id 8) (at 48.26 96.52 0)
-      (effects (font (size 1.27 1.27)) hide)
-    )
-    (property "MPN" "AP2302B" (id 9) (at 48.26 96.52 0)
-      (effects (font (size 1.27 1.27)) hide)
-    )
-    (pin "1")
-    (pin "2")
-    (pin "3")
-  )
-  (symbol (lib_id "mch2021-rescue:GND-power") (at 50.8 104.14 0) (unit 1)
-    (in_bom yes) (on_board yes)
-    (property "Reference" "#PWR0167" (id 0) (at 50.8 110.49 0)
-      (effects (font (size 1.27 1.27)) hide)
-    )
-    (property "Value" "GND" (id 1) (at 50.927 108.5342 0))
-    (property "Footprint" "" (id 2) (at 50.8 104.14 0)
-      (effects (font (size 1.27 1.27)) hide)
-    )
-    (property "Datasheet" "" (id 3) (at 50.8 104.14 0)
-      (effects (font (size 1.27 1.27)) hide)
-    )
-    (pin "1")
-  )
-  (symbol (lib_id "mch2021-rescue:R-Device") (at 39.37 96.52 90) (unit 1)
-    (in_bom yes) (on_board yes)
-    (property "Reference" "R55" (id 0) (at 40.64 100.33 0))
-    (property "Value" "10k" (id 1) (at 38.1 100.33 0))
-    (property "Footprint" "Resistor_SMD:R_0402_1005Metric" (id 2) (at 39.37 98.298 90)
-      (effects (font (size 1.27 1.27)) hide)
-    )
-    (property "Datasheet" "~" (id 3) (at 39.37 96.52 0)
-      (effects (font (size 1.27 1.27)) hide)
-    )
-    (property "Price" "" (id 4) (at 39.37 96.52 0)
-      (effects (font (size 1.27 1.27)) hide)
-    )
-    (property "LCSC" "C144807" (id 5) (at 39.37 96.52 0)
-      (effects (font (size 1.27 1.27)) hide)
-    )
-    (property "Mouser" "-" (id 6) (at 39.37 96.52 0)
-      (effects (font (size 1.27 1.27)) hide)
-    )
-    (property "Sponsored" "N" (id 7) (at 39.37 96.52 0)
-      (effects (font (size 1.27 1.27)) hide)
-    )
-    (property "MANUFACTURER" "YAGEO" (id 8) (at 39.37 96.52 0)
-      (effects (font (size 1.27 1.27)) hide)
-    )
-    (property "MPN" "AC0402FR-0710KL" (id 9) (at 39.37 96.52 0)
-      (effects (font (size 1.27 1.27)) hide)
-    )
-    (pin "1")
-    (pin "2")
-  )
-  (symbol (lib_id "mch2021-rescue:GND-power") (at 33.02 104.14 0) (unit 1)
-    (in_bom yes) (on_board yes)
-    (property "Reference" "#PWR0163" (id 0) (at 33.02 110.49 0)
-      (effects (font (size 1.27 1.27)) hide)
-    )
-    (property "Value" "GND" (id 1) (at 33.147 108.5342 0))
-    (property "Footprint" "" (id 2) (at 33.02 104.14 0)
-      (effects (font (size 1.27 1.27)) hide)
-    )
-    (property "Datasheet" "" (id 3) (at 33.02 104.14 0)
-      (effects (font (size 1.27 1.27)) hide)
-    )
-    (pin "1")
-  )
-  (symbol (lib_id "mch2021-rescue:R-Device") (at 33.02 100.33 0) (unit 1)
-    (in_bom yes) (on_board yes)
-    (property "Reference" "R53" (id 0) (at 29.21 101.6 0))
-    (property "Value" "100k" (id 1) (at 29.21 99.06 0))
-    (property "Footprint" "Resistor_SMD:R_0402_1005Metric" (id 2) (at 31.242 100.33 90)
-      (effects (font (size 1.27 1.27)) hide)
-    )
-    (property "Datasheet" "~" (id 3) (at 33.02 100.33 0)
-      (effects (font (size 1.27 1.27)) hide)
-    )
-    (property "Price" "" (id 4) (at 33.02 100.33 0)
-      (effects (font (size 1.27 1.27)) hide)
-    )
-    (property "LCSC" "C258090" (id 5) (at 33.02 100.33 0)
-      (effects (font (size 1.27 1.27)) hide)
-    )
-    (property "Mouser" "-" (id 6) (at 33.02 100.33 0)
-      (effects (font (size 1.27 1.27)) hide)
-    )
-    (property "Sponsored" "N" (id 7) (at 33.02 100.33 0)
-      (effects (font (size 1.27 1.27)) hide)
-    )
-    (property "MANUFACTURER" "FH" (id 8) (at 33.02 100.33 0)
-      (effects (font (size 1.27 1.27)) hide)
-    )
-    (property "MPN" "RC-02W1003FT" (id 9) (at 33.02 100.33 0)
-      (effects (font (size 1.27 1.27)) hide)
-    )
-    (pin "1")
-    (pin "2")
-  )
   (symbol (lib_id "mch2021-rescue:C-Device") (at 30.48 41.91 180) (unit 1)

Commit message: Small fixes
Parts:
- removed R51, R52: 0, Resistor_SMD:R_0402_1005Metric, symbol mch2021-rescue:R-Device
- C35, C36: value DNP -> 100n
- R62: value 2k -> 10k
- R68: value 3.4k -> 10k
Connections:
- net 1V2REG_VIN is gone; now on net VIN: C36.1, C39.1, U12.1 (EN), U12.4 (VIN)
- net 3V3REG_VIN is gone; now on net VIN: C35.1, C38.1, U11.1 (EN), U11.4 (VIN)
Other:
- note removed: "Iset = 2A = 6800 / 3.4kOhm"
Changed lines of the file:
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@@
     (company "BADGE.TEAM")
   )
+  (junction (at 29.21 130.81) (diameter 0) (color 0 0 0 0)
+  )
   (junction (at 62.23 86.36) (diameter 0) (color 0 0 0 0)
   )
@@
   (junction (at 43.18 130.81) (diameter 0) (color 0 0 0 0)
   )
-  (junction (at 29.21 130.81) (diameter 0) (color 0 0 0 0)
-  )
   (junction (at 16.51 81.28) (diameter 0) (color 0 0 0 0)
   )
@@
     (stroke (width 0) (type default) (color 0 0 0 0))
   )
-  (wire (pts (xy 26.67 130.81) (xy 29.21 130.81))
-    (stroke (width 0) (type default) (color 0 0 0 0))
-  )
   (wire (pts (xy 50.8 140.97) (xy 50.8 147.32))
     (stroke (width 0) (type default) (color 0 0 0 0))
@@
     (stroke (width 0) (type default) (color 0 0 0 0))
   )
-  (wire (pts (xy 26.67 175.26) (xy 29.21 175.26))
-    (stroke (width 0) (type default) (color 0 0 0 0))
-  )
   (wire (pts (xy 76.2 175.26) (xy 76.2 184.15))
     (stroke (width 0) (type default) (color 0 0 0 0))
@@
     (stroke (width 0) (type default) (color 0 0 0 0))
   )
-  (wire (pts (xy 19.05 175.26) (xy 16.51 175.26))
+  (wire (pts (xy 16.51 175.26) (xy 29.21 175.26))
     (stroke (width 0) (type default) (color 0 0 0 0))
   )
@@
     (stroke (width 0) (type default) (color 0 0 0 0))
   )
-  (wire (pts (xy 19.05 130.81) (xy 16.51 130.81))
+  (wire (pts (xy 16.51 130.81) (xy 29.21 130.81))
     (stroke (width 0) (type default) (color 0 0 0 0))
   )
@@
     (stroke (width 0) (type default) (color 0 0 0 0))
   )
-  (text "Iset = 2A = 6800 / 3.4kOhm" (at 120.65 68.58 180)
+  (text "Iset = 0.68A = 6800 / 10kOhm" (at 120.65 68.58 180)
     (effects (font (size 0.9906 0.9906)) (justify right bottom))
   )
@@
       (effects (font (size 1.27 1.27)) (justify left))
     )
-    (property "Value" "2k" (id 1) (at 70.993 27.432 0)
+    (property "Value" "10k" (id 1) (at 70.993 27.432 0)
       (effects (font (size 1.27 1.27)) (justify left))
     )
@@
       (effects (font (size 1.27 1.27)) (justify left))
     )
-    (property "Value" "DNP" (id 1) (at 32.131 144.653 0)
+    (property "Value" "100n" (id 1) (at 32.131 144.653 0)
       (effects (font (size 1.27 1.27)) (justify left))
     )
@@
     )
     (property "LCSC" "C5674" (id 6) (at 29.21 143.51 0)
-      (effects (font (size 1.27 1.27)) hide)
-    )
-    (pin "1")
-    (pin "2")
-  )
-  (symbol (lib_id "mch2021-rescue:R-Device") (at 22.86 130.81 270) (unit 1)
-    (in_bom yes) (on_board yes)
-    (property "Reference" "R51" (id 0) (at 24.0284 132.588 0)
-      (effects (font (size 1.27 1.27)) (justify left))
-    )
-    (property "Value" "0" (id 1) (at 21.717 132.588 0)
-      (effects (font (size 1.27 1.27)) (justify left))
-    )
-    (property "Footprint" "Resistor_SMD:R_0402_1005Metric" (id 2) (at 22.86 129.032 90)
-      (effects (font (size 1.27 1.27)) hide)
-    )
-    (property "Datasheet" "~" (id 3) (at 22.86 130.81 0)
-      (effects (font (size 1.27 1.27)) hide)
-    )
-    (property "Price" "" (id 4) (at 22.86 130.81 0)
-      (effects (font (size 1.27 1.27)) hide)
-    )
-    (property "LCSC" "C60485" (id 5) (at 22.86 130.81 0)
-      (effects (font (size 1.27 1.27)) hide)
-    )
-    (property "Mouser" "-" (id 6) (at 22.86 130.81 0)
-      (effects (font (size 1.27 1.27)) hide)
-    )
-    (property "Sponsored" "N" (id 7) (at 22.86 130.81 0)
-      (effects (font (size 1.27 1.27)) hide)
-    )
-    (property "MANUFACTURER" "YAGEO" (id 8) (at 22.86 130.81 0)
-      (effects (font (size 1.27 1.27)) hide)
-    )
-    (property "MPN" "RC0402JR-070RL" (id 9) (at 22.86 130.81 0)
       (effects (font (size 1.27 1.27)) hide)
     )
@@
       (effects (font (size 1.27 1.27)) (justify left))
     )
-    (property "Value" "DNP" (id 1) (at 32.131 189.103 0)
+    (property "Value" "100n" (id 1) (at 32.131 189.103 0)
       (effects (font (size 1.27 1.27)) (justify left))
     )
@@
     )
     (property "LCSC" "C5674" (id 6) (at 29.21 187.96 0)
-      (effects (font (size 1.27 1.27)) hide)
-    )
-    (pin "1")
-    (pin "2")
-  )
-  (symbol (lib_id "mch2021-rescue:R-Device") (at 22.86 175.26 270) (unit 1)
-    (in_bom yes) (on_board yes)
-    (property "Reference" "R52" (id 0) (at 24.0284 177.038 0)
-      (effects (font (size 1.27 1.27)) (justify left))
-    )
-    (property "Value" "0" (id 1) (at 21.717 177.038 0)
-      (effects (font (size 1.27 1.27)) (justify left))
-    )
-    (property "Footprint" "Resistor_SMD:R_0402_1005Metric" (id 2) (at 22.86 173.482 90)
-      (effects (font (size 1.27 1.27)) hide)
-    )
-    (property "Datasheet" "~" (id 3) (at 22.86 175.26 0)
-      (effects (font (size 1.27 1.27)) hide)
-    )
-    (property "Price" "" (id 4) (at 22.86 175.26 0)
-      (effects (font (size 1.27 1.27)) hide)
-    )
-    (property "LCSC" "C60485" (id 5) (at 22.86 175.26 0)
-      (effects (font (size 1.27 1.27)) hide)
-    )
-    (property "Mouser" "-" (id 6) (at 22.86 175.26 0)
-      (effects (font (size 1.27 1.27)) hide)
-    )
-    (property "Sponsored" "N" (id 7) (at 22.86 175.26 0)
-      (effects (font (size 1.27 1.27)) hide)
-    )
-    (property "MANUFACTURER" "YAGEO" (id 8) (at 22.86 175.26 0)
-      (effects (font (size 1.27 1.27)) hide)
-    )
-    (property "MPN" "RC0402JR-070RL" (id 9) (at 22.86 175.26 0)
       (effects (font (size 1.27 1.27)) hide)
     )
@@
       (effects (font (size 1.27 1.27)) (justify left))
     )
-    (property "Value" "3.4k" (id 1) (at 149.098 91.313 0)
-      (effects (font (size 1.27 1.27)) (justify left))
-    )
+    (property "Value" "10k" (id 1) (at 149.098 91.313 0)
+      (effects (font (size 1.27 1.27)) (justify left))
+    )

Commit message: Remove IO expander, move around signals
Parts:
- removed R65, R76: 10k, Resistor_SMD:R_0402_1005Metric, symbol mch2021-rescue:R-Device
Connections:
- net PWR_LED_ENABLE is gone; now on net PWR_SDCARD_ENABLE: U16.4 (ON)
- net BATT_TEMP: no longer names the net of BT1.1 (Pin_1)
Changed lines of the file:
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@@
   (title_block
     (title "MCH2021 badge - Power management")
-    (date "2022-01-14")
-    (rev "3.1415")
+    (date "2022-03-11")
+    (rev "4")
     (company "BADGE.TEAM")
   )
@@
   (junction (at 140.97 180.34) (diameter 0) (color 0 0 0 0)
   )
-  (junction (at 124.46 85.09) (diameter 0) (color 0 0 0 0)
-  )
   (junction (at 87.63 69.85) (diameter 0) (color 0 0 0 0)
   )
@@
   (junction (at 140.97 175.26) (diameter 0) (color 0 0 0 0)
   )
-  (junction (at 68.58 52.07) (diameter 0) (color 0 0 0 0)
-  )
   (junction (at 38.1 130.81) (diameter 0) (color 0 0 0 0)
   )
@@
     (stroke (width 0) (type default) (color 0 0 0 0))
   )
-  (wire (pts (xy 124.46 86.36) (xy 124.46 85.09))
-    (stroke (width 0) (type default) (color 0 0 0 0))
-  )
   (wire (pts (xy 124.46 179.07) (xy 124.46 172.72))
     (stroke (width 0) (type default) (color 0 0 0 0))
@@
     (stroke (width 0) (type default) (color 0 0 0 0))
   )
-  (wire (pts (xy 123.19 85.09) (xy 124.46 85.09))
-    (stroke (width 0) (type default) (color 0 0 0 0))
-  )
   (wire (pts (xy 58.42 138.43) (xy 58.42 133.35))
     (stroke (width 0) (type default) (color 0 0 0 0))
@@
     (stroke (width 0) (type default) (color 0 0 0 0))
   )
-  (wire (pts (xy 81.28 44.45) (xy 81.28 52.07))
-    (stroke (width 0) (type default) (color 0 0 0 0))
-  )
   (wire (pts (xy 30.48 38.1) (xy 30.48 26.67))
     (stroke (width 0) (type default) (color 0 0 0 0))
@@
     (stroke (width 0) (type default) (color 0 0 0 0))
   )
+  (wire (pts (xy 123.19 85.09) (xy 125.73 85.09))
+    (stroke (width 0) (type default) (color 0 0 0 0))
+  )
   (polyline (pts (xy 12.7 160.02) (xy 176.53 160.02))
     (stroke (width 0) (type default) (color 0 0 0 0))
@@
     (stroke (width 0) (type default) (color 0 0 0 0))
   )
-  (wire (pts (xy 68.58 52.07) (xy 66.04 52.07))
-    (stroke (width 0) (type default) (color 0 0 0 0))
-  )
   (polyline (pts (xy 176.53 12.7) (xy 176.53 166.37))
     (stroke (width 0) (type default) (color 0 0 0 0))
@@
     (stroke (width 0) (type default) (color 0 0 0 0))
   )
-  (wire (pts (xy 86.36 44.45) (xy 81.28 44.45))
-    (stroke (width 0) (type default) (color 0 0 0 0))
-  )
   (wire (pts (xy 68.58 177.8) (xy 67.31 177.8))
     (stroke (width 0) (type default) (color 0 0 0 0))
@@
     (stroke (width 0) (type default) (color 0 0 0 0))
   )
-  (wire (pts (xy 81.28 52.07) (xy 68.58 52.07))
-    (stroke (width 0) (type default) (color 0 0 0 0))
-  )
   (wire (pts (xy 67.31 138.43) (xy 68.58 138.43))
     (stroke (width 0) (type default) (color 0 0 0 0))
@@
   )
   (wire (pts (xy 58.42 184.15) (xy 58.42 182.88))
-    (stroke (width 0) (type default) (color 0 0 0 0))
-  )
-  (wire (pts (xy 124.46 85.09) (xy 125.73 85.09))
     (stroke (width 0) (type default) (color 0 0 0 0))
   )
@@
     )
   )
-  (hierarchical_label "BATT_TEMP" (shape output) (at 66.04 52.07 180)
-    (effects (font (size 1.27 1.27)) (justify right))
+  (hierarchical_label "PWR_SDCARD_ENABLE" (shape input) (at 123.19 85.09 180)
+    (effects (font (size 0.9906 0.9906)) (justify right))
   )
   (hierarchical_label "SENSE_VUSB" (shape output) (at 158.75 180.34 0)
@@
   (hierarchical_label "CHARGING" (shape output) (at 66.04 36.83 0)
     (effects (font (size 0.9906 0.9906)) (justify left))
-  )
-  (hierarchical_label "PWR_LED_ENABLE" (shape input) (at 123.19 85.09 180)
-    (effects (font (size 0.9906 0.9906)) (justify right))
   )
   (hierarchical_label "PWR_SDCARD_ENABLE" (shape input) (at 123.19 39.37 180)
@@
     )
     (property "Datasheet" "" (id 3) (at 147.32 93.98 0)
-      (effects (font (size 1.27 1.27)) hide)
-    )
-    (pin "1")
-  )
-  (symbol (lib_id "mch2021-rescue:GND-power") (at 124.46 93.98 0) (unit 1)
-    (in_bom yes) (on_board yes)
-    (property "Reference" "#PWR0196" (id 0) (at 124.46 100.33 0)
-      (effects (font (size 1.27 1.27)) hide)
-    )
-    (property "Value" "GND" (id 1) (at 124.587 98.3742 0))
-    (property "Footprint" "" (id 2) (at 124.46 93.98 0)
-      (effects (font (size 1.27 1.27)) hide)
-    )
-    (property "Datasheet" "" (id 3) (at 124.46 93.98 0)
       (effects (font (size 1.27 1.27)) hide)
     )
@@
     (pin "2")
   )
-  (symbol (lib_id "mch2021-rescue:R-Device") (at 124.46 90.17 180) (unit 1)
-    (in_bom yes) (on_board yes)
-    (property "Reference" "R65" (id 0) (at 129.7178 90.17 90))
-    (property "Value" "10k" (id 1) (at 127.4064 90.17 90))
-    (property "Footprint" "Resistor_SMD:R_0402_1005Metric" (id 2) (at 126.238 90.17 90)
-      (effects (font (size 1.27 1.27)) hide)
-    )
-    (property "Datasheet" "~" (id 3) (at 124.46 90.17 0)
-      (effects (font (size 1.27 1.27)) hide)
-    )
-    (property "Price" "" (id 4) (at 124.46 90.17 0)
-      (effects (font (size 1.27 1.27)) hide)
-    )
-    (property "LCSC" "C144807" (id 5) (at 124.46 90.17 0)
-      (effects (font (size 1.27 1.27)) hide)
-    )
-    (property "Mouser" "-" (id 6) (at 124.46 90.17 0)
-      (effects (font (size 1.27 1.27)) hide)
-    )
-    (property "Sponsored" "N" (id 7) (at 124.46 90.17 0)
-      (effects (font (size 1.27 1.27)) hide)
-    )
-    (property "MANUFACTURER" "YAGEO" (id 8) (at 124.46 90.17 0)
-      (effects (font (size 1.27 1.27)) hide)
-    )
-    (property "MPN" "AC0402FR-0710KL" (id 9) (at 124.46 90.17 0)
-      (effects (font (size 1.27 1.27)) hide)
-    )
-    (pin "1")
-    (pin "2")
-  )
   (symbol (lib_id "mch2021-rescue:R-Device") (at 62.23 96.52 180) (unit 1)
     (in_bom yes) (on_board yes)
@@
     (pin "1")
   )
-  (symbol (lib_id "mch2021-rescue:+3.3V-power") (at 68.58 44.45 0) (unit 1)
-    (in_bom yes) (on_board yes)
-    (property "Reference" "#PWR0228" (id 0) (at 68.58 48.26 0)
-      (effects (font (size 1.27 1.27)) hide)
-    )
-    (property "Value" "+3.3V" (id 1) (at 68.58 40.64 0))
-    (property "Footprint" "" (id 2) (at 68.58 44.45 0)
-      (effects (font (size 1.27 1.27)) hide)
-    )
-    (property "Datasheet" "" (id 3) (at 68.58 44.45 0)
-      (effects (font (size 1.27 1.27)) hide)
-    )
-    (pin "1")
-  )
-  (symbol (lib_id "mch2021-rescue:R-Device") (at 68.58 48.26 0) (unit 1)
-    (in_bom yes) (on_board yes)
-    (property "Reference" "R76" (id 0) (at 70.358 47.0916 0)
-      (effects (font (size 1.27 1.27)) (justify left))
-    )
-    (property "Value" "10k" (id 1) (at 70.358 49.403 0)
-      (effects (font (size 1.27 1.27)) (justify left))
-    )
-    (property "Footprint" "Resistor_SMD:R_0402_1005Metric" (id 2) (at 66.802 48.26 90)
-      (effects (font (size 1.27 1.27)) hide)
-    )
-    (property "Datasheet" "~" (id 3) (at 68.58 48.26 0)
-      (effects (font (size 1.27 1.27)) hide)
-    )
-    (property "Price" "" (id 4) (at 68.58 48.26 0)
-      (effects (font (size 1.27 1.27)) hide)
-    )
-    (property "LCSC" "C144807" (id 5) (at 68.58 48.26 0)
-      (effects (font (size 1.27 1.27)) hide)
-    )
-    (property "Mouser" "-" (id 6) (at 68.58 48.26 0)
-      (effects (font (size 1.27 1.27)) hide)
-    )
-    (property "Sponsored" "N" (id 7) (at 68.58 48.26 0)
-      (effects (font (size 1.27 1.27)) hide)
-    )
-    (property "MANUFACTURER" "YAGEO" (id 8) (at 68.58 48.26 0)
-      (effects (font (size 1.27 1.27)) hide)
-    )
-    (property "MPN" "AC0402FR-0710KL" (id 9) (at 68.58 48.26 0)
-      (effects (font (size 1.27 1.27)) hide)
-    )
-    (pin "1")
-    (pin "2")
-  )
   (symbol (lib_id "mch2021-rescue:C-Device") (at 156.21 44.45 0) (unit 1)

Commit message: Remove user I2C bus, connect LCD control signals to ESP32 directly, replace I2S dac
Parts:
- R63: value 10k -> 3k4
Connections:
- net PWR_SDCARD_ENABLE renamed PWR_ENABLE
Other:
- note removed: "Note: All control signals are hierarchical labels while all power rails are global"
- title: MCH2021 badge - Power management -> MCH2022 badge - Power management
- moved on the sheet: C48, C49, C50, D9, R59, R63, R64, R67, R68, RN6, SW7, U14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
