File: power.kicad_sch (KiCad schematic)
At the start: 39 parts, among them SW7 Power switch, U11 SY8079AAC, U12 SY8079AAC, U13 XT4054K421MR-G, U14 SY6280AAC, U15 SY6280AAC, U16 SY6280AAC

Commit message: Bill of materials 1/2
Parts:
- BT1: value LiPo -> (none); footprint Connector_JST:JST_PH_S3B-PH-SM4-TB_1x03-1MP_P2.00mm_Horizontal -> (none); Category (none) -> Connectors; MPN (none) -> S3B-PH-SM4-TB(LF)(SN); Manufacturer (none) -> JST; Sponsored N -> (none)
- C34, C42: value 10u -> (none); footprint Capacitor_SMD:C_0402_1005Metric -> (none); Category (none) -> Capacitors; LCSC C15525 -> (none); Sponsored N -> (none)
- C35, C36: value 100n -> (none); footprint Capacitor_SMD:C_0402_1005Metric -> (none); Category (none) -> Capacitors; LCSC C5674 -> (none); Sponsored N -> (none)
- C37, C48, C50: value 100n -> (none); footprint Capacitor_SMD:C_0402_1005Metric -> (none); Category (none) -> Capacitors; LCSC C83056 -> (none); Sponsored N -> (none)
- C38, C39, C43, C44, C45, C46, C49: value 22u -> (none); footprint Capacitor_SMD:C_0805_2012Metric -> (none); Category (none) -> Capacitors; LCSC C159801 -> (none); Sponsored N -> (none)
- C40, C41: value 22p -> (none); footprint Capacitor_SMD:C_0402_1005Metric -> (none); Category (none) -> Capacitors; LCSC C106203 -> (none); MPN CC0402JRNPO9BN220 -> (none); Sponsored N -> (none)
- D9: value PSBD3D40V1H -> (none); footprint Diode_SMD:D_SOD-323 -> (none); Category (none) -> Diodes; MPN (none) -> PSBD3D40V1H; Manufacturer (none) -> Shanghai Prisemi Elec; Sponsored N -> (none)
- L3, L4: value 2.2u -> (none); footprint custom:Inductor_MSC20FC -> (none); Category (none) -> Inductors; MPN (none) -> MCS20FC-2R2MHC; Manufacturer (none) -> PSA; Sponsored N -> (none)
- R56: value 2k -> (none); footprint Resistor_SMD:R_0402_1005Metric -> (none); Category (none) -> Resistors; Sponsored N -> (none)
- R57, R58, R61, R64, R67: value 10k -> (none); footprint Resistor_SMD:R_0402_1005Metric -> (none); Category (none) -> Resistors; LCSC C144807 -> (none); MPN AC0402FR-0710KL -> (none); Sponsored N -> (none)
- R59: value 100k -> (none); footprint Resistor_SMD:R_0402_1005Metric -> (none); Category (none) -> Resistors; LCSC C258090 -> (none); MPN RC-02W1003FT -> (none); Sponsored N -> (none)
- R60: value 45.3k -> (none); footprint Resistor_SMD:R_0402_1005Metric -> (none); Category (none) -> Resistors; Sponsored N -> (none)
- R62: value 10k -> (none); footprint Resistor_SMD:R_0402_1005Metric -> (none); Category (none) -> Resistors; LCSC C4109 -> (none); MPN 0402WGF2001TCE -> (none); Sponsored N -> (none)
- R63: value 3k4 -> (none); footprint Resistor_SMD:R_0402_1005Metric -> (none); Category (none) -> Resistors; Sponsored N -> (none)
- R68: value 10k -> (none); footprint Resistor_SMD:R_0402_1005Metric -> (none); Category (none) -> Resistors; LCSC C4940 -> (none); MPN 0402WGF3401TCE -> (none); Sponsored N -> (none)
- RN6: value 100k -> (none); footprint Resistor_SMD:R_Array_Convex_4x0603 -> (none); Category (none) -> Resistor arrays; Sponsored N -> (none)
- SW7: value Power switch -> (none); footprint Button_Switch_SMD:SW_SPDT_PCM12 -> (none); Category (none) -> Buttons; Sponsored N -> (none)
- U11, U12: value SY8079AAC -> (none); footprint Package_TO_SOT_SMD:SOT-23-5 -> (none); Buy early (none) -> Y; Category (none) -> ICs; MPN (none) -> SY8079AAC; Manufacturer (none) -> Silergy Corp
- U13: value XT4054K421MR-G -> (none); footprint Package_TO_SOT_SMD:SOT-23-5 -> (none); Buy early (none) -> Y; Category (none) -> ICs; MPN (none) -> XT4054K421MR-G; Manufacturer (none) -> Natlinear
- U14, U15, U16: value SY6280AAC -> (none); footprint Package_TO_SOT_SMD:SOT-23-5 -> (none); Buy early (none) -> Y; Category (none) -> ICs; MPN (none) -> SY6280AAC; Manufacturer (none) -> Silergy Corp

Commit message: Add more info to BOM
Parts:
- added R53: (no value), symbol mch2021-rescue:R-Device
- BT1: Sponsored (none) -> N
- C34, C35, C36, C37, C38, C39, C40, C41, C42, C43, C44, C45, C46, C48, C49, C50, D9, L3, L4, R57, R58, R59, R60, R61, R62, R64, R67, R68: Buy early (none) -> Y; Sponsored (none) -> N
- R56: Buy early (none) -> Y; LCSC C4109 -> C25543; MPN 0402WGF2001TCE -> 0402WGJ0102TCE; Manufacturer (none) -> Uni-royal; Sponsored (none) -> N
- R63: Buy early (none) -> Y; LCSC C144807 -> C25940; MPN AC0402FR-0710KL -> 0402WGJ0472TCE; Manufacturer (none) -> Uni-royal; Sponsored (none) -> N
- RN6: Buy early (none) -> Y; Manufacturer (none) -> Uni-royal; Sponsored (none) -> N
- SW7: Buy early (none) -> Y; MPN (none) -> SK-3296S-01-L1; Manufacturer (none) -> XKB Connectivity; Sponsored (none) -> N
Connections:
- net GND: now also R53.1; no longer R56.2
- net at U13.5 (PROG): now also R56.2; no longer R56.1
- new net: R53.2, R56.1
Other:
- note added: "IBAT = (VPROG / RPROG) * 1000 VPROG = 1V"
- note added: "Iset = 1.44A = 6800 / 4700"
- moved on the sheet: C34, C37, R56

Commit message: Add passives to BOM
Parts:
- BT1: Buy early (none) -> N
- C34, C42: LCSC (none) -> C15525; MPN (none) -> CL05A106MQ5NUNC; Manufacturer (none) -> Samsung Electro-Mechanics; Minimal voltage rating (none) -> 6; Voltage rating (none) -> 6.3
- C35, C36, C37, C48, C50: LCSC (none) -> C307331; MPN (none) -> CL05B104KB54PNC; Manufacturer (none) -> Samsung Electro-Mechanics; Minimal voltage rating (none) -> 10; Voltage rating (none) -> 50
- C38, C39, C43, C44, C45, C46, C49: LCSC (none) -> C602037; MPN (none) -> CL21A226MAYNNNE; Manufacturer (none) -> Samsung Electro-Mechanics; Minimal voltage rating (none) -> 10; Voltage rating (none) -> 25
- C40, C41: LCSC (none) -> C466226; MPN (none) -> TCC0402C0G220J500AT; Manufacturer (none) -> CCTC; Minimal voltage rating (none) -> 10; Voltage rating (none) -> 50
- R53, R56: LCSC C25543 -> C11702; MPN 0402WGJ0102TCE -> 0402WGF1001TCE
- R57, R58, R61, R62, R64, R67, R68: LCSC (none) -> C25744; MPN (none) -> 0402WGF1002TCE; Manufacturer (none) -> Uni-royal
- R59: LCSC (none) -> C25741; MPN (none) -> 0402WGF1003TCE; Manufacturer (none) -> Uni-royal
- R60: Manufacturer (none) -> Uni-royal
- R63: LCSC C25940 -> C25900; MPN 0402WGJ0472TCE -> 0402WGF4701TCE
