File: power.kicad_sch (KiCad schematic)
At the start: 40 parts

Commit message: Artwork stuff
Parts:
- BT1: value (none) -> LiPo; footprint (none) -> Connector_JST:JST_PH_S3B-PH-SM4-TB_1x03-1MP_P2.00mm_Horizontal
- C34, C42: value (none) -> 10u; footprint (none) -> Capacitor_SMD:C_0402_1005Metric
- C35, C36, C37, C48, C50: value (none) -> 100n; footprint (none) -> Capacitor_SMD:C_0402_1005Metric
- C38, C39, C43, C44, C45, C46, C49: value (none) -> 22u; footprint (none) -> Capacitor_SMD:C_0805_2012Metric
- C40, C41: value (none) -> 22p; footprint (none) -> Capacitor_SMD:C_0402_1005Metric
- D9: value (none) -> PSBD3D40V1H; footprint (none) -> Diode_SMD:D_SOD-323
- L3, L4: value (none) -> 2.2u; footprint (none) -> custom:Inductor_MSC20FC
- R53, R56: value (none) -> 1k; footprint (none) -> Resistor_SMD:R_0402_1005Metric
- R57, R58, R61, R62, R64, R67, R68: value (none) -> 10k; footprint (none) -> Resistor_SMD:R_0402_1005Metric
- R59: value (none) -> 100k; footprint (none) -> Resistor_SMD:R_0402_1005Metric
- R60: value (none) -> 45.3k; footprint (none) -> Resistor_SMD:R_0402_1005Metric
- R63: value (none) -> 4.7k; footprint (none) -> Resistor_SMD:R_0402_1005Metric
- RN6: value (none) -> 100k; footprint (none) -> Resistor_SMD:R_Array_Convex_4x0603
- SW7: value (none) -> Switch; footprint (none) -> Button_Switch_SMD:SW_SPDT_PCM12
- U11, U12: value (none) -> SY8079AAC; footprint (none) -> Package_TO_SOT_SMD:SOT-23-5
- U13: value (none) -> XT4054K421MR-G; footprint (none) -> Package_TO_SOT_SMD:SOT-23-5
- U14, U15, U16: value (none) -> SY6280AAC; footprint (none) -> Package_TO_SOT_SMD:SOT-23-5

Commit message: Last minute fixes
Connections:
- no-connect marks 0 -> 2
Changed lines of the file:
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@@
   (junction (at 85.09 31.75) (diameter 0) (color 0 0 0 0)
   )
+  (no_connect (at 138.43 116.84))
+  (no_connect (at 86.36 44.45))
   (wire (pts (xy 241.3 76.2) (xy 251.46 76.2))
     (stroke (width 0) (type default) (color 0 0 0 0))

Commit message: Final version of prototype 4
Parts:
- BT1: value LiPo -> (none); footprint Connector_JST:JST_PH_S3B-PH-SM4-TB_1x03-1MP_P2.00mm_Horizontal -> (none); symbol mch2021-rescue:Conn_01x03_Male-Connector -> Connector_Generic_MountingPin:Conn_01x03_MountingPin
Connections:
- net GND: now also BT1.MP (MountPin)
Other:
- moved on the sheet: BT1
Changed lines of the file:
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@@
+    (stroke (width 0) (type default) (color 0 0 0 0))
+  )
+  (wire (pts (xy 96.52 34.29) (xy 91.44 34.29))
     (stroke (width 0) (type default) (color 0 0 0 0))
   )
@@
   )
   (wire (pts (xy 58.42 85.09) (xy 64.77 85.09))
+    (stroke (width 0) (type default) (color 0 0 0 0))
+  )
+  (wire (pts (xy 96.52 45.72) (xy 96.52 34.29))
     (stroke (width 0) (type default) (color 0 0 0 0))
   )
@@
     (pin "1")
   )
-  (symbol (lib_id "mch2021-rescue:Conn_01x03_Male-Connector") (at 91.44 41.91 180) (unit 1)
-    (in_bom yes) (on_board yes)
-    (property "Reference" "BT1" (id 0) (at 90.17 49.53 0)
+  (symbol (lib_id "Connector_Generic_MountingPin:Conn_01x03_MountingPin") (at 91.44 41.91 0) (mirror x) (unit 1)
+    (in_bom yes) (on_board yes)
+    (property "Reference" "BT1" (id 0) (at 92.71 49.53 0)
       (effects (font (size 1.27 1.27)) (justify right))
     )
-    (property "Value" "LiPo" (id 1) (at 90.17 46.99 0)
+    (property "Value" "" (id 1) (at 92.71 46.99 0)
       (effects (font (size 1.27 1.27)) (justify right))
     )
-    (property "Footprint" "Connector_JST:JST_PH_S3B-PH-SM4-TB_1x03-1MP_P2.00mm_Horizontal" (id 2) (at 91.44 41.91 0)
+    (property "Footprint" "" (id 2) (at 91.44 41.91 0)
       (effects (font (size 1.27 1.27)) hide)
     )
@@
     (pin "2")
     (pin "3")
+    (pin "MP")
   )
   (symbol (lib_id "mch2021-rescue:AAT4610BIGV-1-T1-Power_Management") (at 156.21 109.22 0) (unit 1)
@@
     (pin "2")
   )
+  (symbol (lib_id "mch2021-rescue:GND-power") (at 96.52 45.72 0) (unit 1)
+    (in_bom yes) (on_board yes)
+    (property "Reference" "#PWR?" (id 0) (at 96.52 52.07 0)
+      (effects (font (size 1.27 1.27)) hide)
+    )
+    (property "Value" "GND" (id 1) (at 96.647 50.1142 0))
+    (property "Footprint" "" (id 2) (at 96.52 45.72 0)
+      (effects (font (size 1.27 1.27)) hide)
+    )
+    (property "Datasheet" "" (id 3) (at 96.52 45.72 0)
+      (effects (font (size 1.27 1.27)) hide)
+    )
+    (pin "1")
+  )
 )

Commit message: Small last minute tweaks
Parts:
- removed BT1: (no value), symbol Connector_Generic_MountingPin:Conn_01x03_MountingPin
- added J6: (no value), symbol Connector_Generic_MountingPin:Conn_01x02_MountingPin
Connections:
- net GND: now also J6.2 (Pin_2), J6.MP (MountPin)
- net VBAT: now also J6.1 (Pin_1)
- no-connect marks 2 -> 1
Changed lines of the file:
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@@
   )
   (no_connect (at 138.43 116.84))
-  (no_connect (at 86.36 44.45))
   (wire (pts (xy 241.3 76.2) (xy 251.46 76.2))
     (stroke (width 0) (type default) (color 0 0 0 0))
@@
     (stroke (width 0) (type default) (color 0 0 0 0))
   )
-  (wire (pts (xy 96.52 34.29) (xy 91.44 34.29))
-    (stroke (width 0) (type default) (color 0 0 0 0))
-  )
   (wire (pts (xy 68.58 138.43) (xy 68.58 133.35))
     (stroke (width 0) (type default) (color 0 0 0 0))
@@
     (stroke (width 0) (type default) (color 0 0 0 0))
   )
-  (wire (pts (xy 96.52 45.72) (xy 96.52 34.29))
-    (stroke (width 0) (type default) (color 0 0 0 0))
-  )
   (wire (pts (xy 50.8 140.97) (xy 50.8 147.32))
     (stroke (width 0) (type default) (color 0 0 0 0))
   )
-  (wire (pts (xy 85.09 41.91) (xy 85.09 45.72))
+  (wire (pts (xy 85.09 40.64) (xy 85.09 45.72))
     (stroke (width 0) (type default) (color 0 0 0 0))
   )
@@
     (stroke (width 0) (type default) (color 0 0 0 0))
   )
-  (wire (pts (xy 86.36 41.91) (xy 85.09 41.91))
+  (wire (pts (xy 85.09 38.1) (xy 86.36 38.1))
     (stroke (width 0) (type default) (color 0 0 0 0))
   )
@@
     (stroke (width 0) (type default) (color 0 0 0 0))
   )
+  (wire (pts (xy 86.36 40.64) (xy 85.09 40.64))
+    (stroke (width 0) (type default) (color 0 0 0 0))
+  )
   (wire (pts (xy 58.42 139.7) (xy 58.42 138.43))
     (stroke (width 0) (type default) (color 0 0 0 0))
@@
     (stroke (width 0) (type default) (color 0 0 0 0))
   )
-  (wire (pts (xy 86.36 39.37) (xy 85.09 39.37))
-    (stroke (width 0) (type default) (color 0 0 0 0))
-  )
   (wire (pts (xy 201.93 81.28) (xy 201.93 62.23))
     (stroke (width 0) (type default) (color 0 0 0 0))
@@
     (stroke (width 0) (type default) (color 0 0 0 0))
   )
-  (wire (pts (xy 85.09 31.75) (xy 85.09 39.37))
+  (wire (pts (xy 85.09 31.75) (xy 85.09 38.1))
     (stroke (width 0) (type default) (color 0 0 0 0))
   )
@@
     )
     (pin "1")
-  )
-  (symbol (lib_id "Connector_Generic_MountingPin:Conn_01x03_MountingPin") (at 91.44 41.91 0) (mirror x) (unit 1)
-    (in_bom yes) (on_board yes)
-    (property "Reference" "BT1" (id 0) (at 92.71 49.53 0)
-      (effects (font (size 1.27 1.27)) (justify right))
-    )
-    (property "Value" "" (id 1) (at 92.71 46.99 0)
-      (effects (font (size 1.27 1.27)) (justify right))
-    )
-    (property "Footprint" "" (id 2) (at 91.44 41.91 0)
-      (effects (font (size 1.27 1.27)) hide)
-    )
-    (property "Datasheet" "https://datasheet.lcsc.com/lcsc/1810261109_JST-Sales-America-S3B-PH-SM4-TB-LF-SN_C265101.pdf" (id 3) (at 91.44 41.91 0)
-      (effects (font (size 1.27 1.27)) hide)
-    )
-    (property "LCSC" "C265101" (id 4) (at 91.44 41.91 0)
-      (effects (font (size 1.27 1.27)) hide)
-    )
-    (property "Mouser" "-" (id 5) (at 91.44 41.91 0)
-      (effects (font (size 1.27 1.27)) hide)
-    )
-    (property "Price" "" (id 6) (at 91.44 41.91 0)
-      (effects (font (size 1.27 1.27)) hide)
-    )
-    (property "Sponsored" "N" (id 7) (at 91.44 41.91 0)
-      (effects (font (size 1.27 1.27)) hide)
-    )
-    (property "Category" "Connectors" (id 8) (at 91.44 41.91 0)
-      (effects (font (size 1.27 1.27)) hide)
-    )
-    (property "Description" "Depends on battery" (id 9) (at 91.44 41.91 0)
-      (effects (font (size 1.27 1.27)) hide)
-    )
-    (property "MPN" "S3B-PH-SM4-TB(LF)(SN)" (id 10) (at 91.44 41.91 0)
-      (effects (font (size 1.27 1.27)) hide)
-    )
-    (property "Manufacturer" "JST" (id 11) (at 91.44 41.91 0)
-      (effects (font (size 1.27 1.27)) hide)
-    )
-    (property "Buy early" "N" (id 12) (at 91.44 41.91 0)
-      (effects (font (size 1.27 1.27)) hide)
-    )
-    (pin "1")
-    (pin "2")
-    (pin "3")
-    (pin "MP")
   )
   (symbol (lib_id "mch2021-rescue:AAT4610BIGV-1-T1-Power_Management") (at 156.21 109.22 0) (unit 1)
@@
     (pin "2")
   )
-  (symbol (lib_id "mch2021-rescue:GND-power") (at 96.52 45.72 0) (unit 1)
-    (in_bom yes) (on_board yes)
-    (property "Reference" "#PWR?" (id 0) (at 96.52 52.07 0)
-      (effects (font (size 1.27 1.27)) hide)
-    )
-    (property "Value" "GND" (id 1) (at 96.647 50.1142 0))
-    (property "Footprint" "" (id 2) (at 96.52 45.72 0)
-      (effects (font (size 1.27 1.27)) hide)
-    )
-    (property "Datasheet" "" (id 3) (at 96.52 45.72 0)
-      (effects (font (size 1.27 1.27)) hide)
-    )
+  (symbol (lib_id "Connector_Generic_MountingPin:Conn_01x02_MountingPin") (at 91.44 38.1 0) (unit 1)
+    (in_bom yes) (on_board yes) (fields_autoplaced)
+    (property "Reference" "J6" (id 0) (at 93.472 38.4555 0)
+      (effects (font (size 1.27 1.27)) (justify left))
+    )
+    (property "Value" "" (id 1) (at 93.472 40.9955 0)
+      (effects (font (size 1.27 1.27)) (justify left))
+    )
+    (property "Footprint" "" (id 2) (at 91.44 38.1 0)
+      (effects (font (size 1.27 1.27)) hide)
+    )
+    (property "Datasheet" "~" (id 3) (at 91.44 38.1 0)
+      (effects (font (size 1.27 1.27)) hide)
+    )
+    (pin "1")
+    (pin "2")
+    (pin "MP")
+  )
+  (symbol (lib_id "mch2021-rescue:GND-power") (at 91.44 45.72 0) (unit 1)
+    (in_bom yes) (on_board yes)
+    (property "Reference" "#PWR0224" (id 0) (at 91.44 52.07 0)
+      (effects (font (size 1.27 1.27)) hide)
+    )
+    (property "Value" "GND" (id 1) (at 91.567 50.1142 0))
+    (property "Footprint" "" (id 2) (at 91.44 45.72 0)
+      (effects (font (size 1.27 1.27)) hide)
+    )
+    (property "Datasheet" "" (id 3) (at 91.44 45.72 0)
+      (effects (font (size 1.27 1.27)) hide)
+    )

Commit message: Pre-production final design
Parts:
- C34, C42: value 10u -> (none); footprint Capacitor_SMD:C_0402_1005Metric -> (none)
- C35, C36, C37, C48, C50: value 100n -> (none); footprint Capacitor_SMD:C_0402_1005Metric -> (none)
- C38, C39, C43, C44, C45, C46, C49: value 22u -> (none); footprint Capacitor_SMD:C_0805_2012Metric -> (none)
- C40, C41: value 22p -> (none); footprint Capacitor_SMD:C_0402_1005Metric -> (none)
- D9: value PSBD3D40V1H -> (none); footprint Diode_SMD:D_SOD-323 -> (none)
- J6: Category (none) -> Connectors; LCSC (none) -> C265329; MPN (none) -> S2B-ZR-SM4A-TF(LF)(SN); Manufacturer (none) -> JST
- L3, L4: value 2.2u -> (none); footprint custom:Inductor_MSC20FC -> (none)
- R53, R56: value 1k -> (none); footprint Resistor_SMD:R_0402_1005Metric -> (none)
- R57, R58, R61, R64, R67: value 10k -> (none); footprint Resistor_SMD:R_0402_1005Metric -> (none); MANUFACTURER YAGEO -> UNI-ROYAL
- R59: value 100k -> (none); footprint Resistor_SMD:R_0402_1005Metric -> (none); MANUFACTURER FH -> UNI-ROYAL
- R60: value 45.3k -> (none); footprint Resistor_SMD:R_0402_1005Metric -> (none)
- R62, R68: value 10k -> (none); footprint Resistor_SMD:R_0402_1005Metric -> (none)
- R63: value 4.7k -> (none); footprint Resistor_SMD:R_0402_1005Metric -> (none); MANUFACTURER YAGEO -> UNI-ROYAL
- RN6: value 100k -> (none); footprint Resistor_SMD:R_Array_Convex_4x0603 -> (none)
- SW7: value Switch -> (none); footprint Button_Switch_SMD:SW_SPDT_PCM12 -> (none)
- U11, U12: value SY8079AAC -> (none); footprint Package_TO_SOT_SMD:SOT-23-5 -> (none)
- U13: value XT4054K421MR-G -> (none); footprint Package_TO_SOT_SMD:SOT-23-5 -> (none)
- U14, U15, U16: value SY6280AAC -> (none); footprint Package_TO_SOT_SMD:SOT-23-5 -> (none)

Commit message: Add gerbers, add schematic, finalize design
Parts:
- C34, C42: value (none) -> 10u; footprint (none) -> Capacitor_SMD:C_0402_1005Metric
- C35, C36, C37, C48, C50: value (none) -> 100n; footprint (none) -> Capacitor_SMD:C_0402_1005Metric
- C38, C39, C43, C44, C45, C46, C49: value (none) -> 22u; footprint (none) -> Capacitor_SMD:C_0805_2012Metric
- C40, C41: value (none) -> 22p; footprint (none) -> Capacitor_SMD:C_0402_1005Metric
- D9: value (none) -> PSBD3D40V1H; footprint (none) -> Diode_SMD:D_SOD-323
- J6: value (none) -> Battery; footprint (none) -> custom:JST_S2B-ZR-SM4A-TF(LF)(SN)
- L3, L4: value (none) -> 2.2u; footprint (none) -> custom:Inductor_MSC20FC
- R53, R56: value (none) -> 1k; footprint (none) -> Resistor_SMD:R_0402_1005Metric
- R57, R58, R61, R62, R64, R67, R68: value (none) -> 10k; footprint (none) -> Resistor_SMD:R_0402_1005Metric
- R59: value (none) -> 100k; footprint (none) -> Resistor_SMD:R_0402_1005Metric
- R60: value (none) -> 45.3k; footprint (none) -> Resistor_SMD:R_0402_1005Metric
- R63: value (none) -> 4.7k; footprint (none) -> Resistor_SMD:R_0402_1005Metric
- RN6: value (none) -> 100k; footprint (none) -> Resistor_SMD:R_Array_Convex_4x0603
- SW7: value (none) -> Switch; footprint (none) -> Button_Switch_SMD:SW_SPDT_PCM12
- U11, U12: value (none) -> SY8079AAC; footprint (none) -> Package_TO_SOT_SMD:SOT-23-5
- U13: value (none) -> XT4054K421MR-G; footprint (none) -> Package_TO_SOT_SMD:SOT-23-5
- U14, U15, U16: value (none) -> SY6280AAC; footprint (none) -> Package_TO_SOT_SMD:SOT-23-5

Commit message: have you tried switching the polarity?
Connections:
- net GND: now also J6.1 (Pin_1); no longer J6.2 (Pin_2)
- net VBAT: now also J6.2 (Pin_2); no longer J6.1 (Pin_1)
Other:
- moved on the sheet: J6
Changed lines of the file:
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@@
+    (stroke (width 0) (type default) (color 0 0 0 0))
+  )
+  (wire (pts (xy 103.632 33.02) (xy 91.44 33.02))
     (stroke (width 0) (type default) (color 0 0 0 0))
   )
@@
   )
   (wire (pts (xy 68.58 133.35) (xy 67.31 133.35))
+    (stroke (width 0) (type default) (color 0 0 0 0))
+  )
+  (wire (pts (xy 103.632 45.72) (xy 103.632 33.02))
     (stroke (width 0) (type default) (color 0 0 0 0))
   )
@@
     (pin "2")
   )
-  (symbol (lib_id "Connector_Generic_MountingPin:Conn_01x02_MountingPin") (at 91.44 38.1 0) (unit 1)
+  (symbol (lib_id "Connector_Generic_MountingPin:Conn_01x02_MountingPin") (at 91.44 40.64 0) (mirror x) (unit 1)
     (in_bom yes) (on_board yes) (fields_autoplaced)
-    (property "Reference" "J6" (id 0) (at 93.472 38.4555 0)
-      (effects (font (size 1.27 1.27)) (justify left))
-    )
-    (property "Value" "Battery" (id 1) (at 93.472 40.9955 0)
-      (effects (font (size 1.27 1.27)) (justify left))
-    )
-    (property "Footprint" "custom:JST_S2B-ZR-SM4A-TF(LF)(SN)" (id 2) (at 91.44 38.1 0)
-      (effects (font (size 1.27 1.27)) hide)
-    )
-    (property "Datasheet" "https://datasheet.lcsc.com/lcsc/1912111437_JST-Sales-America-S2B-ZR-SM4A-TF-LF-SN_C265329.pdf" (id 3) (at 91.44 38.1 0)
-      (effects (font (size 1.27 1.27)) hide)
-    )
-    (property "Category" "Connectors" (id 4) (at 91.44 38.1 0)
-      (effects (font (size 1.27 1.27)) hide)
-    )
-    (property "LCSC" "C265329" (id 5) (at 91.44 38.1 0)
-      (effects (font (size 1.27 1.27)) hide)
-    )
-    (property "MPN" "S2B-ZR-SM4A-TF(LF)(SN)" (id 6) (at 91.44 38.1 0)
-      (effects (font (size 1.27 1.27)) hide)
-    )
-    (property "Manufacturer" "JST" (id 7) (at 91.44 38.1 0)
+    (property "Reference" "J6" (id 0) (at 94.488 37.7443 0)
+      (effects (font (size 1.27 1.27)) (justify left))
+    )
+    (property "Value" "Battery" (id 1) (at 94.488 40.2843 0)
+      (effects (font (size 1.27 1.27)) (justify left))
+    )
+    (property "Footprint" "custom:JST_S2B-ZR-SM4A-TF(LF)(SN)" (id 2) (at 91.44 40.64 0)
+      (effects (font (size 1.27 1.27)) hide)
+    )
+    (property "Datasheet" "https://datasheet.lcsc.com/lcsc/1912111437_JST-Sales-America-S2B-ZR-SM4A-TF-LF-SN_C265329.pdf" (id 3) (at 91.44 40.64 0)
+      (effects (font (size 1.27 1.27)) hide)
+    )
+    (property "Category" "Connectors" (id 4) (at 91.44 40.64 0)
+      (effects (font (size 1.27 1.27)) hide)
+    )
+    (property "LCSC" "C265329" (id 5) (at 91.44 40.64 0)
+      (effects (font (size 1.27 1.27)) hide)
+    )
+    (property "MPN" "S2B-ZR-SM4A-TF(LF)(SN)" (id 6) (at 91.44 40.64 0)
+      (effects (font (size 1.27 1.27)) hide)
+    )
+    (property "Manufacturer" "JST" (id 7) (at 91.44 40.64 0)
       (effects (font (size 1.27 1.27)) hide)
     )
@@
     (pin "MP")
   )
-  (symbol (lib_id "mch2021-rescue:GND-power") (at 91.44 45.72 0) (unit 1)
-    (in_bom yes) (on_board yes)
-    (property "Reference" "#PWR0224" (id 0) (at 91.44 52.07 0)
-      (effects (font (size 1.27 1.27)) hide)
-    )
-    (property "Value" "GND" (id 1) (at 91.567 50.1142 0))
-    (property "Footprint" "" (id 2) (at 91.44 45.72 0)
-      (effects (font (size 1.27 1.27)) hide)
-    )
-    (property "Datasheet" "" (id 3) (at 91.44 45.72 0)
-      (effects (font (size 1.27 1.27)) hide)
-    )
+  (symbol (lib_id "mch2021-rescue:GND-power") (at 103.632 45.72 0) (unit 1)
+    (in_bom yes) (on_board yes)
+    (property "Reference" "#PWR0224" (id 0) (at 103.632 52.07 0)
+      (effects (font (size 1.27 1.27)) hide)
+    )
+    (property "Value" "GND" (id 1) (at 103.759 50.1142 0))
+    (property "Footprint" "" (id 2) (at 103.632 45.72 0)
+      (effects (font (size 1.27 1.27)) hide)
+    )
+    (property "Datasheet" "" (id 3) (at 103.632 45.72 0)
+      (effects (font (size 1.27 1.27)) hide)
+    )
