File: power.kicad_sch (KiCad schematic)
At the start: 40 parts, among them J6 Battery, SW7 Switch, U11 SY8079AAC, U12 SY8079AAC, U13 XT4054K421MR-G, U14 SY6280AAC, U15 SY6280AAC, U16 SY6280AAC

Commit message: Mark diode as DNP, replace fuse with SMD0805B110TF
Parts:
- D9: value PSBD3D40V1H -> DNP; Buy early Y -> (none); Category Diodes -> (none); LCSC C110733 -> (none); MPN PSBD3D40V1H -> (none); Manufacturer Shanghai Prisemi Elec -> (none)
Changed lines of the file:
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@@
       (effects (font (size 1.27 1.27)) (justify left))
     )
-    (property "Value" "PSBD3D40V1H" (id 1) (at 162.56 92.71 0)
+    (property "Value" "DNP" (id 1) (at 162.56 92.71 0)
       (effects (font (size 1.27 1.27)) (justify left))
     )
@@
       (effects (font (size 1.27 1.27)) hide)
     )
-    (property "Datasheet" "https://datasheet.lcsc.com/lcsc/1810251323_Shanghai-Prisemi-Elec-PSBD3D40V1H_C110733.pdf" (id 3) (at 156.21 95.25 0)
+    (property "Datasheet" "" (id 3) (at 156.21 95.25 0)
       (effects (font (size 1.27 1.27)) hide)
     )
@@
       (effects (font (size 1.27 1.27)) hide)
     )
-    (property "LCSC" "C110733" (id 5) (at 156.21 95.25 0)
+    (property "LCSC" "" (id 5) (at 156.21 95.25 0)
       (effects (font (size 1.27 1.27)) hide)
     )
-    (property "Category" "Diodes" (id 6) (at 156.21 95.25 0)
+    (property "Category" "" (id 6) (at 156.21 95.25 0)
       (effects (font (size 1.27 1.27)) hide)
     )
-    (property "Description" "Generic part" (id 7) (at 156.21 95.25 0)
+    (property "Description" "" (id 7) (at 156.21 95.25 0)
       (effects (font (size 1.27 1.27)) hide)
     )
-    (property "MPN" "PSBD3D40V1H" (id 8) (at 156.21 95.25 0)
+    (property "MPN" "" (id 8) (at 156.21 95.25 0)
       (effects (font (size 1.27 1.27)) hide)
     )
-    (property "Manufacturer" "Shanghai Prisemi Elec" (id 9) (at 156.21 95.25 0)
+    (property "Manufacturer" "" (id 9) (at 156.21 95.25 0)
       (effects (font (size 1.27 1.27)) hide)
     )
-    (property "Buy early" "Y" (id 10) (at 156.21 95.25 0)
+    (property "Buy early" "" (id 10) (at 156.21 95.25 0)
       (effects (font (size 1.27 1.27)) hide)
     )
