File: bosch.kicad_sch (KiCad schematic)
At the start: 12 parts, among them U8 BNO055, U9 BME680, Y3 32kHz

Commit message: Remove IO expander, move around signals
Parts:
- added TP27: RESET, TestPoint:TestPoint_Pad_1.0x1.0mm, symbol mch2021-rescue:TestPoint-Connector
Connections:
- net RESET: no longer names the net of R47.2, U8.11 (RESET)
- net RESET: now also TP27.1
Changed lines of the file:
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@@
   (title_block
     (title "MCH2022 badge - BOSCH")
-    (date "2022-01-14")
-    (rev "3.1415")
+    (date "2022-03-11")
+    (rev "4")
     (company "BADGE.TEAM")
   )
   (junction (at 85.09 92.71) (diameter 0) (color 0 0 0 0)
   )
+  (junction (at 77.47 100.33) (diameter 0) (color 0 0 0 0)
+  )
   (junction (at 149.86 102.87) (diameter 0) (color 0 0 0 0)
   )
@@
   (junction (at 137.16 95.25) (diameter 0) (color 0 0 0 0)
   )
-  (junction (at 77.47 95.25) (diameter 0) (color 0 0 0 0)
-  )
   (junction (at 87.63 100.33) (diameter 0) (color 0 0 0 0)
   )
@@
     (stroke (width 0) (type default) (color 0 0 0 0))
   )
+  (wire (pts (xy 72.39 100.33) (xy 77.47 100.33))
+    (stroke (width 0) (type default) (color 0 0 0 0))
+  )
   (wire (pts (xy 125.73 104.14) (xy 128.27 104.14))
     (stroke (width 0) (type default) (color 0 0 0 0))
@@
     (stroke (width 0) (type default) (color 0 0 0 0))
   )
-  (wire (pts (xy 77.47 95.25) (xy 77.47 110.49))
+  (wire (pts (xy 77.47 90.17) (xy 77.47 100.33))
     (stroke (width 0) (type default) (color 0 0 0 0))
   )
@@
     (stroke (width 0) (type default) (color 0 0 0 0))
   )
-  (wire (pts (xy 77.47 95.25) (xy 72.39 95.25))
+  (wire (pts (xy 77.47 100.33) (xy 77.47 110.49))
     (stroke (width 0) (type default) (color 0 0 0 0))
   )
@@
   )
   (wire (pts (xy 85.09 92.71) (xy 85.09 90.17))
-    (stroke (width 0) (type default) (color 0 0 0 0))
-  )
-  (wire (pts (xy 77.47 90.17) (xy 77.47 95.25))
     (stroke (width 0) (type default) (color 0 0 0 0))
   )
@@
   )
   (hierarchical_label "SDA" (shape bidirectional) (at 72.39 107.95 180)
-    (effects (font (size 1.27 1.27)) (justify right))
-  )
-  (hierarchical_label "RESET" (shape input) (at 72.39 95.25 180)
     (effects (font (size 1.27 1.27)) (justify right))
   )
@@
       (effects (font (size 1.27 1.27)) hide)
     )
+    (pin "1")
+  )
+  (symbol (lib_id "mch2021-rescue:TestPoint-Connector") (at 72.39 100.33 90) (unit 1)
+    (in_bom yes) (on_board yes)
+    (property "Reference" "TP27" (id 0) (at 70.5612 95.377 90))
+    (property "Value" "RESET" (id 1) (at 70.5612 97.6884 90))
+    (property "Footprint" "TestPoint:TestPoint_Pad_1.0x1.0mm" (id 2) (at 72.39 95.25 0)
+      (effects (font (size 1.27 1.27)) hide)
+    )
+    (property "Datasheet" "~" (id 3) (at 72.39 95.25 0)
+      (effects (font (size 1.27 1.27)) hide)
+    )

Commit message: Remove user I2C bus, connect LCD control signals to ESP32 directly, replace I2S dac
Parts:
- added J3: I2C, custom:1X04_1MM_RA_GND, symbol mch2021-rescue:QWIIC_MCH
- added TP16: SCL, TestPoint:TestPoint_Pad_1.0x1.0mm, symbol mch2021-rescue:TestPoint_Small-Connector
- added TP17: SDA, TestPoint:TestPoint_Pad_1.0x1.0mm, symbol mch2021-rescue:TestPoint_Small-Connector
- added X1: Simple_Addon_v2, Simple_Addon_v2:Simple_Addon_v2-BADGE-2x3-nosilk, symbol Simple_Addon_v2:Simple_Addon_v2
Connections:
- net +3V3: now also J3.2 (VCC), X1.1 (VCC)
- net GND: now also J3.1 (GND), J3.5, J3.6, X1.2 (GND)
- net SCL: now also J3.4 (SCL), TP16.1, X1.4 (SCL)
- net SDA: now also J3.3 (SDA), TP17.1, X1.3 (SDA)
- new net SAO0: X1.5 (GPIO1)
- new net SAO1: X1.6 (GPIO2)
Other:
- note added: "I2C periphereals - BOSCH BNO055 - BOSCH BME680 - SAO expansion header - Qwiic expansion header"
- note removed: "BOSCH BNO055 & BME680 SENSORS"
- moved on the sheet: C26, C27, C28, C29, C30, R47, R48, R49, TP15, TP27, U8, U9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

Commit message: Bill of materials 1/2
Parts:
- C26, C27, C30: value 100n -> (none); footprint Capacitor_SMD:C_0402_1005Metric -> (none); Category (none) -> Capacitors; LCSC C83056 -> (none); Sponsored N -> (none)
- C28, C29: value 22p -> (none); footprint Capacitor_SMD:C_0402_1005Metric -> (none); Category (none) -> Capacitors; LCSC C106203 -> (none); MPN CC0402JRNPO9BN220 -> (none); Sponsored N -> (none)
- J3: value I2C -> (none); footprint custom:1X04_1MM_RA_GND -> (none); Category (none) -> Connectors
- R47, R48, R49: value 4.7k -> (none); footprint Resistor_SMD:R_0402_1005Metric -> (none); Category (none) -> Resistors; Sponsored N -> (none)
- TP15: value BL -> (none); footprint TestPoint:TestPoint_Pad_1.0x1.0mm -> (none); Buy early (none) -> N; Category (none) -> Testpoints; Sponsored (none) -> N
- TP16: value SCL -> (none); footprint TestPoint:TestPoint_Pad_1.0x1.0mm -> (none); Buy early (none) -> N; Category (none) -> Testpoints; Sponsored (none) -> N
- TP17: value SDA -> (none); footprint TestPoint:TestPoint_Pad_1.0x1.0mm -> (none); Buy early (none) -> N; Category (none) -> Testpoints; Sponsored (none) -> N
- TP27: value RESET -> (none); footprint TestPoint:TestPoint_Pad_1.0x1.0mm -> (none); Buy early (none) -> N; Category (none) -> Testpoints; Sponsored (none) -> N
- U8: value BNO055 -> (none); footprint digikey-footprints:LGA-28_5.2x3.8mm_BNO0055 -> (none); Buy early (none) -> N; Category Sensors, Transducers -> ICs
- U9: value BME680 -> (none); footprint Package_LGA:Bosch_LGA-8_3x3mm_P0.8mm_ClockwisePinNumbering -> (none); Buy early (none) -> N; Category (none) -> ICs; Sponsored (none) -> Y
- X1: value Simple_Addon_v2 -> (none); footprint Simple_Addon_v2:Simple_Addon_v2-BADGE-2x3-nosilk -> (none); Buy early (none) -> N; Category (none) -> Connectors; Sponsored (none) -> N
- Y3: value 32kHz -> (none); footprint Crystal:Crystal_SMD_3215-2Pin_3.2x1.5mm -> (none); Buy early (none) -> Y; Category (none) -> Oscillators; MPN (none) -> SF32WK32768D31T002; Manufacturer (none) -> TKD; Sponsored (none) -> N

Commit message: Add more info to BOM
Parts:
- C26, C27, C28, C29, C30, J3: Buy early (none) -> Y; Sponsored (none) -> N
- R47, R48, R49: Buy early (none) -> Y; Manufacturer (none) -> Uni-royal; Sponsored (none) -> N
Changed lines of the file:
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@@
       (effects (font (size 1.27 1.27)) hide)
     )
-    (property "Sponsored" "" (id 7) (at 95.25 119.38 0)
+    (property "Sponsored" "N" (id 7) (at 95.25 119.38 0)
       (effects (font (size 1.27 1.27)) hide)
     )
@@
     )
     (property "Description" "Generic part" (id 9) (at 95.25 119.38 0)
+      (effects (font (size 1.27 1.27)) hide)
+    )
+    (property "Buy early" "Y" (id 10) (at 95.25 119.38 0)
       (effects (font (size 1.27 1.27)) hide)
     )
@@
       (effects (font (size 1.27 1.27)) hide)
     )
-    (property "Sponsored" "" (id 7) (at 104.14 87.63 0)
+    (property "Sponsored" "N" (id 7) (at 104.14 87.63 0)
       (effects (font (size 1.27 1.27)) hide)
     )
@@
       (effects (font (size 1.27 1.27)) hide)
     )
+    (property "Buy early" "Y" (id 11) (at 104.14 87.63 0)
+      (effects (font (size 1.27 1.27)) hide)
+    )
+    (property "Description" "Generic part" (id 12) (at 104.14 87.63 0)
+      (effects (font (size 1.27 1.27)) hide)
+    )
+    (property "Manufacturer" "Uni-royal" (id 13) (at 104.14 87.63 0)
+      (effects (font (size 1.27 1.27)) hide)
+    )
     (pin "1")
     (pin "2")
@@
       (effects (font (size 1.27 1.27)) hide)
     )
-    (property "Sponsored" "" (id 7) (at 52.07 87.63 0)
+    (property "Sponsored" "N" (id 7) (at 52.07 87.63 0)
       (effects (font (size 1.27 1.27)) hide)
     )
@@
     )
     (property "Category" "Resistors" (id 10) (at 52.07 87.63 0)
+      (effects (font (size 1.27 1.27)) hide)
+    )
+    (property "Buy early" "Y" (id 11) (at 52.07 87.63 0)
+      (effects (font (size 1.27 1.27)) hide)
+    )
+    (property "Description" "Generic part" (id 12) (at 52.07 87.63 0)
+      (effects (font (size 1.27 1.27)) hide)
+    )
+    (property "Manufacturer" "Uni-royal" (id 13) (at 52.07 87.63 0)
       (effects (font (size 1.27 1.27)) hide)
     )
@@
       (effects (font (size 1.27 1.27)) hide)
     )
-    (property "Sponsored" "" (id 6) (at 106.68 119.38 0)
+    (property "Sponsored" "N" (id 6) (at 106.68 119.38 0)
       (effects (font (size 1.27 1.27)) hide)
     )
@@
       (effects (font (size 1.27 1.27)) hide)
     )
+    (property "Buy early" "Y" (id 11) (at 106.68 119.38 0)
+      (effects (font (size 1.27 1.27)) hide)
+    )
     (pin "1")
     (pin "2")
@@
       (effects (font (size 1.27 1.27)) hide)
     )
-    (property "Sponsored" "" (id 6) (at 116.84 119.38 0)
+    (property "Sponsored" "N" (id 6) (at 116.84 119.38 0)
       (effects (font (size 1.27 1.27)) hide)
     )
@@
     )
     (property "Description" "Generic part" (id 10) (at 116.84 119.38 0)
+      (effects (font (size 1.27 1.27)) hide)
+    )
+    (property "Buy early" "Y" (id 11) (at 116.84 119.38 0)
       (effects (font (size 1.27 1.27)) hide)
     )
@@
       (effects (font (size 1.27 1.27)) hide)
     )
-    (property "Sponsored" "" (id 7) (at 44.45 87.63 0)
+    (property "Sponsored" "N" (id 7) (at 44.45 87.63 0)
       (effects (font (size 1.27 1.27)) hide)
     )
@@
       (effects (font (size 1.27 1.27)) hide)
     )
+    (property "Buy early" "Y" (id 11) (at 44.45 87.63 0)
+      (effects (font (size 1.27 1.27)) hide)
+    )
+    (property "Description" "Generic part" (id 12) (at 44.45 87.63 0)
+      (effects (font (size 1.27 1.27)) hide)
+    )
+    (property "Manufacturer" "Uni-royal" (id 13) (at 44.45 87.63 0)
+      (effects (font (size 1.27 1.27)) hide)
+    )
     (pin "1")
     (pin "2")
@@
       (effects (font (size 1.27 1.27)) hide)
     )
-    (property "Sponsored" "" (id 7) (at 144.78 119.38 0)
+    (property "Sponsored" "N" (id 7) (at 144.78 119.38 0)
       (effects (font (size 1.27 1.27)) hide)
     )
@@
     )
     (property "Description" "Generic part" (id 9) (at 144.78 119.38 0)
+      (effects (font (size 1.27 1.27)) hide)
+    )
+    (property "Buy early" "Y" (id 10) (at 144.78 119.38 0)
       (effects (font (size 1.27 1.27)) hide)
     )
@@
       (effects (font (size 1.27 1.27)) hide)
     )
-    (property "Sponsored" "" (id 7) (at 27.94 119.38 0)
+    (property "Sponsored" "N" (id 7) (at 27.94 119.38 0)
       (effects (font (size 1.27 1.27)) hide)
     )
@@
     )
     (property "Description" "Generic part" (id 9) (at 27.94 119.38 0)
+      (effects (font (size 1.27 1.27)) hide)
+    )
+    (property "Buy early" "Y" (id 10) (at 27.94 119.38 0)
       (effects (font (size 1.27 1.27)) hide)
     )
@@
       (effects (font (size 1.27 1.27)) hide)
     )
+    (property "Buy early" "Y" (id 10) (at 245.11 76.2 0)
+      (effects (font (size 1.27 1.27)) hide)
+    )
+    (property "Sponsored" "N" (id 11) (at 245.11 76.2 0)
+      (effects (font (size 1.27 1.27)) hide)
+    )

Commit message: Add IR transmitter, modify bill of materials
Parts:
- X1: LCSC (none) -> C92272; MPN (none) -> DS1023-2*3SF11; Manufacturer (none) -> Connfly Elec
Changed lines of the file:
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@@
       (effects (font (size 1.27 1.27)) hide)
     )
-    (property "Datasheet" "~" (id 3) (at 104.14 87.63 0)
+    (property "Datasheet" "" (id 3) (at 104.14 87.63 0)
       (effects (font (size 1.27 1.27)) hide)
     )
@@
       (effects (font (size 1.27 1.27)) hide)
     )
-    (property "Datasheet" "~" (id 3) (at 52.07 87.63 0)
+    (property "Datasheet" "" (id 3) (at 52.07 87.63 0)
       (effects (font (size 1.27 1.27)) hide)
     )
@@
       (effects (font (size 1.27 1.27)) hide)
     )
-    (property "Datasheet" "~" (id 3) (at 44.45 87.63 0)
+    (property "Datasheet" "" (id 3) (at 44.45 87.63 0)
       (effects (font (size 1.27 1.27)) hide)
     )
@@
       (effects (font (size 1.27 1.27)) hide)
     )
-    (property "Datasheet" "~" (id 3) (at 39.37 87.63 0)
+    (property "Datasheet" "" (id 3) (at 39.37 87.63 0)
       (effects (font (size 1.27 1.27)) hide)
     )
@@
       (effects (font (size 1.27 1.27)) hide)
     )
-    (property "Datasheet" "~" (id 3) (at 228.6 72.39 0)
+    (property "Datasheet" "" (id 3) (at 228.6 72.39 0)
       (effects (font (size 1.27 1.27)) hide)
     )
@@
       (effects (font (size 1.27 1.27)) hide)
     )
-    (property "Datasheet" "~" (id 3) (at 226.06 74.93 0)
+    (property "Datasheet" "" (id 3) (at 226.06 74.93 0)
       (effects (font (size 1.27 1.27)) hide)
     )
@@
       (effects (font (size 1.27 1.27)) hide)
     )
-    (property "Datasheet" "" (id 3) (at 246.38 109.22 0)
+    (property "Datasheet" "https://datasheet.lcsc.com/lcsc/2004241810_CONNFLY-Elec-DS1023-2-3SF11_C92272.pdf" (id 3) (at 246.38 109.22 0)
       (effects (font (size 1.27 1.27)) hide)
     )
@@
     )
     (property "Sponsored" "N" (id 7) (at 246.38 114.3 0)
+      (effects (font (size 1.27 1.27)) hide)
+    )
+    (property "LCSC" "C92272" (id 8) (at 246.38 114.3 0)
+      (effects (font (size 1.27 1.27)) hide)
+    )
+    (property "MPN" "DS1023-2*3SF11" (id 9) (at 246.38 114.3 0)
+      (effects (font (size 1.27 1.27)) hide)
+    )
+    (property "Manufacturer" "Connfly Elec" (id 10) (at 246.38 114.3 0)
       (effects (font (size 1.27 1.27)) hide)
     )
@@
       (effects (font (size 1.27 1.27)) hide)
     )
-    (property "Datasheet" "~" (id 3) (at 39.37 95.25 0)
-      (effects (font (size 1.27 1.27)) hide)
-    )
+    (property "Datasheet" "" (id 3) (at 39.37 95.25 0)
+      (effects (font (size 1.27 1.27)) hide)
+    )

Commit message: Add passives to BOM
Parts:
- C26, C27, C30: LCSC (none) -> C307331; MPN (none) -> CL05B104KB54PNC; Manufacturer (none) -> Samsung Electro-Mechanics; Minimal voltage rating (none) -> 10; Voltage rating (none) -> 50
- C28, C29: LCSC (none) -> C466226; MPN (none) -> TCC0402C0G220J500AT; Manufacturer (none) -> CCTC; Minimal voltage rating (none) -> 10; Voltage rating (none) -> 50
- R47, R48, R49: LCSC C25940 -> C25900; MPN 0402WGJ0472TCE -> 0402WGF4701TCE
Changed lines of the file:
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@@
       (effects (font (size 1.27 1.27)) hide)
     )
-    (property "Datasheet" "" (id 3) (at 95.25 119.38 0)
-      (effects (font (size 1.27 1.27)) hide)
-    )
-    (property "LCSC" "" (id 4) (at 95.25 119.38 0)
+    (property "Datasheet" "https://datasheet.lcsc.com/lcsc/1810191222_Samsung-Electro-Mechanics-CL05B104KB54PNC_C307331.pdf" (id 3) (at 95.25 119.38 0)
+      (effects (font (size 1.27 1.27)) hide)
+    )
+    (property "LCSC" "C307331" (id 4) (at 95.25 119.38 0)
       (effects (font (size 1.27 1.27)) hide)
     )
@@
     )
     (property "Buy early" "Y" (id 10) (at 95.25 119.38 0)
+      (effects (font (size 1.27 1.27)) hide)
+    )
+    (property "MPN" "CL05B104KB54PNC" (id 11) (at 95.25 119.38 0)
+      (effects (font (size 1.27 1.27)) hide)
+    )
+    (property "Manufacturer" "Samsung Electro-Mechanics" (id 12) (at 95.25 119.38 0)
+      (effects (font (size 1.27 1.27)) hide)
+    )
+    (property "Minimal voltage rating" "10" (id 13) (at 95.25 119.38 0)
+      (effects (font (size 1.27 1.27)) hide)
+    )
+    (property "Voltage rating" "50" (id 14) (at 95.25 119.38 0)
       (effects (font (size 1.27 1.27)) hide)
     )
@@
       (effects (font (size 1.27 1.27)) hide)
     )
-    (property "Datasheet" "" (id 3) (at 104.14 87.63 0)
+    (property "Datasheet" "https://datasheet.lcsc.com/lcsc/2110260030_UNI-ROYAL-Uniroyal-Elec-0402WGF4701TCE_C25900.pdf" (id 3) (at 104.14 87.63 0)
       (effects (font (size 1.27 1.27)) hide)
     )
@@
       (effects (font (size 1.27 1.27)) hide)
     )
-    (property "LCSC" "C25940" (id 5) (at 104.14 87.63 0)
+    (property "LCSC" "C25900" (id 5) (at 104.14 87.63 0)
       (effects (font (size 1.27 1.27)) hide)
     )
@@
       (effects (font (size 1.27 1.27)) hide)
     )
-    (property "MPN" "0402WGJ0472TCE" (id 9) (at 104.14 87.63 0)
+    (property "MPN" "0402WGF4701TCE" (id 9) (at 104.14 87.63 0)
       (effects (font (size 1.27 1.27)) hide)
     )
@@
       (effects (font (size 1.27 1.27)) hide)
     )
-    (property "Datasheet" "" (id 3) (at 52.07 87.63 0)
+    (property "Datasheet" "https://datasheet.lcsc.com/lcsc/2110260030_UNI-ROYAL-Uniroyal-Elec-0402WGF4701TCE_C25900.pdf" (id 3) (at 52.07 87.63 0)
       (effects (font (size 1.27 1.27)) hide)
     )
@@
       (effects (font (size 1.27 1.27)) hide)
     )
-    (property "LCSC" "C25940" (id 5) (at 52.07 87.63 0)
+    (property "LCSC" "C25900" (id 5) (at 52.07 87.63 0)
       (effects (font (size 1.27 1.27)) hide)
     )
@@
       (effects (font (size 1.27 1.27)) hide)
     )
-    (property "MPN" "0402WGJ0472TCE" (id 9) (at 52.07 87.63 0)
+    (property "MPN" "0402WGF4701TCE" (id 9) (at 52.07 87.63 0)
       (effects (font (size 1.27 1.27)) hide)
     )
@@
       (effects (font (size 1.27 1.27)) hide)
     )
-    (property "Datasheet" "" (id 3) (at 106.68 119.38 0)
-      (effects (font (size 1.27 1.27)) hide)
-    )
-    (property "LCSC" "" (id 4) (at 106.68 119.38 0)
+    (property "Datasheet" "https://datasheet.lcsc.com/lcsc/1912111437_CCTC-TCC0402C0G220J500AT_C466226.pdf" (id 3) (at 106.68 119.38 0)
+      (effects (font (size 1.27 1.27)) hide)
+    )
+    (property "LCSC" "C466226" (id 4) (at 106.68 119.38 0)
       (effects (font (size 1.27 1.27)) hide)
     )
@@
       (effects (font (size 1.27 1.27)) hide)
     )
-    (property "MPN" "" (id 8) (at 106.68 119.38 0)
+    (property "MPN" "TCC0402C0G220J500AT" (id 8) (at 106.68 119.38 0)
       (effects (font (size 1.27 1.27)) hide)
     )
@@
       (effects (font (size 1.27 1.27)) hide)
     )
+    (property "Manufacturer" "CCTC" (id 12) (at 106.68 119.38 0)
+      (effects (font (size 1.27 1.27)) hide)
+    )
+    (property "Minimal voltage rating" "10" (id 13) (at 106.68 119.38 0)
+      (effects (font (size 1.27 1.27)) hide)
+    )
+    (property "Voltage rating" "50" (id 14) (at 106.68 119.38 0)
+      (effects (font (size 1.27 1.27)) hide)
+    )
     (pin "1")
     (pin "2")
@@
       (effects (font (size 1.27 1.27)) hide)
     )
-    (property "Datasheet" "" (id 3) (at 116.84 119.38 0)
-      (effects (font (size 1.27 1.27)) hide)
-    )
-    (property "LCSC" "" (id 4) (at 116.84 119.38 0)
+    (property "Datasheet" "https://datasheet.lcsc.com/lcsc/1912111437_CCTC-TCC0402C0G220J500AT_C466226.pdf" (id 3) (at 116.84 119.38 0)
+      (effects (font (size 1.27 1.27)) hide)
+    )
+    (property "LCSC" "C466226" (id 4) (at 116.84 119.38 0)
       (effects (font (size 1.27 1.27)) hide)
     )
@@
       (effects (font (size 1.27 1.27)) hide)
     )
-    (property "MPN" "" (id 8) (at 116.84 119.38 0)
+    (property "MPN" "TCC0402C0G220J500AT" (id 8) (at 116.84 119.38 0)
       (effects (font (size 1.27 1.27)) hide)
     )
@@
     )
     (property "Buy early" "Y" (id 11) (at 116.84 119.38 0)
+      (effects (font (size 1.27 1.27)) hide)
+    )
+    (property "Manufacturer" "CCTC" (id 12) (at 116.84 119.38 0)
+      (effects (font (size 1.27 1.27)) hide)
+    )
+    (property "Minimal voltage rating" "10" (id 13) (at 116.84 119.38 0)
+      (effects (font (size 1.27 1.27)) hide)
+    )
+    (property "Voltage rating" "50" (id 14) (at 116.84 119.38 0)
       (effects (font (size 1.27 1.27)) hide)
     )
@@
       (effects (font (size 1.27 1.27)) hide)
     )
-    (property "Datasheet" "" (id 3) (at 44.45 87.63 0)
+    (property "Datasheet" "https://datasheet.lcsc.com/lcsc/2110260030_UNI-ROYAL-Uniroyal-Elec-0402WGF4701TCE_C25900.pdf" (id 3) (at 44.45 87.63 0)
       (effects (font (size 1.27 1.27)) hide)
     )
@@
       (effects (font (size 1.27 1.27)) hide)
     )
-    (property "LCSC" "C25940" (id 5) (at 44.45 87.63 0)
+    (property "LCSC" "C25900" (id 5) (at 44.45 87.63 0)
       (effects (font (size 1.27 1.27)) hide)
     )
@@
       (effects (font (size 1.27 1.27)) hide)
     )
-    (property "MPN" "0402WGJ0472TCE" (id 9) (at 44.45 87.63 0)
+    (property "MPN" "0402WGF4701TCE" (id 9) (at 44.45 87.63 0)
       (effects (font (size 1.27 1.27)) hide)
     )
@@
       (effects (font (size 1.27 1.27)) hide)
     )
-    (property "Datasheet" "" (id 3) (at 144.78 119.38 0)
-      (effects (font (size 1.27 1.27)) hide)
-    )
-    (property "LCSC" "" (id 4) (at 144.78 119.38 0)
+    (property "Datasheet" "https://datasheet.lcsc.com/lcsc/1810191222_Samsung-Electro-Mechanics-CL05B104KB54PNC_C307331.pdf" (id 3) (at 144.78 119.38 0)
+      (effects (font (size 1.27 1.27)) hide)
+    )
+    (property "LCSC" "C307331" (id 4) (at 144.78 119.38 0)
       (effects (font (size 1.27 1.27)) hide)
     )
@@
     )
     (property "Buy early" "Y" (id 10) (at 144.78 119.38 0)
+      (effects (font (size 1.27 1.27)) hide)
+    )
+    (property "MPN" "CL05B104KB54PNC" (id 11) (at 144.78 119.38 0)
+      (effects (font (size 1.27 1.27)) hide)
+    )
+    (property "Manufacturer" "Samsung Electro-Mechanics" (id 12) (at 144.78 119.38 0)
+      (effects (font (size 1.27 1.27)) hide)
+    )
+    (property "Minimal voltage rating" "10" (id 13) (at 144.78 119.38 0)
+      (effects (font (size 1.27 1.27)) hide)
+    )
+    (property "Voltage rating" "50" (id 14) (at 144.78 119.38 0)
       (effects (font (size 1.27 1.27)) hide)
     )
@@
       (effects (font (size 1.27 1.27)) hide)
     )
-    (property "Datasheet" "" (id 3) (at 27.94 119.38 0)
-      (effects (font (size 1.27 1.27)) hide)
-    )
-    (property "LCSC" "" (id 4) (at 27.94 119.38 0)
+    (property "Datasheet" "https://datasheet.lcsc.com/lcsc/1810191222_Samsung-Electro-Mechanics-CL05B104KB54PNC_C307331.pdf" (id 3) (at 27.94 119.38 0)
+      (effects (font (size 1.27 1.27)) hide)
+    )
+    (property "LCSC" "C307331" (id 4) (at 27.94 119.38 0)
       (effects (font (size 1.27 1.27)) hide)
     )
@@
       (effects (font (size 1.27 1.27)) hide)
     )
+    (property "MPN" "CL05B104KB54PNC" (id 11) (at 27.94 119.38 0)
+      (effects (font (size 1.27 1.27)) hide)
+    )
+    (property "Manufacturer" "Samsung Electro-Mechanics" (id 12) (at 27.94 119.38 0)
+      (effects (font (size 1.27 1.27)) hide)
+    )
+    (property "Minimal voltage rating" "10" (id 13) (at 27.94 119.38 0)
+      (effects (font (size 1.27 1.27)) hide)
+    )
+    (property "Voltage rating" "50" (id 14) (at 27.94 119.38 0)
+      (effects (font (size 1.27 1.27)) hide)
+    )
