File: bosch.kicad_sch (KiCad schematic)
At the start: 17 parts

Commit message: Artwork stuff
Parts:
- C26, C27, C30: value (none) -> 100n; footprint (none) -> Capacitor_SMD:C_0402_1005Metric
- C28, C29: value (none) -> 22p; footprint (none) -> Capacitor_SMD:C_0402_1005Metric
- J3: value (none) -> I2C; footprint (none) -> custom:1X04_1MM_RA_GND
- R47, R48, R49: value (none) -> 4.7k; footprint (none) -> Resistor_SMD:R_0402_1005Metric
- TP15, TP16, TP17, TP27: value (none) -> Testpoint; footprint (none) -> TestPoint:TestPoint_Pad_1.0x1.0mm
- U8: value (none) -> BNO055; footprint (none) -> digikey-footprints:LGA-28_5.2x3.8mm_BNO0055
- U9: value (none) -> BME680; footprint (none) -> Package_LGA:Bosch_LGA-8_3x3mm_P0.8mm_ClockwisePinNumbering
- X1: value (none) -> Simple_Addon_v2; footprint (none) -> Simple_Addon_v2:Simple_Addon_v2-BADGE-2x3-nosilk
- Y3: value (none) -> 32kHz; footprint (none) -> Crystal:Crystal_SMD_3215-2Pin_3.2x1.5mm
Changed lines of the file:
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@@
       (effects (font (size 1.27 1.27)) (justify right))
     )
-    (property "Value" "" (id 1) (at 157.48 96.52 0)
+    (property "Value" "BME680" (id 1) (at 157.48 96.52 0)
       (effects (font (size 1.27 1.27)) (justify right))
     )
-    (property "Footprint" "" (id 2) (at 199.39 119.38 0)
+    (property "Footprint" "Package_LGA:Bosch_LGA-8_3x3mm_P0.8mm_ClockwisePinNumbering" (id 2) (at 199.39 119.38 0)
       (effects (font (size 1.27 1.27)) hide)
     )
@@
     (in_bom yes) (on_board yes)
     (property "Reference" "U8" (id 0) (at 60.96 88.9 0))
-    (property "Value" "" (id 1) (at 86.36 88.9 0))
-    (property "Footprint" "" (id 2) (at 80.01 97.79 0)
+    (property "Value" "BNO055" (id 1) (at 86.36 88.9 0))
+    (property "Footprint" "digikey-footprints:LGA-28_5.2x3.8mm_BNO0055" (id 2) (at 80.01 97.79 0)
       (effects (font (size 1.524 1.524)) (justify left) hide)
     )
@@
       (effects (font (size 1.27 1.27)) (justify left))
     )
-    (property "Value" "" (id 1) (at 99.06 121.92 90)
-      (effects (font (size 1.27 1.27)) (justify left))
-    )
-    (property "Footprint" "" (id 2) (at 96.2152 123.19 0)
+    (property "Value" "100n" (id 1) (at 99.06 121.92 90)
+      (effects (font (size 1.27 1.27)) (justify left))
+    )
+    (property "Footprint" "Capacitor_SMD:C_0402_1005Metric" (id 2) (at 96.2152 123.19 0)
       (effects (font (size 1.27 1.27)) hide)
     )
@@
       (effects (font (size 1.27 1.27)) (justify left))
     )
-    (property "Value" "" (id 1) (at 105.6386 88.773 0)
-      (effects (font (size 1.27 1.27)) (justify left))
-    )
-    (property "Footprint" "" (id 2) (at 104.14 87.63 0)
+    (property "Value" "4.7k" (id 1) (at 105.6386 88.773 0)
+      (effects (font (size 1.27 1.27)) (justify left))
+    )
+    (property "Footprint" "Resistor_SMD:R_0402_1005Metric" (id 2) (at 104.14 87.63 0)
       (effects (font (size 1.27 1.27)) hide)
     )
@@
       (effects (font (size 1.27 1.27)) (justify left))
     )
-    (property "Value" "" (id 1) (at 53.5686 88.773 0)
-      (effects (font (size 1.27 1.27)) (justify left))
-    )
-    (property "Footprint" "" (id 2) (at 52.07 87.63 0)
+    (property "Value" "4.7k" (id 1) (at 53.5686 88.773 0)
+      (effects (font (size 1.27 1.27)) (justify left))
+    )
+    (property "Footprint" "Resistor_SMD:R_0402_1005Metric" (id 2) (at 52.07 87.63 0)
       (effects (font (size 1.27 1.27)) hide)
     )
@@
       (effects (font (size 1.27 1.27)) (justify left))
     )
-    (property "Value" "" (id 1) (at 111.76 121.92 0)
-      (effects (font (size 1.27 1.27)) (justify left))
-    )
-    (property "Footprint" "" (id 2) (at 105.7148 123.19 0)
+    (property "Value" "22p" (id 1) (at 111.76 121.92 0)
+      (effects (font (size 1.27 1.27)) (justify left))
+    )
+    (property "Footprint" "Capacitor_SMD:C_0402_1005Metric" (id 2) (at 105.7148 123.19 0)
       (effects (font (size 1.27 1.27)) hide)
     )
@@
       (effects (font (size 1.27 1.27)) (justify left))
     )
-    (property "Value" "" (id 1) (at 121.92 121.92 0)
-      (effects (font (size 1.27 1.27)) (justify left))
-    )
-    (property "Footprint" "" (id 2) (at 115.8748 123.19 0)
+    (property "Value" "22p" (id 1) (at 121.92 121.92 0)
+      (effects (font (size 1.27 1.27)) (justify left))
+    )
+    (property "Footprint" "Capacitor_SMD:C_0402_1005Metric" (id 2) (at 115.8748 123.19 0)
       (effects (font (size 1.27 1.27)) hide)
     )
@@
       (effects (font (size 1.27 1.27)) (justify left))
     )
-    (property "Value" "" (id 1) (at 110.617 105.1052 90)
-      (effects (font (size 1.27 1.27)) (justify left))
-    )
-    (property "Footprint" "" (id 2) (at 111.76 102.87 0)
+    (property "Value" "32kHz" (id 1) (at 110.617 105.1052 90)
+      (effects (font (size 1.27 1.27)) (justify left))
+    )
+    (property "Footprint" "Crystal:Crystal_SMD_3215-2Pin_3.2x1.5mm" (id 2) (at 111.76 102.87 0)
       (effects (font (size 1.27 1.27)) hide)
     )
@@
       (effects (font (size 1.27 1.27)) (justify left))
     )
-    (property "Value" "" (id 1) (at 45.9486 88.773 0)
-      (effects (font (size 1.27 1.27)) (justify left))
-    )
-    (property "Footprint" "" (id 2) (at 44.45 87.63 0)
+    (property "Value" "4.7k" (id 1) (at 45.9486 88.773 0)
+      (effects (font (size 1.27 1.27)) (justify left))
+    )
+    (property "Footprint" "Resistor_SMD:R_0402_1005Metric" (id 2) (at 44.45 87.63 0)
       (effects (font (size 1.27 1.27)) hide)
     )
@@
       (effects (font (size 1.27 1.27)) (justify left))
     )
-    (property "Value" "" (id 1) (at 148.59 121.92 90)
-      (effects (font (size 1.27 1.27)) (justify left))
-    )
-    (property "Footprint" "" (id 2) (at 145.7452 123.19 0)
+    (property "Value" "100n" (id 1) (at 148.59 121.92 90)
+      (effects (font (size 1.27 1.27)) (justify left))
+    )
+    (property "Footprint" "Capacitor_SMD:C_0402_1005Metric" (id 2) (at 145.7452 123.19 0)
       (effects (font (size 1.27 1.27)) hide)
     )
@@
       (effects (font (size 1.27 1.27)) (justify left))
     )
-    (property "Value" "" (id 1) (at 31.75 121.92 90)
-      (effects (font (size 1.27 1.27)) (justify left))
-    )
-    (property "Footprint" "" (id 2) (at 28.9052 123.19 0)
+    (property "Value" "100n" (id 1) (at 31.75 121.92 90)
+      (effects (font (size 1.27 1.27)) (justify left))
+    )
+    (property "Footprint" "Capacitor_SMD:C_0402_1005Metric" (id 2) (at 28.9052 123.19 0)
       (effects (font (size 1.27 1.27)) hide)
     )
@@
     (in_bom yes) (on_board yes)
     (property "Reference" "TP15" (id 0) (at 37.5412 87.757 90))
-    (property "Value" "" (id 1) (at 37.5412 90.0684 90))
-    (property "Footprint" "" (id 2) (at 39.37 87.63 0)
+    (property "Value" "Testpoint" (id 1) (at 37.5412 90.0684 90))
+    (property "Footprint" "TestPoint:TestPoint_Pad_1.0x1.0mm" (id 2) (at 39.37 87.63 0)
       (effects (font (size 1.27 1.27)) hide)
     )
@@
       (effects (font (size 1.27 1.27)) (justify left))
     )
-    (property "Value" "" (id 1) (at 232.4608 71.247 0)
+    (property "Value" "Testpoint" (id 1) (at 232.4608 71.247 0)
       (effects (font (size 1.27 1.27)) (justify left) hide)
     )
-    (property "Footprint" "" (id 2) (at 228.6 72.39 0)
+    (property "Footprint" "TestPoint:TestPoint_Pad_1.0x1.0mm" (id 2) (at 228.6 72.39 0)
       (effects (font (size 1.27 1.27)) hide)
     )
@@
       (effects (font (size 1.143 1.143)))
     )
-    (property "Value" "" (id 1) (at 255.27 80.01 90)
+    (property "Value" "I2C" (id 1) (at 255.27 80.01 90)
       (effects (font (size 1.143 1.143)))
     )
-    (property "Footprint" "" (id 2) (at 245.11 88.9 0)
+    (property "Footprint" "custom:1X04_1MM_RA_GND" (id 2) (at 245.11 88.9 0)
       (effects (font (size 0.508 0.508)) hide)
     )
@@
       (effects (font (size 1.27 1.27)) (justify left))
     )
-    (property "Value" "" (id 1) (at 229.9208 73.787 0)
+    (property "Value" "Testpoint" (id 1) (at 229.9208 73.787 0)
       (effects (font (size 1.27 1.27)) (justify left) hide)
     )
-    (property "Footprint" "" (id 2) (at 226.06 74.93 0)
+    (property "Footprint" "TestPoint:TestPoint_Pad_1.0x1.0mm" (id 2) (at 226.06 74.93 0)
       (effects (font (size 1.27 1.27)) hide)
     )
@@
     (in_bom yes) (on_board yes)
     (property "Reference" "X1" (id 0) (at 234.569 114.3 90))
-    (property "Value" "" (id 1) (at 236.8804 114.3 90))
-    (property "Footprint" "" (id 2) (at 246.38 109.22 0)
+    (property "Value" "Simple_Addon_v2" (id 1) (at 236.8804 114.3 90))
+    (property "Footprint" "Simple_Addon_v2:Simple_Addon_v2-BADGE-2x3-nosilk" (id 2) (at 246.38 109.22 0)
       (effects (font (size 1.27 1.27)) hide)
     )
@@
     (in_bom yes) (on_board yes)
     (property "Reference" "TP27" (id 0) (at 37.5412 95.377 90))
-    (property "Value" "" (id 1) (at 37.5412 97.6884 90))
-    (property "Footprint" "" (id 2) (at 39.37 95.25 0)
-      (effects (font (size 1.27 1.27)) hide)
-    )
+    (property "Value" "Testpoint" (id 1) (at 37.5412 97.6884 90))
+    (property "Footprint" "TestPoint:TestPoint_Pad_1.0x1.0mm" (id 2) (at 39.37 95.25 0)
+      (effects (font (size 1.27 1.27)) hide)
+    )

Commit message: Add lanyard holes, component placement
Parts:
- removed TP16, TP17: Testpoint, TestPoint:TestPoint_Pad_1.0x1.0mm, symbol mch2021-rescue:TestPoint_Small-Connector
Changed lines of the file:
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@@
   (junction (at 52.07 92.71) (diameter 0) (color 0 0 0 0)
   )
-  (junction (at 233.68 72.39) (diameter 0) (color 0 0 0 0)
-  )
   (junction (at 44.45 100.33) (diameter 0) (color 0 0 0 0)
   )
@@
   )
   (junction (at 54.61 100.33) (diameter 0) (color 0 0 0 0)
-  )
-  (junction (at 231.14 74.93) (diameter 0) (color 0 0 0 0)
   )
   (junction (at 54.61 102.87) (diameter 0) (color 0 0 0 0)
@@
     (pin "1")
   )
-  (symbol (lib_id "mch2021-rescue:TestPoint_Small-Connector") (at 233.68 72.39 180) (unit 1)
-    (in_bom yes) (on_board yes)
-    (property "Reference" "TP17" (id 0) (at 238.76 72.39 0)
-      (effects (font (size 1.27 1.27)) (justify left))
-    )
-    (property "Value" "Testpoint" (id 1) (at 232.4608 71.247 0)
-      (effects (font (size 1.27 1.27)) (justify left) hide)
-    )
-    (property "Footprint" "TestPoint:TestPoint_Pad_1.0x1.0mm" (id 2) (at 228.6 72.39 0)
-      (effects (font (size 1.27 1.27)) hide)
-    )
-    (property "Datasheet" "" (id 3) (at 228.6 72.39 0)
-      (effects (font (size 1.27 1.27)) hide)
-    )
-    (property "Category" "Testpoints" (id 4) (at 233.68 72.39 0)
-      (effects (font (size 1.27 1.27)) hide)
-    )
-    (property "Buy early" "N" (id 5) (at 233.68 72.39 0)
-      (effects (font (size 1.27 1.27)) hide)
-    )
-    (property "Sponsored" "N" (id 6) (at 233.68 72.39 0)
-      (effects (font (size 1.27 1.27)) hide)
-    )
-    (pin "1")
-  )
   (symbol (lib_id "mch2021-rescue:QWIIC_MCH") (at 245.11 76.2 180) (unit 1)
     (in_bom yes) (on_board yes)
@@
       (effects (font (size 1.27 1.27)) hide)
     )
-    (pin "1")
-  )
-  (symbol (lib_id "mch2021-rescue:TestPoint_Small-Connector") (at 231.14 74.93 180) (unit 1)
-    (in_bom yes) (on_board yes)
-    (property "Reference" "TP16" (id 0) (at 236.22 74.93 0)
-      (effects (font (size 1.27 1.27)) (justify left))
-    )
-    (property "Value" "Testpoint" (id 1) (at 229.9208 73.787 0)
-      (effects (font (size 1.27 1.27)) (justify left) hide)
-    )
-    (property "Footprint" "TestPoint:TestPoint_Pad_1.0x1.0mm" (id 2) (at 226.06 74.93 0)
-      (effects (font (size 1.27 1.27)) hide)
-    )
-    (property "Datasheet" "" (id 3) (at 226.06 74.93 0)
-      (effects (font (size 1.27 1.27)) hide)
-    )
-    (property "Category" "Testpoints" (id 4) (at 231.14 74.93 0)
-      (effects (font (size 1.27 1.27)) hide)
-    )
-    (property "Buy early" "N" (id 5) (at 231.14 74.93 0)
-      (effects (font (size 1.27 1.27)) hide)
-    )
-    (property "Sponsored" "N" (id 6) (at 231.14 74.93 0)
-      (effects (font (size 1.27 1.27)) hide)
-    )
