File: bosch.kicad_sch (KiCad schematic)
At the start: 15 parts, among them J3 I2C, U8 BNO055, U9 BME680, X1 Simple_Addon_v2, Y3 32kHz

Commit message: Pre-production final design
Parts:
- C26, C27, C30: value 100n -> (none); footprint Capacitor_SMD:C_0402_1005Metric -> (none)
- C28, C29: value 22p -> (none); footprint Capacitor_SMD:C_0402_1005Metric -> (none)
- J3: value I2C -> (none); footprint custom:1X04_1MM_RA_GND -> (none)
- R47, R48, R49: value 4.7k -> (none); footprint Resistor_SMD:R_0402_1005Metric -> (none)
- TP15, TP27: value Testpoint -> (none); footprint TestPoint:TestPoint_Pad_1.0x1.0mm -> (none)
- U8: value BNO055 -> (none); footprint digikey-footprints:LGA-28_5.2x3.8mm_BNO0055 -> (none)
- U9: value BME680 -> (none); footprint Package_LGA:Bosch_LGA-8_3x3mm_P0.8mm_ClockwisePinNumbering -> (none)
- X1: value Simple_Addon_v2 -> (none); footprint Simple_Addon_v2:Simple_Addon_v2-BADGE-2x3-nosilk -> (none)
- Y3: value 32kHz -> (none); footprint Crystal:Crystal_SMD_3215-2Pin_3.2x1.5mm -> (none)
Changed lines of the file:
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@@
   (title_block
     (title "MCH2022 badge - BOSCH")
-    (date "2022-03-11")
-    (rev "4")
+    (date "2022-04-24")
+    (rev "Pre-production final")
     (company "BADGE.TEAM")
   )
@@
       (effects (font (size 1.27 1.27)) (justify right))
     )
-    (property "Value" "BME680" (id 1) (at 157.48 96.52 0)
+    (property "Value" "" (id 1) (at 157.48 96.52 0)
       (effects (font (size 1.27 1.27)) (justify right))
     )
-    (property "Footprint" "Package_LGA:Bosch_LGA-8_3x3mm_P0.8mm_ClockwisePinNumbering" (id 2) (at 199.39 119.38 0)
+    (property "Footprint" "" (id 2) (at 199.39 119.38 0)
       (effects (font (size 1.27 1.27)) hide)
     )
@@
     (in_bom yes) (on_board yes)
     (property "Reference" "U8" (id 0) (at 60.96 88.9 0))
-    (property "Value" "BNO055" (id 1) (at 86.36 88.9 0))
-    (property "Footprint" "digikey-footprints:LGA-28_5.2x3.8mm_BNO0055" (id 2) (at 80.01 97.79 0)
+    (property "Value" "" (id 1) (at 86.36 88.9 0))
+    (property "Footprint" "" (id 2) (at 80.01 97.79 0)
       (effects (font (size 1.524 1.524)) (justify left) hide)
     )
@@
       (effects (font (size 1.27 1.27)) (justify left))
     )
-    (property "Value" "100n" (id 1) (at 99.06 121.92 90)
-      (effects (font (size 1.27 1.27)) (justify left))
-    )
-    (property "Footprint" "Capacitor_SMD:C_0402_1005Metric" (id 2) (at 96.2152 123.19 0)
+    (property "Value" "" (id 1) (at 99.06 121.92 90)
+      (effects (font (size 1.27 1.27)) (justify left))
+    )
+    (property "Footprint" "" (id 2) (at 96.2152 123.19 0)
       (effects (font (size 1.27 1.27)) hide)
     )
@@
       (effects (font (size 1.27 1.27)) (justify left))
     )
-    (property "Value" "4.7k" (id 1) (at 105.6386 88.773 0)
-      (effects (font (size 1.27 1.27)) (justify left))
-    )
-    (property "Footprint" "Resistor_SMD:R_0402_1005Metric" (id 2) (at 104.14 87.63 0)
+    (property "Value" "" (id 1) (at 105.6386 88.773 0)
+      (effects (font (size 1.27 1.27)) (justify left))
+    )
+    (property "Footprint" "" (id 2) (at 104.14 87.63 0)
       (effects (font (size 1.27 1.27)) hide)
     )
@@
       (effects (font (size 1.27 1.27)) (justify left))
     )
-    (property "Value" "4.7k" (id 1) (at 53.5686 88.773 0)
-      (effects (font (size 1.27 1.27)) (justify left))
-    )
-    (property "Footprint" "Resistor_SMD:R_0402_1005Metric" (id 2) (at 52.07 87.63 0)
+    (property "Value" "" (id 1) (at 53.5686 88.773 0)
+      (effects (font (size 1.27 1.27)) (justify left))
+    )
+    (property "Footprint" "" (id 2) (at 52.07 87.63 0)
       (effects (font (size 1.27 1.27)) hide)
     )
@@
       (effects (font (size 1.27 1.27)) (justify left))
     )
-    (property "Value" "22p" (id 1) (at 111.76 121.92 0)
-      (effects (font (size 1.27 1.27)) (justify left))
-    )
-    (property "Footprint" "Capacitor_SMD:C_0402_1005Metric" (id 2) (at 105.7148 123.19 0)
+    (property "Value" "" (id 1) (at 111.76 121.92 0)
+      (effects (font (size 1.27 1.27)) (justify left))
+    )
+    (property "Footprint" "" (id 2) (at 105.7148 123.19 0)
       (effects (font (size 1.27 1.27)) hide)
     )
@@
       (effects (font (size 1.27 1.27)) (justify left))
     )
-    (property "Value" "22p" (id 1) (at 121.92 121.92 0)
-      (effects (font (size 1.27 1.27)) (justify left))
-    )
-    (property "Footprint" "Capacitor_SMD:C_0402_1005Metric" (id 2) (at 115.8748 123.19 0)
+    (property "Value" "" (id 1) (at 121.92 121.92 0)
+      (effects (font (size 1.27 1.27)) (justify left))
+    )
+    (property "Footprint" "" (id 2) (at 115.8748 123.19 0)
       (effects (font (size 1.27 1.27)) hide)
     )
@@
       (effects (font (size 1.27 1.27)) (justify left))
     )
-    (property "Value" "32kHz" (id 1) (at 110.617 105.1052 90)
-      (effects (font (size 1.27 1.27)) (justify left))
-    )
-    (property "Footprint" "Crystal:Crystal_SMD_3215-2Pin_3.2x1.5mm" (id 2) (at 111.76 102.87 0)
+    (property "Value" "" (id 1) (at 110.617 105.1052 90)
+      (effects (font (size 1.27 1.27)) (justify left))
+    )
+    (property "Footprint" "" (id 2) (at 111.76 102.87 0)
       (effects (font (size 1.27 1.27)) hide)
     )
@@
       (effects (font (size 1.27 1.27)) (justify left))
     )
-    (property "Value" "4.7k" (id 1) (at 45.9486 88.773 0)
-      (effects (font (size 1.27 1.27)) (justify left))
-    )
-    (property "Footprint" "Resistor_SMD:R_0402_1005Metric" (id 2) (at 44.45 87.63 0)
+    (property "Value" "" (id 1) (at 45.9486 88.773 0)
+      (effects (font (size 1.27 1.27)) (justify left))
+    )
+    (property "Footprint" "" (id 2) (at 44.45 87.63 0)
       (effects (font (size 1.27 1.27)) hide)
     )
@@
       (effects (font (size 1.27 1.27)) (justify left))
     )
-    (property "Value" "100n" (id 1) (at 148.59 121.92 90)
-      (effects (font (size 1.27 1.27)) (justify left))
-    )
-    (property "Footprint" "Capacitor_SMD:C_0402_1005Metric" (id 2) (at 145.7452 123.19 0)
+    (property "Value" "" (id 1) (at 148.59 121.92 90)
+      (effects (font (size 1.27 1.27)) (justify left))
+    )
+    (property "Footprint" "" (id 2) (at 145.7452 123.19 0)
       (effects (font (size 1.27 1.27)) hide)
     )
@@
       (effects (font (size 1.27 1.27)) (justify left))
     )
-    (property "Value" "100n" (id 1) (at 31.75 121.92 90)
-      (effects (font (size 1.27 1.27)) (justify left))
-    )
-    (property "Footprint" "Capacitor_SMD:C_0402_1005Metric" (id 2) (at 28.9052 123.19 0)
+    (property "Value" "" (id 1) (at 31.75 121.92 90)
+      (effects (font (size 1.27 1.27)) (justify left))
+    )
+    (property "Footprint" "" (id 2) (at 28.9052 123.19 0)
       (effects (font (size 1.27 1.27)) hide)
     )
@@
     (in_bom yes) (on_board yes)
     (property "Reference" "TP15" (id 0) (at 37.5412 87.757 90))
-    (property "Value" "Testpoint" (id 1) (at 37.5412 90.0684 90))
-    (property "Footprint" "TestPoint:TestPoint_Pad_1.0x1.0mm" (id 2) (at 39.37 87.63 0)
+    (property "Value" "" (id 1) (at 37.5412 90.0684 90))
+    (property "Footprint" "" (id 2) (at 39.37 87.63 0)
       (effects (font (size 1.27 1.27)) hide)
     )
@@
       (effects (font (size 1.143 1.143)))
     )
-    (property "Value" "I2C" (id 1) (at 255.27 80.01 90)
+    (property "Value" "" (id 1) (at 255.27 80.01 90)
       (effects (font (size 1.143 1.143)))
     )
-    (property "Footprint" "custom:1X04_1MM_RA_GND" (id 2) (at 245.11 88.9 0)
+    (property "Footprint" "" (id 2) (at 245.11 88.9 0)
       (effects (font (size 0.508 0.508)) hide)
     )
@@
     (in_bom yes) (on_board yes)
     (property "Reference" "X1" (id 0) (at 234.569 114.3 90))
-    (property "Value" "Simple_Addon_v2" (id 1) (at 236.8804 114.3 90))
-    (property "Footprint" "Simple_Addon_v2:Simple_Addon_v2-BADGE-2x3-nosilk" (id 2) (at 246.38 109.22 0)
+    (property "Value" "" (id 1) (at 236.8804 114.3 90))
+    (property "Footprint" "" (id 2) (at 246.38 109.22 0)
       (effects (font (size 1.27 1.27)) hide)
     )
@@
     (in_bom yes) (on_board yes)
     (property "Reference" "TP27" (id 0) (at 37.5412 95.377 90))
-    (property "Value" "Testpoint" (id 1) (at 37.5412 97.6884 90))
-    (property "Footprint" "TestPoint:TestPoint_Pad_1.0x1.0mm" (id 2) (at 39.37 95.25 0)
-      (effects (font (size 1.27 1.27)) hide)
-    )
+    (property "Value" "" (id 1) (at 37.5412 97.6884 90))
+    (property "Footprint" "" (id 2) (at 39.37 95.25 0)
+      (effects (font (size 1.27 1.27)) hide)
+    )

Commit message: Add gerbers, add schematic, finalize design
Parts:
- C26, C27, C30: value (none) -> 100n; footprint (none) -> Capacitor_SMD:C_0402_1005Metric
- C28, C29: value (none) -> 22p; footprint (none) -> Capacitor_SMD:C_0402_1005Metric
- J3: value (none) -> I2C; footprint (none) -> custom:1X04_1MM_RA_GND
- R47, R48, R49: value (none) -> 4.7k; footprint (none) -> Resistor_SMD:R_0402_1005Metric
- TP15, TP27: value (none) -> Testpoint; footprint (none) -> TestPoint:TestPoint_Pad_1.0x1.0mm
- U8: value (none) -> BNO055; footprint (none) -> digikey-footprints:LGA-28_5.2x3.8mm_BNO0055
- U9: value (none) -> BME680; footprint (none) -> Package_LGA:Bosch_LGA-8_3x3mm_P0.8mm_ClockwisePinNumbering
- X1: value (none) -> Simple_Addon_v2; footprint (none) -> Simple_Addon_v2:Simple_Addon_v2-BADGE-2x3-nosilk
- Y3: value (none) -> 32kHz; footprint (none) -> Crystal:Crystal_SMD_3215-2Pin_3.2x1.5mm
Changed lines of the file:
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@@
     (title "MCH2022 badge - BOSCH")
     (date "2022-04-24")
-    (rev "Pre-production final")
+    (rev "Final")
     (company "BADGE.TEAM")
+    (comment 1 "License: CERN Open Hardware Licence Version 2 - Permissive")
+    (comment 2 "Contact: renze@badge.team")
+    (comment 3 "Website: mch2022.org / badge.team")
+    (comment 4 "Event badge for May Contain Hackers 2022")
   )
   (junction (at 52.07 92.71) (diameter 0) (color 0 0 0 0)
@@
   )
   (text "I2C periphereals\n - BOSCH BNO055\n - BOSCH BME680\n - SAO expansion header\n - Qwiic expansion header"
-    (at 15.24 54.61 0)
-    (effects (font (size 5.0038 5.0038)) (justify left bottom))
+    (at 14.732 38.862 0)
+    (effects (font (size 3 3)) (justify left bottom))
   )
   (label "BNO055_XIN32" (at 93.98 100.33 0)
@@
       (effects (font (size 1.27 1.27)) (justify right))
     )
-    (property "Value" "" (id 1) (at 157.48 96.52 0)
+    (property "Value" "BME680" (id 1) (at 157.48 96.52 0)
       (effects (font (size 1.27 1.27)) (justify right))
     )
-    (property "Footprint" "" (id 2) (at 199.39 119.38 0)
+    (property "Footprint" "Package_LGA:Bosch_LGA-8_3x3mm_P0.8mm_ClockwisePinNumbering" (id 2) (at 199.39 119.38 0)
       (effects (font (size 1.27 1.27)) hide)
     )
@@
     (in_bom yes) (on_board yes)
     (property "Reference" "U8" (id 0) (at 60.96 88.9 0))
-    (property "Value" "" (id 1) (at 86.36 88.9 0))
-    (property "Footprint" "" (id 2) (at 80.01 97.79 0)
+    (property "Value" "BNO055" (id 1) (at 86.36 88.9 0))
+    (property "Footprint" "digikey-footprints:LGA-28_5.2x3.8mm_BNO0055" (id 2) (at 80.01 97.79 0)
       (effects (font (size 1.524 1.524)) (justify left) hide)
     )
@@
       (effects (font (size 1.27 1.27)) (justify left))
     )
-    (property "Value" "" (id 1) (at 99.06 121.92 90)
-      (effects (font (size 1.27 1.27)) (justify left))
-    )
-    (property "Footprint" "" (id 2) (at 96.2152 123.19 0)
+    (property "Value" "100n" (id 1) (at 99.06 121.92 90)
+      (effects (font (size 1.27 1.27)) (justify left))
+    )
+    (property "Footprint" "Capacitor_SMD:C_0402_1005Metric" (id 2) (at 96.2152 123.19 0)
       (effects (font (size 1.27 1.27)) hide)
     )
@@
       (effects (font (size 1.27 1.27)) (justify left))
     )
-    (property "Value" "" (id 1) (at 105.6386 88.773 0)
-      (effects (font (size 1.27 1.27)) (justify left))
-    )
-    (property "Footprint" "" (id 2) (at 104.14 87.63 0)
+    (property "Value" "4.7k" (id 1) (at 105.6386 88.773 0)
+      (effects (font (size 1.27 1.27)) (justify left))
+    )
+    (property "Footprint" "Resistor_SMD:R_0402_1005Metric" (id 2) (at 104.14 87.63 0)
       (effects (font (size 1.27 1.27)) hide)
     )
@@
       (effects (font (size 1.27 1.27)) (justify left))
     )
-    (property "Value" "" (id 1) (at 53.5686 88.773 0)
-      (effects (font (size 1.27 1.27)) (justify left))
-    )
-    (property "Footprint" "" (id 2) (at 52.07 87.63 0)
+    (property "Value" "4.7k" (id 1) (at 53.5686 88.773 0)
+      (effects (font (size 1.27 1.27)) (justify left))
+    )
+    (property "Footprint" "Resistor_SMD:R_0402_1005Metric" (id 2) (at 52.07 87.63 0)
       (effects (font (size 1.27 1.27)) hide)
     )
@@
       (effects (font (size 1.27 1.27)) (justify left))
     )
-    (property "Value" "" (id 1) (at 111.76 121.92 0)
-      (effects (font (size 1.27 1.27)) (justify left))
-    )
-    (property "Footprint" "" (id 2) (at 105.7148 123.19 0)
+    (property "Value" "22p" (id 1) (at 111.76 121.92 0)
+      (effects (font (size 1.27 1.27)) (justify left))
+    )
+    (property "Footprint" "Capacitor_SMD:C_0402_1005Metric" (id 2) (at 105.7148 123.19 0)
       (effects (font (size 1.27 1.27)) hide)
     )
@@
       (effects (font (size 1.27 1.27)) (justify left))
     )
-    (property "Value" "" (id 1) (at 121.92 121.92 0)
-      (effects (font (size 1.27 1.27)) (justify left))
-    )
-    (property "Footprint" "" (id 2) (at 115.8748 123.19 0)
+    (property "Value" "22p" (id 1) (at 121.92 121.92 0)
+      (effects (font (size 1.27 1.27)) (justify left))
+    )
+    (property "Footprint" "Capacitor_SMD:C_0402_1005Metric" (id 2) (at 115.8748 123.19 0)
       (effects (font (size 1.27 1.27)) hide)
     )
@@
       (effects (font (size 1.27 1.27)) (justify left))
     )
-    (property "Value" "" (id 1) (at 110.617 105.1052 90)
-      (effects (font (size 1.27 1.27)) (justify left))
-    )
-    (property "Footprint" "" (id 2) (at 111.76 102.87 0)
+    (property "Value" "32kHz" (id 1) (at 110.617 105.1052 90)
+      (effects (font (size 1.27 1.27)) (justify left))
+    )
+    (property "Footprint" "Crystal:Crystal_SMD_3215-2Pin_3.2x1.5mm" (id 2) (at 111.76 102.87 0)
       (effects (font (size 1.27 1.27)) hide)
     )
@@
       (effects (font (size 1.27 1.27)) (justify left))
     )
-    (property "Value" "" (id 1) (at 45.9486 88.773 0)
-      (effects (font (size 1.27 1.27)) (justify left))
-    )
-    (property "Footprint" "" (id 2) (at 44.45 87.63 0)
+    (property "Value" "4.7k" (id 1) (at 45.9486 88.773 0)
+      (effects (font (size 1.27 1.27)) (justify left))
+    )
+    (property "Footprint" "Resistor_SMD:R_0402_1005Metric" (id 2) (at 44.45 87.63 0)
       (effects (font (size 1.27 1.27)) hide)
     )
@@
       (effects (font (size 1.27 1.27)) (justify left))
     )
-    (property "Value" "" (id 1) (at 148.59 121.92 90)
-      (effects (font (size 1.27 1.27)) (justify left))
-    )
-    (property "Footprint" "" (id 2) (at 145.7452 123.19 0)
+    (property "Value" "100n" (id 1) (at 148.59 121.92 90)
+      (effects (font (size 1.27 1.27)) (justify left))
+    )
+    (property "Footprint" "Capacitor_SMD:C_0402_1005Metric" (id 2) (at 145.7452 123.19 0)
       (effects (font (size 1.27 1.27)) hide)
     )
@@
       (effects (font (size 1.27 1.27)) (justify left))
     )
-    (property "Value" "" (id 1) (at 31.75 121.92 90)
-      (effects (font (size 1.27 1.27)) (justify left))
-    )
-    (property "Footprint" "" (id 2) (at 28.9052 123.19 0)
+    (property "Value" "100n" (id 1) (at 31.75 121.92 90)
+      (effects (font (size 1.27 1.27)) (justify left))
+    )
+    (property "Footprint" "Capacitor_SMD:C_0402_1005Metric" (id 2) (at 28.9052 123.19 0)
       (effects (font (size 1.27 1.27)) hide)
     )
@@
     (in_bom yes) (on_board yes)
     (property "Reference" "TP15" (id 0) (at 37.5412 87.757 90))
-    (property "Value" "" (id 1) (at 37.5412 90.0684 90))
-    (property "Footprint" "" (id 2) (at 39.37 87.63 0)
+    (property "Value" "Testpoint" (id 1) (at 37.5412 90.0684 90))
+    (property "Footprint" "TestPoint:TestPoint_Pad_1.0x1.0mm" (id 2) (at 39.37 87.63 0)
       (effects (font (size 1.27 1.27)) hide)
     )
@@
       (effects (font (size 1.143 1.143)))
     )
-    (property "Value" "" (id 1) (at 255.27 80.01 90)
+    (property "Value" "I2C" (id 1) (at 255.27 80.01 90)
       (effects (font (size 1.143 1.143)))
     )
-    (property "Footprint" "" (id 2) (at 245.11 88.9 0)
+    (property "Footprint" "custom:1X04_1MM_RA_GND" (id 2) (at 245.11 88.9 0)
       (effects (font (size 0.508 0.508)) hide)
     )
@@
     (in_bom yes) (on_board yes)
     (property "Reference" "X1" (id 0) (at 234.569 114.3 90))
-    (property "Value" "" (id 1) (at 236.8804 114.3 90))
-    (property "Footprint" "" (id 2) (at 246.38 109.22 0)
+    (property "Value" "Simple_Addon_v2" (id 1) (at 236.8804 114.3 90))
+    (property "Footprint" "Simple_Addon_v2:Simple_Addon_v2-BADGE-2x3-nosilk" (id 2) (at 246.38 109.22 0)
       (effects (font (size 1.27 1.27)) hide)
     )
@@
     (in_bom yes) (on_board yes)
     (property "Reference" "TP27" (id 0) (at 37.5412 95.377 90))
-    (property "Value" "" (id 1) (at 37.5412 97.6884 90))
-    (property "Footprint" "" (id 2) (at 39.37 95.25 0)
-      (effects (font (size 1.27 1.27)) hide)
-    )
+    (property "Value" "Testpoint" (id 1) (at 37.5412 97.6884 90))
+    (property "Footprint" "TestPoint:TestPoint_Pad_1.0x1.0mm" (id 2) (at 39.37 95.25 0)
+      (effects (font (size 1.27 1.27)) hide)
+    )
