File: lcd.kicad_sch (KiCad schematic)
At the start: 17 parts, among them J7 LCD, Q1 Q_NMOS_GSD, Q2 Q_NMOS_GSD, U2 74LVC1G125

Commit message: Bill of materials 1/2
Parts:
- J7: value LCD -> (none); footprint Connector_FFC-FPC:Hirose_FH12-40S-0.5SH_1x40-1MP_P0.50mm_Horizontal -> (none); Category (none) -> Connectors; Manufacturer (none) -> XUNPU; Sponsored N -> (none)
- Q1, Q2: value Q_NMOS_GSD -> (none); footprint Package_TO_SOT_SMD:SOT-23 -> (none); Category (none) -> Transistors; Sponsored N -> (none)
- R12, R13, R14, R15: value 47 -> (none); footprint Resistor_SMD:R_0402_1005Metric -> (none); Category (none) -> Resistors; LCSC C25168 -> (none); MPN 0402WGJ0470TCE -> (none); Sponsored N -> (none)
- R16, R17, R18, R19, R20, R21: value 100k -> (none); footprint Resistor_SMD:R_0402_1005Metric -> (none); Category (none) -> Resistors; LCSC C258090 -> (none); MPN RC-02W1003FT -> (none); Sponsored N -> (none)
- RN1: value 47 -> (none); footprint Resistor_SMD:R_Array_Convex_4x0603 -> (none); Category (none) -> Resistor arrays; Sponsored N -> (none)
- RN2, RN3: value 100k -> (none); footprint Resistor_SMD:R_Array_Convex_4x0603 -> (none); Category (none) -> Resistor arrays; Sponsored N -> (none)
- U2: value 74LVC1G125 -> (none); footprint Package_TO_SOT_SMD:SOT-353_SC-70-5 -> (none); Buy early (none) -> Y; Category (none) -> ICs

Commit message: Add more info to BOM
Parts:
- J7, R12, R13, R14, R15, R16, R17, R18, R19, R20, R21: Buy early (none) -> Y; Sponsored (none) -> N
- Q1, Q2: Buy early (none) -> Y; Manufacturer (none) -> Allpower; Sponsored (none) -> N
- RN1, RN2, RN3: Buy early (none) -> Y; Manufacturer (none) -> Uni-royal; Sponsored (none) -> N

Commit message: Add passives to BOM
Parts:
- R12, R13, R14, R15: LCSC (none) -> C25118; MPN (none) -> 0402WGF470JTCE; Manufacturer (none) -> Uni-royal
- R16, R17, R18, R19, R20, R21: LCSC (none) -> C25741; MPN (none) -> 0402WGF1003TCE; Manufacturer (none) -> Uni-royal

Commit message: Artwork stuff
Parts:
- J7: value (none) -> LCD; footprint (none) -> Connector_FFC-FPC:Hirose_FH12-40S-0.5SH_1x40-1MP_P0.50mm_Horizontal
- Q1, Q2: value (none) -> AP2302B; footprint (none) -> Package_TO_SOT_SMD:SOT-23
- R12, R13, R14, R15: value (none) -> 47; footprint (none) -> Resistor_SMD:R_0402_1005Metric
- R16, R17, R18, R19, R20, R21: value (none) -> 100k; footprint (none) -> Resistor_SMD:R_0402_1005Metric
- RN1: value (none) -> 47; footprint (none) -> Resistor_SMD:R_Array_Convex_4x0603
- RN2, RN3: value (none) -> 100k; footprint (none) -> Resistor_SMD:R_Array_Convex_4x0603
- U2: value (none) -> 74LVC1G125; footprint (none) -> Package_TO_SOT_SMD:SOT-353_SC-70-5
Changed lines of the file:
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@@
     (in_bom yes) (on_board yes)
     (property "Reference" "R19" (id 0) (at 110.49 44.45 90))
-    (property "Value" "" (id 1) (at 111.76 39.37 90))
-    (property "Footprint" "" (id 2) (at 109.982 39.37 90)
+    (property "Value" "100k" (id 1) (at 111.76 39.37 90))
+    (property "Footprint" "Resistor_SMD:R_0402_1005Metric" (id 2) (at 109.982 39.37 90)
       (effects (font (size 1.27 1.27)) hide)
     )
@@
     (in_bom yes) (on_board yes)
     (property "Reference" "R18" (id 0) (at 107.95 44.45 90))
-    (property "Value" "" (id 1) (at 109.22 39.37 90))
-    (property "Footprint" "" (id 2) (at 107.442 39.37 90)
+    (property "Value" "100k" (id 1) (at 109.22 39.37 90))
+    (property "Footprint" "Resistor_SMD:R_0402_1005Metric" (id 2) (at 107.442 39.37 90)
       (effects (font (size 1.27 1.27)) hide)
     )
@@
     (in_bom yes) (on_board yes)
     (property "Reference" "R17" (id 0) (at 105.41 44.45 90))
-    (property "Value" "" (id 1) (at 106.68 39.37 90))
-    (property "Footprint" "" (id 2) (at 104.902 39.37 90)
+    (property "Value" "100k" (id 1) (at 106.68 39.37 90))
+    (property "Footprint" "Resistor_SMD:R_0402_1005Metric" (id 2) (at 104.902 39.37 90)
       (effects (font (size 1.27 1.27)) hide)
     )
@@
     (in_bom yes) (on_board yes)
     (property "Reference" "R16" (id 0) (at 102.87 44.45 90))
-    (property "Value" "" (id 1) (at 104.14 39.37 90))
-    (property "Footprint" "" (id 2) (at 102.362 39.37 90)
+    (property "Value" "100k" (id 1) (at 104.14 39.37 90))
+    (property "Footprint" "Resistor_SMD:R_0402_1005Metric" (id 2) (at 102.362 39.37 90)
       (effects (font (size 1.27 1.27)) hide)
     )
@@
     (in_bom yes) (on_board yes)
     (property "Reference" "R12" (id 0) (at 88.9 58.42 90))
-    (property "Value" "" (id 1) (at 93.98 59.69 90))
-    (property "Footprint" "" (id 2) (at 93.98 57.912 90)
+    (property "Value" "47" (id 1) (at 93.98 59.69 90))
+    (property "Footprint" "Resistor_SMD:R_0402_1005Metric" (id 2) (at 93.98 57.912 90)
       (effects (font (size 1.27 1.27)) hide)
     )
@@
     (in_bom yes) (on_board yes)
     (property "Reference" "R13" (id 0) (at 88.9 60.96 90))
-    (property "Value" "" (id 1) (at 93.98 62.23 90))
-    (property "Footprint" "" (id 2) (at 93.98 60.452 90)
+    (property "Value" "47" (id 1) (at 93.98 62.23 90))
+    (property "Footprint" "Resistor_SMD:R_0402_1005Metric" (id 2) (at 93.98 60.452 90)
       (effects (font (size 1.27 1.27)) hide)
     )
@@
     (in_bom yes) (on_board yes)
     (property "Reference" "R14" (id 0) (at 88.9 63.5 90))
-    (property "Value" "" (id 1) (at 93.98 64.77 90))
-    (property "Footprint" "" (id 2) (at 93.98 62.992 90)
+    (property "Value" "47" (id 1) (at 93.98 64.77 90))
+    (property "Footprint" "Resistor_SMD:R_0402_1005Metric" (id 2) (at 93.98 62.992 90)
       (effects (font (size 1.27 1.27)) hide)
     )
@@
     (in_bom yes) (on_board yes)
     (property "Reference" "R15" (id 0) (at 96.52 139.7 90))
-    (property "Value" "" (id 1) (at 96.52 142.24 90))
-    (property "Footprint" "" (id 2) (at 96.52 140.462 90)
+    (property "Value" "47" (id 1) (at 96.52 142.24 90))
+    (property "Footprint" "Resistor_SMD:R_0402_1005Metric" (id 2) (at 96.52 140.462 90)
       (effects (font (size 1.27 1.27)) hide)
     )
@@
     (in_bom yes) (on_board yes)
     (property "Reference" "R21" (id 0) (at 123.19 151.13 90))
-    (property "Value" "" (id 1) (at 124.46 146.05 90))
-    (property "Footprint" "" (id 2) (at 126.238 146.05 90)
+    (property "Value" "100k" (id 1) (at 124.46 146.05 90))
+    (property "Footprint" "Resistor_SMD:R_0402_1005Metric" (id 2) (at 126.238 146.05 90)
       (effects (font (size 1.27 1.27)) hide)
     )
@@
     (in_bom yes) (on_board yes)
     (property "Reference" "R20" (id 0) (at 120.65 151.13 90))
-    (property "Value" "" (id 1) (at 121.92 146.05 90))
-    (property "Footprint" "" (id 2) (at 123.698 146.05 90)
+    (property "Value" "100k" (id 1) (at 121.92 146.05 90))
+    (property "Footprint" "Resistor_SMD:R_0402_1005Metric" (id 2) (at 123.698 146.05 90)
       (effects (font (size 1.27 1.27)) hide)
     )
@@
     (in_bom yes) (on_board yes)
     (property "Reference" "J7" (id 0) (at 176.9872 144.145 0))
-    (property "Value" "" (id 1) (at 176.9872 141.8336 0))
-    (property "Footprint" "" (id 2) (at 179.07 87.63 0)
+    (property "Value" "LCD" (id 1) (at 176.9872 141.8336 0))
+    (property "Footprint" "Connector_FFC-FPC:Hirose_FH12-40S-0.5SH_1x40-1MP_P0.50mm_Horizontal" (id 2) (at 179.07 87.63 0)
       (effects (font (size 1.27 1.27)) hide)
     )
@@
     (in_bom yes) (on_board yes)
     (property "Reference" "U2" (id 0) (at 154.94 54.61 0))
-    (property "Value" "" (id 1) (at 154.94 57.15 0))
-    (property "Footprint" "" (id 2) (at 147.32 59.69 0)
+    (property "Value" "74LVC1G125" (id 1) (at 154.94 57.15 0))
+    (property "Footprint" "Package_TO_SOT_SMD:SOT-353_SC-70-5" (id 2) (at 147.32 59.69 0)
       (effects (font (size 1.27 1.27)) hide)
     )
@@
       (effects (font (size 1.27 1.27)) (justify left))
     )
-    (property "Value" "" (id 1) (at 164.7952 147.193 0)
+    (property "Value" "100k" (id 1) (at 164.7952 147.193 0)
       (effects (font (size 1.27 1.27)) (justify left))
     )
-    (property "Footprint" "" (id 2) (at 167.005 146.05 90)
+    (property "Footprint" "Resistor_SMD:R_Array_Convex_4x0603" (id 2) (at 167.005 146.05 90)
       (effects (font (size 1.27 1.27)) hide)
     )
@@
       (effects (font (size 1.27 1.27)) (justify left))
     )
-    (property "Value" "" (id 1) (at 141.9352 147.193 0)
+    (property "Value" "100k" (id 1) (at 141.9352 147.193 0)
       (effects (font (size 1.27 1.27)) (justify left))
     )
-    (property "Footprint" "" (id 2) (at 144.145 146.05 90)
+    (property "Footprint" "Resistor_SMD:R_Array_Convex_4x0603" (id 2) (at 144.145 146.05 90)
       (effects (font (size 1.27 1.27)) hide)
     )
@@
     (in_bom yes) (on_board yes)
     (property "Reference" "Q1" (id 0) (at 83.82 128.27 90))
-    (property "Value" "" (id 1) (at 81.28 132.08 90))
-    (property "Footprint" "" (id 2) (at 82.55 120.65 0)
+    (property "Value" "AP2302B" (id 1) (at 81.28 132.08 90))
+    (property "Footprint" "Package_TO_SOT_SMD:SOT-23" (id 2) (at 82.55 120.65 0)
       (effects (font (size 1.27 1.27)) hide)
     )
@@
       (effects (font (size 1.27 1.27)) (justify left))
     )
-    (property "Value" "" (id 1) (at 95.123 133.0452 0)
+    (property "Value" "47" (id 1) (at 95.123 133.0452 0)
       (effects (font (size 1.27 1.27)) (justify left))
     )
-    (property "Footprint" "" (id 2) (at 93.98 135.255 90)
+    (property "Footprint" "Resistor_SMD:R_Array_Convex_4x0603" (id 2) (at 93.98 135.255 90)
       (effects (font (size 1.27 1.27)) hide)
     )
@@
     (in_bom yes) (on_board yes)
     (property "Reference" "Q2" (id 0) (at 110.49 147.32 0))
-    (property "Value" "" (id 1) (at 105.41 149.86 0))
-    (property "Footprint" "" (id 2) (at 114.3 139.7 0)
-      (effects (font (size 1.27 1.27)) hide)
-    )
+    (property "Value" "AP2302B" (id 1) (at 105.41 149.86 0))
+    (property "Footprint" "Package_TO_SOT_SMD:SOT-23" (id 2) (at 114.3 139.7 0)
+      (effects (font (size 1.27 1.27)) hide)
+    )

Commit message: Last minute fixes
Changed lines of the file:
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@@
-    (effects (font (size 1.27 1.27)) (justify left bottom))
-  )
-  (label "LCD_RS_SCK_SWITCH" (at 127 54.61 0)
     (effects (font (size 1.27 1.27)) (justify left bottom))
   )

Commit message: Final version of prototype 4
Parts:
- J7: value LCD -> (none); footprint Connector_FFC-FPC:Hirose_FH12-40S-0.5SH_1x40-1MP_P0.50mm_Horizontal -> (none); symbol mch2021-rescue:Conn_01x40-Connector_Generic -> Connector_Generic_MountingPin:Conn_01x40_MountingPin
Connections:
- net GND: now also J7.MP (MountPin)
Changed lines of the file:
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@@
+    (stroke (width 0) (type default) (color 0 0 0 0))
+  )
+  (wire (pts (xy 179.07 143.51) (xy 179.07 153.67))
     (stroke (width 0) (type default) (color 0 0 0 0))
   )
@@
     (pin "2")
   )
-  (symbol (lib_id "mch2021-rescue:Conn_01x40-Connector_Generic") (at 179.07 87.63 0) (unit 1)
-    (in_bom yes) (on_board yes)
-    (property "Reference" "J7" (id 0) (at 176.9872 144.145 0))
-    (property "Value" "LCD" (id 1) (at 176.9872 141.8336 0))
-    (property "Footprint" "Connector_FFC-FPC:Hirose_FH12-40S-0.5SH_1x40-1MP_P0.50mm_Horizontal" (id 2) (at 179.07 87.63 0)
+  (symbol (lib_id "Connector_Generic_MountingPin:Conn_01x40_MountingPin") (at 179.07 87.63 0) (unit 1)
+    (in_bom yes) (on_board yes)
+    (property "Reference" "J7" (id 0) (at 175.006 143.002 0))
+    (property "Value" "" (id 1) (at 175.006 140.97 0))
+    (property "Footprint" "" (id 2) (at 179.07 87.63 0)
       (effects (font (size 1.27 1.27)) hide)
     )
@@
     (pin "8")
     (pin "9")
+    (pin "MP")
   )
   (symbol (lib_id "mch2021-rescue:GND-power") (at 171.45 153.67 0) (unit 1)
@@
       (effects (font (size 1.27 1.27)) hide)
     )
+    (pin "1")
+  )
+  (symbol (lib_id "mch2021-rescue:GND-power") (at 179.07 153.67 0) (unit 1)
+    (in_bom yes) (on_board yes)
+    (property "Reference" "#PWR0223" (id 0) (at 179.07 160.02 0)
+      (effects (font (size 1.27 1.27)) hide)
+    )
+    (property "Value" "GND" (id 1) (at 179.197 158.0642 0))
+    (property "Footprint" "" (id 2) (at 179.07 153.67 0)
+      (effects (font (size 1.27 1.27)) hide)
+    )
+    (property "Datasheet" "" (id 3) (at 179.07 153.67 0)
+      (effects (font (size 1.27 1.27)) hide)
+    )
