File: lcd.kicad_sch (KiCad schematic)
At the start: 17 parts, among them Q1 AP2302B, Q2 AP2302B, U2 74LVC1G125

Commit message: Small last minute tweaks
Parts:
- J7: value (none) -> LCD; footprint (none) -> Connector_FFC-FPC:Hirose_FH12-40S-0.5SH_1x40-1MP_P0.50mm_Horizontal
Changed lines of the file:
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@@
     (in_bom yes) (on_board yes)
     (property "Reference" "J7" (id 0) (at 175.006 143.002 0))
-    (property "Value" "" (id 1) (at 175.006 140.97 0))
-    (property "Footprint" "" (id 2) (at 179.07 87.63 0)
+    (property "Value" "LCD" (id 1) (at 175.006 140.97 0))
+    (property "Footprint" "Connector_FFC-FPC:Hirose_FH12-40S-0.5SH_1x40-1MP_P0.50mm_Horizontal" (id 2) (at 179.07 87.63 0)
       (effects (font (size 1.27 1.27)) hide)
     )

Commit message: Pre-production final design
Parts:
- J7: value LCD -> (none); footprint Connector_FFC-FPC:Hirose_FH12-40S-0.5SH_1x40-1MP_P0.50mm_Horizontal -> (none)
- Q1, Q2: value AP2302B -> (none); footprint Package_TO_SOT_SMD:SOT-23 -> (none)
- R12, R13, R14, R15: value 47 -> (none); footprint Resistor_SMD:R_0402_1005Metric -> (none)
- R16, R17, R18, R19, R20, R21: value 100k -> (none); footprint Resistor_SMD:R_0402_1005Metric -> (none); MANUFACTURER FH -> UNI-ROYAL
- RN1: value 47 -> (none); footprint Resistor_SMD:R_Array_Convex_4x0603 -> (none)
- RN2, RN3: value 100k -> (none); footprint Resistor_SMD:R_Array_Convex_4x0603 -> (none)
- U2: value 74LVC1G125 -> (none); footprint Package_TO_SOT_SMD:SOT-353_SC-70-5 -> (none)
Changed lines of the file:
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@@
   (title_block
     (title "MCH2022 badge - LCD")
-    (date "2022-03-11")
-    (rev "4")
+    (date "2022-04-24")
+    (rev "Pre-production final")
     (company "BADGE.TEAM")
   )
@@
     (in_bom yes) (on_board yes)
     (property "Reference" "R19" (id 0) (at 110.49 44.45 90))
-    (property "Value" "100k" (id 1) (at 111.76 39.37 90))
-    (property "Footprint" "Resistor_SMD:R_0402_1005Metric" (id 2) (at 109.982 39.37 90)
+    (property "Value" "" (id 1) (at 111.76 39.37 90))
+    (property "Footprint" "" (id 2) (at 109.982 39.37 90)
       (effects (font (size 1.27 1.27)) hide)
     )
@@
       (effects (font (size 1.27 1.27)) hide)
     )
-    (property "MANUFACTURER" "FH" (id 8) (at 111.76 39.37 0)
+    (property "MANUFACTURER" "UNI-ROYAL" (id 8) (at 111.76 39.37 0)
       (effects (font (size 1.27 1.27)) hide)
     )
@@
     (in_bom yes) (on_board yes)
     (property "Reference" "R18" (id 0) (at 107.95 44.45 90))
-    (property "Value" "100k" (id 1) (at 109.22 39.37 90))
-    (property "Footprint" "Resistor_SMD:R_0402_1005Metric" (id 2) (at 107.442 39.37 90)
+    (property "Value" "" (id 1) (at 109.22 39.37 90))
+    (property "Footprint" "" (id 2) (at 107.442 39.37 90)
       (effects (font (size 1.27 1.27)) hide)
     )
@@
       (effects (font (size 1.27 1.27)) hide)
     )
-    (property "MANUFACTURER" "FH" (id 8) (at 109.22 39.37 0)
+    (property "MANUFACTURER" "UNI-ROYAL" (id 8) (at 109.22 39.37 0)
       (effects (font (size 1.27 1.27)) hide)
     )
@@
     (in_bom yes) (on_board yes)
     (property "Reference" "R17" (id 0) (at 105.41 44.45 90))
-    (property "Value" "100k" (id 1) (at 106.68 39.37 90))
-    (property "Footprint" "Resistor_SMD:R_0402_1005Metric" (id 2) (at 104.902 39.37 90)
+    (property "Value" "" (id 1) (at 106.68 39.37 90))
+    (property "Footprint" "" (id 2) (at 104.902 39.37 90)
       (effects (font (size 1.27 1.27)) hide)
     )
@@
       (effects (font (size 1.27 1.27)) hide)
     )
-    (property "MANUFACTURER" "FH" (id 8) (at 106.68 39.37 0)
+    (property "MANUFACTURER" "UNI-ROYAL" (id 8) (at 106.68 39.37 0)
       (effects (font (size 1.27 1.27)) hide)
     )
@@
     (in_bom yes) (on_board yes)
     (property "Reference" "R16" (id 0) (at 102.87 44.45 90))
-    (property "Value" "100k" (id 1) (at 104.14 39.37 90))
-    (property "Footprint" "Resistor_SMD:R_0402_1005Metric" (id 2) (at 102.362 39.37 90)
+    (property "Value" "" (id 1) (at 104.14 39.37 90))
+    (property "Footprint" "" (id 2) (at 102.362 39.37 90)
       (effects (font (size 1.27 1.27)) hide)
     )
@@
       (effects (font (size 1.27 1.27)) hide)
     )
-    (property "MANUFACTURER" "FH" (id 8) (at 104.14 39.37 0)
+    (property "MANUFACTURER" "UNI-ROYAL" (id 8) (at 104.14 39.37 0)
       (effects (font (size 1.27 1.27)) hide)
     )
@@
     (in_bom yes) (on_board yes)
     (property "Reference" "R12" (id 0) (at 88.9 58.42 90))
-    (property "Value" "47" (id 1) (at 93.98 59.69 90))
-    (property "Footprint" "Resistor_SMD:R_0402_1005Metric" (id 2) (at 93.98 57.912 90)
+    (property "Value" "" (id 1) (at 93.98 59.69 90))
+    (property "Footprint" "" (id 2) (at 93.98 57.912 90)
       (effects (font (size 1.27 1.27)) hide)
     )
@@
     (in_bom yes) (on_board yes)
     (property "Reference" "R13" (id 0) (at 88.9 60.96 90))
-    (property "Value" "47" (id 1) (at 93.98 62.23 90))
-    (property "Footprint" "Resistor_SMD:R_0402_1005Metric" (id 2) (at 93.98 60.452 90)
+    (property "Value" "" (id 1) (at 93.98 62.23 90))
+    (property "Footprint" "" (id 2) (at 93.98 60.452 90)
       (effects (font (size 1.27 1.27)) hide)
     )
@@
     (in_bom yes) (on_board yes)
     (property "Reference" "R14" (id 0) (at 88.9 63.5 90))
-    (property "Value" "47" (id 1) (at 93.98 64.77 90))
-    (property "Footprint" "Resistor_SMD:R_0402_1005Metric" (id 2) (at 93.98 62.992 90)
+    (property "Value" "" (id 1) (at 93.98 64.77 90))
+    (property "Footprint" "" (id 2) (at 93.98 62.992 90)
       (effects (font (size 1.27 1.27)) hide)
     )
@@
     (in_bom yes) (on_board yes)
     (property "Reference" "R15" (id 0) (at 96.52 139.7 90))
-    (property "Value" "47" (id 1) (at 96.52 142.24 90))
-    (property "Footprint" "Resistor_SMD:R_0402_1005Metric" (id 2) (at 96.52 140.462 90)
+    (property "Value" "" (id 1) (at 96.52 142.24 90))
+    (property "Footprint" "" (id 2) (at 96.52 140.462 90)
       (effects (font (size 1.27 1.27)) hide)
     )
@@
     (in_bom yes) (on_board yes)
     (property "Reference" "R21" (id 0) (at 123.19 151.13 90))
-    (property "Value" "100k" (id 1) (at 124.46 146.05 90))
-    (property "Footprint" "Resistor_SMD:R_0402_1005Metric" (id 2) (at 126.238 146.05 90)
+    (property "Value" "" (id 1) (at 124.46 146.05 90))
+    (property "Footprint" "" (id 2) (at 126.238 146.05 90)
       (effects (font (size 1.27 1.27)) hide)
     )
@@
       (effects (font (size 1.27 1.27)) hide)
     )
-    (property "MANUFACTURER" "FH" (id 8) (at 124.46 146.05 0)
+    (property "MANUFACTURER" "UNI-ROYAL" (id 8) (at 124.46 146.05 0)
       (effects (font (size 1.27 1.27)) hide)
     )
@@
     (in_bom yes) (on_board yes)
     (property "Reference" "R20" (id 0) (at 120.65 151.13 90))
-    (property "Value" "100k" (id 1) (at 121.92 146.05 90))
-    (property "Footprint" "Resistor_SMD:R_0402_1005Metric" (id 2) (at 123.698 146.05 90)
+    (property "Value" "" (id 1) (at 121.92 146.05 90))
+    (property "Footprint" "" (id 2) (at 123.698 146.05 90)
       (effects (font (size 1.27 1.27)) hide)
     )
@@
       (effects (font (size 1.27 1.27)) hide)
     )
-    (property "MANUFACTURER" "FH" (id 8) (at 121.92 146.05 0)
+    (property "MANUFACTURER" "UNI-ROYAL" (id 8) (at 121.92 146.05 0)
       (effects (font (size 1.27 1.27)) hide)
     )
@@
     (in_bom yes) (on_board yes)
     (property "Reference" "J7" (id 0) (at 175.006 143.002 0))
-    (property "Value" "LCD" (id 1) (at 175.006 140.97 0))
-    (property "Footprint" "Connector_FFC-FPC:Hirose_FH12-40S-0.5SH_1x40-1MP_P0.50mm_Horizontal" (id 2) (at 179.07 87.63 0)
+    (property "Value" "" (id 1) (at 175.006 140.97 0))
+    (property "Footprint" "" (id 2) (at 179.07 87.63 0)
       (effects (font (size 1.27 1.27)) hide)
     )
@@
     (in_bom yes) (on_board yes)
     (property "Reference" "U2" (id 0) (at 154.94 54.61 0))
-    (property "Value" "74LVC1G125" (id 1) (at 154.94 57.15 0))
-    (property "Footprint" "Package_TO_SOT_SMD:SOT-353_SC-70-5" (id 2) (at 147.32 59.69 0)
+    (property "Value" "" (id 1) (at 154.94 57.15 0))
+    (property "Footprint" "" (id 2) (at 147.32 59.69 0)
       (effects (font (size 1.27 1.27)) hide)
     )
@@
       (effects (font (size 1.27 1.27)) (justify left))
     )
-    (property "Value" "100k" (id 1) (at 164.7952 147.193 0)
+    (property "Value" "" (id 1) (at 164.7952 147.193 0)
       (effects (font (size 1.27 1.27)) (justify left))
     )
-    (property "Footprint" "Resistor_SMD:R_Array_Convex_4x0603" (id 2) (at 167.005 146.05 90)
+    (property "Footprint" "" (id 2) (at 167.005 146.05 90)
       (effects (font (size 1.27 1.27)) hide)
     )
@@
       (effects (font (size 1.27 1.27)) (justify left))
     )
-    (property "Value" "100k" (id 1) (at 141.9352 147.193 0)
+    (property "Value" "" (id 1) (at 141.9352 147.193 0)
       (effects (font (size 1.27 1.27)) (justify left))
     )
-    (property "Footprint" "Resistor_SMD:R_Array_Convex_4x0603" (id 2) (at 144.145 146.05 90)
+    (property "Footprint" "" (id 2) (at 144.145 146.05 90)
       (effects (font (size 1.27 1.27)) hide)
     )
@@
     (in_bom yes) (on_board yes)
     (property "Reference" "Q1" (id 0) (at 83.82 128.27 90))
-    (property "Value" "AP2302B" (id 1) (at 81.28 132.08 90))
-    (property "Footprint" "Package_TO_SOT_SMD:SOT-23" (id 2) (at 82.55 120.65 0)
+    (property "Value" "" (id 1) (at 81.28 132.08 90))
+    (property "Footprint" "" (id 2) (at 82.55 120.65 0)
       (effects (font (size 1.27 1.27)) hide)
     )
@@
       (effects (font (size 1.27 1.27)) (justify left))
     )
-    (property "Value" "47" (id 1) (at 95.123 133.0452 0)
+    (property "Value" "" (id 1) (at 95.123 133.0452 0)
       (effects (font (size 1.27 1.27)) (justify left))
     )
-    (property "Footprint" "Resistor_SMD:R_Array_Convex_4x0603" (id 2) (at 93.98 135.255 90)
+    (property "Footprint" "" (id 2) (at 93.98 135.255 90)
       (effects (font (size 1.27 1.27)) hide)
     )
@@
     (in_bom yes) (on_board yes)
     (property "Reference" "Q2" (id 0) (at 110.49 147.32 0))
-    (property "Value" "AP2302B" (id 1) (at 105.41 149.86 0))
-    (property "Footprint" "Package_TO_SOT_SMD:SOT-23" (id 2) (at 114.3 139.7 0)
-      (effects (font (size 1.27 1.27)) hide)
-    )
+    (property "Value" "" (id 1) (at 105.41 149.86 0))
+    (property "Footprint" "" (id 2) (at 114.3 139.7 0)
+      (effects (font (size 1.27 1.27)) hide)
+    )

Commit message: Add gerbers, add schematic, finalize design
Parts:
- J7: value (none) -> LCD; footprint (none) -> Connector_FFC-FPC:Hirose_FH12-40S-0.5SH_1x40-1MP_P0.50mm_Horizontal
- Q1, Q2: value (none) -> AP2302B; footprint (none) -> Package_TO_SOT_SMD:SOT-23
- R12, R13, R14, R15: value (none) -> 47; footprint (none) -> Resistor_SMD:R_0402_1005Metric
- R16, R17, R18, R19, R20, R21: value (none) -> 100k; footprint (none) -> Resistor_SMD:R_0402_1005Metric
- RN1: value (none) -> 47; footprint (none) -> Resistor_SMD:R_Array_Convex_4x0603
- RN2, RN3: value (none) -> 100k; footprint (none) -> Resistor_SMD:R_Array_Convex_4x0603
- U2: value (none) -> 74LVC1G125; footprint (none) -> Package_TO_SOT_SMD:SOT-353_SC-70-5
Changed lines of the file:
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@@
     (title "MCH2022 badge - LCD")
     (date "2022-04-24")
-    (rev "Pre-production final")
+    (rev "Final")
     (company "BADGE.TEAM")
+    (comment 1 "License: CERN Open Hardware Licence Version 2 - Permissive")
+    (comment 2 "Contact: renze@badge.team")
+    (comment 3 "Website: mch2022.org / badge.team")
+    (comment 4 "Event badge for May Contain Hackers 2022")
   )
   (junction (at 137.16 152.4) (diameter 0) (color 0 0 0 0)
@@
     (in_bom yes) (on_board yes)
     (property "Reference" "R19" (id 0) (at 110.49 44.45 90))
-    (property "Value" "" (id 1) (at 111.76 39.37 90))
-    (property "Footprint" "" (id 2) (at 109.982 39.37 90)
+    (property "Value" "100k" (id 1) (at 111.76 39.37 90))
+    (property "Footprint" "Resistor_SMD:R_0402_1005Metric" (id 2) (at 109.982 39.37 90)
       (effects (font (size 1.27 1.27)) hide)
     )
@@
     (in_bom yes) (on_board yes)
     (property "Reference" "R18" (id 0) (at 107.95 44.45 90))
-    (property "Value" "" (id 1) (at 109.22 39.37 90))
-    (property "Footprint" "" (id 2) (at 107.442 39.37 90)
+    (property "Value" "100k" (id 1) (at 109.22 39.37 90))
+    (property "Footprint" "Resistor_SMD:R_0402_1005Metric" (id 2) (at 107.442 39.37 90)
       (effects (font (size 1.27 1.27)) hide)
     )
@@
     (in_bom yes) (on_board yes)
     (property "Reference" "R17" (id 0) (at 105.41 44.45 90))
-    (property "Value" "" (id 1) (at 106.68 39.37 90))
-    (property "Footprint" "" (id 2) (at 104.902 39.37 90)
+    (property "Value" "100k" (id 1) (at 106.68 39.37 90))
+    (property "Footprint" "Resistor_SMD:R_0402_1005Metric" (id 2) (at 104.902 39.37 90)
       (effects (font (size 1.27 1.27)) hide)
     )
@@
     (in_bom yes) (on_board yes)
     (property "Reference" "R16" (id 0) (at 102.87 44.45 90))
-    (property "Value" "" (id 1) (at 104.14 39.37 90))
-    (property "Footprint" "" (id 2) (at 102.362 39.37 90)
+    (property "Value" "100k" (id 1) (at 104.14 39.37 90))
+    (property "Footprint" "Resistor_SMD:R_0402_1005Metric" (id 2) (at 102.362 39.37 90)
       (effects (font (size 1.27 1.27)) hide)
     )
@@
     (in_bom yes) (on_board yes)
     (property "Reference" "R12" (id 0) (at 88.9 58.42 90))
-    (property "Value" "" (id 1) (at 93.98 59.69 90))
-    (property "Footprint" "" (id 2) (at 93.98 57.912 90)
+    (property "Value" "47" (id 1) (at 93.98 59.69 90))
+    (property "Footprint" "Resistor_SMD:R_0402_1005Metric" (id 2) (at 93.98 57.912 90)
       (effects (font (size 1.27 1.27)) hide)
     )
@@
     (in_bom yes) (on_board yes)
     (property "Reference" "R13" (id 0) (at 88.9 60.96 90))
-    (property "Value" "" (id 1) (at 93.98 62.23 90))
-    (property "Footprint" "" (id 2) (at 93.98 60.452 90)
+    (property "Value" "47" (id 1) (at 93.98 62.23 90))
+    (property "Footprint" "Resistor_SMD:R_0402_1005Metric" (id 2) (at 93.98 60.452 90)
       (effects (font (size 1.27 1.27)) hide)
     )
@@
     (in_bom yes) (on_board yes)
     (property "Reference" "R14" (id 0) (at 88.9 63.5 90))
-    (property "Value" "" (id 1) (at 93.98 64.77 90))
-    (property "Footprint" "" (id 2) (at 93.98 62.992 90)
+    (property "Value" "47" (id 1) (at 93.98 64.77 90))
+    (property "Footprint" "Resistor_SMD:R_0402_1005Metric" (id 2) (at 93.98 62.992 90)
       (effects (font (size 1.27 1.27)) hide)
     )
@@
     (in_bom yes) (on_board yes)
     (property "Reference" "R15" (id 0) (at 96.52 139.7 90))
-    (property "Value" "" (id 1) (at 96.52 142.24 90))
-    (property "Footprint" "" (id 2) (at 96.52 140.462 90)
+    (property "Value" "47" (id 1) (at 96.52 142.24 90))
+    (property "Footprint" "Resistor_SMD:R_0402_1005Metric" (id 2) (at 96.52 140.462 90)
       (effects (font (size 1.27 1.27)) hide)
     )
@@
     (in_bom yes) (on_board yes)
     (property "Reference" "R21" (id 0) (at 123.19 151.13 90))
-    (property "Value" "" (id 1) (at 124.46 146.05 90))
-    (property "Footprint" "" (id 2) (at 126.238 146.05 90)
+    (property "Value" "100k" (id 1) (at 124.46 146.05 90))
+    (property "Footprint" "Resistor_SMD:R_0402_1005Metric" (id 2) (at 126.238 146.05 90)
       (effects (font (size 1.27 1.27)) hide)
     )
@@
     (in_bom yes) (on_board yes)
     (property "Reference" "R20" (id 0) (at 120.65 151.13 90))
-    (property "Value" "" (id 1) (at 121.92 146.05 90))
-    (property "Footprint" "" (id 2) (at 123.698 146.05 90)
+    (property "Value" "100k" (id 1) (at 121.92 146.05 90))
+    (property "Footprint" "Resistor_SMD:R_0402_1005Metric" (id 2) (at 123.698 146.05 90)
       (effects (font (size 1.27 1.27)) hide)
     )
@@
     (in_bom yes) (on_board yes)
     (property "Reference" "J7" (id 0) (at 175.006 143.002 0))
-    (property "Value" "" (id 1) (at 175.006 140.97 0))
-    (property "Footprint" "" (id 2) (at 179.07 87.63 0)
+    (property "Value" "LCD" (id 1) (at 175.006 140.97 0))
+    (property "Footprint" "Connector_FFC-FPC:Hirose_FH12-40S-0.5SH_1x40-1MP_P0.50mm_Horizontal" (id 2) (at 179.07 87.63 0)
       (effects (font (size 1.27 1.27)) hide)
     )
@@
     (in_bom yes) (on_board yes)
     (property "Reference" "U2" (id 0) (at 154.94 54.61 0))
-    (property "Value" "" (id 1) (at 154.94 57.15 0))
-    (property "Footprint" "" (id 2) (at 147.32 59.69 0)
+    (property "Value" "74LVC1G125" (id 1) (at 154.94 57.15 0))
+    (property "Footprint" "Package_TO_SOT_SMD:SOT-353_SC-70-5" (id 2) (at 147.32 59.69 0)
       (effects (font (size 1.27 1.27)) hide)
     )
@@
       (effects (font (size 1.27 1.27)) (justify left))
     )
-    (property "Value" "" (id 1) (at 164.7952 147.193 0)
+    (property "Value" "100k" (id 1) (at 164.7952 147.193 0)
       (effects (font (size 1.27 1.27)) (justify left))
     )
-    (property "Footprint" "" (id 2) (at 167.005 146.05 90)
+    (property "Footprint" "Resistor_SMD:R_Array_Convex_4x0603" (id 2) (at 167.005 146.05 90)
       (effects (font (size 1.27 1.27)) hide)
     )
@@
       (effects (font (size 1.27 1.27)) (justify left))
     )
-    (property "Value" "" (id 1) (at 141.9352 147.193 0)
+    (property "Value" "100k" (id 1) (at 141.9352 147.193 0)
       (effects (font (size 1.27 1.27)) (justify left))
     )
-    (property "Footprint" "" (id 2) (at 144.145 146.05 90)
+    (property "Footprint" "Resistor_SMD:R_Array_Convex_4x0603" (id 2) (at 144.145 146.05 90)
       (effects (font (size 1.27 1.27)) hide)
     )
@@
     (in_bom yes) (on_board yes)
     (property "Reference" "Q1" (id 0) (at 83.82 128.27 90))
-    (property "Value" "" (id 1) (at 81.28 132.08 90))
-    (property "Footprint" "" (id 2) (at 82.55 120.65 0)
+    (property "Value" "AP2302B" (id 1) (at 81.28 132.08 90))
+    (property "Footprint" "Package_TO_SOT_SMD:SOT-23" (id 2) (at 82.55 120.65 0)
       (effects (font (size 1.27 1.27)) hide)
     )
@@
       (effects (font (size 1.27 1.27)) (justify left))
     )
-    (property "Value" "" (id 1) (at 95.123 133.0452 0)
+    (property "Value" "47" (id 1) (at 95.123 133.0452 0)
       (effects (font (size 1.27 1.27)) (justify left))
     )
-    (property "Footprint" "" (id 2) (at 93.98 135.255 90)
+    (property "Footprint" "Resistor_SMD:R_Array_Convex_4x0603" (id 2) (at 93.98 135.255 90)
       (effects (font (size 1.27 1.27)) hide)
     )
@@
     (in_bom yes) (on_board yes)
     (property "Reference" "Q2" (id 0) (at 110.49 147.32 0))
-    (property "Value" "" (id 1) (at 105.41 149.86 0))
-    (property "Footprint" "" (id 2) (at 114.3 139.7 0)
-      (effects (font (size 1.27 1.27)) hide)
-    )
+    (property "Value" "AP2302B" (id 1) (at 105.41 149.86 0))
+    (property "Footprint" "Package_TO_SOT_SMD:SOT-23" (id 2) (at 114.3 139.7 0)
+      (effects (font (size 1.27 1.27)) hide)
+    )
