File: led.kicad_sch (KiCad schematic)
At the start: 13 parts, among them U10 74LVC1G125

Commit message: Small fixes
Parts:
- removed C33, C55, C56: 1u, Capacitor_SMD:C_0402_1005Metric, symbol mch2021-rescue:C-Device
Changed lines of the file:
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@@
-    )
-  )
-  (global_label "PWR_LED" (shape input) (at 154.94 125.73 90) (fields_autoplaced)
-    (effects (font (size 0.9906 0.9906)) (justify left))
-    (property "Intersheet References" "${INTERSHEET_REFS}" (id 0) (at 0 0 0)
-      (effects (font (size 1.27 1.27)) hide)
     )
   )
@@
     )
   )
-  (global_label "PWR_LED" (shape input) (at 139.7 125.73 90) (fields_autoplaced)
-    (effects (font (size 0.9906 0.9906)) (justify left))
-    (property "Intersheet References" "${INTERSHEET_REFS}" (id 0) (at 0 0 0)
-      (effects (font (size 1.27 1.27)) hide)
-    )
-  )
   (global_label "PWR_LED" (shape input) (at 124.46 125.73 90) (fields_autoplaced)
     (effects (font (size 0.9906 0.9906)) (justify left))
@@
   )
   (global_label "PWR_LED" (shape input) (at 154.94 95.25 90) (fields_autoplaced)
-    (effects (font (size 0.9906 0.9906)) (justify left))
-    (property "Intersheet References" "${INTERSHEET_REFS}" (id 0) (at 0 0 0)
-      (effects (font (size 1.27 1.27)) hide)
-    )
-  )
-  (global_label "PWR_LED" (shape input) (at 170.18 125.73 90) (fields_autoplaced)
     (effects (font (size 0.9906 0.9906)) (justify left))
     (property "Intersheet References" "${INTERSHEET_REFS}" (id 0) (at 0 0 0)
@@
     (pin "4")
   )
-  (symbol (lib_id "mch2021-rescue:C-Device") (at 154.94 129.54 0) (mirror y) (unit 1)
-    (in_bom yes) (on_board yes)
-    (property "Reference" "C55" (id 0) (at 152.019 128.3716 0)
-      (effects (font (size 1.27 1.27)) (justify left))
-    )
-    (property "Value" "1u" (id 1) (at 152.019 130.683 0)
-      (effects (font (size 1.27 1.27)) (justify left))
-    )
-    (property "Footprint" "Capacitor_SMD:C_0402_1005Metric" (id 2) (at 153.9748 133.35 0)
-      (effects (font (size 1.27 1.27)) hide)
-    )
-    (property "Datasheet" "" (id 3) (at 154.94 129.54 0)
-      (effects (font (size 1.27 1.27)) hide)
-    )
-    (property "Price" "" (id 4) (at 154.94 129.54 0)
-      (effects (font (size 1.27 1.27)) hide)
-    )
-    (property "Sponsored" "N" (id 5) (at 154.94 129.54 0)
-      (effects (font (size 1.27 1.27)) hide)
-    )
-    (property "LCSC" "C107372" (id 6) (at 154.94 129.54 0)
-      (effects (font (size 1.27 1.27)) hide)
-    )
-    (pin "1")
-    (pin "2")
-  )
-  (symbol (lib_id "mch2021-rescue:GND-power") (at 154.94 133.35 0) (unit 1)
-    (in_bom yes) (on_board yes)
-    (property "Reference" "#PWR0149" (id 0) (at 154.94 139.7 0)
-      (effects (font (size 1.27 1.27)) hide)
-    )
-    (property "Value" "GND" (id 1) (at 155.067 137.7442 0))
-    (property "Footprint" "" (id 2) (at 154.94 133.35 0)
-      (effects (font (size 1.27 1.27)) hide)
-    )
-    (property "Datasheet" "" (id 3) (at 154.94 133.35 0)
-      (effects (font (size 1.27 1.27)) hide)
-    )
-    (pin "1")
-  )
-  (symbol (lib_id "mch2021-rescue:C-Device") (at 170.18 129.54 0) (mirror y) (unit 1)
-    (in_bom yes) (on_board yes)
-    (property "Reference" "C56" (id 0) (at 167.259 128.3716 0)
-      (effects (font (size 1.27 1.27)) (justify left))
-    )
-    (property "Value" "1u" (id 1) (at 167.259 130.683 0)
-      (effects (font (size 1.27 1.27)) (justify left))
-    )
-    (property "Footprint" "Capacitor_SMD:C_0402_1005Metric" (id 2) (at 169.2148 133.35 0)
-      (effects (font (size 1.27 1.27)) hide)
-    )
-    (property "Datasheet" "" (id 3) (at 170.18 129.54 0)
-      (effects (font (size 1.27 1.27)) hide)
-    )
-    (property "Price" "" (id 4) (at 170.18 129.54 0)
-      (effects (font (size 1.27 1.27)) hide)
-    )
-    (property "Sponsored" "N" (id 5) (at 170.18 129.54 0)
-      (effects (font (size 1.27 1.27)) hide)
-    )
-    (property "LCSC" "C107372" (id 6) (at 170.18 129.54 0)
-      (effects (font (size 1.27 1.27)) hide)
-    )
-    (pin "1")
-    (pin "2")
-  )
-  (symbol (lib_id "mch2021-rescue:GND-power") (at 170.18 133.35 0) (unit 1)
-    (in_bom yes) (on_board yes)
-    (property "Reference" "#PWR0219" (id 0) (at 170.18 139.7 0)
-      (effects (font (size 1.27 1.27)) hide)
-    )
-    (property "Value" "GND" (id 1) (at 170.307 137.7442 0))
-    (property "Footprint" "" (id 2) (at 170.18 133.35 0)
-      (effects (font (size 1.27 1.27)) hide)
-    )
-    (property "Datasheet" "" (id 3) (at 170.18 133.35 0)
-      (effects (font (size 1.27 1.27)) hide)
-    )
-    (pin "1")
-  )
   (symbol (lib_id "mch2021-rescue:GND-power") (at 80.01 110.49 0) (mirror y) (unit 1)
     (in_bom yes) (on_board yes)
@@
       (effects (font (size 1.27 1.27)) hide)
     )
-    (pin "1")
-  )
-  (symbol (lib_id "mch2021-rescue:C-Device") (at 139.7 129.54 0) (mirror y) (unit 1)
-    (in_bom yes) (on_board yes)
-    (property "Reference" "C33" (id 0) (at 136.779 128.3716 0)
-      (effects (font (size 1.27 1.27)) (justify left))
-    )
-    (property "Value" "1u" (id 1) (at 136.779 130.683 0)
-      (effects (font (size 1.27 1.27)) (justify left))
-    )
-    (property "Footprint" "Capacitor_SMD:C_0402_1005Metric" (id 2) (at 138.7348 133.35 0)
-      (effects (font (size 1.27 1.27)) hide)
-    )
-    (property "Datasheet" "" (id 3) (at 139.7 129.54 0)
-      (effects (font (size 1.27 1.27)) hide)
-    )
-    (property "Price" "" (id 4) (at 139.7 129.54 0)
-      (effects (font (size 1.27 1.27)) hide)
-    )
-    (property "Sponsored" "N" (id 5) (at 139.7 129.54 0)
-      (effects (font (size 1.27 1.27)) hide)
-    )
-    (property "LCSC" "C107372" (id 6) (at 139.7 129.54 0)
-      (effects (font (size 1.27 1.27)) hide)
-    )
-    (pin "1")
-    (pin "2")
-  )
-  (symbol (lib_id "mch2021-rescue:GND-power") (at 139.7 133.35 0) (unit 1)
-    (in_bom yes) (on_board yes)
-    (property "Reference" "#PWR0152" (id 0) (at 139.7 139.7 0)
-      (effects (font (size 1.27 1.27)) hide)
-    )
-    (property "Value" "GND" (id 1) (at 139.827 137.7442 0))
-    (property "Footprint" "" (id 2) (at 139.7 133.35 0)
-      (effects (font (size 1.27 1.27)) hide)
-    )
-    (property "Datasheet" "" (id 3) (at 139.7 133.35 0)
-      (effects (font (size 1.27 1.27)) hide)
-    )

Commit message: Bill of materials 1/2
Parts:
- C31, C32: value 1u -> (none); footprint Capacitor_SMD:C_0402_1005Metric -> (none); Category (none) -> Capacitors; LCSC C107372 -> (none); Sponsored N -> (none)
- D3, D4, D5, D6, D7: value SK6805-EC15 -> (none); footprint custom:LED_SK6805_EC15_1.5x1.5mm -> (none); Category (none) -> LEDs; MPN (none) -> SK6805-EC15; Manufacturer (none) -> Normandled; Sponsored N -> (none)
- TP2: value LED_DATA_BUFF -> (none); footprint TestPoint:TestPoint_Pad_1.0x1.0mm -> (none); Buy early (none) -> N; Category (none) -> Testpoints; Sponsored (none) -> N
- TP3: value LED_DATA -> (none); footprint TestPoint:TestPoint_Pad_1.0x1.0mm -> (none); Buy early (none) -> N; Category (none) -> Testpoints; Sponsored (none) -> N
- U10: value 74LVC1G125 -> (none); footprint Package_TO_SOT_SMD:SOT-353_SC-70-5 -> (none); Buy early (none) -> Y; Category Integrated Circuits (ICs) -> ICs

Commit message: Add more info to BOM
Parts:
- C31, C32, D3, D4, D5, D6, D7: Buy early (none) -> Y; Sponsored (none) -> N
Changed lines of the file:
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@@
       (effects (font (size 1.27 1.27)) hide)
     )
-    (property "Sponsored" "" (id 7) (at 109.22 102.87 0)
+    (property "Sponsored" "N" (id 7) (at 109.22 102.87 0)
       (effects (font (size 1.27 1.27)) hide)
     )
@@
     )
     (property "Manufacturer" "Normandled" (id 11) (at 109.22 102.87 0)
+      (effects (font (size 1.27 1.27)) hide)
+    )
+    (property "Buy early" "Y" (id 12) (at 109.22 102.87 0)
       (effects (font (size 1.27 1.27)) hide)
     )
@@
       (effects (font (size 1.27 1.27)) hide)
     )
-    (property "Sponsored" "" (id 7) (at 124.46 102.87 0)
+    (property "Sponsored" "N" (id 7) (at 124.46 102.87 0)
       (effects (font (size 1.27 1.27)) hide)
     )
@@
     )
     (property "Manufacturer" "Normandled" (id 11) (at 124.46 102.87 0)
+      (effects (font (size 1.27 1.27)) hide)
+    )
+    (property "Buy early" "Y" (id 12) (at 124.46 102.87 0)
       (effects (font (size 1.27 1.27)) hide)
     )
@@
       (effects (font (size 1.27 1.27)) hide)
     )
-    (property "Sponsored" "" (id 7) (at 139.7 102.87 0)
+    (property "Sponsored" "N" (id 7) (at 139.7 102.87 0)
       (effects (font (size 1.27 1.27)) hide)
     )
@@
     )
     (property "Manufacturer" "Normandled" (id 11) (at 139.7 102.87 0)
+      (effects (font (size 1.27 1.27)) hide)
+    )
+    (property "Buy early" "Y" (id 12) (at 139.7 102.87 0)
       (effects (font (size 1.27 1.27)) hide)
     )
@@
       (effects (font (size 1.27 1.27)) hide)
     )
-    (property "Sponsored" "" (id 7) (at 154.94 102.87 0)
+    (property "Sponsored" "N" (id 7) (at 154.94 102.87 0)
       (effects (font (size 1.27 1.27)) hide)
     )
@@
     )
     (property "Manufacturer" "Normandled" (id 11) (at 154.94 102.87 0)
+      (effects (font (size 1.27 1.27)) hide)
+    )
+    (property "Buy early" "Y" (id 12) (at 154.94 102.87 0)
       (effects (font (size 1.27 1.27)) hide)
     )
@@
       (effects (font (size 1.27 1.27)) hide)
     )
-    (property "Sponsored" "" (id 7) (at 170.18 102.87 0)
+    (property "Sponsored" "N" (id 7) (at 170.18 102.87 0)
       (effects (font (size 1.27 1.27)) hide)
     )
@@
     )
     (property "Manufacturer" "Normandled" (id 11) (at 170.18 102.87 0)
+      (effects (font (size 1.27 1.27)) hide)
+    )
+    (property "Buy early" "Y" (id 12) (at 170.18 102.87 0)
       (effects (font (size 1.27 1.27)) hide)
     )
@@
       (effects (font (size 1.27 1.27)) hide)
     )
-    (property "Sponsored" "" (id 5) (at 109.22 129.54 0)
+    (property "Sponsored" "N" (id 5) (at 109.22 129.54 0)
       (effects (font (size 1.27 1.27)) hide)
     )
@@
     )
     (property "Description" "Generic part" (id 8) (at 109.22 129.54 0)
+      (effects (font (size 1.27 1.27)) hide)
+    )
+    (property "Buy early" "Y" (id 9) (at 109.22 129.54 0)
       (effects (font (size 1.27 1.27)) hide)
     )
@@
       (effects (font (size 1.27 1.27)) hide)
     )
-    (property "Sponsored" "" (id 5) (at 124.46 129.54 0)
+    (property "Sponsored" "N" (id 5) (at 124.46 129.54 0)
       (effects (font (size 1.27 1.27)) hide)
     )
@@
       (effects (font (size 1.27 1.27)) hide)
     )
+    (property "Buy early" "Y" (id 9) (at 124.46 129.54 0)
+      (effects (font (size 1.27 1.27)) hide)
+    )

Commit message: Add passives to BOM
Parts:
- C31, C32: LCSC (none) -> C107372; MPN (none) -> CL05A105KQ5NNNC; Manufacturer (none) -> Samsung Electro-Mechanics; Minimal voltage rating (none) -> 6; Voltage rating (none) -> 6.3
- D3, D4, D5, D6, D7: LCSC (none) -> -
Changed lines of the file:
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@@
       (effects (font (size 1.27 1.27)) (justify left top) hide)
     )
-    (property "LCSC" "" (id 4) (at 109.22 102.87 0)
+    (property "LCSC" "-" (id 4) (at 109.22 102.87 0)
       (effects (font (size 1.27 1.27)) hide)
     )
@@
       (effects (font (size 1.27 1.27)) (justify left top) hide)
     )
-    (property "LCSC" "" (id 4) (at 124.46 102.87 0)
+    (property "LCSC" "-" (id 4) (at 124.46 102.87 0)
       (effects (font (size 1.27 1.27)) hide)
     )
@@
       (effects (font (size 1.27 1.27)) (justify left top) hide)
     )
-    (property "LCSC" "" (id 4) (at 139.7 102.87 0)
+    (property "LCSC" "-" (id 4) (at 139.7 102.87 0)
       (effects (font (size 1.27 1.27)) hide)
     )
@@
       (effects (font (size 1.27 1.27)) (justify left top) hide)
     )
-    (property "LCSC" "" (id 4) (at 154.94 102.87 0)
+    (property "LCSC" "-" (id 4) (at 154.94 102.87 0)
       (effects (font (size 1.27 1.27)) hide)
     )
@@
       (effects (font (size 1.27 1.27)) (justify left top) hide)
     )
-    (property "LCSC" "" (id 4) (at 170.18 102.87 0)
+    (property "LCSC" "-" (id 4) (at 170.18 102.87 0)
       (effects (font (size 1.27 1.27)) hide)
     )
@@
       (effects (font (size 1.27 1.27)) hide)
     )
-    (property "Datasheet" "" (id 3) (at 109.22 129.54 0)
+    (property "Datasheet" "https://datasheet.lcsc.com/lcsc/1810191216_Samsung-Electro-Mechanics-CL05A105KQ5NNNC_C107372.pdf" (id 3) (at 109.22 129.54 0)
       (effects (font (size 1.27 1.27)) hide)
     )
@@
       (effects (font (size 1.27 1.27)) hide)
     )
-    (property "LCSC" "" (id 6) (at 109.22 129.54 0)
+    (property "LCSC" "C107372" (id 6) (at 109.22 129.54 0)
       (effects (font (size 1.27 1.27)) hide)
     )
@@
     )
     (property "Buy early" "Y" (id 9) (at 109.22 129.54 0)
+      (effects (font (size 1.27 1.27)) hide)
+    )
+    (property "MPN" "CL05A105KQ5NNNC" (id 10) (at 109.22 129.54 0)
+      (effects (font (size 1.27 1.27)) hide)
+    )
+    (property "Manufacturer" "Samsung Electro-Mechanics" (id 11) (at 109.22 129.54 0)
+      (effects (font (size 1.27 1.27)) hide)
+    )
+    (property "Minimal voltage rating" "6" (id 12) (at 109.22 129.54 0)
+      (effects (font (size 1.27 1.27)) hide)
+    )
+    (property "Voltage rating" "6.3" (id 13) (at 109.22 129.54 0)
       (effects (font (size 1.27 1.27)) hide)
     )
@@
       (effects (font (size 1.27 1.27)) hide)
     )
-    (property "Datasheet" "" (id 3) (at 124.46 129.54 0)
+    (property "Datasheet" "https://datasheet.lcsc.com/lcsc/1810191216_Samsung-Electro-Mechanics-CL05A105KQ5NNNC_C107372.pdf" (id 3) (at 124.46 129.54 0)
       (effects (font (size 1.27 1.27)) hide)
     )
@@
       (effects (font (size 1.27 1.27)) hide)
     )
-    (property "LCSC" "" (id 6) (at 124.46 129.54 0)
+    (property "LCSC" "C107372" (id 6) (at 124.46 129.54 0)
       (effects (font (size 1.27 1.27)) hide)
     )
@@
       (effects (font (size 1.27 1.27)) hide)
     )
+    (property "MPN" "CL05A105KQ5NNNC" (id 10) (at 124.46 129.54 0)
+      (effects (font (size 1.27 1.27)) hide)
+    )
+    (property "Manufacturer" "Samsung Electro-Mechanics" (id 11) (at 124.46 129.54 0)
+      (effects (font (size 1.27 1.27)) hide)
+    )
+    (property "Minimal voltage rating" "6" (id 12) (at 124.46 129.54 0)
+      (effects (font (size 1.27 1.27)) hide)
+    )
+    (property "Voltage rating" "6.3" (id 13) (at 124.46 129.54 0)
+      (effects (font (size 1.27 1.27)) hide)
+    )

Commit message: Artwork stuff
Parts:
- C31, C32: value (none) -> 1u; footprint (none) -> Capacitor_SMD:C_0402_1005Metric
- D3, D4, D5, D6, D7: value (none) -> SK6805-EC15; footprint (none) -> custom:LED_SK6805_EC15_1.5x1.5mm
- TP2, TP3: value (none) -> Testpoint; footprint (none) -> TestPoint:TestPoint_Pad_1.0x1.0mm
- U10: value (none) -> 74LVC1G125; footprint (none) -> Package_TO_SOT_SMD:SOT-353_SC-70-5
Changed lines of the file:
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@@
       (effects (font (size 1.27 1.27)) (justify left))
     )
-    (property "Value" "" (id 1) (at 113.03 96.52 90)
-      (effects (font (size 1.27 1.27)) (justify left))
-    )
-    (property "Footprint" "" (id 2) (at 110.49 110.49 0)
+    (property "Value" "SK6805-EC15" (id 1) (at 113.03 96.52 90)
+      (effects (font (size 1.27 1.27)) (justify left))
+    )
+    (property "Footprint" "custom:LED_SK6805_EC15_1.5x1.5mm" (id 2) (at 110.49 110.49 0)
       (effects (font (size 1.27 1.27)) (justify left top) hide)
     )
@@
       (effects (font (size 1.524 1.524)))
     )
-    (property "Value" "" (id 1) (at 91.44 97.79 0)
+    (property "Value" "74LVC1G125" (id 1) (at 91.44 97.79 0)
       (effects (font (size 1.524 1.524)))
     )
-    (property "Footprint" "" (id 2) (at 85.09 95.25 0)
+    (property "Footprint" "Package_TO_SOT_SMD:SOT-353_SC-70-5" (id 2) (at 85.09 95.25 0)
       (effects (font (size 1.524 1.524)) (justify left) hide)
     )
@@
       (effects (font (size 1.27 1.27)) (justify left))
     )
-    (property "Value" "" (id 1) (at 128.27 96.52 90)
-      (effects (font (size 1.27 1.27)) (justify left))
-    )
-    (property "Footprint" "" (id 2) (at 125.73 110.49 0)
+    (property "Value" "SK6805-EC15" (id 1) (at 128.27 96.52 90)
+      (effects (font (size 1.27 1.27)) (justify left))
+    )
+    (property "Footprint" "custom:LED_SK6805_EC15_1.5x1.5mm" (id 2) (at 125.73 110.49 0)
       (effects (font (size 1.27 1.27)) (justify left top) hide)
     )
@@
       (effects (font (size 1.27 1.27)) (justify left))
     )
-    (property "Value" "" (id 1) (at 143.51 96.52 90)
-      (effects (font (size 1.27 1.27)) (justify left))
-    )
-    (property "Footprint" "" (id 2) (at 140.97 110.49 0)
+    (property "Value" "SK6805-EC15" (id 1) (at 143.51 96.52 90)
+      (effects (font (size 1.27 1.27)) (justify left))
+    )
+    (property "Footprint" "custom:LED_SK6805_EC15_1.5x1.5mm" (id 2) (at 140.97 110.49 0)
       (effects (font (size 1.27 1.27)) (justify left top) hide)
     )
@@
       (effects (font (size 1.27 1.27)) (justify left))
     )
-    (property "Value" "" (id 1) (at 158.75 96.52 90)
-      (effects (font (size 1.27 1.27)) (justify left))
-    )
-    (property "Footprint" "" (id 2) (at 156.21 110.49 0)
+    (property "Value" "SK6805-EC15" (id 1) (at 158.75 96.52 90)
+      (effects (font (size 1.27 1.27)) (justify left))
+    )
+    (property "Footprint" "custom:LED_SK6805_EC15_1.5x1.5mm" (id 2) (at 156.21 110.49 0)
       (effects (font (size 1.27 1.27)) (justify left top) hide)
     )
@@
       (effects (font (size 1.27 1.27)) (justify left))
     )
-    (property "Value" "" (id 1) (at 173.99 96.52 90)
-      (effects (font (size 1.27 1.27)) (justify left))
-    )
-    (property "Footprint" "" (id 2) (at 171.45 110.49 0)
+    (property "Value" "SK6805-EC15" (id 1) (at 173.99 96.52 90)
+      (effects (font (size 1.27 1.27)) (justify left))
+    )
+    (property "Footprint" "custom:LED_SK6805_EC15_1.5x1.5mm" (id 2) (at 171.45 110.49 0)
       (effects (font (size 1.27 1.27)) (justify left top) hide)
     )
@@
       (effects (font (size 1.27 1.27)) (justify left))
     )
-    (property "Value" "" (id 1) (at 106.299 130.683 0)
-      (effects (font (size 1.27 1.27)) (justify left))
-    )
-    (property "Footprint" "" (id 2) (at 108.2548 133.35 0)
+    (property "Value" "1u" (id 1) (at 106.299 130.683 0)
+      (effects (font (size 1.27 1.27)) (justify left))
+    )
+    (property "Footprint" "Capacitor_SMD:C_0402_1005Metric" (id 2) (at 108.2548 133.35 0)
       (effects (font (size 1.27 1.27)) hide)
     )
@@
       (effects (font (size 1.27 1.27)) (justify left))
     )
-    (property "Value" "" (id 1) (at 121.539 130.683 0)
-      (effects (font (size 1.27 1.27)) (justify left))
-    )
-    (property "Footprint" "" (id 2) (at 123.4948 133.35 0)
+    (property "Value" "1u" (id 1) (at 121.539 130.683 0)
+      (effects (font (size 1.27 1.27)) (justify left))
+    )
+    (property "Footprint" "Capacitor_SMD:C_0402_1005Metric" (id 2) (at 123.4948 133.35 0)
       (effects (font (size 1.27 1.27)) hide)
     )
@@
       (effects (font (size 1.27 1.27)) (justify right))
     )
-    (property "Value" "" (id 1) (at 88.9 106.68 0)
+    (property "Value" "Testpoint" (id 1) (at 88.9 106.68 0)
       (effects (font (size 1.27 1.27)) (justify right))
     )
-    (property "Footprint" "" (id 2) (at 82.55 102.87 0)
+    (property "Footprint" "TestPoint:TestPoint_Pad_1.0x1.0mm" (id 2) (at 82.55 102.87 0)
       (effects (font (size 1.27 1.27)) hide)
     )
@@
       (effects (font (size 1.27 1.27)) (justify right))
     )
-    (property "Value" "" (id 1) (at 60.96 106.68 0)
+    (property "Value" "Testpoint" (id 1) (at 60.96 106.68 0)
       (effects (font (size 1.27 1.27)) (justify right))
     )
-    (property "Footprint" "" (id 2) (at 54.61 102.87 0)
-      (effects (font (size 1.27 1.27)) hide)
-    )
+    (property "Footprint" "TestPoint:TestPoint_Pad_1.0x1.0mm" (id 2) (at 54.61 102.87 0)
+      (effects (font (size 1.27 1.27)) hide)
+    )
