File: led.kicad_sch (KiCad schematic)
At the start: 10 parts, among them U10 74LVC1G125

Commit message: Pre-production final design
Parts:
- C31, C32: value 1u -> (none); footprint Capacitor_SMD:C_0402_1005Metric -> (none)
- D3, D4, D5, D6, D7: value SK6805-EC15 -> (none); footprint custom:LED_SK6805_EC15_1.5x1.5mm -> (none)
- TP2, TP3: value Testpoint -> (none); footprint TestPoint:TestPoint_Pad_1.0x1.0mm -> (none)
- U10: value 74LVC1G125 -> (none); footprint Package_TO_SOT_SMD:SOT-353_SC-70-5 -> (none)
Changed lines of the file:
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@@
   (paper "A4")
   (title_block
-    (date "2022-03-11")
-    (rev "4")
+    (date "2022-04-24")
+    (rev "Pre-production final")
     (company "BADGE.TEAM")
   )
@@
       (effects (font (size 1.27 1.27)) (justify left))
     )
-    (property "Value" "SK6805-EC15" (id 1) (at 113.03 96.52 90)
-      (effects (font (size 1.27 1.27)) (justify left))
-    )
-    (property "Footprint" "custom:LED_SK6805_EC15_1.5x1.5mm" (id 2) (at 110.49 110.49 0)
+    (property "Value" "" (id 1) (at 113.03 96.52 90)
+      (effects (font (size 1.27 1.27)) (justify left))
+    )
+    (property "Footprint" "" (id 2) (at 110.49 110.49 0)
       (effects (font (size 1.27 1.27)) (justify left top) hide)
     )
@@
       (effects (font (size 1.524 1.524)))
     )
-    (property "Value" "74LVC1G125" (id 1) (at 91.44 97.79 0)
+    (property "Value" "" (id 1) (at 91.44 97.79 0)
       (effects (font (size 1.524 1.524)))
     )
-    (property "Footprint" "Package_TO_SOT_SMD:SOT-353_SC-70-5" (id 2) (at 85.09 95.25 0)
+    (property "Footprint" "" (id 2) (at 85.09 95.25 0)
       (effects (font (size 1.524 1.524)) (justify left) hide)
     )
@@
       (effects (font (size 1.27 1.27)) (justify left))
     )
-    (property "Value" "SK6805-EC15" (id 1) (at 128.27 96.52 90)
-      (effects (font (size 1.27 1.27)) (justify left))
-    )
-    (property "Footprint" "custom:LED_SK6805_EC15_1.5x1.5mm" (id 2) (at 125.73 110.49 0)
+    (property "Value" "" (id 1) (at 128.27 96.52 90)
+      (effects (font (size 1.27 1.27)) (justify left))
+    )
+    (property "Footprint" "" (id 2) (at 125.73 110.49 0)
       (effects (font (size 1.27 1.27)) (justify left top) hide)
     )
@@
       (effects (font (size 1.27 1.27)) (justify left))
     )
-    (property "Value" "SK6805-EC15" (id 1) (at 143.51 96.52 90)
-      (effects (font (size 1.27 1.27)) (justify left))
-    )
-    (property "Footprint" "custom:LED_SK6805_EC15_1.5x1.5mm" (id 2) (at 140.97 110.49 0)
+    (property "Value" "" (id 1) (at 143.51 96.52 90)
+      (effects (font (size 1.27 1.27)) (justify left))
+    )
+    (property "Footprint" "" (id 2) (at 140.97 110.49 0)
       (effects (font (size 1.27 1.27)) (justify left top) hide)
     )
@@
       (effects (font (size 1.27 1.27)) (justify left))
     )
-    (property "Value" "SK6805-EC15" (id 1) (at 158.75 96.52 90)
-      (effects (font (size 1.27 1.27)) (justify left))
-    )
-    (property "Footprint" "custom:LED_SK6805_EC15_1.5x1.5mm" (id 2) (at 156.21 110.49 0)
+    (property "Value" "" (id 1) (at 158.75 96.52 90)
+      (effects (font (size 1.27 1.27)) (justify left))
+    )
+    (property "Footprint" "" (id 2) (at 156.21 110.49 0)
       (effects (font (size 1.27 1.27)) (justify left top) hide)
     )
@@
       (effects (font (size 1.27 1.27)) (justify left))
     )
-    (property "Value" "SK6805-EC15" (id 1) (at 173.99 96.52 90)
-      (effects (font (size 1.27 1.27)) (justify left))
-    )
-    (property "Footprint" "custom:LED_SK6805_EC15_1.5x1.5mm" (id 2) (at 171.45 110.49 0)
+    (property "Value" "" (id 1) (at 173.99 96.52 90)
+      (effects (font (size 1.27 1.27)) (justify left))
+    )
+    (property "Footprint" "" (id 2) (at 171.45 110.49 0)
       (effects (font (size 1.27 1.27)) (justify left top) hide)
     )
@@
       (effects (font (size 1.27 1.27)) (justify left))
     )
-    (property "Value" "1u" (id 1) (at 106.299 130.683 0)
-      (effects (font (size 1.27 1.27)) (justify left))
-    )
-    (property "Footprint" "Capacitor_SMD:C_0402_1005Metric" (id 2) (at 108.2548 133.35 0)
+    (property "Value" "" (id 1) (at 106.299 130.683 0)
+      (effects (font (size 1.27 1.27)) (justify left))
+    )
+    (property "Footprint" "" (id 2) (at 108.2548 133.35 0)
       (effects (font (size 1.27 1.27)) hide)
     )
@@
       (effects (font (size 1.27 1.27)) (justify left))
     )
-    (property "Value" "1u" (id 1) (at 121.539 130.683 0)
-      (effects (font (size 1.27 1.27)) (justify left))
-    )
-    (property "Footprint" "Capacitor_SMD:C_0402_1005Metric" (id 2) (at 123.4948 133.35 0)
+    (property "Value" "" (id 1) (at 121.539 130.683 0)
+      (effects (font (size 1.27 1.27)) (justify left))
+    )
+    (property "Footprint" "" (id 2) (at 123.4948 133.35 0)
       (effects (font (size 1.27 1.27)) hide)
     )
@@
       (effects (font (size 1.27 1.27)) (justify right))
     )
-    (property "Value" "Testpoint" (id 1) (at 88.9 106.68 0)
+    (property "Value" "" (id 1) (at 88.9 106.68 0)
       (effects (font (size 1.27 1.27)) (justify right))
     )
-    (property "Footprint" "TestPoint:TestPoint_Pad_1.0x1.0mm" (id 2) (at 82.55 102.87 0)
+    (property "Footprint" "" (id 2) (at 82.55 102.87 0)
       (effects (font (size 1.27 1.27)) hide)
     )
@@
       (effects (font (size 1.27 1.27)) (justify right))
     )
-    (property "Value" "Testpoint" (id 1) (at 60.96 106.68 0)
+    (property "Value" "" (id 1) (at 60.96 106.68 0)
       (effects (font (size 1.27 1.27)) (justify right))
     )
-    (property "Footprint" "TestPoint:TestPoint_Pad_1.0x1.0mm" (id 2) (at 54.61 102.87 0)
-      (effects (font (size 1.27 1.27)) hide)
-    )
+    (property "Footprint" "" (id 2) (at 54.61 102.87 0)
+      (effects (font (size 1.27 1.27)) hide)
+    )
