File: led.kicad_sch (KiCad schematic)
At the start: 10 parts

Commit message: Add gerbers, add schematic, finalize design
Parts:
- C31, C32: value (none) -> 1u; footprint (none) -> Capacitor_SMD:C_0402_1005Metric
- D3, D4, D5, D6, D7: value (none) -> SK6805-EC15; footprint (none) -> custom:LED_SK6805_EC15_1.5x1.5mm
- TP2, TP3: value (none) -> Testpoint; footprint (none) -> TestPoint:TestPoint_Pad_1.0x1.0mm
- U10: value (none) -> 74LVC1G125; footprint (none) -> Package_TO_SOT_SMD:SOT-353_SC-70-5
Changed lines of the file:
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@@
   (title_block
     (date "2022-04-24")
-    (rev "Pre-production final")
+    (rev "Final")
     (company "BADGE.TEAM")
+    (comment 1 "License: CERN Open Hardware Licence Version 2 - Permissive")
+    (comment 2 "Contact: renze@badge.team")
+    (comment 3 "Website: mch2022.org / badge.team")
+    (comment 4 "Event badge for May Contain Hackers 2022")
   )
   (junction (at 59.69 102.87) (diameter 0) (color 0 0 0 0)
@@
       (effects (font (size 1.27 1.27)) (justify left))
     )
-    (property "Value" "" (id 1) (at 113.03 96.52 90)
-      (effects (font (size 1.27 1.27)) (justify left))
-    )
-    (property "Footprint" "" (id 2) (at 110.49 110.49 0)
+    (property "Value" "SK6805-EC15" (id 1) (at 113.03 96.52 90)
+      (effects (font (size 1.27 1.27)) (justify left))
+    )
+    (property "Footprint" "custom:LED_SK6805_EC15_1.5x1.5mm" (id 2) (at 110.49 110.49 0)
       (effects (font (size 1.27 1.27)) (justify left top) hide)
     )
@@
       (effects (font (size 1.524 1.524)))
     )
-    (property "Value" "" (id 1) (at 91.44 97.79 0)
+    (property "Value" "74LVC1G125" (id 1) (at 91.44 97.79 0)
       (effects (font (size 1.524 1.524)))
     )
-    (property "Footprint" "" (id 2) (at 85.09 95.25 0)
+    (property "Footprint" "Package_TO_SOT_SMD:SOT-353_SC-70-5" (id 2) (at 85.09 95.25 0)
       (effects (font (size 1.524 1.524)) (justify left) hide)
     )
@@
       (effects (font (size 1.27 1.27)) (justify left))
     )
-    (property "Value" "" (id 1) (at 128.27 96.52 90)
-      (effects (font (size 1.27 1.27)) (justify left))
-    )
-    (property "Footprint" "" (id 2) (at 125.73 110.49 0)
+    (property "Value" "SK6805-EC15" (id 1) (at 128.27 96.52 90)
+      (effects (font (size 1.27 1.27)) (justify left))
+    )
+    (property "Footprint" "custom:LED_SK6805_EC15_1.5x1.5mm" (id 2) (at 125.73 110.49 0)
       (effects (font (size 1.27 1.27)) (justify left top) hide)
     )
@@
       (effects (font (size 1.27 1.27)) (justify left))
     )
-    (property "Value" "" (id 1) (at 143.51 96.52 90)
-      (effects (font (size 1.27 1.27)) (justify left))
-    )
-    (property "Footprint" "" (id 2) (at 140.97 110.49 0)
+    (property "Value" "SK6805-EC15" (id 1) (at 143.51 96.52 90)
+      (effects (font (size 1.27 1.27)) (justify left))
+    )
+    (property "Footprint" "custom:LED_SK6805_EC15_1.5x1.5mm" (id 2) (at 140.97 110.49 0)
       (effects (font (size 1.27 1.27)) (justify left top) hide)
     )
@@
       (effects (font (size 1.27 1.27)) (justify left))
     )
-    (property "Value" "" (id 1) (at 158.75 96.52 90)
-      (effects (font (size 1.27 1.27)) (justify left))
-    )
-    (property "Footprint" "" (id 2) (at 156.21 110.49 0)
+    (property "Value" "SK6805-EC15" (id 1) (at 158.75 96.52 90)
+      (effects (font (size 1.27 1.27)) (justify left))
+    )
+    (property "Footprint" "custom:LED_SK6805_EC15_1.5x1.5mm" (id 2) (at 156.21 110.49 0)
       (effects (font (size 1.27 1.27)) (justify left top) hide)
     )
@@
       (effects (font (size 1.27 1.27)) (justify left))
     )
-    (property "Value" "" (id 1) (at 173.99 96.52 90)
-      (effects (font (size 1.27 1.27)) (justify left))
-    )
-    (property "Footprint" "" (id 2) (at 171.45 110.49 0)
+    (property "Value" "SK6805-EC15" (id 1) (at 173.99 96.52 90)
+      (effects (font (size 1.27 1.27)) (justify left))
+    )
+    (property "Footprint" "custom:LED_SK6805_EC15_1.5x1.5mm" (id 2) (at 171.45 110.49 0)
       (effects (font (size 1.27 1.27)) (justify left top) hide)
     )
@@
       (effects (font (size 1.27 1.27)) (justify left))
     )
-    (property "Value" "" (id 1) (at 106.299 130.683 0)
-      (effects (font (size 1.27 1.27)) (justify left))
-    )
-    (property "Footprint" "" (id 2) (at 108.2548 133.35 0)
+    (property "Value" "1u" (id 1) (at 106.299 130.683 0)
+      (effects (font (size 1.27 1.27)) (justify left))
+    )
+    (property "Footprint" "Capacitor_SMD:C_0402_1005Metric" (id 2) (at 108.2548 133.35 0)
       (effects (font (size 1.27 1.27)) hide)
     )
@@
       (effects (font (size 1.27 1.27)) (justify left))
     )
-    (property "Value" "" (id 1) (at 121.539 130.683 0)
-      (effects (font (size 1.27 1.27)) (justify left))
-    )
-    (property "Footprint" "" (id 2) (at 123.4948 133.35 0)
+    (property "Value" "1u" (id 1) (at 121.539 130.683 0)
+      (effects (font (size 1.27 1.27)) (justify left))
+    )
+    (property "Footprint" "Capacitor_SMD:C_0402_1005Metric" (id 2) (at 123.4948 133.35 0)
       (effects (font (size 1.27 1.27)) hide)
     )
@@
       (effects (font (size 1.27 1.27)) (justify right))
     )
-    (property "Value" "" (id 1) (at 88.9 106.68 0)
+    (property "Value" "Testpoint" (id 1) (at 88.9 106.68 0)
       (effects (font (size 1.27 1.27)) (justify right))
     )
-    (property "Footprint" "" (id 2) (at 82.55 102.87 0)
+    (property "Footprint" "TestPoint:TestPoint_Pad_1.0x1.0mm" (id 2) (at 82.55 102.87 0)
       (effects (font (size 1.27 1.27)) hide)
     )
@@
       (effects (font (size 1.27 1.27)) (justify right))
     )
-    (property "Value" "" (id 1) (at 60.96 106.68 0)
+    (property "Value" "Testpoint" (id 1) (at 60.96 106.68 0)
       (effects (font (size 1.27 1.27)) (justify right))
     )
-    (property "Footprint" "" (id 2) (at 54.61 102.87 0)
-      (effects (font (size 1.27 1.27)) hide)
-    )
+    (property "Footprint" "TestPoint:TestPoint_Pad_1.0x1.0mm" (id 2) (at 54.61 102.87 0)
+      (effects (font (size 1.27 1.27)) hide)
+    )
