File: fpga.kicad_sch (KiCad schematic)
At the start: 21 parts, among them U5 ICE40UP5K-SG48ITR, U6 LY68L6400, X2 SG-210STF

Commit message: Remove IO expander, move around signals
Parts:
- R32: value DNP -> 10k
Connections:
- net I2S_CLK renamed LCD_CS
- net I2S_DATA renamed LCD_RST
- net I2S_LR renamed LCD_MODE
Changed lines of the file:
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@@
   (title_block
     (title "MCH2022 badge - ICE40 FPGA")
-    (date "2022-01-14")
-    (rev "3.1415")
+    (date "2022-03-11")
+    (rev "4")
     (company "BADGE.TEAM")
   )
@@
     )
   )
-  (hierarchical_label "I2S_LR" (shape output) (at 85.09 116.84 180)
-    (effects (font (size 0.9906 0.9906)) (justify right))
-  )
   (hierarchical_label "FPGA_RESET" (shape passive) (at 110.49 40.64 90)
     (effects (font (size 1.27 1.27)) (justify left))
@@
     (effects (font (size 1.27 1.27)) (justify right))
   )
+  (hierarchical_label "LCD_RST" (shape output) (at 85.09 114.3 180)
+    (effects (font (size 1 1)) (justify right))
+  )
   (hierarchical_label "LCD_D4" (shape output) (at 85.09 106.68 180)
     (effects (font (size 0.9906 0.9906)) (justify right))
@@
     (effects (font (size 1.27 1.27)) (justify right))
   )
+  (hierarchical_label "LCD_MODE" (shape output) (at 85.09 116.84 180)
+    (effects (font (size 1 1)) (justify right))
+  )
   (hierarchical_label "LCD_D1" (shape output) (at 85.09 93.98 180)
     (effects (font (size 0.9906 0.9906)) (justify right))
@@
     (effects (font (size 0.9906 0.9906)) (justify right))
   )
-  (hierarchical_label "I2S_DATA" (shape output) (at 85.09 114.3 180)
-    (effects (font (size 0.9906 0.9906)) (justify right))
-  )
   (hierarchical_label "LCD_D7" (shape output) (at 85.09 121.92 180)
     (effects (font (size 0.9906 0.9906)) (justify right))
@@
     (effects (font (size 0.9906 0.9906)) (justify right))
   )
-  (hierarchical_label "I2S_CLK" (shape output) (at 85.09 99.06 180)
-    (effects (font (size 0.9906 0.9906)) (justify right))
-  )
   (hierarchical_label "FPGA_CDONE" (shape input) (at 38.1 111.76 180)
     (effects (font (size 1.27 1.27)) (justify right))
+  )
+  (hierarchical_label "LCD_CS" (shape output) (at 85.09 99.06 180)
+    (effects (font (size 1 1)) (justify right))
   )
   (hierarchical_label "PMOD_9" (shape bidirectional) (at 161.29 118.11 180)
@@
       (effects (font (size 1.27 1.27)) (justify left))
     )
-    (property "Value" "DNP" (id 1) (at 119.6086 35.433 0)
-      (effects (font (size 1.27 1.27)) (justify left))
-    )
+    (property "Value" "10k" (id 1) (at 119.6086 35.433 0)
+      (effects (font (size 1.27 1.27)) (justify left))
+    )

Commit message: Bill of materials 1/2
Parts:
- removed JP1: ST, Jumpers:SMT-JUMPER_2_NC_PASTE_NO-SILK, symbol Device:Jumper_NC_Small
- C12, C15, C16, C18, C19, C20, C21, C22: value 100n -> (none); footprint Capacitor_SMD:C_0402_1005Metric -> (none); Category (none) -> Capacitors; LCSC C83056 -> (none); Sponsored N -> (none)
- C17: value 10u -> (none); footprint Capacitor_SMD:C_0402_1005Metric -> (none); Category (none) -> Capacitors; LCSC C15525 -> (none); Sponsored N -> (none)
- R31, R35, R36: value 10k -> (none); footprint Resistor_SMD:R_0402_1005Metric -> (none); Category (none) -> Resistors; LCSC C144807 -> (none); MPN AC0402FR-0710KL -> (none); Sponsored N -> (none)
- R32: value 10k -> (none); footprint Resistor_SMD:R_0402_1005Metric -> (none); Category (none) -> Resistors; Sponsored N -> (none)
- R33: value 47 -> (none); footprint Resistor_SMD:R_0402_1005Metric -> (none); Category (none) -> Resistors; LCSC C25168 -> (none); MPN 0402WGJ0470TCE -> (none); Sponsored N -> (none)
- R34: value 4.7k -> (none); footprint Resistor_SMD:R_0402_1005Metric -> (none); Category (none) -> Resistors; Sponsored N -> (none)
- RN4, RN5: value 47 -> (none); footprint Resistor_SMD:R_Array_Convex_4x0603 -> (none); Category (none) -> Resistor arrays; Sponsored N -> (none)
- U5: value ICE40UP5K-SG48ITR -> (none); footprint Package_DFN_QFN:QFN-48-1EP_7x7mm_P0.5mm_EP5.6x5.6mm -> (none); Buy early (none) -> N; Category (none) -> ICs; LCSC - -> (none); Manufacturer (none) -> Lattice; Sponsored N -> Y
- U6: value LY68L6400 -> (none); footprint Package_SO:SOIC-8_3.9x4.9mm_P1.27mm -> (none); Buy early (none) -> N; Category (none) -> ICs; LCSC C261881 -> (none); Manufacturer (none) -> Espressif Systems
- X2: value SG-210STF -> (none); footprint Oscillator:Oscillator_SMD_SeikoEpson_SG210-4Pin_2.5x2.0mm -> (none); Buy early (none) -> Y; Category (none) -> Oscillators; Sponsored (none) -> N
Connections:
- net FPGA_CDONE: now also X2.1 (~{ST})

Commit message: Add more info to BOM
Parts:
- C12, C15, C16, C17, C18, C19, C20, C21, C22, R31, R32, R33, R35, R36: Buy early (none) -> Y; Sponsored (none) -> N
- R34, RN4, RN5: Buy early (none) -> Y; Manufacturer (none) -> Uni-royal; Sponsored (none) -> N
Changed lines of the file:
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@@
       (effects (font (size 1.27 1.27)) hide)
     )
-    (property "Sponsored" "" (id 7) (at 196.85 57.15 0)
+    (property "Sponsored" "N" (id 7) (at 196.85 57.15 0)
       (effects (font (size 1.27 1.27)) hide)
     )
@@
     )
     (property "Category" "Resistors" (id 10) (at 196.85 57.15 0)
+      (effects (font (size 1.27 1.27)) hide)
+    )
+    (property "Buy early" "Y" (id 11) (at 196.85 57.15 0)
+      (effects (font (size 1.27 1.27)) hide)
+    )
+    (property "Description" "Generic part" (id 12) (at 196.85 57.15 0)
       (effects (font (size 1.27 1.27)) hide)
     )
@@
       (effects (font (size 1.27 1.27)) hide)
     )
-    (property "Sponsored" "" (id 7) (at 175.26 78.74 0)
+    (property "Sponsored" "N" (id 7) (at 175.26 78.74 0)
       (effects (font (size 1.27 1.27)) hide)
     )
@@
     )
     (property "Description" "Generic part" (id 9) (at 175.26 78.74 0)
+      (effects (font (size 1.27 1.27)) hide)
+    )
+    (property "Buy early" "Y" (id 10) (at 175.26 78.74 0)
       (effects (font (size 1.27 1.27)) hide)
     )
@@
       (effects (font (size 1.27 1.27)) hide)
     )
-    (property "Sponsored" "" (id 7) (at 223.52 97.79 0)
+    (property "Sponsored" "N" (id 7) (at 223.52 97.79 0)
       (effects (font (size 1.27 1.27)) hide)
     )
@@
     )
     (property "Description" "Generic part" (id 9) (at 223.52 97.79 0)
+      (effects (font (size 1.27 1.27)) hide)
+    )
+    (property "Buy early" "Y" (id 10) (at 223.52 97.79 0)
       (effects (font (size 1.27 1.27)) hide)
     )
@@
       (effects (font (size 1.27 1.27)) hide)
     )
-    (property "Sponsored" "" (id 7) (at 87.63 43.18 0)
+    (property "Sponsored" "N" (id 7) (at 87.63 43.18 0)
       (effects (font (size 1.27 1.27)) hide)
     )
@@
     )
     (property "Description" "Generic part" (id 9) (at 87.63 43.18 0)
+      (effects (font (size 1.27 1.27)) hide)
+    )
+    (property "Buy early" "Y" (id 10) (at 87.63 43.18 0)
       (effects (font (size 1.27 1.27)) hide)
     )
@@
       (effects (font (size 1.27 1.27)) hide)
     )
-    (property "Sponsored" "" (id 7) (at 106.68 78.74 0)
+    (property "Sponsored" "N" (id 7) (at 106.68 78.74 0)
       (effects (font (size 1.27 1.27)) hide)
     )
@@
     )
     (property "Description" "Generic part" (id 9) (at 106.68 78.74 0)
+      (effects (font (size 1.27 1.27)) hide)
+    )
+    (property "Buy early" "Y" (id 10) (at 106.68 78.74 0)
       (effects (font (size 1.27 1.27)) hide)
     )
@@
       (effects (font (size 1.27 1.27)) hide)
     )
-    (property "Sponsored" "" (id 7) (at 22.86 43.18 0)
+    (property "Sponsored" "N" (id 7) (at 22.86 43.18 0)
       (effects (font (size 1.27 1.27)) hide)
     )
@@
     )
     (property "Description" "Generic part" (id 9) (at 22.86 43.18 0)
+      (effects (font (size 1.27 1.27)) hide)
+    )
+    (property "Buy early" "Y" (id 10) (at 22.86 43.18 0)
       (effects (font (size 1.27 1.27)) hide)
     )
@@
       (effects (font (size 1.27 1.27)) hide)
     )
-    (property "Sponsored" "" (id 7) (at 134.62 34.29 0)
+    (property "Sponsored" "N" (id 7) (at 134.62 34.29 0)
       (effects (font (size 1.27 1.27)) hide)
     )
@@
     )
     (property "Category" "Resistors" (id 10) (at 134.62 34.29 0)
+      (effects (font (size 1.27 1.27)) hide)
+    )
+    (property "Buy early" "Y" (id 11) (at 134.62 34.29 0)
+      (effects (font (size 1.27 1.27)) hide)
+    )
+    (property "Description" "Generic part" (id 12) (at 134.62 34.29 0)
       (effects (font (size 1.27 1.27)) hide)
     )
@@
       (effects (font (size 1.27 1.27)) hide)
     )
-    (property "Sponsored" "" (id 7) (at 43.18 34.29 0)
+    (property "Sponsored" "N" (id 7) (at 43.18 34.29 0)
       (effects (font (size 1.27 1.27)) hide)
     )
@@
       (effects (font (size 1.27 1.27)) hide)
     )
+    (property "Buy early" "Y" (id 11) (at 43.18 34.29 0)
+      (effects (font (size 1.27 1.27)) hide)
+    )
+    (property "Description" "Generic part" (id 12) (at 43.18 34.29 0)
+      (effects (font (size 1.27 1.27)) hide)
+    )
     (pin "1")
     (pin "2")
@@
       (effects (font (size 1.27 1.27)) hide)
     )
-    (property "Sponsored" "" (id 7) (at 127 34.29 0)
+    (property "Sponsored" "N" (id 7) (at 127 34.29 0)
       (effects (font (size 1.27 1.27)) hide)
     )
@@
     )
     (property "Category" "Resistors" (id 10) (at 127 34.29 0)
+      (effects (font (size 1.27 1.27)) hide)
+    )
+    (property "Buy early" "Y" (id 11) (at 127 34.29 0)
+      (effects (font (size 1.27 1.27)) hide)
+    )
+    (property "Description" "Generic part" (id 12) (at 127 34.29 0)
+      (effects (font (size 1.27 1.27)) hide)
+    )
+    (property "Manufacturer" "Uni-royal" (id 13) (at 127 34.29 0)
       (effects (font (size 1.27 1.27)) hide)
     )
@@
       (effects (font (size 1.27 1.27)) hide)
     )
-    (property "Sponsored" "" (id 7) (at 33.02 43.18 0)
+    (property "Sponsored" "N" (id 7) (at 33.02 43.18 0)
       (effects (font (size 1.27 1.27)) hide)
     )
@@
       (effects (font (size 1.27 1.27)) hide)
     )
+    (property "Buy early" "Y" (id 10) (at 33.02 43.18 0)
+      (effects (font (size 1.27 1.27)) hide)
+    )
     (pin "1")
     (pin "2")
@@
       (effects (font (size 1.27 1.27)) hide)
     )
-    (property "Sponsored" "" (id 5) (at 43.18 43.18 0)
+    (property "Sponsored" "N" (id 5) (at 43.18 43.18 0)
       (effects (font (size 1.27 1.27)) hide)
     )
@@
       (effects (font (size 1.27 1.27)) hide)
     )
+    (property "Buy early" "Y" (id 9) (at 43.18 43.18 0)
+      (effects (font (size 1.27 1.27)) hide)
+    )
     (pin "1")
     (pin "2")
@@
       (effects (font (size 1.27 1.27)) hide)
     )
-    (property "Sponsored" "" (id 7) (at 53.34 43.18 0)
+    (property "Sponsored" "N" (id 7) (at 53.34 43.18 0)
       (effects (font (size 1.27 1.27)) hide)
     )
@@
     )
     (property "Description" "Generic part" (id 9) (at 53.34 43.18 0)
+      (effects (font (size 1.27 1.27)) hide)
+    )
+    (property "Buy early" "Y" (id 10) (at 53.34 43.18 0)
       (effects (font (size 1.27 1.27)) hide)
     )
@@
       (effects (font (size 1.27 1.27)) hide)
     )
-    (property "Sponsored" "" (id 7) (at 110.49 43.18 0)
+    (property "Sponsored" "N" (id 7) (at 110.49 43.18 0)
       (effects (font (size 1.27 1.27)) hide)
     )
@@
       (effects (font (size 1.27 1.27)) hide)
     )
+    (property "Buy early" "Y" (id 11) (at 110.49 43.18 0)
+      (effects (font (size 1.27 1.27)) hide)
+    )
+    (property "Description" "Generic part" (id 12) (at 110.49 43.18 0)
+      (effects (font (size 1.27 1.27)) hide)
+    )
     (pin "1")
     (pin "2")
@@
       (effects (font (size 1.27 1.27)) hide)
     )
-    (property "Sponsored" "" (id 7) (at 118.11 34.29 0)
+    (property "Sponsored" "N" (id 7) (at 118.11 34.29 0)
       (effects (font (size 1.27 1.27)) hide)
     )
     (property "Category" "Resistors" (id 8) (at 118.11 34.29 0)
+      (effects (font (size 1.27 1.27)) hide)
+    )
+    (property "Buy early" "Y" (id 9) (at 118.11 34.29 0)
+      (effects (font (size 1.27 1.27)) hide)
+    )
+    (property "Description" "Generic part" (id 10) (at 118.11 34.29 0)
       (effects (font (size 1.27 1.27)) hide)
     )
@@
       (effects (font (size 1.27 1.27)) hide)
     )
-    (property "Sponsored" "" (id 7) (at 166.37 113.03 0)
+    (property "Sponsored" "N" (id 7) (at 166.37 113.03 0)
       (effects (font (size 1.27 1.27)) hide)
     )
@@
     )
     (property "Category" "Resistor arrays" (id 10) (at 166.37 113.03 0)
+      (effects (font (size 1.27 1.27)) hide)
+    )
+    (property "Buy early" "Y" (id 11) (at 166.37 113.03 0)
+      (effects (font (size 1.27 1.27)) hide)
+    )
+    (property "Description" "Generic part" (id 12) (at 166.37 113.03 0)
+      (effects (font (size 1.27 1.27)) hide)
+    )
+    (property "Manufacturer" "Uni-royal" (id 13) (at 166.37 113.03 0)
       (effects (font (size 1.27 1.27)) hide)
     )
@@
       (effects (font (size 1.27 1.27)) hide)
     )
-    (property "Sponsored" "" (id 7) (at 166.37 123.19 0)
+    (property "Sponsored" "N" (id 7) (at 166.37 123.19 0)
       (effects (font (size 1.27 1.27)) hide)
     )
@@
     )
     (property "Category" "Resistor arrays" (id 10) (at 166.37 123.19 0)
+      (effects (font (size 1.27 1.27)) hide)
+    )
+    (property "Buy early" "Y" (id 11) (at 166.37 123.19 0)
+      (effects (font (size 1.27 1.27)) hide)
+    )
+    (property "Description" "Generic part" (id 12) (at 166.37 123.19 0)
+      (effects (font (size 1.27 1.27)) hide)
+    )
+    (property "Manufacturer" "Uni-royal" (id 13) (at 166.37 123.19 0)
       (effects (font (size 1.27 1.27)) hide)
     )
@@
       (effects (font (size 1.27 1.27)) hide)
     )
-    (property "Sponsored" "" (id 7) (at 16.51 111.76 0)
+    (property "Sponsored" "N" (id 7) (at 16.51 111.76 0)
       (effects (font (size 1.27 1.27)) hide)
     )
@@
       (effects (font (size 1.27 1.27)) hide)
     )
+    (property "Buy early" "Y" (id 10) (at 16.51 111.76 0)
+      (effects (font (size 1.27 1.27)) hide)
+    )

Commit message: Add passives to BOM
Parts:
- C12, C15, C16, C18, C19, C20, C21, C22: LCSC (none) -> C307331; MPN (none) -> CL05B104KB54PNC; Manufacturer (none) -> Samsung Electro-Mechanics; Minimal voltage rating (none) -> 10; Voltage rating (none) -> 50
- C17: LCSC (none) -> C15525; MPN (none) -> CL05A106MQ5NUNC; Manufacturer (none) -> Samsung Electro-Mechanics; Minimal voltage rating (none) -> 6; Voltage rating (none) -> 6.3
- R31, R32, R35, R36: LCSC (none) -> C25744; MPN (none) -> 0402WGF1002TCE; Manufacturer (none) -> Uni-royal
- R33: LCSC (none) -> C25118; MPN (none) -> 0402WGF470JTCE; Manufacturer (none) -> Uni-royal
- R34: LCSC C25940 -> C25900; MPN 0402WGJ0472TCE -> 0402WGF4701TCE

Commit message: Artwork stuff
Parts:
- C12, C15, C16, C18, C19, C20, C21, C22: value (none) -> 100n; footprint (none) -> Capacitor_SMD:C_0402_1005Metric
- C17: value (none) -> 10u; footprint (none) -> Capacitor_SMD:C_0402_1005Metric
- R31, R32, R35, R36: value (none) -> 10k; footprint (none) -> Resistor_SMD:R_0402_1005Metric
- R33: value (none) -> 47; footprint (none) -> Resistor_SMD:R_0402_1005Metric
- R34: value (none) -> 4.7k; footprint (none) -> Resistor_SMD:R_0402_1005Metric
- RN4, RN5: value (none) -> 47; footprint (none) -> Resistor_SMD:R_Array_Convex_4x0603
- U5: value (none) -> ICE40UP5K-SG48ITR; footprint (none) -> Package_DFN_QFN:QFN-48-1EP_7x7mm_P0.5mm_EP5.6x5.6mm
- U6: value (none) -> ESP-PSRAM64H; footprint (none) -> Package_SO:SOIC-8_3.9x4.9mm_P1.27mm
- X2: value (none) -> SG-210STF; footprint (none) -> Oscillator:Oscillator_SMD_SeikoEpson_SG210-4Pin_2.5x2.0mm

Commit message: Pre-production final design
Parts:
- C12, C15, C16, C18, C19, C20, C21, C22: value 100n -> (none); footprint Capacitor_SMD:C_0402_1005Metric -> (none)
- C17: value 10u -> (none); footprint Capacitor_SMD:C_0402_1005Metric -> (none)
- R31, R35, R36: value 10k -> (none); footprint Resistor_SMD:R_0402_1005Metric -> (none); MANUFACTURER YAGEO -> UNI-ROYAL
- R32: value 10k -> (none); footprint Resistor_SMD:R_0402_1005Metric -> (none); MANUFACTURER (none) -> UNI-ROYAL
- R33: value 47 -> (none); footprint Resistor_SMD:R_0402_1005Metric -> (none)
- R34: value 4.7k -> (none); footprint Resistor_SMD:R_0402_1005Metric -> (none)
- RN4, RN5: value 47 -> (none); footprint Resistor_SMD:R_Array_Convex_4x0603 -> (none)
- U5: value ICE40UP5K-SG48ITR -> (none); footprint Package_DFN_QFN:QFN-48-1EP_7x7mm_P0.5mm_EP5.6x5.6mm -> (none)
- U6: value ESP-PSRAM64H -> (none); footprint Package_SO:SOIC-8_3.9x4.9mm_P1.27mm -> (none)
- X2: value SG-210STF -> (none); footprint Oscillator:Oscillator_SMD_SeikoEpson_SG210-4Pin_2.5x2.0mm -> (none)

Commit message: Add gerbers, add schematic, finalize design
Parts:
- C12, C15, C16, C18, C19, C20, C21, C22: value (none) -> 100n; footprint (none) -> Capacitor_SMD:C_0402_1005Metric
- C17: value (none) -> 10u; footprint (none) -> Capacitor_SMD:C_0402_1005Metric
- R31, R32, R35, R36: value (none) -> 10k; footprint (none) -> Resistor_SMD:R_0402_1005Metric
- R33: value (none) -> 47; footprint (none) -> Resistor_SMD:R_0402_1005Metric
- R34: value (none) -> 4.7k; footprint (none) -> Resistor_SMD:R_0402_1005Metric
- RN4, RN5: value (none) -> 47; footprint (none) -> Resistor_SMD:R_Array_Convex_4x0603
- U5: value (none) -> ICE40UP5K-SG48ITR; footprint (none) -> Package_DFN_QFN:QFN-48-1EP_7x7mm_P0.5mm_EP5.6x5.6mm
- U6: value (none) -> ESP-PSRAM64H; footprint (none) -> Package_SO:SOIC-8_3.9x4.9mm_P1.27mm
- X2: value (none) -> SG-210STF; footprint (none) -> Oscillator:Oscillator_SMD_SeikoEpson_SG210-4Pin_2.5x2.0mm
