File: fpga.kicad_sch (KiCad schematic)
At the start: 20 parts, among them U5 ICE40UP5K-SG48ITR, U6 ESP-PSRAM64H, X2 SG-210STF

Commit message: Add test points to debug FPGA SPI bus.
Parts:
- added TP36, TP37, TP38, TP39: TestPoint, TestPoint:TestPoint_Pad_1.0x1.0mm, symbol Connector:TestPoint
Connections:
- net SPI_CS: now also TP37.1
- net SPI_MISO: now also TP38.1
- net SPI_MOSI: now also TP39.1
- net SPI_SCK: now also TP36.1
Changed lines of the file:
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@@
     (effects (font (size 1.27 1.27)) (justify right))
+  )
+  (hierarchical_label "SPI_SCK" (shape input) (at 125.73 153.67 180)
+    (effects (font (size 0.9906 0.9906)) (justify right))
   )
   (hierarchical_label "PMOD_4" (shape bidirectional) (at 161.29 125.73 180)
@@
     (effects (font (size 1.27 1.27)) (justify right))
   )
+  (hierarchical_label "SPI_CS" (shape input) (at 125.73 158.75 180)
+    (effects (font (size 0.9906 0.9906)) (justify right))
+  )
   (hierarchical_label "UART_TX" (shape output) (at 124.46 96.52 180)
     (effects (font (size 0.9906 0.9906)) (justify right))
@@
     (effects (font (size 0.9906 0.9906)) (justify right))
   )
+  (hierarchical_label "SPI_MOSI" (shape input) (at 125.73 168.91 180)
+    (effects (font (size 0.9906 0.9906)) (justify right))
+  )
   (hierarchical_label "FPGA_CDONE" (shape input) (at 38.1 111.76 180)
     (effects (font (size 1.27 1.27)) (justify right))
@@
   )
   (hierarchical_label "LCD_D5" (shape output) (at 85.09 109.22 180)
+    (effects (font (size 0.9906 0.9906)) (justify right))
+  )
+  (hierarchical_label "SPI_MISO" (shape output) (at 125.73 163.83 180)
     (effects (font (size 0.9906 0.9906)) (justify right))
   )
@@
       (effects (font (size 1.27 1.27)) hide)
     )
+    (pin "1")
+  )
+  (symbol (lib_id "Connector:TestPoint") (at 125.73 153.67 270) (unit 1)
+    (in_bom yes) (on_board yes) (fields_autoplaced)
+    (property "Reference" "TP36" (id 0) (at 130.81 152.3999 90)
+      (effects (font (size 1.27 1.27)) (justify left))
+    )
+    (property "Value" "TestPoint" (id 1) (at 130.81 154.9399 90)
+      (effects (font (size 1.27 1.27)) (justify left))
+    )
+    (property "Footprint" "TestPoint:TestPoint_Pad_1.0x1.0mm" (id 2) (at 125.73 158.75 0)
+      (effects (font (size 1.27 1.27)) hide)
+    )
+    (property "Datasheet" "~" (id 3) (at 125.73 158.75 0)
+      (effects (font (size 1.27 1.27)) hide)
+    )
+    (pin "1")
+  )
+  (symbol (lib_id "Connector:TestPoint") (at 125.73 158.75 270) (unit 1)
+    (in_bom yes) (on_board yes) (fields_autoplaced)
+    (property "Reference" "TP37" (id 0) (at 130.81 157.4799 90)
+      (effects (font (size 1.27 1.27)) (justify left))
+    )
+    (property "Value" "TestPoint" (id 1) (at 130.81 160.0199 90)
+      (effects (font (size 1.27 1.27)) (justify left))
+    )
+    (property "Footprint" "TestPoint:TestPoint_Pad_1.0x1.0mm" (id 2) (at 125.73 163.83 0)
+      (effects (font (size 1.27 1.27)) hide)
+    )
+    (property "Datasheet" "~" (id 3) (at 125.73 163.83 0)
+      (effects (font (size 1.27 1.27)) hide)
+    )
+    (pin "1")
+  )
+  (symbol (lib_id "Connector:TestPoint") (at 125.73 163.83 270) (unit 1)
+    (in_bom yes) (on_board yes) (fields_autoplaced)
+    (property "Reference" "TP38" (id 0) (at 130.81 162.5599 90)
+      (effects (font (size 1.27 1.27)) (justify left))
+    )
+    (property "Value" "TestPoint" (id 1) (at 130.81 165.0999 90)
+      (effects (font (size 1.27 1.27)) (justify left))
+    )
+    (property "Footprint" "TestPoint:TestPoint_Pad_1.0x1.0mm" (id 2) (at 125.73 168.91 0)
+      (effects (font (size 1.27 1.27)) hide)
+    )
+    (property "Datasheet" "~" (id 3) (at 125.73 168.91 0)
+      (effects (font (size 1.27 1.27)) hide)
+    )
+    (pin "1")
+  )
+  (symbol (lib_id "Connector:TestPoint") (at 125.73 168.91 270) (unit 1)
+    (in_bom yes) (on_board yes) (fields_autoplaced)
+    (property "Reference" "TP39" (id 0) (at 130.81 167.6399 90)
+      (effects (font (size 1.27 1.27)) (justify left))
+    )
+    (property "Value" "TestPoint" (id 1) (at 130.81 170.1799 90)
+      (effects (font (size 1.27 1.27)) (justify left))
+    )
+    (property "Footprint" "TestPoint:TestPoint_Pad_1.0x1.0mm" (id 2) (at 125.73 173.99 0)
+      (effects (font (size 1.27 1.27)) hide)
+    )
+    (property "Datasheet" "~" (id 3) (at 125.73 173.99 0)
+      (effects (font (size 1.27 1.27)) hide)
+    )
