File: mch2022.kicad_sch (KiCad schematic)
At the start: 38 parts

Commit message: Add gerbers, add schematic, finalize design
Parts:
- D2: value (none) -> RGB-5050; footprint (none) -> LED_SMD:LED_RGB_5050-6
- F1: value (none) -> 1A; footprint (none) -> Fuse:Fuse_0805_2012Metric
- FID1, FID2: value (none) -> Fiducial; footprint (none) -> Fiducial:Fiducial_1mm_Mask2mm
- J2: value (none) -> USB_C_Receptacle_USB2.0; footprint (none) -> Connector_USB:USB_C_Receptacle_HRO_TYPE-C-31-M-12
- J4: value (none) -> PMOD; footprint (none) -> Connector_PinSocket_2.54mm:PinSocket_2x06_P2.54mm_Horizontal
- N1: value (none) -> Logo; footprint (none) -> custom:badgeteam
- N2: value (none) -> Artwork; footprint (none) -> custom:prototype4
- N3: value (none) -> May Contain Hardware; footprint (none) -> custom:protoboard-squares-big
- R1, R2: value (none) -> 5.1k; footprint (none) -> Resistor_SMD:R_0402_1005Metric
- R22, R4, R5: value (none) -> 47; footprint (none) -> Resistor_SMD:R_0402_1005Metric
- TP1, TP10, TP11, TP12, TP13, TP18, TP19, TP21, TP22, TP23, TP24, TP25, TP26, TP28, TP29, TP30, TP31, TP32, TP33, TP4, TP5, TP6, TP7, TP8: value (none) -> Testpoint; footprint (none) -> TestPoint:TestPoint_Pad_1.0x1.0mm

Commit message: Mark diode as DNP, replace fuse with SMD0805B110TF
Parts:
- F1: LCSC C269104 -> C269107; MPN SMD0805B050TF -> SMD0805B110TF
Changed lines of the file:
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@@
       (effects (font (size 1.27 1.27)) (justify left) hide)
     )
-    (property "Datasheet" "https://datasheet.lcsc.com/lcsc/1808280424_Brightking-Elec--TAIWAN-SMD0805B050TF_C269104.pdf" (id 3) (at 54.61 27.94 0)
-      (effects (font (size 1.27 1.27)) hide)
-    )
-    (property "LCSC" "C269104" (id 4) (at 54.61 27.94 90)
+    (property "Datasheet" "https://datasheet.lcsc.com/lcsc/1810161745_Brightking-Elec--TAIWAN-SMD0805B110TF_C269107.pdf" (id 3) (at 54.61 27.94 0)
+      (effects (font (size 1.27 1.27)) hide)
+    )
+    (property "LCSC" "C269107" (id 4) (at 54.61 27.94 90)
       (effects (font (size 1.27 1.27)) hide)
     )
@@
       (effects (font (size 1.27 1.27)) hide)
     )
-    (property "MPN" "SMD0805B050TF" (id 7) (at 54.61 27.94 0)
+    (property "MPN" "SMD0805B110TF" (id 7) (at 54.61 27.94 0)
       (effects (font (size 1.27 1.27)) hide)
     )
@@
     )
     (path "/00000000-0000-0000-0000-000060c789de/00000000-0000-0000-0000-00005fc55914"
-      (reference "D9") (unit 1) (value "PSBD3D40V1H") (footprint "Diode_SMD:D_SOD-323")
+      (reference "D9") (unit 1) (value "DNP") (footprint "Diode_SMD:D_SOD-323")
     )
     (path "/00000000-0000-0000-0000-00005ff73718"
